File: Gucci/v1 boards/GucciMain.brd (EAGLE design)
At the start: 43.2 x 46.7 mm, 15 parts

Commit message: Add files via upload
Parts:
- PHOTON: value (none) -> PHOTON; device Spark:PHOTON_STACKABLE -> Particle:PHOTON
- moved C2 9.23 mm to (34.6, 26.7), turned to 180 degrees
- moved C1 6.55 mm to (8.57, 29.2)
- moved C3 5.54 mm to (8.57, 26.7)
- moved C4 4.97 mm to (34.6, 29.2), turned to 180 degrees
- moved L-ESC 1.91 mm to (4.13, 27.9)
- moved R-ESC 1.91 mm to (39.1, 27.9)
- moved RS 1.85 mm to (5.40, 35.2)
- moved PHOTON 1.59 mm to (11.4, 10.5)
- moved U$3 0.95 mm to (4.13, 41.6)
- moved U$4 0.95 mm to (39.1, 41.6)
Connections:
- net 3V3: no longer PHOTON.#24
- net BL: no longer PHOTON.@8
- net BR: no longer PHOTON.@7
- net FL: no longer PHOTON.@10
- net FR: no longer PHOTON.@9
- net GND: no longer PHOTON.#21, PHOTON.@2
- net I1: no longer PHOTON.@4
- net I2: no longer PHOTON.@3
- net L-CONTROL: no longer PHOTON.#15
- net R-CONTROL: no longer PHOTON.#16
- net RS-OUT: no longer PHOTON.#17
- net SCL: no longer PHOTON.#14
- net SDA: no longer PHOTON.#13
- net SHDN1: no longer PHOTON.@12
- net SHDN2: no longer PHOTON.@11
- net SHDN3: no longer PHOTON.@6
- net SHDN4: no longer PHOTON.#18
- net SHDN5: no longer PHOTON.#19
- net SHDN6: no longer PHOTON.#20
- net VBAT: no longer PHOTON.#22
- net VCC: no longer PHOTON.@1
Routing:
- net GND: track 24.5 -> 13.8 mm
- net B1: track 10.1 -> 15.2 mm
- net RS-OUT: track 32.3 -> 27.7 mm
- net VBAT: track 2.54 -> 0.00 mm
- net 3V3: track 2.54 -> 0.00 mm
- net R-CONTROL: track 28.7 -> 26.3 mm
- net A2: track 14.9 -> 16.8 mm
- net B2: track 15.4 -> 17.3 mm
- net A1: track 11.0 -> 12.9 mm
- net I1: track 31.2 -> 29.3 mm
- net L-CONTROL: track 14.8 -> 16.2 mm
- net SHDN6: track 31.4 -> 30.4 mm
- net SHDN4: track 28.0 -> 27.1 mm
- net SHDN5: track 27.6 -> 26.6 mm
- net SHDN3: track 28.8 -> 27.9 mm
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Other:
- board size 43.2 x 46.7 mm -> 43.2 x 45.7 mm

Commit message: Add files via upload
Connections:
- net BR: now also PHOTON.6; no longer PHOTON.7
- net SHDN3: now also PHOTON.5; no longer PHOTON.6
Routing:
- net BR: track 40.1 -> 42.7 mm
- net SHDN3: track 27.9 -> 30.4 mm
Changed lines of the file:
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@@
 </layers>
 <board>
-<fusionsync huburn="a.cGVyc29uYWw6dWUyZDhlY2M3" projecturn="a.cGVyc29uYWw6dWUyZDhlY2M3IzIwMTgwNjIyMTM3MzM5MDA2" f3durn="urn:adsk.wipprod:dm.lineage:oCK5GsSnSQyYjkxJwpRfxw" pcbguid="18f558be-6b05-4ec2-9f37-b6cf3be909b8" lastpulledtime="" lastsyncedchangeguid="d21e2af2-68d8-ea46-7203-759839e72bc3"/>
+<fusionsync huburn="a.cGVyc29uYWw6dWUyZDhlY2M3" projecturn="a.cGVyc29uYWw6dWUyZDhlY2M3IzIwMTgwNjIyMTM3MzM5MDA2" f3durn="urn:adsk.wipprod:dm.lineage:oCK5GsSnSQyYjkxJwpRfxw" pcbguid="18f558be-6b05-4ec2-9f37-b6cf3be909b8" lastpulledtime="" lastsyncedchangeguid="8d8fb52a-4eb0-973f-465f-7277e2d40251"/>
 <plain>
 <wire x1="0" y1="0" x2="43.16" y2="0" width="0" layer="20"/>
@@
 <signal name="BR">
 <contactref element="B-LINES" pad="3"/>
-<contactref element="PHOTON" pad="7"/>
-<wire x1="12.7" y1="27.4955" x2="18.923" y2="21.2725" width="0.3048" layer="16"/>
-<wire x1="18.923" y1="21.2725" x2="19.05" y2="21.2725" width="0.3048" layer="16"/>
-<via x="19.05" y="21.2725" extent="1-16" drill="0.35"/>
+<wire x1="19.05" y1="22.098" x2="19.05" y2="22.225" width="0.3048" layer="16"/>
+<via x="19.05" y="22.225" extent="1-16" drill="0.35"/>
 <wire x1="19.05" y1="10.4775" x2="20.6375" y2="8.89" width="0.3048" layer="1"/>
 <wire x1="20.6375" y1="8.89" x2="36.5125" y2="8.89" width="0.3048" layer="1"/>
 <wire x1="36.5125" y1="8.89" x2="38.1" y2="7.3025" width="0.3048" layer="1"/>
-<wire x1="19.05" y1="21.2725" x2="19.05" y2="10.4775" width="0.3048" layer="1"/>
+<wire x1="19.05" y1="22.225" x2="19.05" y2="10.4775" width="0.3048" layer="1"/>
+<contactref element="PHOTON" pad="6"/>
+<wire x1="12.7" y1="30.0355" x2="19.05" y2="23.6855" width="0.3048" layer="16"/>
+<wire x1="19.05" y1="23.6855" x2="19.05" y2="22.225" width="0.3048" layer="16"/>
 </signal>
 <signal name="L-CONTROL">
@@
 <signal name="SHDN3">
 <contactref element="X1" pad="P$10"/>
-<contactref element="PHOTON" pad="6"/>
-<wire x1="20.09" y1="5.2225" x2="20.09" y2="22.6455" width="0.3048" layer="16"/>
-<wire x1="20.09" y1="22.6455" x2="12.7" y2="30.0355" width="0.3048" layer="16"/>
+<contactref element="PHOTON" pad="5"/>
+<wire x1="12.7" y1="32.5755" x2="20.09" y2="25.1855" width="0.3048" layer="16"/>
+<wire x1="20.09" y1="25.1855" x2="20.09" y2="5.2225" width="0.3048" layer="16"/>
 </signal>
 <signal name="SHDN2">
