File: Gucci/v1 boards/GucciMain.sch (EAGLE design)
At the start: 12 parts

Commit message: Add files via upload
Parts:
- PHOTON: value PHOTON_WITH_STACKABLE_HEADERS -> PHOTON; device Spark:PHOTON_WITH_STACKABLE_HEADERS -> Particle:PHOTON_WITH_HEADERS

Commit message: Add files via upload
Connections:
- net BR: now also PHOTON.DAC; no longer PHOTON.A5
- net SHDN3: now also PHOTON.WKP; no longer PHOTON.DAC
Changed lines of the file:
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@@
 </segment>
 <segment>
-<pinref part="PHOTON" gate="G$1" pin="A5"/>
-<wire x1="81.28" y1="66.04" x2="50.8" y2="66.04" width="0.1524" layer="91"/>
-<label x="50.8" y="66.04" size="1.778" layer="95"/>
+<pinref part="PHOTON" gate="G$1" pin="DAC"/>
+<wire x1="81.28" y1="71.12" x2="55.88" y2="71.12" width="0.1524" layer="91"/>
+<label x="55.88" y="71.12" size="1.778" layer="95"/>
 </segment>
 </net>
@@
 </segment>
 <segment>
-<pinref part="PHOTON" gate="G$1" pin="DAC"/>
-<wire x1="81.28" y1="71.12" x2="55.88" y2="71.12" width="0.1524" layer="91"/>
-<label x="55.88" y="71.12" size="1.778" layer="95"/>
+<pinref part="PHOTON" gate="G$1" pin="WKP"/>
+<wire x1="81.28" y1="76.2" x2="50.8" y2="76.2" width="0.1524" layer="91"/>
+<label x="50.8" y="76.2" size="1.778" layer="95"/>
 </segment>
 </net>
