File: Gucci/v1 boards/GucciAux.brd (EAGLE design)
At the start: 47 x 37.5 mm, 19 parts

Commit message: Add files via upload
Parts:
- removed U$1, U$2: (no value), holes:2,8
- moved TOF2 3.18 mm to (7.30, 30.2)
- moved TOF4 3.18 mm to (23.5, 30.2)
- moved TOF6 3.18 mm to (39.7, 30.2)
- moved C3 2.54 mm to (42.9, 26.4)
- moved C4 2.54 mm to (4.13, 26.4)
- moved C5 2.54 mm to (26.7, 26.4)
- moved TOF1 1.91 mm to (7.30, 22.2)
- moved TOF3 1.91 mm to (23.5, 22.2)
- moved TOF5 1.91 mm to (39.7, 22.2)
- moved C1 0.32 mm to (23.5, 10.8)
Routing:
- net SDA: track 70.3 -> 77.8 mm
- net SCL: track 80.7 -> 87.6 mm
- net SHDN6: track 31.3 -> 34.5 mm
- net SHDN4: track 26.7 -> 29.9 mm
- net SHDN2: track 25.4 -> 28.5 mm
- net SHDN1: track 25.3 -> 27.6 mm
- net GND: track 28.5 -> 30.8 mm
- net SHDN5: track 22.6 -> 24.5 mm
- net SHDN3: track 15.7 -> 17.6 mm
