File: Gucci/v2 pcb/Gucci_ControlBoard.brd (EAGLE design)
At the start: 66 x 56 mm, 34 parts

Commit message: revisions to pcb
Parts:
- removed 3.3V_PWR, 5V_PWR: Green, SparkFun-LED:LED-0603
- removed IMU: BMI088, Gucci_ControlBoard:BMI088
- removed LINE_LF, LINE_RF: JST_PH_1X03, Gucci_ControlBoard:JST_PH_1X03
- added C1, C11, C16, C17, C18, C2, C3, C4, C5, C6, C7, C8: 0.1uF, SparkFun-Capacitors:0603
- added C10, C9: 1uF, SparkFun-Capacitors:0603
- added C12, C13, C14, C15: 4.7uF, SparkFun-Capacitors:0603
- added D1, D2: Green, SparkFun-LED:LED-0603
- added J10, J9: JST_PH_1X03, Gucci_ControlBoard:JST_PH_1X03
- added R15, R16: 10k, SparkFun-Resistors:0603
- added U$2: (no value), RoboJackets-Aesthetics:ROBOBUZZ_1.4X
- added U$3: (no value), RoboJackets-Aesthetics:ROBOBUZZ_0.4X
- added U2: AP2114H-3.3TRG1, Gucci_ControlBoard:SOT-223
- added U3: AP2114H-1.8TRG1, Gucci_ControlBoard:SOT-223
- added U4: ICM-20948, ICM-20948:QFN40P300X300X105-25N
- U$1: device RoboJackets-Aesthetics:ROBOBUZZ_0.4X -> RoboJackets-Aesthetics:ROBOJACKETS
- moved U$1 33.5 mm to (33.0, 38.0), flipped to the bottom
- moved R14 28.8 mm to (9.00, 41.0)
- moved R13 25.2 mm to (-4.00, 38.0)
- renumbered LINE_LB to J7, LINE_RB to J8, L_ENCODER to J14, L_ESC to J11, R_ENCODER to J13, R_ESC to J12, START to J15, TEENSY_3.6 to U1, TOF0 to J1, TOF1 to J2, TOF2 to J3, TOF3 to J4, TOF4 to J5, TOF5 to J6
Connections:
- removed net 3.3V: 3.3V_PWR.A, IMU.11, IMU.14, IMU.3, IMU.7, J1.1, J15.2, J2.1, J3.1, J4.1, J5.1, J6.1, J7.3, J8.3, LINE_LF.3, LINE_RF.3, U1.3.3V, U1.3.3V3
- removed net A0_ACCEL: IMU.15, U1.10
- removed net A0_GYRO: IMU.10, U1.12
- removed net INT_ACCEL: IMU.16, U1.9
- removed net INT_GYRO: IMU.12, U1.11
- new net 1.8V: C15.1, C17.1, C18.1, R15.2, R16.2, U3.2, U3.4, U4.13, U4.22, U4.8
- new net 3V3: C1.1, C13.1, C14.1, C2.1, C3.1, C4.1, C5.1, C6.1, C7.1, C8.1, D2.A, J1.1, J10.3, J15.2, J2.1, J3.1, J4.1, J5.1, J6.1, J7.3, J8.3, J9.3, U2.2, U2.4, U3.3
- new net IMU_AD0: U1.9, U4.9
- new net IMU_INT: U1.12, U4.12
- new net N$3: C16.1, U4.10
- net 5V: now also C10.1, C11.1, C12.1, C9.1, D1.A, U2.3; no longer 5V_PWR.A
- net GND: now also C1.2, C10.2, C11.2, C12.2, C13.2, C14.2, C15.2, C16.2, C17.2, C18.2, C2.2, C3.2, C4.2, C5.2, C6.2, C7.2, C8.2, C9.2, J10.1, J9.1, U2.1, U3.1, U4.11, U4.18, U4.20; no longer IMU.2, IMU.4, IMU.6, LINE_LF.1, LINE_RF.1
- net LINE_LF: now also J9.2; no longer LINE_LF.2
- net LINE_RF: now also J10.2; no longer LINE_RF.2
- net N$1: now also D1.C; no longer 5V_PWR.C
- net N$2: now also D2.C; no longer 3.3V_PWR.C
- net SCL1: now also R16.1, U4.23; no longer IMU.8
- net SDA1: now also R15.1, U4.24; no longer IMU.9
Routing:
- net 3V3: track 0.00 -> 90.6 mm
- net 3.3V: track 80.8 -> 0.00 mm
- net GND: track 9.97 -> 81.1 mm, vias 9 -> 13
- net IMU_INT: track 0.00 -> 16.7 mm, vias 0 -> 1
- net IMU_AD0: track 0.00 -> 16.0 mm, vias 0 -> 1
- net A0_GYRO: track 12.7 -> 0.00 mm, vias 1 -> 0
- net 1.8V: track 0.00 -> 12.0 mm
- net LINE_RF: track 53.8 -> 43.7 mm
- net LINE_LF: track 52.5 -> 42.4 mm
- net INT_GYRO: track 10.0 -> 0.00 mm
- net SDA0: track 130.7 -> 121.6 mm
- net INT_ACCEL: track 8.98 -> 0.00 mm
- net A0_ACCEL: track 8.94 -> 0.00 mm
- net SCL0: track 131.0 -> 123.6 mm
- net SCL1: track 23.9 -> 28.2 mm, vias 0 -> 1
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- added copper zone on layer 1, net 1.8V
- added copper zone on layer 1, net 3V3
- removed copper zone on layer 1, net 3.3V
Other:
- board text added: "Gucci Controller Board V2.0"
- board text removed: "Gucci Controller Board Ver 2.0"

Commit message: FInal Check for Rev 2.0
Routing:
- net 3V3: track 90.6 -> 89.9 mm

Commit message: added comparator and updated library for gucci v2
Parts:
- added C19: 0.1uF, SparkFun-Capacitors:0603
- added R17, R18, R19, R20: 1k, SparkFun-Resistors:0603
- added U5: LM339-14-SOIC, Gucci_ControlBoard:14-SOIC
- moved C13 18.4 mm to (32.0, 42.0), turned to 0 degrees
- moved R14 14.1 mm to (23.0, 39.0)
- moved D2 11.0 mm to (24.0, 43.0)
- moved U2 9.00 mm to (28.0, 39.0)
- moved C12 6.71 mm to (32.0, 33.0)
- moved R12 3.00 mm to (44.0, 41.0)
- moved R4 3.00 mm to (38.0, 41.0)
- moved R8 3.00 mm to (41.0, 41.0)
- moved R10 2.00 mm to (4.00, 41.0)
- moved R2 2.00 mm to (-2.00, 41.0)
- moved R6 2.00 mm to (1.00, 41.0)
- moved C11 1.00 mm to (-9.00, 42.0)
- moved D1 1.00 mm to (-9.00, 39.0)
- moved R13 1.00 mm to (-5.00, 38.0)
Connections:
- new net LB_INT: R20.1, U1.17/A3, U5.13
- new net LF_INT: R18.1, U1.11, U5.2
- new net LINE_REF: U1.16/A2, U5.10, U5.4, U5.6, U5.8
- new net RB_INT: R19.1, U1.18/A4, U5.14
- new net RF_INT: R17.1, U1.10, U5.1
- net 3V3: now also R17.2, R18.2, R19.2, R20.2
- net 5V: now also C19.1, U5.3
- net GND: now also C19.2, U5.12
- net LINE_LB: now also U5.11
- net LINE_LF: now also U5.5
- net LINE_RB: now also U5.9
- net LINE_RF: now also U5.7
Routing:
- net LINE_RF: track 43.7 -> 79.9 mm, vias 0 -> 1
- net LINE_RB: track 6.67 -> 34.2 mm, vias 0 -> 1
- net LINE_REF: track 0.00 -> 19.7 mm, vias 0 -> 1
- net GND: track 81.1 -> 99.7 mm, vias 13 -> 12
- net LF_INT: track 0.00 -> 17.2 mm
- net RF_INT: track 0.00 -> 15.3 mm
- net LINE_LF: track 42.4 -> 57.6 mm, vias 0 -> 1
- net RB_INT: track 0.00 -> 14.7 mm
- net LB_INT: track 0.00 -> 14.2 mm, vias 0 -> 1
- net LINE_LB: track 6.45 -> 18.4 mm, vias 0 -> 1
- net 3V3: track 89.9 -> 98.9 mm
- net 3V_ENCODER2_I: track 10.6 -> 12.3 mm
- net 3V_ENCODER2_B: track 8.45 -> 9.43 mm
- net 3V_ENCODER1_A: track 10.6 -> 11.5 mm
- net 3V_ENCODER1_B: track 8.04 -> 8.67 mm
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
Commit message: moved start and line_ref pins
Connections:
- net LINE_REF: now also U1.A22; no longer U1.16/A2
- net START: now also U1.16/A2; no longer U1.15/A1
Routing:
- net LINE_REF: track 19.7 -> 31.6 mm
- net LINE_RF: track 79.9 -> 80.5 mm
Changed lines of the file:
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@@
 <drawing>
 <settings>
-<setting alwaysvectorfont="yes"/>
+<setting alwaysvectorfont="no"/>
 <setting verticaltext="up"/>
 </settings>
@@
 <contactref element="U5" pad="9"/>
 <wire x1="30" y1="52" x2="30" y2="48" width="0.2" layer="16"/>
-<wire x1="30" y1="48" x2="29" y2="47" width="0.2" layer="16"/>
-<wire x1="29" y1="47" x2="20" y2="47" width="0.2" layer="16"/>
-<wire x1="20" y1="47" x2="19" y2="46" width="0.2" layer="16"/>
-<wire x1="19" y1="46" x2="19" y2="42" width="0.2" layer="16"/>
-<wire x1="17" y1="40" x2="19" y2="42" width="0.2" layer="16"/>
+<wire x1="29.3" y1="47.3" x2="30" y2="48" width="0.2" layer="16"/>
 <wire x1="13.55" y1="41.7" x2="13.55" y2="40.45" width="0.2" layer="1"/>
 <wire x1="13.55" y1="40.45" x2="14" y2="40" width="0.2" layer="1"/>
 <via x="14" y="40" extent="1-16" drill="0.4"/>
-<wire x1="14" y1="40" x2="17" y2="40" width="0.2" layer="16"/>
+<wire x1="14" y1="40" x2="15" y2="40" width="0.2" layer="16"/>
+<wire x1="15" y1="40" x2="16.7" y2="41.7" width="0.2" layer="16"/>
+<wire x1="16.7" y1="45.7186625" x2="18.2813375" y2="47.3" width="0.2" layer="16"/>
+<wire x1="16.7" y1="41.7" x2="16.7" y2="45.7186625" width="0.2" layer="16"/>
+<wire x1="18.2813375" y1="47.3" x2="29.3" y2="47.3" width="0.2" layer="16"/>
 </signal>
 <signal name="LINE_RF">
@@
 <via x="17" y="37" extent="1-16" drill="0.4"/>
 <wire x1="17" y1="37" x2="18" y2="38" width="0.2" layer="16"/>
-<wire x1="18" y1="38" x2="18" y2="40" width="0.2" layer="16"/>
-<wire x1="18" y1="40" x2="22" y2="44" width="0.2" layer="16"/>
-<wire x1="22" y1="44" x2="35" y2="44" width="0.2" layer="16"/>
+<wire x1="18" y1="38" x2="18" y2="41" width="0.2" layer="16"/>
+<wire x1="18" y1="41" x2="21" y2="44" width="0.2" layer="16"/>
+<wire x1="21" y1="44" x2="35" y2="44" width="0.2" layer="16"/>
 <wire x1="35" y1="44" x2="36" y2="43" width="0.2" layer="16"/>
 <wire x1="36" y1="43" x2="36" y2="40" width="0.2" layer="16"/>
@@
 <signal name="START">
 <contactref element="J15" pad="3"/>
-<contactref element="U1" pad="15/A1"/>
-<wire x1="17" y1="52" x2="17" y2="46.62" width="0.2" layer="1"/>
-<wire x1="17" y1="46.62" x2="18" y2="45.62" width="0.2" layer="1"/>
+<contactref element="U1" pad="16/A2"/>
+<wire x1="15.46" y1="45.62" x2="17" y2="47.16" width="0.2" layer="1"/>
+<wire x1="17" y1="47.16" x2="17" y2="52" width="0.2" layer="1"/>
 </signal>
 <signal name="ENCODER1_A">
@@
 <contactref element="U5" pad="10"/>
 <contactref element="U5" pad="8"/>
-<contactref element="U1" pad="16/A2"/>
-<wire x1="16" y1="42" x2="15.46" y2="42.54" width="0.2" layer="16"/>
-<via x="16" y="42" extent="1-16" drill="0.4"/>
 <wire x1="13.55" y1="38.55" x2="13.55" y2="36.3" width="0.2" layer="1"/>
-<wire x1="14.82" y1="39.82" x2="14" y2="39" width="0.2" layer="1"/>
 <wire x1="14" y1="39" x2="13.55" y2="38.55" width="0.2" layer="1"/>
-<wire x1="14.82" y1="39.82" x2="16" y2="41" width="0.2" layer="1"/>
-<wire x1="16" y1="41" x2="16" y2="42" width="0.2" layer="1"/>
-<wire x1="14.82" y1="41.7" x2="15.7" y2="41.7" width="0.2" layer="1"/>
-<wire x1="15.7" y1="41.7" x2="16" y2="42" width="0.2" layer="1"/>
+<wire x1="14" y1="39" x2="16" y2="41" width="0.2" layer="1"/>
 <wire x1="11.01" y1="36.3" x2="11.01" y2="35.59" width="0.2" layer="1"/>
 <wire x1="11.01" y1="35.59" x2="11.6" y2="35" width="0.2" layer="1"/>
@@
 <wire x1="13.0226" y1="40.9574" x2="13.0226" y2="40.0502375" width="0.2" layer="1"/>
 <wire x1="13.0226" y1="40.0502375" x2="14" y2="39.0728375" width="0.2" layer="1"/>
-<wire x1="15.46" y1="42.54" x2="15.46" y2="45.62" width="0.2" layer="16"/>
+<contactref element="U1" pad="A22"/>
+<wire x1="16" y1="41" x2="17" y2="41" width="0.2" layer="1"/>
+<via x="17" y="41" extent="1-16" drill="0.4"/>
+<wire x1="17" y1="41" x2="19" y2="43" width="0.2" layer="16"/>
+<wire x1="19" y1="45.6" x2="20.1" y2="46.7" width="0.2" layer="16"/>
+<wire x1="20.1" y1="46.7" x2="27.08" y2="46.7" width="0.2" layer="16"/>
+<wire x1="27.08" y1="46.7" x2="28.16" y2="45.62" width="0.2" layer="16"/>
+<wire x1="19" y1="43" x2="19" y2="45.6" width="0.2" layer="16"/>
+<wire x1="14.82" y1="41.7" x2="15.52" y2="41" width="0.2" layer="1"/>
+<wire x1="15.52" y1="41" x2="16" y2="41" width="0.2" layer="1"/>
 </signal>
 <signal name="RB_INT">
