File: Gucci/v2 pcb/Gucci_ControlBoard.brd (EAGLE design)
At the start: 66 x 56 mm, 64 parts, among them J1 JST_PH_1X05_90, J10 JST_PH_1X03, J11 JST_PHD_2X04, J12 JST_PHD_2X04, J15 JST_PH_1X03_90, J2 JST_PH_1X05_90, J3 JST_PH_1X05_90, J4 JST_PH_1X05_90, J5 JST_PH_1X05_90, J6 JST_PH_1X05_90, J7 JST_PH_1X03_90, J8 JST_PH_1X03_90, J9 JST_PH_1X03, U1 TEENSY_3.6_DIL, U2 AP2114H-3.3TRG1, U3 AP2114H-1.8TRG1, U4 ICM-20948, U5 LM339-14-SOIC

Commit message: level shifter
added level shifter to gucci and kirbi. the part is in gucci's library. the relevant area on the boards should be very similar, but not identical
Parts:
- added R21: 200k, SparkFun-Resistors:0603
- added R22, R23: 10k, SparkFun-Resistors:0603
- added U6: PCA9306_LSSOP, Gucci_ControlBoard:8-LSSOP
- moved C16 4.00 mm to (23.0, 17.0)
- moved C17 4.00 mm to (27.0, 22.0)
- moved C18 4.00 mm to (18.0, 18.0)
- moved U4 4.00 mm to (23.0, 21.0)
- moved R16 3.27 mm to (12.0, 23.7), turned to 90 degrees
- moved R15 3.00 mm to (14.4, 23.7), turned to 90 degrees
Connections:
- new net N$7: R21.1, U6.P$7, U6.P$8
- new net SCL2: R16.1, U1.3, U6.P$6
- new net SDA2: R15.1, U1.4, U6.P$5
- net 1.8V: now also R22.2, R23.2, U6.P$2; no longer R15.2, R16.2
- net 3V3: now also R15.2, R16.2, R21.2
- net GND: now also U6.P$1
- net SCL1: now also R23.1, U6.P$3; no longer R16.1, U1.3
- net SDA1: now also R22.1, U6.P$4; no longer R15.1, U1.4
Routing:
- net SCL2: track 0.00 -> 21.4 mm
- net 3V3: track 98.9 -> 119.0 mm
- net SDA2: track 0.00 -> 18.7 mm
- net SCL1: track 28.2 -> 15.1 mm, vias 1 -> 0
- net SDA1: track 23.4 -> 10.3 mm, vias 1 -> 0
- net N$7: track 0.00 -> 2.47 mm
- net GND: track 99.7 -> 101.9 mm
- net IMU_AD0: track 16.0 -> 17.2 mm

Commit message: fixed silkscreens
Parts:
- moved U$3 5.10 mm to (30.0, 14.0)
Changed lines of the file:
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@@
 <layer number="14" name="Route14" color="22" fill="1" visible="no" active="no"/>
 <layer number="15" name="Route15" color="23" fill="1" visible="no" active="no"/>
-<layer number="16" name="Bottom" color="1" fill="1" visible="yes" active="yes"/>
+<layer number="16" name="Bottom" color="1" fill="1" visible="no" active="yes"/>
 <layer number="17" name="Pads" color="2" fill="1" visible="yes" active="yes"/>
 <layer number="18" name="Vias" color="2" fill="1" visible="yes" active="yes"/>
@@
 <layer number="20" name="Dimension" color="24" fill="1" visible="yes" active="yes"/>
 <layer number="21" name="tPlace" color="7" fill="1" visible="yes" active="yes"/>
-<layer number="22" name="bPlace" color="7" fill="1" visible="yes" active="yes"/>
+<layer number="22" name="bPlace" color="7" fill="1" visible="no" active="yes"/>
 <layer number="23" name="tOrigins" color="15" fill="1" visible="yes" active="yes"/>
-<layer number="24" name="bOrigins" color="15" fill="1" visible="yes" active="yes"/>
+<layer number="24" name="bOrigins" color="15" fill="1" visible="no" active="yes"/>
 <layer number="25" name="tNames" color="7" fill="1" visible="yes" active="yes"/>
-<layer number="26" name="bNames" color="7" fill="1" visible="yes" active="yes"/>
-<layer number="27" name="tValues" color="7" fill="1" visible="no" active="yes"/>
+<layer number="26" name="bNames" color="7" fill="1" visible="no" active="yes"/>
+<layer number="27" name="tValues" color="7" fill="1" visible="yes" active="yes"/>
 <layer number="28" name="bValues" color="7" fill="1" visible="no" active="yes"/>
 <layer number="29" name="tStop" color="7" fill="3" visible="no" active="yes"/>
@@
 <layer number="38" name="bTest" color="7" fill="1" visible="no" active="yes"/>
 <layer number="39" name="tKeepout" color="4" fill="11" visible="yes" active="yes"/>
-<layer number="40" name="bKeepout" color="1" fill="11" visible="yes" active="yes"/>
+<layer number="40" name="bKeepout" color="1" fill="11" visible="no" active="yes"/>
 <layer number="41" name="tRestrict" color="4" fill="10" visible="yes" active="yes"/>
-<layer number="42" name="bRestrict" color="1" fill="10" visible="yes" active="yes"/>
+<layer number="42" name="bRestrict" color="1" fill="10" visible="no" active="yes"/>
 <layer number="43" name="vRestrict" color="2" fill="10" visible="no" active="yes"/>
 <layer number="44" name="Drills" color="7" fill="1" visible="no" active="yes"/>
@@
 <layer number="50" name="dxf" color="7" fill="1" visible="no" active="no"/>
 <layer number="51" name="tDocu" color="7" fill="1" visible="yes" active="yes"/>
-<layer number="52" name="bDocu" color="7" fill="1" visible="yes" active="yes"/>
+<layer number="52" name="bDocu" color="7" fill="1" visible="no" active="yes"/>
 <layer number="53" name="tGND_GNDA" color="7" fill="9" visible="no" active="no"/>
 <layer number="54" name="bGND_GNDA" color="1" fill="9" visible="no" active="no"/>
@@
 </element>
 <element name="R15" library="SparkFun-Resistors" package="0603" value="10k" x="14.4" y="23.7" smashed="yes" rot="R90">
-<attribute name="NAME" x="13.638" y="23.7" size="0.8128" layer="25" font="vector" ratio="20" rot="R90" align="bottom-center"/>
+<attribute name="NAME" x="14.3" y="26.138" size="0.8128" layer="25" font="vector" ratio="20" rot="R180" align="bottom-center"/>
 <attribute name="PROD_ID" value="RES-07856" x="14.4" y="23.7" size="1.778" layer="27" rot="R90" display="off"/>
-<attribute name="VALUE" x="15.162" y="23.7" size="0.8128" layer="21" font="vector" ratio="20" rot="R90" align="top-center"/>
+<attribute name="VALUE" x="14.2" y="21.938" size="0.8128" layer="21" font="vector" ratio="20" align="top-center"/>
 </element>
 <element name="R16" library="SparkFun-Resistors" package="0603" value="10k" x="12" y="23.7" smashed="yes" rot="R90">
-<attribute name="NAME" x="11.238" y="23.7" size="0.8128" layer="25" font="vector" ratio="20" rot="R90" align="bottom-center"/>
+<attribute name="NAME" x="12" y="26.138" size="0.8128" layer="25" font="vector" ratio="20" rot="R180" align="bottom-center"/>
 <attribute name="PROD_ID" value="RES-07856" x="12" y="23.7" size="1.778" layer="27" rot="R90" display="off"/>
-<attribute name="VALUE" x="12.762" y="23.7" size="0.8128" layer="21" font="vector" ratio="20" rot="R90" align="top-center"/>
+<attribute name="VALUE" x="11.7" y="21.938" size="0.8128" layer="21" font="vector" ratio="20" align="top-center"/>
 </element>
 <element name="C16" library="SparkFun-Capacitors" library_urn="urn:adsk.eagle:library:510" package="0603" package3d_urn="urn:adsk.eagle:package:37414/1" value="0.1uF" x="23" y="17" smashed="yes">
-<attribute name="NAME" x="20" y="15.762" size="0.8128" layer="25" font="vector" ratio="20" align="bottom-center"/>
+<attribute name="NAME" x="23" y="17.762" size="0.8128" layer="25" font="vector" ratio="20" align="bottom-center"/>
 <attribute name="PROD_ID" value="CAP-00810" x="23" y="17" size="1.778" layer="27" display="off"/>
 <attribute name="VALUE" x="23" y="16.238" size="0.8128" layer="21" font="vector" ratio="20" align="top-center"/>
@@
 <element name="U$1" library="RoboJackets-Aesthetics" package="ROBOJACKETS" value="" x="33" y="38" smashed="yes" rot="MR0"/>
 <element name="U$2" library="RoboJackets-Aesthetics" package="ROBOBUZZ_1.4X" value="" x="20" y="8" smashed="yes" rot="MR0"/>
-<element name="U$3" library="RoboJackets-Aesthetics" package="ROBOBUZZ_0.4X" value="" x="25" y="13" smashed="yes"/>
+<element name="U$3" library="RoboJackets-Aesthetics" package="ROBOBUZZ_0.4X" value="" x="30" y="14" smashed="yes"/>
 <element name="U5" library="Gucci_ControlBoard" package="14-SOIC" value="LM339-14-SOIC" x="11" y="39" smashed="yes">
 <attribute name="NAME" x="7.8" y="43.9" size="1.27" layer="25" rot="R180"/>
@@
 <attribute name="VALUE" x="5" y="33.362" size="0.8128" layer="21" font="vector" ratio="20" rot="R180" align="top-center"/>
 </element>
-<element name="U6" library="Gucci_ControlBoard" package="8-LSSOP" value="PCA9306_LSSOP" x="12" y="19" rot="R180"/>
-<element name="R21" library="SparkFun-Resistors" package="0603" value="200k" x="9" y="15.6" rot="R270">
+<element name="U6" library="Gucci_ControlBoard" package="8-LSSOP" value="PCA9306_LSSOP" x="12" y="19" smashed="yes" rot="R180">
+<attribute name="NAME" x="13.5" y="16.4" size="1.27" layer="25" rot="R180"/>
+<attribute name="VALUE" x="14" y="21" size="0.8128" layer="27" rot="R180"/>
+</element>
+<element name="R21" library="SparkFun-Resistors" package="0603" value="200k" x="9" y="15.6" smashed="yes" rot="R270">
+<attribute name="NAME" x="9.762" y="15.6" size="0.8128" layer="25" font="vector" ratio="20" rot="R270" align="bottom-center"/>
 <attribute name="PROD_ID" value="RES-07856" x="9" y="15.6" size="1.778" layer="27" rot="R270" display="off"/>
-</element>
-<element name="R22" library="SparkFun-Resistors" package="0603" value="10k" x="18.9" y="23.7" rot="R90">
+<attribute name="VALUE" x="8.238" y="15.6" size="0.8128" layer="21" font="vector" ratio="20" rot="R270" align="top-center"/>
+</element>
+<element name="R22" library="SparkFun-Resistors" package="0603" value="10k" x="18.9" y="23.7" smashed="yes" rot="R90">
+<attribute name="NAME" x="18.9" y="26.138" size="0.8128" layer="25" font="vector" ratio="20" rot="R180" align="bottom-center"/>
 <attribute name="PROD_ID" value="RES-07856" x="18.9" y="23.7" size="1.778" layer="27" rot="R90" display="off"/>
-</element>
-<element name="R23" library="SparkFun-Resistors" package="0603" value="10k" x="16.7" y="23.7" rot="R90">
+<attribute name="VALUE" x="18.9" y="21.938" size="0.8128" layer="21" font="vector" ratio="20" align="top-center"/>
+</element>
+<element name="R23" library="SparkFun-Resistors" package="0603" value="10k" x="16.7" y="23.7" smashed="yes" rot="R90">
+<attribute name="NAME" x="16.6" y="26.138" size="0.8128" layer="25" font="vector" ratio="20" rot="R180" align="bottom-center"/>
 <attribute name="PROD_ID" value="RES-07856" x="16.7" y="23.7" size="1.778" layer="27" rot="R90" display="off"/>
+<attribute name="VALUE" x="16.6" y="21.938" size="0.8128" layer="21" font="vector" ratio="20" align="top-center"/>
 </element>
 </elements>

Commit message: idc connectors
gucci should be done now
Parts:
- removed C7: 0.1uF, SparkFun-Capacitors:0603
- removed J1, J2, J3, J4, J5, J6: JST_PH_1X05_90, Gucci_ControlBoard:JST_PH_1X05_90
- removed J10, J9: JST_PH_1X03, Gucci_ControlBoard:JST_PH_1X03
- removed J15, J7, J8: JST_PH_1X03_90, Gucci_ControlBoard:JST_PH_1X03_90
- removed R20: 1k, SparkFun-Resistors:0603
- removed U6: PCA9306_LSSOP, Gucci_ControlBoard:8-LSSOP
- added D3: 1.8V, SparkFun-LED:LED-0603
- added IMU: ICM-20948, ICM-20948:QFN40P300X300X105-25N
- added LINE_LF, LINE_RF, START: AMPHENOL_2X02_2.54MM_SHROUD, Gucci_ControlBoard:AMPHENOL_2X02_2.54MM_SHROUD
- added TOF2, TOF3, TOF4, TOF5, TOF_0, TOF_1: AMPHENOL_2X03_2.54MM_SHROUD, Gucci_ControlBoard:AMPHENOL_2X03_2.54MM_SHROUD
- D1: value Green -> 5V
- D2: value Green -> 3.3V
- R13: value 330 -> 1650
- R14: value 220 -> 800
- R19: value 1k -> 50
- U4: value ICM-20948 -> LM339-14-SOIC; device ICM-20948:QFN40P300X300X105-25N -> Gucci_ControlBoard:14-SOIC
- U5: value LM339-14-SOIC -> PCA9306_LSSOP; device Gucci_ControlBoard:14-SOIC -> Gucci_ControlBoard:8-LSSOP
- moved R19 31.0 mm to (27.0, 14.0)
- moved U4 21.6 mm to (11.0, 39.0)
- moved U5 20.0 mm to (12.0, 19.0), turned to 180 degrees
- moved C5 9.22 mm to (36.0, 3.00), turned to 90 degrees
- moved C3 7.21 mm to (2.00, 3.00), turned to 90 degrees
- moved C4 7.21 mm to (19.0, 3.00), turned to 90 degrees
- moved U$2 6.00 mm to (20.0, 2.00)
- moved C8 2.79 mm to (25.2, 52.0), turned to 90 degrees
- moved C6 2.24 mm to (44.0, 19.0)
- moved C15 1.14 mm to (13.7, 10.9), turned to 270 degrees
- moved C14 1.08 mm to (24.4, 10.9), turned to 270 degrees
- moved C1 1.00 mm to (-6.00, 25.0)
- moved R17 0.50 mm to (19.0, 32.5)
- renumbered J11 to R_ESC, J12 to L_ESC, J13 to R_ENC, J14 to L_ENC
Connections:
- removed net LB_INT: R20.1, U1.17/A3, U5.13
- removed net LINE_LB: J7.2, U1.19/A5, U5.11
- removed net LINE_RB: J8.2, U1.A21, U5.9
- removed net RB_INT: R19.1, U1.18/A4, U5.14
- new net N$4: D3.C, R19.1
- net 1.8V: now also D3.A, IMU.13, IMU.22, IMU.8, U5.P$2; no longer U4.13, U4.22, U4.8, U6.P$2
- net 3V3: now also LINE_LF.1, LINE_RF.1, START.3, TOF2.6, TOF3.6, TOF4.6, TOF5.6, TOF_0.6, TOF_1.6; no longer C7.1, J1.1, J10.3, J15.2, J2.1, J3.1, J4.1, J5.1, J6.1, J7.3, J8.3, J9.3, R19.2, R20.2
- net 5V: now also U4.3; no longer U5.3
- net GND: now also IMU.11, IMU.18, IMU.20, LINE_LF.3, LINE_RF.3, R19.2, START.2, TOF2.5, TOF3.5, TOF4.5, TOF5.5, TOF_0.5, TOF_1.5, U4.12, U5.P$1; no longer C7.2, J1.2, J10.1, J15.1, J2.2, J3.2, J4.2, J5.2, J6.2, J7.1, J8.1, J9.1, U4.11, U4.18, U4.20, U5.12, U6.P$1
- net IMU_AD0: now also IMU.9; no longer U4.9
- net IMU_INT: now also IMU.12; no longer U4.12
- net LF_INT: now also R17.1, U1.10, U4.1; no longer R18.1, U1.11, U5.2
- net LINE_LF: now also LINE_LF.2, U1.35/A16, U4.7; no longer J9.2, U1.23/A9, U5.5
- net LINE_REF: now also U4.4, U4.6; no longer U5.10, U5.4, U5.6, U5.8
- net LINE_RF: now also LINE_RF.2, U1.23/A9, U4.5; no longer J10.2, U1.35/A16, U5.7
- net N$3: now also IMU.10; no longer U4.10
- net N$7: now also U5.P$7, U5.P$8; no longer U6.P$7, U6.P$8
- net RF_INT: now also R18.1, U1.11, U4.2; no longer R17.1, U1.10, U5.1
- net SCL0: now also TOF2.2, TOF3.2, TOF4.2, TOF5.2, TOF_0.2, TOF_1.2; no longer J1.4, J2.4, J3.4, J4.4, J5.4, J6.4
- net SCL1: now also IMU.23, U5.P$3; no longer U4.23, U6.P$3
- net SCL2: now also U5.P$6; no longer U6.P$6
- net SDA0: now also TOF2.1, TOF3.1, TOF4.1, TOF5.1, TOF_0.1, TOF_1.1; no longer J1.5, J2.5, J3.5, J4.5, J5.5, J6.5
- net SDA1: now also IMU.24, U5.P$4; no longer U4.24, U6.P$4
- net SDA2: now also U5.P$5; no longer U6.P$5
- net SHDN0: now also TOF_0.3; no longer J1.3
- net SHDN1: now also TOF_1.3; no longer J2.3
- net SHDN2: now also TOF2.3; no longer J3.3
- net SHDN3: now also TOF3.3; no longer J4.3
- net SHDN4: now also TOF4.3; no longer J5.3
- net SHDN5: now also TOF5.3; no longer J6.3
- net START: now also START.1; no longer J15.3
Routing:
- net 3V3: track 119.0 -> 82.0 mm
- net LINE_RB: track 34.2 -> 0.00 mm, vias 1 -> 0
- net SDA0: track 121.6 -> 150.7 mm
- net LINE_LF: track 57.6 -> 80.3 mm
- net LINE_RF: track 80.5 -> 60.0 mm
- net LINE_LB: track 18.4 -> 0.00 mm, vias 1 -> 0
- net GND: track 101.9 -> 119.4 mm, vias 12 -> 10
- net RB_INT: track 14.7 -> 0.00 mm
- net LB_INT: track 14.2 -> 0.00 mm, vias 1 -> 0
- net LINE_REF: track 31.6 -> 27.5 mm
- net N$4: track 0.00 -> 2.27 mm
- net RF_INT: track 15.3 -> 17.2 mm
- net SCL0: track 123.6 -> 125.5 mm
- net LF_INT: track 17.2 -> 15.6 mm
- net SHDN1: track 22.0 -> 20.9 mm
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
Commit message: finished v2 pcb and updated library
Parts:
- removed R23: 10k, SparkFun-Resistors:0603
- removed TOF4: AMPHENOL_2X03_2.54MM_SHROUD, Gucci_ControlBoard:AMPHENOL_2X03_2.54MM_SHROUD
- added C20: 4.7uF, SparkFun-Capacitors:0603
- added C7: 0.1uF, SparkFun-Capacitors:0603
- added L_MOT, R_MOT: (no value), pinhead:1X02
- added R20: 200k, SparkFun-Resistors:0603
- added TOF_6: AMPHENOL_2X03_2.54MM_SHROUD, Gucci_ControlBoard:AMPHENOL_2X03_2.54MM_SHROUD
- added U6: MAX4173-SOT-23, Gucci_ControlBoard:SOT-23
- added U7: LM393-8-SOIC, Gucci_ControlBoard:8-SOIC
- C1, C2: value 0.1uF -> 15pF
- C10, C9: value 1uF -> 0.1uF
- C12, C13: value 4.7uF -> 1uF
- C14, C15: value 4.7uF -> 0.1uF
- C17, C18, C19: value 0.1uF -> 4.7uF
- D1: value 5V -> 1.8V
- D3: value 1.8V -> 5V
- R10, R4, R8: value 3k -> 2k
- R11, R3, R7: value 2k -> 3k
- R12: value 3k -> 10k
- R13: value 1650 -> 10k
- R14: value 800 -> 1k
- R15: value 10k -> 3k
- R16: value 10k -> 800
- R17: value 1k -> 1.65k
- R18: value 1k -> 10k
- R19: value 50 -> 10k
- R21: value 200k -> 50
- R22: value 10k -> 1k
- U2: value AP2114H-3.3TRG1 -> PCA9306_LSSOP; device Gucci_ControlBoard:SOT-223 -> Gucci_ControlBoard:8-LSSOP
- U3: value AP2114H-1.8TRG1 -> AP2114H-3.3TRG1
- U4: value LM339-14-SOIC -> AP2114H-1.8TRG1; device Gucci_ControlBoard:14-SOIC -> Gucci_ControlBoard:SOT-223
- U5: value PCA9306_LSSOP -> MAX4173-SOT-23; device Gucci_ControlBoard:8-LSSOP -> Gucci_ControlBoard:SOT-23
- moved C8 49.4 mm to (19.0, 3.00)
- moved R1 48.0 mm to (42.0, 49.0), turned to 180 degrees
- moved TOF_1 48.0 mm to (43.0, 9.00), turned to 225 degrees
- moved R8 47.7 mm to (-6.00, 49.0), turned to 0 degrees
- moved C5 47.4 mm to (-6.00, 25.0), turned to 270 degrees
- moved R9 45.2 mm to (47.0, 49.0), turned to 180 degrees
- moved C6 44.6 mm to (0.00, 12.0), turned to 0 degrees
- moved R7 41.8 mm to (1.00, 41.0), turned to 90 degrees
- moved C16 40.6 mm to (-9.00, 42.0)
- moved D1 40.6 mm to (23.0, 14.0)
- moved D3 40.6 mm to (-9.00, 39.0)
- moved R2 40.0 mm to (38.0, 41.0)
- moved U5 34.5 mm to (29.0, 49.0), turned to 90 degrees
- moved R12 34.3 mm to (14.4, 23.7)
- moved C9 34.0 mm to (36.0, 3.00), turned to 90 degrees
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- renumbered TOF2 to TOF_3, TOF3 to TOF_4, TOF5 to TOF_2, TOF_0 to TOF_5
Connections:
- new net CURRENT_L: U1.A21, U5.P$6
- new net CURRENT_R: U1.13, U6.P$6
- new net L_MOT+: L_MOT.2, U5.P$4
- new net L_MOT-: L_MOT.1, U5.P$5
- new net R_MOT+: R_MOT.2, U6.P$4
- new net R_MOT-: R_MOT.1, U6.P$5
- net 1.8V: now also C20.1, C3.1, C4.1, D1.A, R18.2, R19.2, U2.P$2, U4.2, U4.4; no longer C15.1, C17.1, C18.1, D3.A, R22.2, R23.2, U3.2, U3.4, U5.P$2
- net 3V3: now also C10.1, C11.1, C18.1, C19.1, C7.1, C9.1, R12.2, R13.2, R14.2, R20.2, R22.2, TOF_6.6, U3.2, U3.4, U4.3; no longer C1.1, C13.1, C14.1, C2.1, C3.1, C4.1, R15.2, R16.2, R17.2, R18.2, R21.2, TOF4.6, U2.2, U2.4, U3.3
- net 3V_ENCODER1_A: now also R6.2, R8.2; no longer R1.2, R2.2
- net 3V_ENCODER1_B: now also R7.2; no longer R6.2
- net 3V_ENCODER1_I: now also R15.2; no longer R9.2
- net 3V_ENCODER2_A: now also R2.2; no longer R3.2
- net 3V_ENCODER2_B: now also R1.2, R3.2; no longer R7.2, R8.2
- net 3V_ENCODER2_I: now also R9.2; no longer R12.2
- net 5V: now also C13.1, C14.1, C16.1, C17.1, D3.A, U3.3, U5.P$3, U6.P$3, U7.P$8; no longer C10.1, C11.1, C19.1, C9.1, D1.A, U2.3, U4.3
- net ENCODER1_A: now also R8.1; no longer R1.1
- net ENCODER2_A: now also R4.1; no longer R3.1
- net ENCODER2_B: now also R1.1; no longer R7.1
- net GND: now also C20.2, C7.2, R11.1, R15.1, R16.2, R17.2, R21.2, R3.1, R7.1, TOF_6.5, U2.P$1, U4.1, U5.P$2, U6.P$1, U6.P$2, U7.P$4; no longer R10.1, R12.1, R13.2, R14.2, R19.2, R4.1, R8.1, TOF4.5, U2.1, U4.12
- net LF_INT: now also C2.1, R22.1, U1.18/A4, U7.P$7; no longer R17.1, U1.10, U4.1
- net LINE_LF: now also U7.P$5; no longer U4.7
- net LINE_REF: now also U7.P$2, U7.P$6; no longer U4.4, U4.6
- net LINE_RF: now also U7.P$3; no longer U4.5
- net N$1: now also D3.C, R17.1; no longer D1.C, R13.1
- net N$2: now also R16.1; no longer R14.1
- net N$3: now also C15.1; no longer C16.1
- net N$4: now also D1.C, R21.1; no longer D3.C, R19.1
- net N$5: now also R10.1; no longer R9.1
- net N$7: now also R20.1, U2.P$7, U2.P$8; no longer R21.1, U5.P$7, U5.P$8
- net N$8: now also R9.1; no longer R11.1
- net RF_INT: now also C1.1, R14.1, U1.19/A5, U7.P$1; no longer R18.1, U1.11, U4.2
- net SCL0: now also TOF_6.2; no longer TOF4.2
- net SCL1: now also R19.1, U2.P$3; no longer R23.1, U5.P$3
- net SCL2: now also R13.1, U2.P$6; no longer R16.1, U5.P$6
- net SDA0: now also TOF_6.1; no longer TOF4.1
- net SDA1: now also R18.1, U2.P$4; no longer R22.1, U5.P$4
- net SDA2: now also R12.1, U2.P$5; no longer R15.1, U5.P$5
- net SHDN1: now also TOF_6.3; no longer TOF_1.3
- net SHDN4: now also TOF_1.3; no longer TOF4.3
- net START: now also U1.17/A3; no longer U1.16/A2
Routing:
- net GND: track 119.4 -> 128.8 mm, vias 10 -> 11
- net RF_INT: track 17.2 -> 9.72 mm
- net L_MOT-: track 0.00 -> 7.33 mm
- net R_MOT+: track 0.00 -> 7.31 mm
- net CURRENT_L: track 0.00 -> 6.41 mm
- net LINE_RF: track 60.0 -> 54.1 mm
- net 3V3: track 82.0 -> 87.5 mm
- net CURRENT_R: track 0.00 -> 5.46 mm
- net L_MOT+: track 0.00 -> 4.12 mm
- net R_MOT-: track 0.00 -> 4.10 mm
- net SCL2: track 21.4 -> 24.4 mm
- net LF_INT: track 15.6 -> 12.8 mm
- net LINE_REF: track 27.5 -> 30.2 mm
- net SDA2: track 18.7 -> 21.0 mm
- net LINE_LF: track 80.3 -> 81.2 mm
Other:
- board text added: "+"
- board text added: "-"
