File: Gucci/v2 pcb/Gucci_ControlBoard.brd (EAGLE design)
At the start: 66 x 56 mm, 71 parts, among them U1 TEENSY_3.6_DIL, U2 PCA9306_LSSOP, U3 AP2114H-3.3TRG1, U4 AP2114H-1.8TRG1, U5 MAX4173-SOT-23, U6 MAX4173-SOT-23, U7 LM393-8-SOIC

Commit message: silkscreen tweaks
Parts:
- C1, C2: value 15pF -> 0.1uF
- C12, C13: value 1uF -> 0.1uF
- C15, C16: value 0.1uF -> 15pF
- C5, C7: value 0.1uF -> 1uF
- D1: value 1.8V -> 5V
- D3: value 5V -> 1.8V
- R10, R4, R8: value 2k -> 3k
- R11, R3, R7: value 3k -> 2k
- R12: value 10k -> 3k
- R13: value 10k -> 200k
- R14: value 1k -> 10k
- R15: value 3k -> 10k
- R16: value 800 -> 10k
- R17: value 1.65k -> 10k
- R18: value 10k -> 1.65k
- R19: value 10k -> 800
- R20: value 200k -> 50
- R21: value 50 -> 1k
- U1: value TEENSY_3.6_DIL -> PCA9306_LSSOP; device Teensy_3_and_LC_Series_Boards_v1.4:TEENSY_3.6_DIL -> Gucci_ControlBoard:8-LSSOP
- U2: value PCA9306_LSSOP -> TEENSY_3.6_DIL; device Gucci_ControlBoard:8-LSSOP -> Teensy_3_and_LC_Series_Boards_v1.4:TEENSY_3.6_DIL
- U3: value AP2114H-3.3TRG1 -> MAX4173-SOT-23; device Gucci_ControlBoard:SOT-223 -> Gucci_ControlBoard:SOT-23
- U4: value AP2114H-1.8TRG1 -> MAX4173-SOT-23; device Gucci_ControlBoard:SOT-223 -> Gucci_ControlBoard:SOT-23
- U5: value MAX4173-SOT-23 -> LM393-8-SOIC; device Gucci_ControlBoard:SOT-23 -> Gucci_ControlBoard:8-SOIC
- U6: value MAX4173-SOT-23 -> AP2114H-1.8TRG1; device Gucci_ControlBoard:SOT-23 -> Gucci_ControlBoard:SOT-223
- U7: value LM393-8-SOIC -> AP2114H-3.3TRG1; device Gucci_ControlBoard:8-SOIC -> Gucci_ControlBoard:SOT-223
- moved C11 51.7 mm to (19.0, 3.00)
- moved C8 51.7 mm to (6.00, 53.0)
- moved R8 50.6 mm to (44.0, 41.0), turned to 90 degrees
- moved TOF_1 48.0 mm to (-5.00, 9.00), turned to 135 degrees
- moved TOF_6 48.0 mm to (43.0, 9.00), turned to 225 degrees
- moved R7 46.7 mm to (47.0, 49.0), turned to 180 degrees
- moved R3 41.8 mm to (0.00, 49.0), turned to 0 degrees
- moved R10 40.8 mm to (41.0, 41.0), turned to 90 degrees
- moved D1 40.6 mm to (-9.00, 39.0)
- moved D3 40.6 mm to (23.0, 14.0)
- moved R1 40.2 mm to (2.00, 53.0), turned to 270 degrees
- moved U4 39.3 mm to (29.0, 49.0), turned to 90 degrees
- moved U6 38.3 mm to (19.0, 11.0), turned to 0 degrees
- moved C5 38.1 mm to (32.0, 23.0), turned to 90 degrees
- moved R21 37.4 mm to (11.4, 48.0)
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Connections:
- net 1.8V: now also C1.1, C17.1, C2.1, D3.A, R14.2, R15.2, U1.P$2, U6.2, U6.4; no longer C20.1, C3.1, C4.1, D1.A, R18.2, R19.2, U2.P$2, U4.2, U4.4
- net 3V3: now also C12.1, C13.1, C14.1, R16.2, R17.2, R21.2, U6.3, U7.2, U7.4; no longer C5.1, C6.1, C7.1, R12.2, R14.2, R20.2, U3.2, U3.4, U4.3
- net 3V_ENCODER1_A: now also R5.2, U2.22/A8; no longer R8.2, U1.22/A8
- net 3V_ENCODER1_B: now also R3.2, R4.2, U2.21/A7; no longer R5.2, R7.2, U1.21/A7
- net 3V_ENCODER1_I: now also R1.2, R2.2, U2.20/A6; no longer R10.2, R15.2, U1.20/A6
- net 3V_ENCODER2_A: now also R11.2, R12.2, U2.38/A19; no longer R2.2, R4.2, U1.38/A19
- net 3V_ENCODER2_B: now also R10.2, R9.2, U2.37/A18; no longer R1.2, R3.2, U1.37/A18
- net 3V_ENCODER2_I: now also R7.2, R8.2, U2.36/A17; no longer R11.2, R9.2, U1.36/A17
- net 5V: now also C20.1, C4.1, C5.1, C6.1, C7.1, D1.A, U2.VIN, U3.P$3, U4.P$3, U5.P$8, U7.3; no longer C12.1, C13.1, C14.1, C16.1, C17.1, D3.A, U1.VIN, U3.3, U5.P$3, U6.P$3, U7.P$8
- net CURRENT_L: now also U2.A21, U4.P$6; no longer U1.A21, U5.P$6
- net CURRENT_R: now also U2.13, U3.P$6; no longer U1.13, U6.P$6
- net ENCODER1_A: now also R5.1; no longer R8.1
- net ENCODER1_B: now also R3.1; no longer R5.1
- net ENCODER2_A: now also R11.1; no longer R4.1
- net ENCODER2_B: now also R9.1; no longer R1.1
- net GND: now also R10.1, R12.1, R18.2, R19.2, R20.2, R4.1, R8.1, U1.P$1, U2.AGND, U2.GND, U2.GND1, U3.P$1, U3.P$2, U4.P$1, U4.P$2, U5.P$4, U6.1, U7.1; no longer R11.1, R15.1, R16.2, R17.2, R21.2, R3.1, R7.1, U1.AGND, U1.GND, U1.GND1, U2.P$1, U3.1, U4.1, U5.P$1, U5.P$2, U6.P$1, U6.P$2, U7.P$4
- net IMU_AD0: now also U2.9; no longer U1.9
- net IMU_INT: now also U2.12; no longer U1.12
- net LF_INT: now also C15.1, R21.1, U2.18/A4, U5.P$7; no longer C2.1, R22.1, U1.18/A4, U7.P$7
- net LINE_LF: now also U2.35/A16, U5.P$5; no longer U1.35/A16, U7.P$5
- net LINE_REF: now also U2.A22, U5.P$2, U5.P$6; no longer U1.A22, U7.P$2, U7.P$6
- net LINE_RF: now also U2.23/A9, U5.P$3; no longer U1.23/A9, U7.P$3
- net L_MOT+: now also U4.P$4; no longer U5.P$4
- net L_MOT-: now also U4.P$5; no longer U5.P$5
- net N$1: now also D1.C, R18.1; no longer D3.C, R17.1
- net N$2: now also R19.1; no longer R16.1
- net N$3: now also C3.1; no longer C15.1
- net N$4: now also D3.C, R20.1; no longer D1.C, R21.1
- net N$5: now also R1.1; no longer R10.1
- net N$7: now also R13.1, U1.P$7, U1.P$8; no longer R20.1, U2.P$7, U2.P$8
- net N$8: now also R7.1; no longer R9.1
- net RF_INT: now also C16.1, R22.1, U2.19/A5, U5.P$1; no longer C1.1, R14.1, U1.19/A5, U7.P$1
- net RX0: now also U2.7; no longer U1.7
- net RX1: now also U2.27; no longer U1.27
- net R_MOT+: now also U3.P$4; no longer U6.P$4
- net R_MOT-: now also U3.P$5; no longer U6.P$5
- net SCL0: now also U2.33/A14; no longer U1.33/A14
- net SCL1: now also R14.1, U1.P$3; no longer R19.1, U2.P$3
- net SCL2: now also R16.1, U1.P$6, U2.3; no longer R13.1, U1.3, U2.P$6
- net SDA0: now also U2.34/A15; no longer U1.34/A15
- net SDA1: now also R15.1, U1.P$4; no longer R18.1, U2.P$4
- net SDA2: now also R17.1, U1.P$5, U2.4; no longer R12.1, U1.4, U2.P$5
- net SHDN0: now also TOF_3.3, U2.0; no longer TOF_5.3, U1.0
- net SHDN1: now also TOF_1.3, U2.1; no longer TOF_6.3, U1.1
- net SHDN2: now also TOF_5.3, U2.2; no longer TOF_3.3, U1.2
- net SHDN3: now also TOF_2.3, U2.30; no longer TOF_4.3, U1.30
- net SHDN4: now also TOF_6.3, U2.31/A12; no longer TOF_1.3, U1.31/A12
- net SHDN5: now also TOF_4.3, U2.32/A13; no longer TOF_2.3, U1.32/A13
- net START: now also U2.17/A3; no longer U1.17/A3
- net TX0: now also U2.8; no longer U1.8
- net TX1: now also U2.26; no longer U1.26

Commit message: missed decoup caps and silkscreen changes
Parts:
- added C21, C22: 4.7uF, SparkFun-Capacitors:0603
- added U$4: (no value), RoboJackets-Aesthetics:ROBOBUZZ_0.4X
- C15, C16: value 15pF -> 0.1uF
- C17, C18: value 4.7uF -> 15pF
- moved C9 51.0 mm to (6.00, 53.0)
- moved C8 46.3 mm to (31.0, 14.0), turned to 0 degrees
- moved C18 36.8 mm to (6.50, 43.0), turned to 90 degrees
- moved C19 35.1 mm to (13.7, 9.90), turned to 270 degrees
- moved C16 33.9 mm to (-8.40, 12.6), turned to 45 degrees
- moved TOF_2 33.5 mm to (-5.00, 9.00), turned to 135 degrees
- moved TOF_5 33.5 mm to (43.0, 9.00), turned to 225 degrees
- moved C17 32.1 mm to (12.0, 43.0), turned to 90 degrees
- moved TOF_3 28.3 mm to (10.0, 3.00), turned to 180 degrees
- moved TOF_4 28.3 mm to (28.0, 3.00), turned to 180 degrees
- moved C20 28.2 mm to (24.4, 9.90)
- moved C15 28.0 mm to (-11.0, 27.0), turned to 0 degrees
- moved C12 21.0 mm to (23.0, 3.00)
- moved C11 20.7 mm to (39.5, 5.70), turned to 135 degrees
- moved C10 19.1 mm to (49.0, 17.0), turned to 180 degrees
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Connections:
- net 1.8V: now also C19.1; no longer C17.1
- net 3V3: now also C15.1, C16.1, C20.1, C21.1; no longer C18.1, C19.1
- net 5V: now also C22.1; no longer C20.1
- net CURRENT_R: now also U2.14/A0; no longer U2.13
- net GND: now also C21.2, C22.2
- net LF_INT: now also C17.1; no longer C15.1
- net RF_INT: now also C18.1; no longer C16.1
- net SHDN0: now also TOF_1.3; no longer TOF_3.3
- net SHDN1: now also TOF_2.3; no longer TOF_1.3
- net SHDN2: now also TOF_3.3; no longer TOF_5.3
- net SHDN3: now also TOF_4.3; no longer TOF_2.3
- net SHDN4: now also TOF_5.3; no longer TOF_6.3
- net SHDN5: now also TOF_6.3; no longer TOF_4.3
Routing:
- net GND: track 128.8 -> 119.1 mm, vias 11 -> 9
- net 3V3: track 87.5 -> 93.4 mm
- net CURRENT_R: track 5.46 -> 6.21 mm
