File: Gucci/v2 pcb/Gucci_ControlBoard.brd (EAGLE design)
At the start: 66 x 56 mm, 61 parts, among them U1 PCA9306_LSSOP, U2 TEENSY_3.6_DIL, U3 MAX4173-SOT-23, U4 MAX4173-SOT-23, U5 LM393-8-SOIC, U6 AP2114H-1.8TRG1, U7 AP2114H-3.3TRG1

Commit message: NeoPixel for Kirbi/Fixed IMU
Added NeoPixel/Deleted IMU Interuppt/Tied IMU Address to Ground
Connections:
- removed net IMU_AD0: IMU.9, U2.9
- removed net IMU_INT: IMU.12, U2.12
- net GND: now also IMU.9
Routing:
- net IMU_AD0: track 17.2 -> 0.00 mm, vias 1 -> 0
- net IMU_INT: track 17.0 -> 0.00 mm, vias 1 -> 0
- net GND: track 107.0 -> 113.1 mm
Changed lines of the file:
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@@
 <contactref element="IMU" pad="20"/>
 <contactref element="IMU" pad="18"/>
-<contactref element="IMU" pad="11"/>
 <contactref element="C3" pad="2"/>
 <contactref element="C2" pad="2"/>
 <contactref element="C1" pad="2"/>
-<wire x1="23.6" y1="19.455" x2="23.6" y2="17.25" width="0.2" layer="1"/>
 <wire x1="23.6" y1="17.25" x2="23.85" y2="17" width="0.2" layer="1"/>
 <wire x1="-8.15" y1="42" x2="-7" y2="42" width="0.2" layer="1"/>
@@
 <wire x1="45.8" y1="49" x2="45" y2="49" width="0.2" layer="1"/>
 <via x="45" y="49" extent="1-16" drill="0.4"/>
+<contactref element="IMU" pad="11"/>
+<contactref element="IMU" pad="9"/>
+<wire x1="23.6" y1="19.455" x2="23.6" y2="17.25" width="0.2" layer="1"/>
+<wire x1="22.8" y1="19.455" x2="22.8" y2="18.8" width="0.2" layer="1"/>
+<wire x1="22.8" y1="18.8" x2="22" y2="18" width="0.2" layer="1"/>
+<wire x1="19.25" y1="18" x2="18.4" y2="17.15" width="0.2" layer="1"/>
+<wire x1="18.4" y1="17.15" x2="18" y2="17.15" width="0.2" layer="1"/>
+<wire x1="22" y1="18" x2="19.25" y2="18" width="0.2" layer="1"/>
 <wire x1="4.075" y1="40.075" x2="4.15" y2="40.15" width="0" layer="19" extent="1-1"/>
 <wire x1="12" y1="43.85" x2="6.5" y2="43.85" width="0" layer="19" extent="1-1"/>
@@
 <wire x1="18.25" y1="10.75" x2="19" y2="10" width="0.2" layer="1"/>
 </signal>
-<signal name="IMU_INT">
-<contactref element="U2" pad="12"/>
-<contactref element="IMU" pad="12"/>
-<wire x1="24" y1="19.455" x2="24.455" y2="19" width="0.2" layer="1"/>
-<wire x1="24.455" y1="19" x2="26" y2="19" width="0.2" layer="1"/>
-<via x="26" y="19" extent="1-16" drill="0.4"/>
-<wire x1="27" y1="19" x2="28" y2="20" width="0.2" layer="16"/>
-<wire x1="28" y1="20" x2="28" y2="25.46" width="0.2" layer="16"/>
-<wire x1="28" y1="25.46" x2="23.08" y2="30.38" width="0.2" layer="16"/>
-<wire x1="26" y1="19" x2="27" y2="19" width="0.2" layer="16"/>
-</signal>
-<signal name="IMU_AD0">
-<contactref element="U2" pad="9"/>
-<contactref element="IMU" pad="9"/>
-<wire x1="22.8" y1="19.455" x2="22.8376" y2="19.4174" width="0.2" layer="1"/>
-<wire x1="22.8376" y1="19.4174" x2="22.8376" y2="19.0465625" width="0.2" layer="1"/>
-<wire x1="22.8376" y1="19.0465625" x2="22.8476" y2="19.0365625" width="0.2" layer="1"/>
-<wire x1="22.8476" y1="19.0365625" x2="22.8476" y2="19" width="0.2" layer="1"/>
-<wire x1="22.8476" y1="19" x2="22.1476" y2="18.3" width="0.2" layer="1"/>
-<wire x1="22.1476" y1="18.3" x2="20.6" y2="18.3" width="0.2" layer="1"/>
-<via x="20.6" y="18.3" extent="1-16" drill="0.4"/>
-<wire x1="19" y1="26.84" x2="15.46" y2="30.38" width="0.2" layer="16"/>
-<wire x1="20.6" y1="18.3" x2="19" y2="19.9" width="0.2" layer="16"/>
-<wire x1="19" y1="19.9" x2="19" y2="26.84" width="0.2" layer="16"/>
-</signal>
 <signal name="EXP_PAD">

Commit message: Updated power switch and connector
Parts:
- removed L_ESC, R_ESC: JST_PHD_2X04, Gucci_ControlBoard:JST_PHD_2X04
- added R1: 50, SparkFun-Resistors:0603
- added U$5: POWER_SWITCH, Gucci_ControlBoard:ELUMEESAQ7C12
- added U$6: MOLEX_1.25MM_4PIN_SMT, Gucci_ControlBoard:MOLEX_1.25MM_4PIN_SMT
- moved C7 40.9 mm to (44.0, 34.0), flipped to the bottom, turned to 90 degrees
- moved C5 24.2 mm to (45.5, 43.1), flipped to the bottom, turned to 180 degrees
- moved C21 3.00 mm to (25.0, 42.0)
- moved C22 3.00 mm to (25.8, 39.1)
- moved U7 3.00 mm to (21.0, 39.0)
Connections:
- new net IMU_AD0: IMU.9, U2.9
- new net IMU_INT: IMU.12, U2.12
- new net N$5: R1.1, U$5.P1
- new net N$6: U$5.P4, U$6.P$6
- net 5V: now also U$5.P3, U$5.P5; no longer L_ESC.6, L_ESC.7, R_ESC.2, R_ESC.3
- net GND: now also R1.2, U$6.P$3; no longer IMU.9, L_ESC.5, L_ESC.8, R_ESC.1, R_ESC.4
- net RX0: no longer R_ESC.7
- net RX1: no longer L_ESC.2
- net TX0: no longer R_ESC.5
- net TX1: no longer L_ESC.4
Routing:
- net RX1: track 20.0 -> 0.16 mm
- net GND: track 113.1 -> 94.6 mm
- net TX1: track 17.7 -> 0.00 mm
- net IMU_AD0: track 0.00 -> 17.2 mm, vias 0 -> 1
- net IMU_INT: track 0.00 -> 17.0 mm, vias 0 -> 1
- net TX0: track 14.5 -> 0.00 mm
- net RX0: track 11.1 -> 0.00 mm
- net 5V: track 4.51 -> 0.17 mm
- net 3.3V: track 108.0 -> 106.6 mm

Commit message: Fixed Gucci IMU connections
Parts:
- removed C7: 10uF, SparkFun-Capacitors:0603
- moved C5 19.7 mm to (27.5, 35.1), flipped to the top, turned to 90 degrees
- moved R18 12.2 mm to (3.00, 26.0)
- moved D1 8.00 mm to (-3.00, 26.0), turned to 0 degrees
Connections:
- removed net IMU_AD0: IMU.9, U2.9
- removed net IMU_INT: IMU.12, U2.12
- net 5V: no longer C7.1
- net GND: now also IMU.9; no longer C7.2
Routing:
- net IMU_AD0: track 17.2 -> 0.00 mm, vias 1 -> 0
- net IMU_INT: track 17.0 -> 0.00 mm, vias 1 -> 0
- net N$6: track 0.00 -> 5.39 mm, vias 0 -> 1
- net 5V: track 0.17 -> 3.02 mm
- net N$5: track 0.00 -> 2.72 mm
- net N$1: track 5.69 -> 4.27 mm
- net GND: track 94.6 -> 95.4 mm, vias 10 -> 12

Commit message: Rearranged capacitors/Created 6 Pin SMD Connector Footprint
Parts:
- removed L_MOT, R_MOT: (no value), pinhead:1X02
- removed U3, U4: MAX4173-SOT-23, Gucci_ControlBoard:SOT-23
- moved R1 2.91 mm to (27.8, 42.9)
- moved C5 1.80 mm to (25.7, 35.0)
Connections:
- removed net CURRENT_L: U2.A21, U4.P$6
- removed net CURRENT_R: U2.14/A0, U3.P$6
- removed net L_MOT+: L_MOT.2, U4.P$4
- removed net L_MOT-: L_MOT.1, U4.P$5
- removed net R_MOT+: R_MOT.2, U3.P$4
- removed net R_MOT-: R_MOT.1, U3.P$5
- net 3.3V: no longer U3.P$3, U4.P$3
- net GND: no longer U3.P$1, U3.P$2, U4.P$1, U4.P$2
Routing:
- net 3.3V: track 106.6 -> 92.2 mm, vias 2 -> 0
- net L_MOT-: track 7.33 -> 0.00 mm
- net R_MOT+: track 7.31 -> 0.00 mm
- net GND: track 95.4 -> 89.0 mm, vias 12 -> 14
- net CURRENT_L: track 6.41 -> 0.00 mm
- net CURRENT_R: track 6.21 -> 0.00 mm
- net L_MOT+: track 4.12 -> 0.00 mm
- net R_MOT-: track 4.10 -> 0.00 mm
Other:
- board text removed: "+"
- board text removed: "-"

Commit message: Moved LEDs and NeoPixel to bottom
Parts:
- moved D2 33.2 mm to (11.0, 28.0), flipped to the bottom, turned to 180 degrees
- moved LED1 31.6 mm to (30.0, 26.0), flipped to the bottom, turned to 180 degrees
- moved R19 30.1 mm to (15.0, 28.0), flipped to the bottom, turned to 180 degrees
- moved D3 14.3 mm to (20.0, 28.0), flipped to the bottom, turned to 180 degrees
- moved R20 14.3 mm to (24.0, 28.0), flipped to the bottom, turned to 180 degrees
- moved D1 5.33 mm to (1.90, 28.1), flipped to the bottom, turned to 180 degrees
- moved R18 3.11 mm to (5.30, 28.1), flipped to the bottom, turned to 180 degrees
Routing:
- net GND: track 89.0 -> 80.7 mm, vias 14 -> 11
- net NEO_DI: track 16.3 -> 21.4 mm, vias 0 -> 1
- net 3.3V: track 92.2 -> 96.4 mm, vias 0 -> 1
- net 5V: track 2.99 -> 7.07 mm, vias 0 -> 2
- net 1.8V: track 11.7 -> 15.6 mm, vias 0 -> 1
- net N$1: track 4.27 -> 1.67 mm
- net NEO_DO: track 22.0 -> 22.9 mm, vias 0 -> 1

Commit message: Moved NeoPixel to the center
Parts:
- moved LED1 11.4 mm to (19.0, 23.0)
- moved D1 0.10 mm to (1.90, 28.0)
- moved R18 0.10 mm to (5.30, 28.0)
Connections:
- net NEO_DI: now also U2.11; no longer U2.38/A19
Routing:
- net NEO_DO: track 22.9 -> 0.00 mm, vias 1 -> 0
- net NEO_DI: track 21.4 -> 8.06 mm, vias 1 -> 0
- net 5V: track 7.07 -> 7.73 mm
Changed lines of the file:
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@@
 <attribute name="NAME" x="-8.025" y="32.985" size="1.6764" layer="25" rot="R180"/>
 </element>
-<element name="R18" library="SparkFun-Resistors" package="0603" value="1.65k" x="5.3" y="28.1" smashed="yes" rot="MR180">
-<attribute name="NAME" x="5.3" y="27.338" size="1.016" layer="26" font="vector" ratio="20" rot="MR180" align="bottom-center"/>
-<attribute name="PROD_ID" value="RES-07856" x="5.3" y="28.1" size="1.778" layer="28" rot="MR180" display="off"/>
-<attribute name="VALUE" x="5.3" y="28.862" size="0.8128" layer="28" font="vector" ratio="20" rot="MR180" align="top-center"/>
+<element name="R18" library="SparkFun-Resistors" package="0603" value="1.65k" x="5.3" y="28" smashed="yes" rot="MR180">
+<attribute name="NAME" x="5.3" y="27.238" size="1.016" layer="26" font="vector" ratio="20" rot="MR180" align="bottom-center"/>
+<attribute name="PROD_ID" value="RES-07856" x="5.3" y="28" size="1.778" layer="28" rot="MR180" display="off"/>
+<attribute name="VALUE" x="5.3" y="28.762" size="0.8128" layer="28" font="vector" ratio="20" rot="MR180" align="top-center"/>
 </element>
 <element name="R19" library="SparkFun-Resistors" package="0603" value="800" x="15" y="28" smashed="yes" rot="MR180">
-<attribute name="NAME" x="15" y="25.762" size="1.016" layer="26" font="vector" ratio="20" rot="MR0" align="bottom-center"/>
+<attribute name="NAME" x="15" y="26.062" size="1.016" layer="26" font="vector" ratio="20" rot="MR0" align="bottom-center"/>
 <attribute name="PROD_ID" value="RES-07856" x="15" y="28" size="1.778" layer="28" rot="MR180" display="off"/>
 <attribute name="VALUE" x="15.238" y="30" size="0.8128" layer="28" font="vector" ratio="20" rot="MR90" align="top-center"/>
 </element>
-<element name="D1" library="SparkFun-LED" package="LED-0603" value="5V" x="1.9" y="28.1" smashed="yes" rot="MR180">
-<attribute name="NAME" x="1.9" y="27.465" size="1.016" layer="26" font="vector" ratio="20" rot="MR180" align="bottom-center"/>
-<attribute name="VALUE" x="0.3" y="28.035" size="1.016" layer="22" font="vector" ratio="20" rot="MR90" align="top-center"/>
+<element name="D1" library="SparkFun-LED" package="LED-0603" value="5V" x="1.9" y="28" smashed="yes" rot="MR180">
+<attribute name="NAME" x="1.9" y="27.365" size="0.8128" layer="26" font="vector" ratio="20" rot="MR180" align="bottom-center"/>
+<attribute name="VALUE" x="0.4" y="28.2" size="0.8128" layer="22" font="vector" ratio="20" rot="MR90" align="top-center"/>
 </element>
 <element name="D2" library="SparkFun-LED" package="LED-0603" value="3.3V" x="11" y="28" smashed="yes" rot="MR180">
-<attribute name="NAME" x="11.7" y="26.365" size="1.016" layer="26" font="vector" ratio="20" rot="MR0" align="bottom-center"/>
-<attribute name="VALUE" x="8.5" y="27.435" size="1.016" layer="22" font="vector" ratio="20" rot="MR270" align="top-center"/>
+<attribute name="NAME" x="11.1" y="26.565" size="0.8128" layer="26" font="vector" ratio="20" rot="MR0" align="bottom-center"/>
+<attribute name="VALUE" x="8.6" y="27.635" size="0.8128" layer="22" font="vector" ratio="20" rot="MR270" align="top-center"/>
 </element>
 <element name="C15" library="SparkFun-Capacitors" library_urn="urn:adsk.eagle:library:510" package="0603" package3d_urn="urn:adsk.eagle:package:37414/1" value="0.1uF" x="-11" y="27" smashed="yes">
@@
 <element name="D3" library="SparkFun-LED" package="LED-0603" value="1.8V" x="20" y="28" smashed="yes" rot="MR180">
 <attribute name="NAME" x="20" y="27.265" size="0.8128" layer="26" font="vector" ratio="20" rot="MR180" align="bottom-center"/>
-<attribute name="VALUE" x="18.4" y="27.735" size="0.8128" layer="22" font="vector" ratio="20" rot="MR90" align="top-center"/>
+<attribute name="VALUE" x="18.4" y="27.635" size="0.8128" layer="22" font="vector" ratio="20" rot="MR90" align="top-center"/>
 </element>
 <element name="R20" library="SparkFun-Resistors" package="0603" value="50" x="24" y="28" smashed="yes" rot="MR180">
@@
 </element>
 <element name="U$4" library="RoboJackets-Aesthetics" package="ROBOBUZZ_0.4X" value="" x="-6" y="15" smashed="yes"/>
-<element name="LED1" library="adafruit" library_urn="urn:adsk.eagle:library:420" package="WS2812B" package3d_urn="urn:adsk.eagle:package:6240942/1" value="WS2812B5050" x="30" y="26" smashed="yes" rot="MR180">
-<attribute name="NAME" x="31.3925" y="22.6125" size="1.016" layer="26" ratio="10" rot="MR180"/>
+<element name="LED1" library="adafruit" library_urn="urn:adsk.eagle:library:420" package="WS2812B" package3d_urn="urn:adsk.eagle:package:6240942/1" value="WS2812B5050" x="19" y="23" smashed="yes" rot="MR180">
+<attribute name="NAME" x="20.3925" y="19.6125" size="1.016" layer="26" ratio="10" rot="MR180"/>
 </element>
 <element name="U$5" library="Gucci_ControlBoard" package="ELUMEESAQ7C12" value="POWER_SWITCH" x="40" y="38" smashed="yes" rot="R180">
@@
 <contactref element="U$5" pad="P3"/>
 <contactref element="U$5" pad="P5"/>
-<wire x1="1.023" y1="28.1" x2="-0.3" y2="26.777" width="0.2" layer="16"/>
+<wire x1="1.023" y1="28" x2="-0.3" y2="26.777" width="0.2" layer="16"/>
 <wire x1="-0.3" y1="26.777" x2="-0.3" y2="26.6" width="0.2" layer="16"/>
 <via x="-0.3" y="26.6" extent="1-16" drill="0.4"/>
 <wire x1="-0.3" y1="26.6" x2="-0.3" y2="28.4" width="0.2" layer="1"/>
-<wire x1="32.45" y1="27.65" x2="33.35" y2="27.65" width="0.2" layer="16"/>
-<wire x1="33.35" y1="27.65" x2="34" y2="27" width="0.2" layer="16"/>
-<via x="34" y="27" extent="1-16" drill="0.4"/>
-<wire x1="34" y1="27" x2="34" y2="28.4" width="0.2" layer="1"/>
+<wire x1="21.45" y1="24.65" x2="21.56358125" y2="24.76358125" width="0.2" layer="16"/>
+<wire x1="21.56358125" y1="24.76358125" x2="21.56358125" y2="26.73641875" width="0.2" layer="16"/>
+<via x="21.56358125" y="26.73641875" extent="1-16" drill="0.4"/>
+<wire x1="21.56358125" y1="26.73641875" x2="21.7" y2="26.8728375" width="0.2" layer="1"/>
+<wire x1="21.7" y1="26.8728375" x2="21.7" y2="28.5" width="0.2" layer="1"/>
 </signal>
 <signal name="3.3V">
@@
 <contactref element="D1" pad="C"/>
 <contactref element="R18" pad="1"/>
-<wire x1="2.777" y1="28.1" x2="4.45" y2="28.1" width="0.2" layer="16"/>
+<wire x1="2.777" y1="28" x2="4.45" y2="28" width="0.2" layer="16"/>
 </signal>
 <signal name="N$2">
@@
 </signal>
 <signal name="NEO_DI">
-<contactref element="U2" pad="38/A19"/>
 <contactref element="LED1" pad="4-DIN"/>
-<wire x1="27.55" y1="27.65" x2="29.6" y2="29.7" width="0.2" layer="16"/>
-<via x="35" y="41" extent="1-16" drill="0.4"/>
-<wire x1="35" y1="41" x2="35" y2="44.84" width="0.2" layer="1"/>
-<wire x1="35" y1="44.84" x2="35.78" y2="45.62" width="0.2" layer="1"/>
-<wire x1="29.6" y1="35.6" x2="35" y2="41" width="0.2" layer="16"/>
-<wire x1="29.6" y1="29.7" x2="29.6" y2="35.6" width="0.2" layer="16"/>
+<contactref element="U2" pad="11"/>
+<wire x1="16.55" y1="24.65" x2="17" y2="25.1" width="0.2" layer="16"/>
+<wire x1="17" y1="25.1" x2="17" y2="28" width="0.2" layer="16"/>
+<wire x1="17" y1="28" x2="18.391" y2="29.391" width="0.2" layer="16"/>
+<wire x1="18.391" y1="29.391" x2="18.4096625" y2="29.391" width="0.2" layer="16"/>
+<wire x1="19.3986625" y1="30.38" x2="20.54" y2="30.38" width="0.2" layer="16"/>
+<wire x1="18.4096625" y1="29.391" x2="19.3986625" y2="30.38" width="0.2" layer="16"/>
 </signal>
 <signal name="NEO_DO">
 <contactref element="U2" pad="39/A20"/>
 <contactref element="LED1" pad="2-DOUT"/>
-<via x="34" y="39" extent="1-16" drill="0.4"/>
-<wire x1="34" y1="39" x2="34.791" y2="38.209" width="0.2" layer="16"/>
-<wire x1="34.791" y1="38.209" x2="34.791" y2="26.691" width="0.2" layer="16"/>
-<wire x1="34" y1="39" x2="34" y2="44.86" width="0.2" layer="1"/>
-<wire x1="34" y1="44.86" x2="33.24" y2="45.62" width="0.2" layer="1"/>
-<wire x1="34.791" y1="26.691" x2="32.45" y2="24.35" width="0.2" layer="16"/>
+<wire x1="21.45" y1="21.35" x2="33.24" y2="45.62" width="0" layer="19" extent="16-16"/>
 </signal>
 <signal name="N$5">

Commit message: Removed NeoPixel DO Connector
Connections:
- net NEO_DO: no longer LED1.2-DOUT
Changed lines of the file:
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@@
 <drawing>
 <settings>
-<setting alwaysvectorfont="yes"/>
+<setting alwaysvectorfont="no"/>
 <setting verticaltext="up"/>
 </settings>
@@
 <signal name="NEO_DO">
 <contactref element="U2" pad="39/A20"/>
-<contactref element="LED1" pad="2-DOUT"/>
-<wire x1="21.45" y1="21.35" x2="33.24" y2="45.62" width="0" layer="19" extent="16-16"/>
 </signal>
 <signal name="N$5">

Commit message: Style Guide Adjustments
Parts:
- moved R18 6.70 mm to (12.0, 28.0)
- moved D1 6.10 mm to (8.00, 28.0)
- moved D2 6.00 mm to (17.0, 28.0)
- moved D3 6.00 mm to (26.0, 28.0)
- moved R19 6.00 mm to (21.0, 28.0)
- moved R20 6.00 mm to (30.0, 28.0)
- moved U$4 5.66 mm to (-2.00, 19.0)
- moved U$3 5.00 mm to (40.0, 19.0)
- renumbered U$5 to POWER, U$6 to ESC
Routing:
- net 3.3V: track 96.4 -> 94.3 mm
- net LINE_LF: track 81.2 -> 80.1 mm
- net 5V: track 7.73 -> 8.53 mm
- net N$1: track 1.67 -> 2.27 mm
