File: Gucci/v2 pcb/Gucci_ControlBoard.sch (EAGLE design)
At the start: 61 parts, among them J1 JST_PH_1X05_90, J10 JST_PH_1X03, J11 JST_PHD_2X04, J12 JST_PHD_2X04, J15 JST_PH_1X03_90, J2 JST_PH_1X05_90, J3 JST_PH_1X05_90, J4 JST_PH_1X05_90, J5 JST_PH_1X05_90, J6 JST_PH_1X05_90, J7 JST_PH_1X03_90, J8 JST_PH_1X03_90, J9 JST_PH_1X03, U1 TEENSY_3.6_DIL, U2 AP2114H-3.3TRG1, U3 AP2114H-1.8TRG1, U4 ICM-20948, U5 LM339-14-SOIC

Commit message: level shifter
added level shifter to gucci and kirbi. the part is in gucci's library. the relevant area on the boards should be very similar, but not identical
Parts:
- added R21: 200k, SparkFun-Resistors:1KOHM-0603-1/10W-1%
- added R22, R23: 10k, SparkFun-Resistors:1KOHM-0603-1/10W-1%
- added U6: PCA9306_LSSOP, Gucci_ControlBoard:PCA9306_LSSOP
Connections:
- new net N$7: R21.1, U6.EN, U6.VREF2
- new net SCL2: R16.1, U1.3/CAN0-TX/SCL2/PWM, U6.SCL2
- new net SDA2: R15.1, U1.4/CAN0-RX/SDA2/PWM, U6.SDA2
- net 1.8V: now also R22.2, R23.2, U6.VREF1; no longer R15.2, R16.2
- net 3V3: now also R15.2, R16.2, R21.2
- net GND: now also U6.GND
- net SCL1: now also R23.1, U6.SCL1; no longer R16.1, U1.3/CAN0-TX/SCL2/PWM
- net SDA1: now also R22.1, U6.SDA1; no longer R15.1, U1.4/CAN0-RX/SDA2/PWM
Other:
- moved on the sheet: C16, C17, C18, J13, J14, R1, R10, R11, R12, R15, R2, R3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

Commit message: idc connectors
gucci should be done now
Parts:
- removed C7: 0.1uF, SparkFun-Capacitors:0.1UF-0603-25V-(+80/-20%)
- removed J1, J2, J3, J4, J5, J6: JST_PH_1X05_90, Gucci_ControlBoard:JST_PH_1X05_90
- removed J10, J9: JST_PH_1X03, Gucci_ControlBoard:JST_PH_1X03
- removed J11, J12: JST_PHD_2X04, Gucci_ControlBoard:JST_PHD_2X04
- removed J15, J7, J8: JST_PH_1X03_90, Gucci_ControlBoard:JST_PH_1X03_90
- removed R20: 1k, SparkFun-Resistors:1KOHM-0603-1/10W-1%
- removed U6: PCA9306_LSSOP, Gucci_ControlBoard:PCA9306_LSSOP
- added D3: 1.8V, SparkFun-LED:LED0603
- added IMU: ICM-20948, ICM-20948:ICM-20948
- added LINE_LF, LINE_RF, START: AMPHENOL_2X02_2.54MM_SHROUD, Gucci_ControlBoard:AMPHENOL_2X02_2.54MM_SHROUD
- added L_ESC, R_ESC: JST_PHD_2X04, Gucci_ControlBoard:JST_PHD_2X04
- added TOF2, TOF3, TOF4, TOF5, TOF_0, TOF_1: AMPHENOL_2X03_2.54MM_SHROUD, Gucci_ControlBoard:AMPHENOL_2X03_2.54MM_SHROUD
- D1: value Green -> 5V
- D2: value Green -> 3.3V
- R13: value 330 -> 1650
- R14: value 220 -> 800
- R19: value 1k -> 50
- U4: value ICM-20948 -> LM339-14-SOIC; device ICM-20948:ICM-20948 -> Gucci_ControlBoard:LM339-14-SOIC
- U5: value LM339-14-SOIC -> PCA9306_LSSOP; device Gucci_ControlBoard:LM339-14-SOIC -> Gucci_ControlBoard:PCA9306_LSSOP
- renumbered J13 to R_ENC, J14 to L_ENC
Connections:
- removed net LB_INT: R20.1, U1.17/A3/T/PWM, U5.OUT4
- removed net LINE_LB: J7.2, U1.19/A5/T/SCL0, U5.4IN+
- removed net LINE_RB: J8.2, U1.A21/DAC0, U5.3IN+
- removed net RB_INT: R19.1, U1.18/A4/T/SDA0, U5.OUT3
- new net N$4: D3.C, R19.1
- net 1.8V: now also D3.A, IMU.NCS, IMU.VDD, IMU.VDDIO, U5.VREF1; no longer U4.NCS, U4.VDD, U4.VDDIO, U6.VREF1
- net 3V3: now also LINE_LF.1, LINE_RF.1, START.3, TOF2.6, TOF3.6, TOF4.6, TOF5.6, TOF_0.6, TOF_1.6; no longer C7.1, J1.1, J10.3, J15.2, J2.1, J3.1, J4.1, J5.1, J6.1, J7.3, J8.3, J9.3, R19.2, R20.2
- net 5V: now also L_ESC.6, L_ESC.7, R_ESC.2, R_ESC.3, U4.VCC; no longer J11.2, J11.3, J12.6, J12.7, U5.VCC
- net ENCODER1_A: now also R_ESC.6; no longer J11.6
- net ENCODER1_B: now also R_ESC.8; no longer J11.8
- net ENCODER2_A: now also L_ESC.3; no longer J12.3
- net ENCODER2_B: now also L_ESC.1; no longer J12.1
- net GND: now also IMU.FSYNC, IMU.GND, IMU.RESV_20, LINE_LF.3, LINE_RF.3, L_ESC.5, L_ESC.8, R19.2, R_ESC.1, R_ESC.4, START.2, TOF2.5, TOF3.5, TOF4.5, TOF5.5, TOF_0.5, TOF_1.5; no longer C7.2, J1.2, J10.1, J11.1, J11.4, J12.5, J12.8, J15.1, J2.2, J3.2, J4.2, J5.2, J6.2, J7.1, J8.1, J9.1, U4.FSYNC, U4.RESV_20, U6.GND
- net IMU_AD0: now also IMU.AD0/SDO; no longer U4.AD0/SDO
- net IMU_INT: now also IMU.INT1; no longer U4.INT1
- net LF_INT: now also R17.1, U1.10/TX2/PWM, U4.1OUT; no longer R18.1, U1.11/MOSI0, U5.2OUT
- net LINE_LF: now also LINE_LF.2, U1.35/A16/PWM, U4.1IN+; no longer J9.2, U1.23/A9/T/PWM, U5.2IN+
- net LINE_REF: now also U4.1IN-, U4.2IN-; no longer U5.1IN-, U5.2IN-, U5.3IN-, U5.4IN-
- net LINE_RF: now also LINE_RF.2, U1.23/A9/T/PWM, U4.2IN+; no longer J10.2, U1.35/A16/PWM, U5.1IN+
- net N$3: now also IMU.REGOUT; no longer U4.REGOUT
- net N$7: now also U5.EN, U5.VREF2; no longer U6.EN, U6.VREF2
- net RF_INT: now also R18.1, U1.11/MOSI0, U4.2OUT; no longer R17.1, U1.10/TX2/PWM, U5.1OUT
- net RX0: now also R_ESC.7; no longer J11.7
- net RX1: now also L_ESC.2; no longer J12.2
- net SCL0: now also TOF2.2, TOF3.2, TOF4.2, TOF5.2, TOF_0.2, TOF_1.2; no longer J1.4, J2.4, J3.4, J4.4, J5.4, J6.4
- net SCL1: now also IMU.SCL/SCLK, U5.SCL1; no longer U4.SCL/SCLK, U6.SCL1
- net SCL2: now also U5.SCL2; no longer U6.SCL2
- net SDA0: now also TOF2.1, TOF3.1, TOF4.1, TOF5.1, TOF_0.1, TOF_1.1; no longer J1.5, J2.5, J3.5, J4.5, J5.5, J6.5
- net SDA1: now also IMU.SDA/SDI, U5.SDA1; no longer U4.SDA/SDI, U6.SDA1
- net SDA2: now also U5.SDA2; no longer U6.SDA2
- net SHDN0: now also TOF_0.3; no longer J1.3
- net SHDN1: now also TOF_1.3; no longer J2.3
- net SHDN2: now also TOF2.3; no longer J3.3
- net SHDN3: now also TOF3.3; no longer J4.3
- net SHDN4: now also TOF4.3; no longer J5.3
- net SHDN5: now also TOF5.3; no longer J6.3
- net START: now also START.1; no longer J15.3
- net TX0: now also R_ESC.5; no longer J11.5
- net TX1: now also L_ESC.4; no longer J12.4
Other:
- moved on the sheet: D1, D2, R13, R14, R19

Commit message: finished v2 pcb and updated library
Parts:
- removed R23: 10k, SparkFun-Resistors:1KOHM-0603-1/10W-1%
- removed TOF4: AMPHENOL_2X03_2.54MM_SHROUD, Gucci_ControlBoard:AMPHENOL_2X03_2.54MM_SHROUD
- added C20: 4.7uF, SparkFun-Capacitors:0.1UF-0603-25V-(+80/-20%)
- added C7: 0.1uF, SparkFun-Capacitors:0.1UF-0603-25V-(+80/-20%)
- added L_MOT, R_MOT: (no value), pinhead:PINHD-1X2
- added R20: 200k, SparkFun-Resistors:1KOHM-0603-1/10W-1%
- added TOF_6: AMPHENOL_2X03_2.54MM_SHROUD, Gucci_ControlBoard:AMPHENOL_2X03_2.54MM_SHROUD
- added U6: MAX4173-SOT-23, Gucci_ControlBoard:MAX4173-SOT-23
- added U7: LM393-8-SOIC, Gucci_ControlBoard:LM393-8-SOIC
- C1, C2: value 0.1uF -> 15pF
- C10, C9: value 1uF -> 0.1uF
- C12, C13: value 4.7uF -> 1uF
- C14, C15: value 4.7uF -> 0.1uF
- C17, C18, C19: value 0.1uF -> 4.7uF
- D1: value 5V -> 1.8V
- D3: value 1.8V -> 5V
- R10, R4, R8: value 3k -> 2k
- R11, R3, R7: value 2k -> 3k
- R12: value 3k -> 10k
- R13: value 1650 -> 10k
- R14: value 800 -> 1k
- R15: value 10k -> 3k
- R16: value 10k -> 800
- R17: value 1k -> 1.65k
- R18: value 1k -> 10k
- R19: value 50 -> 10k
- R21: value 200k -> 50
- R22: value 10k -> 1k
- U2: value AP2114H-3.3TRG1 -> PCA9306_LSSOP; device Gucci_ControlBoard:AP2114H-3.3TRG1 -> Gucci_ControlBoard:PCA9306_LSSOP
- U3: value AP2114H-1.8TRG1 -> AP2114H-3.3TRG1; device Gucci_ControlBoard:AP2114H-1.8TRG1 -> Gucci_ControlBoard:AP2114H-3.3TRG1
- U4: value LM339-14-SOIC -> AP2114H-1.8TRG1; device Gucci_ControlBoard:LM339-14-SOIC -> Gucci_ControlBoard:AP2114H-1.8TRG1
- U5: value PCA9306_LSSOP -> MAX4173-SOT-23; device Gucci_ControlBoard:PCA9306_LSSOP -> Gucci_ControlBoard:MAX4173-SOT-23
- renumbered TOF2 to TOF_3, TOF3 to TOF_4, TOF5 to TOF_2, TOF_0 to TOF_5
Connections:
- new net CURRENT_L: U1.A21/DAC0, U5.OUT
- new net CURRENT_R: U1.13/SCK0/LED, U6.OUT
- new net L_MOT+: L_MOT.2, U5.RS+
- new net L_MOT-: L_MOT.1, U5.RS-
- new net R_MOT+: R_MOT.2, U6.RS+
- new net R_MOT-: R_MOT.1, U6.RS-
- net 1.8V: now also C20.1, C3.1, C4.1, D1.A, R18.2, R19.2, U2.VREF1, U4.EPAD, U4.VOUT; no longer C15.1, C17.1, C18.1, D3.A, R22.2, R23.2, U3.EPAD, U3.VOUT, U5.VREF1
- net 3V3: now also C10.1, C11.1, C18.1, C19.1, C7.1, C9.1, R12.2, R13.2, R14.2, R20.2, R22.2, TOF_6.6, U3.EPAD, U3.VOUT, U4.VIN; no longer C1.1, C13.1, C14.1, C2.1, C3.1, C4.1, R15.2, R16.2, R17.2, R18.2, R21.2, TOF4.6, U2.EPAD, U2.VOUT, U3.VIN
- net 3V_ENCODER1_A: now also R6.2, R8.2; no longer R1.2, R2.2
- net 3V_ENCODER1_B: now also R7.2; no longer R6.2
- net 3V_ENCODER1_I: now also R15.2; no longer R9.2
- net 3V_ENCODER2_A: now also R2.2; no longer R3.2
- net 3V_ENCODER2_B: now also R1.2, R3.2; no longer R7.2, R8.2
- net 3V_ENCODER2_I: now also R9.2; no longer R12.2
- net 5V: now also C13.1, C14.1, C16.1, C17.1, D3.A, U3.VIN, U5.VCC, U6.VCC, U7.VCC; no longer C10.1, C11.1, C19.1, C9.1, D1.A, U2.VIN, U4.VCC
- net ENCODER1_A: now also R8.1; no longer R1.1
- net ENCODER2_A: now also R4.1; no longer R3.1
- net ENCODER2_B: now also R1.1; no longer R7.1
- net GND: now also C20.2, C7.2, R11.1, R15.1, R16.2, R17.2, R21.2, R3.1, R7.1, TOF_6.5, U6.GND, U7.GND; no longer R10.1, R12.1, R13.2, R14.2, R19.2, R4.1, R8.1, TOF4.5
- net LF_INT: now also C2.1, R22.1, U1.18/A4/T/SDA0, U7.OUT2; no longer R17.1, U1.10/TX2/PWM, U4.1OUT
- net LINE_LF: now also U7.IN2+; no longer U4.1IN+
- net LINE_REF: now also U7.IN1-, U7.IN2-; no longer U4.1IN-, U4.2IN-
- net LINE_RF: now also U7.IN1+; no longer U4.2IN+
- net N$1: now also D3.C, R17.1; no longer D1.C, R13.1
- net N$2: now also R16.1; no longer R14.1
- net N$3: now also C15.1; no longer C16.1
- net N$4: now also D1.C, R21.1; no longer D3.C, R19.1
- net N$5: now also R10.1; no longer R9.1
- net N$7: now also R20.1, U2.EN, U2.VREF2; no longer R21.1, U5.EN, U5.VREF2
- net N$8: now also R9.1; no longer R11.1
- net RF_INT: now also C1.1, R14.1, U1.19/A5/T/SCL0, U7.OUT1; no longer R18.1, U1.11/MOSI0, U4.2OUT
- net SCL0: now also TOF_6.2; no longer TOF4.2
- net SCL1: now also R19.1, U2.SCL1; no longer R23.1, U5.SCL1
- net SCL2: now also R13.1, U2.SCL2; no longer R16.1, U5.SCL2
- net SDA0: now also TOF_6.1; no longer TOF4.1
- net SDA1: now also R18.1, U2.SDA1; no longer R22.1, U5.SDA1
- net SDA2: now also R12.1, U2.SDA2; no longer R15.1, U5.SDA2
- net SHDN1: now also TOF_6.3; no longer TOF_1.3
- net SHDN4: now also TOF_1.3; no longer TOF4.3
- net START: now also U1.17/A3/T/PWM; no longer U1.16/A2/T/PWM
Other:
- note added: "Current Sensing"
- moved on the sheet: C1, C10, C11, C12, C13, C14, C15, C16, C17, C18, C19, C2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

Commit message: silkscreen tweaks
Parts:
- C1, C2: value 15pF -> 0.1uF
- C12, C13: value 1uF -> 0.1uF
- C15, C16: value 0.1uF -> 15pF
- C5, C7: value 0.1uF -> 1uF
- D1: value 1.8V -> 5V
- D3: value 5V -> 1.8V
- R10, R4, R8: value 2k -> 3k
- R11, R3, R7: value 3k -> 2k
- R12: value 10k -> 3k
- R13: value 10k -> 200k
- R14: value 1k -> 10k
- R15: value 3k -> 10k
- R16: value 800 -> 10k
- R17: value 1.65k -> 10k
- R18: value 10k -> 1.65k
- R19: value 10k -> 800
- R20: value 200k -> 50
- R21: value 50 -> 1k
- U1: value TEENSY_3.6_DIL -> PCA9306_LSSOP; device Teensy_3_and_LC_Series_Boards_v1.4:TEENSY_3.6_DIL -> Gucci_ControlBoard:PCA9306_LSSOP
- U2: value PCA9306_LSSOP -> TEENSY_3.6_DIL; device Gucci_ControlBoard:PCA9306_LSSOP -> Teensy_3_and_LC_Series_Boards_v1.4:TEENSY_3.6_DIL
- U3: value AP2114H-3.3TRG1 -> MAX4173-SOT-23; device Gucci_ControlBoard:AP2114H-3.3TRG1 -> Gucci_ControlBoard:MAX4173-SOT-23
- U4: value AP2114H-1.8TRG1 -> MAX4173-SOT-23; device Gucci_ControlBoard:AP2114H-1.8TRG1 -> Gucci_ControlBoard:MAX4173-SOT-23
- U5: value MAX4173-SOT-23 -> LM393-8-SOIC; device Gucci_ControlBoard:MAX4173-SOT-23 -> Gucci_ControlBoard:LM393-8-SOIC
- U6: value MAX4173-SOT-23 -> AP2114H-1.8TRG1; device Gucci_ControlBoard:MAX4173-SOT-23 -> Gucci_ControlBoard:AP2114H-1.8TRG1
- U7: value LM393-8-SOIC -> AP2114H-3.3TRG1; device Gucci_ControlBoard:LM393-8-SOIC -> Gucci_ControlBoard:AP2114H-3.3TRG1
Connections:
- net 1.8V: now also C1.1, C17.1, C2.1, D3.A, R14.2, R15.2, U1.VREF1, U6.EPAD, U6.VOUT; no longer C20.1, C3.1, C4.1, D1.A, R18.2, R19.2, U2.VREF1, U4.EPAD, U4.VOUT
- net 3V3: now also C12.1, C13.1, C14.1, R16.2, R17.2, R21.2, U6.VIN, U7.EPAD, U7.VOUT; no longer C5.1, C6.1, C7.1, R12.2, R14.2, R20.2, U3.EPAD, U3.VOUT, U4.VIN
- net 3V_ENCODER1_A: now also R5.2, U2.22/A8/T/PWM; no longer R8.2, U1.22/A8/T/PWM
- net 3V_ENCODER1_B: now also R3.2, R4.2, U2.21/A7/PWM; no longer R5.2, R7.2, U1.21/A7/PWM
- net 3V_ENCODER1_I: now also R1.2, R2.2, U2.20/A6/PWM; no longer R10.2, R15.2, U1.20/A6/PWM
- net 3V_ENCODER2_A: now also R11.2, R12.2, U2.38/A19/SDA1/PWM; no longer R2.2, R4.2, U1.38/A19/SDA1/PWM
- net 3V_ENCODER2_B: now also R10.2, R9.2, U2.37/A18/SCL1/PWM; no longer R1.2, R3.2, U1.37/A18/SCL1/PWM
- net 3V_ENCODER2_I: now also R7.2, R8.2, U2.36/A17/PWM; no longer R11.2, R9.2, U1.36/A17/PWM
- net 5V: now also C20.1, C4.1, C5.1, C6.1, C7.1, D1.A, U2.VIN, U3.VCC, U4.VCC, U7.VIN; no longer C12.1, C13.1, C14.1, C16.1, C17.1, D3.A, U1.VIN, U3.VIN, U6.VCC, U7.VCC
- net CURRENT_L: now also U2.A21/DAC0, U4.OUT; no longer U1.A21/DAC0, U5.OUT
- net CURRENT_R: now also U2.13/SCK0/LED, U3.OUT; no longer U1.13/SCK0/LED, U6.OUT
- net ENCODER1_A: now also R5.1; no longer R8.1
- net ENCODER1_B: now also R3.1; no longer R5.1
- net ENCODER2_A: now also R11.1; no longer R4.1
- net ENCODER2_B: now also R9.1; no longer R1.1
- net GND: now also R10.1, R12.1, R18.2, R19.2, R20.2, R4.1, R8.1, U2.AGND; no longer R11.1, R15.1, R16.2, R17.2, R21.2, R3.1, R7.1, U1.AGND
- net IMU_AD0: now also U2.9/RX2/PWM; no longer U1.9/RX2/PWM
- net IMU_INT: now also U2.12/MISO0; no longer U1.12/MISO0
- net LF_INT: now also C15.1, R21.1, U2.18/A4/T/SDA0, U5.OUT2; no longer C2.1, R22.1, U1.18/A4/T/SDA0, U7.OUT2
- net LINE_LF: now also U2.35/A16/PWM, U5.IN2+; no longer U1.35/A16/PWM, U7.IN2+
- net LINE_REF: now also U2.A22/DAC1, U5.IN1-, U5.IN2-; no longer U1.A22/DAC1, U7.IN1-, U7.IN2-
- net LINE_RF: now also U2.23/A9/T/PWM, U5.IN1+; no longer U1.23/A9/T/PWM, U7.IN1+
- net L_MOT+: now also U4.RS+; no longer U5.RS+
- net L_MOT-: now also U4.RS-; no longer U5.RS-
- net N$1: now also D1.C, R18.1; no longer D3.C, R17.1
- net N$2: now also R19.1; no longer R16.1
- net N$3: now also C3.1; no longer C15.1
- net N$4: now also D3.C, R20.1; no longer D1.C, R21.1
- net N$5: now also R1.1; no longer R10.1
- net N$7: now also R13.1, U1.EN, U1.VREF2; no longer R20.1, U2.EN, U2.VREF2
- net N$8: now also R7.1; no longer R9.1
- net RF_INT: now also C16.1, R22.1, U2.19/A5/T/SCL0, U5.OUT1; no longer C1.1, R14.1, U1.19/A5/T/SCL0, U7.OUT1
- net RX0: now also U2.7/RX3/PWM; no longer U1.7/RX3/PWM
- net RX1: now also U2.27; no longer U1.27
- net R_MOT+: now also U3.RS+; no longer U6.RS+
- net R_MOT-: now also U3.RS-; no longer U6.RS-
- net SCL0: now also U2.33/A14/TX5/CAN1-TX; no longer U1.33/A14/TX5/CAN1-TX
- net SCL1: now also R14.1, U1.SCL1; no longer R19.1, U2.SCL1
- net SCL2: now also R16.1, U1.SCL2, U2.3/CAN0-TX/SCL2/PWM; no longer R13.1, U1.3/CAN0-TX/SCL2/PWM, U2.SCL2
- net SDA0: now also U2.34/A15/RX5/CAN1-RX; no longer U1.34/A15/RX5/CAN1-RX
- net SDA1: now also R15.1, U1.SDA1; no longer R18.1, U2.SDA1
- net SDA2: now also R17.1, U1.SDA2, U2.4/CAN0-RX/SDA2/PWM; no longer R12.1, U1.4/CAN0-RX/SDA2/PWM, U2.SDA2
- net SHDN0: now also TOF_3.3, U2.0/RX1/MOSI1/T; no longer TOF_5.3, U1.0/RX1/MOSI1/T
- net SHDN1: now also TOF_1.3, U2.1/TX1/MISO1/T; no longer TOF_6.3, U1.1/TX1/MISO1/T
- net SHDN2: now also TOF_5.3, U2.2/PWM; no longer TOF_3.3, U1.2/PWM
- net SHDN3: now also TOF_2.3, U2.30/T/PWM; no longer TOF_4.3, U1.30/T/PWM
- net SHDN4: now also TOF_6.3, U2.31/A12/RX4; no longer TOF_1.3, U1.31/A12/RX4
- net SHDN5: now also TOF_4.3, U2.32/A13/TX4; no longer TOF_2.3, U1.32/A13/TX4
- net START: now also U2.17/A3/T/PWM; no longer U1.17/A3/T/PWM
- net TX0: now also U2.8/TX3/PWM; no longer U1.8/TX3/PWM
- net TX1: now also U2.26; no longer U1.26
Other:
- moved on the sheet: C1, C10, C11, C12, C13, C14, C15, C16, C17, C18, C19, C2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

Commit message: missed decoup caps and silkscreen changes
Parts:
- added C21, C22: 4.7uF, SparkFun-Capacitors:0.1UF-0603-25V-(+80/-20%)
- C15, C16: value 15pF -> 0.1uF
- C17, C18: value 4.7uF -> 15pF
Connections:
- net 1.8V: now also C19.1; no longer C17.1
- net 3V3: now also C15.1, C16.1, C20.1, C21.1; no longer C18.1, C19.1
- net 5V: now also C22.1; no longer C20.1
- net CURRENT_R: now also U2.14/A0/PWM; no longer U2.13/SCK0/LED
- net GND: now also C21.2, C22.2
- net LF_INT: now also C17.1; no longer C15.1
- net RF_INT: now also C18.1; no longer C16.1
- net SHDN0: now also TOF_1.3; no longer TOF_3.3
- net SHDN1: now also TOF_2.3; no longer TOF_1.3
- net SHDN2: now also TOF_3.3; no longer TOF_5.3
- net SHDN3: now also TOF_4.3; no longer TOF_2.3
- net SHDN4: now also TOF_5.3; no longer TOF_6.3
- net SHDN5: now also TOF_6.3; no longer TOF_4.3
Other:
- moved on the sheet: C10, C11, C12, C13, C14, C15, C16, C17, C18, C19, C20, C8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

Commit message: current sense opamps now powered by 3v3
Parts:
- C5, C7: value 1uF -> 10uF
Connections:
- net 3V3: now also U3.VCC, U4.VCC
- net 5V: no longer U3.VCC, U4.VCC
Changed lines of the file:
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@@
 <part name="C10" library="SparkFun-Capacitors" library_urn="urn:adsk.eagle:library:510" deviceset="0.1UF" device="-0603-25V-(+80/-20%)" package3d_urn="urn:adsk.eagle:package:37414/1" value="0.1uF"/>
 <part name="C9" library="SparkFun-Capacitors" library_urn="urn:adsk.eagle:library:510" deviceset="0.1UF" device="-0603-25V-(+80/-20%)" package3d_urn="urn:adsk.eagle:package:37414/1" value="0.1uF"/>
-<part name="C7" library="SparkFun-Capacitors" library_urn="urn:adsk.eagle:library:510" deviceset="0.1UF" device="-0603-25V-(+80/-20%)" package3d_urn="urn:adsk.eagle:package:37414/1" value="1uF"/>
-<part name="C5" library="SparkFun-Capacitors" library_urn="urn:adsk.eagle:library:510" deviceset="0.1UF" device="-0603-25V-(+80/-20%)" package3d_urn="urn:adsk.eagle:package:37414/1" value="1uF"/>
+<part name="C7" library="SparkFun-Capacitors" library_urn="urn:adsk.eagle:library:510" deviceset="0.1UF" device="-0603-25V-(+80/-20%)" package3d_urn="urn:adsk.eagle:package:37414/1" value="10uF"/>
+<part name="C5" library="SparkFun-Capacitors" library_urn="urn:adsk.eagle:library:510" deviceset="0.1UF" device="-0603-25V-(+80/-20%)" package3d_urn="urn:adsk.eagle:package:37414/1" value="10uF"/>
 <part name="GND26" library="SparkFun-PowerSymbols" library_urn="urn:adsk.eagle:library:530" deviceset="GND" device=""/>
 <part name="SUPPLY8" library="SparkFun-PowerSymbols" library_urn="urn:adsk.eagle:library:530" deviceset="3.3V" device=""/>
@@
 <part name="GND28" library="SparkFun-PowerSymbols" library_urn="urn:adsk.eagle:library:530" deviceset="GND" device=""/>
 <part name="GND29" library="SparkFun-PowerSymbols" library_urn="urn:adsk.eagle:library:530" deviceset="GND" device=""/>
-<part name="SUPPLY30" library="SparkFun-PowerSymbols" deviceset="5V" device=""/>
-<part name="SUPPLY31" library="SparkFun-PowerSymbols" deviceset="5V" device=""/>
 <part name="C8" library="SparkFun-Capacitors" library_urn="urn:adsk.eagle:library:510" deviceset="0.1UF" device="-0603-25V-(+80/-20%)" package3d_urn="urn:adsk.eagle:package:37414/1" value="0.1uF"/>
 <part name="C16" library="SparkFun-Capacitors" library_urn="urn:adsk.eagle:library:510" deviceset="0.1UF" device="-0603-25V-(+80/-20%)" package3d_urn="urn:adsk.eagle:package:37414/1" value="0.1uF"/>
+<part name="SUPPLY30" library="SparkFun-PowerSymbols" library_urn="urn:adsk.eagle:library:530" deviceset="3.3V" device=""/>
+<part name="SUPPLY31" library="SparkFun-PowerSymbols" library_urn="urn:adsk.eagle:library:530" deviceset="3.3V" device=""/>
 </parts>
 <sheets>
@@
 <attribute name="VALUE" x="233.68" y="37.846" size="1.778" layer="96" align="top-center"/>
 </instance>
-<instance part="SUPPLY30" gate="G$1" x="233.68" y="66.04" smashed="yes">
-<attribute name="VALUE" x="233.68" y="68.834" size="1.778" layer="96" align="bottom-center"/>
-</instance>
-<instance part="SUPPLY31" gate="G$1" x="193.04" y="66.04" smashed="yes">
-<attribute name="VALUE" x="193.04" y="68.834" size="1.778" layer="96" align="bottom-center"/>
-</instance>
 <instance part="C8" gate="G$1" x="391.16" y="58.42" smashed="yes">
 <attribute name="NAME" x="392.684" y="61.341" size="1.778" layer="95" font="vector"/>
@@
 <attribute name="NAME" x="331.724" y="61.341" size="1.778" layer="95" font="vector"/>
 <attribute name="VALUE" x="331.724" y="56.261" size="1.778" layer="96" font="vector"/>
+</instance>
+<instance part="SUPPLY30" gate="G$1" x="193.04" y="66.04" smashed="yes">
+<attribute name="VALUE" x="193.04" y="68.834" size="1.778" layer="96" align="bottom-center"/>
+</instance>
+<instance part="SUPPLY31" gate="G$1" x="233.68" y="66.04" smashed="yes">
+<attribute name="VALUE" x="233.68" y="68.834" size="1.778" layer="96" align="bottom-center"/>
 </instance>
 </instances>
@@
 <pinref part="U5" gate="G$1" pin="VCC"/>
 <pinref part="SUPPLY14" gate="G$1" pin="5V"/>
-</segment>
-<segment>
-<pinref part="U3" gate="G$1" pin="VCC"/>
-<pinref part="SUPPLY30" gate="G$1" pin="5V"/>
-</segment>
-<segment>
-<pinref part="U4" gate="G$1" pin="VCC"/>
-<pinref part="SUPPLY31" gate="G$1" pin="5V"/>
 </segment>
 </net>
@@
 <wire x1="175.26" y1="109.22" x2="175.26" y2="106.68" width="0.1524" layer="91"/>
 </segment>
+<segment>
+<pinref part="SUPPLY30" gate="G$1" pin="3.3V"/>
+<pinref part="U4" gate="G$1" pin="VCC"/>
+</segment>
+<segment>
+<pinref part="SUPPLY31" gate="G$1" pin="3.3V"/>
+<pinref part="U3" gate="G$1" pin="VCC"/>
+</segment>
 </net>

Commit message: board changes per core reviews
Connections:
- net 3V3 renamed 3.3V
Changed lines of the file:
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@@
 </segment>
 </net>
-<net name="3V3" class="0">
+<net name="3.3V" class="0">
 <segment>
 <pinref part="D2" gate="G$1" pin="A"/>
@@
 <junction x="375.92" y="66.04"/>
 <pinref part="C9" gate="G$1" pin="1"/>
-<wire x1="383.54" y1="66.04" x2="383.54" y2="63.5" width="0.1524" layer="91"/>
 <junction x="383.54" y="66.04"/>
 <pinref part="SUPPLY8" gate="G$1" pin="3.3V"/>
@@
 <junction x="375.92" y="53.34"/>
 <pinref part="C9" gate="G$1" pin="2"/>
-<wire x1="383.54" y1="53.34" x2="383.54" y2="55.88" width="0.1524" layer="91"/>
 <junction x="383.54" y="53.34"/>
 <pinref part="GND26" gate="1" pin="GND"/>
