File: Gucci/v2 pcb/Gucci_ControlBoard.sch (EAGLE design)
At the start: 58 parts, among them U1 PCA9306_LSSOP, U2 TEENSY_3.6_DIL, U3 MAX4173-SOT-23, U4 MAX4173-SOT-23, U5 LM393-8-SOIC, U6 AP2114H-1.8TRG1, U7 AP2114H-3.3TRG1

Commit message: Implemented NeoPixel Status LED for debugging
Parts:
- removed D4: 5V, SparkFun-LED:LED0603
- removed R1: 1.65k, SparkFun-Resistors:1KOHM-0603-1/10W-1%
- added LED1: WS2812B5050, adafruit:WS2812B5050
Connections:
- removed net N$5: D4.C, R1.1
- new net NEO_DI: LED1.DI, U2.38/A19/SDA1/PWM
- new net NEO_DO: LED1.DO, U2.39/A20
- net 5V: now also LED1.VDD; no longer D4.A
- net GND: now also LED1.GND; no longer R1.2
Other:
- note added: "NeoPixel Status"
- moved on the sheet: L_ESC, R_ESC

Commit message: NeoPixel for Kirbi/Fixed IMU
Added NeoPixel/Deleted IMU Interuppt/Tied IMU Address to Ground
Connections:
- removed net IMU_AD0: IMU.AD0/SDO, U2.9/RX2/PWM
- removed net IMU_INT: IMU.INT1, U2.12/MISO0
- net GND: now also IMU.AD0/SDO
Changed lines of the file:
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@@
 <part name="IMU" library="ICM-20948" deviceset="ICM-20948" device=""/>
 <part name="SUPPLY26" library="SparkFun-PowerSymbols" library_urn="urn:adsk.eagle:library:530" deviceset="1.8V" device=""/>
-<part name="GND27" library="SparkFun-PowerSymbols" library_urn="urn:adsk.eagle:library:530" deviceset="GND" device=""/>
 <part name="C4" library="SparkFun-Capacitors" library_urn="urn:adsk.eagle:library:510" deviceset="0.1UF" device="-0603-25V-(+80/-20%)" package3d_urn="urn:adsk.eagle:package:37414/1" value="0.1uF"/>
 <part name="U1" library="Gucci_ControlBoard" deviceset="PCA9306_LSSOP" device=""/>
@@
 <part name="GND19" library="supply1" library_urn="urn:adsk.eagle:library:371" deviceset="GND" device=""/>
 <part name="SUPPLY19" library="SparkFun-PowerSymbols" deviceset="5V" device=""/>
+<part name="GND18" library="SparkFun-PowerSymbols" library_urn="urn:adsk.eagle:library:530" deviceset="GND" device=""/>
 </parts>
 <sheets>
@@
 <attribute name="VALUE" x="398.78" y="172.974" size="1.778" layer="96" align="bottom-center"/>
 </instance>
-<instance part="GND27" gate="1" x="350.52" y="149.86" smashed="yes">
-<attribute name="VALUE" x="350.52" y="149.606" size="1.778" layer="96" align="top-center"/>
-</instance>
 <instance part="C4" gate="G$1" x="414.02" y="58.42" smashed="yes">
 <attribute name="NAME" x="415.544" y="61.341" size="1.778" layer="95" font="vector"/>
@@
 <instance part="SUPPLY19" gate="G$1" x="299.72" y="233.68" smashed="yes">
 <attribute name="VALUE" x="299.72" y="236.474" size="1.778" layer="96" align="bottom-center"/>
+</instance>
+<instance part="GND18" gate="1" x="340.36" y="139.7" smashed="yes">
+<attribute name="VALUE" x="340.36" y="139.446" size="1.778" layer="96" align="top-center"/>
 </instance>
 </instances>
@@
 </segment>
 <segment>
-<pinref part="IMU" gate="G$1" pin="FSYNC"/>
-<wire x1="355.6" y1="152.4" x2="350.52" y2="152.4" width="0.1524" layer="91"/>
-<pinref part="GND27" gate="1" pin="GND"/>
-</segment>
-<segment>
 <pinref part="TOF_1" gate="G$1" pin="5"/>
 <wire x1="34.29" y1="220.98" x2="27.94" y2="220.98" width="0.1524" layer="91"/>
@@
 <pinref part="GND19" gate="1" pin="GND"/>
 <wire x1="294.64" y1="205.74" x2="294.64" y2="203.2" width="0.1524" layer="91"/>
+</segment>
+<segment>
+<pinref part="IMU" gate="G$1" pin="FSYNC"/>
+<wire x1="355.6" y1="152.4" x2="340.36" y2="152.4" width="0.1524" layer="91"/>
+<pinref part="IMU" gate="G$1" pin="AD0/SDO"/>
+<wire x1="355.6" y1="142.24" x2="340.36" y2="142.24" width="0.1524" layer="91"/>
+<wire x1="340.36" y1="142.24" x2="340.36" y2="152.4" width="0.1524" layer="91"/>
+<pinref part="GND18" gate="1" pin="GND"/>
+<junction x="340.36" y="142.24"/>
 </segment>
 </net>
@@
 </segment>
 </net>
-<net name="IMU_INT" class="0">
-<segment>
-<pinref part="U2" gate="G$1" pin="12/MISO0"/>
-<wire x1="165.1" y1="205.74" x2="160.02" y2="205.74" width="0.1524" layer="91"/>
-<label x="160.02" y="205.74" size="1.778" layer="95" rot="R180" xref="yes"/>
-</segment>
-<segment>
-<pinref part="IMU" gate="G$1" pin="INT1"/>
-<wire x1="396.24" y1="149.86" x2="398.78" y2="149.86" width="0.1524" layer="91"/>
-<label x="398.78" y="149.86" size="1.778" layer="95" xref="yes"/>
-</segment>
-</net>
-<net name="IMU_AD0" class="0">
-<segment>
-<pinref part="U2" gate="G$1" pin="9/RX2/PWM"/>
-<wire x1="165.1" y1="213.36" x2="160.02" y2="213.36" width="0.1524" layer="91"/>
-<label x="160.02" y="213.36" size="1.778" layer="95" rot="R180" xref="yes"/>
-</segment>
-<segment>
-<pinref part="IMU" gate="G$1" pin="AD0/SDO"/>
-<wire x1="355.6" y1="142.24" x2="353.06" y2="142.24" width="0.1524" layer="91"/>
-<label x="353.06" y="142.24" size="1.778" layer="95" rot="R180" xref="yes"/>
-</segment>
-</net>

Commit message: Updated power switch and connector
Parts:
- removed L_ESC, R_ESC: JST_PHD_2X04, Gucci_ControlBoard:JST_PHD_2X04
- added R1: 50, SparkFun-Resistors:1KOHM-0603-1/10W-1%
- added U$5: POWER_SWITCH, Gucci_ControlBoard:POWER_SWITCH
- added U$6: MOLEX_1.25MM_4PIN_SMT, Gucci_ControlBoard:MOLEX_1.25MM_4PIN_SMT
Connections:
- new net IMU_AD0: IMU.AD0/SDO, U2.9/RX2/PWM
- new net IMU_INT: IMU.INT1, U2.12/MISO0
- new net N$5: R1.1, U$5.P1
- new net N$6: U$5.P4, U$6.4
- net 5V: now also U$5.P3, U$5.P5; no longer L_ESC.6, L_ESC.7, R_ESC.2, R_ESC.3
- net GND: now also R1.2, U$6.1; no longer IMU.AD0/SDO, L_ESC.5, L_ESC.8, R_ESC.1, R_ESC.4
- net RX0: no longer R_ESC.7
- net RX1: no longer L_ESC.2
- net TX0: no longer R_ESC.5
- net TX1: no longer L_ESC.4
Other:
- note added: "Power"

Commit message: Fixed Gucci IMU connections
Parts:
- removed C7: 10uF, SparkFun-Capacitors:0.1UF-0603-25V-(+80/-20%)
Connections:
- removed net IMU_AD0: IMU.AD0/SDO, U2.9/RX2/PWM
- removed net IMU_INT: IMU.INT1, U2.12/MISO0
- net 5V: no longer C7.1
- net GND: now also IMU.AD0/SDO; no longer C7.2
Changed lines of the file:
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@@
 <layer number="91" name="Nets" color="2" fill="1" visible="yes" active="yes"/>
 <layer number="92" name="Busses" color="1" fill="1" visible="yes" active="yes"/>
-<layer number="93" name="Pins" color="2" fill="1" visible="no" active="yes"/>
+<layer number="93" name="Pins" color="2" fill="1" visible="yes" active="yes"/>
 <layer number="94" name="Symbols" color="4" fill="1" visible="yes" active="yes"/>
 <layer number="95" name="Names" color="7" fill="1" visible="yes" active="yes"/>
@@
 <part name="C10" library="SparkFun-Capacitors" library_urn="urn:adsk.eagle:library:510" deviceset="0.1UF" device="-0603-25V-(+80/-20%)" package3d_urn="urn:adsk.eagle:package:37414/1" value="0.1uF"/>
 <part name="C9" library="SparkFun-Capacitors" library_urn="urn:adsk.eagle:library:510" deviceset="0.1UF" device="-0603-25V-(+80/-20%)" package3d_urn="urn:adsk.eagle:package:37414/1" value="0.1uF"/>
-<part name="C7" library="SparkFun-Capacitors" library_urn="urn:adsk.eagle:library:510" deviceset="0.1UF" device="-0603-25V-(+80/-20%)" package3d_urn="urn:adsk.eagle:package:37414/1" value="10uF"/>
 <part name="C5" library="SparkFun-Capacitors" library_urn="urn:adsk.eagle:library:510" deviceset="0.1UF" device="-0603-25V-(+80/-20%)" package3d_urn="urn:adsk.eagle:package:37414/1" value="10uF"/>
 <part name="GND26" library="SparkFun-PowerSymbols" library_urn="urn:adsk.eagle:library:530" deviceset="GND" device=""/>
@@
 <attribute name="VALUE" x="385.064" y="56.261" size="1.778" layer="96" font="vector"/>
 </instance>
-<instance part="C7" gate="G$1" x="398.78" y="58.42" smashed="yes">
-<attribute name="NAME" x="400.304" y="61.341" size="1.778" layer="95" font="vector"/>
-<attribute name="VALUE" x="400.304" y="56.261" size="1.778" layer="96" font="vector"/>
-</instance>
 <instance part="C5" gate="G$1" x="406.4" y="58.42" smashed="yes">
 <attribute name="NAME" x="407.924" y="61.341" size="1.778" layer="95" font="vector"/>
@@
 <attribute name="VALUE" x="398.78" y="172.974" size="1.778" layer="96" align="bottom-center"/>
 </instance>
-<instance part="GND27" gate="1" x="350.52" y="149.86" smashed="yes">
-<attribute name="VALUE" x="350.52" y="149.606" size="1.778" layer="96" align="top-center"/>
+<instance part="GND27" gate="1" x="340.868" y="139.446" smashed="yes">
+<attribute name="VALUE" x="340.868" y="139.192" size="1.778" layer="96" align="top-center"/>
 </instance>
 <instance part="C4" gate="G$1" x="414.02" y="58.42" smashed="yes">
@@
 </segment>
 <segment>
-<pinref part="C7" gate="G$1" pin="1"/>
-<wire x1="398.78" y1="63.5" x2="398.78" y2="66.04" width="0.1524" layer="91"/>
-<wire x1="398.78" y1="66.04" x2="406.4" y2="66.04" width="0.1524" layer="91"/>
 <pinref part="C5" gate="G$1" pin="1"/>
 <wire x1="406.4" y1="66.04" x2="406.4" y2="63.5" width="0.1524" layer="91"/>
@@
 <wire x1="383.54" y1="53.34" x2="391.16" y2="53.34" width="0.1524" layer="91"/>
 <junction x="383.54" y="53.34"/>
-<pinref part="C7" gate="G$1" pin="2"/>
-<wire x1="391.16" y1="53.34" x2="398.78" y2="53.34" width="0.1524" layer="91"/>
-<wire x1="398.78" y1="53.34" x2="398.78" y2="55.88" width="0.1524" layer="91"/>
-<wire x1="398.78" y1="53.34" x2="406.4" y2="53.34" width="0.1524" layer="91"/>
-<junction x="398.78" y="53.34"/>
+<wire x1="391.16" y1="53.34" x2="406.4" y2="53.34" width="0.1524" layer="91"/>
 <pinref part="C5" gate="G$1" pin="2"/>
 <wire x1="406.4" y1="53.34" x2="406.4" y2="55.88" width="0.1524" layer="91"/>
@@
 </segment>
 <segment>
-<pinref part="IMU" gate="G$1" pin="FSYNC"/>
-<wire x1="355.6" y1="152.4" x2="350.52" y2="152.4" width="0.1524" layer="91"/>
-<pinref part="GND27" gate="1" pin="GND"/>
-</segment>
-<segment>
 <pinref part="TOF_1" gate="G$1" pin="5"/>
 <wire x1="34.29" y1="220.98" x2="27.94" y2="220.98" width="0.1524" layer="91"/>
@@
 <wire x1="274.32" y1="142.24" x2="276.86" y2="142.24" width="0.1524" layer="91"/>
 <wire x1="276.86" y1="142.24" x2="276.86" y2="132.08" width="0.1524" layer="91"/>
+</segment>
+<segment>
+<pinref part="IMU" gate="G$1" pin="FSYNC"/>
+<pinref part="GND27" gate="1" pin="GND"/>
+<wire x1="355.6" y1="152.4" x2="340.868" y2="152.4" width="0.1524" layer="91"/>
+<wire x1="340.868" y1="152.4" x2="340.868" y2="141.986" width="0.1524" layer="91"/>
+<pinref part="IMU" gate="G$1" pin="AD0/SDO"/>
+<wire x1="355.6" y1="142.24" x2="340.868" y2="142.24" width="0.1524" layer="91"/>
+<wire x1="340.868" y1="142.24" x2="340.868" y2="141.986" width="0.1524" layer="91"/>
+<junction x="340.868" y="141.986"/>
 </segment>
 </net>
@@
 </segment>
 </net>
-<net name="IMU_INT" class="0">
-<segment>
-<pinref part="U2" gate="G$1" pin="12/MISO0"/>
-<wire x1="165.1" y1="205.74" x2="160.02" y2="205.74" width="0.1524" layer="91"/>
-<label x="160.02" y="205.74" size="1.778" layer="95" rot="R180" xref="yes"/>
-</segment>
-<segment>
-<pinref part="IMU" gate="G$1" pin="INT1"/>
-<wire x1="396.24" y1="149.86" x2="398.78" y2="149.86" width="0.1524" layer="91"/>
-<label x="398.78" y="149.86" size="1.778" layer="95" xref="yes"/>
-</segment>
-</net>
-<net name="IMU_AD0" class="0">
-<segment>
-<pinref part="U2" gate="G$1" pin="9/RX2/PWM"/>
-<wire x1="165.1" y1="213.36" x2="160.02" y2="213.36" width="0.1524" layer="91"/>
-<label x="160.02" y="213.36" size="1.778" layer="95" rot="R180" xref="yes"/>
-</segment>
-<segment>
-<pinref part="IMU" gate="G$1" pin="AD0/SDO"/>
-<wire x1="355.6" y1="142.24" x2="353.06" y2="142.24" width="0.1524" layer="91"/>
-<label x="353.06" y="142.24" size="1.778" layer="95" rot="R180" xref="yes"/>
-</segment>
-</net>

Commit message: Rearranged capacitors/Created 6 Pin SMD Connector Footprint
Parts:
- removed L_MOT, R_MOT: (no value), pinhead:PINHD-1X2
- removed U3, U4: MAX4173-SOT-23, Gucci_ControlBoard:MAX4173-SOT-23
Connections:
- removed net CURRENT_L: U2.A21/DAC0, U4.OUT
- removed net CURRENT_R: U2.14/A0/PWM, U3.OUT
- removed net L_MOT+: L_MOT.2, U4.RS+
- removed net L_MOT-: L_MOT.1, U4.RS-
- removed net R_MOT+: R_MOT.2, U3.RS+
- removed net R_MOT-: R_MOT.1, U3.RS-
- net 3.3V: no longer U3.VCC, U4.VCC
- net GND: no longer U3.GND, U4.GND
Other:
- note removed: "Current Sensing"
Changed lines of the file:
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@@
 <part name="C18" library="SparkFun-Capacitors" library_urn="urn:adsk.eagle:library:510" deviceset="0.1UF" device="-0603-25V-(+80/-20%)" package3d_urn="urn:adsk.eagle:package:37414/1" value="15pF"/>
 <part name="C17" library="SparkFun-Capacitors" library_urn="urn:adsk.eagle:library:510" deviceset="0.1UF" device="-0603-25V-(+80/-20%)" package3d_urn="urn:adsk.eagle:package:37414/1" value="15pF"/>
-<part name="L_MOT" library="pinhead" library_urn="urn:adsk.eagle:library:325" deviceset="PINHD-1X2" device="" package3d_urn="urn:adsk.eagle:package:22435/2"/>
-<part name="R_MOT" library="pinhead" library_urn="urn:adsk.eagle:library:325" deviceset="PINHD-1X2" device="" package3d_urn="urn:adsk.eagle:package:22435/2"/>
-<part name="U4" library="Gucci_ControlBoard" deviceset="MAX4173-SOT-23" device=""/>
-<part name="U3" library="Gucci_ControlBoard" deviceset="MAX4173-SOT-23" device=""/>
-<part name="GND28" library="SparkFun-PowerSymbols" library_urn="urn:adsk.eagle:library:530" deviceset="GND" device=""/>
-<part name="GND29" library="SparkFun-PowerSymbols" library_urn="urn:adsk.eagle:library:530" deviceset="GND" device=""/>
 <part name="C8" library="SparkFun-Capacitors" library_urn="urn:adsk.eagle:library:510" deviceset="0.1UF" device="-0603-25V-(+80/-20%)" package3d_urn="urn:adsk.eagle:package:37414/1" value="0.1uF"/>
 <part name="C16" library="SparkFun-Capacitors" library_urn="urn:adsk.eagle:library:510" deviceset="0.1UF" device="-0603-25V-(+80/-20%)" package3d_urn="urn:adsk.eagle:package:37414/1" value="0.1uF"/>
-<part name="SUPPLY30" library="SparkFun-PowerSymbols" library_urn="urn:adsk.eagle:library:530" deviceset="3.3V" device=""/>
-<part name="SUPPLY31" library="SparkFun-PowerSymbols" library_urn="urn:adsk.eagle:library:530" deviceset="3.3V" device=""/>
 <part name="LED1" library="adafruit" library_urn="urn:adsk.eagle:library:420" deviceset="WS2812B" device="5050" package3d_urn="urn:adsk.eagle:package:6240942/1"/>
 <part name="GND19" library="supply1" library_urn="urn:adsk.eagle:library:371" deviceset="GND" device=""/>
@@
 <wire x1="15.24" y1="127" x2="116.84" y2="127" width="1.27" layer="97" style="shortdash"/>
 <wire x1="187.96" y1="127" x2="187.96" y2="78.74" width="1.27" layer="97" style="shortdash"/>
-<text x="187.96" y="71.12" size="5.08" layer="97">Current Sensing</text>
 <wire x1="335.28" y1="177.8" x2="335.28" y2="261.62" width="1.27" layer="97" style="shortdash"/>
 <text x="269.24" y="243.84" size="5.08" layer="97">NeoPixel Status</text>
@@
 <attribute name="VALUE" x="176.784" y="89.281" size="1.778" layer="96" font="vector"/>
 </instance>
-<instance part="L_MOT" gate="G$1" x="190.5" y="30.48" smashed="yes" rot="R180">
-<attribute name="NAME" x="196.85" y="24.765" size="1.778" layer="95" rot="R180"/>
-<attribute name="VALUE" x="196.85" y="35.56" size="1.778" layer="96" rot="R180"/>
-</instance>
-<instance part="R_MOT" gate="G$1" x="228.6" y="30.48" smashed="yes" rot="R180">
-<attribute name="NAME" x="234.95" y="24.765" size="1.778" layer="95" rot="R180"/>
-<attribute name="VALUE" x="234.95" y="35.56" size="1.778" layer="96" rot="R180"/>
-</instance>
-<instance part="U4" gate="G$1" x="193.04" y="53.34" smashed="yes">
-<attribute name="NAME" x="182.88" y="60.96" size="2.54" layer="95"/>
-<attribute name="VALUE" x="182.88" y="43.18" size="2.54" layer="96"/>
-</instance>
-<instance part="U3" gate="G$1" x="233.68" y="53.34" smashed="yes">
-<attribute name="NAME" x="223.52" y="60.96" size="2.54" layer="95"/>
-<attribute name="VALUE" x="223.52" y="43.18" size="2.54" layer="96"/>
-</instance>
-<instance part="GND28" gate="1" x="193.04" y="38.1" smashed="yes">
-<attribute name="VALUE" x="193.04" y="37.846" size="1.778" layer="96" align="top-center"/>
-</instance>
-<instance part="GND29" gate="1" x="233.68" y="38.1" smashed="yes">
-<attribute name="VALUE" x="233.68" y="37.846" size="1.778" layer="96" align="top-center"/>
-</instance>
 <instance part="C8" gate="G$1" x="391.16" y="58.42" smashed="yes">
 <attribute name="NAME" x="392.684" y="61.341" size="1.778" layer="95" font="vector"/>
@@
 <attribute name="NAME" x="331.724" y="61.341" size="1.778" layer="95" font="vector"/>
 <attribute name="VALUE" x="331.724" y="56.261" size="1.778" layer="96" font="vector"/>
-</instance>
-<instance part="SUPPLY30" gate="G$1" x="193.04" y="66.04" smashed="yes">
-<attribute name="VALUE" x="193.04" y="68.834" size="1.778" layer="96" align="bottom-center"/>
-</instance>
-<instance part="SUPPLY31" gate="G$1" x="233.68" y="66.04" smashed="yes">
-<attribute name="VALUE" x="233.68" y="68.834" size="1.778" layer="96" align="bottom-center"/>
 </instance>
 <instance part="LED1" gate="G$1" x="294.64" y="215.9" smashed="yes"/>
@@
 <pinref part="SUPPLY29" gate="G$1" pin="3.3V"/>
 <wire x1="175.26" y1="109.22" x2="175.26" y2="106.68" width="0.1524" layer="91"/>
-</segment>
-<segment>
-<pinref part="SUPPLY30" gate="G$1" pin="3.3V"/>
-<pinref part="U4" gate="G$1" pin="VCC"/>
-</segment>
-<segment>
-<pinref part="SUPPLY31" gate="G$1" pin="3.3V"/>
-<pinref part="U3" gate="G$1" pin="VCC"/>
 </segment>
 </net>
@@
 </segment>
 <segment>
-<pinref part="U4" gate="G$1" pin="GND"/>
-<pinref part="GND28" gate="1" pin="GND"/>
-</segment>
-<segment>
-<pinref part="U3" gate="G$1" pin="GND"/>
-<pinref part="GND29" gate="1" pin="GND"/>
-</segment>
-<segment>
 <pinref part="LED1" gate="G$1" pin="GND"/>
 <pinref part="GND19" gate="1" pin="GND"/>
@@
 </segment>
 </net>
-<net name="CURRENT_L" class="0">
-<segment>
-<pinref part="U4" gate="G$1" pin="OUT"/>
-<wire x1="208.28" y1="53.34" x2="210.82" y2="53.34" width="0.1524" layer="91"/>
-<label x="210.82" y="53.34" size="1.778" layer="95" rot="R90" xref="yes"/>
-</segment>
-<segment>
-<pinref part="U2" gate="G$1" pin="A21/DAC0"/>
-<wire x1="218.44" y1="185.42" x2="223.52" y2="185.42" width="0.1524" layer="91"/>
-<label x="223.52" y="185.42" size="1.778" layer="95" xref="yes"/>
-</segment>
-</net>
-<net name="CURRENT_R" class="0">
-<segment>
-<pinref part="U3" gate="G$1" pin="OUT"/>
-<wire x1="248.92" y1="53.34" x2="251.46" y2="53.34" width="0.1524" layer="91"/>
-<label x="251.46" y="53.34" size="1.778" layer="95" rot="R90" xref="yes"/>
-</segment>
-<segment>
-<label x="160.02" y="200.66" size="1.778" layer="95" rot="R180" xref="yes"/>
-<pinref part="U2" gate="G$1" pin="14/A0/PWM"/>
-<wire x1="165.1" y1="200.66" x2="160.02" y2="200.66" width="0.1524" layer="91"/>
-</segment>
-</net>
-<net name="L_MOT+" class="0">
-<segment>
-<pinref part="U4" gate="G$1" pin="RS+"/>
-<wire x1="177.8" y1="55.88" x2="175.26" y2="55.88" width="0.1524" layer="91"/>
-<label x="175.26" y="55.88" size="1.778" layer="95" rot="R90" xref="yes"/>
-</segment>
-<segment>
-<pinref part="L_MOT" gate="G$1" pin="2"/>
-<wire x1="193.04" y1="30.48" x2="198.12" y2="30.48" width="0.1524" layer="91"/>
-<label x="198.12" y="30.48" size="1.778" layer="95" xref="yes"/>
-</segment>
-</net>
-<net name="L_MOT-" class="0">
-<segment>
-<pinref part="U4" gate="G$1" pin="RS-"/>
-<wire x1="177.8" y1="50.8" x2="175.26" y2="50.8" width="0.1524" layer="91"/>
-<label x="175.26" y="50.8" size="1.778" layer="95" rot="R270" xref="yes"/>
-</segment>
-<segment>
-<pinref part="L_MOT" gate="G$1" pin="1"/>
-<wire x1="193.04" y1="27.94" x2="198.12" y2="27.94" width="0.1524" layer="91"/>
-<label x="198.12" y="27.94" size="1.778" layer="95" xref="yes"/>
-</segment>
-</net>
-<net name="R_MOT+" class="0">
-<segment>
-<pinref part="U3" gate="G$1" pin="RS+"/>
-<wire x1="218.44" y1="55.88" x2="215.9" y2="55.88" width="0.1524" layer="91"/>
-<label x="215.9" y="55.88" size="1.778" layer="95" rot="R90" xref="yes"/>
-</segment>
-<segment>
-<pinref part="R_MOT" gate="G$1" pin="2"/>
-<wire x1="231.14" y1="30.48" x2="236.22" y2="30.48" width="0.1524" layer="91"/>
-<label x="236.22" y="30.48" size="1.778" layer="95" xref="yes"/>
-</segment>
-</net>
-<net name="R_MOT-" class="0">
-<segment>
-<pinref part="U3" gate="G$1" pin="RS-"/>
-<wire x1="218.44" y1="50.8" x2="215.9" y2="50.8" width="0.1524" layer="91"/>
-<label x="215.9" y="50.8" size="1.778" layer="95" rot="R270" xref="yes"/>
-</segment>
-<segment>
-<pinref part="R_MOT" gate="G$1" pin="1"/>
-<wire x1="231.14" y1="27.94" x2="236.22" y2="27.94" width="0.1524" layer="91"/>
-<label x="236.22" y="27.94" size="1.778" layer="95" xref="yes"/>
-</segment>
-</net>

Commit message: Moved NeoPixel to the center
Connections:
- net NEO_DI: now also U2.11/MOSI0; no longer U2.38/A19/SDA1/PWM
Changed lines of the file:
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@@
 <net name="NEO_DI" class="0">
 <segment>
-<pinref part="U2" gate="G$1" pin="38/A19/SDA1/PWM"/>
-<wire x1="165.1" y1="139.7" x2="160.02" y2="139.7" width="0.1524" layer="91"/>
-<label x="160.02" y="139.7" size="1.778" layer="95" rot="R180" xref="yes"/>
+<label x="160.02" y="208.28" size="1.778" layer="95" rot="R180" xref="yes"/>
+<pinref part="U2" gate="G$1" pin="11/MOSI0"/>
+<wire x1="160.02" y1="208.28" x2="165.1" y2="208.28" width="0.1524" layer="91"/>
 </segment>
 <segment>

Commit message: Removed NeoPixel DO Connector
Connections:
- net NEO_DO: no longer LED1.DO
Changed lines of the file:
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@@
 <label x="160.02" y="137.16" size="1.778" layer="95" rot="R180" xref="yes"/>
-</segment>
-<segment>
-<pinref part="LED1" gate="G$1" pin="DO"/>
-<wire x1="307.34" y1="213.36" x2="314.96" y2="213.36" width="0.1524" layer="91"/>
-<label x="314.96" y="213.36" size="1.778" layer="95" xref="yes"/>
 </segment>
 </net>
