File: Gucci/v2 pcb/Gucci_ControlBoard.sch (EAGLE design)
At the start: 53 parts, among them U1 PCA9306_LSSOP, U2 TEENSY_3.6_DIL, U5 LM393-8-SOIC, U6 AP2114H-1.8TRG1, U7 AP2114H-3.3TRG1

Commit message: Wired Radio Tranceiver to Teensi
Added a pin header and connected to respective pins on Teensi/Changed NeoPixel pin to Pin 24
Parts:
- added TRANSCEIVER: (no value), adafruit:PINHD-1X8BIG
Connections:
- new net +3V3: TRANSCEIVER.8
- new net DIO0: TRANSCEIVER.6, U2.14/A0/PWM
- new net MISO: TRANSCEIVER.1, U2.12/MISO0
- new net MOSI: TRANSCEIVER.2, U2.11/MOSI0
- new net NSS: TRANSCEIVER.4, U2.10/TX2/PWM
- new net SCK: TRANSCEIVER.3, U2.13/SCK0/LED
- net GND: now also TRANSCEIVER.7
- net NEO_DI: now also U2.24; no longer U2.11/MOSI0
Changed lines of the file:
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@@
 <part name="SUPPLY15" library="SparkFun-PowerSymbols" deviceset="5V" device=""/>
 <part name="GND15" library="SparkFun-PowerSymbols" library_urn="urn:adsk.eagle:library:530" deviceset="GND" device=""/>
+<part name="TRANSCEIVER" library="adafruit" library_urn="urn:adsk.eagle:library:420" deviceset="PINHD-1X8" device="BIG" package3d_urn="urn:adsk.eagle:package:6240707/1"/>
+<part name="GND16" library="supply1" library_urn="urn:adsk.eagle:library:371" deviceset="GND" device=""/>
+<part name="+3V11" library="supply1" library_urn="urn:adsk.eagle:library:371" deviceset="+3V3" device=""/>
 </parts>
 <sheets>
@@
 <attribute name="VALUE" x="276.86" y="129.286" size="1.778" layer="96" align="top-center"/>
 </instance>
+<instance part="TRANSCEIVER" gate="G$1" x="231.14" y="53.34" smashed="yes">
+<attribute name="NAME" x="224.79" y="64.897" size="1.778" layer="95"/>
+<attribute name="VALUE" x="224.79" y="38.1" size="1.778" layer="96"/>
+</instance>
+<instance part="GND16" gate="1" x="210.82" y="38.1" smashed="yes">
+<attribute name="VALUE" x="208.28" y="35.56" size="1.778" layer="96"/>
+</instance>
+<instance part="+3V11" gate="G$1" x="218.44" y="45.72" smashed="yes">
+<attribute name="VALUE" x="215.9" y="40.64" size="1.778" layer="96" rot="R90"/>
+</instance>
 </instances>
 <busses>
@@
 <junction x="340.868" y="141.986"/>
 </segment>
+<segment>
+<pinref part="GND16" gate="1" pin="GND"/>
+<pinref part="TRANSCEIVER" gate="G$1" pin="7"/>
+<wire x1="210.82" y1="40.64" x2="210.82" y2="45.72" width="0.1524" layer="91"/>
+<wire x1="210.82" y1="45.72" x2="228.6" y2="45.72" width="0.1524" layer="91"/>
+</segment>
 </net>
 <net name="SHDN0" class="0">
@@
 <net name="NEO_DI" class="0">
 <segment>
-<label x="160.02" y="208.28" size="1.778" layer="95" rot="R180" xref="yes"/>
-<pinref part="U2" gate="G$1" pin="11/MOSI0"/>
-<wire x1="160.02" y1="208.28" x2="165.1" y2="208.28" width="0.1524" layer="91"/>
+<label x="160.02" y="175.26" size="1.778" layer="95" rot="R180" xref="yes"/>
+<pinref part="U2" gate="G$1" pin="24"/>
+<wire x1="165.1" y1="175.26" x2="160.02" y2="175.26" width="0.1524" layer="91"/>
 </segment>
 <segment>
@@
 </segment>
 </net>
+<net name="MISO" class="0">
+<segment>
+<label x="223.52" y="60.96" size="1.778" layer="95" rot="R180" xref="yes"/>
+<pinref part="TRANSCEIVER" gate="G$1" pin="1"/>
+<wire x1="228.6" y1="60.96" x2="223.52" y2="60.96" width="0.1524" layer="91"/>
+</segment>
+<segment>
+<pinref part="U2" gate="G$1" pin="12/MISO0"/>
+<wire x1="165.1" y1="205.74" x2="160.02" y2="205.74" width="0.1524" layer="91"/>
+<label x="160.02" y="205.74" size="1.778" layer="95" rot="R180" xref="yes"/>
+</segment>
+</net>
+<net name="MOSI" class="0">
+<segment>
+<label x="223.52" y="58.42" size="1.778" layer="95" rot="R180" xref="yes"/>
+<pinref part="TRANSCEIVER" gate="G$1" pin="2"/>
+<wire x1="228.6" y1="58.42" x2="223.52" y2="58.42" width="0.1524" layer="91"/>
+</segment>
+<segment>
+<pinref part="U2" gate="G$1" pin="11/MOSI0"/>
+<wire x1="165.1" y1="208.28" x2="160.02" y2="208.28" width="0.1524" layer="91"/>
+<label x="160.02" y="208.28" size="1.778" layer="95" rot="R180" xref="yes"/>
+</segment>
+</net>
+<net name="SCK" class="0">
+<segment>
+<label x="223.52" y="55.88" size="1.778" layer="95" rot="R180" xref="yes"/>
+<pinref part="TRANSCEIVER" gate="G$1" pin="3"/>
+<wire x1="228.6" y1="55.88" x2="223.52" y2="55.88" width="0.1524" layer="91"/>
+</segment>
+<segment>
+<pinref part="U2" gate="G$1" pin="13/SCK0/LED"/>
+<wire x1="165.1" y1="203.2" x2="160.02" y2="203.2" width="0.1524" layer="91"/>
+<label x="160.02" y="203.2" size="1.778" layer="95" rot="R180" xref="yes"/>
+</segment>
+</net>
+<net name="+3V3" class="0">
+<segment>
+<pinref part="+3V11" gate="G$1" pin="+3V3"/>
+<pinref part="TRANSCEIVER" gate="G$1" pin="8"/>
+<wire x1="218.44" y1="43.18" x2="228.6" y2="43.18" width="0.1524" layer="91"/>
+</segment>
+</net>
+<net name="NSS" class="0">
+<segment>
+<pinref part="TRANSCEIVER" gate="G$1" pin="4"/>
+<wire x1="228.6" y1="53.34" x2="223.52" y2="53.34" width="0.1524" layer="91"/>
+<label x="223.52" y="53.34" size="1.778" layer="95" rot="R180" xref="yes"/>
+</segment>
+<segment>
+<pinref part="U2" gate="G$1" pin="10/TX2/PWM"/>
+<wire x1="165.1" y1="210.82" x2="160.02" y2="210.82" width="0.1524" layer="91"/>
+<label x="160.02" y="210.82" size="1.778" layer="95" rot="R180" xref="yes"/>
+</segment>
+</net>
+<net name="DIO0" class="0">
+<segment>
+<pinref part="TRANSCEIVER" gate="G$1" pin="6"/>
+<wire x1="228.6" y1="48.26" x2="223.52" y2="48.26" width="0.1524" layer="91"/>
+<label x="223.52" y="48.26" size="1.778" layer="95" rot="R180" xref="yes"/>
+</segment>
+<segment>
+<pinref part="U2" gate="G$1" pin="14/A0/PWM"/>
+<wire x1="165.1" y1="200.66" x2="160.02" y2="200.66" width="0.1524" layer="91"/>
+<label x="160.02" y="200.66" size="1.778" layer="95" rot="R180" xref="yes"/>
+</segment>
+</net>

Commit message: Replace Omiron Sensors/Fixed Wiring
Replaced the Omiron Distance Sensors (Still need to add multiplexers to wire to Teensi)
Fixed some wiring and naming of the radio transciever.
Connections:
- net DIO0 renamed RADIO_DIO0
- net NSS renamed RADIO_NSS
- net SCK renamed RADIO_SCK
Changed lines of the file:
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@@
 </segment>
 </net>
-<net name="SCK" class="0">
+<net name="RADIO_SCK" class="0">
 <segment>
 <label x="223.52" y="55.88" size="1.778" layer="95" rot="R180" xref="yes"/>
@@
 </segment>
 </net>
-<net name="NSS" class="0">
+<net name="RADIO_NSS" class="0">
 <segment>
 <pinref part="TRANSCEIVER" gate="G$1" pin="4"/>
@@
 </segment>
 </net>
-<net name="DIO0" class="0">
+<net name="RADIO_DIO0" class="0">
 <segment>
 <pinref part="TRANSCEIVER" gate="G$1" pin="6"/>

Commit message: Fixed Github versioning
Gucci:
V2 - 9/11/2019 (last push before competition)
V3 - current
Kirbi:
V1 - 9/11/2019 (last push before competition)
V2 - current
Parts:
- removed ESC: MOLEX_1.25MM_4PIN_SMT, Gucci_ControlBoard:MOLEX_1.25MM_4PIN_SMT
- removed LED1: WS2812B5050, adafruit:WS2812B5050
- removed POWER: POWER_SWITCH, Gucci_ControlBoard:POWER_SWITCH
- removed TRANSCEIVER: (no value), adafruit:PINHD-1X8BIG
- added C7: 10uF, SparkFun-Capacitors:0.1UF-0603-25V-(+80/-20%)
- added L_ENC, R_ENC: (no value), pinhead:PINHD-2X5/90
- added L_ESC, R_ESC: JST_PHD_2X04, Gucci_ControlBoard:JST_PHD_2X04
- added L_MOT, R_MOT: (no value), pinhead:PINHD-1X2
- added R10, R12, R2, R4, R6, R8: 3k, SparkFun-Resistors:1KOHM-0603-1/10W-1%
- added R11, R3, R5, R7, R9: 2k, SparkFun-Resistors:1KOHM-0603-1/10W-1%
- added U3, U4: MAX4173-SOT-23, Gucci_ControlBoard:MAX4173-SOT-23
- R1: value 50 -> 2k
Connections:
- removed net +3V3: TRANSCEIVER.8
- removed net MISO: TRANSCEIVER.1, U2.12/MISO0
- removed net MOSI: TRANSCEIVER.2, U2.11/MOSI0
- removed net N$6: ESC.4, POWER.P4
- removed net NEO_DI: LED1.DI, U2.24
- removed net NEO_DO: U2.39/A20
- removed net RADIO_DIO0: TRANSCEIVER.6, U2.14/A0/PWM
- removed net RADIO_NSS: TRANSCEIVER.4, U2.10/TX2/PWM
- removed net RADIO_SCK: TRANSCEIVER.3, U2.13/SCK0/LED
- new net 3V_ENCODER1_A: R5.2, R6.2, U2.22/A8/T/PWM
- new net 3V_ENCODER1_B: R3.2, R4.2, U2.21/A7/PWM
- new net 3V_ENCODER1_I: R1.2, R2.2, U2.20/A6/PWM
- new net 3V_ENCODER2_A: R11.2, R12.2, U2.38/A19/SDA1/PWM
- new net 3V_ENCODER2_B: R10.2, R9.2, U2.37/A18/SCL1/PWM
- new net 3V_ENCODER2_I: R7.2, R8.2, U2.36/A17/PWM
- new net CURRENT_L: U2.A21/DAC0, U4.OUT
- new net CURRENT_R: U2.14/A0/PWM, U3.OUT
- new net ENCODER1_A: R5.1, R_ENC.6, R_ESC.6
- new net ENCODER1_B: R3.1, R_ENC.8, R_ESC.8
- new net ENCODER2_A: L_ENC.6, L_ESC.3, R11.1
- new net ENCODER2_B: L_ENC.8, L_ESC.1, R9.1
- new net IMU_AD0: IMU.AD0/SDO, U2.9/RX2/PWM
- new net IMU_INT: IMU.INT1, U2.12/MISO0
- new net L_MOT+: L_MOT.2, U4.RS+
- new net L_MOT-: L_MOT.1, U4.RS-
- new net N$8: L_ENC.10, R7.1
- new net R_MOT+: R_MOT.2, U3.RS+
- new net R_MOT-: R_MOT.1, U3.RS-
- net 3.3V: now also U3.VCC, U4.VCC
- net 5V: now also C7.1, L_ENC.2, L_ESC.6, L_ESC.7, R_ENC.2, R_ESC.2, R_ESC.3; no longer LED1.VDD, POWER.P3, POWER.P5
- net GND: now also C7.2, L_ENC.3, L_ESC.5, L_ESC.8, R10.1, R12.1, R2.1, R4.1, R6.1, R8.1, R_ENC.3, R_ESC.1, R_ESC.4, U3.GND, U4.GND; no longer ESC.1, IMU.AD0/SDO, LED1.GND, R1.2, TRANSCEIVER.7
- net N$5: now also R_ENC.10; no longer POWER.P1
- net RX0: now also R_ESC.7
- net RX1: now also L_ESC.2
- net TX0: now also R_ESC.5
- net TX1: now also L_ESC.4
Other:
- note added: "Current Sensing"
- note added: "Encoder Connectos And Signal Shifting For Teensy"
- note removed: "NeoPixel Status"
- note removed: "Power"
- moved on the sheet: D1, D2, D3, R1, R18, R19, R20
