File: Kirbi/Kirbi_ControlBoard.sch (EAGLE design)
At the start: 47 parts, among them J10 JST_PH_1X03, J15 JST_PH_1X03_90, J7 JST_PH_1X03_90, J8 JST_PH_1X03_90, J9 JST_PH_1X03, U1 TEENSY_3.6_DIL, U2 AP2114H-3.3TRG1, U3 AP2114H-1.8TRG1, U4 ICM-20948, U5 LM339-14-SOIC

Commit message: kirbi iteration with modified libraries
Parts:
- added C1, C4: 1uF, SparkFun-Capacitors:0.1UF-0603-25V-(+80/-20%)
- added C10, C9: 0.1uF, SparkFun-Capacitors:0.1UF-0603-25V-(+80/-20%)
- added C3, C6: 10uF, SparkFun-Capacitors:0.1UF-0603-25V-(+80/-20%)
- added J1, J2, J5, J6: JST_PH_1X03_90, Gucci_ControlBoard:JST_PH_1X03_90
- added J11: TE_02X01_3.96MM, Kirbi_ControlBoard:TE_02X01_3.96MM
- added J12, J3, J4: MOLEX_1.25MM_4PIN_90, Kirbi_ControlBoard:MOLEX_1.25MM_4PIN_90
- added R21, R23, R25, R28: 6.98k, SparkFun-Resistors:1KOHM-0603-1/10W-1%
- added R22, R24, R26, R27: 1k, SparkFun-Resistors:1KOHM-0603-1/10W-1%
Connections:
- new net +5V: C19.1
- new net 24V: C10.1, C4.1, C6.1, C9.1, J1.3, J11.+, J2.1, J5.3, J6.1
- new net DIST_L: R23.1, R24.2, U1.30/T/PWM
- new net DIST_L_24: J6.2, R23.2
- new net DIST_L_45: R25.1, R26.2, U1.29/T/PWM
- new net DIST_L_45_24: J5.2, R25.2
- new net DIST_R: R21.1, R22.2, U1.2/PWM
- new net DIST_R_24: J1.2, R21.2
- new net DIST_R_45: R27.2, R28.1, U1.3/CAN0-TX/SCL2/PWM
- new net DIST_R_45_24: J2.2, R28.2
- new net RX1: J3.3, U1.0/RX1/MOSI1/T
- new net RX2: J4.3, U1.31/A12/RX4
- new net S1/TX: J12.2, U1.33/A14/TX5/CAN1-TX
- new net S2: J12.1, U1.34/A15/RX5/CAN1-RX
- new net TX1: J3.2, U1.1/TX1/MISO1/T
- new net TX2: J4.2, U1.32/A13/TX4
- net 5V: now also C1.1, C3.1, J12.3, J3.1, J4.1; no longer C19.1
- net GND: now also C1.2, C10.2, C3.2, C4.2, C6.2, C9.2, J1.1, J11.-, J12.4, J2.3, J3.4, J4.4, J5.1, J6.3, R22.1, R24.1, R26.1, R27.1
- net SCL1: now also U1.7/RX3/PWM; no longer U1.3/CAN0-TX/SCL2/PWM
- net SDA1: now also U1.8/TX3/PWM; no longer U1.4/CAN0-RX/SDA2/PWM
Other:
- note added: "Battery Connector"
- note added: "ESC Connector"
- note added: "Lidar Connectors"
- note added: "Omron Distance Sensors"
- note removed: "ESC Connectors"
- note removed: "Time of Flight Connectors"
- moved on the sheet: C19, C2, C5, C7, C8, R15, R16

Commit message: level shifter
added level shifter to gucci and kirbi. the part is in gucci's library. the relevant area on the boards should be very similar, but not identical
Parts:
- added R29: 200k, SparkFun-Resistors:1KOHM-0603-1/10W-1%
- added R30, R31: 10k, SparkFun-Resistors:1KOHM-0603-1/10W-1%
- added U6: PCA9306_LSSOP, Gucci_ControlBoard:PCA9306_LSSOP
Connections:
- new net N$4: R29.1, U6.EN, U6.VREF2
- new net SCL2: R16.1, U1.7/RX3/PWM, U6.SCL2
- new net SDA2: R15.1, U1.8/TX3/PWM, U6.SDA2
- net 1.8V: now also R30.2, R31.2, U6.VREF1; no longer R15.2, R16.2
- net 3V3: now also R15.2, R16.2, R29.2
- net GND: now also U6.GND
- net SCL1: now also R31.1, U6.SCL1; no longer R16.1, U1.7/RX3/PWM
- net SDA1: now also R30.1, U6.SDA1; no longer R15.1, U1.8/TX3/PWM
Other:
- moved on the sheet: C16, C17, C18, J13, J14, R1, R10, R11, R12, R15, R2, R3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
