File: Kirbi/Kirbi_ControlBoard.brd (EAGLE design)
At the start: 66 x 56 mm, 50 parts, among them J10 JST_PH_1X03, J15 JST_PH_1X03_90, J7 JST_PH_1X03_90, J8 JST_PH_1X03_90, J9 JST_PH_1X03, U1 TEENSY_3.6_DIL, U2 AP2114H-3.3TRG1, U3 AP2114H-1.8TRG1, U4 ICM-20948, U5 LM339-14-SOIC

Commit message: kirbi iteration with modified libraries
Parts:
- added C1, C4: 1uF, SparkFun-Capacitors:0603
- added C10, C9: 0.1uF, SparkFun-Capacitors:0603
- added C3, C6: 10uF, SparkFun-Capacitors:0603
- added J1, J2, J5, J6: JST_PH_1X03_90, Gucci_ControlBoard:JST_PH_1X03_90
- added J11: TE_02X01_3.96MM, Kirbi_ControlBoard:TE_02X01_3.96MM
- added J12, J3, J4: MOLEX_1.25MM_4PIN_90, Kirbi_ControlBoard:MOLEX_1.25MM_4PIN_90
- added R21, R23, R25, R28: 6.98k, SparkFun-Resistors:0603
- added R22, R24, R26, R27: 1k, SparkFun-Resistors:0603
- added U$4: (no value), RoboJackets-Aesthetics:ROBOBUZZ_0.4X
- moved U$3 8.94 mm to (33.0, 17.0)
- moved C14 1.00 mm to (25.0, 11.0)
- moved C15 1.00 mm to (13.0, 11.0)
- moved U3 1.00 mm to (19.0, 12.0)
Connections:
- new net +5V: C19.1
- new net 24V: C10.1, C4.1, C6.1, C9.1, J1.3, J11.P$1, J2.1, J5.3, J6.1
- new net DIST_L: R23.1, R24.2, U1.30
- new net DIST_L_24: J6.2, R23.2
- new net DIST_L_45: R25.1, R26.2, U1.29
- new net DIST_L_45_24: J5.2, R25.2
- new net DIST_R: R21.1, R22.2, U1.2
- new net DIST_R_24: J1.2, R21.2
- new net DIST_R_45: R27.2, R28.1, U1.3
- new net DIST_R_45_24: J2.2, R28.2
- new net RX1: J3.P$3, U1.0
- new net RX2: J4.P$3, U1.31/A12
- new net S1/TX: J12.P$2, U1.33/A14
- new net S2: J12.P$1, U1.34/A15
- new net TX1: J3.P$2, U1.1
- new net TX2: J4.P$2, U1.32/A13
- net 5V: now also C1.1, C3.1, J12.P$3, J3.P$1, J4.P$1; no longer C19.1
- net GND: now also C1.2, C10.2, C3.2, C4.2, C6.2, C9.2, J1.1, J11.P$2, J12.P$4, J2.3, J3.P$4, J4.P$4, J5.1, J6.3, R22.1, R24.1, R26.1, R27.1
- net SCL1: now also U1.7; no longer U1.3
- net SDA1: now also U1.8; no longer U1.4
Routing:
- net 24V: track 0.00 -> 95.4 mm
- net 3V3: track 98.9 -> 152.7 mm
- net RX1: track 0.00 -> 46.7 mm
- net TX2: track 0.00 -> 45.2 mm
- net GND: track 87.8 -> 133.0 mm, vias 10 -> 12
- net TX1: track 0.00 -> 43.7 mm
- net RX2: track 0.00 -> 42.8 mm
- net DIST_L_45: track 0.00 -> 17.2 mm
- net DIST_R_45: track 0.00 -> 17.0 mm
- net SCL1: track 28.2 -> 13.5 mm
- net DIST_R: track 0.00 -> 11.6 mm
- net S2: track 0.00 -> 10.7 mm
- net DIST_L: track 0.00 -> 10.6 mm
- net SDA1: track 23.4 -> 13.6 mm, vias 1 -> 0
- net S1/TX: track 0.00 -> 9.62 mm
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- removed copper zone on layer 1, net 3V3

Commit message: level shifter
added level shifter to gucci and kirbi. the part is in gucci's library. the relevant area on the boards should be very similar, but not identical
Parts:
- added R29: 200k, SparkFun-Resistors:0603
- added R30, R31: 10k, SparkFun-Resistors:0603
- added U6: PCA9306_LSSOP, Gucci_ControlBoard:8-LSSOP
- moved C16 4.00 mm to (23.0, 17.0)
- moved C17 4.00 mm to (27.0, 22.0)
- moved C18 4.00 mm to (18.0, 18.0)
- moved U4 4.00 mm to (23.0, 21.0)
- moved R16 3.27 mm to (12.0, 23.7), turned to 90 degrees
- moved R15 3.00 mm to (14.4, 23.7), turned to 90 degrees
Connections:
- new net N$4: R29.1, U6.P$7, U6.P$8
- new net SCL2: R16.1, U1.7, U6.P$6
- new net SDA2: R15.1, U1.8, U6.P$5
- net 1.8V: now also R30.2, R31.2, U6.P$2; no longer R15.2, R16.2
- net 3V3: now also R15.2, R16.2, R29.2
- net GND: now also U6.P$1
- net SCL1: now also R31.1, U6.P$3; no longer R16.1, U1.7
- net SDA1: now also R30.1, U6.P$4; no longer R15.1, U1.8
Routing:
- net 3V3: track 152.7 -> 172.8 mm
- net SDA2: track 0.00 -> 18.1 mm
- net SCL2: track 0.00 -> 16.3 mm
- net SDA1: track 13.6 -> 10.4 mm
- net IMU_AD0: track 16.0 -> 18.5 mm
- net N$4: track 0.00 -> 2.47 mm
- net SCL1: track 13.5 -> 15.3 mm, vias 1 -> 0

Commit message: fixed silkscreens
Changed lines of the file:
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@@
 <drawing>
 <settings>
-<setting alwaysvectorfont="no"/>
+<setting alwaysvectorfont="yes"/>
 <setting verticaltext="up"/>
 </settings>
@@
 </element>
 <element name="R15" library="SparkFun-Resistors" package="0603" value="10k" x="14.4" y="23.7" smashed="yes" rot="R90">
-<attribute name="NAME" x="13.638" y="23.7" size="0.8128" layer="25" font="vector" ratio="20" rot="R90" align="bottom-center"/>
+<attribute name="NAME" x="14.4" y="26.238" size="0.8128" layer="25" font="vector" ratio="20" rot="R180" align="bottom-center"/>
 <attribute name="PROD_ID" value="RES-07856" x="14.4" y="23.7" size="1.778" layer="27" rot="R90" display="off"/>
-<attribute name="VALUE" x="15.162" y="23.7" size="0.8128" layer="21" font="vector" ratio="20" rot="R90" align="top-center"/>
+<attribute name="VALUE" x="14.4" y="22.038" size="0.8128" layer="21" font="vector" ratio="20" align="top-center"/>
 </element>
 <element name="R16" library="SparkFun-Resistors" package="0603" value="10k" x="12" y="23.7" smashed="yes" rot="R90">
-<attribute name="NAME" x="11.238" y="23.7" size="0.8128" layer="25" font="vector" ratio="20" rot="R90" align="bottom-center"/>
+<attribute name="NAME" x="12" y="26.238" size="0.8128" layer="25" font="vector" ratio="20" rot="R180" align="bottom-center"/>
 <attribute name="PROD_ID" value="RES-07856" x="12" y="23.7" size="1.778" layer="27" rot="R90" display="off"/>
-<attribute name="VALUE" x="12.762" y="23.7" size="0.8128" layer="21" font="vector" ratio="20" rot="R90" align="top-center"/>
+<attribute name="VALUE" x="12" y="22.038" size="0.8128" layer="21" font="vector" ratio="20" align="top-center"/>
 </element>
 <element name="C16" library="SparkFun-Capacitors" library_urn="urn:adsk.eagle:library:510" package="0603" package3d_urn="urn:adsk.eagle:package:37414/1" value="0.1uF" x="23" y="17" smashed="yes">
-<attribute name="NAME" x="20" y="15.762" size="0.8128" layer="25" font="vector" ratio="20" align="bottom-center"/>
+<attribute name="NAME" x="23.1" y="14.562" size="0.8128" layer="25" font="vector" ratio="20" align="bottom-center"/>
 <attribute name="PROD_ID" value="CAP-00810" x="23" y="17" size="1.778" layer="27" display="off"/>
-<attribute name="VALUE" x="19.8" y="15.738" size="0.8128" layer="21" font="vector" ratio="20" align="top-center"/>
+<attribute name="VALUE" x="23" y="16.238" size="0.8128" layer="21" font="vector" ratio="20" align="top-center"/>
 </element>
 <element name="C17" library="SparkFun-Capacitors" library_urn="urn:adsk.eagle:library:510" package="0603" package3d_urn="urn:adsk.eagle:package:37414/1" value="0.1uF" x="27" y="22" smashed="yes" rot="R90">
@@
 </element>
 <element name="U$4" library="RoboJackets-Aesthetics" package="ROBOBUZZ_0.4X" value="" x="5" y="17" smashed="yes"/>
-<element name="U6" library="Gucci_ControlBoard" package="8-LSSOP" value="PCA9306_LSSOP" x="12" y="19" rot="R180"/>
-<element name="R29" library="SparkFun-Resistors" package="0603" value="200k" x="9" y="15.6" rot="R270">
+<element name="U6" library="Gucci_ControlBoard" package="8-LSSOP" value="PCA9306_LSSOP" x="12" y="19" smashed="yes" rot="R180">
+<attribute name="NAME" x="13.1" y="16.5" size="1.27" layer="25" rot="R180"/>
+<attribute name="VALUE" x="14" y="21" size="0.8128" layer="27" rot="R180"/>
+</element>
+<element name="R29" library="SparkFun-Resistors" package="0603" value="200k" x="9" y="15.6" smashed="yes" rot="R270">
+<attribute name="NAME" x="9.762" y="15.6" size="0.8128" layer="25" font="vector" ratio="20" rot="R270" align="bottom-center"/>
 <attribute name="PROD_ID" value="RES-07856" x="9" y="15.6" size="1.778" layer="27" rot="R270" display="off"/>
-</element>
-<element name="R30" library="SparkFun-Resistors" package="0603" value="10k" x="18.9" y="23.7" rot="R90">
+<attribute name="VALUE" x="8.238" y="15.6" size="0.8128" layer="21" font="vector" ratio="20" rot="R270" align="top-center"/>
+</element>
+<element name="R30" library="SparkFun-Resistors" package="0603" value="10k" x="18.9" y="23.7" smashed="yes" rot="R90">
+<attribute name="NAME" x="18.9" y="26.238" size="0.8128" layer="25" font="vector" ratio="20" rot="R180" align="bottom-center"/>
 <attribute name="PROD_ID" value="RES-07856" x="18.9" y="23.7" size="1.778" layer="27" rot="R90" display="off"/>
-</element>
-<element name="R31" library="SparkFun-Resistors" package="0603" value="10k" x="16.7" y="23.7" rot="R90">
+<attribute name="VALUE" x="18.9" y="22.038" size="0.8128" layer="21" font="vector" ratio="20" align="top-center"/>
+</element>
+<element name="R31" library="SparkFun-Resistors" package="0603" value="10k" x="16.7" y="23.7" smashed="yes" rot="R90">
+<attribute name="NAME" x="16.7" y="26.238" size="0.8128" layer="25" font="vector" ratio="20" rot="R180" align="bottom-center"/>
 <attribute name="PROD_ID" value="RES-07856" x="16.7" y="23.7" size="1.778" layer="27" rot="R90" display="off"/>
+<attribute name="VALUE" x="16.7" y="22.038" size="0.8128" layer="21" font="vector" ratio="20" align="top-center"/>
 </element>
 </elements>
