File: Kirbi/v1 pcb/Kirbi_ControlBoard.brd (EAGLE design)
At the start: 66 x 56 mm, 72 parts, among them U1 PCA9306_LSSOP, U2 TEENSY_3.6_DIL, U3 MAX4173-SOT-23, U4 MAX4173-SOT-23, U5 LM393-8-SOIC, U6 AP2114H-1.8TRG1, U7 AP2114H-3.3TRG1

Commit message: NeoPixel for Kirbi/Fixed IMU
Added NeoPixel/Deleted IMU Interuppt/Tied IMU Address to Ground
Parts:
- added LED1: WS2812B5050, adafruit:WS2812B
- moved R20 24.0 mm to (36.0, 22.0)
- moved D3 23.3 mm to (36.0, 26.0), turned to 270 degrees
- turned C20 to 270 degrees
Connections:
- removed net 5V: C11.1, C12.1, C13.1, C24.1, C6.1, C7.1, C8.1, D2.A, ESC.P$3, LIDAR_L.P$1, LIDAR_R.P$1, U2.VIN, U5.P$8, U7.3
- removed net IMU_AD0: IMU.9, U2.9
- removed net IMU_INT: IMU.12, U2.12
- new net +5V: C11.1, C12.1, C13.1, C24.1, C6.1, C7.1, C8.1, D2.A, ESC.P$3, LED1.1-VDD, LIDAR_L.P$1, LIDAR_R.P$1, U2.VIN, U5.P$8, U7.3
- new net NEO_DI: LED1.4-DIN, U2.38/A19
- new net NEO_DO: LED1.2-DOUT, U2.39/A20
- net GND: now also IMU.9, LED1.3-GND
Routing:
- net NEO_DO: track 0.00 -> 22.1 mm
- net IMU_AD0: track 18.5 -> 0.00 mm, vias 1 -> 0
- net IMU_INT: track 17.0 -> 0.00 mm, vias 1 -> 0
- net +3.3V: track 138.6 -> 155.2 mm
- net NEO_DI: track 0.00 -> 16.5 mm
- net GND: track 140.9 -> 144.0 mm, vias 10 -> 12
- net 5V: track 2.12 -> 0.00 mm
- net +5V: track 0.00 -> 2.12 mm
- net RF_INT: track 9.74 -> 10.5 mm
- added copper zone on layer 1, net +5V
- removed copper zone on layer 1, net 5V

Commit message: Added Molex SMD Connectors (ESC and LIDAR)
Parts:
- ESC, LIDAR_L, LIDAR_R: value MOLEX_1.25MM_4PIN_90 -> MOLEX_1.25MM_4PIN_SMT; device Kirbi_ControlBoard:MOLEX_1.25MM_4PIN_90 -> Kirbi_ControlBoard:MOLEX_1.25MM_4PIN_SMT
- moved C12 3.00 mm to (10.0, 5.00)
- moved LIDAR_L 2.82 mm to (32.5, 1.70)
- moved C13 2.00 mm to (28.0, 5.00)
- moved LIDAR_R 1.84 mm to (5.60, 1.80)
- moved ESC 1.10 mm to (50.0, 37.4), flipped to the bottom, turned to 270 degrees
Connections:
- net +5V: now also ESC.P$4, LIDAR_L.P$6, LIDAR_R.P$6; no longer ESC.P$3, LIDAR_L.P$1, LIDAR_R.P$1
- net GND: now also ESC.P$3, LIDAR_L.P$3, LIDAR_R.P$3; no longer ESC.P$4, LIDAR_L.P$4, LIDAR_R.P$4
- net RX1: now also LIDAR_R.P$4; no longer LIDAR_R.P$3
- net RX2: now also LIDAR_L.P$4; no longer LIDAR_L.P$3
- net S1/TX: now also ESC.P$5; no longer ESC.P$2
- net S2: now also ESC.P$6; no longer ESC.P$1
- net TX1: now also LIDAR_R.P$5; no longer LIDAR_R.P$2
- net TX2: now also LIDAR_L.P$5; no longer LIDAR_L.P$2
Routing:
- net TX2: track 46.4 -> 11.4 mm
- net RX1: track 48.1 -> 13.4 mm
- net S2: track 17.1 -> 12.0 mm
- net TX1: track 42.4 -> 46.2 mm
- net GND: track 144.0 -> 140.7 mm
- net +5V: track 2.12 -> 4.66 mm, vias 0 -> 1
- net RX2: track 40.9 -> 42.1 mm

Commit message: Finished wiring Molex connectors/Cleaned up wiring
Parts:
- moved D2 1.00 mm to (1.00, 27.0)
- moved C15 0.10 mm to (13.0, 2.90)
- moved LIDAR_L 0.10 mm to (32.5, 1.80)
Routing:
- net TX2: track 11.4 -> 44.9 mm, vias 0 -> 1
- net RX1: track 13.4 -> 45.9 mm, vias 0 -> 1
- net TX1: track 46.2 -> 36.9 mm, vias 0 -> 1
- net GND: track 140.7 -> 132.2 mm, vias 12 -> 18
- net RX2: track 42.1 -> 34.4 mm, vias 0 -> 1
- net +3.3V: track 155.2 -> 147.6 mm
- net +5V: track 4.66 -> 2.22 mm
- net 24V: track 118.2 -> 116.5 mm
- net N$1: track 2.27 -> 3.27 mm
- net N$2: track 3.00 -> 2.27 mm

Commit message: Started to add power button
Parts:
- added R1: 50, SparkFun-Resistors:0603
- added U$5: POWER_SWITCH, Kirbi_ControlBoard:ELUMEESAQ7C12
- moved C7 18.3 mm to (25.9, 35.0), turned to 90 degrees
- moved C8 15.2 mm to (25.9, 38.8)
- moved C23 3.00 mm to (25.0, 42.0)
- moved U7 3.00 mm to (21.0, 39.0)
- moved C24 2.24 mm to (27.8, 41.1)
- moved C11 1.00 mm to (15.4, 39.0)
- moved ESC 0.81 mm to (49.6, 38.1)
Connections:
- new net N$5: U$5.P4
- new net N$8: R1.2, U$5.P1
- net +5V: now also U$5.P3, U$5.P5
- net GND: now also R1.1
Routing:
- net +3.3V: track 147.6 -> 151.6 mm
- net +5V: track 2.22 -> 0.00 mm, vias 1 -> 0
- net S1/TX: track 9.79 -> 8.22 mm
- net S2: track 11.6 -> 11.0 mm
- net GND: track 132.2 -> 132.3 mm, vias 18 -> 17

Commit message: Connected the power button to the ESC
Parts:
- moved R1 83.1 mm to (27.9, 37.4), turned to 90 degrees
- moved U$5 72.6 mm to (40.0, 38.0), turned to 180 degrees
Connections:
- removed net N$5: U$5.P4
- net +5V: no longer ESC.P$4
- net S2: now also U$5.P4
Routing:
- net S2: track 11.0 -> 16.3 mm, vias 0 -> 1
- net N$8: track 0.00 -> 5.07 mm
- net GND: track 132.3 -> 133.8 mm
- net S1/TX: track 8.22 -> 8.99 mm
Changed lines of the file:
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@@
 </element>
 <element name="ESC" library="Kirbi_ControlBoard" package="MOLEX_1.25MM_4PIN_SMT" value="MOLEX_1.25MM_4PIN_SMT" x="49.6" y="38.1" smashed="yes" rot="MR270">
-<attribute name="NAME" x="42.6" y="33.1" size="1.6" layer="25"/>
+<attribute name="NAME" x="41.5" y="32.9" size="1.6" layer="25"/>
 <attribute name="VALUE" x="53.6" y="42.1" size="1.6" layer="28" rot="MR270"/>
 </element>
@@
 <attribute name="VALUE" x="28.5" y="-2.2" size="1.6" layer="27"/>
 </element>
-<element name="U$5" library="Kirbi_ControlBoard" package="ELUMEESAQ7C12" value="POWER_SWITCH" x="-5" y="-19" smashed="yes">
-<attribute name="NAME" x="-12" y="-13" size="1.27" layer="25"/>
-<attribute name="VALUE" x="-12" y="-26.3" size="1.27" layer="27"/>
+<element name="U$5" library="Kirbi_ControlBoard" package="ELUMEESAQ7C12" value="POWER_SWITCH" x="40" y="38" smashed="yes" rot="R180">
+<attribute name="NAME" x="47" y="32" size="1.27" layer="25" rot="R180"/>
+<attribute name="VALUE" x="47" y="45.3" size="1.27" layer="27" rot="R180"/>
 </element>
-<element name="R1" library="SparkFun-Resistors" library_urn="urn:adsk.eagle:library:532" package="0603" package3d_urn="urn:adsk.eagle:package:39650/1" value="50" x="-22" y="-29" smashed="yes">
-<attribute name="NAME" x="-22" y="-28.238" size="0.6096" layer="25" font="vector" ratio="20" align="bottom-center"/>
-<attribute name="PROD_ID" value="RES-07856" x="-22" y="-29" size="1.778" layer="27" display="off"/>
-<attribute name="VALUE" x="-22" y="-29.762" size="0.6096" layer="27" font="vector" ratio="20" align="top-center"/>
+<element name="R1" library="SparkFun-Resistors" library_urn="urn:adsk.eagle:library:532" package="0603" package3d_urn="urn:adsk.eagle:package:39650/1" value="50" x="27.9" y="37.4" smashed="yes" rot="R90">
+<attribute name="NAME" x="27.138" y="37.4" size="0.6096" layer="25" font="vector" ratio="20" rot="R90" align="bottom-center"/>
+<attribute name="PROD_ID" value="RES-07856" x="27.9" y="37.4" size="1.778" layer="27" rot="R90" display="off"/>
+<attribute name="VALUE" x="28.662" y="37.4" size="0.6096" layer="27" font="vector" ratio="20" rot="R90" align="top-center"/>
 </element>
 </elements>
@@
 <wire x1="45.8" y1="49" x2="45" y2="49" width="0.2" layer="1"/>
 <via x="45" y="49" extent="1-16" drill="0.4"/>
-<wire x1="15.25" y1="38" x2="15.4" y2="38.15" width="0.2" layer="1"/>
 <wire x1="6.5" y1="42.15" x2="4.8" y2="40.45" width="0.2" layer="1"/>
 <wire x1="7.4" y1="36.495" x2="5.805" y2="36.495" width="0.2" layer="1"/>
@@
 <contactref element="R1" pad="1"/>
 <contactref element="ESC" pad="P$3"/>
-<wire x1="46.7" y1="39.975" x2="45" y2="49" width="0" layer="19" extent="16-16"/>
-<wire x1="29" y1="47.8" x2="45" y2="49" width="0" layer="19" extent="1-1"/>
-<wire x1="25.9" y1="37.95" x2="25.85" y2="42" width="0" layer="19" extent="1-1"/>
-<wire x1="19" y1="34" x2="25.9" y2="35.85" width="0" layer="19" extent="1-1"/>
-<wire x1="13.1" y1="43.8" x2="15.4" y2="38.15" width="0" layer="19" extent="1-1"/>
-<wire x1="6.5" y1="42.15" x2="12" y2="43.85" width="0" layer="19" extent="1-1"/>
-<wire x1="11.13" y1="54.27" x2="12" y2="43.85" width="0" layer="19" extent="1-1"/>
-<wire x1="25.1" y1="23.6" x2="27.4" y2="35.1" width="0" layer="19" extent="1-1"/>
-<wire x1="23.6" y1="19.455" x2="24.545" y2="22" width="0" layer="19" extent="1-1"/>
-<wire x1="22.8" y1="19.455" x2="23.6" y2="19.455" width="0" layer="19" extent="1-1"/>
-<wire x1="27.85" y1="14.7" x2="25" y2="17" width="0" layer="19" extent="1-1"/>
-<wire x1="29.73" y1="11.27" x2="27.85" y2="14.7" width="0" layer="19" extent="1-1"/>
-<wire x1="32.85" y1="14" x2="29.73" y2="11.27" width="0" layer="19" extent="1-1"/>
-<wire x1="28.85" y1="5" x2="29.73" y2="11.27" width="0" layer="19" extent="1-1"/>
-<wire x1="25" y1="3.85" x2="28.85" y2="5" width="0" layer="19" extent="1-1"/>
-<wire x1="18" y1="8" x2="20.96" y2="3" width="0" layer="19" extent="1-1"/>
-<wire x1="13" y1="5.1" x2="13.7" y2="10.05" width="0" layer="19" extent="1-1"/>
-<wire x1="3.725" y1="4.7" x2="10.85" y2="5" width="0" layer="19" extent="1-1"/>
-<wire x1="-3.203946875" y1="9" x2="2.3327625" y2="5.1944" width="0" layer="19" extent="1-1"/>
-<wire x1="-2.7" y1="13.7" x2="-6.79895625" y2="12.001040625" width="0" layer="19" extent="1-1"/>
-<wire x1="1.1" y1="15.6" x2="-3" y2="15.15" width="0" layer="19" extent="1-1"/>
-<wire x1="5.15" y1="14" x2="1.1" y2="15.6" width="0" layer="19" extent="1-1"/>
-<wire x1="-6.85" y1="20" x2="-3" y2="15.15" width="0" layer="19" extent="1-1"/>
-<wire x1="43" y1="10.79605" x2="37.15" y2="17" width="0" layer="19" extent="1-1"/>
-<wire x1="48.05" y1="17.5" x2="44.79895625" y2="12.101040625" width="0" layer="19" extent="1-1"/>
-<wire x1="-9.94" y1="30.38" x2="-9.73" y2="19.73" width="0" layer="19" extent="1-1"/>
-<wire x1="-8.15" y1="42" x2="-9.94" y2="30.38" width="0" layer="19" extent="1-1"/>
-<wire x1="-7.4" y1="45.62" x2="-7" y2="42" width="0" layer="19" extent="1-1"/>
-<wire x1="-22.85" y1="-29" x2="2.3327625" y2="5.1944" width="0" layer="19" extent="1-1"/>
+<wire x1="27.9" y1="36.55" x2="27.9" y2="35.6" width="0.2" layer="1"/>
+<wire x1="27.9" y1="35.6" x2="27.4" y2="35.1" width="0.2" layer="1"/>
 </signal>
 <signal name="+5V">
@@
 <contactref element="U$5" pad="P3"/>
 <contactref element="U$5" pad="P5"/>
-<contactref element="ESC" pad="P$4"/>
-<wire x1="46.7" y1="37.475" x2="49.65" y2="54.45" width="0" layer="19" extent="1-16"/>
-<wire x1="27.8" y1="40.25" x2="46.7" y2="37.475" width="0" layer="19" extent="1-16"/>
-<wire x1="25.9" y1="39.65" x2="27.8" y2="40.25" width="0" layer="19" extent="1-1"/>
-<wire x1="23.3" y1="35.975" x2="25.9" y2="39.65" width="0" layer="19" extent="1-1"/>
-<wire x1="25.9" y1="34.15" x2="23.3" y2="35.975" width="0" layer="19" extent="1-1"/>
-<wire x1="15.4" y1="39.85" x2="23.3" y2="35.975" width="0" layer="19" extent="1-1"/>
-<wire x1="12.8" y1="40.305" x2="15.4" y2="39.85" width="0" layer="19" extent="1-1"/>
-<wire x1="1" y1="27.877" x2="12.8" y2="40.305" width="0" layer="19" extent="1-1"/>
-<wire x1="-9.85" y1="42" x2="1" y2="27.877" width="0" layer="19" extent="1-1"/>
-<wire x1="-9.94" y1="45.62" x2="-9.85" y2="42" width="0" layer="19" extent="1-1"/>
-<wire x1="7.475" y1="4.7" x2="1" y2="27.877" width="0" layer="19" extent="1-1"/>
-<wire x1="9.15" y1="5" x2="7.475" y2="4.7" width="0" layer="19" extent="1-1"/>
-<wire x1="27.15" y1="5" x2="9.15" y2="5" width="0" layer="19" extent="1-1"/>
-<wire x1="34.375" y1="4.7" x2="27.15" y2="5" width="0" layer="19" extent="1-1"/>
-<wire x1="4.93" y1="-14.58" x2="7.475" y2="4.7" width="0" layer="19" extent="1-1"/>
-<wire x1="-14.93" y1="-23.42" x2="4.93" y2="-14.58" width="0" layer="19" extent="1-1"/>
 </signal>
 <signal name="+3.3V">
@@
 <contactref element="ESC" pad="P$5"/>
 <wire x1="46.603571875" y1="38.596428125" x2="46.7" y2="38.725" width="0.2" layer="16"/>
-<wire x1="45.5" y1="39.7" x2="45.5" y2="40" width="0.2" layer="16"/>
-<wire x1="45.5" y1="40" x2="45.5" y2="42.64" width="0.2" layer="16"/>
+<wire x1="45.5" y1="39.5" x2="45.5" y2="42.64" width="0.2" layer="16"/>
 <wire x1="45.5" y1="42.64" x2="48.48" y2="45.62" width="0.2" layer="16"/>
-<wire x1="45.5" y1="39.7" x2="45.5" y2="39.5" width="0.2" layer="16"/>
-<wire x1="45.5" y1="39.5" x2="46" y2="39" width="0.2" layer="16"/>
-<wire x1="46" y1="39" x2="46.603571875" y2="38.596428125" width="0" layer="19" extent="16-16"/>
+<wire x1="46.403571875" y1="38.596428125" x2="46.603571875" y2="38.596428125" width="0.2" layer="16"/>
+<wire x1="45.5" y1="39.5" x2="46.403571875" y2="38.596428125" width="0.2" layer="16"/>
 </signal>
 <signal name="S2">
 <contactref element="U2" pad="34/A15"/>
 <contactref element="ESC" pad="P$6"/>
-<wire x1="46.7" y1="36.225" x2="45.7" y2="36.225" width="0.2" layer="16"/>
-<wire x1="45.71824375" y1="36.28175625" x2="45.7" y2="36.225" width="0.2" layer="16"/>
 <wire x1="45.1" y1="44.78" x2="45.94" y2="45.62" width="0.2" layer="16"/>
-<wire x1="45.71824375" y1="36.28175625" x2="45.1" y2="36.9" width="0.2" layer="16"/>
-<wire x1="45.1" y1="36.9" x2="45.1" y2="44.78" width="0.2" layer="16"/>
+<wire x1="46.7" y1="36.225" x2="45.675" y2="36.225" width="0.2" layer="16"/>
+<wire x1="45.675" y1="36.225" x2="45.1" y2="36.8" width="0.2" layer="16"/>
+<wire x1="45.1" y1="36.8" x2="45.1" y2="44.78" width="0.2" layer="16"/>
+<contactref element="U$5" pad="P4"/>
+<wire x1="46.7" y1="36.225" x2="46.7" y2="34.6" width="0.2" layer="16"/>
+<via x="46.7" y="34.6" extent="1-16" drill="0.4"/>
+<wire x1="46.7" y1="34.6" x2="47.72" y2="33.58" width="0.2" layer="1"/>
+<wire x1="47.72" y1="33.58" x2="49.93" y2="33.58" width="0.2" layer="1"/>
 </signal>
 <signal name="SCL2">
@@
 <wire x1="35.78" y1="46.38" x2="35.78" y2="45.62" width="0.2" layer="1"/>
 </signal>
-<signal name="N$5">
-<contactref element="U$5" pad="P4"/>
-</signal>
 <signal name="N$8">
 <contactref element="U$5" pad="P1"/>
 <contactref element="R1" pad="2"/>
-<wire x1="4.93" y1="-23.42" x2="-21.15" y2="-29" width="0" layer="19" extent="1-1"/>
+<wire x1="30.07" y1="42.42" x2="30.07" y2="40.42" width="0.2" layer="1"/>
+<wire x1="30.07" y1="40.42" x2="27.9" y2="38.25" width="0.2" layer="1"/>
 </signal>
 </signals>

Commit message: Rearranged capacitors/Created 6 Pin SMD Connector Footprint
Parts:
- removed L_MOT, R_MOT: (no value), pinhead:1X02
- removed U3, U4: MAX4173-SOT-23, Gucci_ControlBoard:SOT-23
- moved R1 5.50 mm to (27.9, 42.9)
- moved C24 1.80 mm to (27.9, 39.3), turned to 270 degrees
- moved C8 0.40 mm to (25.9, 38.4)
- moved C7 0.30 mm to (25.9, 34.7)
Connections:
- removed net CURRENT_L: U2.A21, U4.P$6
- removed net CURRENT_R: U2.14/A0, U3.P$6
- removed net L_MOT+: L_MOT.2, U4.P$4
- removed net L_MOT-: L_MOT.1, U4.P$5
- removed net R_MOT+: R_MOT.2, U3.P$4
- removed net R_MOT-: R_MOT.1, U3.P$5
- net +3.3V: no longer U3.P$3, U4.P$3
- net GND: no longer U3.P$1, U3.P$2, U4.P$1, U4.P$2
Routing:
- net +3.3V: track 151.6 -> 135.0 mm, vias 2 -> 0
- net GND: track 133.8 -> 123.4 mm, vias 17 -> 18
- net R_MOT+: track 7.35 -> 0.00 mm
- net L_MOT-: track 7.33 -> 0.00 mm
- net CURRENT_L: track 6.53 -> 0.00 mm
- net CURRENT_R: track 6.12 -> 0.00 mm
- net L_MOT+: track 4.12 -> 0.00 mm
- net R_MOT-: track 4.10 -> 0.00 mm
- net N$8: track 5.07 -> 2.72 mm

Commit message: Moved LEDs and NeoPixel to bottom
Parts:
- moved LED1 27.3 mm to (39.8, 26.0), flipped to the bottom, turned to 180 degrees
- moved D3 16.1 mm to (20.0, 28.0), flipped to the bottom, turned to 180 degrees
- moved R19 15.2 mm to (15.0, 28.0), flipped to the bottom, turned to 180 degrees
- moved R18 15.1 mm to (6.20, 28.0), flipped to the bottom, turned to 180 degrees
- moved D4 14.4 mm to (28.5, 28.0), flipped to the bottom, turned to 180 degrees
- moved R21 14.2 mm to (32.0, 28.0), flipped to the bottom, turned to 180 degrees
- moved D1 13.5 mm to (1.90, 28.0), flipped to the bottom, turned to 180 degrees
- moved R20 13.4 mm to (24.0, 28.0), flipped to the bottom, turned to 180 degrees
- moved D2 10.0 mm to (11.0, 28.0), flipped to the bottom, turned to 180 degrees
Routing:
- net NEO_DO: track 22.1 -> 0.06 mm
- net 24V: track 116.5 -> 135.9 mm, vias 0 -> 1
- net NEO_DI: track 16.5 -> 0.00 mm
- net GND: track 123.4 -> 107.9 mm, vias 18 -> 19
- net +3.3V: track 135.0 -> 127.9 mm, vias 0 -> 1
- net +5V: track 0.00 -> 4.00 mm, vias 0 -> 1
- net LINE_LF: track 81.5 -> 83.7 mm
- net N$6: track 2.19 -> 4.27 mm
- net 1.8V: track 14.9 -> 16.1 mm, vias 0 -> 2
- net N$1: track 3.27 -> 2.27 mm
- net N$10: track 2.27 -> 1.77 mm

Commit message: Moved NeoPixel to the center
Parts:
- moved LED1 21.0 mm to (19.0, 23.0)
Connections:
- net NEO_DI: now also U2.11; no longer U2.38/A19
- net NEO_DO: no longer U2.39/A20
Routing:
- net NEO_DI: track 0.00 -> 7.77 mm
- net +5V: track 4.00 -> 8.00 mm, vias 1 -> 2
- net N$6: track 4.27 -> 2.57 mm
- net 24V: track 135.9 -> 134.9 mm
Changed lines of the file:
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@@
 <attribute name="VALUE" x="28" y="4.238" size="0.6096" layer="27" font="vector" ratio="20" align="top-center"/>
 </element>
-<element name="LED1" library="adafruit" library_urn="urn:adsk.eagle:library:420" package="WS2812B" package3d_urn="urn:adsk.eagle:package:6240942/1" value="WS2812B5050" x="39.8" y="26" smashed="yes" rot="MR180">
-<attribute name="NAME" x="36.2925" y="27.8125" size="0.8128" layer="26" ratio="10" rot="MR270"/>
+<element name="LED1" library="adafruit" library_urn="urn:adsk.eagle:library:420" package="WS2812B" package3d_urn="urn:adsk.eagle:package:6240942/1" value="WS2812B5050" x="19" y="23" smashed="yes" rot="MR180">
+<attribute name="NAME" x="15.4925" y="24.8125" size="0.8128" layer="26" ratio="10" rot="MR270"/>
 </element>
 <element name="ESC" library="Kirbi_ControlBoard" package="MOLEX_1.25MM_4PIN_SMT" value="MOLEX_1.25MM_4PIN_SMT" x="49.6" y="38.1" smashed="yes" rot="MR270">
@@
 <wire x1="12" y1="43.85" x2="12.05" y2="43.8" width="0.2" layer="1"/>
 <wire x1="1" y1="17.15" x2="0.85" y2="17" width="0.2" layer="1"/>
-<wire x1="25.030721875" y1="27.969278125" x2="24.85" y2="28" width="0.2" layer="16"/>
 <contactref element="LED1" pad="3-GND"/>
 <wire x1="6.5" y1="42.15" x2="4.8" y2="40.45" width="0.2" layer="1"/>
@@
 <via x="8.6" y="26.6" extent="1-16" drill="0.4"/>
 <wire x1="8.6" y1="26.6" x2="8.6" y2="28.5" width="0.2" layer="1"/>
-<wire x1="30.07" y1="33.58" x2="42.25" y2="27.65" width="0" layer="19" extent="1-16"/>
+<wire x1="21.45" y1="24.65" x2="21.8" y2="25" width="0.2" layer="16"/>
+<wire x1="21.8" y1="25" x2="21.8" y2="26.6444" width="0.2" layer="16"/>
+<via x="21.8" y="26.6444" extent="1-16" drill="0.4"/>
+<wire x1="21.8" y1="26.6444" x2="21.8" y2="28.5" width="0.2" layer="1"/>
 </signal>
 <signal name="+3.3V">
@@
 <contactref element="R17" pad="2"/>
 <contactref element="R13" pad="2"/>
-<wire x1="14.4" y1="24.55" x2="15.85" y2="26" width="0.2" layer="1"/>
-<wire x1="25.8" y1="26" x2="26.9" y2="27.1" width="0.2" layer="1"/>
-<wire x1="15.85" y1="26" x2="18" y2="26" width="0.2" layer="1"/>
-<wire x1="18.2" y1="26" x2="25.8" y2="26" width="0.2" layer="1"/>
+<wire x1="14.4" y1="24.55" x2="15.55" y2="25.7" width="0.2" layer="1"/>
+<wire x1="25.5" y1="25.7" x2="26.9" y2="27.1" width="0.2" layer="1"/>
+<wire x1="15.55" y1="25.7" x2="18" y2="25.7" width="0.2" layer="1"/>
+<wire x1="18" y1="25.7" x2="25.5" y2="25.7" width="0.2" layer="1"/>
 <wire x1="12" y1="24.55" x2="14.4" y2="24.55" width="0.2" layer="1"/>
 <contactref element="LINE_LF" pad="1"/>
@@
 <wire x1="31.15" y1="14" x2="30" y2="14" width="0.2" layer="1"/>
 <wire x1="30" y1="14" x2="29" y2="15" width="0.2" layer="1"/>
-<wire x1="19.123" y1="28" x2="19.123" y2="26.923" width="0.2" layer="16"/>
-<wire x1="19.123" y1="26.923" x2="18.8" y2="26.6" width="0.2" layer="16"/>
-<via x="18.8" y="26.6" extent="1-16" drill="0.4"/>
-<wire x1="18.8" y1="26.6" x2="18.2" y2="26" width="0.2" layer="1"/>
-<wire x1="18.2" y1="26" x2="18" y2="26" width="0.2" layer="1"/>
+<wire x1="19.123" y1="28" x2="19.123" y2="26.823" width="0.2" layer="16"/>
+<wire x1="19.123" y1="26.823" x2="18.7" y2="26.4" width="0.2" layer="16"/>
+<via x="18.7" y="26.4" extent="1-16" drill="0.4"/>
+<wire x1="18.7" y1="26.4" x2="18" y2="25.7" width="0.2" layer="1"/>
 <wire x1="27.123" y1="26.877" x2="19.123" y2="28" width="0" layer="19" extent="1-16"/>
 </signal>
@@
 <wire x1="-12.27" y1="19.73" x2="-12.27" y2="22.27" width="0.5" layer="16"/>
 <wire x1="-12.27" y1="19.73" x2="-11.95" y2="19.41" width="0.2" layer="1"/>
-<wire x1="-11.95" y1="17.6" x2="-11.1976" y2="16.8476" width="0.2" layer="1"/>
 <wire x1="50.27" y1="14.47395" x2="44.79605" y2="9" width="0.5" layer="16"/>
 <wire x1="50.27" y1="22.27" x2="50.27" y2="19.73" width="0.5" layer="16"/>
@@
 <contactref element="D1" pad="C"/>
 <contactref element="R18" pad="1"/>
-<wire x1="7.05" y1="28" x2="5.35" y2="28" width="0.1524" layer="16"/>
 <wire x1="2.777" y1="28" x2="5.35" y2="28" width="0.2" layer="16"/>
 </signal>
@@
 <signal name="NEO_DO">
 <contactref element="LED1" pad="2-DOUT"/>
-<contactref element="U2" pad="39/A20"/>
-<wire x1="33.24" y1="45.62" x2="33.2" y2="45.66" width="0.2" layer="1"/>
-<wire x1="42.25" y1="24.35" x2="33.24" y2="45.62" width="0" layer="19" extent="16-16"/>
 </signal>
 <signal name="NEO_DI">
 <contactref element="LED1" pad="4-DIN"/>
-<contactref element="U2" pad="38/A19"/>
-<wire x1="37.35" y1="27.65" x2="35.78" y2="45.62" width="0" layer="19" extent="16-16"/>
+<contactref element="U2" pad="11"/>
+<wire x1="16.55" y1="24.65" x2="17.5" y2="25.6" width="0.2" layer="16"/>
+<wire x1="17.5" y1="25.6" x2="17.5" y2="28" width="0.2" layer="16"/>
+<wire x1="17.5" y1="28" x2="19.88" y2="30.38" width="0.2" layer="16"/>
+<wire x1="19.88" y1="30.38" x2="20.54" y2="30.38" width="0.2" layer="16"/>
 </signal>
 <signal name="N$8">
