File: Kirbi/v1 pcb/Kirbi_ControlBoard.brd (EAGLE design)
At the start: 66 x 56 mm, 68 parts, among them U1 PCA9306_LSSOP, U2 TEENSY_3.6_DIL, U5 LM393-8-SOIC, U6 AP2114H-1.8TRG1, U7 AP2114H-3.3TRG1

Commit message: Moved Power Switch/Deleted 24 V parts
Moved power switch to left side of the board (moved around parts accordingly)
Deleted 24 V parts on Kirbi
Parts:
- removed C10, C4, C5, C9: 0.1uF, SparkFun-Capacitors:0603
- removed D1: 24V, SparkFun-LED:LED-0603
- removed R18: 11.15k, SparkFun-Resistors:0603
- moved POWER 42.6 mm to (-2.60, 38.0), turned to 0 degrees
- moved R1 13.9 mm to (15.8, 34.1), turned to 180 degrees
- moved C11 12.6 mm to (27.8, 41.1), turned to 90 degrees
- moved C6 12.2 mm to (4.00, 48.0), turned to 180 degrees
- moved C20 4.90 mm to (11.4, 43.0)
- moved U5 2.60 mm to (12.7, 38.3)
- moved C19 2.00 mm to (14.0, 43.0)
Connections:
- removed net N$6: D1.C, R18.1
- net 24V: no longer C10.1, C4.1, C5.1, C9.1, D1.A
- net GND: no longer C10.2, C4.2, C5.2, C9.2, R18.2
Routing:
- net 24V: track 92.9 -> 17.1 mm, vias 1 -> 0
- net GND: track 91.1 -> 71.5 mm, vias 20 -> 17
- net LF_INT: track 13.0 -> 20.1 mm
- net SCL2: track 14.9 -> 21.8 mm
- net N$8: track 2.46 -> 7.84 mm
- net S2: track 16.3 -> 11.0 mm, vias 1 -> 0
- net LINE_RF: track 53.4 -> 57.1 mm
- net SDA2: track 17.4 -> 21.0 mm
- net LINE_LF: track 84.2 -> 81.6 mm
- net N$6: track 2.27 -> 0.00 mm
- net LINE_REF: track 30.3 -> 29.1 mm

Commit message: Fixed MUXs and Centered LEDs
Connectted Tx (Connectors) to Rx (Teensi) and Rx (Connectors) to Tx (Teensi)
Parts:
- moved D2 4.50 mm to (8.00, 28.0)
- moved D3 4.50 mm to (17.0, 28.0)
- moved R19 4.50 mm to (12.0, 28.0)
- moved R20 4.50 mm to (21.0, 28.0)
- moved D4 4.00 mm to (26.0, 28.0)
- moved R21 4.00 mm to (30.0, 28.0)
Connections:
- net MUXS1: now also MUX_RX1.P$6, MUX_TX1.P$6; no longer MUX_RX1.P$4, MUX_TX1.P$4
- net MUXS2: now also MUX_RX2.P$6, MUX_TX2.P$6; no longer MUX_RX2.P$4, MUX_TX2.P$4
- net RXO1: now also MUX_TX1.P$4; no longer MUX_RX1.P$6
- net RXO2: now also MUX_TX2.P$4; no longer MUX_RX2.P$6
- net TXO1: now also MUX_RX1.P$4; no longer MUX_TX1.P$6
- net TXO2: now also MUX_RX2.P$4; no longer MUX_TX2.P$6
Routing:
- net NEO_DI: track 14.3 -> 17.9 mm
- net 1.8V: track 16.7 -> 13.5 mm
- net +3.3V: track 134.0 -> 130.9 mm
- net +5V: track 10.2 -> 7.73 mm
- net SDA2: track 21.0 -> 21.7 mm

Commit message: Finished Multiplexing
Changed schematic of multiplexer (Tx to Teensi TX etc.)/Wired on board
Parts:
- removed BATT: TE_02X01_3.96MM, Kirbi_ControlBoard:TE_02X01_3.96MM
- removed C15: 10uF, SparkFun-Capacitors:0603
- removed C16: 1uF, SparkFun-Capacitors:0603
- removed LIDAR_L, LIDAR_R: MOLEX_1.25MM_4PIN_SMT, Kirbi_ControlBoard:MOLEX_1.25MM_4PIN_SMT
- added DIST_5, DIST_6: MOLEX_1.25MM_4PIN_SMT, Kirbi_ControlBoard:MOLEX_1.25MM_4PIN_SMT
- R1: value 50 -> 1.65k
- moved DIST_3 40.2 mm to (5.60, 1.80), turned to 0 degrees
- moved DIST_4 26.7 mm to (32.5, 1.80), turned to 0 degrees
- moved TRANSCEIVER 9.00 mm to (39.0, 58.0)
- moved MUX_RX1 6.08 mm to (3.00, 18.0)
- moved MUX_RX2 6.08 mm to (35.0, 18.0)
- moved MUX_TX1 3.16 mm to (-2.00, 18.0)
- moved MUX_TX2 3.16 mm to (40.0, 18.0)
- moved R1 0.36 mm to (15.5, 33.9)
Connections:
- removed net +3V3: MUX_RX1.P$5, MUX_RX2.P$5, MUX_TX1.P$5, MUX_TX2.P$5, TRANSCEIVER.8
- removed net 24V: BATT.P$1, C15.1, C16.1
- removed net RX1: LIDAR_R.P$4, U2.0
- removed net RX2: LIDAR_L.P$4, U2.31/A12
- removed net RXO1: MUX_TX1.P$4, U2.9
- removed net RXO2: MUX_TX2.P$4, U2.7
- removed net TX1: LIDAR_R.P$5, U2.1
- removed net TX2: LIDAR_L.P$5, U2.32/A13
- removed net TXO1: MUX_RX1.P$4, U2.10
- removed net TXO2: MUX_RX2.P$4, U2.8
- new net RXD5: DIST_5.P$4, MUX_RX2.P$3
- new net RXD6: DIST_6.P$4, MUX_RX2.P$1
- new net TRX1: MUX_RX1.P$4, U2.7
- new net TRX2: MUX_RX2.P$4, U2.9
- new net TTX1: MUX_TX1.P$4, U2.8
- new net TTX2: MUX_TX2.P$4, U2.10
- new net TXD5: DIST_5.P$5, MUX_TX2.P$3
- new net TXD6: DIST_6.P$5, MUX_TX2.P$1
- net +3.3V: now also MUX_RX1.P$5, MUX_RX2.P$5, MUX_TX1.P$5, MUX_TX2.P$5, TRANSCEIVER.8
- net +5V: now also DIST_5.P$6, DIST_6.P$6; no longer LIDAR_L.P$6, LIDAR_R.P$6
- net GND: now also DIST_5.P$3, DIST_6.P$3; no longer BATT.P$2, C15.2, C16.2, ESC.P$3, LIDAR_L.P$3, LIDAR_R.P$3
- net MUXS1: now also U2.2; no longer U2.15/A1
- net MUXS2: now also U2.25; no longer U2.16/A2
- net RXD3: now also U2.0; no longer MUX_RX2.P$3
- net RXD4: now also U2.31/A12; no longer MUX_RX2.P$1
- net S2: no longer ESC.P$6
- net TXD3: now also U2.1; no longer MUX_TX2.P$3
- net TXD4: now also U2.32/A13; no longer MUX_TX2.P$1
Routing:
- net S2: track 11.0 -> 79.2 mm
- net RX1: track 45.9 -> 0.00 mm, vias 1 -> 0
- net TX2: track 44.9 -> 0.00 mm, vias 1 -> 0
- net RXD3: track 0.00 -> 43.4 mm, vias 0 -> 1
- net TXD4: track 0.00 -> 42.4 mm, vias 0 -> 1
- net TTX2: track 0.00 -> 39.2 mm, vias 0 -> 1
- net TX1: track 36.9 -> 0.00 mm, vias 1 -> 0
- net TXD3: track 0.00 -> 36.9 mm, vias 0 -> 1
- net RX2: track 34.4 -> 0.00 mm, vias 1 -> 0
- net RXD4: track 0.00 -> 32.9 mm, vias 0 -> 1
- net TRX2: track 0.00 -> 30.5 mm, vias 0 -> 1
- net MUXS2: track 0.00 -> 27.4 mm
- net RADIO_DIO0: track 25.7 -> 0.00 mm
- net TRX1: track 0.00 -> 25.7 mm
- net MOSI: track 24.2 -> 0.00 mm, vias 1 -> 0
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
Commit message: Deleted Traceiver Breakout Board/Wired Tranceiver Module
Added Radio Tranceiver Module and wired it on back of board
Parts:
- added C4: 0.1uF, SparkFun-Capacitors:0603
- TRANSCEIVER: device adafruit:1X08-BIG -> Kirbi_ControlBoard:RFMHCW_SMT
- moved TRANSCEIVER 52.0 mm to (19.0, 10.0), flipped to the bottom
Connections:
- net +3.3V: now also C4.1, TRANSCEIVER.5P; no longer TRANSCEIVER.8
- net GND: now also C4.2, TRANSCEIVER.16P, TRANSCEIVER.2P, TRANSCEIVER.9P; no longer TRANSCEIVER.7
- net MISO: now also TRANSCEIVER.10P; no longer TRANSCEIVER.1
- net MOSI: now also TRANSCEIVER.11P; no longer TRANSCEIVER.2
- net RADIO_DIO0: now also TRANSCEIVER.6P, U2.5; no longer TRANSCEIVER.6, U2.14/A0
- net RADIO_NSS: now also TRANSCEIVER.13P; no longer TRANSCEIVER.4
- net RADIO_SCK: now also TRANSCEIVER.12P; no longer TRANSCEIVER.3
Routing:
- net RADIO_SCK: track 0.00 -> 75.9 mm
- net MOSI: track 0.00 -> 36.0 mm, vias 0 -> 1
- net MISO: track 0.00 -> 34.6 mm, vias 0 -> 1
- net RADIO_NSS: track 0.00 -> 31.6 mm, vias 0 -> 1
- net RADIO_DIO0: track 0.00 -> 31.0 mm
- net +3.3V: track 154.3 -> 164.7 mm
- net S2: track 79.2 -> 70.0 mm
- net LINE_REF: track 29.0 -> 25.0 mm
- net TXD4: track 42.4 -> 44.9 mm
- net RXD3: track 43.4 -> 45.9 mm
- net RXD4: track 32.9 -> 34.4 mm
- net LINE_LF: track 81.6 -> 80.9 mm

Commit message: Fixed Wiring/Added Antenna
Added through hole Antenna for radio tranceiver.
Parts:
- added JP1: (no value), pinhead:1X01
- moved C4 11.5 mm to (8.30, 5.90), turned to 270 degrees
Connections:
- removed net S2: POWER.P4, U2.34/A15
- new net N$5: JP1.1, TRANSCEIVER.1P
Routing:
- net S2: track 70.0 -> 0.00 mm
- net N$5: track 0.00 -> 13.6 mm
- net LINE_LF: track 80.9 -> 74.6 mm
- net LINE_RF: track 57.1 -> 62.4 mm, vias 1 -> 0
- net +3.3V: track 164.7 -> 162.2 mm
- net RXD3: track 45.9 -> 46.8 mm

Commit message: Decoupling Capacitors/Wiring/Moved Antenna
Added decoupling capacitors distance sensors
Re-routed some of the multiplexers
Moved Antenna to bottom of the board
Parts:
- removed U$2: (no value), RoboJackets-Aesthetics:ROBOBUZZ_1.4X
- added C10, C15, C16, C25, C5, C9: 0.1uF, SparkFun-Capacitors:0603
- moved JP1 20.4 mm to (19.0, 2.10)
- moved TRANSCEIVER 2.00 mm to (19.0, 12.0)
Connections:
- net +5V: now also C10.1, C15.1, C16.1, C25.1, C5.1, C9.1
- net GND: now also C10.2, C15.2, C16.2, C25.2, C5.2, C9.2
Routing:
- net +5V: track 8.83 -> 43.6 mm
- net TTX1: track 23.4 -> 41.8 mm, vias 1 -> 2
- net TTX2: track 39.3 -> 54.2 mm
- net TRX2: track 30.0 -> 43.7 mm
- net RADIO_DIO0: track 31.0 -> 17.7 mm
- net GND: track 84.9 -> 97.2 mm, vias 23 -> 27
- net N$5: track 13.6 -> 9.30 mm
- net RADIO_SCK: track 76.0 -> 78.0 mm
- net MOSI: track 36.0 -> 35.2 mm
- net RADIO_NSS: track 31.6 -> 30.8 mm
- net MISO: track 34.6 -> 33.7 mm
- net +3.3V: track 162.2 -> 163.0 mm
- net TXD6: track 13.6 -> 13.1 mm

Commit message: Re-routed Multiplexer/Fixed Airwires
Re-routed some pins on
the multiplexer/Fixed Airwires
Routing:
- net TTX2: track 54.2 -> 32.5 mm
- net TTX1: track 41.8 -> 24.5 mm, vias 2 -> 1
- net TRX2: track 43.7 -> 37.4 mm
- net 1.8V: track 13.4 -> 18.3 mm
- net MISO: track 33.7 -> 37.3 mm
- net TRX1: track 25.5 -> 22.1 mm, vias 0 -> 1
- net MUXS2: track 27.4 -> 26.0 mm
- net +3.3V: track 163.0 -> 162.1 mm

Commit message: Cleaned up ground plane
Cleaned up ground plane (moved wires to the edge and out of the transceiver) /changed radio_nss to pin 34
Parts:
- moved C5 0.30 mm to (46.2, 16.7)
Connections:
- net RADIO_NSS: now also U2.34/A15; no longer U2.6
Routing:
- net +5V: track 43.6 -> 16.1 mm
- net RADIO_NSS: track 30.8 -> 54.8 mm, vias 1 -> 0
- net LINE_RF: track 62.1 -> 80.3 mm
- net MISO: track 37.3 -> 19.7 mm
- net MOSI: track 35.2 -> 22.3 mm
- net TXD3: track 36.9 -> 43.5 mm
- net LINE_LF: track 74.6 -> 71.1 mm
- net GND: track 97.0 -> 94.6 mm, vias 27 -> 30
- net TRX1: track 22.1 -> 20.7 mm
- net +3.3V: track 162.1 -> 162.9 mm
- net 1.8V: track 18.3 -> 18.1 mm, vias 2 -> 1
