File: Kirbi/v1 pcb/Kirbi_ControlBoard.brd (EAGLE design)
At the start: 66 x 56 mm, 66 parts, among them U1 PCA9306_LSSOP, U2 TEENSY_3.6_DIL, U5 LM393-8-SOIC, U6 AP2114H-1.8TRG1, U7 AP2114H-3.3TRG1

Commit message: Cleaned up silk screen
Cleaned up silk screen/Moved neo pixel up/transceiver down/etc.
Parts:
- moved U$3 2.00 mm to (40.0, 21.0)
- moved U$4 2.00 mm to (-2.00, 21.0)
- moved LED1 0.61 mm to (18.9, 23.6)
- moved TRANSCEIVER 0.20 mm to (19.0, 11.8)
- moved JP1 0.10 mm to (19.0, 2.00)
Routing:
- net +5V: track 16.1 -> 17.1 mm
- net GND: track 88.8 -> 89.7 mm
- net +3.3V: track 158.7 -> 157.8 mm

Commit message: small tweaks
moved a few routes and components
fixed wire stub issue
fixed some of the silkscreen
Parts:
- moved C14 2.30 mm to (15.3, 52.9)
- moved C2 1.49 mm to (27.1, 19.9), turned to 0 degrees
- moved DIST_3 0.30 mm to (5.60, 2.10)
- moved DIST_4 0.30 mm to (32.5, 2.10)
- moved START 0.30 mm to (19.0, 52.7)
- moved C25 0.20 mm to (37.0, 5.10)
- moved C12 0.10 mm to (10.0, 5.10)
Routing:
- net +5V: track 17.1 -> 37.7 mm
- net GND: track 89.7 -> 76.7 mm, vias 35 -> 37
- net RF_INT: track 15.9 -> 13.3 mm
- net LF_INT: track 14.3 -> 12.7 mm
- net LINE_RF: track 80.1 -> 78.7 mm, vias 0 -> 1
- net +3.3V: track 157.8 -> 156.4 mm

Commit message: Fixed fonts/silk screen/Changed resistor values
Fixed fonts: vectorized
Changed resistor values: for LEDs and power button
Re-centered LED on bottom of the board
Parts:
- removed R21: 50, SparkFun-Resistors:0603
- R1: value 1.65k -> 100
- R19: value 1.65k -> 200
- R20: value 800 -> 100
- moved D4 3.00 mm to (29.0, 28.0)
- moved R20 3.00 mm to (24.0, 28.0)
- moved D3 2.00 mm to (19.0, 28.0)
- moved R19 2.00 mm to (14.0, 28.0)
- moved D2 1.00 mm to (9.00, 28.0)
Connections:
- removed net N$10: D4.C, R21.1
- net GND: now also D4.C; no longer R21.2
Routing:
- net +5V: track 37.7 -> 35.0 mm
- net 1.8V: track 18.1 -> 20.4 mm
- net N$10: track 2.27 -> 0.00 mm
- net +3.3V: track 156.4 -> 157.9 mm
- net N$2: track 2.27 -> 3.27 mm
- net N$1: track 2.27 -> 3.27 mm
- net NEO_DI: track 13.8 -> 14.8 mm
- net TTX1: track 24.5 -> 25.0 mm

Commit message: Connected ESCs
Connectted ESCs (Added two multiplexers to Gucci/Changed RADIO_NSS to Pin 30)
Parts:
- ESC: value MOLEX_1.25MM_4PIN_SMT -> MOLEX_1.25MM_3PIN_SMT; device Kirbi_ControlBoard:MOLEX_1.25MM_4PIN_SMT -> Kirbi_ControlBoard:MOLEX_1.25MM_3PIN_SMT
- moved ESC 1.20 mm to (48.4, 38.0)
Connections:
- removed net S1/TX: ESC.P$5, U2.33/A14
- new net S1/TRX: ESC.P$2, U2.34/A15
- new net S1/TTX: ESC.P$1, U2.33/A14
- net GND: now also ESC.P$3
- net RADIO_NSS: now also U2.30; no longer U2.34/A15
Routing:
- net RADIO_NSS: track 54.9 -> 39.8 mm
- net S1/TX: track 8.99 -> 0.00 mm
- net S1/TRX: track 0.00 -> 8.75 mm
- net S1/TTX: track 0.00 -> 6.98 mm
Changed lines of the file:
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@@
 <drawing>
 <settings>
-<setting alwaysvectorfont="yes"/>
+<setting alwaysvectorfont="no"/>
 <setting verticaltext="up"/>
 </settings>
@@
 <attribute name="VALUE" x="27.3" y="27.735" size="0.8128" layer="22" font="vector" ratio="20" rot="MR90" align="top-center"/>
 </element>
-<element name="ESC" library="Kirbi_ControlBoard" package="MOLEX_1.25MM_4PIN_SMT" value="MOLEX_1.25MM_4PIN_SMT" x="49.6" y="38.1" smashed="yes" rot="MR270">
-<attribute name="NAME" x="45.6" y="33" size="1.6" layer="26" font="vector" rot="MR0"/>
-<attribute name="VALUE" x="53.6" y="42.1" size="1.6" layer="28" rot="MR270"/>
-</element>
 <element name="DIST_3" library="Kirbi_ControlBoard" package="MOLEX_1.25MM_4PIN_SMT" value="MOLEX_1.25MM_4PIN_SMT" x="5.6" y="2.1" smashed="yes">
 <attribute name="NAME" x="13.9" y="0.5" size="1.6" layer="25" font="vector" rot="R90"/>
@@
 <attribute name="PROD_ID" value="CAP-00810" x="10" y="5.1" size="1.778" layer="27" display="off"/>
 <attribute name="VALUE" x="10" y="4.338" size="0.6096" layer="27" font="vector" ratio="20" align="top-center"/>
+</element>
+<element name="ESC" library="Kirbi_ControlBoard" package="MOLEX_1.25MM_3PIN_SMT" value="MOLEX_1.25MM_3PIN_SMT" x="48.4" y="38" smashed="yes" rot="MR270">
+<attribute name="NAME" x="45.4" y="43" size="1.778" layer="26" font="vector" rot="MR270"/>
+<attribute name="VALUE" x="54.4" y="43" size="1.778" layer="28" font="vector" rot="MR270"/>
 </element>
 </elements>
@@
 <via x="25.4" y="22.4" extent="1-16" drill="0.4"/>
 <contactref element="D4" pad="C"/>
+<contactref element="ESC" pad="P$3"/>
 </signal>
 <signal name="+5V">
@@
 <wire x1="12.335" y1="37.665" x2="11.065" y2="38.935" width="0.2" layer="1"/>
 </signal>
-<signal name="S1/TX">
-<contactref element="U2" pad="33/A14"/>
-<contactref element="ESC" pad="P$5"/>
-<wire x1="46.603571875" y1="38.596428125" x2="46.7" y2="38.725" width="0.2" layer="16"/>
-<wire x1="45.5" y1="39.5" x2="45.5" y2="42.64" width="0.2" layer="16"/>
-<wire x1="45.5" y1="42.64" x2="48.48" y2="45.62" width="0.2" layer="16"/>
-<wire x1="46.403571875" y1="38.596428125" x2="46.603571875" y2="38.596428125" width="0.2" layer="16"/>
-<wire x1="45.5" y1="39.5" x2="46.403571875" y2="38.596428125" width="0.2" layer="16"/>
-</signal>
 <signal name="SCL2">
 <contactref element="R16" pad="1"/>
@@
 <signal name="RADIO_NSS">
 <contactref element="TRANSCEIVER" pad="13P"/>
-<contactref element="U2" pad="34/A15"/>
 <wire x1="27.1" y1="10.8" x2="28.6156" y2="9.4844" width="0.2" layer="16"/>
 <wire x1="28.6156" y1="9.4844" x2="28.6156" y2="8.00981875" width="0.2" layer="16"/>
@@
 <wire x1="45.2066" y1="16.0066" x2="45.2066" y2="27.3" width="0.2" layer="16"/>
 <via x="45.2066" y="27.3" extent="1-16" drill="0.4"/>
-<wire x1="45.2066" y1="27.3" x2="44.751" y2="27.7556" width="0.2" layer="1"/>
-<wire x1="44.751" y1="44.431" x2="45.94" y2="45.62" width="0.2" layer="1"/>
 <wire x1="35.7" y1="6.5" x2="45.2066" y2="16.0066" width="0.2" layer="16"/>
-<wire x1="44.751" y1="27.7556" x2="44.751" y2="44.431" width="0.2" layer="1"/>
+<contactref element="U2" pad="30"/>
+<wire x1="45.2066" y1="27.3" x2="43.4" y2="29.1066" width="0.2" layer="1"/>
+<wire x1="43.4" y1="29.1066" x2="43.4" y2="30.38" width="0.2" layer="1"/>
 </signal>
 <signal name="RADIO_DIO0">
@@
 <wire x1="-10.95" y1="44" x2="-12.53" y2="42.42" width="0.6" layer="1"/>
 </signal>
+<signal name="S1/TTX">
+<contactref element="U2" pad="33/A14"/>
+<contactref element="ESC" pad="P$1"/>
+<wire x1="47" y1="39.25" x2="47" y2="44.14" width="0.2" layer="16"/>
+<wire x1="47" y1="44.14" x2="48.48" y2="45.62" width="0.2" layer="16"/>
+</signal>
+<signal name="S1/TRX">
+<contactref element="U2" pad="34/A15"/>
+<contactref element="ESC" pad="P$2"/>
+<wire x1="45.94" y1="45.62" x2="45.74" y2="45.42" width="0.2" layer="16"/>
+<wire x1="45.74" y1="45.42" x2="45.74" y2="38.36" width="0.2" layer="16"/>
+<wire x1="45.74" y1="38.36" x2="46.1" y2="38" width="0.2" layer="16"/>
+<wire x1="46.1" y1="38" x2="47" y2="38" width="0.2" layer="16"/>
+</signal>
 </signals>

Commit message: Fixed Silkscreen/Fuse/Added Resistor
Fixed Silkscreen/Fuse (Added label)/Added Resistor (6.2 OHM to 1.8 LED)
Parts:
- removed U$2: BEL_FUSE_C1F_3.5, Kirbi_ControlBoard:BEL_FUSE_C1F_3.5
- added F1: 3.5, Kirbi_ControlBoard:BEL_FUSE_C1F_3.5
- added R2: 6.2, Kirbi_ControlBoard:0603
- moved D4 3.00 mm to (26.0, 28.0)
- moved R20 3.00 mm to (21.0, 28.0)
- moved D3 2.00 mm to (17.0, 28.0)
- moved R19 2.00 mm to (12.0, 28.0)
- moved D2 1.00 mm to (8.00, 28.0)
Connections:
- new net N$9: D4.C, R2.1
- net GND: now also R2.2; no longer D4.C
- net N$6: now also F1.P$2; no longer U$2.P$2
- net N$7: now also F1.P$1; no longer U$2.P$1
Routing:
- net N$6: track 23.4 -> 27.8 mm
- net GND: track 76.6 -> 79.8 mm
- net 1.8V: track 20.4 -> 18.1 mm
- net N$9: track 0.00 -> 2.27 mm
- net LINE_RF: track 78.7 -> 81.0 mm
- net +3.3V: track 157.9 -> 156.3 mm
- net RF_INT: track 13.3 -> 14.7 mm
- net N$2: track 3.27 -> 2.27 mm
- net N$1: track 3.27 -> 2.27 mm
- net N$7: track 6.76 -> 7.63 mm
- net +5V: track 35.0 -> 34.3 mm
- net SDA1: track 10.4 -> 9.75 mm

Commit message: Added Pull-up Resistors/Moved MUXs
Added Pull-up Resistors (1k OHM to RX line)
Added 6.2 OHM to 1.8 V LED
Moved MUXs and rerouted
Fixed SIlkscreen
Parts:
- added R3, R4: 1k, SparkFun-Resistors:0603
- moved R1 0.50 mm to (10.4, 34.0)
Connections:
- net +3.3V: now also R3.2, R4.2
- net TRX1: now also R4.1
- net TRX2: now also R3.1
Routing:
- net +3.3V: track 156.3 -> 168.7 mm
- net TRX2: track 37.3 -> 41.5 mm
- net TRX1: track 20.7 -> 22.9 mm
Changed lines of the file:
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@@
 </element>
 <element name="U5" library="Gucci_ControlBoard" package="8-SOIC" value="LM393-8-SOIC" x="12.7" y="38.3" smashed="yes">
-<attribute name="NAME" x="14.7" y="35.6" size="1" layer="25" font="vector" rot="R180"/>
+<attribute name="NAME" x="16.4" y="41.6" size="1" layer="25" font="vector" rot="R180"/>
 <attribute name="VALUE" x="10.7" y="34.5" size="1" layer="27"/>
 </element>
@@
 </element>
 <element name="C19" library="SparkFun-Capacitors" library_urn="urn:adsk.eagle:library:510" package="0603" package3d_urn="urn:adsk.eagle:package:37414/1" value="15pF" x="14" y="43" smashed="yes" rot="R90">
-<attribute name="NAME" x="15.738" y="42.9" size="0.8128" layer="25" font="vector" ratio="20" rot="R270" align="bottom-center"/>
+<attribute name="NAME" x="15.738" y="43" size="0.8128" layer="25" font="vector" ratio="20" rot="R270" align="bottom-center"/>
 <attribute name="PROD_ID" value="CAP-00810" x="14" y="43" size="1.778" layer="27" rot="R90" display="off"/>
 <attribute name="VALUE" x="14.762" y="43" size="0.6096" layer="27" font="vector" ratio="20" rot="R90" align="top-center"/>
@@
 <attribute name="NAME" x="22.3925" y="22.0125" size="0.8128" layer="26" font="vector" ratio="10" rot="MR90"/>
 </element>
-<element name="R1" library="SparkFun-Resistors" library_urn="urn:adsk.eagle:library:532" package="0603" package3d_urn="urn:adsk.eagle:package:39650/1" value="100" x="10.4" y="33.5" smashed="yes" rot="R180">
-<attribute name="NAME" x="9.8" y="35.238" size="0.8128" layer="25" font="vector" ratio="20" rot="R180" align="bottom-center"/>
-<attribute name="PROD_ID" value="RES-12438" x="10.4" y="33.5" size="1.778" layer="27" rot="R180" display="off"/>
-<attribute name="VALUE" value="100" x="10.4" y="34.262" size="0.6096" layer="27" font="vector" ratio="20" rot="R180" align="top-center"/>
+<element name="R1" library="SparkFun-Resistors" library_urn="urn:adsk.eagle:library:532" package="0603" package3d_urn="urn:adsk.eagle:package:39650/1" value="100" x="10.4" y="34" smashed="yes" rot="R180">
+<attribute name="NAME" x="9.4" y="35.638" size="0.8128" layer="25" font="vector" ratio="20" rot="R180" align="bottom-center"/>
+<attribute name="PROD_ID" value="RES-12438" x="10.4" y="34" size="1.778" layer="27" rot="R180" display="off"/>
+<attribute name="VALUE" value="100" x="10.4" y="34.762" size="0.6096" layer="27" font="vector" ratio="20" rot="R180" align="top-center"/>
 </element>
 <element name="MUX_TX1" library="Kirbi_ControlBoard" package="MUX_74LVC1G157GV" value="MUX_74LVC1G157GV" x="-2" y="18" smashed="yes">
@@
 </element>
 <element name="F1" library="Kirbi_ControlBoard" package="BEL_FUSE_C1F_3.5" value="3.5" x="8.8" y="35.1" smashed="yes" rot="MR180">
-<attribute name="NAME" x="12.852" y="36.095" size="1.778" layer="26" font="vector" rot="MR180"/>
+<attribute name="NAME" x="5.752" y="37.595" size="1.016" layer="26" font="vector" rot="MR180"/>
 <attribute name="VALUE" x="5.879" y="38.656" size="1.778" layer="28" font="vector" rot="MR180"/>
 </element>
 <element name="R2" library="Kirbi_ControlBoard" package="0603" package3d_urn="urn:adsk.eagle:package:39650/1" value="6.2" x="30" y="28" smashed="yes" rot="MR180">
-<attribute name="NAME" x="30" y="27.238" size="0.6096" layer="26" font="vector" ratio="20" rot="MR180" align="bottom-center"/>
+<attribute name="NAME" x="30" y="27.238" size="0.8128" layer="26" font="vector" ratio="20" rot="MR180" align="bottom-center"/>
 <attribute name="PROD_ID" value="P6.2GCT-ND" x="30" y="28" size="1.778" layer="28" rot="MR180" display="off"/>
 <attribute name="VALUE" x="30" y="28.762" size="0.6096" layer="28" font="vector" ratio="20" rot="MR180" align="top-center"/>
+</element>
+<element name="R3" library="SparkFun-Resistors" library_urn="urn:adsk.eagle:library:532" package="0603" package3d_urn="urn:adsk.eagle:package:39650/1" value="1k" x="14.9" y="34" smashed="yes">
+<attribute name="NAME" x="17.438" y="34" size="0.8128" layer="25" font="vector" ratio="20" rot="R90" align="bottom-center"/>
+<attribute name="PROD_ID" value="RES-07856" x="14.9" y="34" size="1.778" layer="27" display="off"/>
+<attribute name="VALUE" x="14.9" y="33.238" size="0.6096" layer="27" font="vector" ratio="20" align="top-center"/>
+</element>
+<element name="R4" library="SparkFun-Resistors" library_urn="urn:adsk.eagle:library:532" package="0603" package3d_urn="urn:adsk.eagle:package:39650/1" value="1k" x="10.3" y="32.2" smashed="yes">
+<attribute name="NAME" x="12.838" y="32.2" size="0.8128" layer="25" font="vector" ratio="20" rot="R90" align="bottom-center"/>
+<attribute name="PROD_ID" value="RES-07856" x="10.3" y="32.2" size="1.778" layer="27" display="off"/>
+<attribute name="VALUE" x="10.3" y="31.438" size="0.6096" layer="27" font="vector" ratio="20" align="top-center"/>
 </element>
 </elements>
@@
 <wire x1="30.625" y1="3.375" x2="30.8" y2="3.2" width="0.2" layer="1"/>
 <via x="30.8" y="3.2" extent="1-16" drill="0.4"/>
-<wire x1="18.7" y1="35.975" x2="18.7" y2="34.7" width="0.2" layer="1"/>
-<wire x1="18.7" y1="34.7" x2="18" y2="34" width="0.2" layer="1"/>
-<via x="18" y="34" extent="1-16" drill="0.4"/>
+<wire x1="18.7" y1="35.975" x2="18.7" y2="34.4" width="0.2" layer="1"/>
+<wire x1="18.7" y1="34.4" x2="18.3" y2="34" width="0.2" layer="1"/>
+<via x="18.3" y="34" extent="1-16" drill="0.4"/>
 <contactref element="DIST_2" pad="P$3"/>
 <contactref element="DIST_5" pad="P$3"/>
@@
 <via x="10.1" y="42.5" extent="1-16" drill="0.4"/>
 <contactref element="POWER_CONN" pad="P$2"/>
-<wire x1="11.25" y1="33.5" x2="12.8" y2="33.5" width="0.2" layer="1"/>
-<wire x1="12.8" y1="33.5" x2="12.9" y2="33.4" width="0.2" layer="1"/>
-<via x="12.9" y="33.4" extent="1-16" drill="0.4"/>
+<via x="12.6" y="33.9" extent="1-16" drill="0.4"/>
 <wire x1="23.6" y1="23.2" x2="23.9" y2="23.5" width="0.2" layer="1"/>
 <wire x1="23.9" y1="23.5" x2="24.8" y2="23.5" width="0.2" layer="1"/>
@@
 <contactref element="ESC" pad="P$3"/>
 <contactref element="R2" pad="2"/>
+<wire x1="11.25" y1="34" x2="12.5" y2="34" width="0.2" layer="1"/>
+<wire x1="12.5" y1="34" x2="12.6" y2="33.9" width="0.2" layer="1"/>
 </signal>
 <signal name="+5V">
@@
 <wire x1="21.4" y1="27.6" x2="19.301" y2="29.699" width="0.5" layer="1"/>
 <wire x1="19.301" y1="34.276" x2="21" y2="35.975" width="0.5" layer="1"/>
-<wire x1="19.301" y1="29.699" x2="19.301" y2="34.276" width="0.5" layer="1"/>
+<wire x1="19.301" y1="29.699" x2="19.301" y2="32" width="0.5" layer="1"/>
+<wire x1="19.301" y1="32" x2="19.301" y2="34.276" width="0.5" layer="1"/>
 <wire x1="15.425" y1="25.575" x2="22.575" y2="25.575" width="0.2" layer="1"/>
 <wire x1="22.575" y1="25.575" x2="24.1" y2="27.1" width="0.2" layer="1"/>
@@
 <wire x1="16.123" y1="28" x2="14.8" y2="26.677" width="0.2" layer="16"/>
 <wire x1="14.8" y1="26.677" x2="14.8" y2="26" width="0.2" layer="16"/>
+<contactref element="R3" pad="2"/>
+<contactref element="R4" pad="2"/>
+<wire x1="15.75" y1="34" x2="17.301" y2="34" width="0.2" layer="1"/>
+<wire x1="17.301" y1="34" x2="19.301" y2="32" width="0.2" layer="1"/>
+<wire x1="11.15" y1="32.2" x2="11.669" y2="31.681" width="0.2" layer="1"/>
+<wire x1="11.669" y1="31.681" x2="11.669" y2="24.881" width="0.2" layer="1"/>
+<wire x1="11.669" y1="24.881" x2="12" y2="24.55" width="0.2" layer="1"/>
 </signal>
 <signal name="LINE_LF">
@@
 <contactref element="R1" pad="2"/>
 <wire x1="9.47" y1="33.58" x2="7.33" y2="33.58" width="0.2" layer="1"/>
-<wire x1="9.55" y1="33.5" x2="9.47" y2="33.58" width="0.2" layer="1"/>
+<wire x1="9.55" y1="34" x2="9.47" y2="33.58" width="0.2" layer="1"/>
 </signal>
 <signal name="MISO">
@@
 <wire x1="3.1" y1="26.2" x2="5.077" y2="24.223" width="0.2" layer="1"/>
 <wire x1="5.077" y1="24.223" x2="5.077" y2="20.42251875" width="0.2" layer="1"/>
+<contactref element="R4" pad="1"/>
+<wire x1="9.45" y1="32.2" x2="10.38" y2="31.27" width="0.2" layer="1"/>
+<wire x1="10.38" y1="31.27" x2="10.38" y2="30.38" width="0.2" layer="1"/>
 </signal>
 <signal name="TXD6">
@@
 <wire x1="37.1" y1="31.7" x2="35.8" y2="33" width="0.2" layer="16"/>
 <wire x1="35.8" y1="33" x2="18" y2="33" width="0.2" layer="16"/>
+<contactref element="R3" pad="1"/>
+<wire x1="14.05" y1="34" x2="14.05" y2="31.79" width="0.2" layer="1"/>
+<wire x1="14.05" y1="31.79" x2="15.46" y2="30.38" width="0.2" layer="1"/>
 </signal>
 <signal name="TTX1">
