File: Kirbi/v1 pcb/Kirbi_ControlBoard.sch (EAGLE design)
At the start: 71 parts, among them U1 PCA9306_LSSOP, U2 TEENSY_3.6_DIL, U3 MAX4173-SOT-23, U4 MAX4173-SOT-23, U5 LM393-8-SOIC, U6 AP2114H-1.8TRG1, U7 AP2114H-3.3TRG1

Commit message: Rearranged capacitors/Created 6 Pin SMD Connector Footprint
Parts:
- removed L_MOT, R_MOT: (no value), pinhead:PINHD-1X2
- removed U3, U4: MAX4173-SOT-23, Gucci_ControlBoard:MAX4173-SOT-23
Connections:
- removed net CURRENT_L: U2.A21/DAC0, U4.OUT
- removed net CURRENT_R: U2.14/A0/PWM, U3.OUT
- removed net L_MOT+: L_MOT.2, U4.RS+
- removed net L_MOT-: L_MOT.1, U4.RS-
- removed net R_MOT+: R_MOT.2, U3.RS+
- removed net R_MOT-: R_MOT.1, U3.RS-
- net +3.3V: no longer U3.VCC, U4.VCC
- net GND: no longer U3.GND, U4.GND
Other:
- note removed: "Current Sensing"
Changed lines of the file:
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@@
 <part name="GND12" library="SparkFun-PowerSymbols" library_urn="urn:adsk.eagle:library:530" deviceset="GND" device=""/>
 <part name="+3V6" library="supply1" library_urn="urn:adsk.eagle:library:371" deviceset="+3V3" device=""/>
-<part name="U4" library="Gucci_ControlBoard" deviceset="MAX4173-SOT-23" device=""/>
-<part name="U3" library="Gucci_ControlBoard" deviceset="MAX4173-SOT-23" device=""/>
-<part name="GND13" library="SparkFun-PowerSymbols" library_urn="urn:adsk.eagle:library:530" deviceset="GND" device=""/>
-<part name="GND15" library="SparkFun-PowerSymbols" library_urn="urn:adsk.eagle:library:530" deviceset="GND" device=""/>
-<part name="L_MOT" library="pinhead" library_urn="urn:adsk.eagle:library:325" deviceset="PINHD-1X2" device="" package3d_urn="urn:adsk.eagle:package:22435/2"/>
-<part name="R_MOT" library="pinhead" library_urn="urn:adsk.eagle:library:325" deviceset="PINHD-1X2" device="" package3d_urn="urn:adsk.eagle:package:22435/2"/>
 <part name="D4" library="SparkFun-LED" deviceset="LED" device="0603" value="1.8V"/>
 <part name="D1" library="SparkFun-LED" deviceset="LED" device="0603" value="24V"/>
@@
 <part name="C12" library="SparkFun-Capacitors" library_urn="urn:adsk.eagle:library:510" deviceset="0.1UF" device="-0603-25V-(+80/-20%)" package3d_urn="urn:adsk.eagle:package:37414/1" value="0.1uF"/>
 <part name="C13" library="SparkFun-Capacitors" library_urn="urn:adsk.eagle:library:510" deviceset="0.1UF" device="-0603-25V-(+80/-20%)" package3d_urn="urn:adsk.eagle:package:37414/1" value="0.1uF"/>
-<part name="+3V11" library="supply1" library_urn="urn:adsk.eagle:library:371" deviceset="+3V3" device=""/>
-<part name="+3V12" library="supply1" library_urn="urn:adsk.eagle:library:371" deviceset="+3V3" device=""/>
 <part name="LED1" library="adafruit" library_urn="urn:adsk.eagle:library:420" deviceset="WS2812B" device="5050" package3d_urn="urn:adsk.eagle:package:6240942/1"/>
 <part name="GND18" library="supply1" library_urn="urn:adsk.eagle:library:371" deviceset="GND" device=""/>
@@
 <text x="266.7" y="111.76" size="5.08" layer="97">Battery Connector</text>
 <wire x1="190.5" y1="127" x2="190.5" y2="78.74" width="1.27" layer="97" style="shortdash"/>
-<text x="185.42" y="71.12" size="5.08" layer="97">Current Sensing</text>
 <text x="312.42" y="157.48" size="5.08" layer="97">Power</text>
 </plain>
@@
 <attribute name="VALUE" x="193.04" y="104.14" size="1.778" layer="96" rot="R90"/>
 </instance>
-<instance part="U4" gate="G$1" x="193.04" y="53.34" smashed="yes">
-<attribute name="NAME" x="182.88" y="60.96" size="2.54" layer="95"/>
-<attribute name="VALUE" x="182.88" y="43.18" size="2.54" layer="96"/>
-</instance>
-<instance part="U3" gate="G$1" x="233.68" y="53.34" smashed="yes">
-<attribute name="NAME" x="223.52" y="60.96" size="2.54" layer="95"/>
-<attribute name="VALUE" x="223.52" y="43.18" size="2.54" layer="96"/>
-</instance>
-<instance part="GND13" gate="1" x="193.04" y="38.1" smashed="yes">
-<attribute name="VALUE" x="193.04" y="37.846" size="1.778" layer="96" align="top-center"/>
-</instance>
-<instance part="GND15" gate="1" x="233.68" y="38.1" smashed="yes">
-<attribute name="VALUE" x="233.68" y="37.846" size="1.778" layer="96" align="top-center"/>
-</instance>
-<instance part="L_MOT" gate="G$1" x="190.5" y="30.48" smashed="yes" rot="R180">
-<attribute name="NAME" x="196.85" y="24.765" size="1.778" layer="95" rot="R180"/>
-<attribute name="VALUE" x="196.85" y="35.56" size="1.778" layer="96" rot="R180"/>
-</instance>
-<instance part="R_MOT" gate="G$1" x="231.14" y="30.48" smashed="yes" rot="R180">
-<attribute name="NAME" x="237.49" y="24.765" size="1.778" layer="95" rot="R180"/>
-<attribute name="VALUE" x="237.49" y="35.56" size="1.778" layer="96" rot="R180"/>
-</instance>
 <instance part="D4" gate="G$1" x="274.32" y="27.94" smashed="yes" rot="R90">
 <attribute name="NAME" x="278.892" y="24.511" size="1.778" layer="95" font="vector" rot="R180"/>
@@
 <attribute name="NAME" x="367.284" y="61.341" size="1.778" layer="95" font="vector"/>
 <attribute name="VALUE" x="367.284" y="56.261" size="1.778" layer="96" font="vector"/>
-</instance>
-<instance part="+3V11" gate="G$1" x="193.04" y="68.58" smashed="yes">
-<attribute name="VALUE" x="190.5" y="63.5" size="1.778" layer="96" rot="R90"/>
-</instance>
-<instance part="+3V12" gate="G$1" x="233.68" y="68.58" smashed="yes">
-<attribute name="VALUE" x="231.14" y="63.5" size="1.778" layer="96" rot="R90"/>
 </instance>
 <instance part="LED1" gate="G$1" x="281.94" y="198.12" smashed="yes"/>
@@
 <wire x1="195.58" y1="100.33" x2="195.58" y2="106.68" width="0.1524" layer="91"/>
 <pinref part="+3V6" gate="G$1" pin="+3V3"/>
-</segment>
-<segment>
-<pinref part="+3V11" gate="G$1" pin="+3V3"/>
-<pinref part="U4" gate="G$1" pin="VCC"/>
-</segment>
-<segment>
-<pinref part="+3V12" gate="G$1" pin="+3V3"/>
-<pinref part="U3" gate="G$1" pin="VCC"/>
 </segment>
 </net>
@@
 </segment>
 <segment>
-<pinref part="U4" gate="G$1" pin="GND"/>
-<pinref part="GND13" gate="1" pin="GND"/>
-</segment>
-<segment>
-<pinref part="U3" gate="G$1" pin="GND"/>
-<pinref part="GND15" gate="1" pin="GND"/>
-</segment>
-<segment>
 <pinref part="R18" gate="G$1" pin="2"/>
 <wire x1="299.72" y1="60.96" x2="304.8" y2="60.96" width="0.1524" layer="91"/>
@@
 <pinref part="U$5" gate="G$1" pin="P3"/>
 <wire x1="297.18" y1="160.02" x2="297.18" y2="154.94" width="0.1524" layer="91"/>
-<pinref part="U$5" gate="G$1" pin="P5"/>
-<wire x1="297.18" y1="154.94" x2="297.18" y2="142.24" width="0.1524" layer="91"/>
-<wire x1="297.18" y1="142.24" x2="292.1" y2="142.24" width="0.1524" layer="91"/>
+<wire x1="297.18" y1="154.94" x2="297.18" y2="147.32" width="0.1524" layer="91"/>
 <junction x="297.18" y="154.94"/>
 <junction x="297.18" y="160.02"/>
 <wire x1="309.88" y1="142.24" x2="309.88" y2="160.02" width="0.1524" layer="91"/>
 <wire x1="309.88" y1="160.02" x2="297.18" y2="160.02" width="0.1524" layer="91"/>
+<wire x1="297.18" y1="147.32" x2="292.1" y2="147.32" width="0.1524" layer="91"/>
+<pinref part="U$5" gate="G$1" pin="P5"/>
+<wire x1="292.1" y1="147.32" x2="292.1" y2="142.24" width="0.1524" layer="91"/>
 </segment>
 <segment>
@@
 <net name="S2" class="0">
 <segment>
-<wire x1="266.7" y1="139.7" x2="271.78" y2="139.7" width="0.1524" layer="91"/>
-<label x="271.78" y="139.7" size="1.778" layer="95" xref="yes"/>
 <pinref part="ESC" gate="G$1" pin="4"/>
 <pinref part="U$5" gate="G$1" pin="P4"/>
 <wire x1="287.02" y1="154.94" x2="266.7" y2="154.94" width="0.1524" layer="91"/>
 <wire x1="266.7" y1="154.94" x2="266.7" y2="139.7" width="0.1524" layer="91"/>
-<junction x="266.7" y="139.7"/>
 </segment>
 <segment>
@@
 </segment>
 </net>
-<net name="L_MOT+" class="0">
-<segment>
-<pinref part="U4" gate="G$1" pin="RS+"/>
-<wire x1="177.8" y1="55.88" x2="175.26" y2="55.88" width="0.1524" layer="91"/>
-<label x="175.26" y="55.88" size="1.778" layer="95" rot="R90" xref="yes"/>
-</segment>
-<segment>
-<pinref part="L_MOT" gate="G$1" pin="2"/>
-<wire x1="193.04" y1="30.48" x2="198.12" y2="30.48" width="0.1524" layer="91"/>
-<label x="198.12" y="30.48" size="1.778" layer="95" xref="yes"/>
-</segment>
-</net>
-<net name="L_MOT-" class="0">
-<segment>
-<pinref part="U4" gate="G$1" pin="RS-"/>
-<wire x1="177.8" y1="50.8" x2="175.26" y2="50.8" width="0.1524" layer="91"/>
-<label x="175.26" y="50.8" size="1.778" layer="95" rot="R270" xref="yes"/>
-</segment>
-<segment>
-<pinref part="L_MOT" gate="G$1" pin="1"/>
-<wire x1="193.04" y1="27.94" x2="198.12" y2="27.94" width="0.1524" layer="91"/>
-<label x="198.12" y="27.94" size="1.778" layer="95" xref="yes"/>
-</segment>
-</net>
-<net name="CURRENT_L" class="0">
-<segment>
-<pinref part="U4" gate="G$1" pin="OUT"/>
-<wire x1="208.28" y1="53.34" x2="210.82" y2="53.34" width="0.1524" layer="91"/>
-<label x="210.82" y="53.34" size="1.778" layer="95" rot="R90" xref="yes"/>
-</segment>
-<segment>
-<pinref part="U2" gate="G$1" pin="A21/DAC0"/>
-<wire x1="218.44" y1="185.42" x2="223.52" y2="185.42" width="0.1524" layer="91"/>
-<label x="223.52" y="185.42" size="1.778" layer="95" xref="yes"/>
-</segment>
-</net>
-<net name="R_MOT+" class="0">
-<segment>
-<pinref part="U3" gate="G$1" pin="RS+"/>
-<wire x1="218.44" y1="55.88" x2="215.9" y2="55.88" width="0.1524" layer="91"/>
-<label x="215.9" y="55.88" size="1.778" layer="95" rot="R90" xref="yes"/>
-</segment>
-<segment>
-<pinref part="R_MOT" gate="G$1" pin="2"/>
-<wire x1="233.68" y1="30.48" x2="238.76" y2="30.48" width="0.1524" layer="91"/>
-<label x="238.76" y="30.48" size="1.778" layer="95" xref="yes"/>
-</segment>
-</net>
-<net name="R_MOT-" class="0">
-<segment>
-<pinref part="U3" gate="G$1" pin="RS-"/>
-<wire x1="218.44" y1="50.8" x2="215.9" y2="50.8" width="0.1524" layer="91"/>
-<label x="215.9" y="50.8" size="1.778" layer="95" rot="R270" xref="yes"/>
-</segment>
-<segment>
-<pinref part="R_MOT" gate="G$1" pin="1"/>
-<wire x1="233.68" y1="27.94" x2="238.76" y2="27.94" width="0.1524" layer="91"/>
-<label x="238.76" y="27.94" size="1.778" layer="95" xref="yes"/>
-</segment>
-</net>
-<net name="CURRENT_R" class="0">
-<segment>
-<pinref part="U3" gate="G$1" pin="OUT"/>
-<wire x1="248.92" y1="53.34" x2="251.46" y2="53.34" width="0.1524" layer="91"/>
-<label x="251.46" y="53.34" size="1.778" layer="95" rot="R90" xref="yes"/>
-</segment>
-<segment>
-<label x="160.02" y="200.66" size="1.778" layer="95" rot="R180" xref="yes"/>
-<pinref part="U2" gate="G$1" pin="14/A0/PWM"/>
-<wire x1="165.1" y1="200.66" x2="160.02" y2="200.66" width="0.1524" layer="91"/>
-</segment>
-</net>

Commit message: Moved NeoPixel to the center
Connections:
- net NEO_DI: now also U2.11/MOSI0; no longer U2.38/A19/SDA1/PWM
- net NEO_DO: no longer U2.39/A20
Changed lines of the file:
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@@
 <label x="297.18" y="195.58" size="1.778" layer="95" xref="yes"/>
-</segment>
-<segment>
-<pinref part="U2" gate="G$1" pin="39/A20"/>
-<wire x1="165.1" y1="137.16" x2="162.56" y2="137.16" width="0.1524" layer="91"/>
-<label x="162.56" y="137.16" size="1.778" layer="95" rot="R180" xref="yes"/>
 </segment>
 </net>
@@
 </segment>
 <segment>
-<pinref part="U2" gate="G$1" pin="38/A19/SDA1/PWM"/>
-<wire x1="165.1" y1="139.7" x2="162.56" y2="139.7" width="0.1524" layer="91"/>
-<label x="162.56" y="139.7" size="1.778" layer="95" rot="R180" xref="yes"/>
+<label x="160.02" y="208.28" size="1.778" layer="95" rot="R180" xref="yes"/>
+<pinref part="U2" gate="G$1" pin="11/MOSI0"/>
+<wire x1="160.02" y1="208.28" x2="165.1" y2="208.28" width="0.1524" layer="91"/>
 </segment>
 </net>

Commit message: Removed NeoPixel DO Connector
Connections:
- removed net NEO_DO: LED1.DO
Changed lines of the file:
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@@
-</segment>
-</net>
-<net name="NEO_DO" class="0">
-<segment>
-<pinref part="LED1" gate="G$1" pin="DO"/>
-<wire x1="294.64" y1="195.58" x2="297.18" y2="195.58" width="0.1524" layer="91"/>
-<label x="297.18" y="195.58" size="1.778" layer="95" xref="yes"/>
 </segment>
 </net>

Commit message: Style Guide Adjustments
Parts:
- renumbered U$5 to POWER
Changed lines of the file:
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@@
 <part name="LIDAR_R" library="Kirbi_ControlBoard" deviceset="MOLEX_1.25MM_4PIN_SMT" device=""/>
 <part name="LIDAR_L" library="Kirbi_ControlBoard" deviceset="MOLEX_1.25MM_4PIN_SMT" device=""/>
-<part name="U$5" library="Kirbi_ControlBoard" deviceset="POWER_SWITCH" device=""/>
+<part name="POWER" library="Kirbi_ControlBoard" deviceset="POWER_SWITCH" device=""/>
 <part name="P+3" library="supply1" library_urn="urn:adsk.eagle:library:371" deviceset="+5V" device=""/>
 <part name="R1" library="SparkFun-Resistors" library_urn="urn:adsk.eagle:library:532" deviceset="1KOHM" device="-0603-1/10W-1%" package3d_urn="urn:adsk.eagle:package:39650/1" value="50"/>
@@
 <attribute name="NAME" x="66.04" y="236.728" size="1.778" layer="95" font="vector"/>
 </instance>
-<instance part="U$5" gate="G$1" x="297.18" y="149.86" smashed="yes">
+<instance part="POWER" gate="G$1" x="297.18" y="149.86" smashed="yes">
 <attribute name="NAME" x="294.64" y="149.86" size="1.27" layer="97"/>
 </instance>
@@
 <junction x="317.5" y="142.24"/>
 <pinref part="P+3" gate="1" pin="+5V"/>
-<pinref part="U$5" gate="G$1" pin="P3"/>
+<pinref part="POWER" gate="G$1" pin="P3"/>
 <wire x1="297.18" y1="160.02" x2="297.18" y2="154.94" width="0.1524" layer="91"/>
 <wire x1="297.18" y1="154.94" x2="297.18" y2="147.32" width="0.1524" layer="91"/>
@@
 <wire x1="309.88" y1="160.02" x2="297.18" y2="160.02" width="0.1524" layer="91"/>
 <wire x1="297.18" y1="147.32" x2="292.1" y2="147.32" width="0.1524" layer="91"/>
-<pinref part="U$5" gate="G$1" pin="P5"/>
+<pinref part="POWER" gate="G$1" pin="P5"/>
 <wire x1="292.1" y1="147.32" x2="292.1" y2="142.24" width="0.1524" layer="91"/>
 </segment>
@@
 <segment>
 <pinref part="ESC" gate="G$1" pin="4"/>
-<pinref part="U$5" gate="G$1" pin="P4"/>
+<pinref part="POWER" gate="G$1" pin="P4"/>
 <wire x1="287.02" y1="154.94" x2="266.7" y2="154.94" width="0.1524" layer="91"/>
 <wire x1="266.7" y1="154.94" x2="266.7" y2="139.7" width="0.1524" layer="91"/>
@@
 <net name="N$8" class="0">
 <segment>
-<pinref part="U$5" gate="G$1" pin="P1"/>
+<pinref part="POWER" gate="G$1" pin="P1"/>
 <pinref part="R1" gate="G$1" pin="2"/>
 <wire x1="304.8" y1="139.7" x2="304.8" y2="142.24" width="0.1524" layer="91"/>

Commit message: Wired Radio Tranceiver to Teensi
Added a pin header and connected to respective pins on Teensi/Changed NeoPixel pin to Pin 24
Parts:
- added TRANSCEIVER: (no value), adafruit:PINHD-1X8BIG
Connections:
- new net +3V3: TRANSCEIVER.8
- new net DIO0: TRANSCEIVER.6, U2.14/A0/PWM
- new net MISO: TRANSCEIVER.1, U2.12/MISO0
- new net MOSI: TRANSCEIVER.2, U2.11/MOSI0
- new net NSS: TRANSCEIVER.4, U2.10/TX2/PWM
- new net SCK: TRANSCEIVER.3, U2.13/SCK0/LED
- net GND: now also TRANSCEIVER.7
- net NEO_DI: now also U2.24; no longer U2.11/MOSI0
Changed lines of the file:
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@@
 <part name="P+3" library="supply1" library_urn="urn:adsk.eagle:library:371" deviceset="+5V" device=""/>
 <part name="R1" library="SparkFun-Resistors" library_urn="urn:adsk.eagle:library:532" deviceset="1KOHM" device="-0603-1/10W-1%" package3d_urn="urn:adsk.eagle:package:39650/1" value="50"/>
+<part name="TRANSCEIVER" library="adafruit" library_urn="urn:adsk.eagle:library:420" deviceset="PINHD-1X8" device="BIG" package3d_urn="urn:adsk.eagle:package:6240707/1"/>
+<part name="GND13" library="supply1" library_urn="urn:adsk.eagle:library:371" deviceset="GND" device=""/>
+<part name="+3V11" library="supply1" library_urn="urn:adsk.eagle:library:371" deviceset="+3V3" device=""/>
 </parts>
 <sheets>
@@
 <attribute name="VALUE" x="306.324" y="134.62" size="1.778" layer="96" font="vector" rot="R90" align="top-center"/>
 </instance>
+<instance part="TRANSCEIVER" gate="G$1" x="322.58" y="200.66" smashed="yes">
+<attribute name="NAME" x="316.23" y="212.217" size="1.778" layer="95"/>
+<attribute name="VALUE" x="316.23" y="185.42" size="1.778" layer="96"/>
+</instance>
+<instance part="GND13" gate="1" x="302.26" y="185.42" smashed="yes">
+<attribute name="VALUE" x="299.72" y="182.88" size="1.778" layer="96"/>
+</instance>
+<instance part="+3V11" gate="G$1" x="309.88" y="193.04" smashed="yes">
+<attribute name="VALUE" x="307.34" y="187.96" size="1.778" layer="96" rot="R90"/>
+</instance>
 </instances>
 <busses>
@@
 <junction x="340.36" y="142.24"/>
 </segment>
+<segment>
+<pinref part="GND13" gate="1" pin="GND"/>
+<pinref part="TRANSCEIVER" gate="G$1" pin="7"/>
+<wire x1="302.26" y1="187.96" x2="302.26" y2="193.04" width="0.1524" layer="91"/>
+<wire x1="302.26" y1="193.04" x2="320.04" y2="193.04" width="0.1524" layer="91"/>
+</segment>
 </net>
 <net name="LINE_LF" class="0">
@@
 </segment>
 <segment>
-<label x="160.02" y="208.28" size="1.778" layer="95" rot="R180" xref="yes"/>
-<pinref part="U2" gate="G$1" pin="11/MOSI0"/>
-<wire x1="160.02" y1="208.28" x2="165.1" y2="208.28" width="0.1524" layer="91"/>
+<label x="160.02" y="175.26" size="1.778" layer="95" rot="R180" xref="yes"/>
+<pinref part="U2" gate="G$1" pin="24"/>
+<wire x1="165.1" y1="175.26" x2="160.02" y2="175.26" width="0.1524" layer="91"/>
 </segment>
 </net>
@@
 </segment>
 </net>
+<net name="MISO" class="0">
+<segment>
+<label x="314.96" y="208.28" size="1.778" layer="95" rot="R180" xref="yes"/>
+<pinref part="TRANSCEIVER" gate="G$1" pin="1"/>
+<wire x1="320.04" y1="208.28" x2="314.96" y2="208.28" width="0.1524" layer="91"/>
+</segment>
+<segment>
+<pinref part="U2" gate="G$1" pin="12/MISO0"/>
+<wire x1="165.1" y1="205.74" x2="160.02" y2="205.74" width="0.1524" layer="91"/>
+<label x="160.02" y="205.74" size="1.778" layer="95" rot="R180" xref="yes"/>
+</segment>
+</net>
+<net name="MOSI" class="0">
+<segment>
+<label x="314.96" y="205.74" size="1.778" layer="95" rot="R180" xref="yes"/>
+<pinref part="TRANSCEIVER" gate="G$1" pin="2"/>
+<wire x1="320.04" y1="205.74" x2="314.96" y2="205.74" width="0.1524" layer="91"/>
+</segment>
+<segment>
+<pinref part="U2" gate="G$1" pin="11/MOSI0"/>
+<wire x1="165.1" y1="208.28" x2="160.02" y2="208.28" width="0.1524" layer="91"/>
+<label x="160.02" y="208.28" size="1.778" layer="95" rot="R180" xref="yes"/>
+</segment>
+</net>
+<net name="SCK" class="0">
+<segment>
+<label x="314.96" y="203.2" size="1.778" layer="95" rot="R180" xref="yes"/>
+<pinref part="TRANSCEIVER" gate="G$1" pin="3"/>
+<wire x1="320.04" y1="203.2" x2="314.96" y2="203.2" width="0.1524" layer="91"/>
+</segment>
+<segment>
+<label x="160.02" y="203.2" size="1.778" layer="95" rot="R180" xref="yes"/>
+<pinref part="U2" gate="G$1" pin="13/SCK0/LED"/>
+<wire x1="165.1" y1="203.2" x2="160.02" y2="203.2" width="0.1524" layer="91"/>
+</segment>
+</net>
+<net name="+3V3" class="0">
+<segment>
+<pinref part="+3V11" gate="G$1" pin="+3V3"/>
+<pinref part="TRANSCEIVER" gate="G$1" pin="8"/>
+<wire x1="309.88" y1="190.5" x2="320.04" y2="190.5" width="0.1524" layer="91"/>
+</segment>
+</net>
+<net name="NSS" class="0">
+<segment>
+<pinref part="U2" gate="G$1" pin="10/TX2/PWM"/>
+<wire x1="165.1" y1="210.82" x2="160.02" y2="210.82" width="0.1524" layer="91"/>
+<label x="160.02" y="210.82" size="1.778" layer="95" rot="R180" xref="yes"/>
+</segment>
+<segment>
+<pinref part="TRANSCEIVER" gate="G$1" pin="4"/>
+<wire x1="320.04" y1="200.66" x2="314.96" y2="200.66" width="0.1524" layer="91"/>
+<label x="314.96" y="200.66" size="1.778" layer="95" rot="R180" xref="yes"/>
+</segment>
+</net>
+<net name="DIO0" class="0">
+<segment>
+<pinref part="U2" gate="G$1" pin="14/A0/PWM"/>
+<wire x1="165.1" y1="200.66" x2="160.02" y2="200.66" width="0.1524" layer="91"/>
+<label x="160.02" y="200.66" size="1.778" layer="95" rot="R180" xref="yes"/>
+</segment>
+<segment>
+<pinref part="TRANSCEIVER" gate="G$1" pin="6"/>
+<wire x1="320.04" y1="195.58" x2="314.96" y2="195.58" width="0.1524" layer="91"/>
+<label x="314.96" y="195.58" size="1.778" layer="95" rot="R180" xref="yes"/>
+</segment>
+</net>
