File: Kirbi/v1 pcb/Kirbi_ControlBoard.sch (EAGLE design)
At the start: 68 parts, among them U1 PCA9306_LSSOP, U2 TEENSY_3.6_DIL, U5 LM393-8-SOIC, U6 AP2114H-1.8TRG1, U7 AP2114H-3.3TRG1

Commit message: Replace Omiron Sensors/Fixed Wiring
Replaced the Omiron Distance Sensors (Still need to add multiplexers to wire to Teensi)
Fixed some wiring and naming of the radio transciever.
Parts:
- removed R22, R26, R28, R30: 6.98k, SparkFun-Resistors:1KOHM-0603-1/10W-1%
- removed R23, R27, R29, R31: 1k, SparkFun-Resistors:1KOHM-0603-1/10W-1%
- DIST_1, DIST_2, DIST_3, DIST_4: value AMPHENOL_2X02_2.54MM_SHROUD -> MOLEX_1.25MM_4PIN_SMT; device Gucci_ControlBoard:AMPHENOL_2X02_2.54MM_SHROUD -> Kirbi_ControlBoard:MOLEX_1.25MM_4PIN_SMT
Connections:
- net DIO0 renamed RADIO_DIO0
- net NSS renamed RADIO_NSS
- net SCK renamed RADIO_SCK
- removed net N$11: DIST_3.3, R26.2
- removed net N$12: DIST_2.3, R30.2
- removed net N$7: DIST_1.3, R28.2
- removed net N$9: DIST_4.3, R22.2
- net +5V: now also DIST_1.4, DIST_2.4, DIST_3.4, DIST_4.4
- net 24V: no longer DIST_1.2, DIST_1.4, DIST_2.2, DIST_2.4, DIST_3.2, DIST_3.4, DIST_4.2, DIST_4.4
- net DIST_L: no longer R22.1, R23.2
- net DIST_L_45: no longer R26.1, R27.2
- net DIST_R: no longer R28.1, R29.2
- net DIST_R_45: no longer R30.1, R31.2
- net GND: no longer R23.1, R27.1, R29.1, R31.1
- net RX1: now also DIST_1.2, DIST_2.2, DIST_3.2, DIST_4.2
- net TX1: now also DIST_1.3, DIST_2.3, DIST_3.3, DIST_4.3
Other:
- note removed: "Omron Distance Sensors"
- moved on the sheet: DIST_1, DIST_2, DIST_3, DIST_4

Commit message: Added MUX Distance Sensors
Added MUX Distance Sensors on the Schematic/Changed SCL2/SDA2/RADIO_NSS Pins on Teensi
Parts:
- added MUX_RX1, MUX_RX2, MUX_TX1, MUX_TX2: MUX_74LVC1G157GV, Kirbi_ControlBoard:MUX_74LVC1G157GV
Connections:
- removed net DIST_L: U2.30/T/PWM
- removed net DIST_L_45: U2.28
- removed net DIST_R: U2.2/PWM
- removed net DIST_R_45: U2.3/CAN0-TX/SCL2/PWM
- new net MUXS1: MUX_RX1.P$3, MUX_TX1.P$3, U2.15/A1/T
- new net MUXS2: MUX_RX2.P$3, MUX_TX2.P$3, U2.16/A2/T/PWM
- new net RXD1: DIST_1.2, MUX_RX1.P$1
- new net RXD2: DIST_2.2, MUX_RX1.P$2
- new net RXD3: DIST_3.2, MUX_RX2.P$1
- new net RXD4: DIST_4.2, MUX_RX2.P$2
- new net RXO1: MUX_RX1.P$4, U2.9/RX2/PWM
- new net RXO2: MUX_RX2.P$4, U2.7/RX3/PWM
- new net TXD1: DIST_1.3, MUX_TX1.P$1
- new net TXD2: DIST_2.3, MUX_TX1.P$2
- new net TXD3: DIST_3.3, MUX_TX2.P$1
- new net TXD4: DIST_4.3, MUX_TX2.P$2
- new net TXO1: MUX_TX1.P$4, U2.10/TX2/PWM
- new net TXO2: MUX_TX2.P$4, U2.8/TX3/PWM
- net +3V3: now also MUX_RX1.P$6, MUX_RX2.P$6, MUX_TX1.P$6, MUX_TX2.P$6
- net GND: now also MUX_RX1.P$5, MUX_RX2.P$5, MUX_TX1.P$5, MUX_TX2.P$5
- net RADIO_NSS: now also U2.6/PWM; no longer U2.10/TX2/PWM
- net RX1: no longer DIST_1.2, DIST_2.2, DIST_3.2, DIST_4.2
- net SCL2: now also U2.3/CAN0-TX/SCL2/PWM; no longer U2.7/RX3/PWM
- net SDA2: now also U2.4/CAN0-RX/SDA2/PWM; no longer U2.8/TX3/PWM
- net TX1: no longer DIST_1.3, DIST_2.3, DIST_3.3, DIST_4.3
Other:
- moved on the sheet: R16, R17, TRANSCEIVER

Commit message: Moved Power Switch/Deleted 24 V parts
Moved power switch to left side of the board (moved around parts accordingly)
Deleted 24 V parts on Kirbi
Parts:
- removed C10, C4, C5, C9: 0.1uF, SparkFun-Capacitors:0.1UF-0603-25V-(+80/-20%)
- removed D1: 24V, SparkFun-LED:LED0603
- removed R18: 11.15k, SparkFun-Resistors:1KOHM-0603-1/10W-1%
Connections:
- removed net N$6: D1.C, R18.1
- net 24V: no longer C10.1, C4.1, C5.1, C9.1, D1.A
- net GND: no longer C10.2, C4.2, C5.2, C9.2, R18.2

Commit message: Fixed MUXs and Centered LEDs
Connectted Tx (Connectors) to Rx (Teensi) and Rx (Connectors) to Tx (Teensi)
Connections:
- net RXO1: now also MUX_TX1.P$4; no longer MUX_RX1.P$4
- net RXO2: now also MUX_TX2.P$4; no longer MUX_RX2.P$4
- net TXO1: now also MUX_RX1.P$4; no longer MUX_TX1.P$4
- net TXO2: now also MUX_RX2.P$4; no longer MUX_TX2.P$4
Changed lines of the file:
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@@
 <net name="TXO1" class="0">
+<segment>
+<pinref part="U2" gate="G$1" pin="10/TX2/PWM"/>
+<wire x1="165.1" y1="210.82" x2="160.02" y2="210.82" width="0.1524" layer="91"/>
+<label x="160.02" y="210.82" size="1.778" layer="95" rot="MR0" xref="yes"/>
+</segment>
+<segment>
+<pinref part="MUX_RX1" gate="G$1" pin="P$4"/>
+<wire x1="370.84" y1="213.36" x2="373.38" y2="213.36" width="0.1524" layer="91"/>
+<label x="370.84" y="213.36" size="1.778" layer="95" xref="yes"/>
+</segment>
+</net>
+<net name="TXO2" class="0">
+<segment>
+<pinref part="U2" gate="G$1" pin="8/TX3/PWM"/>
+<wire x1="165.1" y1="215.9" x2="160.02" y2="215.9" width="0.1524" layer="91"/>
+<label x="160.02" y="215.9" size="1.778" layer="95" rot="MR0" xref="yes"/>
+</segment>
+<segment>
+<pinref part="MUX_RX2" gate="G$1" pin="P$4"/>
+<wire x1="406.4" y1="213.36" x2="408.94" y2="213.36" width="0.1524" layer="91"/>
+<label x="408.94" y="213.36" size="1.778" layer="95" xref="yes"/>
+</segment>
+</net>
+<net name="RXO1" class="0">
+<segment>
+<pinref part="U2" gate="G$1" pin="9/RX2/PWM"/>
+<wire x1="165.1" y1="213.36" x2="160.02" y2="213.36" width="0.1524" layer="91"/>
+<label x="160.02" y="213.36" size="1.778" layer="95" rot="MR0" xref="yes"/>
+</segment>
 <segment>
 <pinref part="MUX_TX1" gate="G$1" pin="P$4"/>
@@
 <label x="292.1" y="213.36" size="1.778" layer="95" xref="yes"/>
 </segment>
+</net>
+<net name="RXO2" class="0">
 <segment>
-<pinref part="U2" gate="G$1" pin="10/TX2/PWM"/>
-<wire x1="165.1" y1="210.82" x2="160.02" y2="210.82" width="0.1524" layer="91"/>
-<label x="160.02" y="210.82" size="1.778" layer="95" rot="MR0" xref="yes"/>
+<pinref part="U2" gate="G$1" pin="7/RX3/PWM"/>
+<wire x1="165.1" y1="218.44" x2="160.02" y2="218.44" width="0.1524" layer="91"/>
+<label x="160.02" y="218.44" size="1.778" layer="95" rot="MR0" xref="yes"/>
 </segment>
-</net>
-<net name="TXO2" class="0">
 <segment>
 <pinref part="MUX_TX2" gate="G$1" pin="P$4"/>
@@
 <label x="330.2" y="213.36" size="1.778" layer="95" xref="yes"/>
 </segment>
-<segment>
-<pinref part="U2" gate="G$1" pin="8/TX3/PWM"/>
-<wire x1="165.1" y1="215.9" x2="160.02" y2="215.9" width="0.1524" layer="91"/>
-<label x="160.02" y="215.9" size="1.778" layer="95" rot="MR0" xref="yes"/>
-</segment>
 </net>
-<net name="RXO1" class="0">
-<segment>
-<pinref part="MUX_RX1" gate="G$1" pin="P$4"/>
-<wire x1="370.84" y1="213.36" x2="373.38" y2="213.36" width="0.1524" layer="91"/>
-<label x="370.84" y="213.36" size="1.778" layer="95" xref="yes"/>
-</segment>
-<segment>
-<pinref part="U2" gate="G$1" pin="9/RX2/PWM"/>
-<wire x1="165.1" y1="213.36" x2="160.02" y2="213.36" width="0.1524" layer="91"/>
-<label x="160.02" y="213.36" size="1.778" layer="95" rot="MR0" xref="yes"/>
-</segment>
-</net>
-<net name="RXO2" class="0">
-<segment>
-<pinref part="MUX_RX2" gate="G$1" pin="P$4"/>
-<wire x1="406.4" y1="213.36" x2="408.94" y2="213.36" width="0.1524" layer="91"/>
-<label x="408.94" y="213.36" size="1.778" layer="95" xref="yes"/>
-</segment>
-<segment>
-<pinref part="U2" gate="G$1" pin="7/RX3/PWM"/>
-<wire x1="165.1" y1="218.44" x2="160.02" y2="218.44" width="0.1524" layer="91"/>
-<label x="160.02" y="218.44" size="1.778" layer="95" rot="MR0" xref="yes"/>
-</segment>
-</net>

Commit message: Finished Multiplexing
Changed schematic of multiplexer (Tx to Teensi TX etc.)/Wired on board
Parts:
- removed BATT: TE_02X01_3.96MM, Kirbi_ControlBoard:TE_02X01_3.96MM
- removed C15: 10uF, SparkFun-Capacitors:0.1UF-0603-25V-(+80/-20%)
- removed C16: 1uF, SparkFun-Capacitors:0.1UF-0603-25V-(+80/-20%)
- removed LIDAR_L, LIDAR_R: MOLEX_1.25MM_4PIN_SMT, Kirbi_ControlBoard:MOLEX_1.25MM_4PIN_SMT
- added DIST_5, DIST_6: MOLEX_1.25MM_4PIN_SMT, Kirbi_ControlBoard:MOLEX_1.25MM_4PIN_SMT
- R1: value 50 -> 1.65k
Connections:
- removed net +3V3: MUX_RX1.P$6, MUX_RX2.P$6, MUX_TX1.P$6, MUX_TX2.P$6, TRANSCEIVER.8
- removed net 24V: BATT.+, C15.1, C16.1
- removed net RX1: LIDAR_R.2, U2.0/RX1/MOSI1/T
- removed net RX2: LIDAR_L.2, U2.31/A12/RX4
- removed net RXO1: MUX_TX1.P$4, U2.9/RX2/PWM
- removed net RXO2: MUX_TX2.P$4, U2.7/RX3/PWM
- removed net TX1: LIDAR_R.3, U2.1/TX1/MISO1/T
- removed net TX2: LIDAR_L.3, U2.32/A13/TX4
- removed net TXO1: MUX_RX1.P$4, U2.10/TX2/PWM
- removed net TXO2: MUX_RX2.P$4, U2.8/TX3/PWM
- new net RXD5: DIST_5.2, MUX_RX2.I0
- new net RXD6: DIST_6.2, MUX_RX2.I1
- new net TRX1: MUX_RX1.Y, U2.7/RX3/PWM
- new net TRX2: MUX_RX2.Y, U2.9/RX2/PWM
- new net TTX1: MUX_TX1.Y, U2.8/TX3/PWM
- new net TTX2: MUX_TX2.Y, U2.10/TX2/PWM
- new net TXD5: DIST_5.3, MUX_TX2.I0
- new net TXD6: DIST_6.3, MUX_TX2.I1
- net +3.3V: now also MUX_RX1.V, MUX_RX2.V, MUX_TX1.V, MUX_TX2.V, TRANSCEIVER.8
- net +5V: now also DIST_5.4, DIST_6.4; no longer LIDAR_L.4, LIDAR_R.4
- net GND: now also DIST_5.1, DIST_6.1, MUX_RX1.GND, MUX_RX2.GND, MUX_TX1.GND, MUX_TX2.GND; no longer BATT.-, C15.2, C16.2, ESC.1, LIDAR_L.1, LIDAR_R.1, MUX_RX1.P$5, MUX_RX2.P$5, MUX_TX1.P$5, MUX_TX2.P$5
- net MUXS1: now also MUX_RX1.S, MUX_TX1.S, U2.2/PWM; no longer MUX_RX1.P$3, MUX_TX1.P$3, U2.15/A1/T
- net MUXS2: now also MUX_RX2.S, MUX_TX2.S, U2.25; no longer MUX_RX2.P$3, MUX_TX2.P$3, U2.16/A2/T/PWM
- net RXD1: now also MUX_RX1.I0; no longer MUX_RX1.P$1
- net RXD2: now also MUX_RX1.I1; no longer MUX_RX1.P$2
- net RXD3: now also U2.0/RX1/MOSI1/T; no longer MUX_RX2.P$1
- net RXD4: now also U2.31/A12/RX4; no longer MUX_RX2.P$2
- net S2: no longer ESC.4
- net TXD1: now also MUX_TX1.I0; no longer MUX_TX1.P$1
- net TXD2: now also MUX_TX1.I1; no longer MUX_TX1.P$2
- net TXD3: now also U2.1/TX1/MISO1/T; no longer MUX_TX2.P$1
- net TXD4: now also U2.32/A13/TX4; no longer MUX_TX2.P$2
Other:
- note added: "Multiplexers"
- note added: "Power Input"
- note added: "Radio Transciever"
- note removed: "Battery Connector"
- note removed: "Power"
- moved on the sheet: C11, C12, C13, C14, C17, C18, C7, C8, D2, D3, D4, DIST_1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

Commit message: Deleted Traceiver Breakout Board/Wired Tranceiver Module
Added Radio Tranceiver Module and wired it on back of board
Parts:
- added C4: 0.1uF, SparkFun-Capacitors:0.1UF-0603-25V-(+80/-20%)
- TRANSCEIVER: device adafruit:PINHD-1X8BIG -> Kirbi_ControlBoard:RFM69HCW_SMT
Connections:
- net +3.3V: now also C4.1, TRANSCEIVER.VDD; no longer TRANSCEIVER.8
- net GND: now also C4.2, TRANSCEIVER.GND@1, TRANSCEIVER.GND@2, TRANSCEIVER.GND@3; no longer TRANSCEIVER.7
- net MISO: now also TRANSCEIVER.MISO; no longer TRANSCEIVER.1
- net MOSI: now also TRANSCEIVER.MOSI; no longer TRANSCEIVER.2
- net RADIO_DIO0: now also TRANSCEIVER.DIO0, U2.5/PWM; no longer TRANSCEIVER.6, U2.14/A0/PWM
- net RADIO_NSS: now also TRANSCEIVER.NSS; no longer TRANSCEIVER.4
- net RADIO_SCK: now also TRANSCEIVER.SCK; no longer TRANSCEIVER.3
Other:
- note added: "Radio Transceiver"
- note removed: "Radio Transciever"

Commit message: Fixed Wiring/Added Antenna
Added through hole Antenna for radio tranceiver.
Parts:
- added JP1: (no value), pinhead:PINHD-1X1
Connections:
- removed net S2: POWER.P4, U2.34/A15/RX5/CAN1-RX
- new net N$5: JP1.1, TRANSCEIVER.ANT
Changed lines of the file:
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@@
 <part name="+3V11" library="supply1" library_urn="urn:adsk.eagle:library:371" deviceset="+3V3" device=""/>
 <part name="C4" library="SparkFun-Capacitors" library_urn="urn:adsk.eagle:library:510" deviceset="0.1UF" device="-0603-25V-(+80/-20%)" package3d_urn="urn:adsk.eagle:package:37414/1" value="0.1uF"/>
+<part name="JP1" library="pinhead" library_urn="urn:adsk.eagle:library:325" deviceset="PINHD-1X1" device="" package3d_urn="urn:adsk.eagle:package:22485/2"/>
 </parts>
 <sheets>
@@
 <attribute name="VALUE" x="237.744" y="38.481" size="1.778" layer="96" font="vector"/>
 </instance>
+<instance part="JP1" gate="G$1" x="233.68" y="30.48" smashed="yes">
+<attribute name="NAME" x="227.33" y="33.655" size="1.778" layer="95"/>
+<attribute name="VALUE" x="227.33" y="25.4" size="1.778" layer="96"/>
+</instance>
 </instances>
 <busses>
@@
 </segment>
 </net>
-<net name="S2" class="0">
-<segment>
-<pinref part="POWER" gate="G$1" pin="P4"/>
-<wire x1="286.512" y1="110.49" x2="278.13" y2="110.49" width="0.1524" layer="91"/>
-</segment>
-<segment>
-<pinref part="U2" gate="G$1" pin="34/A15/RX5/CAN1-RX"/>
-<wire x1="165.1" y1="149.86" x2="160.02" y2="149.86" width="0.1524" layer="91"/>
-<label x="160.02" y="149.86" size="1.778" layer="95" rot="R180" xref="yes"/>
-</segment>
-</net>
 <net name="SCL2" class="0">
 <segment>
@@
 </segment>
 </net>
+<net name="N$5" class="0">
+<segment>
+<pinref part="JP1" gate="G$1" pin="1"/>
+<pinref part="TRANSCEIVER" gate="RFM59HCW" pin="ANT"/>
+<wire x1="231.14" y1="30.48" x2="226.06" y2="30.48" width="0.1524" layer="91"/>
+<wire x1="226.06" y1="30.48" x2="226.06" y2="35.56" width="0.1524" layer="91"/>
+</segment>
+</net>

Commit message: Decoupling Capacitors/Wiring/Moved Antenna
Added decoupling capacitors distance sensors
Re-routed some of the multiplexers
Moved Antenna to bottom of the board
Parts:
- added C10, C15, C16, C25, C5, C9: 0.1uF, SparkFun-Capacitors:0.1UF-0603-25V-(+80/-20%)
Connections:
- net +5V: now also C10.1, C15.1, C16.1, C25.1, C5.1, C9.1
- net GND: now also C10.2, C15.2, C16.2, C25.2, C5.2, C9.2
Changed lines of the file:
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@@
 <part name="C4" library="SparkFun-Capacitors" library_urn="urn:adsk.eagle:library:510" deviceset="0.1UF" device="-0603-25V-(+80/-20%)" package3d_urn="urn:adsk.eagle:package:37414/1" value="0.1uF"/>
 <part name="JP1" library="pinhead" library_urn="urn:adsk.eagle:library:325" deviceset="PINHD-1X1" device="" package3d_urn="urn:adsk.eagle:package:22485/2"/>
+<part name="C5" library="SparkFun-Capacitors" library_urn="urn:adsk.eagle:library:510" deviceset="0.1UF" device="-0603-25V-(+80/-20%)" package3d_urn="urn:adsk.eagle:package:37414/1" value="0.1uF"/>
+<part name="C9" library="SparkFun-Capacitors" library_urn="urn:adsk.eagle:library:510" deviceset="0.1UF" device="-0603-25V-(+80/-20%)" package3d_urn="urn:adsk.eagle:package:37414/1" value="0.1uF"/>
+<part name="C10" library="SparkFun-Capacitors" library_urn="urn:adsk.eagle:library:510" deviceset="0.1UF" device="-0603-25V-(+80/-20%)" package3d_urn="urn:adsk.eagle:package:37414/1" value="0.1uF"/>
+<part name="C15" library="SparkFun-Capacitors" library_urn="urn:adsk.eagle:library:510" deviceset="0.1UF" device="-0603-25V-(+80/-20%)" package3d_urn="urn:adsk.eagle:package:37414/1" value="0.1uF"/>
+<part name="C16" library="SparkFun-Capacitors" library_urn="urn:adsk.eagle:library:510" deviceset="0.1UF" device="-0603-25V-(+80/-20%)" package3d_urn="urn:adsk.eagle:package:37414/1" value="0.1uF"/>
+<part name="C25" library="SparkFun-Capacitors" library_urn="urn:adsk.eagle:library:510" deviceset="0.1UF" device="-0603-25V-(+80/-20%)" package3d_urn="urn:adsk.eagle:package:37414/1" value="0.1uF"/>
 </parts>
 <sheets>
@@
 <attribute name="VALUE" x="55.88" y="238.76" size="1.778" layer="96" rot="R90"/>
 </instance>
-<instance part="P+13" gate="1" x="101.346" y="244.094" smashed="yes">
-<attribute name="VALUE" x="104.14" y="239.522" size="1.778" layer="96" rot="R90"/>
+<instance part="P+13" gate="1" x="101.854" y="243.84" smashed="yes">
+<attribute name="VALUE" x="104.648" y="239.268" size="1.778" layer="96" rot="R90"/>
 </instance>
 <instance part="GND7" gate="1" x="58.42" y="220.98" smashed="yes">
@@
 <attribute name="NAME" x="227.33" y="33.655" size="1.778" layer="95"/>
 <attribute name="VALUE" x="227.33" y="25.4" size="1.778" layer="96"/>
+</instance>
+<instance part="C5" gate="G$1" x="101.6" y="154.94" smashed="yes">
+<attribute name="NAME" x="103.124" y="157.861" size="1.778" layer="95" font="vector"/>
+<attribute name="VALUE" x="103.124" y="152.781" size="1.778" layer="96" font="vector"/>
+</instance>
+<instance part="C9" gate="G$1" x="58.42" y="154.94" smashed="yes">
+<attribute name="NAME" x="59.944" y="157.861" size="1.778" layer="95" font="vector"/>
+<attribute name="VALUE" x="59.944" y="152.781" size="1.778" layer="96" font="vector"/>
+</instance>
+<instance part="C10" gate="G$1" x="58.42" y="190.5" smashed="yes">
+<attribute name="NAME" x="59.944" y="193.421" size="1.778" layer="95" font="vector"/>
+<attribute name="VALUE" x="59.944" y="188.341" size="1.778" layer="96" font="vector"/>
+</instance>
+<instance part="C15" gate="G$1" x="101.6" y="190.5" smashed="yes">
+<attribute name="NAME" x="103.124" y="193.421" size="1.778" layer="95" font="vector"/>
+<attribute name="VALUE" x="103.124" y="188.341" size="1.778" layer="96" font="vector"/>
+</instance>
+<instance part="C16" gate="G$1" x="58.42" y="228.6" smashed="yes">
+<attribute name="NAME" x="59.944" y="231.521" size="1.778" layer="95" font="vector"/>
+<attribute name="VALUE" x="59.944" y="226.441" size="1.778" layer="96" font="vector"/>
+</instance>
+<instance part="C25" gate="G$1" x="101.854" y="229.108" smashed="yes">
+<attribute name="NAME" x="103.378" y="232.029" size="1.778" layer="95" font="vector"/>
+<attribute name="VALUE" x="103.378" y="226.949" size="1.778" layer="96" font="vector"/>
 </instance>
 </instances>
@@
 <pinref part="GND7" gate="1" pin="GND"/>
 <pinref part="DIST_3" gate="G$1" pin="1"/>
+<pinref part="C16" gate="G$1" pin="2"/>
+<junction x="58.42" y="226.06"/>
 </segment>
 <segment>
@@
 <pinref part="GND8" gate="1" pin="GND"/>
 <pinref part="DIST_4" gate="G$1" pin="1"/>
+<pinref part="C25" gate="G$1" pin="2"/>
+<junction x="101.854" y="226.568"/>
 </segment>
 <segment>
@@
 <pinref part="GND4" gate="1" pin="GND"/>
 <pinref part="DIST_2" gate="G$1" pin="1"/>
+<pinref part="C15" gate="G$1" pin="2"/>
+<junction x="101.6" y="187.96"/>
 </segment>
 <segment>
@@
 <pinref part="GND5" gate="1" pin="GND"/>
 <pinref part="DIST_5" gate="G$1" pin="1"/>
+<pinref part="C9" gate="G$1" pin="2"/>
+<junction x="58.42" y="152.4"/>
 </segment>
 <segment>
@@
 <pinref part="GND6" gate="1" pin="GND"/>
 <pinref part="DIST_6" gate="G$1" pin="1"/>
+<pinref part="C5" gate="G$1" pin="2"/>
+<junction x="101.6" y="152.4"/>
 </segment>
 <segment>
@@
 <pinref part="GND1" gate="1" pin="GND"/>
 <pinref part="DIST_1" gate="G$1" pin="1"/>
+<pinref part="C10" gate="G$1" pin="2"/>
+<junction x="58.42" y="187.96"/>
 </segment>
 <segment>
@@
 <wire x1="58.42" y1="233.68" x2="58.42" y2="241.3" width="0.1524" layer="91"/>
 <pinref part="DIST_3" gate="G$1" pin="4"/>
+<pinref part="C16" gate="G$1" pin="1"/>
+<junction x="58.42" y="233.68"/>
 </segment>
 <segment>
 <pinref part="P+13" gate="1" pin="+5V"/>
 <wire x1="81.534" y1="234.188" x2="101.854" y2="234.188" width="0.1524" layer="91"/>
-<wire x1="101.854" y1="234.188" x2="101.346" y2="241.554" width="0.1524" layer="91"/>
+<wire x1="101.854" y1="234.188" x2="101.854" y2="241.3" width="0.1524" layer="91"/>
 <pinref part="DIST_4" gate="G$1" pin="4"/>
+<pinref part="C25" gate="G$1" pin="1"/>
+<junction x="101.854" y="234.188"/>
 </segment>
 <segment>
@@
 <wire x1="101.6" y1="195.58" x2="101.6" y2="203.2" width="0.1524" layer="91"/>
 <pinref part="DIST_2" gate="G$1" pin="4"/>
+<pinref part="C15" gate="G$1" pin="1"/>
+<junction x="101.6" y="195.58"/>
 </segment>
 <segment>
@@
 <wire x1="58.42" y1="160.02" x2="58.42" y2="167.64" width="0.1524" layer="91"/>
 <pinref part="DIST_5" gate="G$1" pin="4"/>
+<pinref part="C9" gate="G$1" pin="1"/>
+<junction x="58.42" y="160.02"/>
 </segment>
 <segment>
@@
 <wire x1="101.6" y1="160.02" x2="101.6" y2="167.64" width="0.1524" layer="91"/>
 <pinref part="DIST_6" gate="G$1" pin="4"/>
+<pinref part="C5" gate="G$1" pin="1"/>
+<junction x="101.6" y="160.02"/>
 </segment>
 <segment>
@@
 <wire x1="58.42" y1="195.58" x2="58.42" y2="203.2" width="0.1524" layer="91"/>
 <pinref part="DIST_1" gate="G$1" pin="4"/>
-</segment>
-<segment>
+<pinref part="C10" gate="G$1" pin="1"/>
+<junction x="58.42" y="195.58"/>
+</segment>
+<segment>
