File: Kirbi/v1 pcb/Kirbi_ControlBoard.sch (EAGLE design)
At the start: 63 parts, among them U1 PCA9306_LSSOP, U2 TEENSY_3.6_DIL, U5 LM393-8-SOIC, U6 AP2114H-1.8TRG1, U7 AP2114H-3.3TRG1

Commit message: Fixed fonts/silk screen/Changed resistor values
Fixed fonts: vectorized
Changed resistor values: for LEDs and power button
Re-centered LED on bottom of the board
Parts:
- removed R21: 50, SparkFun-Resistors:1KOHM-0603-1/10W-1%
- R1: value 1.65k -> 100; device SparkFun-Resistors:1KOHM-0603-1/10W-1% -> SparkFun-Resistors:100OHM-0603-1/4W-5%
- R19: value 1.65k -> 200; device SparkFun-Resistors:1KOHM-0603-1/10W-1% -> SparkFun-Resistors:200OHM-0603-1/10W-1%
- R20: value 800 -> 100; device SparkFun-Resistors:1KOHM-0603-1/10W-1% -> SparkFun-Resistors:100OHM-0603-1/4W-5%
Connections:
- removed net N$10: D4.C, R21.1
- net GND: now also D4.C; no longer R21.2
Changed lines of the file:
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@@
 <part name="GND2" library="SparkFun-PowerSymbols" library_urn="urn:adsk.eagle:library:530" deviceset="GND" device=""/>
 <part name="GND3" library="SparkFun-PowerSymbols" library_urn="urn:adsk.eagle:library:530" deviceset="GND" device=""/>
-<part name="R19" library="SparkFun-Resistors" deviceset="1KOHM" device="-0603-1/10W-1%" value="1.65k"/>
-<part name="R20" library="SparkFun-Resistors" deviceset="1KOHM" device="-0603-1/10W-1%" value="800"/>
+<part name="R19" library="SparkFun-Resistors" library_urn="urn:adsk.eagle:library:532" deviceset="200OHM" device="-0603-1/10W-1%" package3d_urn="urn:adsk.eagle:package:39650/1" value="200"/>
+<part name="R20" library="SparkFun-Resistors" library_urn="urn:adsk.eagle:library:532" deviceset="100OHM" device="-0603-1/4W-5%" package3d_urn="urn:adsk.eagle:package:39650/1" value="100"/>
 <part name="D2" library="SparkFun-LED" deviceset="LED" device="0603" value="5V"/>
 <part name="D3" library="SparkFun-LED" deviceset="LED" device="0603" value="3.3V"/>
@@
 <part name="+3V6" library="supply1" library_urn="urn:adsk.eagle:library:371" deviceset="+3V3" device=""/>
 <part name="D4" library="SparkFun-LED" deviceset="LED" device="0603" value="1.8V"/>
-<part name="R21" library="SparkFun-Resistors" deviceset="1KOHM" device="-0603-1/10W-1%" value="50"/>
 <part name="SUPPLY1" library="SparkFun-PowerSymbols" library_urn="urn:adsk.eagle:library:530" deviceset="1.8V" device=""/>
 <part name="GND28" library="SparkFun-PowerSymbols" library_urn="urn:adsk.eagle:library:530" deviceset="GND" device=""/>
@@
 <part name="GND18" library="supply1" library_urn="urn:adsk.eagle:library:371" deviceset="GND" device=""/>
 <part name="P+2" library="supply1" library_urn="urn:adsk.eagle:library:371" deviceset="+5V" device=""/>
-<part name="R1" library="SparkFun-Resistors" deviceset="1KOHM" device="-0603-1/10W-1%" value="1.65k"/>
+<part name="R1" library="SparkFun-Resistors" library_urn="urn:adsk.eagle:library:532" deviceset="100OHM" device="-0603-1/4W-5%" package3d_urn="urn:adsk.eagle:package:39650/1" value="100"/>
 <part name="MUX_TX1" library="Kirbi_ControlBoard" deviceset="MUX_74LVC1G157GV" device=""/>
 <part name="MUX_TX2" library="Kirbi_ControlBoard" deviceset="MUX_74LVC1G157GV" device=""/>
@@
 <attribute name="VALUE" x="278.892" y="34.925" size="1.778" layer="96" font="vector" rot="R180" align="top-left"/>
 </instance>
-<instance part="R21" gate="G$1" x="294.64" y="33.02" smashed="yes">
-<attribute name="NAME" x="294.64" y="34.544" size="1.778" layer="95" font="vector" align="bottom-center"/>
-<attribute name="VALUE" x="294.64" y="31.496" size="1.778" layer="96" font="vector" align="top-center"/>
-</instance>
 <instance part="SUPPLY1" gate="G$1" x="266.7" y="35.56" smashed="yes">
 <attribute name="VALUE" x="266.7" y="38.354" size="1.778" layer="96" align="bottom-center"/>
@@
 </segment>
 <segment>
-<pinref part="R21" gate="G$1" pin="2"/>
-<wire x1="299.72" y1="33.02" x2="304.8" y2="33.02" width="0.1524" layer="91"/>
-<wire x1="304.8" y1="33.02" x2="304.8" y2="30.48" width="0.1524" layer="91"/>
-<pinref part="GND28" gate="1" pin="GND"/>
-</segment>
-<segment>
 <pinref part="IMU" gate="G$1" pin="FSYNC"/>
 <wire x1="355.6" y1="152.4" x2="340.36" y2="152.4" width="0.1524" layer="91"/>
@@
 <wire x1="198.12" y1="33.02" x2="190.5" y2="33.02" width="0.1524" layer="91"/>
 <junction x="190.5" y="33.02"/>
+</segment>
+<segment>
+<pinref part="D4" gate="G$1" pin="C"/>
+<pinref part="GND28" gate="1" pin="GND"/>
+<wire x1="304.8" y1="30.48" x2="304.8" y2="33.02" width="0.1524" layer="91"/>
+<wire x1="304.8" y1="33.02" x2="279.4" y2="33.02" width="0.1524" layer="91"/>
 </segment>
 </net>
@@
 </segment>
 </net>
-<net name="N$10" class="0">
-<segment>
-<pinref part="D4" gate="G$1" pin="C"/>
-<pinref part="R21" gate="G$1" pin="1"/>
-<wire x1="279.4" y1="33.02" x2="289.56" y2="33.02" width="0.1524" layer="91"/>
-</segment>
-</net>

Commit message: Connected ESCs
Connectted ESCs (Added two multiplexers to Gucci/Changed RADIO_NSS to Pin 30)
Parts:
- ESC: value MOLEX_1.25MM_4PIN_SMT -> MOLEX_1.25MM_3PIN_SMT; device Kirbi_ControlBoard:MOLEX_1.25MM_4PIN_SMT -> Kirbi_ControlBoard:MOLEX_1.25MM_3PIN_SMT
Connections:
- net S1/TX renamed S1/TTX
- new net S1/TRX: ESC.2, U2.34/A15/RX5/CAN1-RX
- net GND: now also ESC.1
- net RADIO_NSS: now also U2.30/T/PWM; no longer U2.34/A15/RX5/CAN1-RX
Changed lines of the file:
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@@
 <part name="GND28" library="SparkFun-PowerSymbols" library_urn="urn:adsk.eagle:library:530" deviceset="GND" device=""/>
 <part name="GND19" library="SparkFun-PowerSymbols" library_urn="urn:adsk.eagle:library:530" deviceset="GND" device=""/>
-<part name="ESC" library="Kirbi_ControlBoard" deviceset="MOLEX_1.25MM_4PIN_SMT" device=""/>
 <part name="DIST_3" library="Kirbi_ControlBoard" deviceset="MOLEX_1.25MM_4PIN_SMT" device=""/>
 <part name="DIST_4" library="Kirbi_ControlBoard" deviceset="MOLEX_1.25MM_4PIN_SMT" device=""/>
@@
 <part name="U$2" library="Kirbi_ControlBoard" deviceset="BEL_FUSE_C1F_3.5" device=""/>
 <part name="C12" library="SparkFun-Capacitors" library_urn="urn:adsk.eagle:library:510" deviceset="0.1UF" device="-0603-25V-(+80/-20%)" package3d_urn="urn:adsk.eagle:package:37414/1" value="0.1uF"/>
+<part name="ESC" library="Kirbi_ControlBoard" deviceset="MOLEX_1.25MM_3PIN_SMT" device=""/>
+<part name="GND21" library="SparkFun-PowerSymbols" library_urn="urn:adsk.eagle:library:530" deviceset="GND" device=""/>
 </parts>
 <sheets>
@@
 <attribute name="VALUE" x="340.36" y="139.446" size="1.778" layer="96" align="top-center"/>
 </instance>
-<instance part="ESC" gate="G$1" x="271.78" y="149.86" smashed="yes">
-<attribute name="VALUE" x="266.7" y="142.494" size="1.778" layer="96" font="vector"/>
-<attribute name="NAME" x="266.7" y="157.988" size="1.778" layer="95" font="vector"/>
-</instance>
 <instance part="DIST_3" gate="G$1" x="33.02" y="228.6" smashed="yes">
 <attribute name="VALUE" x="27.94" y="221.234" size="1.778" layer="96" font="vector"/>
@@
 <attribute name="NAME" x="59.944" y="231.521" size="1.778" layer="95" font="vector"/>
 <attribute name="VALUE" x="59.944" y="226.441" size="1.778" layer="96" font="vector"/>
+</instance>
+<instance part="ESC" gate="G$1" x="271.78" y="149.86" smashed="yes">
+<attribute name="VALUE" x="269.24" y="142.494" size="1.778" layer="96" font="vector"/>
+<attribute name="NAME" x="269.24" y="155.448" size="1.778" layer="95" font="vector"/>
+</instance>
+<instance part="GND21" gate="1" x="279.908" y="136.906" smashed="yes">
+<attribute name="VALUE" x="279.908" y="136.652" size="1.778" layer="96" align="top-center"/>
 </instance>
 </instances>
@@
 <wire x1="304.8" y1="33.02" x2="279.4" y2="33.02" width="0.1524" layer="91"/>
 </segment>
+<segment>
+<pinref part="ESC" gate="G$1" pin="1"/>
+<pinref part="GND21" gate="1" pin="GND"/>
+<wire x1="279.4" y1="147.32" x2="279.908" y2="147.32" width="0.1524" layer="91"/>
+<wire x1="279.908" y1="147.32" x2="279.908" y2="139.446" width="0.1524" layer="91"/>
+</segment>
 </net>
 <net name="LINE_LF" class="0">
@@
 </segment>
 </net>
-<net name="S1/TX" class="0">
-<segment>
-<wire x1="276.86" y1="152.4" x2="281.94" y2="152.4" width="0.1524" layer="91"/>
-<label x="281.94" y="152.4" size="1.778" layer="95" xref="yes"/>
-<pinref part="ESC" gate="G$1" pin="3"/>
-</segment>
-<segment>
-<pinref part="U2" gate="G$1" pin="33/A14/TX5/CAN1-TX"/>
-<wire x1="165.1" y1="152.4" x2="160.02" y2="152.4" width="0.1524" layer="91"/>
-<label x="160.02" y="152.4" size="1.778" layer="95" rot="R180" xref="yes"/>
-</segment>
-</net>
 <net name="SCL2" class="0">
 <segment>
@@
 </segment>
 <segment>
-<pinref part="U2" gate="G$1" pin="34/A15/RX5/CAN1-RX"/>
-<wire x1="165.1" y1="149.86" x2="160.02" y2="149.86" width="0.1524" layer="91"/>
-<label x="160.02" y="149.86" size="1.778" layer="95" rot="R180" xref="yes"/>
+<pinref part="U2" gate="G$1" pin="30/T/PWM"/>
+<wire x1="165.1" y1="160.02" x2="160.02" y2="160.02" width="0.1524" layer="91"/>
+<label x="160.02" y="160.02" size="1.778" layer="95" rot="R180" xref="yes"/>
 </segment>
 </net>
@@
 </segment>
 </net>
+<net name="S1/TTX" class="0">
+<segment>
+<pinref part="U2" gate="G$1" pin="33/A14/TX5/CAN1-TX"/>
+<wire x1="165.1" y1="152.4" x2="160.02" y2="152.4" width="0.1524" layer="91"/>
+<label x="160.02" y="152.4" size="1.778" layer="95" rot="R180" xref="yes"/>
+</segment>
+<segment>
+<pinref part="ESC" gate="G$1" pin="3"/>
+<wire x1="279.4" y1="152.4" x2="281.94" y2="152.4" width="0.1524" layer="91"/>
+<label x="281.94" y="152.4" size="1.778" layer="95" xref="yes"/>
+</segment>
+</net>
+<net name="S1/TRX" class="0">
+<segment>
+<pinref part="U2" gate="G$1" pin="34/A15/RX5/CAN1-RX"/>
+<wire x1="165.1" y1="149.86" x2="160.02" y2="149.86" width="0.1524" layer="91"/>
+<label x="160.02" y="149.86" size="1.778" layer="95" rot="MR0" xref="yes"/>
+</segment>
+<segment>
+<pinref part="ESC" gate="G$1" pin="2"/>
+<wire x1="279.4" y1="149.86" x2="281.94" y2="149.86" width="0.1524" layer="91"/>
+<label x="281.94" y="149.86" size="1.778" layer="95" xref="yes"/>
+</segment>
+</net>

Commit message: Fixed Silkscreen/Fuse/Added Resistor
Fixed Silkscreen/Fuse (Added label)/Added Resistor (6.2 OHM to 1.8 LED)
Parts:
- added R2: 6.2, Kirbi_ControlBoard:6.2OHM-0603-1/10W-5%
- F1: value BEL_FUSE_C1F_3.5 -> 3.5
- renumbered U$2 to F1
Connections:
- new net N$9: D4.C, R2.1
- net GND: now also R2.2; no longer D4.C
Changed lines of the file:
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@@
 <part name="C25" library="SparkFun-Capacitors" library_urn="urn:adsk.eagle:library:510" deviceset="0.1UF" device="-0603-25V-(+80/-20%)" package3d_urn="urn:adsk.eagle:package:37414/1" value="0.1uF"/>
 <part name="POWER_CONN" library="Kirbi_ControlBoard" deviceset="MOLEX_2.54MM_2PIN" device=""/>
-<part name="U$2" library="Kirbi_ControlBoard" deviceset="BEL_FUSE_C1F_3.5" device=""/>
 <part name="C12" library="SparkFun-Capacitors" library_urn="urn:adsk.eagle:library:510" deviceset="0.1UF" device="-0603-25V-(+80/-20%)" package3d_urn="urn:adsk.eagle:package:37414/1" value="0.1uF"/>
 <part name="ESC" library="Kirbi_ControlBoard" deviceset="MOLEX_1.25MM_3PIN_SMT" device=""/>
 <part name="GND21" library="SparkFun-PowerSymbols" library_urn="urn:adsk.eagle:library:530" deviceset="GND" device=""/>
+<part name="F1" library="Kirbi_ControlBoard" deviceset="BEL_FUSE_C1F_3.5" device="" value="3.5"/>
+<part name="R2" library="Kirbi_ControlBoard" deviceset="6.2OHM" device="-0603-1/10W-5%" package3d_urn="urn:adsk.eagle:package:39650/1" value="6.2"/>
 </parts>
 <sheets>
@@
 <attribute name="VALUE" x="262.636" y="93.98" size="1.778" layer="95"/>
 </instance>
-<instance part="U$2" gate="G$1" x="279.4" y="104.14" smashed="yes"/>
 <instance part="C12" gate="G$1" x="58.42" y="228.6" smashed="yes">
 <attribute name="NAME" x="59.944" y="231.521" size="1.778" layer="95" font="vector"/>
@@
 <instance part="GND21" gate="1" x="279.908" y="136.906" smashed="yes">
 <attribute name="VALUE" x="279.908" y="136.652" size="1.778" layer="96" align="top-center"/>
+</instance>
+<instance part="F1" gate="G$1" x="279.4" y="104.14" smashed="yes">
+<attribute name="NAME" x="276.86" y="106.68" size="1.778" layer="95"/>
+<attribute name="VALUE" x="276.86" y="100.33" size="1.778" layer="96"/>
+</instance>
+<instance part="R2" gate="G$1" x="294.894" y="33.02" smashed="yes">
+<attribute name="NAME" x="294.894" y="34.544" size="1.778" layer="95" font="vector" align="bottom-center"/>
+<attribute name="VALUE" x="294.894" y="31.496" size="1.778" layer="96" font="vector" align="top-center"/>
 </instance>
 </instances>
@@
 </segment>
 <segment>
-<pinref part="D4" gate="G$1" pin="C"/>
 <pinref part="GND28" gate="1" pin="GND"/>
 <wire x1="304.8" y1="30.48" x2="304.8" y2="33.02" width="0.1524" layer="91"/>
-<wire x1="304.8" y1="33.02" x2="279.4" y2="33.02" width="0.1524" layer="91"/>
+<pinref part="R2" gate="G$1" pin="2"/>
+<wire x1="304.8" y1="33.02" x2="299.974" y2="33.02" width="0.1524" layer="91"/>
 </segment>
 <segment>
@@
 <net name="N$7" class="0">
 <segment>
-<pinref part="U$2" gate="G$1" pin="P$1"/>
 <pinref part="POWER_CONN" gate="G$1" pin="P$1"/>
 <wire x1="274.32" y1="104.14" x2="276.86" y2="104.14" width="0.1524" layer="91"/>
+<pinref part="F1" gate="G$1" pin="P$1"/>
 </segment>
 </net>
 <net name="N$6" class="0">
 <segment>
-<pinref part="U$2" gate="G$1" pin="P$2"/>
 <wire x1="281.94" y1="104.14" x2="284.48" y2="104.14" width="0.1524" layer="91"/>
 <wire x1="284.48" y1="104.14" x2="284.48" y2="110.49" width="0.1524" layer="91"/>
 <pinref part="POWER" gate="G$1" pin="P4"/>
 <wire x1="284.48" y1="110.49" x2="286.512" y2="110.49" width="0.1524" layer="91"/>
+<pinref part="F1" gate="G$1" pin="P$2"/>
 </segment>
 </net>
@@
 </segment>
 </net>
+<net name="N$9" class="0">
+<segment>
+<pinref part="D4" gate="G$1" pin="C"/>
+<pinref part="R2" gate="G$1" pin="1"/>
+<wire x1="279.4" y1="33.02" x2="289.814" y2="33.02" width="0.1524" layer="91"/>
+</segment>
+</net>

Commit message: Added Pull-up Resistors/Moved MUXs
Added Pull-up Resistors (1k OHM to RX line)
Added 6.2 OHM to 1.8 V LED
Moved MUXs and rerouted
Fixed SIlkscreen
Parts:
- added R3, R4: 1k, SparkFun-Resistors:1KOHM-0603-1/10W-1%
Connections:
- net +3.3V: now also R3.2, R4.2
- net TRX1: now also R4.1
- net TRX2: now also R3.1
Changed lines of the file:
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@@
 <part name="F1" library="Kirbi_ControlBoard" deviceset="BEL_FUSE_C1F_3.5" device="" value="3.5"/>
 <part name="R2" library="Kirbi_ControlBoard" deviceset="6.2OHM" device="-0603-1/10W-5%" package3d_urn="urn:adsk.eagle:package:39650/1" value="6.2"/>
+<part name="R3" library="SparkFun-Resistors" library_urn="urn:adsk.eagle:library:532" deviceset="1KOHM" device="-0603-1/10W-1%" package3d_urn="urn:adsk.eagle:package:39650/1" value="1k"/>
+<part name="R4" library="SparkFun-Resistors" library_urn="urn:adsk.eagle:library:532" deviceset="1KOHM" device="-0603-1/10W-1%" package3d_urn="urn:adsk.eagle:package:39650/1" value="1k"/>
+<part name="+3V16" library="supply1" library_urn="urn:adsk.eagle:library:371" deviceset="+3V3" device=""/>
 </parts>
 <sheets>
@@
 <attribute name="VALUE" x="294.894" y="31.496" size="1.778" layer="96" font="vector" align="top-center"/>
 </instance>
+<instance part="R3" gate="G$1" x="121.158" y="214.63" smashed="yes" rot="R90">
+<attribute name="NAME" x="119.634" y="214.63" size="1.778" layer="95" font="vector" rot="R90" align="bottom-center"/>
+<attribute name="VALUE" x="122.682" y="214.63" size="1.778" layer="96" font="vector" rot="R90" align="top-center"/>
+</instance>
+<instance part="R4" gate="G$1" x="129.032" y="214.63" smashed="yes" rot="R90">
+<attribute name="NAME" x="127.508" y="214.63" size="1.778" layer="95" font="vector" rot="R90" align="bottom-center"/>
+<attribute name="VALUE" x="130.556" y="214.63" size="1.778" layer="96" font="vector" rot="R90" align="top-center"/>
+</instance>
+<instance part="+3V16" gate="G$1" x="121.158" y="224.028" smashed="yes">
+<attribute name="VALUE" x="119.634" y="219.202" size="1.778" layer="96" rot="R90"/>
+</instance>
 </instances>
 <busses>
@@
 <pinref part="C4" gate="G$1" pin="1"/>
 <junction x="236.22" y="45.72"/>
+</segment>
+<segment>
+<pinref part="+3V16" gate="G$1" pin="+3V3"/>
+<pinref part="R3" gate="G$1" pin="2"/>
+<wire x1="121.158" y1="221.488" x2="121.158" y2="219.71" width="0.1524" layer="91"/>
+<pinref part="R4" gate="G$1" pin="2"/>
+<wire x1="129.032" y1="219.71" x2="121.158" y2="219.71" width="0.1524" layer="91"/>
+<junction x="121.158" y="219.71"/>
 </segment>
 </net>
@@
 <segment>
 <pinref part="U2" gate="G$1" pin="7/RX3/PWM"/>
-<wire x1="165.1" y1="218.44" x2="160.02" y2="218.44" width="0.1524" layer="91"/>
-<label x="160.02" y="218.44" size="1.778" layer="95" rot="MR0" xref="yes"/>
+<wire x1="165.1" y1="218.44" x2="144.78" y2="218.44" width="0.1524" layer="91"/>
+<label x="143.002" y="218.44" size="1.778" layer="95" rot="MR0" xref="yes"/>
+<pinref part="R4" gate="G$1" pin="1"/>
+<wire x1="144.78" y1="218.44" x2="143.002" y2="218.44" width="0.1524" layer="91"/>
+<wire x1="129.032" y1="209.55" x2="132.842" y2="209.55" width="0.1524" layer="91"/>
+<wire x1="132.842" y1="209.55" x2="132.842" y2="220.98" width="0.1524" layer="91"/>
+<wire x1="132.842" y1="220.98" x2="144.78" y2="220.98" width="0.1524" layer="91"/>
+<wire x1="144.78" y1="220.98" x2="144.78" y2="218.44" width="0.1524" layer="91"/>
+<junction x="144.78" y="218.44"/>
 </segment>
 </net>
@@
 <segment>
 <pinref part="U2" gate="G$1" pin="9/RX2/PWM"/>
-<wire x1="165.1" y1="213.36" x2="160.02" y2="213.36" width="0.1524" layer="91"/>
-<label x="160.02" y="213.36" size="1.778" layer="95" rot="MR0" xref="yes"/>
-</segment>
-</net>
+<wire x1="165.1" y1="213.36" x2="144.78" y2="213.36" width="0.1524" layer="91"/>
+<label x="143.764" y="213.36" size="1.778" layer="95" rot="MR0" xref="yes"/>
+<pinref part="R3" gate="G$1" pin="1"/>
+<wire x1="144.78" y1="213.36" x2="143.764" y2="213.36" width="0.1524" layer="91"/>
+<wire x1="121.158" y1="209.55" x2="121.158" y2="205.74" width="0.1524" layer="91"/>
+<wire x1="121.158" y1="205.74" x2="144.78" y2="205.74" width="0.1524" layer="91"/>
+<wire x1="144.78" y1="205.74" x2="144.78" y2="213.36" width="0.1524" layer="91"/>
+<junction x="144.78" y="213.36"/>
+</segment>
+</net>

Commit message: Added Pull up Resistors
Finished on Gucci/Still need to route on Kirbi
Parts:
- removed R4: 1k, SparkFun-Resistors:1KOHM-0603-1/10W-1%
- added R10, R11, R5, R6, R7: 1k, SparkFun-Resistors:1KOHM-0603-1/10W-1%
Connections:
- net +3.3V: now also R10.2, R11.2, R5.2, R6.2, R7.2; no longer R4.2
- net TRX1: now also R10.1; no longer R4.1
- net TRX2: now also R11.1; no longer R3.1
- net TXD1: now also R3.1
- net TXD2: now also R5.1
- net TXD5: now also R6.1
- net TXD6: now also R7.1
Other:
- note added: "*Note: The TX and RX labels refer to the respective Teensy connection (not the sensor pins)"
- moved on the sheet: R3
