File: Kirbi/v1 pcb/Kirbi_ControlBoard.sch (EAGLE design)
At the start: 69 parts, among them U1 PCA9306_LSSOP, U2 TEENSY_3.6_DIL, U5 LM393-8-SOIC, U6 AP2114H-1.8TRG1, U7 AP2114H-3.3TRG1

Commit message: Fixed Github versioning
Gucci:
V2 - 9/11/2019 (last push before competition)
V3 - current
Kirbi:
V1 - 9/11/2019 (last push before competition)
V2 - current
Parts:
- removed C25: 0.1uF, SparkFun-Capacitors:0.1UF-0603-25V-(+80/-20%)
- removed DIST_5, DIST_6: MOLEX_1.25MM_4PIN_SMT, Kirbi_ControlBoard:MOLEX_1.25MM_4PIN_SMT
- removed F1: 3.5, Kirbi_ControlBoard:BEL_FUSE_C1F_3.5
- removed JP1: (no value), pinhead:PINHD-1X1
- removed LED1: WS2812B5050, adafruit:WS2812B5050
- removed MUX_RX1, MUX_RX2, MUX_TX1, MUX_TX2: MUX_74LVC1G157GV, Kirbi_ControlBoard:MUX_74LVC1G157GV
- removed POWER: POWER_SWITCH, Kirbi_ControlBoard:POWER_SWITCH
- removed POWER_CONN: MOLEX_2.54MM_2PIN, Kirbi_ControlBoard:MOLEX_2.54MM_2PIN
- removed TRANSCEIVER: (no value), Kirbi_ControlBoard:RFM69HCW_SMT
- added BATT: TE_02X01_3.96MM, Kirbi_ControlBoard:TE_02X01_3.96MM
- added C13: 0.1uF, SparkFun-Capacitors:0.1UF-0603-25V-(+80/-20%)
- added C16: 1uF, SparkFun-Capacitors:0.1UF-0603-25V-(+80/-20%)
- added D1: 24V, SparkFun-LED:LED0603
- added LIDAR_L, LIDAR_R: MOLEX_1.25MM_4PIN_90, Kirbi_ControlBoard:MOLEX_1.25MM_4PIN_90
- added L_ENC, R_ENC: (no value), pinhead:PINHD-2X5/90
- added L_MOT, R_MOT: (no value), pinhead:PINHD-1X2
- added R12, R4, R8: 3k, SparkFun-Resistors:1KOHM-0603-1/10W-1%
- added R18: 11.15k, SparkFun-Resistors:1KOHM-0603-1/10W-1%
- added R21: 50, SparkFun-Resistors:1KOHM-0603-1/10W-1%
- added R22, R26, R28, R30: 6.98k, SparkFun-Resistors:1KOHM-0603-1/10W-1%
- added R23, R27, R29, R31: 1k, SparkFun-Resistors:1KOHM-0603-1/10W-1%
- added R9: 2k, SparkFun-Resistors:1KOHM-0603-1/10W-1%
- added U3, U4: MAX4173-SOT-23, Gucci_ControlBoard:MAX4173-SOT-23
- C15: value 0.1uF -> 10uF
- DIST_1, DIST_2, DIST_3, DIST_4: value MOLEX_1.25MM_4PIN_SMT -> AMPHENOL_2X02_2.54MM_SHROUD; device Kirbi_ControlBoard:MOLEX_1.25MM_4PIN_SMT -> Gucci_ControlBoard:AMPHENOL_2X02_2.54MM_SHROUD
- ESC: value MOLEX_1.25MM_3PIN_SMT -> MOLEX_1.25MM_4PIN_90; device Kirbi_ControlBoard:MOLEX_1.25MM_3PIN_SMT -> Kirbi_ControlBoard:MOLEX_1.25MM_4PIN_90
- R1: value 100 -> 2k; device SparkFun-Resistors:100OHM-0603-1/4W-5% -> SparkFun-Resistors:1KOHM-0603-1/10W-1%
- R10, R6: value 1k -> 3k
- R11, R3, R5, R7: value 1k -> 2k
- R19: value 200 -> 1.65k; device SparkFun-Resistors:200OHM-0603-1/10W-1% -> SparkFun-Resistors:1KOHM-0603-1/10W-1%
- R2: value 6.2 -> 3k; device Kirbi_ControlBoard:6.2OHM-0603-1/10W-5% -> SparkFun-Resistors:1KOHM-0603-1/10W-1%
- R20: value 100 -> 800; device SparkFun-Resistors:100OHM-0603-1/4W-5% -> SparkFun-Resistors:1KOHM-0603-1/10W-1%
Connections:
- removed net +5V: C10.1, C11.1, C12.1, C15.1, C24.1, C25.1, C5.1, C6.1, C7.1, C8.1, C9.1, D2.A, DIST_1.4, DIST_2.4, DIST_3.4, DIST_4.4, DIST_5.4, DIST_6.4, LED1.VDD, POWER.P3, POWER.P5, U2.VIN, U5.VCC, U7.VIN
- removed net MISO: TRANSCEIVER.MISO, U2.12/MISO0
- removed net MOSI: TRANSCEIVER.MOSI, U2.11/MOSI0
- removed net MUXS1: MUX_RX1.S, MUX_TX1.S, U2.2/PWM
- removed net MUXS2: MUX_RX2.S, MUX_TX2.S, U2.25
- removed net NEO_DI: LED1.DI, U2.24
- removed net RADIO_DIO0: TRANSCEIVER.DIO0, U2.5/PWM
- removed net RADIO_NSS: TRANSCEIVER.NSS, U2.30/T/PWM
- removed net RADIO_RESET: TRANSCEIVER.RESET, U2.29/T/PWM
- removed net RADIO_SCK: TRANSCEIVER.SCK, U2.13/SCK0/LED
- removed net RXD1: DIST_1.2, MUX_RX1.I0
- removed net RXD2: DIST_2.2, MUX_RX1.I1
- removed net RXD3: DIST_3.2, U2.0/RX1/MOSI1/T
- removed net RXD4: DIST_4.2, U2.31/A12/RX4
- removed net RXD5: DIST_5.2, MUX_RX2.I0
- removed net RXD6: DIST_6.2, MUX_RX2.I1
- removed net S1/TRX: ESC.2, U2.34/A15/RX5/CAN1-RX
- removed net S1/TTX: ESC.3, U2.33/A14/TX5/CAN1-TX
- removed net TRX1: MUX_RX1.Y, R10.1, U2.7/RX3/PWM
- removed net TRX2: MUX_RX2.Y, R11.1, U2.9/RX2/PWM
- removed net TTX1: MUX_TX1.Y, U2.8/TX3/PWM
- removed net TTX2: MUX_TX2.Y, U2.10/TX2/PWM
- removed net TXD1: DIST_1.3, MUX_TX1.I0, R3.1
- removed net TXD2: DIST_2.3, MUX_TX1.I1, R5.1
- removed net TXD3: DIST_3.3, U2.1/TX1/MISO1/T
- removed net TXD4: DIST_4.3, U2.32/A13/TX4
- removed net TXD5: DIST_5.3, MUX_TX2.I0, R6.1
- removed net TXD6: DIST_6.3, MUX_TX2.I1, R7.1
- new net 24V: BATT.+, C10.1, C15.1, C16.1, C4.1, C5.1, C9.1, D1.A, DIST_1.2, DIST_1.4, DIST_2.2, DIST_2.4, DIST_3.2, DIST_3.4, DIST_4.2, DIST_4.4
- new net 3V_ENCODER1_A: R5.2, R6.2, U2.22/A8/T/PWM
- new net 3V_ENCODER1_B: R3.2, R4.2, U2.21/A7/PWM
- new net 3V_ENCODER1_I: R1.2, R2.2, U2.20/A6/PWM
- new net 3V_ENCODER2_A: R11.2, R12.2, U2.38/A19/SDA1/PWM
- new net 3V_ENCODER2_B: R10.2, R9.2, U2.37/A18/SCL1/PWM
- new net 3V_ENCODER2_I: R7.2, R8.2, U2.36/A17/PWM
- new net 5V: C11.1, C12.1, C13.1, C24.1, C6.1, C7.1, C8.1, D2.A, ESC.3, LIDAR_L.1, LIDAR_R.1, L_ENC.2, R_ENC.2, U2.VIN, U5.VCC, U7.VIN
- new net CURRENT_L: U2.A21/DAC0, U4.OUT
- new net CURRENT_R: U2.14/A0/PWM, U3.OUT
- new net DIST_L: R22.1, R23.2, U2.30/T/PWM
- new net DIST_L_45: R26.1, R27.2, U2.28
- new net DIST_R: R28.1, R29.2, U2.2/PWM
- new net DIST_R_45: R30.1, R31.2, U2.3/CAN0-TX/SCL2/PWM
- new net ENCODER1_A: R5.1, R_ENC.6
- new net ENCODER1_B: R3.1, R_ENC.8
- new net ENCODER2_A: L_ENC.6, R11.1
- new net ENCODER2_B: L_ENC.8, R9.1
- new net IMU_AD0: IMU.AD0/SDO, U2.9/RX2/PWM
- new net IMU_INT: IMU.INT1, U2.12/MISO0
- new net L_MOT+: L_MOT.2, U4.RS+
- new net L_MOT-: L_MOT.1, U4.RS-
- new net N$10: D4.C, R21.1
- new net N$11: DIST_3.3, R26.2
- new net N$12: DIST_2.3, R30.2
- new net RX1: LIDAR_R.3, U2.0/RX1/MOSI1/T
- new net RX2: LIDAR_L.3, U2.31/A12/RX4
- new net R_MOT+: R_MOT.2, U3.RS+
- new net R_MOT-: R_MOT.1, U3.RS-
- new net S1/TX: ESC.2, U2.33/A14/TX5/CAN1-TX
- new net S2: ESC.1, U2.34/A15/RX5/CAN1-RX
- new net TX1: LIDAR_R.2, U2.1/TX1/MISO1/T
- new net TX2: LIDAR_L.2, U2.32/A13/TX4
- net +3.3V: now also U3.VCC, U4.VCC; no longer C4.1, MUX_RX1.V, MUX_RX2.V, MUX_TX1.V, MUX_TX2.V, R10.2, R11.2, R3.2, R5.2, R6.2, R7.2, TRANSCEIVER.VDD
- net GND: now also BATT.-, C13.2, C16.2, ESC.4, LIDAR_L.4, LIDAR_R.4, L_ENC.3, R10.1, R12.1, R18.2, R2.1, R21.2, R23.1, R27.1, R29.1, R31.1, R4.1, R6.1, R8.1, R_ENC.3, U3.GND, U4.GND; no longer C25.2, DIST_5.1, DIST_6.1, ESC.1, IMU.AD0/SDO, LED1.GND, MUX_RX1.GND, MUX_RX2.GND, MUX_TX1.GND, MUX_TX2.GND, POWER_CONN.P$2, R1.1, R2.2, TRANSCEIVER.GND@1, TRANSCEIVER.GND@2, TRANSCEIVER.GND@3
- net LF_INT: now also U2.18/A4/T/SDA0; no longer U2.15/A1/T
- net N$5: now also R1.1, R_ENC.10; no longer JP1.1, TRANSCEIVER.ANT
- net N$6: now also D1.C, R18.1; no longer F1.P$2, POWER.P4
- net N$7: now also DIST_1.3, R28.2; no longer F1.P$1, POWER_CONN.P$1
- net N$8: now also L_ENC.10, R7.1; no longer POWER.P1, R1.2
- net N$9: now also DIST_4.3, R22.2; no longer D4.C, R2.1
- net RF_INT: now also U2.19/A5/T/SCL0; no longer U2.16/A2/T/PWM
- net SCL2: now also U2.7/RX3/PWM; no longer U2.3/CAN0-TX/SCL2/PWM
- net SDA2: now also U2.8/TX3/PWM; no longer U2.4/CAN0-RX/SDA2/PWM
- net START: now also U2.17/A3/T/PWM; no longer U2.14/A0/PWM
Other:
- note added: "Battery Connector"
- note added: "Current Sensing"
- note added: "Encoder Connectos And Signal Shifting For Teensy"
- note added: "Omron Distance Sensors"
- note removed: "*Note: The TX and RX labels refer to the respective Teensy connection (not the sensor pins)"
- note removed: "Multiplexers"
- note removed: "Power Input"
- note removed: "Radio Transceiver"
- moved on the sheet: C10, C11, C12, C14, C15, C17, C18, C4, C5, C7, C8, C9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
