File: CurrentSensingBoard/sensor.sch (EAGLE design)
At the start: 14 parts

Commit message: routing
Parts:
- removed CONNECTOR: B2B-PH-K-S(LF)(SN), B2B-PH-K-S_LF__SN_:B2B-PH-K-S(LF)(SN)
- added Q1, Q2: (no value), Adafruit FET 4-Channel Shifter:ADAFRUIT_MOSFET-NREFLOW
- added R3, R4, R5, R6: 10k, rcl:R-US_R0603
- added U$2: MOLEX_1.25MM_4PIN_90, Kirbi_ControlBoard:MOLEX_1.25MM_4PIN_90
Connections:
- new net +3V3: Q1.G, Q2.G, R3.1, R5.1, U$1.3.3V
- new net RX_NANO: Q1.D, R6.2, U$1.RX1
- new net TX_NANO: Q2.D, R4.2, U$1.TX0
- net +5V: now also R4.1, R6.1, U$2.4
- net GND: now also U$2.1
- net RX_TEENSY: now also Q2.S, R3.2, U$2.3; no longer CONNECTOR.2, U$1.TX0
- net TX_TEENSY: now also Q1.S, R5.2, U$2.2; no longer CONNECTOR.1, U$1.RX1
Other:
- note added: "Level Shifters"
