File: CurrentSensingBoard/powerDistribution.brd (EAGLE design)
At the start: 48 x 46 mm, 37 parts, among them J1 XT-60BATT_LABEL, U1 MAX11635EEE+, U2 LM2678SX-5.0/NOPB, U7 AP2114H-3.3TRG1

Commit message: started layout of power board
Parts:
- added J2, J3: XT-60BATT_LABEL, RoboJackets-Connectors:XT-60
- moved F2 352.1 mm to (64.0, 64.0), turned to 90 degrees
- moved C14 327.8 mm to (43.0, 50.0)
- moved F1 322.6 mm to (8.00, 64.0), turned to 270 degrees
- moved C13 313.0 mm to (43.0, 44.0)
- moved C11 304.0 mm to (29.0, 50.0), turned to 180 degrees
- moved U$2 273.2 mm to (31.0, 33.0)
- moved C10 272.4 mm to (34.0, 23.0), turned to 90 degrees
- moved C7 272.4 mm to (41.0, 23.0), turned to 90 degrees
- moved C15 240.2 mm to (34.0, 40.0), turned to 180 degrees
- moved C12 229.9 mm to (29.0, 46.0), turned to 180 degrees
- moved J1 214.0 mm to (36.0, 70.0), turned to 180 degrees
- moved U2 203.6 mm to (48.0, 34.0), turned to 270 degrees
- moved U$1 174.0 mm to (24.0, 33.0)
- moved C4 164.2 mm to (68.0, 25.0)
- moved R14 160.3 mm to (65.0, 26.0), turned to 90 degrees
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Connections:
- removed net MOTOR1: F1.1, F1.LEG1
- removed net MOTOR2: F2.1, F2.LEG1
- removed net N$5: C5.1
- removed net VDD: U1.11
- removed net VSS: C2.1, C3.2, R7.1, R8.2, U$4.1, U$4.3, U$4.5, U1.10
- net +24V: now also F1.1, F1.LEG1, F2.1, F2.LEG1
- net +3V3: now also U1.11
- net GND: now also C2.1, C3.2, J2.GND, J3.GND, R7.1, R8.2, U$4.1, U$4.3, U$4.5, U1.10
- net N1: now also J2.BATT
- net N2: now also J3.BATT
- net VREF: now also C5.1
Routing:
- removed copper zone on layer 1, net +5V
- removed copper zone on layer 16, net GND
Other:
- board size 48 x 46 mm -> 80 x 71 mm
