File: CurrentSensingBoard/powerDistribution.brd (EAGLE design)
At the start: 80 x 71 mm, 39 parts, among them J1 XT-60BATT_LABEL, J2 XT-60BATT_LABEL, J3 XT-60BATT_LABEL, U1 MAX11635EEE+, U2 LM2678SX-5.0/NOPB, U7 AP2114H-3.3TRG1

Commit message: added power LEDs
Parts:
- added D1, D2, D3: LED-SMD, RoboJackets-LEDs:CHIP-LED0603
- added R3: 100Ω, rcl:R0603
- added R4: 200Ω, rcl:R0603
- added R5: 1200Ω, rcl:R0603
- U$2: value MBRD835LT4G -> SD2114S040S8R0; device CurrentSensing:SCHDIODE -> CurrentSensing:SD2114S040S8R0
- moved U$2 74.4 mm to (-18.0, -23.0)
Connections:
- new net N$5: D1.A, R3.1
- new net N$8: D2.A, R4.1
- new net N$9: D3.A, R5.1
- net +24V: now also R5.2
- net +3V3: now also R3.2
- net +5V: now also R4.2
- net GND: now also D1.C, D2.C, D3.C; no longer U$2.3
- net N$6: now also U$2.2; no longer U$2.4
Changed lines of the file:
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@@
 <attribute name="VALUE" x="34.635" y="41.905" size="1.27" layer="27" rot="R180"/>
-</element>
-<element name="U$2" library="CurrentSensing" package="SCHDIODE" value="MBRD835LT4G" x="31" y="33" smashed="yes">
-<attribute name="NAME" x="28.46" y="36.81" size="1.27" layer="25" ratio="6"/>
-<attribute name="VALUE" x="28.46" y="27.92" size="1.27" layer="27" ratio="6"/>
 </element>
 <element name="C7" library="CurrentSensing" package="860010373009" value="180uF" x="41" y="23" smashed="yes" rot="R90">
@@
 <element name="J3" library="RoboJackets-Connectors" package="XT-60" value="XT-60BATT_LABEL" x="71" y="39" smashed="yes" rot="R180">
 <attribute name="NAME" x="75.5" y="39" size="1" layer="25" font="vector" ratio="10" rot="R270"/>
+</element>
+<element name="R3" library="rcl" library_urn="urn:adsk.eagle:library:334" package="R0603" package3d_urn="urn:adsk.eagle:package:23555/3" value="100Ω" x="-6" y="-9" smashed="yes">
+<attribute name="NAME" x="-6.635" y="-8.365" size="1.27" layer="25"/>
+<attribute name="POPULARITY" value="77" x="-6" y="-9" size="1.778" layer="27" display="off"/>
+<attribute name="SPICEPREFIX" value="R" x="-6" y="-9" size="1.778" layer="27" display="off"/>
+<attribute name="VALUE" x="-6.635" y="-10.905" size="1.27" layer="27"/>
+</element>
+<element name="R4" library="rcl" library_urn="urn:adsk.eagle:library:334" package="R0603" package3d_urn="urn:adsk.eagle:package:23555/3" value="200Ω" x="-6" y="-13" smashed="yes">
+<attribute name="NAME" x="-6.635" y="-12.365" size="1.27" layer="25"/>
+<attribute name="POPULARITY" value="77" x="-6" y="-13" size="1.778" layer="27" display="off"/>
+<attribute name="SPICEPREFIX" value="R" x="-6" y="-13" size="1.778" layer="27" display="off"/>
+<attribute name="VALUE" x="-6.635" y="-14.905" size="1.27" layer="27"/>
+</element>
+<element name="R5" library="rcl" library_urn="urn:adsk.eagle:library:334" package="R0603" package3d_urn="urn:adsk.eagle:package:23555/3" value="1200Ω" x="-6" y="-17" smashed="yes">
+<attribute name="NAME" x="-6.635" y="-16.365" size="1.27" layer="25"/>
+<attribute name="POPULARITY" value="77" x="-6" y="-17" size="1.778" layer="27" display="off"/>
+<attribute name="SPICEPREFIX" value="R" x="-6" y="-17" size="1.778" layer="27" display="off"/>
+<attribute name="VALUE" x="-6.635" y="-18.905" size="1.27" layer="27"/>
+</element>
+<element name="D1" library="RoboJackets-LEDs" package="CHIP-LED0603" value="LED-SMD" x="-11" y="-16" smashed="yes">
+<attribute name="DIGIKEY" value="" x="-11" y="-16" size="1.778" layer="27" display="off"/>
+<attribute name="MPN" value="" x="-11" y="-16" size="1.778" layer="27" display="off"/>
+<attribute name="NAME" x="-11.635" y="-16.635" size="1.27" layer="25" rot="R90"/>
+<attribute name="VALUE" x="-9.095" y="-16.635" size="1.27" layer="27" rot="R90"/>
+</element>
+<element name="D2" library="RoboJackets-LEDs" package="CHIP-LED0603" value="LED-SMD" x="-16" y="-16" smashed="yes">
+<attribute name="DIGIKEY" value="" x="-16" y="-16" size="1.778" layer="27" display="off"/>
+<attribute name="MPN" value="" x="-16" y="-16" size="1.778" layer="27" display="off"/>
+<attribute name="NAME" x="-16.635" y="-16.635" size="1.27" layer="25" rot="R90"/>
+<attribute name="VALUE" x="-14.095" y="-16.635" size="1.27" layer="27" rot="R90"/>
+</element>
+<element name="D3" library="RoboJackets-LEDs" package="CHIP-LED0603" value="LED-SMD" x="-21" y="-16" smashed="yes">
+<attribute name="DIGIKEY" value="" x="-21" y="-16" size="1.778" layer="27" display="off"/>
+<attribute name="MPN" value="" x="-21" y="-16" size="1.778" layer="27" display="off"/>
+<attribute name="NAME" x="-21.635" y="-16.635" size="1.27" layer="25" rot="R90"/>
+<attribute name="VALUE" x="-19.095" y="-16.635" size="1.27" layer="27" rot="R90"/>
+</element>
+<element name="U$2" library="CurrentSensing" package="SD2114S040S8R0" value="SD2114S040S8R0" x="-18" y="-23" smashed="yes">
+<attribute name="NAME" x="-22" y="-21" size="1" layer="25"/>
+<attribute name="VALUE" x="-22" y="-25" size="1" layer="27" align="top-left"/>
 </element>
 </elements>
@@
 <contactref element="R12" pad="2"/>
 <contactref element="C4" pad="2"/>
-<contactref element="U$2" pad="1"/>
-<contactref element="U$2" pad="3"/>
 <contactref element="U2" pad="8"/>
 <contactref element="U2" pad="4"/>
@@
 <contactref element="J2" pad="GND"/>
 <contactref element="J3" pad="GND"/>
+<contactref element="D1" pad="C"/>
+<contactref element="D2" pad="C"/>
+<contactref element="D3" pad="C"/>
+<contactref element="U$2" pad="1"/>
 <wire x1="60" y1="37.4" x2="62.54" y2="37.4" width="0" layer="19" extent="1-1"/>
 <wire x1="57.46" y1="37.4" x2="60" y2="37.4" width="0" layer="19" extent="1-1"/>
@@
 <wire x1="25.85" y1="50" x2="36" y2="58.908" width="0" layer="19" extent="1-1"/>
 <wire x1="28.15" y1="46" x2="25.85" y2="50" width="0" layer="19" extent="1-1"/>
-<wire x1="35.0894" y1="35.286" x2="27.11" y2="4.81" width="0" layer="19" extent="1-1"/>
-<wire x1="35.0894" y1="30.714" x2="35.0894" y2="35.286" width="0" layer="19" extent="1-1"/>
+<wire x1="-11" y1="-15.25" x2="19" y2="13.15" width="0" layer="19" extent="1-1"/>
+<wire x1="-16" y1="-15.25" x2="-11" y2="-15.25" width="0" layer="19" extent="1-1"/>
+<wire x1="-21" y1="-15.25" x2="-16" y2="-15.25" width="0" layer="19" extent="1-1"/>
+<wire x1="-20.325" y1="-23" x2="-21" y2="-15.25" width="0" layer="19" extent="1-1"/>
 </signal>
 <signal name="+5V">
@@
 <contactref element="C7" pad="1"/>
 <contactref element="C10" pad="1"/>
+<contactref element="R4" pad="2"/>
 <wire x1="60.85" y1="30" x2="58.73" y2="35.2" width="0" layer="19" extent="1-1"/>
 <wire x1="56" y1="29.15" x2="60.85" y2="30" width="0" layer="19" extent="1-1"/>
@@
 <wire x1="10.73" y1="35.2" x2="8.85" y2="30" width="0" layer="19" extent="1-1"/>
 <wire x1="44.89" y1="4.81" x2="41" y2="24.25" width="0" layer="19" extent="1-1"/>
+<wire x1="-5.15" y1="-13" x2="19" y2="14.85" width="0" layer="19" extent="1-1"/>
 </signal>
 <signal name="AIN1">
@@
 <contactref element="U1" pad="11"/>
 <contactref element="C6" pad="1"/>
+<contactref element="R3" pad="2"/>
 <wire x1="36.15" y1="10" x2="36.0475" y2="12.27585" width="0" layer="19" extent="1-1"/>
 <wire x1="29" y1="13.15" x2="36.0475" y2="12.27585" width="0" layer="19" extent="1-1"/>
 <wire x1="24" y1="10.975" x2="29" y2="13.15" width="0" layer="19" extent="1-1"/>
 <wire x1="24" y1="17.025" x2="24" y2="10.975" width="0" layer="19" extent="1-1"/>
+<wire x1="-5.15" y1="-9" x2="24" y2="10.975" width="0" layer="19" extent="1-1"/>
 </signal>
 <signal name="N$3">
@@
 <contactref element="F2" pad="1" route="any" routetag="G$1.1"/>
 <contactref element="F2" pad="LEG1" route="any" routetag="G$1.1"/>
+<contactref element="R5" pad="2"/>
 <wire x1="39.85" y1="50" x2="58.92" y2="59.935" width="0" layer="19" extent="1-1"/>
 <wire x1="39.85" y1="44" x2="39.85" y2="50" width="0" layer="19" extent="1-1"/>
@@
 <wire x1="36" y1="65.8455" x2="39.85" y2="50" width="0" layer="19" extent="1-1"/>
 <wire x1="13.08" y1="68.065" x2="36" y2="65.8455" width="0" layer="19" extent="1-1"/>
+<wire x1="-5.15" y1="-17" x2="39.68" y2="36.54" width="0" layer="19" extent="1-1"/>
 </signal>
 <signal name="N$6">
-<contactref element="U$2" pad="4"/>
 <contactref element="U$1" pad="P$1"/>
 <contactref element="U2" pad="1"/>
 <contactref element="C15" pad="2"/>
+<contactref element="U$2" pad="2"/>
 <wire x1="33.15" y1="40" x2="39.68" y2="37.81" width="0" layer="19" extent="1-1"/>
 <wire x1="24" y1="37.95" x2="33.15" y2="40" width="0" layer="19" extent="1-1"/>
-<wire x1="27.9012" y1="33" x2="24" y2="37.95" width="0" layer="19" extent="1-1"/>
+<wire x1="-15.675" y1="-23" x2="24" y2="37.95" width="0" layer="19" extent="1-1"/>
 </signal>
 <signal name="N$7">
@@
 <wire x1="71" y1="34.8455" x2="53.575" y2="49" width="0" layer="19" extent="1-1"/>
 </signal>
+<signal name="N$5">
+<contactref element="R3" pad="1"/>
+<contactref element="D1" pad="A"/>
+<wire x1="-6.85" y1="-9" x2="-11" y2="-16.75" width="0" layer="19" extent="1-1"/>
+</signal>
+<signal name="N$8">
+<contactref element="R4" pad="1"/>
+<contactref element="D2" pad="A"/>
+<wire x1="-6.85" y1="-13" x2="-16" y2="-16.75" width="0" layer="19" extent="1-1"/>
+</signal>
+<signal name="N$9">
+<contactref element="R5" pad="1"/>
+<contactref element="D3" pad="A"/>
+<wire x1="-6.85" y1="-17" x2="-21" y2="-16.75" width="0" layer="19" extent="1-1"/>
+</signal>
 </signals>

Commit message: started routing
Parts:
- moved D3 82.8 mm to (29.0, 50.0)
- moved U$2 82.4 mm to (30.0, 44.0), turned to 90 degrees
- moved R5 76.5 mm to (31.0, 50.0), turned to 90 degrees
- moved D2 45.3 mm to (18.0, 14.0)
- moved D1 44.1 mm to (26.0, 8.00)
- moved R3 38.0 mm to (28.0, 8.00), turned to 90 degrees
- moved R4 37.5 mm to (20.0, 14.0), turned to 90 degrees
- moved C11 27.3 mm to (40.0, 25.0), turned to 270 degrees
- moved C12 24.2 mm to (44.0, 27.0), turned to 270 degrees
- moved C7 15.0 mm to (56.0, 24.0)
- moved C10 14.6 mm to (48.6, 24.0)
- moved C14 9.22 mm to (49.0, 43.0)
- moved C15 8.49 mm to (40.0, 46.0)
- moved U$5 6.00 mm to (66.0, 49.0)
- moved C13 5.83 mm to (40.0, 39.0), turned to 270 degrees
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Connections:
- new net N$14: JP1.6
- net !EOC!: now also JP1.3; no longer JP1.6
- net MISO: now also JP1.4; no longer JP1.5
- net MOSI: now also JP1.5; no longer JP1.4
- net SCLK: no longer JP1.3
Routing:
- net +24V: track 0.00 -> 62.7 mm
- net GND: track 0.00 -> 32.1 mm, vias 0 -> 12
- net P2: track 0.00 -> 31.4 mm
- net P1: track 0.00 -> 22.9 mm
- net !CNVST!: track 0.00 -> 18.4 mm
- net +5V: track 0.00 -> 11.6 mm
- net !CS!: track 0.00 -> 11.4 mm
- net MOSI: track 0.00 -> 8.80 mm
- net +3V3: track 0.00 -> 8.70 mm
- net MISO: track 0.00 -> 8.01 mm
- net !EOC!: track 0.00 -> 7.71 mm
- net VREF: track 0.00 -> 6.34 mm
- net N$4: track 0.00 -> 5.71 mm
- net N$2: track 0.00 -> 5.13 mm
- net N$1: track 0.00 -> 5.08 mm
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- added copper zone on layer 1, net +5V
- added copper zone on layer 16, net GND

Commit message: updated board layout and routing
Parts:
- removed F1, F2: (no value), RoboJackets-Fuses:FUSEHOLDER_3549_X2
- added U$6, U$7: 3550, CurrentSensing:3550
- moved C11 31.0 mm to (48.0, 55.0), turned to 0 degrees
- moved C13 12.8 mm to (48.0, 49.0), turned to 0 degrees
- moved C12 11.2 mm to (39.0, 37.0)
- moved C8 11.0 mm to (12.0, 15.0)
- moved C9 11.0 mm to (22.0, 15.0)
- moved D1 11.0 mm to (15.0, 9.00)
- moved D2 11.0 mm to (7.00, 15.0)
- moved R3 11.0 mm to (17.0, 9.00)
- moved R4 11.0 mm to (9.00, 15.0)
- moved U7 11.0 mm to (17.0, 15.0)
- moved C2 10.8 mm to (11.0, 31.0), turned to 0 degrees
- moved C15 9.22 mm to (42.0, 37.0), turned to 90 degrees
- moved C6 8.06 mm to (36.0, 17.0), turned to 90 degrees
- moved C5 7.28 mm to (39.0, 19.0), turned to 180 degrees
- moved U$3 5.39 mm to (7.13, 2.77)
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Connections:
- removed net N$14: JP1.6
- net +24V: now also U$6.P$2, U$7.P$2; no longer F1.1, F1.LEG1, F2.1, F2.LEG1
- net P1: now also U$6.P$1; no longer F1.2, F1.LEG2
- net P2: now also U$7.P$1; no longer F2.2, F2.LEG2
- net SCLK: now also JP1.6
Routing:
- net VREF: track 6.34 -> 68.3 mm
- net +24V: track 62.7 -> 9.00 mm, vias 0 -> 6
- net GND: track 32.1 -> 68.4 mm, vias 12 -> 25
- net AIN0: track 2.21 -> 36.7 mm, vias 0 -> 2
- net AIN1: track 2.21 -> 35.9 mm
- net N2: track 0.00 -> 23.5 mm
- net +3V3: track 8.70 -> 32.0 mm
- net N$6: track 0.00 -> 20.8 mm
- net N1: track 0.00 -> 15.6 mm
- net P2: track 31.4 -> 16.1 mm
- net SCLK: track 0.00 -> 13.2 mm
- net !EOC!: track 7.71 -> 15.2 mm
- net MISO: track 8.01 -> 13.4 mm
- net +5V: track 11.6 -> 6.89 mm, vias 0 -> 2
- net MOSI: track 8.80 -> 13.2 mm
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- added copper zone on layer 1, net +24V

Commit message: helped Caleb
Routing:
- net P1: track 22.7 -> 0.00 mm
- net N1: track 15.6 -> 0.00 mm
- added copper zone on layer 1, net N1
- added copper zone on layer 1, net P1
Changed lines of the file:
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@@
 <setting verticaltext="up"/>
 </settings>
-<grid distance="1" unitdist="mm" unit="mm" style="lines" multiple="1" display="yes" altdistance="0.01" altunitdist="mm" altunit="mm"/>
+<grid distance="1" unitdist="mm" unit="mm" style="lines" multiple="1" display="no" altdistance="0.01" altunitdist="mm" altunit="mm"/>
 <layers>
 <layer number="1" name="Top" color="4" fill="1" visible="yes" active="yes"/>
@@
 </element>
 <element name="C2" library="rcl" library_urn="urn:adsk.eagle:library:334" package="C0603" package3d_urn="urn:adsk.eagle:package:23616/2" value="0.1uF" x="11" y="31" smashed="yes">
-<attribute name="NAME" x="10.365" y="31.635" size="1.27" layer="25"/>
+<attribute name="NAME" x="10.365" y="31.635" size="0.8128" layer="25"/>
 <attribute name="POPULARITY" value="37" x="11" y="31" size="1.778" layer="27" display="off"/>
 <attribute name="SPICEPREFIX" value="C" x="11" y="31" size="1.778" layer="27" display="off"/>
@@
 <wire x1="67" y1="32" x2="67.15" y2="32" width="0.2" layer="1"/>
 <wire x1="67.15" y1="32" x2="68.15" y2="31" width="0.2" layer="1"/>
+<wire x1="65" y1="37.4" x2="67.54" y2="37.4" width="0" layer="19" extent="1-1"/>
+<wire x1="62.46" y1="37.4" x2="65" y2="37.4" width="0" layer="19" extent="1-1"/>
+<wire x1="67" y1="32" x2="67.54" y2="37.4" width="0" layer="19" extent="1-1"/>
+<wire x1="66" y1="27.15" x2="68.15" y2="31" width="0" layer="19" extent="1-1"/>
+<wire x1="60" y1="28.85" x2="64.85" y2="26" width="0" layer="19" extent="1-1"/>
+<wire x1="60.15" y1="31" x2="59" y2="30" width="0" layer="19" extent="1-1"/>
+<wire x1="53" y1="34" x2="59" y2="32" width="0" layer="19" extent="1-1"/>
+<wire x1="39" y1="35" x2="42" y2="34" width="0" layer="19" extent="1-1"/>
+<wire x1="56" y1="22.75" x2="60" y2="28.85" width="0" layer="19" extent="1-1"/>
+<wire x1="48.56" y1="22.75" x2="56" y2="22.75" width="0" layer="19" extent="1-1"/>
+<wire x1="46" y1="16" x2="48.56" y2="22.75" width="0" layer="19" extent="1-1"/>
+<wire x1="40" y1="16" x2="43.72415" y2="16.5875" width="0" layer="19" extent="1-1"/>
+<wire x1="38.15" y1="19" x2="38.27585" y2="16.5875" width="0" layer="19" extent="1-1"/>
+<wire x1="36" y1="17.85" x2="37" y2="20" width="0" layer="19" extent="1-1"/>
+<wire x1="75" y1="27.908" x2="68.15" y2="31" width="0" layer="19" extent="1-1"/>
+<wire x1="49" y1="42" x2="53" y2="34" width="0" layer="19" extent="1-1"/>
+<wire x1="49" y1="48" x2="51.15" y2="43" width="0" layer="19" extent="1-1"/>
+<wire x1="49" y1="54" x2="51.15" y2="49" width="0" layer="19" extent="1-1"/>
+<wire x1="23" y1="17" x2="34" y2="17" width="0" layer="19" extent="1-1"/>
+<wire x1="19.3" y1="18.025" x2="22" y2="15.85" width="0" layer="19" extent="1-1"/>
+<wire x1="18" y1="26" x2="21" y2="20" width="0" layer="19" extent="1-1"/>
+<wire x1="19.85" y1="31" x2="17" y2="27.15" width="0" layer="19" extent="1-1"/>
+<wire x1="12" y1="26" x2="17" y2="27.15" width="0" layer="19" extent="1-1"/>
+<wire x1="10.15" y1="31" x2="11" y2="27.15" width="0" layer="19" extent="1-1"/>
+<wire x1="5" y1="27.908" x2="8" y2="31" width="0" layer="19" extent="1-1"/>
+<wire x1="17.54" y1="37.4" x2="21" y2="32" width="0" layer="19" extent="1-1"/>
+<wire x1="15" y1="37.4" x2="17.54" y2="37.4" width="0" layer="19" extent="1-1"/>
+<wire x1="12.46" y1="37.4" x2="15" y2="37.4" width="0" layer="19" extent="1-1"/>
+<wire x1="12" y1="14.15" x2="19.3" y2="18.025" width="0" layer="19" extent="1-1"/>
+<wire x1="14" y1="10" x2="11" y2="13" width="0" layer="19" extent="1-1"/>
+<wire x1="19" y1="8" x2="15" y2="9.75" width="0" layer="19" extent="1-1"/>
+<wire x1="7" y1="15.75" x2="11" y2="13" width="0" layer="19" extent="1-1"/>
+<wire x1="38" y1="58.908" x2="49" y2="54" width="0" layer="19" extent="1-1"/>
+<wire x1="29" y1="50.75" x2="38" y2="58.908" width="0" layer="19" extent="1-1"/>
+<wire x1="30" y1="46.325" x2="29" y2="50.75" width="0" layer="19" extent="1-1"/>
 </signal>
 <signal name="+5V">
@@
 <vertex x="0" y="0"/>
 <vertex x="80" y="0"/>
-<vertex x="80" y="33.38"/>
-<vertex x="0" y="33.38"/>
+<vertex x="80" y="31.38"/>
+<vertex x="0" y="31.38"/>
 </polygon>
 <polygon width="0.1524" layer="1" thermals="no">
-<vertex x="0" y="32"/>
-<vertex x="0" y="40"/>
+<vertex x="10" y="31"/>
+<vertex x="10" y="40"/>
 <vertex x="20" y="40"/>
-<vertex x="20" y="32"/>
+<vertex x="20" y="31"/>
 </polygon>
 <polygon width="0.1524" layer="1" thermals="no">
@@
 <wire x1="53" y1="27" x2="54.25" y2="27" width="0.2" layer="16"/>
 <wire x1="54.25" y1="27" x2="56" y2="25.25" width="0.2" layer="16"/>
+<wire x1="61.85" y1="31" x2="63.73" y2="35.2" width="0" layer="19" extent="1-1"/>
+<wire x1="63" y1="28.85" x2="61.85" y2="31" width="0" layer="19" extent="1-1"/>
+<wire x1="56" y1="25.25" x2="63" y2="28.85" width="0" layer="19" extent="1-1"/>
+<wire x1="51" y1="27" x2="53" y2="27" width="0" layer="19" extent="1-1"/>
+<wire x1="44.68" y1="31.46" x2="48.56" y2="25.25" width="0" layer="19" extent="1-1"/>
+<wire x1="28" y1="28.05" x2="44.68" y2="31.46" width="0" layer="19" extent="1-1"/>
+<wire x1="14" y1="28.85" x2="28" y2="28.05" width="0" layer="19" extent="1-1"/>
+<wire x1="11.85" y1="31" x2="14" y2="28.85" width="0" layer="19" extent="1-1"/>
+<wire x1="13.73" y1="35.2" x2="11.85" y2="31" width="0" layer="19" extent="1-1"/>
+<wire x1="14.7" y1="18.025" x2="14" y2="28.85" width="0" layer="19" extent="1-1"/>
+<wire x1="12" y1="15.85" x2="14.7" y2="18.025" width="0" layer="19" extent="1-1"/>
+<wire x1="9" y1="15.85" x2="12" y2="15.85" width="0" layer="19" extent="1-1"/>
+<wire x1="48.89" y1="4.81" x2="48.56" y2="25.25" width="0" layer="19" extent="1-1"/>
 </signal>
 <signal name="AIN1">
@@
 <contactref element="C14" pad="1"/>
 <contactref element="R5" pad="2"/>
-<polygon width="0.1524" layer="1" thermals="no">
-<vertex x="0" y="71"/>
-<vertex x="0" y="41"/>
-<vertex x="26" y="41"/>
-<vertex x="27" y="40"/>
-<vertex x="43" y="40"/>
-<vertex x="49" y="40"/>
-<vertex x="49" y="57"/>
-<vertex x="50" y="58"/>
-<vertex x="80" y="58"/>
-<vertex x="80" y="71"/>
-</polygon>
 <via x="41" y="55" extent="1-16" drill="1"/>
 <via x="44" y="55" extent="1-16" drill="1"/>
@@
 <contactref element="U$6" pad="P$2"/>
 <contactref element="U$7" pad="P$2"/>
+<polygon width="0.1524" layer="1" thermals="no">
+<vertex x="11" y="71"/>
+<vertex x="11" y="61"/>
+<vertex x="68" y="61"/>
+<vertex x="68" y="71"/>
+</polygon>
+<wire x1="44" y1="55" x2="44.85" y2="55" width="0" layer="19" extent="1-1"/>
+<wire x1="44.85" y1="49" x2="44.85" y2="55" width="0" layer="19" extent="1-1"/>
+<wire x1="44" y1="49" x2="44.85" y2="49" width="0" layer="19" extent="1-1"/>
+<wire x1="44.85" y1="43" x2="44.85" y2="49" width="0" layer="19" extent="1-1"/>
+<wire x1="44" y1="43" x2="44.85" y2="43" width="0" layer="19" extent="1-1"/>
+<wire x1="39" y1="37.85" x2="41" y2="43" width="0" layer="19" extent="1-1"/>
+<wire x1="31" y1="50.85" x2="41" y2="49" width="0" layer="19" extent="1-1"/>
+<wire x1="38" y1="65.8455" x2="41" y2="55" width="0" layer="19" extent="1-1"/>
 </signal>
 <signal name="N$6">
@@
 <contactref element="U$4" pad="7"/>
 <contactref element="J2" pad="BATT"/>
-<wire x1="8.575" y1="49" x2="5" y2="45.425" width="2" layer="1"/>
-<wire x1="5" y1="45.425" x2="5" y2="34.8455" width="2" layer="1"/>
+<polygon width="0.1524" layer="1" thermals="no">
+<vertex x="0" y="32"/>
+<vertex x="9" y="32"/>
+<vertex x="9" y="41"/>
+<vertex x="15" y="41"/>
+<vertex x="15" y="55"/>
+<vertex x="0" y="55"/>
+</polygon>
 </signal>
 <signal name="P1">
 <contactref element="U$4" pad="6"/>
 <contactref element="U$6" pad="P$1"/>
-<wire x1="4.92" y1="64" x2="6.425" y2="64" width="1.55" layer="1"/>
-<wire x1="6.425" y1="64" x2="21.425" y2="49" width="1.55" layer="1"/>
+<polygon width="0.1524" layer="1" thermals="no">
+<vertex x="16" y="42"/>
+<vertex x="27" y="42"/>
+<vertex x="27" y="60"/>
+<vertex x="10" y="60"/>
+<vertex x="10" y="71"/>
+<vertex x="0" y="71"/>
+<vertex x="0" y="56"/>
+<vertex x="16" y="56"/>
+</polygon>
 </signal>
 <signal name="P2">

Commit message: made some revisions
fixd 24V fuse
added 5A fuse
labled LEDs
Parts:
- removed D1, D2, D3: LED-SMD, RoboJackets-LEDs:CHIP-LED0603
- added +24V, +3.3V, +5V: LED-SMD, RoboJackets-LEDs:CHIP-LED0603
- added U$8: ERB-RE5R00V, CurrentSensing:ERB-RE5R00V
- U$6, U$7: value 3550 -> 3550(2)
- moved R5 33.6 mm to (14.0, 21.0), turned to 0 degrees
- moved J1 12.0 mm to (39.0, 82.0)
- moved R3 7.62 mm to (14.0, 16.0), turned to 0 degrees
- moved U$6 7.28 mm to (12.0, 71.0)
- moved U$7 6.08 mm to (68.0, 70.0)
- moved R4 6.04 mm to (14.0, 18.4), turned to 0 degrees
- moved C10 5.39 mm to (43.6, 26.0)
- moved C7 5.00 mm to (51.0, 24.0)
- moved C15 4.24 mm to (45.0, 40.0), turned to 180 degrees
- moved C8 3.61 mm to (15.0, 13.0)
- moved C9 3.61 mm to (25.0, 13.0)
- moved U7 3.61 mm to (20.0, 13.0)
- moved C12 3.00 mm to (42.0, 37.0)
- moved C11 1.00 mm to (48.0, 56.0)
- moved C13 1.00 mm to (48.0, 50.0)
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Connections:
- new net N$10: C10.1, C7.1, U$1.P$2, U$8.P$1, U2.6
- net +24V: now also U$6.P$4, U$7.P$4
- net +5V: now also U$8.P$2; no longer C10.1, C7.1, U$1.P$2, U2.6
- net GND: now also +24V.C, +3.3V.C, +5V.C; no longer D1.C, D2.C, D3.C
- net N$5: now also +3.3V.A; no longer D1.A
- net N$8: now also +5V.A; no longer D2.A
- net N$9: now also +24V.A; no longer D3.A
- net P1: now also U$6.P$3
- net P2: now also U$7.P$3
Routing:
- net N2: track 23.5 -> 0.00 mm
- net P2: track 16.1 -> 0.00 mm
- net +24V: track 9.00 -> 20.6 mm, vias 6 -> 2
- net GND: track 68.4 -> 61.3 mm
- net +5V: track 6.89 -> 0.00 mm, vias 2 -> 0
- net N$9: track 2.04 -> 8.81 mm
- net N$8: track 2.04 -> 8.70 mm
- net N$5: track 2.04 -> 8.40 mm
- net N$7: track 3.04 -> 6.72 mm
- net +3V3: track 32.0 -> 35.1 mm
- net N$6: track 20.8 -> 21.8 mm, vias 0 -> 2
- added copper zone on layer 1, net N$10
- added copper zone on layer 1, net N2
- added copper zone on layer 1, net P2
Other:
- board size 80 x 71 mm -> 80 x 82 mm

Commit message: made some small revisions on the board and silkscreen
Parts:
- moved C7 13.0 mm to (38.0, 24.0), turned to 180 degrees
- moved C10 6.76 mm to (39.0, 31.0), turned to 180 degrees
- moved U$7 2.83 mm to (70.0, 72.0), turned to 0 degrees
- moved U$6 1.41 mm to (13.0, 72.0)
- moved U$1 0.23 mm to (28.2, 33.2)
Connections:
- net +24V: now also U$7.P$1, U$7.P$3; no longer U$7.P$2, U$7.P$4
- net P2: now also U$7.P$2, U$7.P$4; no longer U$7.P$1, U$7.P$3
Routing:
- net GND: track 61.3 -> 66.1 mm
- net AIN1: track 35.9 -> 38.2 mm
- net VREF: track 68.3 -> 69.5 mm
- net N$5: track 8.40 -> 9.09 mm
