File: CurrentSensingBoard/powerDistribution.brd (EAGLE design)
At the start: 80 x 82 mm, 46 parts, among them J1 XT-60BATT_LABEL, J2 XT-60BATT_LABEL, J3 XT-60BATT_LABEL, U1 MAX11635EEE+, U2 LM2678SX-5.0/NOPB, U7 AP2114H-3.3TRG1

Commit message: cleaned up power planes a bit
Connections:
- net N2: now also U$5.6; no longer U$5.7
- net P2: now also U$5.7; no longer U$5.6
Routing:
- net +24V: track 20.6 -> 16.8 mm
- net AIN1: track 38.2 -> 40.2 mm

Commit message: fixed silkscreen somemore
Parts:
- removed U$3: (no value), RoboJackets-Aesthetics:ROBOBUZZ_0.4X
- added D1: SD2114S040S8R0, CurrentSensing:SD2114S040S8R0
- added L1: 22uH, CurrentSensing:INDUCTOR22
- added U3, U4: CQ2065, CurrentSensing:CQ2065
- J2, J3: value XT-60BATT_LABEL -> CONNECTOR; device RoboJackets-Connectors:XT-60 -> CurrentSensing:XT-60
- U$1: value 22uH -> (none); device CurrentSensing:INDUCTOR22 -> RoboJackets-Aesthetics:ROBOJACKETS
- U$2: value SD2114S040S8R0 -> (none); device CurrentSensing:SD2114S040S8R0 -> RoboJackets-Aesthetics:ROBOBUZZ_0.2X
- U$4: value CQ2065 -> (none); device CurrentSensing:CQ2065 -> RoboJackets-Aesthetics:ROBOBUZZ_0.4X
- U$5: value CQ2065 -> (none); device CurrentSensing:CQ2065 -> RoboJackets-Aesthetics:ROBOBUZZ_0.6X
- moved U$4 67.9 mm to (67.5, 5.90)
- moved U$2 49.7 mm to (62.0, 6.00), turned to 0 degrees
- moved U$5 44.1 mm to (75.0, 6.00)
- moved U$1 39.4 mm to (51.0, 1.00)
- renumbered U$6 to XF1, U$7 to XF2, U$8 to F1
Connections:
- net +5V: now also U3.2, U4.2; no longer U$4.2, U$5.2
- net GND: now also D1.1, U3.1, U3.3, U3.5, U4.1, U4.3, U4.5; no longer U$2.1, U$4.1, U$4.3, U$4.5, U$5.1, U$5.3, U$5.5
- net N$1: now also U4.4; no longer U$5.4
- net N$10: now also L1.P$2; no longer U$1.P$2
- net N$3: now also U3.4; no longer U$4.4
- net N$6: now also D1.2, L1.P$1; no longer U$1.P$1, U$2.2
- net N1: now also U3.7; no longer U$4.7
- net N2: now also U4.6; no longer U$5.6
- net P1: now also U3.6; no longer U$4.6
- net P2: now also U4.7; no longer U$5.7
Routing:
- net GND: track 66.0 -> 65.4 mm
Other:
- board text added: "Power Distribution Board v1.0"
