File: CurrentSensingBoard/powerDistribution.sch (EAGLE design)
At the start: 20 parts

Commit message: repurpose current sensing board
current sengins board becomes power distribution board
using stm32 instead of nano
Parts:
- added U$4: STM32F0, STM32F031C4T6:STM32F0
Changed lines of the file:
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@@
 <part name="P+8" library="supply1" library_urn="urn:adsk.eagle:library:371" deviceset="+5V" device=""/>
 <part name="GND10" library="supply1" library_urn="urn:adsk.eagle:library:371" deviceset="GND" device=""/>
+<part name="U$4" library="STM32F031C4T6" deviceset="STM32F0" device=""/>
 </parts>
 <sheets>
@@
 <attribute name="VALUE" x="143.002" y="82.296" size="1.778" layer="96"/>
 </instance>
+<instance part="U$4" gate="G$1" x="-66.04" y="40.64" smashed="yes">
+<attribute name="NAME" x="-71.374" y="72.39" size="1.778" layer="95"/>
+<attribute name="VALUE" x="-71.12" y="5.08" size="1.778" layer="96"/>
+</instance>
 </instances>

Commit message: switched back to Nano
Parts:
- removed 12-BIT_ADC: MAX11634EEE+T21-0055H_16-L, CurrentSensing:MAX11634EEE+T21-0055H_16-L
- removed SENSOR_0, SENSOR_1: CQ2065, CurrentSensing:CQ2065
- added C8, C9: 4.7uF, rcl:C-USC0603
- added R10, R14: RF1, rcl:R-US_R0603
- added R11, R12, R7, R8: 39k, rcl:R-US_R0603
- added R13, R9: 20k, rcl:R-US_R0603
- added U$5: CQ2065, CurrentSensing:CQ2065
- added U1: MAX11635EEE+, CurrentSensing:MAX11635EEE+
- added U7: AP2114H-3.3TRG1, Gucci_ControlBoard:AP2114H-3.3TRG1
- C1: value CF0 -> 0.1uF
- C2: value CF1 -> 0.1uF
- C3, C4: value 0.1uF -> CF1
- R1: value RF0 -> 20k
- R2: value RF1 -> 20k
- U$4: value STM32F0 -> CQ2065; device STM32F031C4T6:STM32F0 -> CurrentSensing:CQ2065
Connections:
- removed net N$5: R1.1, SENSOR_0.VOUT
- new net N$1: R1.1, U$5.VOUT
- new net N$2: R10.2, R2.2, R7.2
- new net N$4: R1.2, R11.2, R14.2
- new net VDD: C6.1, U1.VDD
- new net VREF: R12.1, R13.1, R8.1, R9.1, U1.REF+
- new net VSS: C1.1, C2.1, C3.2, C4.2, R11.1, R12.2, R7.1, R8.2, U$4.DATA_IO, U$4.SCLK, U$4.VSS, U$5.DATA_IO, U$5.SCLK, U$5.VSS, U1.GND
- net !CNVST!: now also U1.!CNVST; no longer 12-BIT_ADC.!CNVST
- net !CS!: now also U1.!CS; no longer 12-BIT_ADC.!CS
- net !EOC!: now also U1.!EOC; no longer 12-BIT_ADC.!EOC
- net +3V3: now also C9.1, U7.EPAD, U7.VOUT
- net +5V: now also C1.2, C2.2, C8.1, R13.2, R9.2, U$4.VDD, U$5.VDD, U7.VIN; no longer 12-BIT_ADC.REF+, 12-BIT_ADC.VDD, C3.2, C4.2, C6.1, SENSOR_0.VDD, SENSOR_1.VDD
- net AIN0: now also C3.1, R10.1, U1.AIN0; no longer 12-BIT_ADC.AIN0, C1.1, R1.2
- net AIN1: now also C4.1, R14.1, U1.AIN1; no longer 12-BIT_ADC.AIN1, C2.1, R2.2
- net DIN: now also U1.DIN; no longer 12-BIT_ADC.DIN
- net DOUT: now also U1.DOUT; no longer 12-BIT_ADC.DOUT
- net GND: now also C8.2, C9.2, U1.REF-, U7.GND; no longer 12-BIT_ADC.GND, 12-BIT_ADC.REF-, C1.2, C2.2, C3.1, C4.1, SENSOR_0.DATA_IO, SENSOR_0.SCLK, SENSOR_0.VSS, SENSOR_1.DATA_IO, SENSOR_1.SCLK, SENSOR_1.VSS
- net N$3: now also U$4.VOUT; no longer SENSOR_1.VOUT
- net SCLK: now also U1.SCLK; no longer 12-BIT_ADC.SCLK
Other:
- note added: "Voltage Regulator"
- moved on the sheet: C1, C2, C3, C4, C5, C6, Q1, Q2, R1, R2, R3, R4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

Commit message: added data line connector
Parts:
- removed C7: 0.1uF, rcl:C-USC0603
- removed Q1, Q2: (no value), Adafruit FET 4-Channel Shifter:ADAFRUIT_MOSFET-NREFLOW
- removed R3, R4, R5, R6: 10k, rcl:R-US_R0603
- removed U$1: NANO, I'mRADIOactive:NANO
- removed U$2: MOLEX_1.25MM_4PIN_90, Kirbi_ControlBoard:MOLEX_1.25MM_4PIN_90
- added JP1: (no value), pinhead:PINHD-1X8/90
Connections:
- removed net DIN: U$1.D4, U1.DIN
- removed net DOUT: U$1.D5, U1.DOUT
- removed net RX_NANO: Q1.D, R6.2, U$1.RX1
- removed net RX_TEENSY: Q2.S, R3.2, U$2.3
- removed net TX_NANO: Q2.D, R4.2, U$1.TX0
- removed net TX_TEENSY: Q1.S, R5.2, U$2.2
- new net MISO: JP1.5, U1.DOUT
- new net MOSI: JP1.4, U1.DIN
- net !CNVST!: now also JP1.2; no longer U$1.D7
- net !CS!: now also JP1.7; no longer U$1.D2
- net !EOC!: now also JP1.6; no longer U$1.D6
- net +3V3: now also C5.1, C6.1; no longer Q1.G, Q2.G, R3.1, R5.1, U$1.3.3V
- net +5V: now also JP1.1; no longer C5.1, C7.1, R4.1, R6.1, U$1.RAW, U$2.4
- net GND: now also JP1.8; no longer C7.2, U$1.GND, U$1.GND2, U$2.1
- net SCLK: now also JP1.3; no longer U$1.D3
- net VDD: no longer C6.1
Other:
- note removed: "Arduino Nano Microcontroller"
- note removed: "Level Shifters"
- moved on the sheet: C5, C6, C8, C9, U1, U7

Commit message: put in 24v-5v
Parts:
- added C10, C11, C13, C14, C7: 15uF, rcl:C-USC0603
- added C12: 47uF, rcl:C-USC0603
- added C15: 100nF, rcl:C-USC0603
- added J1: XT-60BATT_LABEL, RoboJackets-Connectors:XT-60BATT_LABEL
- added U$1: 22uH, CurrentSensing:7447709220
- added U$2: MBRD835LT4G, CurrentSensing:MBRD835LT4G
- added U2: LM2678SX-5.0/NOPB, CurrentSensing:LM2678SX-5.0/NOPB
Connections:
- new net +24V: J1.1
- new net CB: C15.1, U2.CB
- new net FB: C13.1, C14.1, U$1.2, U2.FB
- new net N$5: C5.1
- new net SW: C15.2, U$1.1, U$2.4, U2.SW
- new net VIN: C10.1, C11.1, C12.1, C7.1, U2.VIN
- net +3V3: no longer C5.1
- net +5V: now also U2.ON/~OFF
- net GND: now also C1.1, C10.2, C11.2, C12.2, C13.2, C14.2, C4.2, C7.2, J1.2, R11.1, R12.2, U$2.1, U$2.3, U$5.DATA_IO, U$5.SCLK, U$5.VSS, U2.GND
- net VSS: no longer C1.1, C4.2, R11.1, R12.2, U$5.DATA_IO, U$5.SCLK, U$5.VSS

Commit message: added capictors
Parts:
- removed C10, C11, C13, C14, C7: 15uF, rcl:C-USC0603
- added U$10, U$8, U$9: 15uF, CurrentSensing:TR3E156M050C0300
- added U$6, U$7: 180uF, CurrentSensing:860010373009
- C12: value 47uF -> 0.47uF
Connections:
- net FB: now also U$6.P$1, U$7.P$1; no longer C13.1, C14.1
- net GND: now also U$10.P$2, U$6.P$2, U$7.P$2, U$8.P$2, U$9.P$2; no longer C10.2, C11.2, C13.2, C14.2, C7.2
- net VIN: now also U$10.P$1, U$8.P$1, U$9.P$1; no longer C10.1, C11.1, C7.1
Other:
- moved on the sheet: C12

Commit message: fixed Caleb's mess
changed caps and diode symbols
24v regulator footprint was weird
24v regulator schematic looking clean now
deleted unnecessary stuff in library
Parts:
- removed U$10, U$8, U$9: 15uF, CurrentSensing:TR3E156M050C0300
- removed U$6, U$7: 180uF, CurrentSensing:860010373009
- added C10, C7: 180uF, CurrentSensing:860010373009
- added C11, C13, C14: 15uF, CurrentSensing:TR3E156M050C0300
Connections:
- net CB renamed N$7
- removed net FB: U$1.2, U$6.P$1, U$7.P$1, U2.FB
- removed net SW: C15.2, U$1.1, U$2.4, U2.SW
- removed net VIN: C12.1, U$10.P$1, U$8.P$1, U$9.P$1, U2.VIN
- new net N$6: C15.2, U$1.1, U$2.C, U2.SW
- net +24V: now also C11.+, C12.1, C13.+, C14.+, U2.VIN
- net +5V: now also C10.+, C7.+, U$1.2, U2.FB; no longer U2.ON/~OFF
- net GND: now also C10.-, C11.-, C13.-, C14.-, C7.-, U$2.A; no longer U$10.P$2, U$2.1, U$2.3, U$6.P$2, U$7.P$2, U$8.P$2, U$9.P$2
Other:
- moved on the sheet: C12, C15, J1, U$1

Commit message: added fuseholders
Parts:
- added F1, F2: (no value), RoboJackets-Fuses:FUSEHOLDER_3549_X2
Connections:
- new net MOTOR1: F1.1
- new net MOTOR2: F2.1
- new net N1: U$4.I_N
- new net N2: U$5.I_N
- new net P1: F1.2, U$4.I_P
- new net P2: F2.2, U$5.I_P
Other:
- moved on the sheet: C2, C3, R10, R2, R7, R8, R9

Commit message: started layout of power board
Parts:
- added J2, J3: XT-60BATT_LABEL, RoboJackets-Connectors:XT-60BATT_LABEL
Connections:
- removed net MOTOR1: F1.1
- removed net MOTOR2: F2.1
- removed net N$5: C5.1
- removed net VDD: U1.VDD
- removed net VSS: C2.1, C3.2, R7.1, R8.2, U$4.DATA_IO, U$4.SCLK, U$4.VSS, U1.GND
- net +24V: now also F1.1, F2.1
- net +3V3: now also U1.VDD
- net GND: now also C2.1, C3.2, J2.2, J3.2, R7.1, R8.2, U$4.DATA_IO, U$4.SCLK, U$4.VSS, U1.GND
- net N1: now also J2.1
- net N2: now also J3.1
- net VREF: now also C5.1
Other:
- moved on the sheet: C5, C6, F1, F2
