File: CurrentSensingBoard/powerDistribution.sch (EAGLE design)
At the start: 38 parts, among them J1 XT-60BATT_LABEL, J2 XT-60BATT_LABEL, J3 XT-60BATT_LABEL, U1 MAX11635EEE+, U2 LM2678SX-5.0/NOPB, U7 AP2114H-3.3TRG1

Commit message: added power LEDs
Parts:
- added D1, D2, D3: LED-SMD, RoboJackets-LEDs:LED-SMD
- added R3: 100Ω, rcl:R-US_R0603
- added R4: 200Ω, rcl:R-US_R0603
- added R5: 1200Ω, rcl:R-US_R0603
- U$2: value MBRD835LT4G -> SD2114S040S8R0; device CurrentSensing:MBRD835LT4G -> CurrentSensing:SD2114S040S8R0
Connections:
- new net N$5: D1.A, R3.1
- new net N$8: D2.A, R4.1
- new net N$9: D3.A, R5.1
- net +24V: now also R5.2
- net +3V3: now also R3.2
- net +5V: now also R4.2
- net GND: now also D1.K, D2.K, D3.K
Other:
- note added: "Motor & Battery Connector"
- moved on the sheet: C8, C9, J1, J2, J3, U7

Commit message: started routing
Connections:
- new net N$14: JP1.6
- net !EOC!: now also JP1.3; no longer JP1.6
- net MISO: now also JP1.4; no longer JP1.5
- net MOSI: now also JP1.5; no longer JP1.4
- net SCLK: no longer JP1.3
Changed lines of the file:
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@@
 </segment>
 <segment>
-<label x="20.32" y="127" size="1.27" layer="95" rot="R180" xref="yes"/>
-<pinref part="JP1" gate="A" pin="6"/>
-<wire x1="20.32" y1="127" x2="26.67" y2="127" width="0.1524" layer="91"/>
+<label x="20.32" y="134.62" size="1.27" layer="95" rot="R180" xref="yes"/>
+<pinref part="JP1" gate="A" pin="3"/>
+<wire x1="20.32" y1="134.62" x2="26.67" y2="134.62" width="0.1524" layer="91"/>
 </segment>
 </net>
@@
 </segment>
 <segment>
+<label x="20.32" y="132.08" size="1.27" layer="95" rot="R180" xref="yes"/>
+<pinref part="JP1" gate="A" pin="4"/>
+<wire x1="20.32" y1="132.08" x2="26.67" y2="132.08" width="0.1524" layer="91"/>
+</segment>
+</net>
+<net name="MOSI" class="0">
+<segment>
+<pinref part="U1" gate="A" pin="DIN"/>
+<wire x1="85.09" y1="186.69" x2="87.63" y2="186.69" width="0.1524" layer="91"/>
+<label x="87.63" y="186.69" size="1.27" layer="95" xref="yes"/>
+</segment>
+<segment>
 <label x="20.32" y="129.54" size="1.27" layer="95" rot="R180" xref="yes"/>
 <pinref part="JP1" gate="A" pin="5"/>
@@
 </segment>
 </net>
-<net name="MOSI" class="0">
-<segment>
-<pinref part="U1" gate="A" pin="DIN"/>
-<wire x1="85.09" y1="186.69" x2="87.63" y2="186.69" width="0.1524" layer="91"/>
-<label x="87.63" y="186.69" size="1.27" layer="95" xref="yes"/>
-</segment>
-<segment>
-<label x="20.32" y="132.08" size="1.27" layer="95" rot="R180" xref="yes"/>
-<pinref part="JP1" gate="A" pin="4"/>
-<wire x1="20.32" y1="132.08" x2="26.67" y2="132.08" width="0.1524" layer="91"/>
-</segment>
-</net>
 <net name="SCLK" class="0">
 <segment>
@@
 <wire x1="85.09" y1="184.15" x2="87.63" y2="184.15" width="0.1524" layer="91"/>
 <label x="87.63" y="184.15" size="1.27" layer="95" xref="yes"/>
-</segment>
-<segment>
-<label x="20.32" y="134.62" size="1.27" layer="95" rot="R180" xref="yes"/>
-<pinref part="JP1" gate="A" pin="3"/>
-<wire x1="20.32" y1="134.62" x2="26.67" y2="134.62" width="0.1524" layer="91"/>
 </segment>
 </net>
@@
 </segment>
 </net>
+<net name="N$14" class="0">
+<segment>
+<pinref part="JP1" gate="A" pin="6"/>
+<wire x1="20.32" y1="127" x2="26.67" y2="127" width="0.1524" layer="91"/>
+<label x="20.32" y="127" size="1.27" layer="95" rot="R180" xref="yes"/>
+</segment>
+</net>

Commit message: updated board layout and routing
Parts:
- removed F1, F2: (no value), RoboJackets-Fuses:FUSEHOLDER_3549_X2
- added U$6, U$7: 3550, CurrentSensing:3550
Connections:
- removed net N$14: JP1.6
- net +24V: now also U$6.2, U$7.2; no longer F1.1, F2.1
- net P1: now also U$6.1; no longer F1.2
- net P2: now also U$7.1; no longer F2.2
- net SCLK: now also JP1.6
Other:
- note added: "Status LEDs"
- moved on the sheet: C10, C11, C12, C13, C14, C15, C7, C8, C9, D1, D2, D3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

Commit message: helped Caleb
Other:
- note added: "Voltage Regulators"
- note removed: "Voltage Regulator"
Changed lines of the file:
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@@
 <wire x1="170.18" y1="2.54" x2="170.18" y2="45.72" width="0.1524" layer="97" style="shortdash"/>
 <wire x1="147.574" y1="165.1" x2="148.082" y2="165.1" width="0.1524" layer="97" style="shortdash"/>
-<text x="8.89" y="85.09" size="5.08" layer="97" font="vector" ratio="12">Voltage Regulator</text>
+<text x="8.89" y="85.09" size="5.08" layer="97" font="vector" ratio="12">Voltage Regulators</text>
 <wire x1="170.18" y1="45.72" x2="170.18" y2="95.25" width="0.1524" layer="97" style="shortdash"/>
 <text x="100.584" y="147.066" size="6.35" layer="97" font="vector" ratio="12" distance="12" rot="MR0">Motor &amp; Battery Connector</text>

Commit message: made some revisions
fixd 24V fuse
added 5A fuse
labled LEDs
Parts:
- added U$8: ERB-RE5R00V, CurrentSensing:ERB-RE5R00V
- U$6, U$7: value 3550 -> 3550(2); device CurrentSensing:3550 -> CurrentSensing:3550(2)
- renumbered D1 to +3.3V, D2 to +5V, D3 to +24V
Connections:
- new net N$10: C10.+, C7.+, U$1.2, U$8.1, U2.FB
- net +5V: now also U$8.2; no longer C10.+, C7.+, U$1.2, U2.FB
Changed lines of the file:
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@@
 <part name="R4" library="rcl" library_urn="urn:adsk.eagle:library:334" deviceset="R-US_" device="R0603" package3d_urn="urn:adsk.eagle:package:23555/3" value="200Ω"/>
 <part name="R5" library="rcl" library_urn="urn:adsk.eagle:library:334" deviceset="R-US_" device="R0603" package3d_urn="urn:adsk.eagle:package:23555/3" value="1200Ω"/>
-<part name="D1" library="RoboJackets-LEDs" deviceset="LED-SMD" device=""/>
-<part name="D2" library="RoboJackets-LEDs" deviceset="LED-SMD" device=""/>
-<part name="D3" library="RoboJackets-LEDs" deviceset="LED-SMD" device=""/>
+<part name="+3.3V" library="RoboJackets-LEDs" deviceset="LED-SMD" device=""/>
+<part name="+5V" library="RoboJackets-LEDs" deviceset="LED-SMD" device=""/>
+<part name="+24V" library="RoboJackets-LEDs" deviceset="LED-SMD" device=""/>
 <part name="GND13" library="supply1" library_urn="urn:adsk.eagle:library:371" deviceset="GND" device=""/>
 <part name="GND14" library="supply1" library_urn="urn:adsk.eagle:library:371" deviceset="GND" device=""/>
 <part name="GND15" library="supply1" library_urn="urn:adsk.eagle:library:371" deviceset="GND" device=""/>
 <part name="U$2" library="CurrentSensing" deviceset="SD2114S040S8R0" device=""/>
-<part name="U$6" library="CurrentSensing" deviceset="3550" device=""/>
-<part name="U$7" library="CurrentSensing" deviceset="3550" device=""/>
+<part name="U$6" library="CurrentSensing" deviceset="3550(2)" device=""/>
+<part name="U$7" library="CurrentSensing" deviceset="3550(2)" device=""/>
+<part name="U$8" library="CurrentSensing" deviceset="ERB-RE5R00V" device=""/>
 </parts>
 <sheets>
@@
 <attribute name="VALUE" x="111.76" y="7.62" size="1.778" layer="96"/>
 </instance>
-<instance part="P+6" gate="1" x="138.43" y="44.45" smashed="yes">
-<attribute name="VALUE" x="143.51" y="45.72" size="1.778" layer="96" rot="R180"/>
+<instance part="P+6" gate="1" x="138.43" y="50.8" smashed="yes">
+<attribute name="VALUE" x="143.51" y="52.07" size="1.778" layer="96" rot="R180"/>
 </instance>
 <instance part="C15" gate="G$1" x="106.68" y="33.02" smashed="yes" rot="R90">
@@
 <attribute name="VALUE" x="155.702" y="123.19" size="1.778" layer="96" rot="R90"/>
 </instance>
-<instance part="D1" gate="G$1" x="115.57" y="114.3" smashed="yes">
+<instance part="+3.3V" gate="G$1" x="115.57" y="114.3" smashed="yes">
 <attribute name="NAME" x="118.11" y="116.84" size="1.778" layer="95"/>
 <attribute name="VALUE" x="118.11" y="114.3" size="1.778" layer="96"/>
 </instance>
-<instance part="D2" gate="G$1" x="134.62" y="114.3" smashed="yes">
+<instance part="+5V" gate="G$1" x="134.62" y="114.3" smashed="yes">
 <attribute name="NAME" x="137.16" y="116.84" size="1.778" layer="95"/>
 <attribute name="VALUE" x="137.16" y="114.3" size="1.778" layer="96"/>
 </instance>
-<instance part="D3" gate="G$1" x="152.4" y="114.3" smashed="yes">
+<instance part="+24V" gate="G$1" x="152.4" y="114.3" smashed="yes">
 <attribute name="NAME" x="154.94" y="116.84" size="1.778" layer="95"/>
 <attribute name="VALUE" x="154.94" y="114.3" size="1.778" layer="96"/>
@@
 <attribute name="NAME" x="204.47" y="124.46" size="1.778" layer="95"/>
 <attribute name="VALUE" x="204.47" y="119.38" size="1.778" layer="96" align="top-left"/>
+</instance>
+<instance part="U$8" gate="G$1" x="138.43" y="43.18" smashed="yes" rot="R90">
+<attribute name="NAME" x="135.89" y="40.64" size="1.778" layer="95" rot="R90"/>
+<attribute name="VALUE" x="140.97" y="40.64" size="1.778" layer="96" rot="R90" align="top-left"/>
 </instance>
 </instances>
@@
 </segment>
 <segment>
-<pinref part="D1" gate="G$1" pin="K"/>
+<pinref part="+3.3V" gate="G$1" pin="K"/>
 <pinref part="GND13" gate="1" pin="GND"/>
 <wire x1="115.57" y1="111.76" x2="115.57" y2="109.22" width="0.1524" layer="91"/>
 </segment>
 <segment>
-<pinref part="D2" gate="G$1" pin="K"/>
+<pinref part="+5V" gate="G$1" pin="K"/>
 <pinref part="GND14" gate="1" pin="GND"/>
 <wire x1="134.62" y1="111.76" x2="134.62" y2="109.22" width="0.1524" layer="91"/>
 </segment>
 <segment>
-<pinref part="D3" gate="G$1" pin="K"/>
+<pinref part="+24V" gate="G$1" pin="K"/>
 <pinref part="GND15" gate="1" pin="GND"/>
 <wire x1="152.4" y1="111.76" x2="152.4" y2="109.22" width="0.1524" layer="91"/>
@@
 </segment>
 <segment>
-<pinref part="U$1" gate="G$1" pin="2"/>
-<wire x1="135.89" y1="27.94" x2="138.43" y2="27.94" width="0.1524" layer="91"/>
-<pinref part="U2" gate="G$1" pin="FB"/>
-<wire x1="138.43" y1="27.94" x2="138.43" y2="38.1" width="0.1524" layer="91"/>
-<wire x1="138.43" y1="38.1" x2="99.06" y2="38.1" width="0.1524" layer="91"/>
-<pinref part="P+6" gate="1" pin="+5V"/>
-<wire x1="138.43" y1="41.91" x2="138.43" y2="38.1" width="0.1524" layer="91"/>
-<junction x="138.43" y="38.1"/>
-<pinref part="C7" gate="G$1" pin="+"/>
-<wire x1="138.43" y1="24.13" x2="138.43" y2="27.94" width="0.1524" layer="91"/>
-<junction x="138.43" y="27.94"/>
-<wire x1="138.43" y1="27.94" x2="148.59" y2="27.94" width="0.1524" layer="91"/>
-<pinref part="C10" gate="G$1" pin="+"/>
-<wire x1="148.59" y1="27.94" x2="148.59" y2="24.13" width="0.1524" layer="91"/>
-</segment>
-<segment>
 <pinref part="P+10" gate="1" pin="+5V"/>
 <pinref part="R4" gate="G$1" pin="2"/>
 <wire x1="134.62" y1="137.16" x2="134.62" y2="132.08" width="0.1524" layer="91"/>
+</segment>
+<segment>
+<pinref part="U$8" gate="G$1" pin="2"/>
+<wire x1="138.43" y1="45.72" x2="138.43" y2="48.26" width="0.1524" layer="91"/>
+<pinref part="P+6" gate="1" pin="+5V"/>
 </segment>
 </net>
@@
 <pinref part="P+7" gate="1" pin="+24V"/>
 <wire x1="214.63" y1="191.77" x2="214.63" y2="194.31" width="0.1524" layer="91"/>
+<wire x1="209.55" y1="191.77" x2="214.63" y2="191.77" width="0.1524" layer="91"/>
 <pinref part="U$6" gate="G$1" pin="2"/>
-<wire x1="209.55" y1="191.77" x2="214.63" y2="191.77" width="0.1524" layer="91"/>
 </segment>
 <segment>
 <pinref part="P+8" gate="1" pin="+24V"/>
 <wire x1="214.63" y1="121.92" x2="214.63" y2="124.46" width="0.1524" layer="91"/>
+<wire x1="209.55" y1="121.92" x2="214.63" y2="121.92" width="0.1524" layer="91"/>
 <pinref part="U$7" gate="G$1" pin="2"/>
-<wire x1="209.55" y1="121.92" x2="214.63" y2="121.92" width="0.1524" layer="91"/>
 </segment>
 <segment>
@@
 <pinref part="U$4" gate="G$1" pin="I_P"/>
 <wire x1="184.15" y1="189.23" x2="184.15" y2="191.77" width="0.1524" layer="91"/>
+<wire x1="184.15" y1="191.77" x2="204.47" y2="191.77" width="0.1524" layer="91"/>
 <pinref part="U$6" gate="G$1" pin="1"/>
-<wire x1="184.15" y1="191.77" x2="204.47" y2="191.77" width="0.1524" layer="91"/>
 </segment>
 </net>
@@
 <pinref part="U$5" gate="G$1" pin="I_P"/>
 <wire x1="184.15" y1="119.38" x2="184.15" y2="121.92" width="0.1524" layer="91"/>
+<wire x1="184.15" y1="121.92" x2="204.47" y2="121.92" width="0.1524" layer="91"/>
 <pinref part="U$7" gate="G$1" pin="1"/>
-<wire x1="184.15" y1="121.92" x2="204.47" y2="121.92" width="0.1524" layer="91"/>
 </segment>
 </net>
@@
 <segment>
 <pinref part="R3" gate="G$1" pin="1"/>
-<pinref part="D1" gate="G$1" pin="A"/>
+<pinref part="+3.3V" gate="G$1" pin="A"/>
 <wire x1="115.57" y1="121.92" x2="115.57" y2="119.38" width="0.1524" layer="91"/>
 </segment>
@@
 <segment>
 <pinref part="R4" gate="G$1" pin="1"/>
-<pinref part="D2" gate="G$1" pin="A"/>
+<pinref part="+5V" gate="G$1" pin="A"/>
 <wire x1="134.62" y1="121.92" x2="134.62" y2="119.38" width="0.1524" layer="91"/>
 </segment>
@@
 <segment>
 <pinref part="R5" gate="G$1" pin="1"/>
-<pinref part="D3" gate="G$1" pin="A"/>
+<pinref part="+24V" gate="G$1" pin="A"/>
 <wire x1="152.4" y1="121.92" x2="152.4" y2="119.38" width="0.1524" layer="91"/>
 </segment>
 </net>
+<net name="N$10" class="0">
+<segment>
+<pinref part="U$1" gate="G$1" pin="2"/>
+<wire x1="135.89" y1="27.94" x2="138.43" y2="27.94" width="0.1524" layer="91"/>
+<pinref part="U2" gate="G$1" pin="FB"/>
+<wire x1="138.43" y1="27.94" x2="138.43" y2="38.1" width="0.1524" layer="91"/>
+<wire x1="138.43" y1="38.1" x2="99.06" y2="38.1" width="0.1524" layer="91"/>
+<pinref part="C7" gate="G$1" pin="+"/>
+<wire x1="138.43" y1="24.13" x2="138.43" y2="27.94" width="0.1524" layer="91"/>
+<junction x="138.43" y="27.94"/>
+<wire x1="138.43" y1="27.94" x2="148.59" y2="27.94" width="0.1524" layer="91"/>
+<pinref part="C10" gate="G$1" pin="+"/>
+<wire x1="148.59" y1="27.94" x2="148.59" y2="24.13" width="0.1524" layer="91"/>
+<pinref part="U$8" gate="G$1" pin="1"/>
+<wire x1="138.43" y1="40.64" x2="138.43" y2="38.1" width="0.1524" layer="91"/>
+</segment>
+</net>

Commit message: made some small revisions on the board and silkscreen
Connections:
- net +24V: now also U$7.1; no longer U$7.2
- net P2: now also U$7.2; no longer U$7.1
Changed lines of the file:
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@@
 <part name="GND15" library="supply1" library_urn="urn:adsk.eagle:library:371" deviceset="GND" device=""/>
 <part name="U$2" library="CurrentSensing" deviceset="SD2114S040S8R0" device=""/>
+<part name="U$8" library="CurrentSensing" deviceset="ERB-RE5R00V" device=""/>
 <part name="U$6" library="CurrentSensing" deviceset="3550(2)" device=""/>
 <part name="U$7" library="CurrentSensing" deviceset="3550(2)" device=""/>
-<part name="U$8" library="CurrentSensing" deviceset="ERB-RE5R00V" device=""/>
 </parts>
 <sheets>
@@
 <attribute name="VALUE" x="212.09" y="191.77" size="1.778" layer="96" rot="R90"/>
 </instance>
-<instance part="P+8" gate="1" x="214.63" y="127" smashed="yes">
-<attribute name="VALUE" x="212.09" y="121.92" size="1.778" layer="96" rot="R90"/>
+<instance part="P+8" gate="1" x="214.63" y="128.27" smashed="yes">
+<attribute name="VALUE" x="212.09" y="123.19" size="1.778" layer="96" rot="R90"/>
 </instance>
 <instance part="GND4" gate="1" x="55.88" y="114.3" smashed="yes">
@@
 <attribute name="VALUE" x="116.332" y="19.05" size="1.778" layer="96" font="vector" rot="R90" align="top-left"/>
 </instance>
+<instance part="U$8" gate="G$1" x="138.43" y="43.18" smashed="yes" rot="R90">
+<attribute name="NAME" x="135.89" y="40.64" size="1.778" layer="95" rot="R90"/>
+<attribute name="VALUE" x="140.97" y="40.64" size="1.778" layer="96" rot="R90" align="top-left"/>
+</instance>
 <instance part="U$6" gate="G$1" x="207.01" y="191.77" smashed="yes">
 <attribute name="NAME" x="204.47" y="194.31" size="1.778" layer="95"/>
@@
 <attribute name="NAME" x="204.47" y="124.46" size="1.778" layer="95"/>
 <attribute name="VALUE" x="204.47" y="119.38" size="1.778" layer="96" align="top-left"/>
-</instance>
-<instance part="U$8" gate="G$1" x="138.43" y="43.18" smashed="yes" rot="R90">
-<attribute name="NAME" x="135.89" y="40.64" size="1.778" layer="95" rot="R90"/>
-<attribute name="VALUE" x="140.97" y="40.64" size="1.778" layer="96" rot="R90" align="top-left"/>
 </instance>
 </instances>
@@
 </segment>
 <segment>
-<pinref part="P+8" gate="1" pin="+24V"/>
-<wire x1="214.63" y1="121.92" x2="214.63" y2="124.46" width="0.1524" layer="91"/>
-<wire x1="209.55" y1="121.92" x2="214.63" y2="121.92" width="0.1524" layer="91"/>
-<pinref part="U$7" gate="G$1" pin="2"/>
-</segment>
-<segment>
 <pinref part="P+11" gate="1" pin="+24V"/>
 <pinref part="R5" gate="G$1" pin="2"/>
 <wire x1="152.4" y1="135.89" x2="152.4" y2="132.08" width="0.1524" layer="91"/>
+</segment>
+<segment>
+<pinref part="U$7" gate="G$1" pin="1"/>
+<wire x1="204.47" y1="121.92" x2="204.47" y2="124.46" width="0.1524" layer="91"/>
+<wire x1="204.47" y1="124.46" x2="214.63" y2="124.46" width="0.1524" layer="91"/>
+<pinref part="P+8" gate="1" pin="+24V"/>
+<wire x1="214.63" y1="124.46" x2="214.63" y2="125.73" width="0.1524" layer="91"/>
 </segment>
 </net>
@@
 <segment>
 <pinref part="U$5" gate="G$1" pin="I_P"/>
-<wire x1="184.15" y1="119.38" x2="184.15" y2="121.92" width="0.1524" layer="91"/>
-<wire x1="184.15" y1="121.92" x2="204.47" y2="121.92" width="0.1524" layer="91"/>
-<pinref part="U$7" gate="G$1" pin="1"/>
-</segment>
-</net>
+<pinref part="U$7" gate="G$1" pin="2"/>
+<wire x1="209.55" y1="121.92" x2="209.55" y2="119.38" width="0.1524" layer="91"/>
+<wire x1="209.55" y1="119.38" x2="184.15" y2="119.38" width="0.1524" layer="91"/>
+</segment>
+</net>

Commit message: cleaned up power planes a bit
Connections:
- net N2: now also U$5.I_P; no longer U$5.I_N
- net P2: now also U$5.I_N; no longer U$5.I_P
Other:
- moved on the sheet: U$7
Changed lines of the file:
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@@
 <attribute name="VALUE" x="212.09" y="191.77" size="1.778" layer="96" rot="R90"/>
 </instance>
-<instance part="P+8" gate="1" x="214.63" y="128.27" smashed="yes">
-<attribute name="VALUE" x="212.09" y="123.19" size="1.778" layer="96" rot="R90"/>
+<instance part="P+8" gate="1" x="203.2" y="60.96" smashed="yes">
+<attribute name="VALUE" x="200.66" y="55.88" size="1.778" layer="96" rot="R90"/>
 </instance>
 <instance part="GND4" gate="1" x="55.88" y="114.3" smashed="yes">
@@
 <attribute name="VALUE" x="204.47" y="189.23" size="1.778" layer="96" align="top-left"/>
 </instance>
-<instance part="U$7" gate="G$1" x="207.01" y="121.92" smashed="yes">
-<attribute name="NAME" x="204.47" y="124.46" size="1.778" layer="95"/>
-<attribute name="VALUE" x="204.47" y="119.38" size="1.778" layer="96" align="top-left"/>
+<instance part="U$7" gate="G$1" x="195.58" y="54.61" smashed="yes">
+<attribute name="NAME" x="193.04" y="57.15" size="1.778" layer="95"/>
+<attribute name="VALUE" x="193.04" y="52.07" size="1.778" layer="96" align="top-left"/>
 </instance>
 </instances>
@@
 <segment>
 <pinref part="U$7" gate="G$1" pin="1"/>
-<wire x1="204.47" y1="121.92" x2="204.47" y2="124.46" width="0.1524" layer="91"/>
-<wire x1="204.47" y1="124.46" x2="214.63" y2="124.46" width="0.1524" layer="91"/>
+<wire x1="193.04" y1="54.61" x2="193.04" y2="57.15" width="0.1524" layer="91"/>
+<wire x1="193.04" y1="57.15" x2="203.2" y2="57.15" width="0.1524" layer="91"/>
 <pinref part="P+8" gate="1" pin="+24V"/>
-<wire x1="214.63" y1="124.46" x2="214.63" y2="125.73" width="0.1524" layer="91"/>
+<wire x1="203.2" y1="57.15" x2="203.2" y2="58.42" width="0.1524" layer="91"/>
 </segment>
 </net>
@@
 </segment>
 </net>
-<net name="P2" class="0">
-<segment>
-<pinref part="U$5" gate="G$1" pin="I_P"/>
-<pinref part="U$7" gate="G$1" pin="2"/>
-<wire x1="209.55" y1="121.92" x2="209.55" y2="119.38" width="0.1524" layer="91"/>
-<wire x1="209.55" y1="119.38" x2="184.15" y2="119.38" width="0.1524" layer="91"/>
-</segment>
-</net>
 <net name="N2" class="0">
-<segment>
-<pinref part="U$5" gate="G$1" pin="I_N"/>
-<wire x1="184.15" y1="58.42" x2="184.15" y2="55.88" width="0.1524" layer="91"/>
-<wire x1="184.15" y1="55.88" x2="186.69" y2="55.88" width="0.1524" layer="91"/>
-<label x="186.69" y="55.88" size="1.27" layer="95" xref="yes"/>
-</segment>
 <segment>
 <pinref part="J3" gate="G$1" pin="1"/>
@@
 <wire x1="87.63" y1="124.46" x2="87.63" y2="128.27" width="0.1524" layer="91"/>
 <label x="87.63" y="128.27" size="1.778" layer="95" rot="R90" xref="yes"/>
+</segment>
+<segment>
+<pinref part="U$5" gate="G$1" pin="I_P"/>
+<wire x1="184.15" y1="119.38" x2="184.15" y2="121.92" width="0.1524" layer="91"/>
+<wire x1="184.15" y1="121.92" x2="186.69" y2="121.92" width="0.1524" layer="91"/>
+<label x="186.69" y="121.92" size="1.27" layer="95" xref="yes"/>
 </segment>
 </net>
@@
 </segment>
 </net>
+<net name="P2" class="0">
+<segment>
+<pinref part="U$7" gate="G$1" pin="2"/>
+<wire x1="198.12" y1="54.61" x2="198.12" y2="50.8" width="0.1524" layer="91"/>
+<pinref part="U$5" gate="G$1" pin="I_N"/>
+<wire x1="198.12" y1="50.8" x2="184.15" y2="50.8" width="0.1524" layer="91"/>
+<wire x1="184.15" y1="50.8" x2="184.15" y2="58.42" width="0.1524" layer="91"/>
+</segment>
+</net>

Commit message: fixed silkscreen somemore
Parts:
- J2, J3: value XT-60BATT_LABEL -> CONNECTOR; device RoboJackets-Connectors:XT-60BATT_LABEL -> CurrentSensing:CONNECTOR
- renumbered U$1 to L1, U$2 to D1, U$4 to U3, U$5 to U4, U$6 to XF1, U$7 to XF2, U$8 to F1
