File: Radio/Radii/Radii.brd (EAGLE design)
At the start: 43.1 x 44.3 mm, 14 parts, among them U2 74HC4050D,653

Commit message: Updated board with Level Shifter
Parts:
- U2: value 74HC4050D,653 -> LEV_SHIFT
- moved C6 60.1 mm to (30.0, 42.0)
- moved U2 43.9 mm to (24.2, 37.7), turned to 0 degrees
- moved JP1 24.0 mm to (41.6, 34.2), turned to 90 degrees
- moved U1 14.0 mm to (29.9, 20.3)
- moved C3 13.0 mm to (40.7, 23.4)
- moved JP2 13.0 mm to (40.0, 10.0)
- moved C2 6.32 mm to (34.4, 10.5)
Routing:
- net 5V: track 55.5 -> 124.4 mm
- net SCK5: track 26.8 -> 67.2 mm
- net SS3: track 0.00 -> 32.3 mm, vias 0 -> 4
- net MOSI3: track 0.00 -> 26.0 mm, vias 0 -> 2
- net SS5: track 8.88 -> 33.6 mm
- net INT5: track 0.00 -> 23.2 mm
- net 3.3V: track 63.2 -> 82.0 mm, vias 2 -> 0
- net MISO3: track 0.00 -> 18.4 mm
- net DISP_RESET: track 22.1 -> 33.8 mm, vias 0 -> 1
- net DC_SELECT: track 17.8 -> 28.8 mm, vias 0 -> 1
- net INT: track 33.2 -> 25.1 mm
- net SCK3: track 20.8 -> 17.4 mm
- net MISO5: track 1.58 -> 4.05 mm
- net CS5: track 25.7 -> 24.3 mm, vias 0 -> 1
- net N$3: track 5.10 -> 4.10 mm
Other:
- board size 43.1 x 44.3 mm -> 44.2 x 44.3 mm

Commit message: Radii Style Guide Changes
Parts:
- moved C6 23.0 mm to (7.40, 37.6)
- moved U2 16.6 mm to (9.20, 30.7)
- moved JP1 13.9 mm to (29.6, 41.2), turned to 0 degrees
- moved C1 3.01 mm to (5.77, 7.46), turned to 0 degrees
- moved U1 3.00 mm to (29.9, 23.3)
- moved C2 2.92 mm to (36.9, 12.0), turned to 0 degrees
- moved C3 1.90 mm to (40.7, 25.3)
- renumbered CN1 to P1, U$1 to U4, U$2 to U3
Connections:
- removed net MISO3: U1.10P, U2.2
- removed net MISO5: U2.3, U4.D12
- new net MISO: U1.10P, U4.D12
Routing:
- net 5V: track 124.4 -> 84.3 mm, vias 0 -> 2
- net SS5: track 33.6 -> 7.60 mm, vias 0 -> 1
- net SCK5: track 67.2 -> 42.0 mm
- net MISO3: track 18.4 -> 0.00 mm
- net MISO: track 0.00 -> 14.9 mm
- net SS3: track 32.3 -> 18.2 mm, vias 4 -> 0
- net DISP_RESET: track 33.8 -> 21.0 mm, vias 1 -> 0
- net INT5: track 23.2 -> 12.7 mm
- net CS5: track 24.3 -> 16.7 mm, vias 1 -> 0
- net MOSI3: track 26.0 -> 18.7 mm
- net SCK3: track 17.4 -> 23.0 mm
- net DC_SELECT: track 28.8 -> 23.9 mm, vias 1 -> 0
- net MISO5: track 4.05 -> 0.00 mm
- net INT: track 25.1 -> 28.5 mm
- net N$3: track 4.10 -> 7.10 mm
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- added copper zone on layer 16, net GND
Other:
- board size 44.2 x 44.3 mm -> 42.6 x 44.3 mm
