File: Radio/Radii/Radii.brd (EAGLE design)
At the start: 42.6 x 44.3 mm, 14 parts, among them U2 LEV_SHIFT, U3 XC9140C501MR-G, U4 NANO

Commit message: Changed to MCU
Parts:
- removed C5: 10uF, SparkFun-Capacitors:0603
- removed C6: 0.1uF, SparkFun-Capacitors:0603
- removed L1: 4.7μH, I'mRADIOactive:IND_BOURNS_SRN3015
- removed U2: LEV_SHIFT, I'mRADIOactive:SOIC127P600X175-16N
- removed U3: XC9140C501MR-G, I'mRADIOactive:XC9140C501MR-G
- removed U4: NANO, I'mRADIOactive:NANO
- added U$1: STM32F0, I'mRADIOactive:QFP50P900X900X160-48N
- C4: value 4.7pF -> 0.1uF
- moved C4 44.5 mm to (-10.0, -14.0), turned to 0 degrees
Connections:
- removed net 5V: C1.1, C2.1, C5.1, JP1.1, U3.5, U4.RAW
- removed net INT5: U2.11, U4.D4
- removed net MOSI5: JP1.4, U2.5, U4.D11
- removed net N$1: L1.1, U3.1
- removed net N$2: U3.2
- removed net SCK5: JP1.3, U2.7, U4.D13
- removed net SS5: U2.9, U4.D5
- new net CS3: JP1.5
- new net RESET: U$1.7
- net 3.3V: now also C1.1, C2.1, JP1.1, U$1.23, U$1.47, U$1.8; no longer C6.1, L1.2, U2.1, U3.3
- net CS5: now also U$1.25; no longer JP1.5, U4.D10
- net DC_SELECT: now also U$1.13, U$1.27; no longer U4.D8
- net DISP_RESET: now also U$1.12, U$1.26; no longer U4.D9
- net GND: now also U$1.24, U$1.48, U$1.9; no longer C5.2, C6.2, U2.8, U3.4, U4.GND
- net INT: now also U$1.11; no longer U2.12
- net MISO: now also U$1.16; no longer U4.D12
- net MOSI3: now also JP1.4, U$1.17; no longer U2.4
- net SCK3: now also JP1.3, U$1.15; no longer U2.6
- net SS3: now also U$1.14; no longer U2.10
Routing:
- net 5V: track 84.3 -> 0.00 mm, vias 2 -> 0
- net SCK5: track 42.0 -> 0.00 mm, vias 1 -> 0
- net MOSI5: track 28.8 -> 0.00 mm
- net SCK3: track 23.0 -> 48.6 mm
- net CS5: track 16.7 -> 0.00 mm
- net CS3: track 0.00 -> 14.4 mm
- net INT5: track 12.7 -> 0.00 mm
- net MOSI3: track 18.7 -> 30.9 mm
- net 3.3V: track 84.9 -> 73.1 mm
- net SS5: track 7.60 -> 0.00 mm, vias 1 -> 0
- net DC_SELECT: track 23.9 -> 17.1 mm
- net N$1: track 3.30 -> 0.00 mm
- net SS3: track 18.2 -> 17.2 mm
- net INT: track 28.5 -> 27.5 mm
- net MISO: track 14.9 -> 14.2 mm

Commit message: Updated Power Regulators
Parts:
- added C5: 10uF, SparkFun-Capacitors:0603
- added C6: 0.1uF, SparkFun-Capacitors:0603
- added C7: 44uF, SparkFun-Capacitors:0603
- added L1: SRN3015-4R7M, I'mRADIOactive:IND_BOURNS_SRN3015
- added U$2, U$3: AP63203WU-7, I'mRADIOactive:POWERREG
Connections:
- new net N$1: C6.2, L1.2, U$3.5
- new net N$2: C6.1, U$3.6
- new net RADIO_RESET: U$1.18, U1.14P
- net 3.3V: now also C5.1, C7.1, L1.1, U$3.1, U$3.2, U$3.3
- net GND: now also C5.2, C7.2, U$3.4
Changed lines of the file:
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@@
 <attribute name="VALUE" x="-10" y="-14.762" size="0.6096" layer="27" font="vector" ratio="20" align="top-center"/>
+</element>
+<element name="U$2" library="I'mRADIOactive" package="POWERREG" value="AP63203WU-7" x="-7" y="-20" smashed="yes">
+<attribute name="NAME" x="-11.318" y="-18.222" size="1.778" layer="21"/>
+<attribute name="VALUE" x="-11.445" y="-23.556" size="1.778" layer="21"/>
+</element>
+<element name="U$3" library="I'mRADIOactive" package="POWERREG" value="AP63203WU-7" x="-7" y="-29" smashed="yes">
+<attribute name="NAME" x="-11.318" y="-27.222" size="1.778" layer="21"/>
+<attribute name="VALUE" x="-11.445" y="-32.556" size="1.778" layer="21"/>
+</element>
+<element name="C5" library="SparkFun-Capacitors" library_urn="urn:adsk.eagle:library:510" package="0603" package3d_urn="urn:adsk.eagle:package:37414/1" value="10uF" x="-10" y="-35" smashed="yes">
+<attribute name="NAME" x="-10" y="-34.238" size="0.6096" layer="25" font="vector" ratio="20" align="bottom-center"/>
+<attribute name="PROD_ID" value="CAP-11015" x="-10" y="-35" size="1.778" layer="27" display="off"/>
+<attribute name="VALUE" x="-10" y="-35.762" size="0.6096" layer="27" font="vector" ratio="20" align="top-center"/>
+</element>
+<element name="C6" library="SparkFun-Capacitors" library_urn="urn:adsk.eagle:library:510" package="0603" package3d_urn="urn:adsk.eagle:package:37414/1" value="0.1uF" x="-10" y="-39" smashed="yes">
+<attribute name="NAME" x="-10" y="-38.238" size="0.6096" layer="25" font="vector" ratio="20" align="bottom-center"/>
+<attribute name="PROD_ID" value="CAP-00810" x="-10" y="-39" size="1.778" layer="27" display="off"/>
+<attribute name="VALUE" x="-10" y="-39.762" size="0.6096" layer="27" font="vector" ratio="20" align="top-center"/>
+</element>
+<element name="C7" library="SparkFun-Capacitors" library_urn="urn:adsk.eagle:library:510" package="0603" package3d_urn="urn:adsk.eagle:package:37414/1" value="44uF" x="-10" y="-43" smashed="yes">
+<attribute name="NAME" x="-10" y="-42.238" size="0.6096" layer="25" font="vector" ratio="20" align="bottom-center"/>
+<attribute name="PROD_ID" value="CAP-11015" x="-10" y="-43" size="1.778" layer="27" display="off"/>
+<attribute name="VALUE" x="-10" y="-43.762" size="0.6096" layer="27" font="vector" ratio="20" align="top-center"/>
+</element>
+<element name="L1" library="I'mRADIOactive" package="IND_BOURNS_SRN3015" value="SRN3015-4R7M" x="-16" y="-40" smashed="yes">
+<attribute name="BUILT_BY" value="EMA_UL_Team" x="-16" y="-40" size="1.778" layer="27" display="off"/>
+<attribute name="MANUFACTURER_PART_NUMBER" value="SRN3015-4R7M" x="-16" y="-40" size="1.778" layer="27" display="off"/>
+<attribute name="NAME" x="-18.8956" y="-38.222" size="1.27" layer="25" ratio="6" rot="SR0"/>
+<attribute name="VALUE" x="-18.9972" y="-43.175" size="1.27" layer="27" ratio="6" rot="SR0"/>
+<attribute name="VENDOR" value="Bourns Electronics" x="-16" y="-40" size="1.778" layer="27" display="off"/>
 </element>
 </elements>
@@
 <contactref element="U$1" pad="48"/>
 <contactref element="U$1" pad="24"/>
+<contactref element="C5" pad="2"/>
+<contactref element="U$3" pad="4"/>
+<contactref element="C7" pad="2"/>
 <wire x1="38.045" y1="18.295" x2="40.69" y2="26.11" width="0" layer="19" extent="1-1"/>
 <wire x1="37.73" y1="12.02" x2="38.045" y2="18.295" width="0" layer="19" extent="1-1"/>
@@
 <wire x1="-3.25" y1="-8.18" x2="-10.18" y2="-5.25" width="0" layer="19" extent="1-1"/>
 <wire x1="-9.15" y1="-14" x2="-3.25" y2="-8.18" width="0" layer="19" extent="1-1"/>
+<wire x1="-5.9005" y1="-29.95" x2="-9.15" y2="-14" width="0" layer="19" extent="1-1"/>
+<wire x1="-9.15" y1="-35" x2="-5.9005" y2="-29.95" width="0" layer="19" extent="1-1"/>
+<wire x1="-9.15" y1="-43" x2="-9.15" y2="-35" width="0" layer="19" extent="1-1"/>
 </signal>
 <signal name="DISP_RESET">
@@
 <contactref element="U$1" pad="47"/>
 <contactref element="U$1" pad="23"/>
+<contactref element="U$3" pad="3"/>
+<contactref element="U$3" pad="2"/>
+<contactref element="C5" pad="1"/>
+<contactref element="L1" pad="1"/>
+<contactref element="C7" pad="1"/>
+<contactref element="U$3" pad="1"/>
 <wire x1="6.40465" y1="35.145" x2="21.95" y2="41.23" width="0" layer="19" extent="1-1"/>
 <wire x1="31.9078" y1="8.9078" x2="31.25" y2="3.75" width="0" layer="19" extent="1-1"/>
@@
 <wire x1="-3.75" y1="-8.18" x2="-10.18" y2="-4.75" width="0" layer="19" extent="1-1"/>
 <wire x1="-10.85" y1="-14" x2="-3.75" y2="-8.18" width="0" layer="19" extent="1-1"/>
+<wire x1="-8.0995" y1="-28.05" x2="-10.85" y2="-14" width="0" layer="19" extent="1-1"/>
+<wire x1="-8.0995" y1="-29" x2="-8.0995" y2="-28.05" width="0" layer="19" extent="1-1"/>
+<wire x1="-8.0995" y1="-29.95" x2="-8.0995" y2="-29" width="0" layer="19" extent="1-1"/>
+<wire x1="-10.85" y1="-35" x2="-8.0995" y2="-29.95" width="0" layer="19" extent="1-1"/>
+<wire x1="-17.0922" y1="-40" x2="-10.85" y2="-35" width="0" layer="19" extent="1-1"/>
+<wire x1="-10.85" y1="-43" x2="-17.0922" y2="-40" width="0" layer="19" extent="1-1"/>
 </signal>
 <signal name="N$3">
@@
 <contactref element="U$1" pad="25"/>
 </signal>
+<signal name="RADIO_RESET">
+<contactref element="U1" pad="14P"/>
+<contactref element="U$1" pad="18"/>
+<wire x1="-6.25" y1="-8.18" x2="21.845" y2="20.295" width="0" layer="19" extent="1-1"/>
+</signal>
+<signal name="N$1">
+<contactref element="U$3" pad="5"/>
+<contactref element="L1" pad="2"/>
+<contactref element="C6" pad="2"/>
+<wire x1="-9.15" y1="-39" x2="-14.9078" y2="-40" width="0" layer="19" extent="1-1"/>
+<wire x1="-5.9005" y1="-29" x2="-9.15" y2="-39" width="0" layer="19" extent="1-1"/>
+</signal>
+<signal name="N$2">
+<contactref element="U$3" pad="6"/>
+<contactref element="C6" pad="1"/>
+<wire x1="-5.9005" y1="-28.05" x2="-10.85" y2="-39" width="0" layer="19" extent="1-1"/>
+</signal>
 </signals>

Commit message: Wired radio board
Parts:
- removed L1: SRN3015-4R7M, I'mRADIOactive:IND_BOURNS_SRN3015
- added C8: 22UF-1210-16V-20%, SparkFun-Capacitors:1210
- C7: value 44uF -> 22UF-1210-16V-20%; device SparkFun-Capacitors:0603 -> SparkFun-Capacitors:1210
- U$2: value AP63203WU-7 -> IND_1255AY-3R9N=P3; device I'mRADIOactive:POWERREG -> I'mRADIOactive:IND_1255AY-3R9N=P3
- moved C7 64.9 mm to (17.0, 16.0), turned to 270 degrees
- moved C6 58.2 mm to (6.00, 17.0), turned to 270 degrees
- moved C4 54.5 mm to (33.8, 18.5)
- moved C5 49.7 mm to (3.00, 13.0)
- moved U$3 47.1 mm to (3.00, 17.0)
- moved U$2 41.1 mm to (11.0, 17.0), turned to 90 degrees
- moved C2 27.7 mm to (9.18, 11.3), turned to 180 degrees
- moved U$1 25.5 mm to (17.0, 7.00), turned to 90 degrees
- moved JP1 20.6 mm to (24.6, 21.2)
- moved P1 19.0 mm to (5.42, 4.36)
- moved U1 14.3 mm to (32.9, 9.29)
- moved C1 13.3 mm to (2.77, 20.5), turned to 180 degrees
- moved JP2 10.0 mm to (41.0, 20.0)
- moved C3 7.43 mm to (37.7, 18.5), turned to 0 degrees
Connections:
- new net 9V: C5.1, P1.1, U$3.2, U$3.3
- net 3.3V: now also C8.1, U$2.2; no longer C5.1, L1.1, P1.1, U$3.2, U$3.3
- net DC_SELECT: now also U$1.26; no longer U$1.13, U$1.27
- net DISP_RESET: now also U$1.27; no longer U$1.12, U$1.26
- net GND: now also C8.2
- net N$1: now also U$2.1; no longer L1.2
- net RADIO_RESET: now also U$1.13; no longer U$1.18
Routing:
- net SCK3: track 48.6 -> 28.4 mm, vias 0 -> 1
- net 3.3V: track 73.1 -> 88.2 mm, vias 2 -> 0
- net CS3: track 14.4 -> 0.00 mm
- net SS3: track 17.2 -> 5.49 mm
- net N$3: track 7.10 -> 18.5 mm, vias 0 -> 1
- net 9V: track 0.00 -> 9.98 mm
- net N$1: track 0.00 -> 7.87 mm
- net RADIO_RESET: track 0.00 -> 4.51 mm
- net DISP_RESET: track 20.7 -> 16.4 mm, vias 0 -> 1
- net MOSI3: track 30.9 -> 27.8 mm
- net INT: track 27.5 -> 29.8 mm
- net N$2: track 0.00 -> 1.94 mm
- net MISO: track 14.2 -> 12.4 mm
- net DC_SELECT: track 17.1 -> 17.7 mm, vias 0 -> 1

Commit message: Took out MCU from Radio
Parts:
- removed U$1: STM32F0, I'mRADIOactive:QFP50P900X900X160-48N
Connections:
- removed net CS5: U$1.25
- removed net RESET: U$1.7
- net 3.3V: no longer U$1.23, U$1.47, U$1.8
- net DC_SELECT: no longer U$1.26
- net DISP_RESET: no longer U$1.27
- net GND: no longer U$1.24, U$1.48, U$1.9
- net INT: no longer U$1.11
- net MISO: no longer U$1.16
- net MOSI3: no longer U$1.17
- net RADIO_RESET: no longer U$1.13
- net SCK3: no longer U$1.15
- net SS3: no longer U$1.14
Routing:
- net 3.3V: track 88.2 -> 73.4 mm
- net SCK3: track 28.4 -> 26.3 mm
- net RADIO_RESET: track 4.51 -> 2.89 mm
- net DISP_RESET: track 16.4 -> 15.0 mm
- net MOSI3: track 27.8 -> 26.4 mm
- net DC_SELECT: track 17.7 -> 16.7 mm
- net INT: track 29.8 -> 28.7 mm
- net SS3: track 5.49 -> 4.76 mm
- net MISO: track 12.4 -> 11.6 mm
Changed lines of the file:
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@@
 <attribute name="VALUE" x="39.73" y="16.825" size="1.27" layer="27"/>
-</element>
-<element name="U$1" library="I'mRADIOactive" package="QFP50P900X900X160-48N" value="STM32F0" x="17" y="7" smashed="yes" rot="R90">
-<attribute name="NAME" x="11" y="2" size="1.27" layer="25" rot="R90"/>
-<attribute name="VALUE" x="23" y="2" size="1.27" layer="27" rot="R90" align="top-left"/>
 </element>
 <element name="C4" library="SparkFun-Capacitors" library_urn="urn:adsk.eagle:library:510" package="0603" package3d_urn="urn:adsk.eagle:package:37414/1" value="0.1uF" x="33.8" y="18.5" smashed="yes">
@@
 <signal name="MISO">
 <contactref element="U1" pad="10P"/>
-<contactref element="U$1" pad="16"/>
 <wire x1="26.0736" y1="12.7896875" x2="26.0736" y2="11.8003125" width="0.1524" layer="1"/>
 <wire x1="24.845" y1="14.295" x2="24.845" y2="14.0182875" width="0.1524" layer="1"/>
@@
 <wire x1="23.7503125" y1="10.9236" x2="22.8838" y2="10.0570875" width="0.1524" layer="1"/>
 <wire x1="22.8838" y1="6.7310125" x2="21.9027875" y2="5.75" width="0.1524" layer="1"/>
-<wire x1="21.9027875" y1="5.75" x2="21.18" y2="5.75" width="0.1524" layer="1"/>
 <wire x1="22.8838" y1="10.0570875" x2="22.8838" y2="6.7310125" width="0.1524" layer="1"/>
 </signal>
@@
 <vertex x="0" y="44.3"/>
 </polygon>
-<contactref element="U$1" pad="9"/>
 <contactref element="C4" pad="2"/>
-<contactref element="U$1" pad="48"/>
-<contactref element="U$1" pad="24"/>
 <contactref element="C5" pad="2"/>
 <contactref element="C7" pad="2"/>
@@
 <signal name="DISP_RESET">
 <contactref element="JP1" pad="6"/>
-<contactref element="U$1" pad="27"/>
-<wire x1="18.75" y1="11.18" x2="18.75" y2="12.65" width="0.1524" layer="1"/>
 <wire x1="18.75" y1="12.65" x2="18.5" y2="12.9" width="0.1524" layer="1"/>
 <via x="18.5" y="12.9" extent="1-16" drill="0.381"/>
@@
 <signal name="DC_SELECT">
 <contactref element="JP1" pad="7"/>
-<contactref element="U$1" pad="26"/>
-<wire x1="19.25" y1="11.18" x2="19.25" y2="12.25" width="0.1524" layer="1"/>
 <wire x1="19.25" y1="12.25" x2="19.8" y2="12.8" width="0.1524" layer="1"/>
 <via x="19.8" y="12.8" extent="1-16" drill="0.381"/>
@@
 <signal name="INT">
 <contactref element="U1" pad="6P"/>
-<contactref element="U$1" pad="11"/>
-<wire x1="19.25" y1="2.82" x2="19.25" y2="1.75" width="0.1524" layer="1"/>
 <wire x1="19.25" y1="1.75" x2="20" y2="1" width="0.1524" layer="1"/>
 <via x="20" y="1" extent="1-16" drill="0.381"/>
@@
 <contactref element="JP1" pad="1"/>
 <contactref element="C1" pad="1"/>
-<contactref element="U$1" pad="8"/>
 <contactref element="C4" pad="1"/>
-<contactref element="U$1" pad="47"/>
-<contactref element="U$1" pad="23"/>
 <contactref element="U$2" pad="2"/>
 <contactref element="C7" pad="1"/>
@@
 <wire x1="17" y1="17.755" x2="21" y2="17.755" width="0.1524" layer="1"/>
 <wire x1="22.0341875" y1="9.3814" x2="21.3114" y2="9.3814" width="0.1524" layer="1"/>
-<wire x1="21.3114" y1="9.3814" x2="21.18" y2="9.25" width="0.1524" layer="1"/>
 <wire x1="21" y1="17.755" x2="22.2586" y2="16.4964" width="0.1524" layer="1"/>
 <wire x1="22.2586" y1="16.4964" x2="22.2586" y2="9.6058125" width="0.1524" layer="1"/>
 <wire x1="22.2586" y1="9.6058125" x2="22.0341875" y2="9.3814" width="0.1524" layer="1"/>
 <wire x1="11.9658125" y1="4.8814" x2="12.6886" y2="4.8814" width="0.1524" layer="1"/>
-<wire x1="12.6886" y1="4.8814" x2="12.82" y2="4.75" width="0.1524" layer="1"/>
 <wire x1="10.03" y1="11.32" x2="10.03" y2="6.8172125" width="0.1524" layer="1"/>
 <wire x1="10.03" y1="6.8172125" x2="11.9658125" y2="4.8814" width="0.1524" layer="1"/>
-<wire x1="17.6186" y1="3.6741875" x2="17.6186" y2="2.9514" width="0.1524" layer="1"/>
-<wire x1="17.6186" y1="2.9514" x2="17.75" y2="2.82" width="0.1524" layer="1"/>
-<wire x1="12.82" y1="4.75" x2="16.5427875" y2="4.75" width="0.1524" layer="1"/>
-<wire x1="16.5427875" y1="4.75" x2="17.6186" y2="3.6741875" width="0.1524" layer="1"/>
-<wire x1="21.18" y1="9.25" x2="21.0486" y2="9.1186" width="0.1524" layer="1"/>
-<wire x1="21.0486" y1="9.1186" x2="20.3258125" y2="9.1186" width="0.1524" layer="1"/>
-<wire x1="20.3258125" y1="9.1186" x2="17.75" y2="6.5427875" width="0.1524" layer="1"/>
-<wire x1="17.75" y1="6.5427875" x2="17.75" y2="2.82" width="0.1524" layer="1"/>
 <wire x1="21" y1="17.755" x2="21.745" y2="18.5" width="0.1524" layer="1"/>
 <wire x1="21.745" y1="18.5" x2="32.95" y2="18.5" width="0.1524" layer="1"/>
+<wire x1="10.03" y1="11.32" x2="11" y2="19.35" width="0" layer="19" extent="1-1"/>
 </signal>
 <signal name="N$3">
@@
 <signal name="MOSI3">
 <contactref element="U1" pad="11P"/>
-<contactref element="U$1" pad="17"/>
 <contactref element="JP1" pad="4"/>
-<wire x1="21.18" y1="6.25" x2="19.75" y2="6.25" width="0.1524" layer="1"/>
 <wire x1="19.75" y1="6.25" x2="19.043640625" y2="6.956359375" width="0.1524" layer="1"/>
 <via x="19.043640625" y="6.956359375" extent="1-16" drill="0.381"/>
@@
 <signal name="SCK3">
 <contactref element="U1" pad="12P"/>
-<contactref element="U$1" pad="15"/>
 <contactref element="JP1" pad="3"/>
-<wire x1="21.18" y1="5.25" x2="21.3114" y2="5.3814" width="0.1524" layer="1"/>
 <wire x1="21.3114" y1="5.3814" x2="22.0341875" y2="5.3814" width="0.1524" layer="1"/>
 <wire x1="22.0341875" y1="5.3814" x2="23.1886" y2="6.5358125" width="0.1524" layer="1"/>
@@
 <via x="19" y="5" extent="1-16" drill="0.381"/>
 <wire x1="19" y1="5" x2="19.25" y2="5.25" width="0.1524" layer="1"/>
-<wire x1="19.25" y1="5.25" x2="21.18" y2="5.25" width="0.1524" layer="1"/>
 <wire x1="17" y1="16.2" x2="17" y2="7" width="0.1524" layer="16"/>
+<wire x1="19.25" y1="5.25" x2="21.3114" y2="5.3814" width="0" layer="19" extent="1-1"/>
 </signal>
 <signal name="SS3">
 <contactref element="U1" pad="13P"/>
-<contactref element="U$1" pad="14"/>
 <wire x1="23.5886" y1="7.0386" x2="24.845" y2="8.295" width="0.1524" layer="1"/>
 <wire x1="23.5886" y1="6.4358125" x2="23.5886" y2="7.0386" width="0.1524" layer="1"/>
-<wire x1="21.18" y1="4.75" x2="21.9027875" y2="4.75" width="0.1524" layer="1"/>
 <wire x1="21.9027875" y1="4.75" x2="23.5886" y2="6.4358125" width="0.1524" layer="1"/>
 </signal>
@@
 <contactref element="JP1" pad="5"/>
 </signal>
-<signal name="RESET">
-<contactref element="U$1" pad="7"/>
-</signal>
-<signal name="CS5">
-<contactref element="U$1" pad="25"/>
-</signal>
 <signal name="RADIO_RESET">
 <contactref element="U1" pad="14P"/>
-<contactref element="U$1" pad="13"/>
-<wire x1="21.18" y1="4.25" x2="22.8" y2="4.25" width="0.1524" layer="1"/>
 <wire x1="22.8" y1="4.25" x2="24.845" y2="6.295" width="0.1524" layer="1"/>
 </signal>

Commit message: Added 22uH inductor
Parts:
- added U2: ATMEGA32U4-AU, I'mRADIOactive:QFP80P1200X1200X120-44N
Connections:
- new net AVCC: U2.44
- new net AVCC_2: U2.24
- new net UCAP: U2.6
- new net UVCC: U2.2
- new net VCC: U2.34
- net 9V: now also U2.14
Changed lines of the file:
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@@
 <attribute name="VALUE" x="16.08" y="13.19" size="1.27" layer="27" rot="R90"/>
+</element>
+<element name="U2" library="I'mRADIOactive" package="QFP80P1200X1200X120-44N" value="ATMEGA32U4-AU" x="-11" y="11" smashed="yes">
+<attribute name="AVAILABILITY" value="Unavailable" x="-11" y="11" size="1.778" layer="27" display="off"/>
+<attribute name="DESCRIPTION" value=" AVR AVR® ATmega Microcontroller IC 8-Bit 16MHz 32KB (16K x 16) FLASH 44-TQFP (10x10) " x="-11" y="11" size="1.778" layer="27" display="off"/>
+<attribute name="DIGIKEY-PURCHASE-URL" value="https://snapeda.com/shop?store=DigiKey&amp;id=4251478" x="-11" y="11" size="1.778" layer="27" display="off"/>
+<attribute name="MF" value="Microchip Technology" x="-11" y="11" size="1.778" layer="27" display="off"/>
+<attribute name="MP" value="ATMEGA32U4-AU" x="-11" y="11" size="1.778" layer="27" display="off"/>
+<attribute name="NAME" x="-15.16611875" y="0.9149" size="2.083059375" layer="25" ratio="10" rot="SR0"/>
+<attribute name="PACKAGE" value="TQFP-44 Microchip Technology" x="-11" y="11" size="1.778" layer="27" display="off"/>
+<attribute name="PRICE" value="None" x="-11" y="11" size="1.778" layer="27" display="off"/>
+<attribute name="VALUE" x="-14.45928125" y="21.098" size="2.085740625" layer="27" ratio="10" rot="SR0"/>
 </element>
 </elements>
@@
 <wire x1="2.15" y1="15.8005" x2="2.15" y2="13" width="0.1524" layer="1"/>
 <wire x1="1.9005" y1="17" x2="1.9005" y2="16.05" width="0.1524" layer="1"/>
+<contactref element="U2" pad="14"/>
+<wire x1="-13.3876" y1="5.2596" x2="2.15" y2="13" width="0" layer="19" extent="1-1"/>
+</signal>
+<signal name="VCC">
+<contactref element="U2" pad="34"/>
+</signal>
+<signal name="UVCC">
+<contactref element="U2" pad="2"/>
+</signal>
+<signal name="AVCC_2">
+<contactref element="U2" pad="24"/>
+</signal>
+<signal name="AVCC">
+<contactref element="U2" pad="44"/>
+</signal>
+<signal name="UCAP">
+<contactref element="U2" pad="6"/>
 </signal>
 </signals>

Commit message: Organized board with 32u4
Parts:
- removed U$2: IND_1255AY-3R9N=P3, I'mRADIOactive:IND_1255AY-3R9N=P3
- removed U$3: AP63203WU-7, I'mRADIOactive:POWERREG
- added J1: 10118193-0001LF, I'mRADIOactive:FCI_10118193-0001LF
- added R1, R2: 22Ω, adafruit:R0603
- added U3: (no value), I'mRADIOactive:POWERREG
- added U4: IND_1255AY-3R9N=P3, I'mRADIOactive:IND_1255AY-3R9N=P3
- C1, C4: value 0.1uF -> 1.0uF
- U2: value ATMEGA32U4-AU -> ATMEGA32U4-AUR
- moved C4 28.4 mm to (5.90, 13.0), turned to 180 degrees
- moved U2 27.5 mm to (16.3, 7.70)
- moved P1 16.4 mm to (3.42, 20.7), turned to 90 degrees
- moved C1 11.7 mm to (2.00, 8.80)
- moved C2 4.69 mm to (4.58, 10.4), turned to 270 degrees
- moved JP1 3.16 mm to (27.6, 22.2)
- moved C5 2.33 mm to (2.00, 10.9)
- moved C6 1.90 mm to (5.90, 15.1), turned to 0 degrees
- moved C7 1.77 mm to (18.2, 17.3)
- moved C8 1.48 mm to (21.7, 17.3)
- turned C3 to 180 degrees
Connections:
- removed net AVCC: U2.44
- removed net AVCC_2: U2.24
- removed net UCAP: U2.6
- removed net UVCC: U2.2
- removed net VCC: U2.34
- new net DIFF_N: J1.2, R1.1
- new net DIFF_P: J1.3, R2.1
- new net N$4: J1.1, U2.7
- new net N$5: C4.1, U2.6
- new net N$6: R1.2, U2.3
- new net N$8: R2.2, U2.4
- new net RESET: U2.13
- net 3.3V: now also U2.14, U2.2, U2.24, U2.34, U2.44, U3.1, U4.2; no longer C4.1, U$2.2, U$3.1
- net 9V: now also U3.2, U3.3; no longer U$3.2, U$3.3, U2.14
- net CS3: now also U2.38
- net DC_SELECT: now also U2.36
- net DISP_RESET: now also U2.37
- net GND: now also J1.5, J1.S1, J1.S2, J1.S3, J1.S4, J1.S5, J1.S6, U2.15, U2.23, U2.35, U2.43, U2.5, U3.4; no longer U$3.4
- net INT: now also U2.30
- net MISO: now also U2.11
- net MOSI3: now also U2.10
- net N$1: now also U3.5, U4.1; no longer U$2.1, U$3.5
- net N$2: now also U3.6; no longer U$3.6
- net RADIO_RESET: now also U2.28
- net SCK3: now also U2.9
- net SS3: now also U2.29
Routing:
- net 3.3V: track 73.4 -> 101.5 mm
- net CS3: track 0.00 -> 19.9 mm, vias 0 -> 1
- net N$5: track 0.00 -> 10.6 mm, vias 0 -> 2
- net N$4: track 0.00 -> 9.34 mm
- net MISO: track 11.6 -> 20.7 mm, vias 0 -> 2
- net DIFF_N: track 0.00 -> 6.53 mm
- net DISP_RESET: track 15.0 -> 21.2 mm
- net DC_SELECT: track 16.7 -> 22.8 mm
- net INT: track 28.7 -> 22.7 mm
- net SCK3: track 26.3 -> 31.5 mm, vias 1 -> 2
- net N$1: track 7.87 -> 12.9 mm
- net 9V: track 9.98 -> 14.8 mm
- net DIFF_P: track 0.00 -> 4.66 mm
- net MOSI3: track 26.4 -> 28.8 mm, vias 2 -> 3
- net N$6: track 0.00 -> 2.06 mm
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