File: Radio/Radii/Radii.brd (EAGLE design)
At the start: 42.6 x 44.3 mm, 18 parts, among them J1 10118193-0001LF, U2 ATMEGA32U4-AUR, U4 IND_1255AY-3R9N=P3

Commit message: Redoing radio board
Parts:
- added C10, C11, C9: 0.1uF, SparkFun-Capacitors:0603
- added C12: 10nF, SparkFun-Capacitors:0603
- C1: value 1.0uF -> 0.1uF
- moved U1 19.2 mm to (20.9, 24.3), turned to 90 degrees
- moved C8 16.3 mm to (7.50, 9.30), turned to 180 degrees
- moved JP1 15.7 mm to (41.6, 29.2)
- moved C7 11.6 mm to (7.50, 12.9), turned to 180 degrees
- moved C2 11.5 mm to (13.8, 3.52), turned to 180 degrees
- moved C4 9.38 mm to (13.8, 8.00)
- moved C1 8.97 mm to (10.4, 5.80)
- moved R1 6.81 mm to (1.20, 10.4), turned to 90 degrees
- moved U2 6.00 mm to (22.3, 7.70)
- moved C6 5.14 mm to (2.55, 19.0)
- moved P1 5.00 mm to (3.42, 25.7)
- moved R2 5.00 mm to (3.30, 10.4), turned to 90 degrees
- moved U4 4.90 mm to (8.30, 17.9), turned to 0 degrees
- moved C5 2.65 mm to (2.52, 13.5)
- moved U3 2.62 mm to (2.52, 16.5)
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Connections:
- net N$6 renamed DIFF1_N
- net N$8 renamed DIFF1_P
- new net N$7: C12.1, U2.42
- new net UVCC: U2.2
- net 3.3V: now also C10.1, C11.1, C9.1; no longer U2.2
- net GND: now also C10.2, C11.2, C12.2, C9.2
Routing:
- net 3.3V: track 101.5 -> 13.2 mm, vias 0 -> 2
- net SCK3: track 31.5 -> 0.00 mm, vias 2 -> 0
- net MOSI3: track 28.8 -> 0.00 mm, vias 3 -> 0
- net DC_SELECT: track 22.8 -> 0.00 mm, vias 1 -> 0
- net INT: track 22.7 -> 0.00 mm, vias 2 -> 0
- net DISP_RESET: track 21.2 -> 0.00 mm, vias 1 -> 0
- net MISO: track 20.7 -> 0.00 mm, vias 2 -> 0
- net CS3: track 19.9 -> 0.00 mm, vias 1 -> 0
- net DIFF1_N: track 2.06 -> 20.9 mm, vias 0 -> 2
- net N$3: track 18.8 -> 0.00 mm, vias 1 -> 0
- net DIFF1_P: track 2.02 -> 20.1 mm, vias 0 -> 2
- net GND: track 0.00 -> 13.4 mm
- net N$1: track 12.9 -> 0.00 mm
- net N$5: track 10.6 -> 0.00 mm, vias 2 -> 0
- net N$4: track 9.34 -> 0.00 mm
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- added copper zone on layer 1, net 3.3V
- added copper zone on layer 1, net 9V
- added copper zone on layer 1, net N$1

Commit message: Updated radio board
Parts:
- moved JP1 20.0 mm to (40.6, 9.23), turned to 270 degrees
- moved JP2 12.0 mm to (41.0, 32.0)
- moved C12 6.00 mm to (13.8, 11.9)
- moved C11 3.40 mm to (13.8, 1.25)
- moved C10 2.48 mm to (13.8, 3.52)
- moved C2 2.30 mm to (13.8, 5.82)
- moved C3 2.24 mm to (36.7, 16.5)
Routing:
- net GND: track 13.4 -> 34.4 mm, vias 0 -> 4
- net N$5: track 0.00 -> 2.05 mm
