File: Radio/Radii/Radii.brd (EAGLE design)
At the start: 42.6 x 44.3 mm, 22 parts, among them J1 10118193-0001LF, U2 ATMEGA32U4-AUR, U4 IND_1255AY-3R9N=P3

Commit message: Edited radio board
Parts:
- moved C3 23.7 mm to (13.9, 10.1)
- moved C12 0.40 mm to (13.8, 12.3)
- moved C1 0.40 mm to (10.4, 5.40)
- moved C9 0.30 mm to (10.4, 3.23)
Routing:
- net GND: track 34.4 -> 35.8 mm
Changed lines of the file:
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@@
 <attribute name="VALUE" x="13.845" y="6.582" size="0.6096" layer="27" font="vector" ratio="20" rot="R180" align="top-center"/>
 </element>
-<element name="C3" library="SparkFun-Capacitors" library_urn="urn:adsk.eagle:library:510" package="0603" package3d_urn="urn:adsk.eagle:package:37414/1" value="0.1uF" x="36.69" y="16.46" smashed="yes" rot="R180">
-<attribute name="NAME" x="36.69" y="15.698" size="0.6096" layer="25" font="vector" ratio="20" rot="R180" align="bottom-center"/>
-<attribute name="PROD_ID" value="CAP-00810" x="36.69" y="16.46" size="1.778" layer="27" rot="R180" display="off"/>
-<attribute name="VALUE" x="36.69" y="17.222" size="0.6096" layer="27" font="vector" ratio="20" rot="R180" align="top-center"/>
+<element name="C3" library="SparkFun-Capacitors" library_urn="urn:adsk.eagle:library:510" package="0603" package3d_urn="urn:adsk.eagle:package:37414/1" value="0.1uF" x="13.89" y="10.06" smashed="yes" rot="R180">
+<attribute name="NAME" x="13.89" y="11.398" size="0.6096" layer="25" font="vector" ratio="20" rot="R180" align="bottom-center"/>
+<attribute name="PROD_ID" value="CAP-00810" x="13.89" y="10.06" size="1.778" layer="27" rot="R180" display="off"/>
+<attribute name="VALUE" x="13.89" y="10.822" size="0.6096" layer="27" font="vector" ratio="20" rot="R180" align="top-center"/>
 </element>
 <element name="P1" library="adafruit" library_urn="urn:adsk.eagle:library:420" package="JST-PH-2-SMT-RA" package3d_urn="urn:adsk.eagle:package:6240692/1" value="" x="3.418" y="25.658" smashed="yes" rot="R90">
@@
 <attribute name="VALUE" x="5.332" y="9.511" size="1.27" layer="27" rot="R90"/>
 </element>
-<element name="C1" library="SparkFun-Capacitors" library_urn="urn:adsk.eagle:library:510" package="0603" package3d_urn="urn:adsk.eagle:package:37414/1" value="0.1uF" x="10.45" y="5.8" smashed="yes" rot="R180">
-<attribute name="NAME" x="10.45" y="7.138" size="0.6096" layer="25" font="vector" ratio="20" rot="R180" align="bottom-center"/>
-<attribute name="PROD_ID" value="CAP-00810" x="10.45" y="5.8" size="1.778" layer="27" rot="R180" display="off"/>
-<attribute name="VALUE" x="10.45" y="6.562" size="0.6096" layer="27" font="vector" ratio="20" rot="R180" align="top-center"/>
-</element>
-<element name="C9" library="SparkFun-Capacitors" library_urn="urn:adsk.eagle:library:510" package="0603" package3d_urn="urn:adsk.eagle:package:37414/1" value="0.1uF" x="10.45" y="3.525" smashed="yes" rot="R180">
-<attribute name="NAME" x="10.45" y="4.863" size="0.6096" layer="25" font="vector" ratio="20" rot="R180" align="bottom-center"/>
-<attribute name="PROD_ID" value="CAP-00810" x="10.45" y="3.525" size="1.778" layer="27" rot="R180" display="off"/>
-<attribute name="VALUE" x="10.45" y="4.287" size="0.6096" layer="27" font="vector" ratio="20" rot="R180" align="top-center"/>
+<element name="C1" library="SparkFun-Capacitors" library_urn="urn:adsk.eagle:library:510" package="0603" package3d_urn="urn:adsk.eagle:package:37414/1" value="0.1uF" x="10.45" y="5.4" smashed="yes" rot="R180">
+<attribute name="NAME" x="10.45" y="6.738" size="0.6096" layer="25" font="vector" ratio="20" rot="R180" align="bottom-center"/>
+<attribute name="PROD_ID" value="CAP-00810" x="10.45" y="5.4" size="1.778" layer="27" rot="R180" display="off"/>
+<attribute name="VALUE" x="10.45" y="6.162" size="0.6096" layer="27" font="vector" ratio="20" rot="R180" align="top-center"/>
+</element>
+<element name="C9" library="SparkFun-Capacitors" library_urn="urn:adsk.eagle:library:510" package="0603" package3d_urn="urn:adsk.eagle:package:37414/1" value="0.1uF" x="10.45" y="3.225" smashed="yes" rot="R180">
+<attribute name="NAME" x="10.45" y="4.563" size="0.6096" layer="25" font="vector" ratio="20" rot="R180" align="bottom-center"/>
+<attribute name="PROD_ID" value="CAP-00810" x="10.45" y="3.225" size="1.778" layer="27" rot="R180" display="off"/>
+<attribute name="VALUE" x="10.45" y="3.987" size="0.6096" layer="27" font="vector" ratio="20" rot="R180" align="top-center"/>
 </element>
 <element name="C10" library="SparkFun-Capacitors" library_urn="urn:adsk.eagle:library:510" package="0603" package3d_urn="urn:adsk.eagle:package:37414/1" value="0.1uF" x="13.845" y="3.525" smashed="yes" rot="R180">
@@
 <attribute name="VALUE" x="13.845" y="2.012" size="0.6096" layer="27" font="vector" ratio="20" rot="R180" align="top-center"/>
 </element>
-<element name="C12" library="SparkFun-Capacitors" library_urn="urn:adsk.eagle:library:510" package="0603" package3d_urn="urn:adsk.eagle:package:37414/1" value="10nF" x="13.84" y="11.9" smashed="yes" rot="R180">
-<attribute name="NAME" x="13.84" y="13.038" size="0.6096" layer="25" font="vector" ratio="20" rot="R180" align="bottom-center"/>
-<attribute name="PROD_ID" value="CAP-00867" x="13.84" y="11.9" size="1.778" layer="27" rot="R180" display="off"/>
-<attribute name="VALUE" x="13.84" y="12.662" size="0.6096" layer="27" font="vector" ratio="20" rot="R180" align="top-center"/>
+<element name="C12" library="SparkFun-Capacitors" library_urn="urn:adsk.eagle:library:510" package="0603" package3d_urn="urn:adsk.eagle:package:37414/1" value="10nF" x="13.84" y="12.3" smashed="yes" rot="R180">
+<attribute name="NAME" x="13.84" y="13.638" size="0.6096" layer="25" font="vector" ratio="20" rot="R180" align="bottom-center"/>
+<attribute name="PROD_ID" value="CAP-00867" x="13.84" y="12.3" size="1.778" layer="27" rot="R180" display="off"/>
+<attribute name="VALUE" x="13.84" y="13.062" size="0.6096" layer="27" font="vector" ratio="20" rot="R180" align="top-center"/>
 </element>
 </elements>
@@
 <wire x1="8" y1="23.776" x2="8" y2="23" width="0.508" layer="1"/>
 <via x="8" y="23" extent="1-16" drill="0.381"/>
-<wire x1="9.6" y1="5.8" x2="9.6" y2="3.525" width="0.4064" layer="1"/>
+<wire x1="9.6" y1="5.4" x2="9.6" y2="3.225" width="0.4064" layer="1"/>
 <wire x1="12.995" y1="5.82" x2="12.995" y2="3.525" width="0.4064" layer="1"/>
 <wire x1="12.995" y1="3.525" x2="12.995" y2="1.25" width="0.4064" layer="1"/>
@@
 <wire x1="12.745" y1="1" x2="11" y2="1" width="0.4064" layer="1"/>
 <via x="11" y="1" extent="1-16" drill="0.381"/>
-<wire x1="9.6" y1="3.525" x2="11" y2="2.125" width="0.4064" layer="1"/>
-<wire x1="11" y1="2.125" x2="11" y2="1" width="0.4064" layer="1"/>
+<wire x1="9.6" y1="3.225" x2="11" y2="1.825" width="0.4064" layer="1"/>
+<wire x1="11" y1="1.825" x2="11" y2="1" width="0.4064" layer="1"/>
 <wire x1="12.995" y1="8" x2="12.995" y2="5.82" width="0.4064" layer="1"/>
-<wire x1="12.99" y1="11.9" x2="12.99" y2="13.99" width="0.4064" layer="1"/>
+<wire x1="12.99" y1="12.3" x2="12.99" y2="13.99" width="0.4064" layer="1"/>
 <wire x1="12.99" y1="13.99" x2="13" y2="14" width="0.4064" layer="1"/>
 <via x="13" y="14" extent="1-16" drill="0.381"/>
 <wire x1="13.945" y1="16.195" x2="13.945" y2="14.945" width="0.4064" layer="1"/>
 <wire x1="13.945" y1="14.945" x2="13" y2="14" width="0.4064" layer="1"/>
+<wire x1="13.04" y1="10.06" x2="12.99" y2="10.11" width="0.4064" layer="1"/>
+<wire x1="12.99" y1="10.11" x2="12.99" y2="12.3" width="0.4064" layer="1"/>
 <wire x1="27.945" y1="16.195" x2="25.945" y2="32.395" width="0" layer="19" extent="1-1"/>
 <wire x1="25.5" y1="13.38" x2="27.945" y2="16.195" width="0" layer="19" extent="1-1"/>
@@
 <wire x1="16.62" y1="8.5" x2="19.1" y2="13.38" width="0" layer="19" extent="1-1"/>
 <wire x1="12.995" y1="8" x2="16.62" y2="8.5" width="0" layer="19" extent="1-1"/>
-<wire x1="7.6" y1="3.3" x2="9.6" y2="3.525" width="0" layer="19" extent="1-1"/>
-<wire x1="7.5" y1="5.75" x2="9.6" y2="5.8" width="0" layer="19" extent="1-1"/>
 <wire x1="0.5468" y1="3.3" x2="1" y2="3.3" width="0" layer="19" extent="1-1"/>
-<wire x1="5.745" y1="9.3" x2="5.6" y2="5.975" width="0" layer="19" extent="1-1"/>
-<wire x1="5" y1="11" x2="5.745" y2="9.3" width="0" layer="19" extent="1-1"/>
-<wire x1="5.745" y1="12.9" x2="5" y2="11" width="0" layer="19" extent="1-1"/>
-<wire x1="3.372675" y1="13.5" x2="5.745" y2="12.9" width="0" layer="19" extent="1-1"/>
-<wire x1="3.622175" y1="15.55" x2="3.372675" y2="13.5" width="0" layer="19" extent="1-1"/>
-<wire x1="12.99" y1="11.9" x2="12.995" y2="8" width="0" layer="19" extent="1-1"/>
 <wire x1="20.7" y1="2.02" x2="16.62" y2="8.5" width="0" layer="19" extent="1-1"/>
 <wire x1="27.98" y1="3.7" x2="20.7" y2="2.02" width="0" layer="19" extent="1-1"/>
-<wire x1="35.84" y1="16.46" x2="27.945" y2="16.195" width="0" layer="19" extent="1-1"/>
-<wire x1="40.57" y1="14.31" x2="35.84" y2="16.46" width="0" layer="19" extent="1-1"/>
-<wire x1="8" y1="23" x2="3.622175" y2="15.55" width="0" layer="19" extent="1-1"/>
 </signal>
 <signal name="DISP_RESET">
@@
 <vertex x="43" y="33"/>
 </polygon>
-<wire x1="11.3" y1="3.525" x2="11.3" y2="5.8" width="0" layer="19" extent="1-1"/>
-<wire x1="14.695" y1="5.82" x2="11.3" y2="5.8" width="0" layer="19" extent="1-1"/>
+<wire x1="11.3" y1="3.225" x2="11.3" y2="5.4" width="0" layer="19" extent="1-1"/>
+<wire x1="14.695" y1="5.82" x2="11.3" y2="5.4" width="0" layer="19" extent="1-1"/>
 </signal>
 <signal name="N$3">
@@
 <contactref element="U2" pad="42"/>
 <contactref element="C12" pad="1"/>
-<wire x1="14.69" y1="11.9" x2="19.9" y2="13.38" width="0" layer="19" extent="1-1"/>
+<wire x1="14.69" y1="12.3" x2="19.9" y2="13.38" width="0" layer="19" extent="1-1"/>
 </signal>
 <signal name="N$1">

Commit message: Rearranged radio board
Parts:
- added C13, C14: 33pF, SparkFun-Capacitors:0603
- added D1: 9V, RoboJackets-LEDs:CHIP-LED0603
- added D2: 3.3V, RoboJackets-LEDs:CHIP-LED0603
- added R3: 3.9K, SparkFun-Resistors:0603
- added R4: 800Ω, SparkFun-Resistors:0603-RES
- added U$1, U$2, U$3, U$4, U$5: BUTTON, I'mRADIOactive:1X02
- added Y1: ECS-80-20-5PX-TR, I'mRADIOactive:XTAL_ECS-80-20-5PX-TR
- R1, R2: device adafruit:R0603 -> SparkFun-Resistors:0603-RES
- moved C2 36.1 mm to (37.1, 33.4)
- moved C3 27.9 mm to (19.1, 37.5)
- moved C9 17.1 mm to (27.4, 5.22), turned to 270 degrees
- moved C10 15.5 mm to (22.6, 16.3)
- moved JP1 15.0 mm to (40.6, 24.2)
- moved C1 11.6 mm to (14.4, 16.3), turned to 0 degrees
- moved C12 6.17 mm to (18.5, 16.3), turned to 0 degrees
- moved C4 4.22 mm to (10.2, 5.80)
- moved U2 3.35 mm to (19.1, 8.70)
- moved JP2 3.00 mm to (41.0, 35.0)
- moved U1 3.00 mm to (20.9, 27.3)
- moved C11 1.26 mm to (15.0, 0.85)
- moved R1 0.22 mm to (1.30, 10.2)
- moved R2 0.22 mm to (3.20, 10.2)
Connections:
- new net N$10: D2.C, R4.1
- new net N$6: C13.1, U2.16, Y1.2
- new net N$8: C14.1, U2.17, Y1.1
- new net N$9: D1.C, R3.1
- net 3.3V: now also D2.A
- net 9V: now also D1.A
- net CS3: now also U2.30; no longer U2.38
- net DC_SELECT: now also U2.28; no longer U2.36
- net DISP_RESET: now also U2.29; no longer U2.37
- net GND: now also C13.2, C14.2, R3.2, R4.2
- net INT: now also U2.36; no longer U2.30
- net RADIO_RESET: now also U2.37; no longer U2.28
- net SS3: now also U2.38; no longer U2.29
Routing:
- net DIFF1_N: track 20.6 -> 0.00 mm, vias 2 -> 0
- net DIFF1_P: track 19.9 -> 0.00 mm, vias 2 -> 0
- net N$6: track 0.00 -> 16.5 mm
- net INT: track 0.00 -> 15.3 mm, vias 0 -> 1
- net N$3: track 0.00 -> 13.2 mm
- net N$8: track 0.00 -> 4.73 mm
- net N$5: track 2.05 -> 0.00 mm
- net GND: track 35.8 -> 34.1 mm, vias 4 -> 9
- net SS3: track 0.00 -> 1.63 mm
- net MOSI3: track 0.00 -> 1.49 mm
- net N$4: track 0.00 -> 1.44 mm, vias 0 -> 1
- net SCK3: track 0.00 -> 1.35 mm
- net MISO: track 0.00 -> 1.35 mm

Commit message: Wired radio board
Parts:
- removed U$2, U$3, U$4, U$5: BUTTON, I'mRADIOactive:1X02
- added R5, R6, R7, R8, R9: 10K, SparkFun-Resistors:0603-RES
- added U5, U7, U8, U9: BUTTON, I'mRADIOactive:1X02
- D1: value 9V -> GREEN
- D2: value 3.3V -> GREEN
- R3: value 3.9K -> 400Ω; device SparkFun-Resistors:0603 -> SparkFun-Resistors:0603-RES
- R4: value 800Ω -> 100Ω
- moved C3 1.70 mm to (20.8, 37.4), turned to 0 degrees
- moved C9 1.00 mm to (27.4, 4.22)
- moved C4 0.51 mm to (10.3, 6.30)
- renumbered U$1 to U6
Connections:
- new net N$11: R5.1, U2.20, U5.2
- new net N$12: R6.1, U2.21, U6.2
- new net N$13: R7.1, U2.25, U7.2
- new net N$14: R8.1, U2.26, U8.2
- new net N$15: R9.1, U2.27, U9.2
- net 3.3V: now also U5.1, U6.1, U7.1, U9.1
- net GND: now also R5.2, R6.2, R7.2, R8.2, R9.2
Routing:
- net GND: track 34.1 -> 80.3 mm, vias 9 -> 23
- net MOSI3: track 1.49 -> 46.2 mm, vias 0 -> 3
- net SCK3: track 1.35 -> 43.2 mm, vias 0 -> 3
- net N$11: track 0.00 -> 27.2 mm, vias 0 -> 2
- net N$8: track 4.73 -> 29.4 mm
- net CS3: track 0.00 -> 24.3 mm, vias 0 -> 1
- net DISP_RESET: track 0.00 -> 23.1 mm, vias 0 -> 1
- net N$6: track 16.5 -> 39.2 mm
- net DC_SELECT: track 0.00 -> 22.7 mm, vias 0 -> 1
- net N$4: track 1.44 -> 24.0 mm, vias 1 -> 2
- net N$12: track 0.00 -> 20.1 mm, vias 0 -> 2
- net N$13: track 0.00 -> 19.8 mm
- net MISO: track 1.35 -> 19.7 mm, vias 0 -> 2
- net 3.3V: track 13.2 -> 28.4 mm
- net N$15: track 0.00 -> 14.9 mm
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
Commit message: Finished wiring Radio pcb
Parts:
- U3: value (none) -> AP63203WU-7
- renumbered U5 to J2, U6 to J3, U7 to J4
Connections:
- net 3.3V: now also U8.1
- net N$14: now also U2.22; no longer U2.26
Routing:
- net N$4: track 24.0 -> 15.7 mm
- net N$14: track 12.6 -> 17.1 mm, vias 0 -> 2
- net RADIO_RESET: track 11.3 -> 13.9 mm
- net GND: track 80.3 -> 82.1 mm
- net MISO: track 19.7 -> 21.2 mm
- net SS3: track 9.41 -> 10.6 mm
- net N$6: vias 0 -> 2
- net N$8: vias 0 -> 2

Commit message: Added reset button
Parts:
- added C15: 0.1uF, SparkFun-Capacitors:0603
- added R10: 10K, SparkFun-Resistors:0603-RES
- added S1: KMR2, RoboJackets-Switches:KMR2
- C7, C8: value 22UF-1210-16V-20% -> 22uF
- moved D1 7.13 mm to (1.90, 31.4)
- moved R4 5.35 mm to (8.20, 33.8)
- moved D2 3.69 mm to (8.20, 31.4)
- moved R3 1.97 mm to (2.10, 33.8), turned to 0 degrees
- renumbered U8 to J5, U9 to J6
Connections:
- removed net RESET: U2.13
- new net N$17: C15.1, R10.2, S1.1.1, S1.1.2, U2.13
- net 3.3V: now also R10.1
- net GND: now also C15.2, S1.2.1, S1.2.2
Routing:
- net N$17: track 0.00 -> 43.9 mm, vias 0 -> 2
- net 3.3V: track 28.4 -> 45.4 mm
- net GND: track 82.1 -> 91.9 mm, vias 23 -> 24
- net N$9: track 4.40 -> 2.39 mm
- net N$10: track 4.40 -> 3.01 mm
Other:
- board size 42.6 x 44.3 mm -> 42.6 x 38.3 mm
