File: Radio/Radii/Radii.sch (EAGLE design)
At the start: 14 parts, among them U2 LEV_SHIFT

Commit message: Radii Style Guide Changes
Parts:
- removed CN1: (no value), adafruit:JST_2PIN-SMT-RA
- removed U$1: NANO, I'mRADIOactive:NANO
- removed U$2: XC9140C501MR-G, I'mRADIOactive:XC9140C501MR-G
- added P1: (no value), adafruit:JST_2PIN-SMT-RA
- added U3: XC9140C501MR-G, I'mRADIOactive:XC9140C501MR-G
- added U4: NANO, I'mRADIOactive:NANO
Connections:
- removed net MISO3: U1.MISO, U2.1Y
- removed net MISO5: U$1.D12, U2.1A
- new net MISO: U1.MISO, U4.D12
- net 3.3V: now also P1.2, U3.VBAT; no longer CN1.2, U$2.VBAT
- net 5V: now also U3.VOUT, U4.RAW; no longer U$1.RAW, U$2.VOUT
- net CS5: now also U4.D10; no longer U$1.D10
- net DC_SELECT: now also U4.D8; no longer U$1.D8
- net DISP_RESET: now also U4.D9; no longer U$1.D9
- net GND: now also P1.1, U3.GND, U4.GND; no longer CN1.1, U$1.GND, U$2.GND
- net INT5: now also U4.D4; no longer U$1.D4
- net MOSI5: now also U4.D11; no longer U$1.D11
- net N$1: now also U3.LX; no longer U$2.LX
- net N$2: now also U3.CE; no longer U$2.CE
- net SCK5: now also U4.D13; no longer U$1.D13
- net SS5: now also U4.D5; no longer U$1.D5
Other:
- note added: "5V to 3V Level Shifter"
- note added: "Arduino Nano Pinout"
- note added: "Do not ever activate pin D12 as output"
- note added: "LCD Display"
- note added: "Power"
- note added: "Radio Debugging Device for Sumo Bot"
- note added: "Radio Module"
- note added: "RoboWrestling"
- moved on the sheet: C1, C2, C3, C4, C5, C6, JP1, JP2, L1, U1, U2

Commit message: Changed to MCU
Parts:
- removed C5: 10uF, SparkFun-Capacitors:10UF-0603-6.3V-20%
- removed C6: 0.1uF, SparkFun-Capacitors:0.1UF-0603-25V-(+80/-20%)
- removed L1: 4.7μH, I'mRADIOactive:SRN3015-4R7M
- removed U2: LEV_SHIFT, I'mRADIOactive:74HC4050D,653
- removed U3: XC9140C501MR-G, I'mRADIOactive:XC9140C501MR-G
- removed U4: NANO, I'mRADIOactive:NANO
- added U$1: STM32F0, I'mRADIOactive:STM32F0
- C4: value 4.7pF -> 0.1uF; device SparkFun-Capacitors:4.7PF-0603-50V-5% -> SparkFun-Capacitors:0.1UF-0603-25V-(+80/-20%)
Connections:
- removed net 5V: C1.1, C2.1, C5.1, JP1.1, U3.VOUT, U4.RAW
- removed net INT5: U2.5A, U4.D4
- removed net MOSI5: JP1.4, U2.2A, U4.D11
- removed net N$1: L1.1, U3.LX
- removed net N$2: U3.CE
- removed net SCK5: JP1.3, U2.3A, U4.D13
- removed net SS5: U2.4A, U4.D5
- new net CS3: JP1.5
- new net RESET: U$1.NRST
- net 3.3V: now also C1.1, C2.1, JP1.1, U$1.VSS, U$1.VSSA; no longer C6.1, L1.2, U2.VCC, U3.VBAT
- net CS5: now also U$1.PB12; no longer JP1.5, U4.D10
- net DC_SELECT: now also U$1.PA3, U$1.PB14; no longer U4.D8
- net DISP_RESET: now also U$1.PA2, U$1.PB13; no longer U4.D9
- net GND: now also U$1.VDD, U$1.VDDA; no longer C5.2, C6.2, U2.GND, U3.GND, U4.GND
- net INT: now also U$1.PA1; no longer U2.5Y
- net MISO: now also U$1.PA6; no longer U4.D12
- net MOSI3: now also JP1.4, U$1.PA7; no longer U2.2Y
- net SCK3: now also JP1.3, U$1.PA5; no longer U2.3Y
- net SS3: now also U$1.PA4; no longer U2.4Y
Other:
- note added: "MCU Pinout"
- note removed: "5V to 3V Level Shifter"
- note removed: "Arduino Nano Pinout"
- note removed: "Do not ever activate pin D12 as output"
- moved on the sheet: C1, C2, C4, JP1, P1

Commit message: Updated Power Regulators
Parts:
- added C5: 10uF, SparkFun-Capacitors:10UF-0603-6.3V-20%
- added C6: 0.1uF, SparkFun-Capacitors:0.1UF-0603-25V-(+80/-20%)
- added C7: 44uF, SparkFun-Capacitors:10UF-0603-6.3V-20%
- added L1: SRN3015-4R7M, I'mRADIOactive:SRN3015-4R7M
- added U$2, U$3: AP63203WU-7, I'mRADIOactive:AP63203WU-7
Connections:
- new net N$1: C6.2, L1.2, U$3.SW
- new net N$2: C6.1, U$3.BST
- new net RADIO_RESET: U$1.PB0, U1.RESET
- net 3.3V: now also C5.1, C7.1, L1.1, U$3.EN, U$3.FB, U$3.VIN
- net GND: now also C5.2, C7.2, U$3.GND
Other:
- note added: "44uF capacitor doesn't exist"
- moved on the sheet: C4, P1

Commit message: Wired radio board
Parts:
- removed L1: SRN3015-4R7M, I'mRADIOactive:SRN3015-4R7M
- added C8: 22UF-1210-16V-20%, SparkFun-Capacitors:22UF-1210-16V-20%
- C7: value 44uF -> 22UF-1210-16V-20%; device SparkFun-Capacitors:10UF-0603-6.3V-20% -> SparkFun-Capacitors:22UF-1210-16V-20%
- U$2: value AP63203WU-7 -> IND_1255AY-3R9N=P3; device I'mRADIOactive:AP63203WU-7 -> I'mRADIOactive:IND_1255AY-3R9N=P3
Connections:
- new net 9V: C5.1, P1.2, U$3.EN, U$3.VIN
- net 3.3V: now also C8.1, U$2.2; no longer C5.1, L1.1, P1.2, U$3.EN, U$3.VIN
- net DC_SELECT: now also U$1.PB13; no longer U$1.PA3, U$1.PB14
- net DISP_RESET: now also U$1.PB14; no longer U$1.PA2, U$1.PB13
- net GND: now also C8.2
- net N$1: now also U$2.1; no longer L1.2
- net RADIO_RESET: now also U$1.PA3; no longer U$1.PB0
Other:
- note removed: "44uF capacitor doesn't exist"

Commit message: Took out MCU from Radio
Parts:
- removed U$1: STM32F0, I'mRADIOactive:STM32F0
Connections:
- removed net CS5: U$1.PB12
- removed net RESET: U$1.NRST
- net 3.3V: no longer U$1.VSS, U$1.VSSA
- net DC_SELECT: no longer U$1.PB13
- net DISP_RESET: no longer U$1.PB14
- net GND: no longer U$1.VDD, U$1.VDDA
- net INT: no longer U$1.PA1
- net MISO: no longer U$1.PA6
- net MOSI3: no longer U$1.PA7
- net RADIO_RESET: no longer U$1.PA3
- net SCK3: no longer U$1.PA5
- net SS3: no longer U$1.PA4
Changed lines of the file:
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@@
 <part name="JP2" library="pinhead" library_urn="urn:adsk.eagle:library:325" deviceset="PINHD-1X1" device="" package3d_urn="urn:adsk.eagle:package:22485/2"/>
 <part name="FRAME1" library="RoboJackets-Frames" deviceset="FRAME_A_L" device=""/>
-<part name="U$1" library="I'mRADIOactive" deviceset="STM32F0" device=""/>
 <part name="SUPPLY2" library="SparkFun-PowerSymbols" library_urn="urn:adsk.eagle:library:530" deviceset="3.3V" device=""/>
 <part name="SUPPLY1" library="SparkFun-PowerSymbols" library_urn="urn:adsk.eagle:library:530" deviceset="3.3V" device=""/>
@@
 <attribute name="DRAWING_NAME" x="185.42" y="19.05" size="2.54" layer="94" font="vector"/>
 </instance>
-<instance part="U$1" gate="G$1" x="76.2" y="160.02" smashed="yes">
-<attribute name="NAME" x="70.866" y="191.77" size="1.778" layer="95"/>
-<attribute name="VALUE" x="71.12" y="124.46" size="1.778" layer="96"/>
-</instance>
 <instance part="SUPPLY2" gate="G$1" x="205.74" y="175.26" smashed="yes">
 <attribute name="VALUE" x="205.74" y="178.054" size="1.778" layer="96" align="bottom-center"/>
@@
 </segment>
 <segment>
-<pinref part="U$1" gate="G$1" pin="PA6"/>
 <wire x1="55.88" y1="149.86" x2="30.48" y2="149.86" width="0.1524" layer="91"/>
 <label x="30.48" y="149.86" size="1.778" layer="95" rot="R180" xref="yes"/>
@@
 <wire x1="55.88" y1="167.64" x2="49.022" y2="167.64" width="0.1524" layer="91"/>
 <junction x="49.022" y="167.64"/>
-<pinref part="U$1" gate="G$1" pin="VDDA"/>
 </segment>
 <segment>
@@
 <wire x1="55.88" y1="129.54" x2="41.402" y2="129.54" width="0.1524" layer="91"/>
 <junction x="41.402" y="129.54"/>
-<pinref part="U$1" gate="G$1" pin="VDD"/>
 </segment>
 <segment>
@@
 <wire x1="96.52" y1="187.96" x2="106.68" y2="187.96" width="0.1524" layer="91"/>
 <label x="106.68" y="187.96" size="1.778" layer="95" xref="yes"/>
-<pinref part="U$1" gate="G$1" pin="PB12"/>
 </segment>
 </net>
@@
 </segment>
 <segment>
-<pinref part="U$1" gate="G$1" pin="PB14"/>
 <wire x1="96.52" y1="182.88" x2="99.06" y2="182.88" width="0.1524" layer="91"/>
 <label x="99.06" y="182.88" size="1.778" layer="95" xref="yes"/>
@@
 </segment>
 <segment>
-<pinref part="U$1" gate="G$1" pin="PB13"/>
 <wire x1="96.52" y1="185.42" x2="116.84" y2="185.42" width="0.1524" layer="91"/>
 <label x="116.84" y="185.42" size="1.778" layer="95" xref="yes"/>
@@
 </segment>
 <segment>
-<pinref part="U$1" gate="G$1" pin="PA1"/>
 <wire x1="55.88" y1="162.56" x2="40.64" y2="162.56" width="0.1524" layer="91"/>
 <label x="40.64" y="162.56" size="1.778" layer="95" rot="R180" xref="yes"/>
@@
 <wire x1="36.322" y1="185.42" x2="31.242" y2="185.42" width="0.1524" layer="91"/>
 <wire x1="31.242" y1="185.42" x2="31.242" y2="180.34" width="0.1524" layer="91"/>
-<pinref part="U$1" gate="G$1" pin="VSSA"/>
 <pinref part="SUPPLY1" gate="G$1" pin="3.3V"/>
 <junction x="36.322" y="185.42"/>
@@
 <pinref part="SUPPLY4" gate="G$1" pin="3.3V"/>
 <junction x="28.702" y="139.7"/>
-<pinref part="U$1" gate="G$1" pin="VSS"/>
 </segment>
 <segment>
@@
 </segment>
 <segment>
-<pinref part="U$1" gate="G$1" pin="PA7"/>
 <wire x1="55.88" y1="147.32" x2="43.18" y2="147.32" width="0.1524" layer="91"/>
 <label x="43.18" y="147.32" size="1.778" layer="95" rot="R180" xref="yes"/>
@@
 </segment>
 <segment>
-<pinref part="U$1" gate="G$1" pin="PA5"/>
 <wire x1="55.88" y1="152.4" x2="40.64" y2="152.4" width="0.1524" layer="91"/>
 <label x="40.64" y="152.4" size="1.778" layer="95" rot="R180" xref="yes"/>
@@
 </segment>
 <segment>
-<pinref part="U$1" gate="G$1" pin="PA4"/>
 <wire x1="55.88" y1="154.94" x2="30.48" y2="154.94" width="0.1524" layer="91"/>
 <label x="30.48" y="154.94" size="1.778" layer="95" rot="R180" xref="yes"/>
@@
 <net name="RESET" class="0">
 <segment>
-<pinref part="U$1" gate="G$1" pin="NRST"/>
 <wire x1="55.88" y1="172.72" x2="53.34" y2="172.72" width="0.1524" layer="91"/>
 <label x="53.34" y="172.72" size="1.778" layer="95" rot="R180" xref="yes"/>
@@
 <segment>
 <label x="53.34" y="157.48" size="1.778" layer="95" rot="R180" xref="yes"/>
-<wire x1="54.864" y1="157.48" x2="53.34" y2="157.48" width="0.1524" layer="91"/>
-<pinref part="U$1" gate="G$1" pin="PA3"/>
-<wire x1="55.88" y1="157.48" x2="54.864" y2="157.48" width="0.1524" layer="91"/>
-</segment>
-</net>
+<wire x1="55.88" y1="157.48" x2="53.34" y2="157.48" width="0.1524" layer="91"/>
+</segment>
+</net>

Commit message: Added 22uH inductor
Parts:
- added U2: ATMEGA32U4-AU, I'mRADIOactive:ATMEGA32U4-AU
Changed lines of the file:
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@@
 <part name="SUPPLY5" library="SparkFun-PowerSymbols" library_urn="urn:adsk.eagle:library:530" deviceset="VCC_2" device="" value="9V"/>
 <part name="SUPPLY6" library="SparkFun-PowerSymbols" library_urn="urn:adsk.eagle:library:530" deviceset="VCC_2" device="" value="9V"/>
+<part name="U2" library="I'mRADIOactive" deviceset="ATMEGA32U4-AU" device=""/>
 </parts>
 <sheets>
@@
 <attribute name="VALUE" x="198.12" y="94.234" size="1.778" layer="96" align="bottom-center"/>
 </instance>
+<instance part="U2" gate="A" x="76.2" y="154.94" smashed="yes">
+<attribute name="NAME" x="70.402559375" y="189.4195" size="2.085040625" layer="95" ratio="10" rot="SR0"/>
+<attribute name="VALUE" x="72.56615" y="111.3338" size="2.08375" layer="96" ratio="10" rot="SR0"/>
+</instance>
 </instances>

Commit message: Organized board with 32u4
Parts:
- added J1: 10118193-0001LF, I'mRADIOactive:10118193-0001LF
- added R1, R2: 22Ω, adafruit:R-US_R0603
- C1, C4: value 0.1uF -> 1.0uF; device SparkFun-Capacitors:0.1UF-0603-25V-(+80/-20%) -> SparkFun-Capacitors:1.0UF-0603-16V-10%
- U2: value ATMEGA32U4-AU -> ATMEGA32U4-AUR; device I'mRADIOactive:ATMEGA32U4-AU -> I'mRADIOactive:ATMEGA32U4-AUR
- renumbered U$2 to U4, U$3 to U3
Connections:
- new net DIFF_N: J1.D-, R1.1
- new net DIFF_P: J1.D+, R2.1
- new net N$4: J1.VUSB, U2.VBUS
- new net N$5: C4.1, U2.UCAP
- new net N$6: R1.2, U2.D-
- new net N$8: R2.2, U2.D+
- new net RESET: U2.!RESET
- net 3.3V: now also U2.AVCC, U2.UVCC, U2.VCC; no longer C4.1
- net CS3: now also U2.PF5(ADC5/TMS)
- net DC_SELECT: now also U2.PF7(ADC7/TDI)
- net DISP_RESET: now also U2.PF6(ADC6/TDO)
- net GND: now also J1.GND, J1.SHIELD, U2.GND, U2.UGND
- net INT: now also U2.PB6(PCINT6/OC1B/OC4B/ADC)
- net MISO: now also U2.PB3(PDO/PCINT3/MISO)
- net MOSI3: now also U2.PB2(PDI/PCINT2/MOSI)
- net RADIO_RESET: now also U2.PB4(PCINT4/ADC11)
- net SCK3: now also U2.PB1(PCINT1/SCLK)
- net SS3: now also U2.PB5(PCINT5/OC1A/OC4B/ADC)
Other:
- note added: "AU and AUR have the same package, the AUR symbol was better, I'm using AU"
- moved on the sheet: C1, C4

Commit message: Redoing radio board
Parts:
- added C10, C11, C9: 0.1uF, SparkFun-Capacitors:0.1UF-0603-25V-(+80/-20%)
- added C12: 10nF, SparkFun-Capacitors:10NF-0603-50V-10%
- C1: value 1.0uF -> 0.1uF; device SparkFun-Capacitors:1.0UF-0603-16V-10% -> SparkFun-Capacitors:0.1UF-0603-25V-(+80/-20%)
Connections:
- net N$6 renamed DIFF1_N
- net N$8 renamed DIFF1_P
- new net N$7: C12.1, U2.AREF
- net 3.3V: now also C10.1, C11.1, C9.1; no longer U2.UVCC
- net GND: now also C10.2, C11.2, C12.2, C9.2
