File: Gucci/v4 pcb/Gucci_ControlBoard.sch (EAGLE design)
At the start: 69 parts, among them U1 PCA9306_LSSOP, U2 TEENSY_3.6_DIL, U5 LM393-8-SOIC, U6 AP2114H-1.8TRG1, U7 AP2114H-3.3TRG1

Commit message: Added Pull up Resistors
Finished on Gucci/Still need to route on Kirbi
Parts:
- added R10, R11, R6, R7, R8, R9: 1k, SparkFun-Resistors:1KOHM-0603-1/10W-1%
Connections:
- net +3.3V: now also R10.2, R11.2, R6.2, R7.2, R8.2, R9.2
- net ESC_TRX: now also R9.1; no longer R5.1
- net S1/TX: now also R10.1
- net S2/TX: now also R11.1
- net TRX1: now also R7.1; no longer R4.1
- net TRX2: now also R8.1; no longer R3.1
- net TXD1: now also R5.1
- net TXD2: now also R3.1
- net TXD5: now also R4.1
- net TXD6: now also R6.1
Other:
- note added: "*Note: The TX and RX labels refer to the respective Teensy connection (not the ESC pins)"
- note added: "*Note: The TX and RX labels refer to the respective Teensy connection (not the sensor pins)"
- moved on the sheet: R3, R4, R5
