File: Gucci/v4 pcb/Gucci_ControlBoard.brd (EAGLE design)
At the start: 66 x 56 mm, 65 parts, among them U1 PCA9306_LSSOP, U2 TEENSY_3.6_DIL, U5 LM393-8-SOIC, U6 AP2114H-1.8TRG1, U7 AP2114H-3.3TRG1

Commit message: Connected ESCs
Connectted ESCs (Added two multiplexers to Gucci/Changed RADIO_NSS to Pin 30)
Parts:
- removed ESC: MOLEX_1.25MM_4PIN_SMT, Kirbi_ControlBoard:MOLEX_1.25MM_4PIN_SMT
- added ESC1, ESC2: MOLEX_1.25MM_3PIN_SMT, Kirbi_ControlBoard:MOLEX_1.25MM_3PIN_SMT
- added ESC_RX, ESC_TX: MUX_74LVC1G157GV, Kirbi_ControlBoard:MUX_74LVC1G157GV
Connections:
- new net ESC_S: ESC_RX.P$6, ESC_TX.P$6, U2.36/A17
- new net ESC_TRX: ESC_RX.P$4, U2.34/A15
- new net ESC_TTX: ESC_TX.P$4, U2.33/A14
- new net S1/RX: ESC1.P$2, ESC_RX.P$3
- new net S2/RX: ESC2.P$2, ESC_RX.P$1
- new net S2/TX: ESC2.P$1, ESC_TX.P$1
- net +3.3V: now also ESC_RX.P$5, ESC_TX.P$5
- net GND: now also ESC1.P$3, ESC2.P$3
- net RADIO_NSS: now also U2.30; no longer U2.34/A15
- net S1/TX: now also ESC1.P$1, ESC_TX.P$3; no longer ESC.P$5, U2.33/A14
Routing:
- net +3.3V: track 157.9 -> 183.1 mm, vias 1 -> 3
- net S1/RX: track 0.00 -> 22.6 mm, vias 0 -> 2
- net ESC_S: track 0.00 -> 16.4 mm
- net S2/RX: track 0.00 -> 15.3 mm
- net RADIO_NSS: track 54.9 -> 39.8 mm
- net ESC_TRX: track 0.00 -> 13.2 mm
- net ESC_TTX: track 0.00 -> 10.7 mm
- net S1/TX: track 8.99 -> 17.4 mm, vias 0 -> 2
- net RADIO_SCK: track 78.3 -> 70.1 mm, vias 0 -> 2
- net S2/TX: track 0.00 -> 7.96 mm
Other:
- board text added: "Gucci Controller Board V2.0"

Commit message: Added Pull-up Resistors/Moved MUXs
Added Pull-up Resistors (1k OHM to RX line)
Added 6.2 OHM to 1.8 V LED
Moved MUXs and rerouted
Fixed SIlkscreen
Parts:
- removed U$2: BEL_FUSE_C1F_3.5, Kirbi_ControlBoard:BEL_FUSE_C1F_3.5
- added F1: 3.5, Kirbi_ControlBoard:BEL_FUSE_C1F_3.5
- added R2: 6.2, Kirbi_ControlBoard:0603
- added R3, R4, R5: 1k, SparkFun-Resistors:0603
- moved ESC_RX 14.6 mm to (43.6, 41.0)
- moved ESC_TX 11.0 mm to (40.0, 41.0)
- moved D4 3.00 mm to (26.0, 28.0)
- moved R20 3.00 mm to (21.0, 28.0)
- moved D3 2.00 mm to (17.0, 28.0)
- moved R19 2.00 mm to (12.0, 28.0)
- moved D2 1.00 mm to (8.00, 28.0)
- moved R1 0.50 mm to (10.4, 34.0)
- moved ESC2 0.30 mm to (46.4, 52.4)
Connections:
- new net N$9: D4.C, R2.1
- net +3.3V: now also R3.2, R4.2, R5.2
- net ESC_TRX: now also R5.1
- net GND: now also R2.2; no longer D4.C
- net N$6: now also F1.P$2; no longer U$2.P$2
- net N$7: now also F1.P$1; no longer U$2.P$1
- net TRX1: now also R4.1
- net TRX2: now also R3.1
Routing:
- net +3.3V: track 183.1 -> 212.3 mm, vias 3 -> 4
- net S1/RX: track 22.6 -> 8.85 mm
- net S1/TX: track 17.4 -> 8.21 mm
- net S2/RX: track 15.3 -> 10.4 mm
- net N$6: track 23.4 -> 27.8 mm
- net ESC_S: track 16.4 -> 12.0 mm
- net ESC_TRX: track 13.2 -> 8.90 mm
- net TRX2: track 37.3 -> 41.5 mm
- net S2/TX: track 7.96 -> 12.1 mm
- net GND: track 76.6 -> 79.7 mm
- net LINE_RF: track 78.7 -> 81.2 mm
- net ESC_TTX: track 10.7 -> 13.2 mm
- net 1.8V: track 20.4 -> 18.1 mm
- net N$9: track 0.00 -> 2.27 mm
- net TRX1: track 20.7 -> 22.9 mm
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Other:
- board text removed: "Kirbi Controller Board V1.0"

Commit message: esc routing fix
Parts:
- moved ESC_RX 11.0 mm to (50.0, 50.0), turned to 270 degrees
- moved ESC_TX 9.22 mm to (42.0, 50.0), turned to 270 degrees
Connections:
- net GND: now also ESC_RX.P$2, ESC_TX.P$2
Routing:
- net +3.3V: track 212.3 -> 202.0 mm, vias 4 -> 3
- net S2/TX: track 12.1 -> 2.05 mm
- net ESC_S: track 12.0 -> 17.4 mm, vias 0 -> 2
- net S2/RX: track 10.4 -> 5.91 mm
- net S1/RX: track 8.85 -> 12.9 mm, vias 2 -> 0
- net S1/TX: track 8.21 -> 11.6 mm, vias 2 -> 0
- net TXD4: track 45.2 -> 47.4 mm
- net ESC_TTX: track 13.2 -> 11.5 mm, vias 0 -> 1
- net ESC_TRX: track 8.90 -> 7.55 mm
- net LINE_LF: track 71.1 -> 71.8 mm, vias 2 -> 1

Commit message: Added Pull up Resistors
Finished on Gucci/Still need to route on Kirbi
Parts:
- added R10, R11, R6, R7, R8, R9: 1k, SparkFun-Resistors:0603
- moved R5 56.2 mm to (0.30, 14.0), turned to 0 degrees
- moved R4 32.0 mm to (36.6, 14.0), turned to 180 degrees
- moved R3 27.9 mm to (0.20, 10.3), turned to 315 degrees
- moved C15 0.36 mm to (-1.10, 9.00)
Connections:
- net +3.3V: now also R10.2, R11.2, R6.2, R7.2, R8.2, R9.2
- net ESC_TRX: now also R9.1; no longer R5.1
- net S1/TX: now also R10.1
- net S2/TX: now also R11.1
- net TRX1: now also R7.1; no longer R4.1
- net TRX2: now also R8.1; no longer R3.1
- net TXD1: now also R5.1
- net TXD2: now also R3.1
- net TXD5: now also R4.1
- net TXD6: now also R6.1
Routing:
- net +3.3V: track 202.0 -> 235.5 mm, vias 3 -> 4
- net TXD2: track 5.39 -> 15.1 mm, vias 0 -> 2
- net S2/TX: track 2.05 -> 9.77 mm, vias 0 -> 2
- net TXD1: track 11.6 -> 18.6 mm, vias 0 -> 2
- net RADIO_SCK: track 68.9 -> 74.9 mm
- net TXD6: track 13.1 -> 16.4 mm, vias 0 -> 1
- net S1/TX: track 11.6 -> 13.9 mm
- net TXD5: track 8.45 -> 10.1 mm
- net GND: track 79.7 -> 78.8 mm
- net RXD2: track 9.82 -> 9.00 mm
- net LINE_LF: track 71.8 -> 72.3 mm

Commit message: Finished routing pull-up resistors
Finished routing pull-up resistors (mainly on Kirbi)
Changed lines of the file:
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@@
 <drawing>
 <settings>
-<setting alwaysvectorfont="yes"/>
+<setting alwaysvectorfont="no"/>
 <setting verticaltext="up"/>
 </settings>
@@
 </element>
 <element name="R5" library="SparkFun-Resistors" library_urn="urn:adsk.eagle:library:532" package="0603" package3d_urn="urn:adsk.eagle:package:39650/1" value="1k" x="0.3" y="14" smashed="yes">
-<attribute name="NAME" x="0.3" y="14.762" size="0.8128" layer="25" font="vector" ratio="20" align="bottom-center"/>
+<attribute name="NAME" x="2.7" y="13.662" size="0.8128" layer="25" font="vector" ratio="20" align="bottom-center"/>
 <attribute name="PROD_ID" value="RES-07856" x="0.3" y="14" size="1.778" layer="27" display="off"/>
 <attribute name="VALUE" x="0.3" y="13.238" size="0.6096" layer="27" font="vector" ratio="20" align="top-center"/>
