File: Radio/Radii.brd (EAGLE design)
At the start: 42.6 x 38.3 mm, 42 parts, among them J1 10118193-0001LF, J2 BUTTON, J3 BUTTON, J4 BUTTON, J5 BUTTON, J6 BUTTON, U2 ATMEGA32U4-AU, U3 AP63203WU-7, U4 IND_1255AY-3R9N=P3, Y1 ECS-80-20-5PX-TR

Commit message: Added pFET
Parts:
- added Q1: (no value), RoboJackets-Discrete:SOT-23-3
- added R11: 10K, SparkFun-Resistors:0603-RES
- moved C10 3.60 mm to (26.2, 16.3)
- moved C8 2.00 mm to (7.50, 7.30)
- moved C4 2.00 mm to (10.3, 4.30)
- moved C5 2.00 mm to (2.52, 11.5)
- moved C6 2.00 mm to (2.65, 17.7)
- moved C7 2.00 mm to (7.50, 10.9)
- moved P1 2.00 mm to (3.42, 23.7)
- moved R1 2.00 mm to (1.30, 8.20)
- moved R2 2.00 mm to (3.20, 8.20)
- moved U3 2.00 mm to (2.52, 14.5)
- moved U4 2.00 mm to (8.30, 15.9)
- moved J1 1.80 mm to (4.20, 1.50)
Connections:
- new net VCC: P1.1, Q1.3
- net 3.3V: now also R11.2
- net 9V: now also Q1.2; no longer P1.1
- net GND: now also Q1.1
- net SS3: now also R11.1
Routing:
- net 9V: track 22.5 -> 31.9 mm
- net VCC: track 0.00 -> 6.90 mm
- net VUSB: track 16.0 -> 19.7 mm
- net GND: track 85.6 -> 89.0 mm, vias 30 -> 28
- net SS3: track 10.4 -> 13.3 mm
- net N$5: track 3.67 -> 5.63 mm
- net DIFF1_P: track 13.0 -> 14.6 mm
- net DIFF1_N: track 15.0 -> 15.8 mm
- net 3.3V: track 48.1 -> 48.7 mm

Commit message: Added debouncing filters for buttons
Parts:
- added C16, C17, C18, C19, C20: 0.1uF, SparkFun-Capacitors:0603
- added R12, R14, R16: 1K, SparkFun-Resistors:0603-RES
- added R13, R15: 10K, SparkFun-Resistors:0603-RES
- R7, R9: value 10K -> 1K
- moved R7 12.3 mm to (29.8, 5.15), turned to 270 degrees
- moved R8 8.08 mm to (41.7, 12.6), turned to 270 degrees
- moved R9 5.26 mm to (36.1, 9.10), turned to 270 degrees
- moved J6 3.33 mm to (33.5, 16.2)
- moved J5 1.26 mm to (30.3, 9.05)
- moved J4 1.12 mm to (38.4, 9.05)
- moved R5 0.92 mm to (41.7, 5.15), turned to 270 degrees
- moved R6 0.92 mm to (34.7, 5.15), turned to 270 degrees
- moved C9 0.80 mm to (27.4, 5.03)
- moved J3 0.73 mm to (30.3, 1.80)
- moved J2 0.50 mm to (38.4, 1.70)
Connections:
- net CS3 renamed CS
- net MOSI3 renamed MOSI
- net SCK3 renamed SCK
- net SS3 renamed SS
- new net N$11: J2.2, R12.2, R5.2
- new net N$12: J4.2, R8.2, R9.2
- new net N$13: J5.2, R13.2, R14.2
- new net N$14: J6.2, R15.2, R16.2
- new net N$4: J3.2, R6.2, R7.2
- net BUTTON1: now also C17.1, R7.1; no longer J2.2, R5.1
- net BUTTON2: now also C16.1, R12.1; no longer J3.2, R6.1
- net BUTTON3: now also C19.1, R14.1; no longer J4.2, R7.1
- net BUTTON4: now also C18.1, R9.1; no longer J5.2, R8.1
- net BUTTON5: now also C20.1, R16.1; no longer J6.2, R9.1
- net GND: now also C16.2, C17.2, C18.2, C19.2, C20.2, R13.1, R15.1, R5.1, R6.1, R8.1; no longer R5.2, R6.2, R7.2, R8.2, R9.2
Routing:
- net BUTTON1: track 27.4 -> 14.3 mm, vias 2 -> 0
- net BUTTON3: track 19.8 -> 9.58 mm
- net N$12: track 0.00 -> 8.49 mm
- net N$14: track 0.00 -> 8.13 mm
- net N$11: track 0.00 -> 7.63 mm
- net N$4: track 0.00 -> 7.35 mm
- net N$13: track 0.00 -> 7.29 mm
- net GND: track 89.0 -> 94.9 mm
- net BUTTON4: track 17.1 -> 21.9 mm
- net BUTTON2: track 20.3 -> 22.6 mm
- net VUSB: track 19.7 -> 17.6 mm
- net BUTTON5: track 14.9 -> 16.9 mm, vias 0 -> 2
- net DC_SELECT: track 23.1 -> 25.0 mm
- net DIFF1_P: track 14.6 -> 13.2 mm
- net CS: track 24.6 -> 23.9 mm
Other:
- board size 42.6 x 38.3 mm -> 42.6 x 44.3 mm

Commit message: Added pullup to display
Parts:
- added R17: 10K, SparkFun-Resistors:0603-RES
Connections:
- removed net N$5: C4.1, U2.6
- net 3.3V: now also C4.1, R17.2, U2.6
- net CS: now also R17.1
Routing:
- net N$5: track 5.65 -> 0.00 mm
- net 3.3V: track 48.4 -> 54.0 mm
- net CS: track 23.9 -> 29.2 mm, vias 1 -> 2
- net GND: track 94.9 -> 90.7 mm, vias 28 -> 29
- net DIFF1_N: track 15.8 -> 14.5 mm
- net DIFF1_P: track 13.2 -> 12.2 mm
Changed lines of the file:
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@@
 <attribute name="VALUE" x="33.838" y="12.6" size="0.6096" layer="27" font="vector" ratio="20" rot="R270" align="top-center"/>
+</element>
+<element name="R17" library="SparkFun-Resistors" package="0603-RES" value="10K" x="37.4" y="26" smashed="yes" rot="R90">
+<attribute name="NAME" x="36.638" y="25.111" size="0.4064" layer="25" font="vector" rot="R90"/>
+<attribute name="PROD_ID" value="RES-00824" x="37.4" y="26" size="1.778" layer="27" rot="R90" display="off"/>
+<attribute name="VALUE" x="38.543" y="24.984" size="0.4064" layer="27" font="vector" rot="R90"/>
 </element>
 </elements>
@@
 <contactref element="C13" pad="2"/>
 <contactref element="C14" pad="2"/>
-<wire x1="37.4" y1="29.65" x2="37.4" y2="22.15" width="0.4064" layer="1"/>
 <wire x1="40.57" y1="29.31" x2="39.57" y2="28.31" width="0.4064" layer="1"/>
 <wire x1="39.57" y1="28.31" x2="38.74" y2="28.31" width="0.4064" layer="1"/>
@@
 <wire x1="19.39" y1="16.3" x2="20.6" y2="16.3" width="0.1524" layer="1"/>
 <via x="20.6" y="16.3" extent="1-16" drill="0.35"/>
-<wire x1="9.495" y1="4.3" x2="9.195" y2="4.3" width="0.1524" layer="1"/>
 <wire x1="24.78" y1="4.7" x2="24.8" y2="4.68" width="0.4064" layer="1"/>
 <wire x1="24.8" y1="4.68" x2="24.8" y2="3.7" width="0.4064" layer="1"/>
@@
 <wire x1="41.7" y1="13.45" x2="40.6" y2="14.55" width="0.2" layer="1"/>
 <wire x1="40.6" y1="14.55" x2="40.6" y2="14.6" width="0.2" layer="1"/>
-<wire x1="7.4" y1="3.95" x2="7.75" y2="4.3" width="0.2" layer="1"/>
-<wire x1="7.75" y1="4.3" x2="9.495" y2="4.3" width="0.2" layer="1"/>
-<wire x1="37.4" y1="29.65" x2="36.295" y2="33.42" width="0" layer="19" extent="1-1"/>
-<wire x1="40.6" y1="14.6" x2="37.4" y2="22.15" width="0" layer="19" extent="1-1"/>
-<wire x1="37" y1="11.75" x2="39.5" y2="13.45" width="0" layer="19" extent="1-1"/>
-<wire x1="36" y1="7" x2="35.8" y2="11.3" width="0" layer="19" extent="1-1"/>
-<wire x1="39.5" y1="6" x2="36" y2="7" width="0" layer="19" extent="1-1"/>
-<wire x1="30" y1="13.1628" x2="34.6" y2="11.75" width="0" layer="19" extent="1-1"/>
-<wire x1="27.095" y1="16.325" x2="28.65" y2="13.4" width="0" layer="19" extent="1-1"/>
-<wire x1="28.9777" y1="18.1777" x2="27.095" y2="16.325" width="0" layer="19" extent="1-1"/>
-<wire x1="22.3" y1="14.38" x2="25" y2="15" width="0" layer="19" extent="1-1"/>
-<wire x1="20.6" y1="16.3" x2="22.3" y2="14.38" width="0" layer="19" extent="1-1"/>
-<wire x1="16.5" y1="16.3" x2="19.39" y2="16.3" width="0" layer="19" extent="1-1"/>
-<wire x1="15.9" y1="14.38" x2="15.3" y2="16.3" width="0" layer="19" extent="1-1"/>
-<wire x1="12.9" y1="18" x2="15.3" y2="16.3" width="0" layer="19" extent="1-1"/>
-<wire x1="13.42" y1="9.5" x2="15.9223" y2="12.7" width="0" layer="19" extent="1-1"/>
-<wire x1="9.495" y1="4.3" x2="11" y2="7" width="0" layer="19" extent="1-1"/>
-<wire x1="7.5" y1="1.5" x2="5.4" y2="1.5" width="0" layer="19" extent="1-1"/>
-<wire x1="0.9" y1="1.5" x2="3" y2="1.5" width="0" layer="19" extent="1-1"/>
-<wire x1="5.745" y1="7.3" x2="5.5" y2="4.175" width="0" layer="19" extent="1-1"/>
-<wire x1="4.5" y1="7.2" x2="5.745" y2="7.3" width="0" layer="19" extent="1-1"/>
-<wire x1="5.7" y1="9.1" x2="5.745" y2="7.3" width="0" layer="19" extent="1-1"/>
-<wire x1="4.5" y1="10.2" x2="5.7" y2="9.1" width="0" layer="19" extent="1-1"/>
-<wire x1="5.745" y1="10.9" x2="4.5" y2="10.2" width="0" layer="19" extent="1-1"/>
-<wire x1="3.372675" y1="11.5" x2="4.5" y2="10.2" width="0" layer="19" extent="1-1"/>
-<wire x1="3.5" y1="12.6" x2="3.372675" y2="11.5" width="0" layer="19" extent="1-1"/>
-<wire x1="3.622175" y1="13.55" x2="3.5" y2="12.6" width="0" layer="19" extent="1-1"/>
-<wire x1="12.7" y1="0.9" x2="9.495" y2="4.3" width="0" layer="19" extent="1-1"/>
-<wire x1="18" y1="1" x2="14.195" y2="0.85" width="0" layer="19" extent="1-1"/>
-<wire x1="27.45" y1="4.175" x2="32.2" y2="6" width="0" layer="19" extent="1-1"/>
-<wire x1="24.8" y1="3.7" x2="26.1" y2="3.6556" width="0" layer="19" extent="1-1"/>
-<wire x1="7.3" y1="21.5" x2="12.9" y2="18" width="0" layer="19" extent="1-1"/>
-<wire x1="4.2" y1="32.5" x2="4.35" y2="28.4" width="0" layer="19" extent="1-1"/>
-<wire x1="6.1" y1="32.5" x2="4.2" y2="32.5" width="0" layer="19" extent="1-1"/>
-<wire x1="7.3" y1="37.15" x2="7.35" y2="33.75" width="0" layer="19" extent="1-1"/>
-<wire x1="25.945" y1="35.395" x2="35" y2="34" width="0" layer="19" extent="1-1"/>
-<wire x1="23.1" y1="37.4" x2="26" y2="37" width="0" layer="19" extent="1-1"/>
+<wire x1="0.9" y1="1.5" x2="3" y2="1.5" width="0.1524" layer="1"/>
+<wire x1="7.4" y1="3.95" x2="7.75" y2="4.3" width="0.4064" layer="1"/>
+<wire x1="7.75" y1="4.3" x2="9.495" y2="4.3" width="0.4064" layer="1"/>
+<wire x1="37.4" y1="22.15" x2="36.85" y2="22.7" width="0.2" layer="1"/>
+<wire x1="36.85" y1="22.7" x2="36.2" y2="22.7" width="0.2" layer="1"/>
+<via x="36.2" y="22.7" extent="1-16" drill="0.35"/>
 </signal>
 <signal name="DISP_RESET">
@@
 <contactref element="J5" pad="1"/>
 <contactref element="J6" pad="1"/>
+<contactref element="U2" pad="6"/>
+<contactref element="C4" pad="1"/>
+<wire x1="12.56624375" y1="8.402" x2="13.122" y2="8.402" width="0.2" layer="1"/>
+<wire x1="13.122" y1="8.402" x2="13.42" y2="8.7" width="0.2" layer="1"/>
+<wire x1="11.195" y1="4.3" x2="11.195" y2="6.2678375" width="0.2" layer="1"/>
+<wire x1="11.195" y1="6.2678375" x2="12.066" y2="7.1388375" width="0.2" layer="1"/>
+<wire x1="12.066" y1="7.1388375" x2="12.066" y2="7.90175625" width="0.2" layer="1"/>
+<wire x1="12.066" y1="7.90175625" x2="12.56624375" y2="8.402" width="0.2" layer="1"/>
+<contactref element="R17" pad="2"/>
 </signal>
 <signal name="N$3">
@@
 <wire x1="25.05070625" y1="10.7589" x2="35.98180625" y2="21.69" width="0.2" layer="16"/>
 <wire x1="35.98180625" y1="21.69" x2="40.57" y2="21.69" width="0.2" layer="16"/>
+<contactref element="R17" pad="1"/>
+<wire x1="37.4" y1="25.15" x2="37.4" y2="23.8694" width="0.2" layer="1"/>
+<via x="37.4" y="23.8694" extent="1-16" drill="0.35"/>
+<wire x1="37.4" y1="23.8694" x2="39.5794" y2="21.69" width="0.2" layer="16"/>
+<wire x1="39.5794" y1="21.69" x2="40.57" y2="21.69" width="0.2" layer="16"/>
 </signal>
 <signal name="RADIO_RESET">
@@
 <wire x1="12.393" y1="4.126975" x2="11.839025" y2="3.573" width="0.2" layer="1"/>
 </signal>
-<signal name="N$5">
-<contactref element="U2" pad="6"/>
-<contactref element="C4" pad="1"/>
-<wire x1="12.56624375" y1="8.402" x2="13.122" y2="8.402" width="0.2" layer="1"/>
-<wire x1="13.122" y1="8.402" x2="13.42" y2="8.7" width="0.2" layer="1"/>
-<wire x1="11.195" y1="4.3" x2="11.195" y2="6.2678375" width="0.2" layer="1"/>
-<wire x1="11.195" y1="6.2678375" x2="12.066" y2="7.1388375" width="0.2" layer="1"/>
-<wire x1="12.066" y1="7.1388375" x2="12.066" y2="7.90175625" width="0.2" layer="1"/>
-<wire x1="12.066" y1="7.90175625" x2="12.56624375" y2="8.402" width="0.2" layer="1"/>
-</signal>
 <signal name="DIFF1_N">
 <contactref element="U2" pad="3"/>
@@
 <via x="1.2801" y="10.3" extent="1-16" drill="0.35"/>
 <wire x1="1.2801" y1="10.3" x2="2.3325" y2="11.3524" width="0.2" layer="16"/>
-<wire x1="7.145975" y1="11.3524" x2="9.2491875" y2="9.2491875" width="0.2" layer="16"/>
-<wire x1="9.4491875" y1="9.2491875" x2="11.7" y2="11.5" width="0.2" layer="16"/>
-<wire x1="9.2491875" y1="9.2491875" x2="9.4491875" y2="9.2491875" width="0.2" layer="16"/>
+<wire x1="7.145975" y1="11.3524" x2="7.6491875" y2="10.8491875" width="0.2" layer="16"/>
+<wire x1="11.0491875" y1="10.8491875" x2="11.7" y2="11.5" width="0.2" layer="16"/>
+<wire x1="7.6491875" y1="10.8491875" x2="11.0491875" y2="10.8491875" width="0.2" layer="16"/>
 <wire x1="2.3325" y1="11.3524" x2="7.145975" y2="11.3524" width="0.2" layer="16"/>
 </signal>
@@
 <via x="3.2199" y="10.3" extent="1-16" drill="0.35"/>
 <wire x1="3.2199" y1="10.3" x2="3.9199" y2="11" width="0.2" layer="16"/>
-<wire x1="10.4179375" y1="8.8781375" x2="11.7" y2="10.1602" width="0.2" layer="16"/>
-<wire x1="9.1218625" y1="8.8781375" x2="10.4179375" y2="8.8781375" width="0.2" layer="16"/>
+<wire x1="11.7" y1="10.1602" x2="11.3" y2="10.1602" width="0.2" layer="16"/>
+<wire x1="11.3" y1="10.1602" x2="11.0820625" y2="10.3781375" width="0.2" layer="16"/>
+<wire x1="11.0820625" y1="10.3781375" x2="7.6218625" y2="10.3781375" width="0.2" layer="16"/>
 <wire x1="3.9199" y1="11" x2="7" y2="11" width="0.2" layer="16"/>
-<wire x1="7" y1="11" x2="9.1218625" y2="8.8781375" width="0.2" layer="16"/>
+<wire x1="7" y1="11" x2="7.6218625" y2="10.3781375" width="0.2" layer="16"/>
 </signal>
 <signal name="UVCC">
