File: Radio/Radii.brd (EAGLE design)
At the start: 42.6 x 44.9 mm, 55 parts, among them J1 10118193-0001LF, J2 BUTTON, J3 BUTTON, J4 BUTTON, J5 BUTTON, J6 BUTTON, U2 ATMEGA32U4-AU, U3 AP63203WU-7, U4 IND_1255AY-3R9N=P3, Y1 ECS-80-20-5PX-TR

Commit message: Fixed silkscreens and added designs
Parts:
- removed P1: (no value), adafruit:JST-PH-2-SMT-RA
- added J7: S2B-PH-SM4-TB(LF)(SN), I'mRADIOactive:JST_S2B-PH-SM4-TB(LF)(SN)
- added U$1: (no value), RoboJackets-Aesthetics:ROBOBUZZ_0.8X
- added U$2: (no value), RoboJackets-Aesthetics:ROBOJACKETS
Connections:
- net GND: now also J7.2, J7.S1, J7.S2; no longer P1.2
- net VCC: now also J7.1; no longer P1.1
Routing:
- net GND: track 90.7 -> 100.5 mm
Other:
- board text added: "3.3V"
- board text added: "9V"
- board text added: "Radio Board v1.0 RoboWrestling 2020"
Changed lines of the file:
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@@
 <drawing>
 <settings>
-<setting alwaysvectorfont="no"/>
+<setting alwaysvectorfont="yes"/>
 <setting verticaltext="up"/>
 </settings>
@@
 <circle x="3.1" y="41.7" radius="3" width="0.1524" layer="21"/>
 <circle x="39.5" y="41.8" radius="3" width="0.1524" layer="21"/>
+<text x="3.3" y="31.1" size="0.6096" layer="21">9V</text>
+<text x="9.7" y="31.1" size="0.6096" layer="21">3.3V</text>
+<text x="17" y="41" size="0.6096" layer="21">Radio Board v1.0
+RoboWrestling 2020</text>
 </plain>
 <attributes>
@@
 <attribute name="VALUE" x="20.99" y="36.698" size="0.6096" layer="27" font="vector" ratio="20" align="top-center"/>
 </element>
-<element name="P1" library="adafruit" library_urn="urn:adsk.eagle:library:420" package="JST-PH-2-SMT-RA" package3d_urn="urn:adsk.eagle:package:6240692/1" value="" x="3.418" y="23.658" smashed="yes" rot="R90">
-<attribute name="NAME" x="6.708" y="21.018" size="0.6096" layer="25" font="vector" rot="R90"/>
-<attribute name="VALUE" x="11.038" y="21.118" size="1.27" layer="27" font="vector" rot="R90"/>
-</element>
 <element name="JP2" library="pinhead" library_urn="urn:adsk.eagle:library:325" package="1X01" package3d_urn="urn:adsk.eagle:package:22485/2" value="" x="41" y="35" smashed="yes">
 <attribute name="NAME" x="39.6538" y="36.8288" size="0.6096" layer="25" font="vector"/>
@@
 <attribute name="VALUE" x="38.543" y="24.984" size="0.4064" layer="27" font="vector" rot="R90"/>
 </element>
+<element name="J7" library="I'mRADIOactive" package="JST_S2B-PH-SM4-TB(LF)(SN)" value="S2B-PH-SM4-TB(LF)(SN)" x="7.7" y="24.1" smashed="yes" rot="R270">
+<attribute name="DESCRIPTION" value=" Connector Header Surface Mount, Right Angle 2 position 0.079 (2.00mm) " x="7.7" y="24.1" size="1.778" layer="27" rot="R270" display="off"/>
+<attribute name="DIGI-KEY_PART_NUMBER" value="455-1749-1-ND" x="7.7" y="24.1" size="1.778" layer="27" rot="R270" display="off"/>
+<attribute name="MF" value="JST Sales" x="7.7" y="24.1" size="1.778" layer="27" rot="R270" display="off"/>
+<attribute name="MP" value="S2B-PH-SM4-TB(LF)(SN)" x="7.7" y="24.1" size="1.778" layer="27" rot="R270" display="off"/>
+<attribute name="NAME" x="10.247609375" y="27.97423125" size="1.27278125" layer="25" rot="R270"/>
+<attribute name="PACKAGE" value="None" x="7.7" y="24.1" size="1.778" layer="27" rot="R270" display="off"/>
+<attribute name="VALUE" x="-2.4187" y="27.85341875" size="1.274540625" layer="27" rot="R270"/>
+</element>
+<element name="U$2" library="RoboJackets-Aesthetics" package="ROBOJACKETS" value="" x="35" y="40" smashed="yes" rot="MR0"/>
+<element name="U$1" library="RoboJackets-Aesthetics" package="ROBOBUZZ_0.8X" value="" x="29" y="23" smashed="yes" rot="MR0"/>
 </elements>
 <signals>
@@
 <wire x1="15.9694" y1="14.3106" x2="15.9694" y2="12.7471" width="0.4064" layer="1"/>
 <contactref element="R3" pad="2"/>
-<contactref element="P1" pad="2"/>
 <contactref element="U3" pad="4"/>
 <contactref element="C5" pad="2"/>
@@
 <via x="25" y="15" extent="1-16" drill="0.4"/>
 <contactref element="Q1" pad="1"/>
-<wire x1="7.118" y1="22.658" x2="7.118" y2="21.682" width="0.508" layer="1"/>
-<wire x1="7.118" y1="21.682" x2="7.3" y2="21.5" width="0.508" layer="1"/>
-<via x="7.3" y="21.5" extent="1-16" drill="0.35"/>
-<wire x1="4.6601875" y1="23.777" x2="5.999" y2="23.777" width="0.508" layer="1"/>
-<wire x1="5.999" y1="23.777" x2="7.118" y2="22.658" width="0.508" layer="1"/>
-<wire x1="4.35" y1="28.4" x2="4.35" y2="24.0871875" width="0.508" layer="1"/>
+<wire x1="4.35" y1="28.4" x2="4.35" y2="27" width="0.508" layer="1"/>
+<wire x1="4.35" y1="27" x2="4.35" y2="24.0871875" width="0.508" layer="1"/>
 <wire x1="4.35" y1="24.0871875" x2="4.6601875" y2="23.777" width="0.508" layer="1"/>
 <contactref element="R5" pad="1"/>
@@
 <wire x1="36.85" y1="22.7" x2="36.2" y2="22.7" width="0.2" layer="1"/>
 <via x="36.2" y="22.7" extent="1-16" drill="0.35"/>
+<contactref element="J7" pad="2"/>
+<contactref element="J7" pad="S1"/>
+<contactref element="J7" pad="S2"/>
+<wire x1="7.023" y1="23.777" x2="7.7" y2="23.1" width="0.508" layer="1"/>
+<wire x1="4.6601875" y1="23.777" x2="7.023" y2="23.777" width="0.508" layer="1"/>
+<wire x1="7.7" y1="23.1" x2="7.7" y2="22.7" width="0.508" layer="1"/>
+<wire x1="7.7" y1="22.7" x2="7" y2="22" width="0.508" layer="1"/>
+<via x="7" y="22" extent="1-16" drill="0.35"/>
+<wire x1="1.95" y1="20.75" x2="4.3" y2="23.1" width="0.508" layer="1"/>
+<wire x1="4.3" y1="23.1" x2="7.7" y2="23.1" width="0.508" layer="1"/>
+<wire x1="1.95" y1="27.45" x2="3.9" y2="27.45" width="0.508" layer="1"/>
+<wire x1="3.9" y1="27.45" x2="4.35" y2="27" width="0.508" layer="1"/>
 </signal>
 <signal name="DISP_RESET">
@@
 </signal>
 <signal name="VCC">
-<contactref element="P1" pad="1"/>
 <contactref element="Q1" pad="3"/>
-<wire x1="7.118" y1="24.658" x2="5.3" y2="26.476" width="0.508" layer="1"/>
-<wire x1="5.3" y1="26.476" x2="5.3" y2="30.8" width="0.508" layer="1"/>
+<wire x1="5.3" y1="30.8" x2="5.3" y2="26.476" width="0.508" layer="1"/>
+<contactref element="J7" pad="1"/>
+<wire x1="5.3" y1="26.476" x2="6.676" y2="25.1" width="0.508" layer="1"/>
+<wire x1="6.676" y1="25.1" x2="7.7" y2="25.1" width="0.508" layer="1"/>
 </signal>
 <signal name="N$11">
@@
 </drawing>
 <compatibility>
+<note version="6.3" minversion="6.2.2" severity="warning">
+Since Version 6.2.2 text objects can contain more than one line,
+which will not be processed correctly with this version.
+</note>
 <note version="8.2" severity="warning">
 Since Version 8.2, EAGLE supports online libraries. The ids

Commit message: Updated board with styled parts
Parts:
- U2: device I'mRADIOactive:QFP80P1200X1200X120-44N -> I'mRADIOactive:44-TQFP(10X10)
- U3: device I'mRADIOactive:POWERREG -> I'mRADIOactive:TSOT-23-6
- U4: value IND_1255AY-3R9N=P3 -> 3.9uH; device I'mRADIOactive:IND_1255AY-3R9N=P3 -> I'mRADIOactive:1255AY-3R9N=P3
- Y1: value ECS-80-20-5PX-TR -> 8.000 MHz
- moved J7 3.00 mm to (4.70, 24.1)
- moved J2 1.30 mm to (39.7, 1.70)
- moved J4 1.30 mm to (39.7, 9.05)
- moved J3 1.30 mm to (31.6, 1.80)
- moved J5 1.30 mm to (31.6, 9.05)
- moved J6 1.30 mm to (34.8, 16.2)
Connections:
- removed net UVCC: U2.2
Routing:
- net N$11: track 7.63 -> 8.39 mm
- net GND: track 100.5 -> 101.2 mm

Commit message: fixed mcu on radio schematic
Parts:
- R3: value 400Ω -> (none); device SparkFun-Resistors:0603-RES -> SparkFun-Resistors:0603
- R4: value 100Ω -> (none); device SparkFun-Resistors:0603-RES -> SparkFun-Resistors:0603
