File: Radio/Radii.sch (EAGLE design)
At the start: 42 parts, among them J1 10118193-0001LF, J2 BUTTON, J3 BUTTON, J4 BUTTON, J5 BUTTON, J6 BUTTON, U2 ATMEGA32U4-AU, U3 AP63203WU-7, U4 IND_1255AY-3R9N=P3, Y1 ECS-80-20-5PX-TR

Commit message: Added pFET
Parts:
- added Q1: (no value), RoboJackets-Discrete:PMOS
- added R11: 10K, SparkFun-Resistors:10KOHM-1/10W-1%(0603)0603
Connections:
- new net VCC: P1.2, Q1.D
- net 3.3V: now also R11.2
- net 9V: now also Q1.S; no longer P1.2
- net GND: now also Q1.G
- net SS3: now also R11.1
Changed lines of the file:
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@@
 <part name="R10" library="SparkFun-Resistors" deviceset="10KOHM-1/10W-1%(0603)" device="0603" value="10K"/>
 <part name="GND10" library="supply1" library_urn="urn:adsk.eagle:library:371" deviceset="GND" device=""/>
+<part name="Q1" library="RoboJackets-Discrete" deviceset="PMOS" device=""/>
+<part name="SUPPLY11" library="SparkFun-PowerSymbols" library_urn="urn:adsk.eagle:library:530" deviceset="3.3V" device=""/>
+<part name="R11" library="SparkFun-Resistors" deviceset="10KOHM-1/10W-1%(0603)" device="0603" value="10K"/>
 </parts>
 <sheets>
@@
 <attribute name="VALUE" x="255.27" y="91.44" size="1.778" layer="96" rot="R90"/>
 </instance>
-<instance part="SUPPLY5" gate="G$1" x="182.88" y="111.76" smashed="yes">
-<attribute name="VALUE" x="182.88" y="114.554" size="1.778" layer="96" align="bottom-center"/>
+<instance part="SUPPLY5" gate="G$1" x="198.12" y="111.76" smashed="yes">
+<attribute name="VALUE" x="198.12" y="114.554" size="1.778" layer="96" align="bottom-center"/>
 </instance>
 <instance part="SUPPLY6" gate="G$1" x="198.12" y="91.44" smashed="yes">
@@
 <instance part="GND10" gate="1" x="139.446" y="19.812" smashed="yes">
 <attribute name="VALUE" x="136.906" y="17.272" size="1.778" layer="96"/>
+</instance>
+<instance part="Q1" gate="G$1" x="187.96" y="106.68" smashed="yes" rot="MR180">
+<attribute name="VALUE" x="190.5" y="106.68" size="1.778" layer="96" rot="MR180"/>
+<attribute name="NAME" x="190.5" y="104.14" size="1.778" layer="95" rot="MR180"/>
+</instance>
+<instance part="SUPPLY11" gate="G$1" x="21.082" y="58.42" smashed="yes">
+<attribute name="VALUE" x="21.082" y="61.214" size="1.778" layer="96" align="bottom-center"/>
+</instance>
+<instance part="R11" gate="G$1" x="21.082" y="51.054" smashed="yes" rot="R90">
+<attribute name="NAME" x="19.5834" y="47.244" size="1.778" layer="95" rot="R90"/>
+<attribute name="VALUE" x="24.384" y="47.244" size="1.778" layer="96" rot="R90"/>
 </instance>
 </instances>
@@
 <wire x1="175.26" y1="104.14" x2="182.88" y2="104.14" width="0.1524" layer="91"/>
 <wire x1="182.88" y1="104.14" x2="182.88" y2="101.6" width="0.1524" layer="91"/>
+<pinref part="Q1" gate="G$1" pin="G"/>
+<junction x="182.88" y="104.14"/>
 </segment>
 <segment>
@@
 <wire x1="137.077834375" y1="195.58" x2="137.077834375" y2="195.59219375" width="0.1524" layer="91"/>
 </segment>
+<segment>
+<pinref part="SUPPLY11" gate="G$1" pin="3.3V"/>
+<pinref part="R11" gate="G$1" pin="2"/>
+<wire x1="21.082" y1="58.42" x2="21.082" y2="56.134" width="0.1524" layer="91"/>
+</segment>
 </net>
 <net name="N$3" class="0">
@@
 <segment>
 <pinref part="U1" gate="RFM59HCW" pin="NSS"/>
-<wire x1="50.8" y1="33.02" x2="38.1" y2="33.02" width="0.1524" layer="91"/>
-<label x="38.1" y="33.02" size="1.778" layer="95" rot="R180" xref="yes"/>
+<wire x1="50.8" y1="33.02" x2="21.082" y2="33.02" width="0.1524" layer="91"/>
+<label x="20.32" y="33.02" size="1.778" layer="95" rot="R180" xref="yes"/>
+<pinref part="R11" gate="G$1" pin="1"/>
+<wire x1="21.082" y1="45.974" x2="21.082" y2="33.02" width="0.1524" layer="91"/>
+<wire x1="21.082" y1="33.02" x2="20.32" y2="33.02" width="0.1524" layer="91"/>
 </segment>
 <segment>
@@
 <net name="9V" class="0">
 <segment>
-<pinref part="P1" gate="G$1" pin="2"/>
-<wire x1="182.88" y1="111.76" x2="182.88" y2="106.68" width="0.1524" layer="91"/>
-<wire x1="182.88" y1="106.68" x2="175.26" y2="106.68" width="0.1524" layer="91"/>
-<pinref part="SUPPLY5" gate="G$1" pin="VCC_2"/>
-</segment>
-<segment>
-<pinref part="U3" gate="G$1" pin="VIN"/>
-<wire x1="210.82" y1="84.328" x2="198.12" y2="84.328" width="0.1524" layer="91"/>
+<wire x1="198.12" y1="81.28" x2="198.12" y2="84.328" width="0.1524" layer="91"/>
+<pinref part="C5" gate="G$1" pin="1"/>
+<pinref part="SUPPLY6" gate="G$1" pin="VCC_2"/>
 <pinref part="U3" gate="G$1" pin="EN"/>
 <wire x1="198.12" y1="84.328" x2="198.12" y2="90.17" width="0.1524" layer="91"/>
 <wire x1="198.12" y1="90.17" x2="198.12" y2="91.44" width="0.1524" layer="91"/>
 <wire x1="210.82" y1="90.17" x2="198.12" y2="90.17" width="0.1524" layer="91"/>
-<pinref part="C5" gate="G$1" pin="1"/>
-<wire x1="198.12" y1="81.28" x2="198.12" y2="84.328" width="0.1524" layer="91"/>
-<pinref part="SUPPLY6" gate="G$1" pin="VCC_2"/>
+<junction x="198.12" y="90.17"/>
+<pinref part="U3" gate="G$1" pin="VIN"/>
+<wire x1="210.82" y1="84.328" x2="198.12" y2="84.328" width="0.1524" layer="91"/>
+<junction x="198.12" y="84.328"/>
 </segment>
 <segment>
@@
 <pinref part="D1" gate="G$1" pin="A"/>
 <wire x1="167.64" y1="86.36" x2="170.18" y2="86.36" width="0.1524" layer="91"/>
+</segment>
+<segment>
+<pinref part="Q1" gate="G$1" pin="S"/>
+<wire x1="187.96" y1="101.6" x2="198.12" y2="101.6" width="0.1524" layer="91"/>
+<pinref part="SUPPLY5" gate="G$1" pin="VCC_2"/>
+<wire x1="198.12" y1="101.6" x2="198.12" y2="111.76" width="0.1524" layer="91"/>
 </segment>
 </net>
@@
 </segment>
 </net>
+<net name="VCC" class="0">
+<segment>
+<pinref part="P1" gate="G$1" pin="2"/>
+<wire x1="182.88" y1="106.68" x2="175.26" y2="106.68" width="0.1524" layer="91"/>
+<pinref part="Q1" gate="G$1" pin="D"/>
+<wire x1="182.88" y1="106.68" x2="182.88" y2="111.76" width="0.1524" layer="91"/>
+<wire x1="182.88" y1="111.76" x2="187.96" y2="111.76" width="0.1524" layer="91"/>
+</segment>
+</net>

Commit message: Added debouncing filters for buttons
Parts:
- added C16, C17, C18, C19, C20: 0.1uF, SparkFun-Capacitors:0.1UF-0603-25V-(+80/-20%)
- added R12, R14, R16: 1K, SparkFun-Resistors:10KOHM-1/10W-1%(0603)0603
- added R13, R15: 10K, SparkFun-Resistors:10KOHM-1/10W-1%(0603)0603
- R7, R9: value 10K -> 1K
Connections:
- net CS3 renamed CS
- net MOSI3 renamed MOSI
- net SCK3 renamed SCK
- net SS3 renamed SS
- new net N$11: J2.P$2, R12.2, R5.2
- new net N$12: J4.P$2, R8.2, R9.2
- new net N$13: J5.P$2, R13.2, R14.2
- new net N$14: J6.P$2, R15.2, R16.2
- new net N$4: J3.P$2, R6.2, R7.2
- net BUTTON1: now also C17.1, R7.1; no longer J2.P$2, R5.1
- net BUTTON2: now also C16.1, R12.1; no longer J3.P$2, R6.1
- net BUTTON3: now also C19.1, R14.1; no longer J4.P$2, R7.1
- net BUTTON4: now also C18.1, R9.1; no longer J5.P$2, R8.1
- net BUTTON5: now also C20.1, R16.1; no longer J6.P$2, R9.1
- net GND: now also C16.2, C17.2, C18.2, C19.2, C20.2, R13.1, R15.1, R5.1, R6.1, R8.1; no longer R5.2, R6.2, R7.2, R8.2, R9.2
Other:
- moved on the sheet: R5, R6, R7, R8, R9

Commit message: Added pullup to display
Parts:
- added R17: 10K, SparkFun-Resistors:10KOHM-1/10W-1%(0603)0603
Connections:
- removed net N$5: C4.1, U2.UCAP
- net 3.3V: now also C4.1, R17.2, U2.UCAP
- net CS: now also R17.1
Other:
- moved on the sheet: C16, C17, C18, C19, C20, C5, C6, C7, C8, D1, D2, J2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

Commit message: Fixed silkscreens and added designs
Parts:
- removed P1: (no value), adafruit:JST_2PIN-SMT-RA
- added J7: S2B-PH-SM4-TB(LF)(SN), I'mRADIOactive:S2B-PH-SM4-TB(LF)(SN)
Connections:
- net GND: now also J7.2, J7.SHIELD; no longer P1.1
- net VCC: now also J7.1; no longer P1.2
Changed lines of the file:
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@@
 <part name="C2" library="SparkFun-Capacitors" library_urn="urn:adsk.eagle:library:510" deviceset="0.1UF" device="-0603-25V-(+80/-20%)" package3d_urn="urn:adsk.eagle:package:37414/1" value="0.1uF"/>
 <part name="C3" library="SparkFun-Capacitors" library_urn="urn:adsk.eagle:library:510" deviceset="0.1UF" device="-0603-25V-(+80/-20%)" package3d_urn="urn:adsk.eagle:package:37414/1" value="0.1uF"/>
-<part name="P1" library="adafruit" library_urn="urn:adsk.eagle:library:420" deviceset="JST_2PIN" device="-SMT-RA" package3d_urn="urn:adsk.eagle:package:6240692/1"/>
 <part name="GND5" library="supply1" library_urn="urn:adsk.eagle:library:371" deviceset="GND" device=""/>
 <part name="JP2" library="pinhead" library_urn="urn:adsk.eagle:library:325" deviceset="PINHD-1X1" device="" package3d_urn="urn:adsk.eagle:package:22485/2"/>
@@
 <part name="SUPPLY16" library="SparkFun-PowerSymbols" library_urn="urn:adsk.eagle:library:530" deviceset="3.3V" device=""/>
 <part name="R17" library="SparkFun-Resistors" deviceset="10KOHM-1/10W-1%(0603)" device="0603" value="10K"/>
+<part name="J7" library="I'mRADIOactive" deviceset="S2B-PH-SM4-TB(LF)(SN)" device=""/>
 </parts>
 <sheets>
@@
 <attribute name="VALUE" x="103.124" y="23.241" size="1.778" layer="96" font="vector"/>
 </instance>
-<instance part="P1" gate="G$1" x="203.2" y="81.28" smashed="yes" rot="R180">
-<attribute name="NAME" x="209.55" y="75.565" size="1.778" layer="95" rot="R180"/>
-<attribute name="VALUE" x="209.55" y="86.36" size="1.778" layer="96" rot="R180"/>
-</instance>
 <instance part="GND5" gate="1" x="213.36" y="73.66" smashed="yes">
 <attribute name="VALUE" x="210.82" y="71.12" size="1.778" layer="96"/>
@@
 <attribute name="NAME" x="217.7034" y="176.784" size="1.778" layer="95" rot="R90"/>
 <attribute name="VALUE" x="222.504" y="176.784" size="1.778" layer="96" rot="R90"/>
+</instance>
+<instance part="J7" gate="G$1" x="198.12" y="78.74" smashed="yes" rot="MR0">
+<attribute name="NAME" x="203.2029" y="84.33571875" size="1.272509375" layer="95" rot="MR0"/>
+<attribute name="VALUE" x="203.20811875" y="69.31731875" size="1.275409375" layer="96" rot="MR0"/>
 </instance>
 </instances>
@@
 </segment>
 <segment>
-<pinref part="P1" gate="G$1" pin="1"/>
 <pinref part="GND5" gate="1" pin="GND"/>
-<wire x1="205.74" y1="78.74" x2="213.36" y2="78.74" width="0.1524" layer="91"/>
 <wire x1="213.36" y1="78.74" x2="213.36" y2="76.2" width="0.1524" layer="91"/>
 <pinref part="Q1" gate="G$1" pin="G"/>
+<pinref part="J7" gate="G$1" pin="2"/>
+<wire x1="213.36" y1="78.74" x2="205.74" y2="78.74" width="0.1524" layer="91"/>
 <junction x="213.36" y="78.74"/>
+<pinref part="J7" gate="G$1" pin="SHIELD"/>
+<wire x1="205.74" y1="73.66" x2="208.28" y2="73.66" width="0.1524" layer="91"/>
+<wire x1="208.28" y1="73.66" x2="208.28" y2="76.2" width="0.1524" layer="91"/>
+<wire x1="208.28" y1="76.2" x2="213.36" y2="76.2" width="0.1524" layer="91"/>
+<junction x="213.36" y="76.2"/>
 </segment>
 <segment>
@@
 <net name="VCC" class="0">
 <segment>
-<pinref part="P1" gate="G$1" pin="2"/>
-<wire x1="213.36" y1="81.28" x2="205.74" y2="81.28" width="0.1524" layer="91"/>
 <pinref part="Q1" gate="G$1" pin="D"/>
 <wire x1="213.36" y1="81.28" x2="213.36" y2="86.36" width="0.1524" layer="91"/>
 <wire x1="213.36" y1="86.36" x2="218.44" y2="86.36" width="0.1524" layer="91"/>
-</segment>
-</net>
+<pinref part="J7" gate="G$1" pin="1"/>
+<wire x1="205.74" y1="81.28" x2="213.36" y2="81.28" width="0.1524" layer="91"/>
+</segment>
+</net>

Commit message: Updated board with styled parts
Parts:
- U4: value IND_1255AY-3R9N=P3 -> 3.9uH; device I'mRADIOactive:IND_1255AY-3R9N=P3 -> I'mRADIOactive:1255AY-3R9N=P3
- Y1: value ECS-80-20-5PX-TR -> 8.000 MHz
Other:
- moved on the sheet: J1, J7, JP1, U1, U2
Changed lines of the file:
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@@
 <part name="C7" library="SparkFun-Capacitors" library_urn="urn:adsk.eagle:library:510" deviceset="22UF" device="-1210-16V-20%" package3d_urn="urn:adsk.eagle:package:37436/1" value="22uF"/>
 <part name="C8" library="SparkFun-Capacitors" library_urn="urn:adsk.eagle:library:510" deviceset="22UF" device="-1210-16V-20%" package3d_urn="urn:adsk.eagle:package:37436/1" value="22uF"/>
-<part name="U4" library="I'mRADIOactive" deviceset="IND_1255AY-3R9N=P3" device=""/>
+<part name="U4" library="I'mRADIOactive" deviceset="1255AY-3R9N=P3" device="" value="3.9uH"/>
 <part name="SUPPLY5" library="SparkFun-PowerSymbols" library_urn="urn:adsk.eagle:library:530" deviceset="VCC_2" device="" value="9V"/>
 <part name="SUPPLY6" library="SparkFun-PowerSymbols" library_urn="urn:adsk.eagle:library:530" deviceset="VCC_2" device="" value="9V"/>
@@
 <part name="C13" library="SparkFun-Capacitors" library_urn="urn:adsk.eagle:library:510" deviceset="33PF" device="-0603-50V-5%" package3d_urn="urn:adsk.eagle:package:37414/1" value="33pF"/>
 <part name="C14" library="SparkFun-Capacitors" library_urn="urn:adsk.eagle:library:510" deviceset="33PF" device="-0603-50V-5%" package3d_urn="urn:adsk.eagle:package:37414/1" value="33pF"/>
-<part name="Y1" library="I'mRADIOactive" deviceset="ECS-80-20-5PX-TR" device=""/>
+<part name="Y1" library="I'mRADIOactive" deviceset="ECS-80-20-5PX-TR" device="" value="8.000 MHz"/>
 <part name="D1" library="RoboJackets-LEDs" deviceset="LED-SMD" device="" value="GREEN"/>
 <part name="D2" library="RoboJackets-LEDs" deviceset="LED-SMD" device="" value="GREEN"/>
@@
 <segment>
 <pinref part="U1" gate="RFM59HCW" pin="MISO"/>
-<wire x1="50.8" y1="40.64" x2="48.26" y2="40.64" width="0.1524" layer="91"/>
 <label x="48.26" y="40.64" size="1.778" layer="95" rot="R180" xref="yes"/>
 </segment>
@@
 <pinref part="U1" gate="RFM59HCW" pin="GND@3"/>
 <pinref part="GND2" gate="1" pin="GND"/>
-<wire x1="50.8" y1="25.4" x2="33.02" y2="25.4" width="0.1524" layer="91"/>
+<wire x1="78.74" y1="25.4" x2="33.02" y2="25.4" width="0.1524" layer="91"/>
 <wire x1="33.02" y1="25.4" x2="33.02" y2="15.24" width="0.1524" layer="91"/>
 <pinref part="U1" gate="RFM59HCW" pin="GND@2"/>
-<wire x1="50.8" y1="43.18" x2="15.24" y2="43.18" width="0.1524" layer="91"/>
+<wire x1="78.74" y1="27.94" x2="15.24" y2="43.18" width="0.1524" layer="91"/>
 <wire x1="15.24" y1="43.18" x2="15.24" y2="15.24" width="0.1524" layer="91"/>
 <wire x1="15.24" y1="15.24" x2="33.02" y2="15.24" width="0.1524" layer="91"/>
 <junction x="33.02" y="15.24"/>
 <pinref part="U1" gate="RFM59HCW" pin="GND@1"/>
-<wire x1="76.2" y1="27.94" x2="91.44" y2="27.94" width="0.1524" layer="91"/>
+<wire x1="78.74" y1="30.48" x2="91.44" y2="27.94" width="0.1524" layer="91"/>
 <wire x1="91.44" y1="27.94" x2="91.44" y2="15.24" width="0.1524" layer="91"/>
 <wire x1="91.44" y1="15.24" x2="33.02" y2="15.24" width="0.1524" layer="91"/>
@@
 <pinref part="Q1" gate="G$1" pin="G"/>
 <pinref part="J7" gate="G$1" pin="2"/>
-<wire x1="213.36" y1="78.74" x2="205.74" y2="78.74" width="0.1524" layer="91"/>
+<wire x1="213.36" y1="78.74" x2="208.28" y2="78.74" width="0.1524" layer="91"/>
 <junction x="213.36" y="78.74"/>
 <pinref part="J7" gate="G$1" pin="SHIELD"/>
-<wire x1="205.74" y1="73.66" x2="208.28" y2="73.66" width="0.1524" layer="91"/>
 <wire x1="208.28" y1="73.66" x2="208.28" y2="76.2" width="0.1524" layer="91"/>
 <wire x1="208.28" y1="76.2" x2="213.36" y2="76.2" width="0.1524" layer="91"/>
@@
 <pinref part="J1" gate="G$1" pin="SHIELD"/>
 <pinref part="J1" gate="G$1" pin="GND"/>
-<wire x1="139.446" y1="32.512" x2="139.446" y2="27.432" width="0.1524" layer="91"/>
+<wire x1="119.126" y1="27.432" x2="139.446" y2="32.512" width="0.1524" layer="91"/>
 <pinref part="GND10" gate="1" pin="GND"/>
-<wire x1="139.446" y1="27.432" x2="139.446" y2="22.352" width="0.1524" layer="91"/>
-<junction x="139.446" y="27.432"/>
+<wire x1="139.446" y1="32.512" x2="139.446" y2="22.352" width="0.1524" layer="91"/>
+<junction x="139.446" y="32.512"/>
 </segment>
 <segment>
@@
 <segment>
 <pinref part="U1" gate="RFM59HCW" pin="DIO0"/>
-<wire x1="76.2" y1="38.1" x2="88.9" y2="38.1" width="0.1524" layer="91"/>
+<wire x1="78.74" y1="35.56" x2="88.9" y2="38.1" width="0.1524" layer="91"/>
 <label x="88.9" y="38.1" size="1.778" layer="95" xref="yes"/>
 </segment>
@@
 <segment>
 <pinref part="U1" gate="RFM59HCW" pin="VDD"/>
-<wire x1="76.2" y1="35.56" x2="101.6" y2="35.56" width="0.1524" layer="91"/>
+<wire x1="48.26" y1="43.18" x2="101.6" y2="35.56" width="0.1524" layer="91"/>
 <pinref part="SUPPLY3" gate="G$1" pin="3.3V"/>
 <wire x1="101.6" y1="35.56" x2="101.6" y2="38.1" width="0.1524" layer="91"/>
@@
 <wire x1="43.18" y1="200.66" x2="66.04" y2="200.66" width="0.1524" layer="91"/>
 <junction x="43.18" y="200.66"/>
-<wire x1="66.04" y1="200.66" x2="66.04" y2="193.04" width="0.1524" layer="91"/>
+<wire x1="66.04" y1="200.66" x2="132.08" y2="193.04" width="0.1524" layer="91"/>
 <wire x1="43.18" y1="198.12" x2="50.8" y2="198.12" width="0.1524" layer="91"/>
 <junction x="43.18" y="198.12"/>
 <wire x1="50.8" y1="198.12" x2="60.96" y2="198.12" width="0.1524" layer="91"/>
 <wire x1="60.96" y1="198.12" x2="60.96" y2="190.5" width="0.1524" layer="91"/>
-<wire x1="60.96" y1="190.5" x2="66.04" y2="190.5" width="0.1524" layer="91"/>
+<wire x1="60.96" y1="190.5" x2="132.08" y2="190.5" width="0.1524" layer="91"/>
 <pinref part="U2" gate="G$1" pin="VCC"/>
 <pinref part="U2" gate="G$1" pin="AVCC"/>
@@
 <pinref part="U2" gate="G$1" pin="UCAP"/>
 <pinref part="C4" gate="G$1" pin="1"/>
-<wire x1="66.04" y1="185.42" x2="50.8" y2="185.42" width="0.1524" layer="91"/>
+<wire x1="132.08" y1="185.42" x2="50.8" y2="185.42" width="0.1524" layer="91"/>
 <wire x1="50.8" y1="185.42" x2="50.8" y2="198.12" width="0.1524" layer="91"/>
 <junction x="50.8" y="185.42"/>
@@
 <segment>
 <pinref part="U1" gate="RFM59HCW" pin="ANT"/>
-<wire x1="76.2" y1="25.4" x2="78.74" y2="25.4" width="0.1524" layer="91"/>
-<wire x1="78.74" y1="25.4" x2="78.74" y2="22.86" width="0.1524" layer="91"/>
+<wire x1="78.74" y1="33.02" x2="78.74" y2="22.86" width="0.1524" layer="91"/>
 <pinref part="JP2" gate="G$1" pin="1"/>
 <wire x1="78.74" y1="22.86" x2="83.82" y2="22.86" width="0.1524" layer="91"/>
@@
 <segment>
 <pinref part="U1" gate="RFM59HCW" pin="MOSI"/>
-<wire x1="50.8" y1="38.1" x2="33.02" y2="38.1" width="0.1524" layer="91"/>
+<wire x1="48.26" y1="38.1" x2="33.02" y2="38.1" width="0.1524" layer="91"/>
 <label x="33.02" y="38.1" size="1.778" layer="95" rot="R180" xref="yes"/>
 </segment>
@@
 <segment>
 <pinref part="U1" gate="RFM59HCW" pin="SCK"/>
-<wire x1="50.8" y1="35.56" x2="48.26" y2="35.56" width="0.1524" layer="91"/>
 <label x="48.26" y="35.56" size="1.778" layer="95" rot="R180" xref="yes"/>
 </segment>
@@
 <segment>
 <pinref part="U1" gate="RFM59HCW" pin="NSS"/>
-<wire x1="50.8" y1="33.02" x2="21.082" y2="33.02" width="0.1524" layer="91"/>
+<wire x1="48.26" y1="33.02" x2="21.082" y2="33.02" width="0.1524" layer="91"/>
 <label x="20.32" y="33.02" size="1.778" layer="95" rot="R180" xref="yes"/>
 <pinref part="R11" gate="G$1" pin="1"/>
@@
 <segment>
 <pinref part="U1" gate="RFM59HCW" pin="RESET"/>
-<wire x1="50.8" y1="30.48" x2="48.26" y2="30.48" width="0.1524" layer="91"/>
 <label x="48.26" y="30.48" size="1.778" layer="95" rot="R180" xref="yes"/>
 </segment>
@@
 <pinref part="U2" gate="G$1" pin="VBUS"/>
 <label x="64.77" y="182.88" size="1.778" layer="95" rot="R180" xref="yes"/>
-<wire x1="66.04" y1="182.88" x2="64.77" y2="182.88" width="0.1524" layer="91"/>
+<wire x1="132.08" y1="182.88" x2="64.77" y2="182.88" width="0.1524" layer="91"/>
 <wire x1="64.77" y1="182.88" x2="64.77" y2="182.626" width="0.1524" layer="91"/>
 </segment>
@@
 <wire x1="213.36" y1="86.36" x2="218.44" y2="86.36" width="0.1524" layer="91"/>
 <pinref part="J7" gate="G$1" pin="1"/>
-<wire x1="205.74" y1="81.28" x2="213.36" y2="81.28" width="0.1524" layer="91"/>
-</segment>
-</net>
+<wire x1="208.28" y1="81.28" x2="213.36" y2="81.28" width="0.1524" layer="91"/>
+</segment>
+</net>

Commit message: fixed mcu on radio schematic
Parts:
- R3: value 400Ω -> (none)
- R4: value 100Ω -> (none)
Other:
- moved on the sheet: U2
