File: Gucci/v3 pcb/Gucci_ControlBoard.brd (EAGLE design)
At the start: 66 x 56 mm, 89 parts, among them U1 TEENSY_3.6_DIL, U2 ICM-20948, U3 PCA9306_LSSOP, U5 LM393-8-SOIC, U6 AP2114H-1.8TRG1, U7 AP2114H-3.3TRG1

Commit message: mounting holes clearance
Parts:
- moved R22 1.00 mm to (30.4, 27.2)
- moved R18 1.00 mm to (34.3, 27.2)
Routing:
- net +3.3V: track 246.5 -> 244.2 mm

Commit message: Started Implementing 4 Layers
Started Implementing 4 Layers: Adding vias
Routing:
- net GND: track 85.8 -> 88.6 mm, vias 43 -> 45
- added copper zone on layer 15, net +5V
- added copper zone on layer 15, net 1.8V
- added copper zone on layer 2, net GND
- removed copper zone on layer 1, net +5V
- removed copper zone on layer 1, net 1.8V
- removed copper zone on layer 16, net GND

Commit message: Finished 4-layer routing on Gucci
Finished 4-layer routing on Gucci (changed layer names)
Parts:
- moved C7 0.60 mm to (25.9, 34.1)
- moved C11 0.20 mm to (27.8, 41.3)
Routing:
- net +5V: track 31.8 -> 75.0 mm, vias 1 -> 22
- net GND: track 88.6 -> 121.4 mm, vias 45 -> 58
- added copper zone on layer 1, net 1.8V
- removed copper zone on layer 15, net 1.8V

Commit message: Moved Power Connector out/Capacitors
Moved Power Connector out/Moved Capacitors
Parts:
- moved C8 34.0 mm to (-8.10, 39.7)
- moved C7 32.5 mm to (-6.10, 39.7), turned to 270 degrees
- moved C11 5.73 mm to (28.4, 35.6), turned to 270 degrees
- moved D1 3.00 mm to (29.6, 41.9)
- moved POWER_CONN 2.30 mm to (-11.6, 38.0)
- moved C24 2.10 mm to (25.9, 35.6)
- moved F1 0.91 mm to (-1.60, 43.1)
Routing:
- net +5V: track 75.0 -> 48.7 mm, vias 22 -> 23
- net GND: track 121.4 -> 116.6 mm
- net MOSI: track 55.4 -> 51.2 mm, vias 3 -> 2
- net MISO: track 53.1 -> 49.0 mm, vias 3 -> 2
- net LINE_RF: track 81.7 -> 79.4 mm, vias 3 -> 1
- net +3.3V: track 243.9 -> 241.8 mm
- net N$7: track 6.45 -> 4.93 mm
- net N$6: track 10.9 -> 9.99 mm

Commit message: Multiplexed Distance Sensors
Multiplexed Distance Sensors (3-4)/Directly connectted ESCs
Parts:
- removed ESC_RX, ESC_TX: MUX_74LVC1G157GV, Kirbi_ControlBoard:MUX_74LVC1G157GV
- added MUX_RX3, MUX_TX3: MUX_74LVC1G157GV, Kirbi_ControlBoard:MUX_74LVC1G157GV
- moved R10 59.6 mm to (3.90, 1.50), turned to 0 degrees
- moved R27 57.6 mm to (21.8, 1.50), flipped to the bottom, turned to 180 degrees
- moved R11 53.0 mm to (30.9, 1.60), turned to 0 degrees
- moved R26 49.4 mm to (14.7, 5.60), flipped to the top, turned to 0 degrees
- moved R9 46.7 mm to (24.0, 6.30), turned to 90 degrees
- moved JP1 6.00 mm to (13.0, 2.00)
- moved C4 1.26 mm to (7.90, 7.10), turned to 0 degrees
- moved C15 1.20 mm to (-1.00, 10.2)
- moved C22 0.80 mm to (23.6, 11.9)
- moved R23 0.67 mm to (27.4, 5.30)
- moved C12 0.20 mm to (10.0, 5.30)
- moved C25 0.20 mm to (37.0, 5.30)
- moved C10 0.20 mm to (-8.40, 17.0)
- moved R3 0.10 mm to (0.00, 12.2)
Connections:
- removed net ESC_S: ESC_RX.P$6, ESC_TX.P$6, R26.2, R27.2, U1.36/A17
- removed net ESC_TRX: ESC_RX.P$4, R9.1, U1.34/A15
- removed net ESC_TTX: ESC_TX.P$4, U1.33/A14
- removed net S1/RX: ESC1.P$2, ESC_RX.P$3
- removed net S1/TX: ESC1.P$1, ESC_TX.P$3, R10.1
- removed net S2/RX: ESC2.P$2, ESC_RX.P$1
- removed net S2/TX: ESC2.P$1, ESC_TX.P$1, R11.1
- new net ESC_RX4: ESC1.P$2, U1.32/A13
- new net ESC_RX5: ESC2.P$2, U1.34/A15
- new net ESC_TX4: ESC1.P$1, U1.31/A12
- new net ESC_TX5: ESC2.P$1, U1.33/A14
- new net MUXS3: MUX_RX3.P$6, MUX_TX3.P$6, R26.2, R27.2, U1.28
- new net TRX3: MUX_RX3.P$4, R9.1, U1.0
- new net TTX3: MUX_TX3.P$4, U1.1
- net +3.3V: now also MUX_RX3.P$5, MUX_TX3.P$5; no longer ESC_RX.P$5, ESC_TX.P$5
- net GND: now also MUX_RX3.P$2, MUX_TX3.P$2; no longer ESC_RX.P$2, ESC_TX.P$2
- net RXD3: now also MUX_RX3.P$3; no longer U1.0
- net RXD4: now also MUX_RX3.P$1; no longer U1.31/A12
- net TXD3: now also MUX_TX3.P$3, R10.1; no longer U1.1
- net TXD4: now also MUX_TX3.P$1, R11.1; no longer U1.32/A13
Routing:
- net MUXS3: track 0.00 -> 67.2 mm, vias 0 -> 3
- net TRX3: track 0.00 -> 60.4 mm, vias 0 -> 1
- net TTX3: track 0.00 -> 54.8 mm, vias 0 -> 1
- net TXD4: track 47.4 -> 21.4 mm, vias 1 -> 2
- net RXD3: track 47.1 -> 24.0 mm, vias 1 -> 2
- net ESC_S: track 23.0 -> 0.00 mm, vias 2 -> 0
- net TXD3: track 43.8 -> 21.1 mm, vias 1 -> 2
- net RXD4: track 34.7 -> 16.4 mm, vias 1 -> 0
- net S1/TX: track 13.9 -> 0.00 mm
- net S1/RX: track 13.1 -> 0.00 mm
- net ESC_TTX: track 11.5 -> 0.00 mm, vias 1 -> 0
- net ESC_TX5: track 0.00 -> 11.4 mm
- net ESC_TX4: track 0.00 -> 10.9 mm
- net S2/TX: track 10.2 -> 0.00 mm, vias 2 -> 0
- net ESC_RX4: track 0.00 -> 9.32 mm
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
Commit message: Moved/Re-routed Some Parts
Moved/Re-routed Some Parts (Moved components away from the Teensy pins)
Parts:
- moved C6 1.75 mm to (-7.30, 42.2)
- moved C20 1.75 mm to (9.70, 42.6), turned to 180 degrees
- moved F1 1.61 mm to (-0.80, 41.7), turned to 0 degrees
- moved C7 1.60 mm to (-6.10, 38.1)
- moved C8 1.60 mm to (-8.10, 38.1)
- moved R7 1.53 mm to (10.1, 33.7)
- moved C19 0.57 mm to (13.6, 42.6), turned to 180 degrees
- moved R8 0.32 mm to (15.1, 33.7)
Routing:
- net N$6: track 9.99 -> 12.5 mm
- net N$7: track 4.93 -> 6.78 mm
- net TRX1: track 24.5 -> 26.2 mm
- net RF_INT: track 19.4 -> 20.8 mm
- net +3.3V: track 245.2 -> 246.6 mm
- net LINE_RF: track 75.5 -> 76.5 mm
- net GND: track 117.5 -> 116.7 mm
- net RADIO_DIO0: track 36.5 -> 35.9 mm

Commit message: slight tweak to gucci routing
Routing:
- net SCK: track 96.8 -> 94.4 mm, vias 2 -> 1
- net RADIO_NSS: vias 2 -> 1
Changed lines of the file:
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@@
 <?xml version="1.0" encoding="utf-8"?>
 <!DOCTYPE eagle SYSTEM "eagle.dtd">
-<eagle version="9.5.1">
+<eagle version="9.6.2">
 <drawing>
 <settings>
@@
 </layers>
 <board>
-<fusionsync huburn="a.cGVyc29uYWw6dWUyZDhlY2M3" projecturn="a.cGVyc29uYWw6dWUyZDhlY2M3IzIwMTgwNjIyMTM3MzM5MDA2" f3durn="urn:adsk.wipprod:dm.lineage:QPpZktTET7ejCF_ArrbzTw" pcbguid="f848ebd0-78e5-4ff5-950d-ec630e07b391" lastpulledtime="" lastsyncedchangeguid="6a44ac2e-81d3-cdee-9ebe-45ffbfe41bd8"/>
+<fusionsync huburn="a.cGVyc29uYWw6dWUyZDhlY2M3" projecturn="a.cGVyc29uYWw6dWUyZDhlY2M3IzIwMTgwNjIyMTM3MzM5MDA2" f3durn="urn:adsk.wipprod:dm.lineage:QPpZktTET7ejCF_ArrbzTw" pcbguid="f848ebd0-78e5-4ff5-950d-ec630e07b391" lastpulledtime="" lastsyncedchangeguid="6a44ac2e-81d3-cdee-9ebe-45ffbfe41bd8" latestrevisionid="" lastsyncedrevisionid="" lastboardhashguid="" lastpushedtime="" linktopcb3d="false"/>
 <plain>
 <wire x1="52" y1="14" x2="52" y2="56" width="0" layer="20"/>
@@
 <signal name="RADIO_NSS">
 <contactref element="U4" pad="13P"/>
-<wire x1="45.0066" y1="15.8066" x2="45.0066" y2="27.4" width="0.2" layer="16"/>
-<via x="45.0066" y="27.4" extent="1-16" drill="0.4"/>
+<wire x1="45.0066" y1="15.8066" x2="45.0066" y2="27" width="0.2" layer="16"/>
 <wire x1="35.7" y1="6.5" x2="45.0066" y2="15.8066" width="0.2" layer="16"/>
 <contactref element="U1" pad="30"/>
-<wire x1="45.0066" y1="27.4" x2="43.4" y2="29.0066" width="0.2" layer="1"/>
-<wire x1="43.4" y1="29.0066" x2="43.4" y2="30.38" width="0.2" layer="1"/>
 <wire x1="27.1" y1="10.8" x2="30.95" y2="6.95" width="0.2" layer="16"/>
 <wire x1="30.95" y1="6.95" x2="31.4" y2="6.5" width="0.2" layer="16"/>
@@
 <wire x1="29.5186" y1="6.9" x2="29.5686" y2="6.95" width="0.2" layer="16"/>
 <wire x1="29.5686" y1="6.95" x2="30.95" y2="6.95" width="0.2" layer="16"/>
+<wire x1="45.0066" y1="27" x2="43.4" y2="28.6066" width="0.2" layer="16"/>
+<wire x1="43.4" y1="28.6066" x2="43.4" y2="30.38" width="0.2" layer="16"/>
 </signal>
 <signal name="RADIO_DIO0">
@@
 <wire x1="31.9" y1="7.1" x2="35.4" y2="7.1" width="0.2" layer="16"/>
 <wire x1="44.451" y1="16.151" x2="44.451" y2="26.149" width="0.2" layer="16"/>
-<wire x1="44.451" y1="26.149" x2="43.8" y2="26.8" width="0.2" layer="16"/>
-<via x="43.8" y="27" extent="1-16" drill="0.4"/>
-<wire x1="43.8" y1="26.8" x2="43.8" y2="27" width="0.2" layer="16"/>
-<wire x1="41.4" y1="34.2" x2="42.1" y2="33.5" width="0.2" layer="1"/>
-<wire x1="42.1" y1="33.5" x2="42.1" y2="28.7" width="0.2" layer="1"/>
-<wire x1="43.8" y1="27" x2="42.1" y2="28.7" width="0.2" layer="1"/>
-<via x="41.4" y="34.2" extent="1-16" drill="0.4"/>
-<wire x1="41.4" y1="34.2" x2="41.4" y2="40.6" width="0.2" layer="16"/>
-<wire x1="41.4" y1="40.6" x2="37.1" y2="44.9" width="0.2" layer="16"/>
-<wire x1="37.1" y1="44.9" x2="37.1" y2="46.9" width="0.2" layer="16"/>
-<wire x1="37.1" y1="46.9" x2="36.5" y2="47.5" width="0.2" layer="16"/>
-<wire x1="36.5" y1="47.5" x2="24.5" y2="47.5" width="0.2" layer="16"/>
-<wire x1="23.08" y1="46.08" x2="24.5" y2="47.5" width="0.2" layer="16"/>
+<wire x1="44.451" y1="26.149" x2="43.7" y2="26.9" width="0.2" layer="16"/>
+<via x="43.7" y="26.9" extent="1-16" drill="0.4"/>
 <wire x1="30.142425" y1="13.557575" x2="27.857575" y2="13.557575" width="0.2" layer="16"/>
 <wire x1="27.857575" y1="13.557575" x2="27.1" y2="12.8" width="0.2" layer="16"/>
@@
 <wire x1="14.7444" y1="43.3556" x2="20.8156" y2="43.3556" width="0.2" layer="16"/>
 <wire x1="20.8156" y1="43.3556" x2="23.08" y2="45.62" width="0.2" layer="16"/>
-<wire x1="23.08" y1="45.62" x2="23.08" y2="46.08" width="0.2" layer="16"/>
+<wire x1="23.08" y1="45.62" x2="24.7" y2="44" width="0.2" layer="15"/>
+<wire x1="24.7" y1="44" x2="39" y2="44" width="0.2" layer="15"/>
+<wire x1="39" y1="44" x2="42.3" y2="40.7" width="0.2" layer="15"/>
+<wire x1="42.3" y1="28.3" x2="43.7" y2="26.9" width="0.2" layer="15"/>
+<wire x1="42.3" y1="40.7" x2="42.3" y2="28.3" width="0.2" layer="15"/>
 </signal>
 <signal name="ESC_TX5">
@@
 <via x="45.574959375" y="28.474959375" extent="1-16" drill="0.4"/>
 <contactref element="U1" pad="28"/>
-<wire x1="45.574959375" y1="28.474959375" x2="40.225040625" y2="28.474959375" width="0.2" layer="15"/>
-<wire x1="40.225040625" y1="28.474959375" x2="38.32" y2="30.38" width="0.2" layer="15"/>
 <wire x1="15.55" y1="5.6" x2="16.028975" y2="5.121025" width="0.2" layer="1"/>
 <wire x1="16.028975" y1="5.121025" x2="16.028975" y2="4" width="0.2" layer="1"/>
@@
 <wire x1="24.36631875" y1="2.877" x2="22.123" y2="2.877" width="0.2" layer="1"/>
 <wire x1="22.123" y1="2.877" x2="20.9625" y2="4.0375" width="0.2" layer="1"/>
+<wire x1="38.32" y1="30.38" x2="40.225040625" y2="28.474959375" width="0.2" layer="2"/>
+<wire x1="40.225040625" y1="28.474959375" x2="45.574959375" y2="28.474959375" width="0.2" layer="2"/>
 </signal>
 </signals>

Commit message: Replaced parts in Gucci control board
Replaced parts in Gucci control board
Parts:
- DIST_1, DIST_2, DIST_3, DIST_4, DIST_5, DIST_6: value MOLEX_1.25MM_4PIN_SMT -> 0532610471; device Kirbi_ControlBoard:MOLEX_1.25MM_4PIN_SMT -> Kirbi_ControlBoard:0532610471
- ESC1, ESC2: value MOLEX_1.25MM_3PIN_SMT -> 0532610371; device Kirbi_ControlBoard:MOLEX_1.25MM_3PIN_SMT -> Kirbi_ControlBoard:0532610371
- F1: device Kirbi_ControlBoard:BEL_FUSE_C1F_3.5 -> Kirbi_ControlBoard:C1F
- LINE_LF, LINE_RF, START: value AMPHENOL_2X02_2.54MM_SHROUD -> 75869-130LF; device Gucci_ControlBoard:AMPHENOL_2X02_2.54MM_SHROUD -> Gucci_ControlBoard:75869-130LF
- MUX_RX1, MUX_RX2, MUX_RX3, MUX_TX1, MUX_TX2, MUX_TX3: value MUX_74LVC1G157GV -> 74LVC1G157GW,125; device Kirbi_ControlBoard:MUX_74LVC1G157GV -> Kirbi_ControlBoard:TSSOP6
- PDB_CONN: value AMPHENOL_2X3_2.54MM -> 71600-006LF
- POWER_CONN: value MOLEX_2.54MM_2PIN -> 1719770002; device Kirbi_ControlBoard:MOLEX_2.54MM_2PIN -> Kirbi_ControlBoard:1719770002
- U2: device ICM-20948:QFN40P300X300X105-25N -> Gucci_ControlBoard:24-QFN_(3X3)
- U3: value PCA9306_LSSOP -> PCA9306
- U4: value (none) -> RFM69HCW_SMT
- U5: value LM393-8-SOIC -> LM393ADR
- moved R26 0.20 mm to (14.7, 5.40)
Connections:
- net +3.3V: now also MUX_RX1.5, MUX_RX2.5, MUX_RX3.5, MUX_TX1.5, MUX_TX2.5, MUX_TX3.5; no longer MUX_RX1.P$5, MUX_RX2.P$5, MUX_RX3.P$5, MUX_TX1.P$5, MUX_TX2.P$5, MUX_TX3.P$5
- net +5V: now also DIST_1.6, DIST_2.6, DIST_3.6, DIST_4.6, DIST_5.6, DIST_6.6, POWER_SWITCH.P, U5.8; no longer DIST_1.P$6, DIST_2.P$6, DIST_3.P$6, DIST_4.P$6, DIST_5.P$6, DIST_6.P$6, POWER_SWITCH.P$2, U5.P$8
- net 1.8V: now also U3.2; no longer U3.P$2
- net ESC_RX4: now also ESC1.2; no longer ESC1.P$2
- net ESC_RX5: now also ESC2.2; no longer ESC2.P$2
- net ESC_TX4: now also ESC1.1; no longer ESC1.P$1
- net ESC_TX5: now also ESC2.1; no longer ESC2.P$1
- net GND: now also DIST_1.3, DIST_2.3, DIST_3.3, DIST_4.3, DIST_5.3, DIST_6.3, ESC1.3, ESC2.3, MUX_RX1.2, MUX_RX2.2, MUX_RX3.2, MUX_TX1.2, MUX_TX2.2, MUX_TX3.2, POWER_CONN.1, U3.1, U5.4; no longer DIST_1.P$3, DIST_2.P$3, DIST_3.P$3, DIST_4.P$3, DIST_5.P$3, DIST_6.P$3, ESC1.P$3, ESC2.P$3, MUX_RX1.P$2, MUX_RX2.P$2, MUX_RX3.P$2, MUX_TX1.P$2, MUX_TX2.P$2, MUX_TX3.P$2, POWER_CONN.P$2, U3.P$1, U5.P$4
- net LF_INT: now also U5.7; no longer U5.P$7
- net LINE_LF: now also U5.5; no longer U5.P$5
- net LINE_REF: now also U5.2, U5.6; no longer U5.P$2, U5.P$6
- net LINE_RF: now also U5.3; no longer U5.P$3
- net MISO: now also PDB_CONN.5; no longer PDB_CONN.P$5
- net MOSI: now also PDB_CONN.4; no longer PDB_CONN.P$4
- net MUXS1: now also MUX_RX1.6, MUX_TX1.6; no longer MUX_RX1.P$6, MUX_TX1.P$6
- net MUXS2: now also MUX_RX2.6, MUX_TX2.6; no longer MUX_RX2.P$6, MUX_TX2.P$6
- net MUXS3: now also MUX_RX3.6, MUX_TX3.6; no longer MUX_RX3.P$6, MUX_TX3.P$6
- net N$4: now also U3.7, U3.8; no longer U3.P$7, U3.P$8
- net N$6: now also F1.2, POWER_SWITCH.1; no longer F1.P$2, POWER_SWITCH.P$1
- net N$7: now also F1.1, POWER_CONN.2; no longer F1.P$1, POWER_CONN.P$1
- net PDB_!CS!: now also PDB_CONN.6; no longer PDB_CONN.P$6
- net PDB_!EOC!: now also PDB_CONN.2; no longer PDB_CONN.P$2
- net PDB_START: now also PDB_CONN.1; no longer PDB_CONN.P$1
- net RF_INT: now also U5.1; no longer U5.P$1
- net RXD1: now also DIST_1.4, MUX_RX1.3; no longer DIST_1.P$4, MUX_RX1.P$3
- net RXD2: now also DIST_2.4, MUX_RX1.1; no longer DIST_2.P$4, MUX_RX1.P$1
- net RXD3: now also DIST_3.4, MUX_RX3.3; no longer DIST_3.P$4, MUX_RX3.P$3
- net RXD4: now also DIST_4.4, MUX_RX3.1; no longer DIST_4.P$4, MUX_RX3.P$1
- net RXD5: now also DIST_5.4, MUX_RX2.3; no longer DIST_5.P$4, MUX_RX2.P$3
- net RXD6: now also DIST_6.4, MUX_RX2.1; no longer DIST_6.P$4, MUX_RX2.P$1
- net SCK: now also PDB_CONN.3; no longer PDB_CONN.P$3
- net SCL1: now also U3.3; no longer U3.P$3
- net SCL2: now also U3.6; no longer U3.P$6
- net SDA1: now also U3.4; no longer U3.P$4
- net SDA2: now also U3.5; no longer U3.P$5
- net TRX1: now also MUX_RX1.4; no longer MUX_RX1.P$4
- net TRX2: now also MUX_RX2.4; no longer MUX_RX2.P$4
- net TRX3: now also MUX_RX3.4; no longer MUX_RX3.P$4
- net TTX1: now also MUX_TX1.4; no longer MUX_TX1.P$4
- net TTX2: now also MUX_TX2.4; no longer MUX_TX2.P$4
- net TTX3: now also MUX_TX3.4; no longer MUX_TX3.P$4
- net TXD1: now also DIST_1.5, MUX_TX1.3; no longer DIST_1.P$5, MUX_TX1.P$3
- net TXD2: now also DIST_2.5, MUX_TX1.1; no longer DIST_2.P$5, MUX_TX1.P$1
- net TXD3: now also DIST_3.5, MUX_TX3.3; no longer DIST_3.P$5, MUX_TX3.P$3
- net TXD4: now also DIST_4.5, MUX_TX3.1; no longer DIST_4.P$5, MUX_TX3.P$1
- net TXD5: now also DIST_5.5, MUX_TX2.3; no longer DIST_5.P$5, MUX_TX2.P$3
- net TXD6: now also DIST_6.5, MUX_TX2.1; no longer DIST_6.P$5, MUX_TX2.P$1
Routing:
- net TXD1: track 16.2 -> 19.1 mm, vias 1 -> 2
- net GND: track 116.7 -> 117.7 mm
- net MUXS1: track 27.0 -> 27.5 mm
- net TRX3: track 60.4 -> 60.9 mm
