File: Gucci/v3 pcb/Gucci_ControlBoard.brd (EAGLE design)
At the start: 66 x 56 mm, 89 parts, among them U1 TEENSY_3.6_DIL, U2 ICM-20948, U3 PCA9306, U4 RFM69HCW_SMT, U5 LM393ADR, U6 AP2114H-1.8TRG1, U7 AP2114H-3.3TRG1

Commit message: Replaced more parts on Gucci
Replaced more parts on Gucci
Parts:
- D1, D5: value DFLS130L-7_30V_1A -> 30; device Kirbi_ControlBoard:DFLS130L-7_30V_1A -> Kirbi_ControlBoard:DFLS130L-7
Connections:
- net +3.3V: now also D1.2, D5.1; no longer D1.P$2, D5.P$1
- net +5V: now also D1.1; no longer D1.P$1
- net 1.8V: now also D5.2; no longer D5.P$2
Changed lines of the file:
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@@
 <attribute name="VALUE" x="30.9" y="0.838" size="0.6096" layer="28" font="vector" ratio="20" rot="MR0" align="top-center"/>
 </element>
-<element name="D1" library="Kirbi_ControlBoard" package="DFLS130L-7_30V_1A" value="DFLS130L-7_30V_1A" x="29.6" y="41.9" smashed="yes">
+<element name="D1" library="Kirbi_ControlBoard" package="DFLS130L-7" value="30" x="29.6" y="41.9" smashed="yes">
+<attribute name="DKPN" value="DFLS130LDICT-ND" x="29.6" y="41.9" size="1.778" layer="27" display="off"/>
 <attribute name="NAME" x="28.2" y="39.5" size="1.016" layer="25" font="vector"/>
-<attribute name="VALUE" x="27.6" y="39.2" size="1.016" layer="27" font="vector"/>
-</element>
-<element name="D5" library="Kirbi_ControlBoard" package="DFLS130L-7_30V_1A" value="DFLS130L-7_30V_1A" x="19.1" y="18.6" smashed="yes" rot="R270">
+<attribute name="VALUE" value="30" x="27.6" y="39.2" size="1.016" layer="27" font="vector"/>
+</element>
+<element name="D5" library="Kirbi_ControlBoard" package="DFLS130L-7" value="30" x="19.1" y="18.6" smashed="yes" rot="R270">
+<attribute name="DKPN" value="DFLS130LDICT-ND" x="19.1" y="18.6" size="1.778" layer="27" rot="R270" display="off"/>
 <attribute name="NAME" x="18.3" y="20.8" size="1.016" layer="25" font="vector"/>
-<attribute name="VALUE" x="16.4" y="20.6" size="1.016" layer="27" font="vector" rot="R270"/>
+<attribute name="VALUE" value="30" x="16.4" y="20.6" size="1.016" layer="27" font="vector" rot="R270"/>
 </element>
 <element name="R12" library="SparkFun-Resistors" library_urn="urn:adsk.eagle:library:532" package="0603" package3d_urn="urn:adsk.eagle:package:39650/1" value="1k" x="-4.4" y="22.8" smashed="yes" rot="R270">
@@
 <contactref element="C25" pad="1"/>
 <contactref element="C12" pad="1"/>
-<contactref element="D1" pad="P$1"/>
+<contactref element="D1" pad="1"/>
 <contactref element="POWER_SWITCH" pad="P"/>
 <contactref element="5V" pad="A"/>
@@
 <wire x1="6.54" y1="14" x2="8.27" y2="12.27" width="0.2" layer="16"/>
 <wire x1="8.27" y1="14.68" x2="8.27" y2="12.27" width="0.2" layer="1"/>
-<contactref element="D1" pad="P$2"/>
-<contactref element="D5" pad="P$1"/>
+<contactref element="D1" pad="2"/>
+<contactref element="D5" pad="1"/>
 <wire x1="28.65" y1="41.9" x2="28.65" y2="42.3" width="0.3" layer="1"/>
 <wire x1="28.65" y1="42.3" x2="26.6944" y2="44.2556" width="0.3" layer="1"/>
@@
 <wire x1="24" y1="25.6556" x2="24" y2="26.877" width="0.2" layer="16"/>
 <wire x1="24" y1="26.877" x2="25.123" y2="28" width="0.2" layer="16"/>
-<contactref element="D5" pad="P$2"/>
+<contactref element="D5" pad="2"/>
 </signal>
 <signal name="EXP_PAD">

Commit message: Fixed Diodes on Kirbi, Gucci, and PD Board
Fixed Diodes (DFLS130L-7) on Kirbi, Gucci, and PD Board from Kirbi Library
Parts:
- turned D1 to 180 degrees
- turned D5 to 90 degrees
Connections:
- net +3.3V: now also D1.1, D5.2; no longer D1.2, D5.1
- net +5V: now also D1.2; no longer D1.1
- net 1.8V: now also D5.1; no longer D5.2
Routing:
- net +5V: track 49.7 -> 50.3 mm
Changed lines of the file:
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@@
 <attribute name="VALUE" x="30.9" y="0.838" size="0.6096" layer="28" font="vector" ratio="20" rot="MR0" align="top-center"/>
 </element>
-<element name="D1" library="Kirbi_ControlBoard" package="DFLS130L-7" value="30" x="29.6" y="41.9" smashed="yes">
-<attribute name="DKPN" value="DFLS130LDICT-ND" x="29.6" y="41.9" size="1.778" layer="27" display="off"/>
-<attribute name="NAME" x="28.2" y="39.5" size="1.016" layer="25" font="vector"/>
-<attribute name="VALUE" value="30" x="27.6" y="39.2" size="1.016" layer="27" font="vector"/>
-</element>
-<element name="D5" library="Kirbi_ControlBoard" package="DFLS130L-7" value="30" x="19.1" y="18.6" smashed="yes" rot="R270">
-<attribute name="DKPN" value="DFLS130LDICT-ND" x="19.1" y="18.6" size="1.778" layer="27" rot="R270" display="off"/>
-<attribute name="NAME" x="18.3" y="20.8" size="1.016" layer="25" font="vector"/>
-<attribute name="VALUE" value="30" x="16.4" y="20.6" size="1.016" layer="27" font="vector" rot="R270"/>
+<element name="D1" library="Kirbi_ControlBoard" package="DFLS130L-7" value="30" x="29.6" y="41.9" smashed="yes" rot="R180">
+<attribute name="DKPN" value="DFLS130LDICT-ND" x="29.6" y="41.9" size="1.778" layer="27" rot="R180" display="off"/>
+<attribute name="NAME" x="30.3" y="40.7" size="1.016" layer="25" font="vector" rot="R180"/>
+<attribute name="VALUE" value="30" x="31.6" y="44.6" size="1.016" layer="27" font="vector" rot="R180"/>
+</element>
+<element name="D5" library="Kirbi_ControlBoard" package="DFLS130L-7" value="30" x="19.1" y="18.6" smashed="yes" rot="R90">
+<attribute name="DKPN" value="DFLS130LDICT-ND" x="19.1" y="18.6" size="1.778" layer="27" rot="R90" display="off"/>
+<attribute name="NAME" x="19.8" y="22" size="1.016" layer="25" font="vector" rot="R180"/>
+<attribute name="VALUE" value="30" x="21.8" y="16.6" size="1.016" layer="27" font="vector" rot="R90"/>
 </element>
 <element name="R12" library="SparkFun-Resistors" library_urn="urn:adsk.eagle:library:532" package="0603" package3d_urn="urn:adsk.eagle:package:39650/1" value="1k" x="-4.4" y="22.8" smashed="yes" rot="R270">
@@
 <contactref element="C25" pad="1"/>
 <contactref element="C12" pad="1"/>
-<contactref element="D1" pad="1"/>
+<contactref element="D1" pad="2"/>
 <contactref element="POWER_SWITCH" pad="P"/>
 <contactref element="5V" pad="A"/>
@@
 <wire x1="-7.2" y1="41.45" x2="-7.2" y2="40.4" width="0.2" layer="1"/>
 <via x="-7.2" y="40.4" extent="1-16" drill="0.4"/>
-<wire x1="32.4" y1="42.6" x2="31.7" y2="41.9" width="0.2" layer="1"/>
-<wire x1="31.7" y1="41.9" x2="31.2" y2="41.9" width="0.2" layer="1"/>
 <via x="32.4" y="42.6" extent="1-16" drill="0.4"/>
 <wire x1="16.08561875" y1="42.31438125" x2="15.4" y2="41.6287625" width="0.2" layer="1"/>
@@
 <wire x1="24.4" y1="34.875" x2="24.4" y2="34.2" width="0.2" layer="1"/>
 <via x="24.4" y="34.2" extent="1-16" drill="0.4"/>
+<wire x1="30.55" y1="41.9" x2="31.25" y2="42.6" width="0.2" layer="1"/>
+<wire x1="31.25" y1="42.6" x2="32.4" y2="42.6" width="0.2" layer="1"/>
 </signal>
 <signal name="+3.3V">
@@
 <wire x1="6.54" y1="14" x2="8.27" y2="12.27" width="0.2" layer="16"/>
 <wire x1="8.27" y1="14.68" x2="8.27" y2="12.27" width="0.2" layer="1"/>
-<contactref element="D1" pad="2"/>
-<contactref element="D5" pad="1"/>
-<wire x1="28.65" y1="41.9" x2="28.65" y2="42.3" width="0.3" layer="1"/>
-<wire x1="28.65" y1="42.3" x2="26.6944" y2="44.2556" width="0.3" layer="1"/>
-<wire x1="26.6944" y1="44.2556" x2="22.2556" y2="44.2556" width="0.3" layer="1"/>
-<wire x1="19.1" y1="17" x2="19.878975" y2="17" width="0.2" layer="1"/>
-<wire x1="19.878975" y1="17" x2="20.9394875" y2="15.9394875" width="0.2" layer="1"/>
+<contactref element="D1" pad="1"/>
+<contactref element="D5" pad="2"/>
 <wire x1="20.65" y1="53.8" x2="20.65" y2="51.1" width="0.3" layer="1"/>
 <wire x1="20.65" y1="51.1" x2="20.65" y2="48.5" width="0.3" layer="1"/>
@@
 <wire x1="29.2" y1="14.1867125" x2="29.2" y2="14.3" width="0.5" layer="1"/>
 <wire x1="29.2" y1="14.3" x2="29.2" y2="17" width="0.5" layer="1"/>
-<wire x1="20.9394875" y1="15.9394875" x2="28.1394875" y2="15.9394875" width="0.2" layer="1"/>
-<wire x1="28.1394875" y1="15.9394875" x2="29.2" y2="17" width="0.2" layer="1"/>
+<wire x1="29.2" y1="17" x2="28.1394875" y2="15.9394875" width="0.2" layer="1"/>
 <wire x1="29.2" y1="17" x2="29.6" y2="16.6" width="0.2" layer="1"/>
 <wire x1="29.6" y1="16.6" x2="30.85" y2="16.6" width="0.2" layer="1"/>
@@
 <wire x1="23.6" y1="11.05" x2="21.525" y2="8.975" width="0.2" layer="1"/>
 <wire x1="21.525" y1="8.975" x2="21.3" y2="8.975" width="0.2" layer="1"/>
+<wire x1="28.1394875" y1="15.9394875" x2="22.0605125" y2="15.9394875" width="0.2" layer="1"/>
+<wire x1="28" y1="41.9" x2="28" y2="43" width="0.3" layer="1"/>
+<wire x1="28" y1="43" x2="26.7444" y2="44.2556" width="0.3" layer="1"/>
+<wire x1="26.7444" y1="44.2556" x2="22.2556" y2="44.2556" width="0.3" layer="1"/>
+<wire x1="22.0605125" y1="15.9394875" x2="20" y2="18" width="0.2" layer="1"/>
+<wire x1="20" y1="18" x2="19.45" y2="18" width="0.2" layer="1"/>
+<wire x1="19.45" y1="18" x2="19.1" y2="17.65" width="0.2" layer="1"/>
 </signal>
 <signal name="LINE_LF">
@@
 <wire x1="24" y1="25.6556" x2="24" y2="26.877" width="0.2" layer="16"/>
 <wire x1="24" y1="26.877" x2="25.123" y2="28" width="0.2" layer="16"/>
-<contactref element="D5" pad="2"/>
+<contactref element="D5" pad="1"/>
 </signal>
 <signal name="EXP_PAD">

Commit message: Fixed doubled parts in Gucci and Kirbi Library
Fixed doubled parts in Gucci and Kirbi Library (IMU, Teensy)
Parts:
- U1: value TEENSY_3.6_DIL -> TEENSY_3.6; device Teensy_3_and_LC_Series_Boards_v1.4:TEENSY_3.6_DIL -> Gucci_ControlBoard:TEENSY_3.6
Changed lines of the file:
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@@
 </autorouter>
 <elements>
-<element name="U1" library="Teensy_3_and_LC_Series_Boards_v1.4" package="TEENSY_3.6_DIL" value="TEENSY_3.6_DIL" x="18" y="38" smashed="yes" rot="R90">
+<element name="U1" library="Gucci_ControlBoard" package="TEENSY_3.6" value="TEENSY_3.6" x="18" y="38" smashed="yes" rot="R90">
+<attribute name="DKPN" value="1568-1442-ND" x="18" y="38" size="1.778" layer="27" rot="R90" display="off"/>
 <attribute name="NAME" x="47.875" y="44.285" size="1.6764" layer="25" font="vector" rot="R180"/>
 </element>

Commit message: Switched RX4 and TX4 pins on Gucci
Switched RX4 and TX4 on Gucci (make it consistent with the rest of the board)
Connections:
- net ESC_RX4: now also ESC1.1, U1.31/A12; no longer ESC1.2, U1.32/A13
- net ESC_TX4: now also ESC1.2, U1.32/A13; no longer ESC1.1, U1.31/A12
Routing:
- net ESC_TX4: track 10.9 -> 9.32 mm
- net ESC_RX4: track 9.32 -> 10.9 mm
Changed lines of the file:
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@@
 </signal>
 <signal name="ESC_TX4">
+<contactref element="ESC1" pad="2"/>
+<contactref element="U1" pad="32/A13"/>
+<wire x1="48.7" y1="37.5" x2="48.2" y2="38" width="0.2" layer="16"/>
+<wire x1="48.7" y1="37.5" x2="48.7" y2="36" width="0.2" layer="16"/>
+<wire x1="48.7" y1="36" x2="48" y2="35.3" width="0.2" layer="16"/>
+<wire x1="48" y1="35.3" x2="48" y2="30.86" width="0.2" layer="16"/>
+<wire x1="48" y1="30.86" x2="48.48" y2="30.38" width="0.2" layer="16"/>
+<wire x1="48.2" y1="38" x2="47.2" y2="38" width="0.2" layer="16"/>
+</signal>
+<signal name="ESC_RX4">
+<contactref element="ESC1" pad="1"/>
 <contactref element="U1" pad="31/A12"/>
-<contactref element="ESC1" pad="1"/>
 <wire x1="45" y1="38.3" x2="45.95" y2="39.25" width="0.2" layer="16"/>
 <wire x1="45" y1="38.3" x2="45" y2="31.32" width="0.2" layer="16"/>
@@
 <wire x1="45.95" y1="39.25" x2="47.2" y2="39.25" width="0.2" layer="16"/>
 </signal>
-<signal name="ESC_RX4">
-<contactref element="U1" pad="32/A13"/>
-<contactref element="ESC1" pad="2"/>
-<wire x1="47.2" y1="38" x2="48.2" y2="38" width="0.2" layer="16"/>
-<wire x1="48.2" y1="38" x2="48.7" y2="37.5" width="0.2" layer="16"/>
-<wire x1="48.7" y1="37.5" x2="48.7" y2="36" width="0.2" layer="16"/>
-<wire x1="48.7" y1="36" x2="48" y2="35.3" width="0.2" layer="16"/>
-<wire x1="48" y1="35.3" x2="48" y2="30.86" width="0.2" layer="16"/>
-<wire x1="48" y1="30.86" x2="48.48" y2="30.38" width="0.2" layer="16"/>
-</signal>
 <signal name="TRX3">
