File: Gucci/v3 pcb/Gucci_ControlBoard.sch (EAGLE design)
At the start: 57 parts, among them U1 PCA9306_LSSOP, U2 TEENSY_3.6_DIL, U5 LM393-8-SOIC, U6 AP2114H-1.8TRG1, U7 AP2114H-3.3TRG1

Commit message: Starting fixing git versions/Changing connectors
Starting fixing git versions - changed v4 name to v3 (made v3-old will delete later)
Changing connector (replacing the amphenol connector 71600-104LF
to 75869-130LF) - for the start module and line sensors
Parts:
- removed C13: 0.1uF, SparkFun-Capacitors:0.1UF-0603-25V-(+80/-20%)
- removed ESC: MOLEX_1.25MM_4PIN_SMT, Kirbi_ControlBoard:MOLEX_1.25MM_4PIN_SMT
- removed R21: 50, SparkFun-Resistors:1KOHM-0603-1/10W-1%
- added C10, C15, C25, C5, C9: 0.1uF, SparkFun-Capacitors:0.1UF-0603-25V-(+80/-20%)
- added ESC1, ESC2: MOLEX_1.25MM_3PIN_SMT, Kirbi_ControlBoard:MOLEX_1.25MM_3PIN_SMT
- added ESC_RX, ESC_TX: MUX_74LVC1G157GV, Kirbi_ControlBoard:MUX_74LVC1G157GV
- added F1: 3.5, Kirbi_ControlBoard:BEL_FUSE_C1F_3.5
- added POWER_CONN: MOLEX_2.54MM_2PIN, Kirbi_ControlBoard:MOLEX_2.54MM_2PIN
- added R10, R11, R3, R4, R5, R6, R7, R8, R9: 1k, SparkFun-Resistors:1KOHM-0603-1/10W-1%
- added R2: 6.2, Kirbi_ControlBoard:6.2OHM-0603-1/10W-5%
- R1: value 1.65k -> 100; device SparkFun-Resistors:1KOHM-0603-1/10W-1% -> SparkFun-Resistors:100OHM-0603-1/4W-5%
- R19: value 1.65k -> 200; device SparkFun-Resistors:1KOHM-0603-1/10W-1% -> SparkFun-Resistors:200OHM-0603-1/10W-1%
- R20: value 800 -> 100; device SparkFun-Resistors:1KOHM-0603-1/10W-1% -> SparkFun-Resistors:100OHM-0603-1/4W-5%
Connections:
- removed net N$10: D4.C, R21.1
- new net ESC_S: ESC_RX.S, ESC_TX.S, U2.36/A17/PWM
- new net ESC_TRX: ESC_RX.Y, R9.1, U2.34/A15/RX5/CAN1-RX
- new net ESC_TTX: ESC_TX.Y, U2.33/A14/TX5/CAN1-TX
- new net N$6: F1.P$2, POWER.P4
- new net N$7: F1.P$1, POWER_CONN.P$1
- new net N$9: D4.C, R2.1
- new net RADIO_RESET: TRANSCEIVER.RESET, U2.29/T/PWM
- new net S1/RX: ESC1.2, ESC_RX.I0
- new net S2/RX: ESC2.2, ESC_RX.I1
- new net S2/TX: ESC2.3, ESC_TX.I1, R11.1
- net +3.3V: now also ESC_RX.V, ESC_TX.V, R10.2, R11.2, R3.2, R4.2, R5.2, R6.2, R7.2, R8.2, R9.2
- net +5V: now also C10.1, C15.1, C25.1, C5.1, C9.1; no longer C13.1
- net GND: now also C10.2, C15.2, C25.2, C5.2, C9.2, ESC1.1, ESC2.1, ESC_RX.GND, ESC_TX.GND, POWER_CONN.P$2, R2.2; no longer C13.2, R21.2
- net LF_INT: now also U2.15/A1/T; no longer U2.18/A4/T/SDA0
- net RADIO_NSS: now also U2.30/T/PWM; no longer U2.6/PWM
- net RF_INT: now also U2.16/A2/T/PWM; no longer U2.19/A5/T/SCL0
- net S1/TX: now also ESC1.3, ESC_TX.I0, R10.1; no longer ESC.3, U2.33/A14/TX5/CAN1-TX
- net START: now also U2.14/A0/PWM; no longer U2.17/A3/T/PWM
- net TRX1: now also R7.1
- net TRX2: now also R8.1
- net TXD1: now also R5.1
- net TXD2: now also R3.1
- net TXD5: now also R4.1
- net TXD6: now also R6.1
Other:
- note added: "*Note: The TX and RX labels refer to the respective Teensy connection (not the ESC pins)"
- note added: "*Note: The TX and RX labels refer to the respective Teensy connection (not the sensor pins)"
- moved on the sheet: C11, C12

Commit message: Cleaned up Schematic/Silkscreen
Cleaned up Schematic/Silkscreen (moved a few things around)
Changed lines of the file:
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@@
 <part name="R11" library="SparkFun-Resistors" library_urn="urn:adsk.eagle:library:532" deviceset="1KOHM" device="-0603-1/10W-1%" package3d_urn="urn:adsk.eagle:package:39650/1" value="1k"/>
 <part name="+3V26" library="supply1" library_urn="urn:adsk.eagle:library:371" deviceset="+3V3" device=""/>
+<part name="GND31" library="SparkFun-PowerSymbols" library_urn="urn:adsk.eagle:library:530" deviceset="GND" device=""/>
 </parts>
 <sheets>
@@
 </instance>
 <instance part="POWER" gate="G$1" x="296.672" y="105.41" smashed="yes">
-<attribute name="NAME" x="294.132" y="105.41" size="1.27" layer="97"/>
+<attribute name="NAME" x="284.48" y="114.3" size="1.27" layer="97"/>
 </instance>
 <instance part="P+3" gate="1" x="296.672" y="118.11" smashed="yes">
-<attribute name="VALUE" x="294.132" y="113.03" size="1.778" layer="96" rot="R90"/>
+<attribute name="VALUE" x="294.64" y="114.3" size="1.778" layer="96" rot="R90"/>
 </instance>
 <instance part="P+9" gate="1" x="101.6" y="205.74" smashed="yes">
@@
 <instance part="POWER_CONN" gate="G$1" x="266.7" y="101.6" smashed="yes">
 <attribute name="NAME" x="262.89" y="108.204" size="1.778" layer="95"/>
-<attribute name="VALUE" x="262.636" y="93.98" size="1.778" layer="95"/>
+<attribute name="VALUE" x="256.794" y="93.98" size="1.778" layer="95"/>
 </instance>
 <instance part="C12" gate="G$1" x="58.42" y="228.6" smashed="yes">
@@
 <instance part="+3V26" gate="G$1" x="333.248" y="183.896" smashed="yes">
 <attribute name="VALUE" x="332.486" y="179.07" size="1.778" layer="96" rot="R270"/>
+</instance>
+<instance part="GND31" gate="1" x="403.86" y="53.34" smashed="yes">
+<attribute name="VALUE" x="403.86" y="53.086" size="1.778" layer="96" align="top-center"/>
 </instance>
 </instances>
@@
 <wire x1="381" y1="55.88" x2="391.16" y2="55.88" width="0.1524" layer="91"/>
 <junction x="381" y="55.88"/>
-<pinref part="C11" gate="G$1" pin="2"/>
-<wire x1="391.16" y1="55.88" x2="403.86" y2="55.88" width="0.1524" layer="91"/>
-<wire x1="403.86" y1="55.88" x2="403.86" y2="58.42" width="0.1524" layer="91"/>
 <pinref part="C14" gate="G$1" pin="2"/>
 <wire x1="391.16" y1="58.42" x2="391.16" y2="55.88" width="0.1524" layer="91"/>
-<junction x="391.16" y="55.88"/>
 </segment>
 <segment>
@@
 <wire x1="316.992" y1="85.09" x2="304.292" y2="85.09" width="0.1524" layer="91"/>
 <pinref part="R1" gate="G$1" pin="1"/>
-<wire x1="304.292" y1="85.09" x2="283.972" y2="85.09" width="0.1524" layer="91"/>
+<wire x1="304.292" y1="85.09" x2="283.21" y2="85.09" width="0.1524" layer="91"/>
 <junction x="304.292" y="85.09"/>
 <pinref part="POWER_CONN" gate="G$1" pin="P$2"/>
-<wire x1="274.32" y1="99.06" x2="283.972" y2="99.06" width="0.1524" layer="91"/>
-<wire x1="283.972" y1="99.06" x2="283.972" y2="85.09" width="0.1524" layer="91"/>
+<wire x1="274.32" y1="99.06" x2="283.21" y2="99.06" width="0.1524" layer="91"/>
+<wire x1="283.21" y1="99.06" x2="283.21" y2="85.09" width="0.1524" layer="91"/>
 </segment>
 <segment>
@@
 <pinref part="ESC_TX" gate="G$1" pin="GND"/>
 <pinref part="GND29" gate="1" pin="GND"/>
+</segment>
+<segment>
+<pinref part="C11" gate="G$1" pin="2"/>
+<wire x1="403.86" y1="55.88" x2="403.86" y2="58.42" width="0.1524" layer="91"/>
+<pinref part="GND31" gate="1" pin="GND"/>
 </segment>
 </net>
@@
 <wire x1="327.152" y1="97.79" x2="316.992" y2="97.79" width="0.1524" layer="91"/>
 <junction x="316.992" y="97.79"/>
-<wire x1="316.992" y1="97.79" x2="309.372" y2="97.79" width="0.1524" layer="91"/>
+<wire x1="316.992" y1="97.79" x2="313.69" y2="97.79" width="0.1524" layer="91"/>
 <junction x="316.992" y="97.79"/>
 <pinref part="P+3" gate="1" pin="+5V"/>
 <pinref part="POWER" gate="G$1" pin="P3"/>
 <wire x1="296.672" y1="115.57" x2="296.672" y2="110.49" width="0.1524" layer="91"/>
-<wire x1="296.672" y1="110.49" x2="296.672" y2="102.87" width="0.1524" layer="91"/>
+<wire x1="296.672" y1="110.49" x2="301.752" y2="102.87" width="0.1524" layer="91"/>
 <junction x="296.672" y="110.49"/>
 <junction x="296.672" y="115.57"/>
-<wire x1="309.372" y1="97.79" x2="309.372" y2="115.57" width="0.1524" layer="91"/>
-<wire x1="309.372" y1="115.57" x2="296.672" y2="115.57" width="0.1524" layer="91"/>
-<wire x1="296.672" y1="102.87" x2="291.592" y2="102.87" width="0.1524" layer="91"/>
+<wire x1="313.69" y1="97.79" x2="313.69" y2="115.57" width="0.1524" layer="91"/>
+<wire x1="313.69" y1="115.57" x2="296.672" y2="115.57" width="0.1524" layer="91"/>
+<wire x1="301.752" y1="102.87" x2="291.592" y2="102.87" width="0.1524" layer="91"/>
 <pinref part="POWER" gate="G$1" pin="P5"/>
 <wire x1="291.592" y1="102.87" x2="291.592" y2="97.79" width="0.1524" layer="91"/>
@@
 <segment>
 <pinref part="U1" gate="G$1" pin="SCL2"/>
-<wire x1="396.24" y1="96.52" x2="401.32" y2="96.52" width="0.1524" layer="91"/>
-<label x="401.32" y="96.52" size="1.778" layer="95" xref="yes"/>
+<wire x1="396.24" y1="96.52" x2="406.4" y2="96.52" width="0.1524" layer="91"/>
+<label x="406.4" y="96.52" size="1.778" layer="95" rot="R270" xref="yes"/>
 </segment>
 </net>
@@
 <pinref part="U1" gate="G$1" pin="SDA2"/>
 <wire x1="396.24" y1="93.98" x2="401.32" y2="93.98" width="0.1524" layer="91"/>
-<label x="401.32" y="93.98" size="1.778" layer="95" xref="yes"/>
-</segment>
-</net>
+<label x="401.32" y="93.98" size="1.778" layer="95" rot="R270" xref="yes"/>
+</segment>
+</net>

Commit message: PDB Conector/Power Switch/Resistors
Pull Up Resistor - Radio Module
Pull Down Resistors - MUXs
Power Distribution Board Connector (in Kirbi library and on schematic)
Replaced old power switch addded LED
Parts:
- removed POWER: POWER_SWITCH, Kirbi_ControlBoard:POWER_SWITCH
- added D1, D5: DFLS130L-7_30V_1A, Kirbi_ControlBoard:DFLS130L-7_30V_1A
- added D6: 5V, SparkFun-LED:LED0603
- added PDB_CONN: AMPHENOL_2X3_2.54MM, Kirbi_ControlBoard:AMPHENOL_2X3_2.54MM
- added POWER_SWITCH: GPTS202312B, Kirbi_ControlBoard:GPTS202312B
- added R12, R18, R21, R22, R23, R26, R27: 1k, SparkFun-Resistors:1KOHM-0603-1/10W-1%
- R1: value 100 -> 200; device SparkFun-Resistors:100OHM-0603-1/4W-5% -> SparkFun-Resistors:200OHM-0603-1/10W-1%
Connections:
- new net PDB_!CS!: PDB_CONN.1
- new net PDB_!EOC!: PDB_CONN.4
- new net PDB_MISO: PDB_CONN.2, U2.5/PWM
- new net PDB_MOSI: PDB_CONN.5, U2.21/A7/PWM
- new net PDB_SCLK: PDB_CONN.3, U2.20/A6/PWM
- new net PDB_START: PDB_CONN.6
- net +3.3V: now also D1.A, D5.C, R23.2
- net +5V: now also D1.C, D6.A, POWER_SWITCH.COMMON; no longer POWER.P3, POWER.P5
- net 1.8V: now also D5.A
- net ESC_S: now also R26.2, R27.2
- net GND: now also R1.2, R12.1, R18.1, R21.1, R22.1, R26.1, R27.1; no longer R1.1
- net MUXS1: now also R12.2, R21.2
- net MUXS2: now also R18.2, R22.2
- net N$6: now also POWER_SWITCH.B; no longer POWER.P4
- net N$8: now also D6.C, R1.1; no longer POWER.P1, R1.2
- net NEO_DI: now also U2.6/PWM; no longer U2.24
- net RADIO_DIO0: now also U2.22/A8/T/PWM; no longer U2.5/PWM
- net RADIO_NSS: now also R23.1

Commit message: Routed Power Distribution Board
Routed Power Distribution Board
Connections:
- net PDB_!CS!: now also U2.17/A3/T/PWM
- net PDB_!EOC!: now also U2.18/A4/T/SDA0
- net PDB_START: now also U2.19/A5/T/SCL0
Changed lines of the file:
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@@
+</segment>
+</net>
+<net name="PDB_!CS!" class="0">
+<segment>
+<pinref part="U2" gate="G$1" pin="17/A3/T/PWM"/>
+<wire x1="165.1" y1="193.04" x2="160.02" y2="193.04" width="0.1524" layer="91"/>
+<label x="160.02" y="193.04" size="1.778" layer="95" rot="R180" xref="yes"/>
+</segment>
+</net>
+<net name="PDB_!EOC!" class="0">
+<segment>
+<pinref part="U2" gate="G$1" pin="18/A4/T/SDA0"/>
+<wire x1="165.1" y1="190.5" x2="160.02" y2="190.5" width="0.1524" layer="91"/>
+<label x="160.02" y="190.5" size="1.778" layer="95" rot="R180" xref="yes"/>
+</segment>
+</net>
+<net name="PDB_START" class="0">
+<segment>
+<pinref part="U2" gate="G$1" pin="19/A5/T/SCL0"/>
+<wire x1="165.1" y1="187.96" x2="160.02" y2="187.96" width="0.1524" layer="91"/>
+<label x="160.02" y="187.96" size="1.778" layer="95" rot="R180" xref="yes"/>
 </segment>
 </net>

Commit message: Screw Head Clearance/Silkscreen
Screw Head Clearance/Silkscreen cleaned up
Parts:
- renumbered D6 to 5V
Changed lines of the file:
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@@
 <part name="POWER_SWITCH" library="Kirbi_ControlBoard" deviceset="GPTS202312B" device=""/>
 <part name="R1" library="SparkFun-Resistors" library_urn="urn:adsk.eagle:library:532" deviceset="200OHM" device="-0603-1/10W-1%" package3d_urn="urn:adsk.eagle:package:39650/1" value="200"/>
-<part name="D6" library="SparkFun-LED" deviceset="LED" device="0603" value="5V"/>
+<part name="5V" library="SparkFun-LED" deviceset="LED" device="0603" value="5V"/>
 <part name="FRAME2" library="RoboJackets-Frames" deviceset="FRAME_B_L" device=""/>
 <part name="PDB_CONN" library="Kirbi_ControlBoard" deviceset="AMPHENOL_2X3_2.54MM" device=""/>
@@
 <attribute name="VALUE" x="313.436" y="91.44" size="1.778" layer="96" font="vector" rot="R270" align="top-center"/>
 </instance>
-<instance part="D6" gate="G$1" x="307.34" y="96.52" smashed="yes" rot="R90">
+<instance part="5V" gate="G$1" x="307.34" y="96.52" smashed="yes" rot="R90">
 <attribute name="NAME" x="309.372" y="93.091" size="1.778" layer="95" font="vector" rot="R180"/>
 <attribute name="VALUE" x="309.372" y="98.425" size="1.778" layer="96" font="vector" rot="R180" align="top-left"/>
@@
 <wire x1="306.832" y1="104.14" x2="304.8" y2="104.14" width="0.1524" layer="91"/>
 <junction x="306.832" y="115.57"/>
-<pinref part="D6" gate="G$1" pin="A"/>
+<pinref part="5V" gate="G$1" pin="A"/>
 <wire x1="304.8" y1="104.14" x2="304.8" y2="96.52" width="0.1524" layer="91"/>
 <junction x="304.8" y="104.14"/>
@@
 <net name="N$8" class="0">
 <segment>
-<pinref part="D6" gate="G$1" pin="C"/>
+<pinref part="5V" gate="G$1" pin="C"/>
 <pinref part="R1" gate="G$1" pin="1"/>
 <wire x1="314.96" y1="96.52" x2="312.42" y2="96.52" width="0.1524" layer="91"/>

Commit message: Renamed Parts/Routed SPI Interface
Renamed Parts (U1-U7)
Routed SPI Interface (Connectted MISO, MOSI, and SCK) (Fixed routing to avoid islands/breaks in ground plane)
Parts:
- removed IMU: ICM-20948, ICM-20948:ICM-20948
- added U3: PCA9306_LSSOP, Gucci_ControlBoard:PCA9306_LSSOP
- U1: value PCA9306_LSSOP -> TEENSY_3.6_DIL; device Gucci_ControlBoard:PCA9306_LSSOP -> Teensy_3_and_LC_Series_Boards_v1.4:TEENSY_3.6_DIL
- U2: value TEENSY_3.6_DIL -> ICM-20948; device Teensy_3_and_LC_Series_Boards_v1.4:TEENSY_3.6_DIL -> ICM-20948:ICM-20948
- renumbered TRANSCEIVER to U4
Connections:
- removed net PDB_MISO: PDB_CONN.2, U2.5/PWM
- removed net PDB_MOSI: PDB_CONN.5, U2.21/A7/PWM
- removed net PDB_SCLK: PDB_CONN.3, U2.20/A6/PWM
- removed net RADIO_SCK: U2.13/SCK0/LED, U4.SCK
- new net SCK: PDB_CONN.2, U1.13/SCK0/LED, U4.SCK
- net +5V: now also U1.VIN; no longer U2.VIN
- net 1.8V: now also U2.NCS, U2.VDD, U2.VDDIO, U3.VREF1; no longer IMU.NCS, IMU.VDD, IMU.VDDIO, U1.VREF1
- net ESC_S: now also U1.36/A17/PWM; no longer U2.36/A17/PWM
- net ESC_TRX: now also U1.34/A15/RX5/CAN1-RX; no longer U2.34/A15/RX5/CAN1-RX
- net ESC_TTX: now also U1.33/A14/TX5/CAN1-TX; no longer U2.33/A14/TX5/CAN1-TX
- net GND: now also U1.AGND, U2.AD0/SDO, U2.FSYNC, U2.RESV_20, U3.GND; no longer IMU.AD0/SDO, IMU.FSYNC, IMU.GND, IMU.RESV_20, U2.AGND
- net LF_INT: now also U1.15/A1/T; no longer U2.15/A1/T
- net LINE_LF: now also U1.35/A16/PWM; no longer U2.35/A16/PWM
- net LINE_REF: now also U1.A22/DAC1; no longer U2.A22/DAC1
- net LINE_RF: now also U1.23/A9/T/PWM; no longer U2.23/A9/T/PWM
- net MISO: now also PDB_CONN.3, U1.12/MISO0; no longer U2.12/MISO0
- net MOSI: now also PDB_CONN.5, U1.11/MOSI0; no longer U2.11/MOSI0
- net MUXS1: now also U1.2/PWM; no longer U2.2/PWM
- net MUXS2: now also U1.25; no longer U2.25
- net N$3: now also U2.REGOUT; no longer IMU.REGOUT
- net N$4: now also U3.EN, U3.VREF2; no longer U1.EN, U1.VREF2
- net NEO_DI: now also U1.6/PWM; no longer U2.6/PWM
- net PDB_!CS!: now also U1.17/A3/T/PWM; no longer U2.17/A3/T/PWM
- net PDB_!EOC!: now also U1.18/A4/T/SDA0; no longer U2.18/A4/T/SDA0
- net PDB_START: now also U1.19/A5/T/SCL0; no longer U2.19/A5/T/SCL0
- net RADIO_DIO0: now also U1.22/A8/T/PWM; no longer U2.22/A8/T/PWM
- net RADIO_NSS: now also U1.30/T/PWM; no longer U2.30/T/PWM
- net RADIO_RESET: now also U1.29/T/PWM; no longer U2.29/T/PWM
- net RF_INT: now also U1.16/A2/T/PWM; no longer U2.16/A2/T/PWM
- net RXD3: now also U1.0/RX1/MOSI1/T; no longer U2.0/RX1/MOSI1/T
- net RXD4: now also U1.31/A12/RX4; no longer U2.31/A12/RX4
- net SCL1: now also U2.SCL/SCLK, U3.SCL1; no longer IMU.SCL/SCLK, U1.SCL1
- net SCL2: now also U1.3/CAN0-TX/SCL2/PWM, U3.SCL2; no longer U1.SCL2, U2.3/CAN0-TX/SCL2/PWM
- net SDA1: now also U2.SDA/SDI, U3.SDA1; no longer IMU.SDA/SDI, U1.SDA1
- net SDA2: now also U1.4/CAN0-RX/SDA2/PWM, U3.SDA2; no longer U1.SDA2, U2.4/CAN0-RX/SDA2/PWM
- net START: now also U1.14/A0/PWM; no longer U2.14/A0/PWM
- net TRX1: now also U1.7/RX3/PWM; no longer U2.7/RX3/PWM
- net TRX2: now also U1.9/RX2/PWM; no longer U2.9/RX2/PWM
- net TTX1: now also U1.8/TX3/PWM; no longer U2.8/TX3/PWM
- net TTX2: now also U1.10/TX2/PWM; no longer U2.10/TX2/PWM
- net TXD3: now also U1.1/TX1/MISO1/T; no longer U2.1/TX1/MISO1/T
- net TXD4: now also U1.32/A13/TX4; no longer U2.32/A13/TX4

Commit message: Multiplexed Distance Sensors
Multiplexed Distance Sensors (3-4)/Directly connectted ESCs
Parts:
- removed ESC_RX, ESC_TX: MUX_74LVC1G157GV, Kirbi_ControlBoard:MUX_74LVC1G157GV
- added MUX_RX3, MUX_TX3: MUX_74LVC1G157GV, Kirbi_ControlBoard:MUX_74LVC1G157GV
Connections:
- removed net ESC_S: ESC_RX.S, ESC_TX.S, R26.2, R27.2, U1.36/A17/PWM
- removed net ESC_TRX: ESC_RX.Y, R9.1, U1.34/A15/RX5/CAN1-RX
- removed net ESC_TTX: ESC_TX.Y, U1.33/A14/TX5/CAN1-TX
- removed net S1/RX: ESC1.2, ESC_RX.I0
- removed net S1/TX: ESC1.3, ESC_TX.I0, R10.1
- removed net S2/RX: ESC2.2, ESC_RX.I1
- removed net S2/TX: ESC2.3, ESC_TX.I1, R11.1
- new net ESC_RX4: ESC1.2, U1.32/A13/TX4
- new net ESC_RX5: ESC2.2, U1.34/A15/RX5/CAN1-RX
- new net ESC_TX4: ESC1.3, U1.31/A12/RX4
- new net ESC_TX5: ESC2.3, U1.33/A14/TX5/CAN1-TX
- new net MUXS3: MUX_RX3.S, MUX_TX3.S, R26.2, R27.2, U1.28
- new net TRX3: MUX_RX3.Y, R9.1, U1.0/RX1/MOSI1/T
- new net TTX3: MUX_TX3.Y, U1.1/TX1/MISO1/T
- net +3.3V: now also MUX_RX3.V, MUX_TX3.V; no longer ESC_RX.V, ESC_TX.V
- net GND: now also MUX_RX3.GND, MUX_TX3.GND; no longer ESC_RX.GND, ESC_TX.GND
- net RXD3: now also MUX_RX3.I0; no longer U1.0/RX1/MOSI1/T
- net RXD4: now also MUX_RX3.I1; no longer U1.31/A12/RX4
- net TXD3: now also MUX_TX3.I0, R10.1; no longer U1.1/TX1/MISO1/T
- net TXD4: now also MUX_TX3.I1, R11.1; no longer U1.32/A13/TX4
Other:
- note added: "Multiplexers (D1-2,D5-6)"
- note added: "Multiplexers (D3-4)"
- note added: "Power Distribution Board"
- note removed: "Multiplexers"
- moved on the sheet: PDB_CONN, R10, R11, R26, R27, R9

Commit message: Replaced parts in Gucci control board
Replaced parts in Gucci control board
Parts:
- DIST_1, DIST_2, DIST_3, DIST_4, DIST_5, DIST_6: value MOLEX_1.25MM_4PIN_SMT -> 0532610471; device Kirbi_ControlBoard:MOLEX_1.25MM_4PIN_SMT -> Kirbi_ControlBoard:0532610471
- ESC1, ESC2: value MOLEX_1.25MM_3PIN_SMT -> 0532610371; device Kirbi_ControlBoard:MOLEX_1.25MM_3PIN_SMT -> Kirbi_ControlBoard:0532610371
- F1: device Kirbi_ControlBoard:BEL_FUSE_C1F_3.5 -> Kirbi_ControlBoard:C1F3.5
- LINE_LF, LINE_RF, START: value AMPHENOL_2X02_2.54MM_SHROUD -> 75869-130LF; device Gucci_ControlBoard:AMPHENOL_2X02_2.54MM_SHROUD -> Gucci_ControlBoard:75869-130LF
- MUX_RX1, MUX_RX2, MUX_RX3, MUX_TX1, MUX_TX2, MUX_TX3: value MUX_74LVC1G157GV -> 74LVC1G157GW,125; device Kirbi_ControlBoard:MUX_74LVC1G157GV -> Kirbi_ControlBoard:74LVC1G157GW,125
- PDB_CONN: value AMPHENOL_2X3_2.54MM -> 71600-006LF; device Kirbi_ControlBoard:AMPHENOL_2X3_2.54MM -> Kirbi_ControlBoard:71600-006LF
- POWER_CONN: value MOLEX_2.54MM_2PIN -> 1719770002; device Kirbi_ControlBoard:MOLEX_2.54MM_2PIN -> Kirbi_ControlBoard:1719770002
- U2: device ICM-20948:ICM-20948 -> Gucci_ControlBoard:ICM-20948
- U3: value PCA9306_LSSOP -> PCA9306; device Gucci_ControlBoard:PCA9306_LSSOP -> Gucci_ControlBoard:PCA9306
- U4: value (none) -> RFM69HCW_SMT
- U5: value LM393-8-SOIC -> LM393ADR; device Gucci_ControlBoard:LM393-8-SOIC -> Gucci_ControlBoard:LM393ADR
Connections:
- net +5V: now also U5.V+; no longer U5.VCC
- net GND: now also U5.V-; no longer U5.GND
- net LF_INT: now also U5.OUTB; no longer U5.OUT2
- net LINE_LF: now also U5.INB+; no longer U5.IN2+
- net LINE_REF: now also U5.INA-, U5.INB-; no longer U5.IN1-, U5.IN2-
- net LINE_RF: now also U5.INA+; no longer U5.IN1+
- net RF_INT: now also U5.OUTA; no longer U5.OUT1
Other:
- moved on the sheet: C19, C20, D1, D5, DIST_1, DIST_2, DIST_3, DIST_4, DIST_5, DIST_6, ESC1, ESC2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
