File: Gucci/v3 pcb/Gucci_ControlBoard.sch (EAGLE design)
At the start: 86 parts, among them U1 TEENSY_3.6_DIL, U2 ICM-20948, U3 PCA9306, U4 RFM69HCW_SMT, U5 LM393ADR, U6 AP2114H-1.8TRG1, U7 AP2114H-3.3TRG1

Commit message: Replaced more parts on Gucci
Replaced more parts on Gucci
Parts:
- D1, D5: value DFLS130L-7_30V_1A -> 30; device Kirbi_ControlBoard:DFLS130L-7_30V_1A -> Kirbi_ControlBoard:DFLS130L-7
Other:
- moved on the sheet: R2
Changed lines of the file:
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@@
 <part name="+3V26" library="supply1" library_urn="urn:adsk.eagle:library:371" deviceset="+3V3" device=""/>
 <part name="GND31" library="SparkFun-PowerSymbols" library_urn="urn:adsk.eagle:library:530" deviceset="GND" device=""/>
-<part name="D1" library="Kirbi_ControlBoard" deviceset="DFLS130L-7_30V_1A" device=""/>
-<part name="D5" library="Kirbi_ControlBoard" deviceset="DFLS130L-7_30V_1A" device=""/>
+<part name="D1" library="Kirbi_ControlBoard" deviceset="DFLS130L-7" device="" value="30"/>
+<part name="D5" library="Kirbi_ControlBoard" deviceset="DFLS130L-7" device="" value="30"/>
 <part name="R12" library="SparkFun-Resistors" library_urn="urn:adsk.eagle:library:532" deviceset="1KOHM" device="-0603-1/10W-1%" package3d_urn="urn:adsk.eagle:package:39650/1" value="1k"/>
 <part name="GND32" library="SparkFun-PowerSymbols" library_urn="urn:adsk.eagle:library:530" deviceset="GND" device=""/>
@@
 <attribute name="VALUE" x="276.86" y="100.33" size="1.778" layer="96"/>
 </instance>
-<instance part="R2" gate="G$1" x="292.1" y="33.02" smashed="yes">
-<attribute name="NAME" x="292.1" y="34.544" size="1.778" layer="95" font="vector" align="bottom-center"/>
-<attribute name="VALUE" x="292.1" y="31.496" size="1.778" layer="96" font="vector" align="top-center"/>
+<instance part="R2" gate="G$1" x="294.64" y="33.02" smashed="yes">
+<attribute name="NAME" x="294.64" y="34.544" size="1.778" layer="95" font="vector" align="bottom-center"/>
+<attribute name="VALUE" x="294.64" y="31.496" size="1.778" layer="96" font="vector" align="top-center"/>
 </instance>
 <instance part="GND29" gate="1" x="274.32" y="137.16" smashed="yes">
@@
 <wire x1="304.8" y1="30.48" x2="304.8" y2="33.02" width="0.1524" layer="91"/>
 <pinref part="R2" gate="G$1" pin="2"/>
-<wire x1="304.8" y1="33.02" x2="297.18" y2="33.02" width="0.1524" layer="91"/>
+<wire x1="304.8" y1="33.02" x2="299.72" y2="33.02" width="0.1524" layer="91"/>
 </segment>
 <segment>
@@
 <pinref part="R2" gate="G$1" pin="1"/>
 <pinref part="D4" gate="G$1" pin="C"/>
-<wire x1="287.02" y1="33.02" x2="279.4" y2="33.02" width="0.1524" layer="91"/>
-</segment>
-</net>
+<wire x1="289.56" y1="33.02" x2="279.4" y2="33.02" width="0.1524" layer="91"/>
+</segment>
+</net>

Commit message: Fixed doubled parts in Gucci and Kirbi Library
Fixed doubled parts in Gucci and Kirbi Library (IMU, Teensy)
Parts:
- U1: value TEENSY_3.6_DIL -> TEENSY_3.6; device Teensy_3_and_LC_Series_Boards_v1.4:TEENSY_3.6_DIL -> Gucci_ControlBoard:TEENSY_3.6
Changed lines of the file:
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@@
 </classes>
 <parts>
-<part name="U1" library="Teensy_3_and_LC_Series_Boards_v1.4" deviceset="TEENSY_3.6_DIL" device=""/>
+<part name="U1" library="Gucci_ControlBoard" deviceset="TEENSY_3.6" device=""/>
 <part name="GND2" library="SparkFun-PowerSymbols" library_urn="urn:adsk.eagle:library:530" deviceset="GND" device=""/>
 <part name="GND3" library="SparkFun-PowerSymbols" library_urn="urn:adsk.eagle:library:530" deviceset="GND" device=""/>

Commit message: Switched RX4 and TX4 pins on Gucci
Switched RX4 and TX4 on Gucci (make it consistent with the rest of the board)
Connections:
- net ESC_RX4: now also ESC1.3, U1.31/A12/RX4; no longer ESC1.2, U1.32/A13/TX4
- net ESC_TX4: now also ESC1.2, U1.32/A13/TX4; no longer ESC1.3, U1.31/A12/RX4
Changed lines of the file:
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@@
 </segment>
 </net>
-<net name="ESC_TX4" class="0">
+<net name="ESC_RX4" class="0">
 <segment>
 <pinref part="U1" gate="G$1" pin="31/A12/RX4"/>
 <wire x1="165.1" y1="157.48" x2="160.02" y2="157.48" width="0.1524" layer="91"/>
 <label x="160.02" y="157.48" size="1.778" layer="95" rot="R180" xref="yes"/>
-</segment>
-</net>
-<net name="ESC_RX4" class="0">
-<segment>
-<pinref part="U1" gate="G$1" pin="32/A13/TX4"/>
-<wire x1="165.1" y1="154.94" x2="160.02" y2="154.94" width="0.1524" layer="91"/>
-<label x="160.02" y="154.94" size="1.778" layer="95" rot="R180" xref="yes"/>
 </segment>
 </net>
@@
 <pinref part="U1" gate="G$1" pin="28"/>
 <wire x1="165.1" y1="165.1" x2="160.02" y2="165.1" width="0.1524" layer="91"/>
+</segment>
+</net>
+<net name="ESC_TX4" class="0">
+<segment>
+<pinref part="U1" gate="G$1" pin="32/A13/TX4"/>
+<wire x1="165.1" y1="154.94" x2="160.02" y2="154.94" width="0.1524" layer="91"/>
+<label x="160.02" y="154.94" size="1.778" layer="95" rot="R180" xref="yes"/>
 </segment>
 </net>
@@
 </segment>
 </net>
-<net name="ESC_TX4" class="0">
+<net name="ESC_RX4" class="0">
 <segment>
 <pinref part="ESC1" gate="G$1" pin="3"/>
@@
 </segment>
 </net>
-<net name="ESC_RX4" class="0">
+<net name="ESC_TX4" class="0">
 <segment>
 <pinref part="ESC1" gate="G$1" pin="2"/>
