File: Kirbi/v2 pcb/Kirbi_ControlBoard.brd (EAGLE design)
At the start: 66 x 56 mm, 60 parts, among them U1 PCA9306_LSSOP, U2 TEENSY_3.6_DIL, U5 LM393-8-SOIC, U6 AP2114H-1.8TRG1, U7 AP2114H-3.3TRG1

Commit message: Fixed Github versioning
Gucci:
V2 - 9/11/2019 (last push before competition)
V3 - current
Kirbi:
V1 - 9/11/2019 (last push before competition)
V2 - current
Parts:
- removed C13: 0.1uF, SparkFun-Capacitors:0603
- removed R21: 50, SparkFun-Resistors:0603
- removed U$2: (no value), RoboJackets-Aesthetics:ROBOBUZZ_1.4X
- added C10, C15, C25, C5, C9: 0.1uF, SparkFun-Capacitors:0603
- added F1: 3.5, Kirbi_ControlBoard:BEL_FUSE_C1F_3.5
- added JP1: (no value), pinhead:1X01
- added POWER_CONN: MOLEX_2.54MM_2PIN, Kirbi_ControlBoard:MOLEX_2.54MM_2PIN
- added R10, R11, R3, R5, R6, R7: 1k, SparkFun-Resistors:0603
- added R2: 6.2, Kirbi_ControlBoard:0603
- ESC: value MOLEX_1.25MM_4PIN_SMT -> MOLEX_1.25MM_3PIN_SMT; device Kirbi_ControlBoard:MOLEX_1.25MM_4PIN_SMT -> Kirbi_ControlBoard:MOLEX_1.25MM_3PIN_SMT
- R1: value 1.65k -> 100
- R19: value 1.65k -> 200
- R20: value 800 -> 100
- moved C6 13.6 mm to (-9.60, 48.0)
- moved C4 11.5 mm to (8.30, 5.90), turned to 270 degrees
- moved START 6.62 mm to (19.0, 52.5)
- moved R1 5.10 mm to (10.4, 34.0)
- moved C14 4.90 mm to (10.8, 54.0), turned to 0 degrees
- moved R24 3.45 mm to (10.8, 51.4), turned to 180 degrees
- moved R25 3.04 mm to (10.8, 48.5)
- moved C2 2.37 mm to (27.1, 19.9), turned to 0 degrees
- moved U$3 2.00 mm to (40.0, 21.0)
- moved U$4 2.00 mm to (-2.00, 21.0)
- moved TRANSCEIVER 1.80 mm to (19.0, 11.8)
- moved ESC 1.20 mm to (48.4, 38.0)
- moved LED1 0.61 mm to (18.9, 23.6)
- moved DIST_3 0.30 mm to (5.60, 2.10)
- moved DIST_4 0.30 mm to (32.5, 2.10)
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Connections:
- removed net N$10: D4.C, R21.1
- removed net S1/TX: ESC.P$5, U2.33/A14
- removed net S2: POWER.P4, U2.34/A15
- new net N$5: JP1.1, TRANSCEIVER.1P
- new net N$6: F1.P$2, POWER.P4
- new net N$7: F1.P$1, POWER_CONN.P$1
- new net N$9: D4.C, R2.1
- new net RADIO_RESET: TRANSCEIVER.14P, U2.29
- new net S1/TRX: ESC.P$2, U2.34/A15
- new net S1/TTX: ESC.P$1, U2.33/A14
- net +3.3V: now also R10.2, R11.2, R3.2, R5.2, R6.2, R7.2
- net +5V: now also C10.1, C15.1, C25.1, C5.1, C9.1; no longer C13.1
- net GND: now also C10.2, C15.2, C25.2, C5.2, C9.2, ESC.P$3, POWER_CONN.P$2, R2.2; no longer C13.2, R21.2
- net LF_INT: now also U2.15/A1; no longer U2.18/A4
- net RADIO_NSS: now also U2.30; no longer U2.6
- net RF_INT: now also U2.16/A2; no longer U2.19/A5
- net START: now also U2.14/A0; no longer U2.17/A3
- net TRX1: now also R10.1
- net TRX2: now also R11.1
- net TXD1: now also R3.1
- net TXD2: now also R5.1
- net TXD5: now also R6.1
- net TXD6: now also R7.1
Routing:
- net S2: track 70.0 -> 0.00 mm
- net RADIO_RESET: track 0.00 -> 34.9 mm, vias 0 -> 2
- net +3.3V: track 164.7 -> 198.8 mm
- net N$6: track 0.00 -> 27.8 mm, vias 0 -> 1
- net +5V: track 8.83 -> 34.3 mm
- net LINE_RF: track 57.1 -> 81.0 mm
- net MISO: track 34.6 -> 19.8 mm
- net MOSI: track 36.0 -> 22.4 mm
- net RADIO_DIO0: track 31.0 -> 17.8 mm
- net TRX2: track 30.0 -> 41.5 mm
- net TXD2: track 5.39 -> 15.3 mm, vias 0 -> 2
- net N$5: track 0.00 -> 9.16 mm
- net S1/TX: track 8.99 -> 0.00 mm
- net S1/TRX: track 0.00 -> 8.75 mm
- net RADIO_NSS: track 31.6 -> 40.1 mm
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Other:
- board text added: "Kirbi Controller Board V2.0"
- board text removed: "+"
- board text removed: "-"
- board text removed: "Kirbi Controller Board V1.0"

Commit message: Replaced Connectors
Replaced Connectors (for start module/line sensors) /re-routed and moved some resistors/capacitors
Parts:
- moved R6 6.22 mm to (39.5, 19.5), flipped to the bottom, turned to 0 degrees
- moved R7 4.97 mm to (35.3, 19.5)
- moved C18 3.51 mm to (6.30, 17.5), turned to 90 degrees
- moved C17 2.62 mm to (31.7, 16.6)
- moved R13 1.99 mm to (8.40, 17.5)
- moved R5 1.80 mm to (0.10, 12.1), flipped to the bottom, turned to 180 degrees
- moved LINE_LF 1.00 mm to (31.0, 11.0)
- moved LINE_RF 1.00 mm to (7.00, 11.0)
- moved C21 0.76 mm to (14.4, 11.2)
- moved C22 0.76 mm to (23.7, 11.2)
- moved R3 0.30 mm to (0.00, 14.0), flipped to the bottom, turned to 180 degrees
Routing:
- net +3.3V: track 198.8 -> 191.7 mm, vias 1 -> 2
- net LINE_LF: track 74.5 -> 78.6 mm
- net TXD1: track 18.1 -> 15.4 mm, vias 2 -> 1
- net TXD5: track 10.1 -> 12.5 mm
- net TXD2: track 15.3 -> 13.3 mm, vias 2 -> 1
- net RADIO_SCK: track 78.7 -> 80.2 mm
- net RADIO_RESET: track 34.9 -> 33.6 mm
- net TXD6: track 16.5 -> 17.7 mm
- net MOSI: track 22.4 -> 23.5 mm
- net LINE_RF: track 81.0 -> 81.7 mm
- net MISO: track 19.8 -> 19.2 mm
- net 1.8V: track 18.1 -> 17.5 mm
- net GND: track 82.1 -> 82.6 mm, vias 37 -> 38

Commit message: Fixed Clearances  - Changed DRC
Fixed Clearance  - Changed DRC (JLCPCB Layer 2)
Routing:
- net GND: track 82.6 -> 83.8 mm

Commit message: Cleaned up Schematic/Silkscreen
Cleaned up Schematic/Silkscreen (moved a few things around)
Changed lines of the file:
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@@
 </element>
 <element name="DIST_3" library="Kirbi_ControlBoard" package="MOLEX_1.25MM_4PIN_SMT" value="MOLEX_1.25MM_4PIN_SMT" x="5.6" y="2.1" smashed="yes">
-<attribute name="NAME" x="13.9" y="0.5" size="1.6" layer="25" font="vector" rot="R90"/>
+<attribute name="NAME" x="15.1" y="0.4" size="1.6" layer="25" font="vector" rot="R90"/>
 <attribute name="VALUE" x="1.6" y="-1.9" size="1.6" layer="27"/>
 </element>
@@
 <wire x1="46.701040625" y1="16.201040625" x2="47.6" y2="17.1" width="0.2" layer="1"/>
 <via x="47.6" y="17.1" extent="1-16" drill="0.4"/>
-<contactref element="C11" pad="2"/>
 <contactref element="C14" pad="2"/>
-<wire x1="27.8" y1="41.95" x2="28.85" y2="43" width="0.2" layer="1"/>
-<wire x1="28.85" y1="43" x2="29" y2="43" width="0.2" layer="1"/>
-<via x="29" y="43" extent="1-16" drill="0.4"/>
 <wire x1="17.5" y1="54" x2="17.73" y2="53.77" width="0.2" layer="1"/>
 <wire x1="11.65" y1="54" x2="17.5" y2="54" width="0.2" layer="1"/>
@@
 <wire x1="6.8" y1="18.85" x2="6.8" y2="20.6" width="0.2" layer="1"/>
 <via x="6.8" y="20.6" extent="1-16" drill="0.4"/>
+<contactref element="C11" pad="2"/>
+<wire x1="27.8" y1="41.95" x2="29.05" y2="43.2" width="0.2" layer="1"/>
+<wire x1="29.05" y1="43.2" x2="29.2" y2="43.2" width="0.2" layer="1"/>
+<via x="29.2" y="43.2" extent="1-16" drill="0.4"/>
 </signal>
 <signal name="+5V">

Commit message: PDB Conector/Power Switch/Resistors
Pull Up Resistor - Radio Module
Pull Down Resistors - MUXs
Power Distribution Board Connector (in Kirbi library and on schematic)
Replaced old power switch addded LED
Parts:
- removed POWER: POWER_SWITCH, Kirbi_ControlBoard:ELUMEESAQ7C12
- added D1, D5: DFLS130L-7_30V_1A, Kirbi_ControlBoard:DFLS130L-7_30V_1A
- added D6: 5V, SparkFun-LED:LED-0603
- added PDB_CONN: AMPHENOL_2X3_2.54MM, Kirbi_ControlBoard:AMPHENOL_2X3_2.54MM
- added POWER_SWITCH: GPTS202312B, Kirbi_ControlBoard:GPTS202312B
- added R12, R18, R4, R8, R9: 1k, SparkFun-Resistors:0603
- R1: value 100 -> 200
- moved R1 21.5 mm to (-5.90, 48.0)
- moved F1 13.0 mm to (-2.20, 42.1), flipped to the top
- moved R24 9.58 mm to (19.9, 48.4), turned to 0 degrees
- moved R25 9.37 mm to (19.8, 51.1), turned to 0 degrees
- moved START 9.01 mm to (28.0, 52.0)
- moved C14 9.00 mm to (19.8, 54.0), turned to 180 degrees
- moved C6 4.47 mm to (-7.60, 44.0)
- moved C1 1.04 mm to (17.0, 18.3)
- moved C3 0.42 mm to (23.3, 17.3)
Connections:
- new net PDB_!CS!: PDB_CONN.P$6
- new net PDB_!EOC!: PDB_CONN.P$2
- new net PDB_MISO: PDB_CONN.P$3, U2.5
- new net PDB_MOSI: PDB_CONN.P$4, U2.21/A7
- new net PDB_SCLK: PDB_CONN.P$5, U2.20/A6
- new net PDB_START: PDB_CONN.P$1
- net +3.3V: now also D1.P$2, D5.P$1, R4.2
- net +5V: now also D1.P$1, D6.A, POWER_SWITCH.P$2; no longer POWER.P3, POWER.P5
- net 1.8V: now also D5.P$2
- net GND: now also R12.1, R18.1, R8.1, R9.1
- net MUXS1: now also R12.2, R8.2
- net MUXS2: now also R18.2, R9.2
- net N$6: now also POWER_SWITCH.P$1; no longer POWER.P4
- net N$8: now also D6.C; no longer POWER.P1
- net NEO_DI: now also U2.6; no longer U2.24
- net RADIO_DIO0: now also U2.22/A8; no longer U2.5
- net RADIO_NSS: now also R4.1
Routing:
- net RADIO_DIO0: track 17.8 -> 0.00 mm
- net +3.3V: track 191.7 -> 209.5 mm
- net N$6: track 27.8 -> 11.1 mm, vias 1 -> 0
- net MUXS1: track 18.5 -> 26.5 mm, vias 0 -> 1
- net LF_INT: track 18.5 -> 12.6 mm
- net RF_INT: track 16.3 -> 20.3 mm
- net RADIO_NSS: track 39.6 -> 43.3 mm, vias 1 -> 2
- net NEO_DI: track 14.4 -> 11.8 mm
- net +5V: track 34.3 -> 31.8 mm, vias 2 -> 1
- net START: track 6.77 -> 8.31 mm
- net MUXS2: track 26.0 -> 27.4 mm
- net N$7: track 7.63 -> 6.45 mm, vias 0 -> 1
- net N$8: track 2.57 -> 1.97 mm
- net LINE_RF: track 81.7 -> 82.2 mm
- net GND: track 84.1 -> 84.6 mm, vias 38 -> 42

Commit message: Routed Power Distribution Board
Routed Power Distribution Board
Connections:
- net PDB_!CS!: now also U2.17/A3
- net PDB_!EOC!: now also U2.18/A4
- net PDB_START: now also U2.19/A5
Routing:
- net RADIO_DIO0: track 0.00 -> 35.5 mm, vias 0 -> 1
- net PDB_MISO: track 0.00 -> 25.1 mm
- net PDB_!EOC!: track 0.00 -> 8.55 mm
- net PDB_START: track 0.00 -> 8.55 mm
- net PDB_SCLK: track 0.00 -> 6.33 mm
- net PDB_MOSI: track 0.00 -> 6.31 mm
- net PDB_!CS!: track 0.00 -> 6.01 mm
Changed lines of the file:
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@@
 <drawing>
 <settings>
-<setting alwaysvectorfont="yes"/>
+<setting alwaysvectorfont="no"/>
 <setting verticaltext="up"/>
 </settings>
@@
 <wire x1="29.65" y1="25.65" x2="29.3" y2="25.3" width="0.2" layer="1"/>
 <via x="29.3" y="25.3" extent="1-16" drill="0.4"/>
-<wire x1="16.45" y1="21.95" x2="12.85" y2="28" width="0" layer="19" extent="16-16"/>
 </signal>
 <signal name="+5V">
@@
 <wire x1="20.971025" y1="24.871025" x2="21.35" y2="25.25" width="0.2" layer="16"/>
 <wire x1="20.971025" y1="24.871025" x2="20.971025" y2="24.85" width="0.2" layer="16"/>
-<wire x1="20.494025" y1="24.373" x2="20.971025" y2="24.85" width="0.2" layer="16"/>
-<wire x1="7.123" y1="28" x2="10.75" y2="24.373" width="0.2" layer="16"/>
-<wire x1="10.75" y1="24.373" x2="20.494025" y2="24.373" width="0.2" layer="16"/>
+<wire x1="20.194025" y1="24.073" x2="20.971025" y2="24.85" width="0.2" layer="16"/>
+<wire x1="7.123" y1="28" x2="11.05" y2="24.073" width="0.2" layer="16"/>
+<wire x1="11.05" y1="24.073" x2="20.194025" y2="24.073" width="0.2" layer="16"/>
 </signal>
 <signal name="+3.3V">
@@
 <wire x1="28.5626" y1="12.7493125" x2="22.90664375" y2="7.09335625" width="0.5" layer="1"/>
 <wire x1="22.90664375" y1="7.09335625" x2="22.8132875" y2="7" width="0.5" layer="1"/>
-<wire x1="29.2" y1="16.113953125" x2="29.2" y2="22" width="0.5" layer="1"/>
-<wire x1="29.2" y1="16" x2="29.2" y2="13.39095625" width="0.5" layer="1"/>
-<wire x1="29.2" y1="13.39095625" x2="28.5626" y2="12.75355625" width="0.5" layer="1"/>
+<wire x1="29.24644375" y1="13.4374" x2="28.5626" y2="12.75355625" width="0.5" layer="1"/>
 <wire x1="28.5626" y1="12.75355625" x2="28.5626" y2="12.7493125" width="0.5" layer="1"/>
-<wire x1="29.24644375" y1="13.4374" x2="29.2" y2="13.39095625" width="0.5" layer="1"/>
 <wire x1="32.27" y1="12.27" x2="31.1026" y2="13.4374" width="0.5" layer="1"/>
 <wire x1="31.1026" y1="13.4374" x2="29.24644375" y2="13.4374" width="0.5" layer="1"/>
@@
 <contactref element="D5" pad="P$1"/>
 <wire x1="19.2" y1="17.1" x2="20.678975" y2="17.1" width="0.2" layer="1"/>
-<wire x1="29.040953125" y1="16.273" x2="29.2" y2="16.113953125" width="0.2" layer="1"/>
-<wire x1="21.665021875" y1="16.113953125" x2="29.2" y2="16.113953125" width="0.2" layer="1"/>
-<wire x1="20.678975" y1="17.1" x2="21.665021875" y2="16.113953125" width="0.2" layer="1"/>
 <wire x1="31.25" y1="43.4" x2="30.45" y2="44.2" width="0.2" layer="1"/>
 <wire x1="30.45" y1="44.2" x2="22.25" y2="44.2" width="0.2" layer="1"/>
@@
 <wire x1="26.15" y1="5" x2="24.05664375" y2="7.09335625" width="0.2" layer="1"/>
 <wire x1="24.05664375" y1="7.09335625" x2="22.90664375" y2="7.09335625" width="0.2" layer="1"/>
-<wire x1="29.2" y1="16" x2="29.040953125" y2="16.273" width="0" layer="19" extent="1-1"/>
+<wire x1="29.2" y1="13.48384375" x2="29.24644375" y2="13.4374" width="0.5" layer="1"/>
+<wire x1="29.2" y1="22" x2="29.2" y2="17" width="0.5" layer="1"/>
+<wire x1="29.2" y1="17" x2="29.2" y2="13.48384375" width="0.5" layer="1"/>
+<wire x1="28.2" y1="16" x2="29.2" y2="17" width="0.2" layer="1"/>
+<wire x1="20.678975" y1="17.1" x2="21.778975" y2="16" width="0.2" layer="1"/>
+<wire x1="21.778975" y1="16" x2="28.2" y2="16" width="0.2" layer="1"/>
 </signal>
 <signal name="LINE_LF">
@@
 <contactref element="TRANSCEIVER" pad="6P"/>
 <contactref element="U2" pad="22/A8"/>
-<wire x1="10.9" y1="14.8" x2="0.22" y2="45.62" width="0" layer="19" extent="16-16"/>
+<wire x1="10.9" y1="14.8" x2="8" y2="17.7" width="0.2" layer="16"/>
+<wire x1="8" y1="17.7" x2="8" y2="25" width="0.2" layer="16"/>
+<via x="8" y="25" extent="1-16" drill="0.4"/>
+<wire x1="8" y1="25" x2="4" y2="29" width="0.2" layer="1"/>
+<wire x1="4" y1="29" x2="4" y2="42.3" width="0.2" layer="1"/>
+<wire x1="4" y1="42.3" x2="0.68" y2="45.62" width="0.2" layer="1"/>
+<wire x1="0.68" y1="45.62" x2="0.22" y2="45.62" width="0.2" layer="1"/>
 </signal>
 <signal name="TXD2">
@@
 <wire x1="-2.95" y1="24" x2="-2.95" y2="29.75" width="0.2" layer="1"/>
 <wire x1="-2.95" y1="29.75" x2="-2.32" y2="30.38" width="0.2" layer="1"/>
-<wire x1="-2.825" y1="24" x2="-2.95" y2="24" width="0.2" layer="1"/>
 <contactref element="R8" pad="2"/>
 <contactref element="R12" pad="2"/>
@@
 <contactref element="POWER_CONN" pad="P$1"/>
 <contactref element="F1" pad="P$1"/>
-<wire x1="1.39" y1="39.27" x2="1.22" y2="39.1" width="0.6" layer="16"/>
 <wire x1="-0.11" y1="42.1" x2="2.5968" y2="42.1" width="0.6" layer="1"/>
 <wire x1="2.5968" y1="42.1" x2="2.8" y2="41.8968" width="0.6" layer="1"/>
@@
 <contactref element="PDB_CONN" pad="P$4"/>
 <contactref element="U2" pad="21/A7"/>
-<wire x1="2.76" y1="45.62" x2="5.66" y2="50.73" width="0" layer="19" extent="1-1"/>
+<wire x1="5.66" y1="50.73" x2="5.66" y2="48.52" width="0.2" layer="1"/>
+<wire x1="5.66" y1="48.52" x2="2.76" y2="45.62" width="0.2" layer="1"/>
 </signal>
 <signal name="PDB_SCLK">
 <contactref element="PDB_CONN" pad="P$5"/>
 <contactref element="U2" pad="20/A6"/>
-<wire x1="5.3" y1="45.62" x2="8.2" y2="50.73" width="0" layer="19" extent="1-1"/>
+<wire x1="8.2" y1="50.73" x2="8.2" y2="49.48955" width="0.2" layer="1"/>
+<wire x1="8.2" y1="49.48955" x2="5.273" y2="46.56255" width="0.2" layer="1"/>
+<wire x1="5.3" y1="46.466" x2="5.273" y2="46.493" width="0.2" layer="1"/>
+<wire x1="5.3" y1="46.466" x2="5.3" y2="45.62" width="0.2" layer="1"/>
+<wire x1="5.273" y1="46.56255" x2="5.273" y2="46.493" width="0.2" layer="1"/>
 </signal>
 <signal name="PDB_!CS!">
 <contactref element="PDB_CONN" pad="P$6"/>
+<contactref element="U2" pad="17/A3"/>
+<wire x1="10.74" y1="50.73" x2="12.92" y2="48.55" width="0.2" layer="16"/>
+<wire x1="12.92" y1="48.55" x2="12.92" y2="45.62" width="0.2" layer="16"/>
 </signal>
 <signal name="PDB_START">
 <contactref element="PDB_CONN" pad="P$1"/>
+<contactref element="U2" pad="19/A5"/>
+<wire x1="5.66" y1="53.27" x2="7" y2="51.93" width="0.2" layer="16"/>
+<wire x1="7" y1="46.46" x2="7.84" y2="45.62" width="0.2" layer="16"/>
+<wire x1="7" y1="51.93" x2="7" y2="46.46" width="0.2" layer="16"/>
 </signal>
 <signal name="PDB_!EOC!">
 <contactref element="PDB_CONN" pad="P$2"/>
+<contactref element="U2" pad="18/A4"/>
+<wire x1="9.548" y1="51.622" x2="8.2" y2="52.97" width="0.2" layer="16"/>
+<wire x1="8.2" y1="53.27" x2="8.2" y2="52.97" width="0.2" layer="16"/>
+<wire x1="9.548" y1="51.622" x2="9.548" y2="46.452" width="0.2" layer="16"/>
+<wire x1="9.548" y1="46.452" x2="10.38" y2="45.62" width="0.2" layer="16"/>
 </signal>
 <signal name="PDB_MISO">
 <contactref element="PDB_CONN" pad="P$3"/>
 <contactref element="U2" pad="5"/>
-<wire x1="5.3" y1="30.38" x2="10.74" y2="53.27" width="0" layer="19" extent="1-1"/>
+<wire x1="10.74" y1="53.27" x2="10.74" y2="52.74" width="0.2" layer="1"/>
+<wire x1="6.6" y1="31.68" x2="5.3" y2="30.38" width="0.2" layer="1"/>
+<wire x1="9.492" y1="51.492" x2="9.492" y2="49.7191" width="0.2" layer="1"/>
+<wire x1="9.492" y1="49.7191" x2="6.6" y2="46.8271" width="0.2" layer="1"/>
+<wire x1="6.6" y1="46.8271" x2="6.6" y2="31.68" width="0.2" layer="1"/>
+<wire x1="10.74" y1="52.74" x2="9.492" y2="51.492" width="0.2" layer="1"/>
 </signal>
 </signals>

Commit message: Screw Head Clearance/Silkscreen
Screw Head Clearance/Silkscreen cleaned up
Parts:
- moved R6 1.10 mm to (39.5, 18.4)
- moved R7 1.10 mm to (35.3, 18.4)
- moved R18 0.50 mm to (30.5, 26.2)
- moved R9 0.50 mm to (34.3, 26.2)
- renumbered D6 to 5V
Routing:
- net TRX1: track 22.9 -> 24.0 mm
- net MUXS2: track 27.4 -> 28.3 mm
- net TXD6: track 17.8 -> 17.2 mm

Commit message: Renamed Parts/Routed SPI Interface
Renamed Parts (U1-U7)
Routed SPI Interface (Connectted MISO, MOSI, and SCK) (Fixed routing to avoid islands/breaks in ground plane)
Parts:
- removed IMU: ICM-20948, ICM-20948:QFN40P300X300X105-25N
- added U3: PCA9306_LSSOP, Gucci_ControlBoard:8-LSSOP
- U1: value PCA9306_LSSOP -> TEENSY_3.6_DIL; device Gucci_ControlBoard:8-LSSOP -> Teensy_3_and_LC_Series_Boards_v1.4:TEENSY_3.6_DIL
- U2: value TEENSY_3.6_DIL -> ICM-20948; device Teensy_3_and_LC_Series_Boards_v1.4:TEENSY_3.6_DIL -> ICM-20948:QFN40P300X300X105-25N
- moved U1 19.9 mm to (18.0, 38.0), turned to 90 degrees
- moved U2 17.7 mm to (23.0, 21.0), turned to 0 degrees
- renumbered TRANSCEIVER to U4
Connections:
- removed net PDB_MISO: PDB_CONN.P$3, U2.5
- removed net PDB_MOSI: PDB_CONN.P$4, U2.21/A7
- removed net PDB_SCLK: PDB_CONN.P$5, U2.20/A6
- removed net RADIO_SCK: U2.13, U4.12P
- new net SCK: PDB_CONN.P$3, U1.13, U4.12P
- net +5V: now also U1.VIN; no longer U2.VIN
- net 1.8V: now also U2.13, U2.22, U2.8, U3.P$2; no longer IMU.13, IMU.22, IMU.8, U1.P$2
- net GND: now also U1.AGND, U1.GND, U1.GND1, U2.11, U2.18, U2.20, U2.9, U3.P$1; no longer IMU.11, IMU.18, IMU.20, IMU.9, U1.P$1, U2.AGND, U2.GND, U2.GND1
- net LF_INT: now also U1.15/A1; no longer U2.15/A1
- net LINE_LF: now also U1.35/A16; no longer U2.35/A16
- net LINE_REF: now also U1.A22; no longer U2.A22
- net LINE_RF: now also U1.23/A9; no longer U2.23/A9
- net MISO: now also PDB_CONN.P$5, U1.12; no longer U2.12
- net MOSI: now also PDB_CONN.P$4, U1.11; no longer U2.11
- net MUXS1: now also U1.2; no longer U2.2
- net MUXS2: now also U1.25; no longer U2.25
- net N$3: now also U2.10; no longer IMU.10
- net N$4: now also U3.P$7, U3.P$8; no longer U1.P$7, U1.P$8
- net NEO_DI: now also U1.6; no longer U2.6
- net PDB_!CS!: now also U1.17/A3; no longer U2.17/A3
- net PDB_!EOC!: now also U1.18/A4; no longer U2.18/A4
- net PDB_START: now also U1.19/A5; no longer U2.19/A5
- net RADIO_DIO0: now also U1.22/A8; no longer U2.22/A8
- net RADIO_NSS: now also U1.30; no longer U2.30
- net RADIO_RESET: now also U1.29; no longer U2.29
- net RF_INT: now also U1.16/A2; no longer U2.16/A2
- net RXD3: now also U1.0; no longer U2.0
- net RXD4: now also U1.31/A12; no longer U2.31/A12
- net S1/TRX: now also U1.34/A15; no longer U2.34/A15
- net S1/TTX: now also U1.33/A14; no longer U2.33/A14
- net SCL1: now also U2.23, U3.P$3; no longer IMU.23, U1.P$3
- net SCL2: now also U1.3, U3.P$6; no longer U1.P$6, U2.3
- net SDA1: now also U2.24, U3.P$4; no longer IMU.24, U1.P$4
- net SDA2: now also U1.4, U3.P$5; no longer U1.P$5, U2.4
- net START: now also U1.14/A0; no longer U2.14/A0
- net TRX1: now also U1.7; no longer U2.7
- net TRX2: now also U1.9; no longer U2.9
- net TTX1: now also U1.8; no longer U2.8
- net TTX2: now also U1.10; no longer U2.10
- net TXD3: now also U1.1; no longer U2.1
- net TXD4: now also U1.32/A13; no longer U2.32/A13
Routing:
- net SCK: track 0.00 -> 101.2 mm
- net RADIO_SCK: track 80.2 -> 0.00 mm
- net MISO: track 19.2 -> 53.2 mm, vias 1 -> 3
- net MOSI: track 23.5 -> 57.0 mm, vias 1 -> 3
- net PDB_MISO: track 25.1 -> 0.00 mm
- net PDB_SCLK: track 6.33 -> 0.00 mm
- net PDB_MOSI: track 6.31 -> 0.00 mm
- net RF_INT: track 20.3 -> 19.5 mm
- net GND: track 85.0 -> 84.4 mm
- net TTX1: track 25.1 -> 25.7 mm
- net LINE_RF: track 82.2 -> 82.0 mm, vias 1 -> 3
- net NEO_DI: track 11.8 -> 11.6 mm, vias 0 -> 1
