File: Kirbi/v2 pcb/Kirbi_ControlBoard.brd (EAGLE design)
At the start: 66 x 56 mm, 81 parts, among them U1 TEENSY_3.6_DIL, U2 ICM-20948, U3 PCA9306_LSSOP, U5 LM393-8-SOIC, U6 AP2114H-1.8TRG1, U7 AP2114H-3.3TRG1

Commit message: mounting holes clearance
Parts:
- moved R18 0.81 mm to (30.6, 27.0)
- moved R9 0.80 mm to (34.3, 27.0)

Commit message: Started Implementing 4 Layers
Started Implementing 4 Layers: Adding vias
Parts:
- moved C7 0.90 mm to (25.9, 33.8)
Routing:
- net +5V: track 32.0 -> 61.4 mm, vias 1 -> 13
- net GND: track 84.2 -> 99.1 mm, vias 42 -> 48
- added copper zone on layer 15, net +5V
- added copper zone on layer 2, net GND
- removed copper zone on layer 1, net +5V
- removed copper zone on layer 16, net GND

Commit message: Re-routed for 4-layers/Changed 5V plane
Re-routed for 4-layers/Changed 5V plane (whole board - 3rd layer)
Routing:
- net GND: track 99.1 -> 112.7 mm, vias 48 -> 52
- net +5V: track 61.4 -> 69.1 mm, vias 13 -> 18
Changed lines of the file:
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@@
 <drawing>
 <settings>
-<setting alwaysvectorfont="yes"/>
+<setting alwaysvectorfont="no"/>
 <setting verticaltext="up"/>
 </settings>
@@
 <wire x1="27.1" y1="4.8" x2="29.2" y2="4.8" width="0.2" layer="16"/>
 <wire x1="29.2" y1="4.8" x2="30.8" y2="3.2" width="0.2" layer="16"/>
-<wire x1="8.3" y1="5.05" x2="8.3" y2="3.3" width="0.2" layer="16"/>
-<wire x1="8.3" y1="3.3" x2="8" y2="3" width="0.2" layer="16"/>
-<via x="8" y="3" extent="1-16" drill="0.4"/>
+<wire x1="8.3" y1="5.05" x2="8.3" y2="4.5" width="0.2" layer="16"/>
+<wire x1="8.3" y1="4.5" x2="7.7" y2="3.9" width="0.2" layer="16"/>
+<wire x1="7.7" y1="3.9" x2="7.7" y2="2.3" width="0.2" layer="16"/>
+<via x="7.7" y="2.3" extent="1-16" drill="0.4"/>
 <wire x1="12.85" y1="28" x2="13.8" y2="27.05" width="0.2" layer="16"/>
 <wire x1="13.8" y1="27.05" x2="13.8" y2="26.3" width="0.2" layer="16"/>
@@
 <wire x1="31.6698" y1="28" x2="32.3" y2="28.6302" width="0.2" layer="16"/>
 <via x="32.3" y="28.6302" extent="1-16" drill="0.4"/>
-<wire x1="27.95" y1="19.9" x2="27.1" y2="18.8" width="0" layer="19" extent="1-16"/>
-<wire x1="10.9" y1="6.8" x2="10.85" y2="5.1" width="0" layer="19" extent="1-16"/>
-<wire x1="-2" y1="22.15" x2="-4.4" y2="23.65" width="0" layer="19" extent="1-16"/>
-<wire x1="16.45" y1="21.95" x2="17" y2="17.45" width="0" layer="19" extent="1-16"/>
+<wire x1="10.9" y1="6.8" x2="12.9" y2="6.8" width="0.2" layer="16"/>
+<wire x1="12.9" y1="6.8" x2="14.1" y2="5.6" width="0.2" layer="16"/>
+<via x="14.1" y="5.6" extent="1-16" drill="0.4"/>
+<wire x1="-2" y1="22.15" x2="-4.75" y2="22.15" width="0.2" layer="16"/>
+<wire x1="-4.75" y1="22.15" x2="-6.6" y2="24" width="0.2" layer="16"/>
+<via x="-6.6" y="24" extent="1-16" drill="0.4"/>
+<wire x1="27.1" y1="18.8" x2="25.7" y2="18.8" width="0.2" layer="16"/>
+<wire x1="25.7" y1="18.8" x2="25.5" y2="18.6" width="0.2" layer="16"/>
+<via x="25.5" y="18.6" extent="1-16" drill="0.4"/>
+<wire x1="16.45" y1="21.95" x2="15.0698" y2="20.5698" width="0.2" layer="16"/>
+<wire x1="15.0698" y1="20.5698" x2="15" y2="20.5698" width="0.2" layer="16"/>
+<via x="15" y="20.5698" extent="1-16" drill="0.4"/>
 </signal>
 <signal name="+5V">
@@
 <contactref element="U7" pad="3"/>
 <contactref element="C24" pad="1"/>
-<polygon width="0.2" layer="15" isolate="0.1524" orphans="yes" thermals="no">
-<vertex x="-14" y="56"/>
-<vertex x="-14" y="28"/>
-<vertex x="52" y="28"/>
-<vertex x="52" y="56"/>
-</polygon>
-<polygon width="0.2" layer="15" isolate="0.1524" thermals="no">
-<vertex x="-14" y="28"/>
-<vertex x="-14" y="14"/>
-<vertex x="0" y="0"/>
-<vertex x="12" y="0"/>
-<vertex x="12" y="6"/>
-<vertex x="4" y="6"/>
-<vertex x="-5" y="15"/>
-<vertex x="-5" y="28"/>
-</polygon>
-<polygon width="0.2" layer="15" isolate="0.1524" thermals="no">
-<vertex x="52" y="28"/>
-<vertex x="52" y="14"/>
-<vertex x="38" y="0"/>
-<vertex x="26" y="0"/>
-<vertex x="26" y="6"/>
-<vertex x="34" y="6"/>
-<vertex x="43" y="15"/>
-<vertex x="43" y="28"/>
-</polygon>
 <contactref element="C8" pad="1"/>
 <contactref element="C7" pad="1"/>
@@
 <wire x1="34.375" y1="3.087" x2="34.462" y2="3" width="0.2" layer="1"/>
 <via x="34.462" y="3" extent="1-16" drill="0.4"/>
-<wire x1="-9.1" y1="20.125" x2="-8.6" y2="19.625" width="0.2" layer="1"/>
-<wire x1="-8.6" y1="19.625" x2="-8.6" y2="17.85" width="0.2" layer="1"/>
 <wire x1="-9.1" y1="20.125" x2="-10.525" y2="20.125" width="0.2" layer="1"/>
 <wire x1="-10.525" y1="20.125" x2="-10.6" y2="20.2" width="0.2" layer="1"/>
@@
 <wire x1="22.75" y1="25.25" x2="23" y2="25" width="0.2" layer="16"/>
 <via x="23" y="25" extent="1-16" drill="0.4"/>
-<wire x1="25.9" y1="32.95" x2="26.288" y2="32.95" width="0.2" layer="1"/>
-<wire x1="26.288" y1="32.95" x2="27.238" y2="33.9" width="0.2" layer="1"/>
 <via x="27.238" y="33.9" extent="1-16" drill="0.4"/>
 <wire x1="25.9" y1="39.25" x2="29.9802" y2="39.25" width="0.2" layer="1"/>
@@
 <wire x1="15.4" y1="41.6287625" x2="16.23561875" y2="42.46438125" width="0.2" layer="1"/>
 <via x="16.23561875" y="42.46438125" extent="1-16" drill="0.4"/>
-<wire x1="25.9" y1="32.95" x2="23" y2="25" width="0" layer="19" extent="1-1"/>
-<wire x1="-3.6340125" y1="10.771853125" x2="-8.6" y2="17.85" width="0" layer="19" extent="1-1"/>
-<wire x1="-1.701040625" y1="9.601040625" x2="-3.6340125" y2="10.771853125" width="0" layer="19" extent="1-1"/>
-<wire x1="7.475" y1="5" x2="-1.701040625" y2="9.601040625" width="0" layer="19" extent="1-1"/>
-<wire x1="9.15" y1="5.1" x2="7.475" y2="5" width="0" layer="19" extent="1-1"/>
+<wire x1="25.9" y1="32.95" x2="26.85" y2="33.9" width="0.2" layer="1"/>
+<wire x1="26.85" y1="33.9" x2="27.238" y2="33.9" width="0.2" layer="1"/>
+<wire x1="7.475" y1="5" x2="7.475" y2="3.81831875" width="0.2" layer="1"/>
+<wire x1="7.475" y1="3.81831875" x2="7.0552" y2="3.39851875" width="0.2" layer="1"/>
+<via x="7.0552" y="3.39851875" extent="1-16" drill="0.4"/>
+<wire x1="9.15" y1="5.1" x2="8.394" y2="4.344" width="0.2" layer="1"/>
+<wire x1="8.394" y1="4.344" x2="8.394" y2="3.4" width="0.2" layer="1"/>
+<via x="8.394" y="3.4" extent="1-16" drill="0.4"/>
+<wire x1="-3.6340125" y1="10.771853125" x2="-4.405865625" y2="10" width="0.2" layer="1"/>
+<wire x1="-4.405865625" y1="10" x2="-5" y2="10" width="0.2" layer="1"/>
+<via x="-5" y="10" extent="1-16" drill="0.4"/>
+<wire x1="-1.701040625" y1="9.601040625" x2="-2.26450625" y2="9.037575" width="0.2" layer="1"/>
+<wire x1="-2.26450625" y1="9.037575" x2="-4.0386375" y2="9.037575" width="0.2" layer="1"/>
+<via x="-4.0386375" y="9.037575" extent="1-16" drill="0.4"/>
+<wire x1="-8.6" y1="17.85" x2="-6.55" y2="17.85" width="0.2" layer="1"/>
+<wire x1="-6.55" y1="17.85" x2="-6.5" y2="17.9" width="0.2" layer="1"/>
+<via x="-6.5" y="17.9" extent="1-16" drill="0.4"/>
+<polygon width="0.2" layer="15">
+<vertex x="-14" y="56"/>
+<vertex x="52" y="56"/>
+<vertex x="52" y="14"/>
+<vertex x="38" y="0"/>
+<vertex x="0" y="0"/>
+<vertex x="-14" y="14"/>
+</polygon>
 </signal>
 <signal name="+3.3V">

Commit message: Finished 4-layer routing on Gucci
Finished 4-layer routing on Gucci (changed layer names)
Routing:
- net +5V: track 69.1 -> 70.5 mm, vias 18 -> 21
Changed lines of the file:
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@@
 <layers>
 <layer number="1" name="Top" color="4" fill="1" visible="yes" active="yes"/>
-<layer number="2" name="Inner1" color="16" fill="1" visible="yes" active="yes"/>
+<layer number="2" name="GND" color="39" fill="1" visible="yes" active="yes"/>
 <layer number="3" name="Route3" color="17" fill="1" visible="no" active="no"/>
 <layer number="4" name="Route4" color="18" fill="1" visible="no" active="no"/>
@@
 <layer number="13" name="Route13" color="21" fill="1" visible="no" active="no"/>
 <layer number="14" name="Route14" color="22" fill="1" visible="no" active="no"/>
-<layer number="15" name="Inner2" color="23" fill="1" visible="yes" active="yes"/>
+<layer number="15" name="5V" color="40" fill="1" visible="yes" active="yes"/>
 <layer number="16" name="Bottom" color="1" fill="1" visible="yes" active="yes"/>
 <layer number="17" name="Pads" color="2" fill="1" visible="yes" active="yes"/>
@@
 <wire x1="7.123" y1="28" x2="11.05" y2="24.073" width="0.2" layer="16"/>
 <wire x1="11.05" y1="24.073" x2="20.194025" y2="24.073" width="0.2" layer="16"/>
-<wire x1="47.1" y1="23.875" x2="47.225" y2="24" width="0.2" layer="1"/>
-<wire x1="47.225" y1="24" x2="49" y2="24" width="0.2" layer="1"/>
-<via x="49" y="24" extent="1-16" drill="0.4"/>
+<wire x1="47.1" y1="23.875" x2="47.375" y2="23.6" width="0.2" layer="1"/>
+<wire x1="49" y1="23.6" x2="47.375" y2="23.6" width="0.2" layer="1"/>
+<via x="49" y="23.6" extent="1-16" drill="0.4"/>
 <wire x1="-6.75" y1="44" x2="-6.75" y2="42.45" width="0.2" layer="1"/>
 <wire x1="-6.75" y1="42.45" x2="-6.6" y2="42.3" width="0.2" layer="1"/>
@@
 <wire x1="-10.477" y1="48" x2="-9.94" y2="47.463" width="0.2" layer="1"/>
 <wire x1="-9.94" y1="47.463" x2="-9.94" y2="45.62" width="0.2" layer="1"/>
-<wire x1="44.352003125" y1="13.39200625" x2="44.37200625" y2="13.372003125" width="0.2" layer="1"/>
-<wire x1="44.37200625" y1="13.372003125" x2="45.344009375" y2="12.4" width="0.2" layer="1"/>
-<wire x1="45.344009375" y1="12.4" x2="45.6" y2="12.4" width="0.2" layer="1"/>
-<via x="45.6" y="12.4" extent="1-16" drill="0.4"/>
-<wire x1="45.39895625" y1="14.99895625" x2="45.39895625" y2="14.398953125" width="0.2" layer="1"/>
-<wire x1="45.39895625" y1="14.398953125" x2="44.37200625" y2="13.372003125" width="0.2" layer="1"/>
-<wire x1="46.99258125" y1="25.45003125" x2="46.99258125" y2="23.98241875" width="0.2" layer="1"/>
-<wire x1="46.99258125" y1="23.98241875" x2="47.1" y2="23.875" width="0.2" layer="1"/>
-<wire x1="36.15" y1="5.1" x2="36.05" y2="5" width="0.2" layer="1"/>
-<wire x1="36.05" y1="5" x2="34.375" y2="5" width="0.2" layer="1"/>
-<wire x1="34.375" y1="5" x2="34.375" y2="3.087" width="0.2" layer="1"/>
-<wire x1="34.375" y1="3.087" x2="34.462" y2="3" width="0.2" layer="1"/>
-<via x="34.462" y="3" extent="1-16" drill="0.4"/>
+<wire x1="44.352003125" y1="13.39200625" x2="45.30000625" y2="12.444003125" width="0.2" layer="1"/>
+<wire x1="45.30000625" y1="12.444003125" x2="45.3" y2="12" width="0.2" layer="1"/>
+<via x="45.3" y="12" extent="1-16" drill="0.4"/>
+<wire x1="34.375" y1="5" x2="34.375" y2="2.9" width="0.2" layer="1"/>
+<wire x1="34.375" y1="2.9" x2="34.362" y2="2.9" width="0.2" layer="1"/>
+<via x="34.362" y="2.9" extent="1-16" drill="0.4"/>
 <wire x1="-9.1" y1="20.125" x2="-10.525" y2="20.125" width="0.2" layer="1"/>
 <wire x1="-10.525" y1="20.125" x2="-10.6" y2="20.2" width="0.2" layer="1"/>
@@
 <vertex x="-14" y="14"/>
 </polygon>
+<via x="35.294" y="3.5" extent="1-16" drill="0.4"/>
+<wire x1="35.294" y1="4.244" x2="35.294" y2="3.5" width="0.2" layer="1"/>
+<wire x1="46.14203125" y1="12.849040625" x2="45.39895625" y2="13.592115625" width="0.2" layer="1"/>
+<via x="46.14203125" y="12.849040625" extent="1-16" drill="0.4"/>
+<wire x1="46.99258125" y1="25.45003125" x2="47.6486125" y2="24.794" width="0.2" layer="1"/>
+<wire x1="47.6486125" y1="24.794" x2="49" y2="24.794" width="0.2" layer="1"/>
+<via x="49" y="24.794" extent="1-16" drill="0.4"/>
+<wire x1="45.39895625" y1="13.592115625" x2="45.39895625" y2="14.99895625" width="0.2" layer="1"/>
+<wire x1="35.294" y1="4.244" x2="36.15" y2="5.1" width="0.2" layer="1"/>
 </signal>
 <signal name="+3.3V">
@@
 <contactref element="DIST_4" pad="P$4"/>
 <contactref element="U1" pad="31/A12"/>
-<via x="33.3" y="3" extent="1-16" drill="0.4"/>
-<wire x1="33.3" y1="3" x2="46.34" y2="15.83366875" width="0.2" layer="16"/>
+<via x="33.1" y="2.9" extent="1-16" drill="0.4"/>
+<wire x1="33.1" y1="2.9" x2="46.34" y2="15.930503125" width="0.2" layer="16"/>
 <wire x1="46.34" y1="29.98" x2="45.94" y2="30.38" width="0.2" layer="16"/>
-<wire x1="46.34" y1="29.98" x2="46.34" y2="15.83366875" width="0.2" layer="16"/>
-<wire x1="33.125" y1="3.175" x2="33.3" y2="3" width="0.2" layer="1"/>
-<wire x1="33.125" y1="5" x2="33.125" y2="3.175" width="0.2" layer="1"/>
+<wire x1="46.34" y1="29.98" x2="46.34" y2="15.930503125" width="0.2" layer="16"/>
+<wire x1="33.125" y1="2.925" x2="33.1" y2="2.9" width="0.2" layer="1"/>
+<wire x1="33.125" y1="5" x2="33.125" y2="2.925" width="0.2" layer="1"/>
 </signal>
 <signal name="N$5">

Commit message: Moved Power Connector out/Capacitors
Moved Power Connector out/Moved Capacitors
Parts:
- moved C8 34.0 mm to (-8.10, 39.7)
- moved C7 32.5 mm to (-6.10, 39.7), turned to 270 degrees
- moved C11 5.53 mm to (28.4, 35.6), turned to 270 degrees
- moved D1 3.04 mm to (29.5, 42.0)
- moved POWER_CONN 2.30 mm to (-11.6, 38.0)
- moved C24 2.10 mm to (25.9, 35.6)
- moved F1 1.56 mm to (-1.00, 43.1)
- moved C6 0.58 mm to (-7.10, 43.7)
Routing:
- net +5V: track 70.5 -> 45.5 mm, vias 21 -> 22
- net GND: track 112.7 -> 108.2 mm
- net MISO: track 53.2 -> 48.8 mm, vias 3 -> 2
- net MOSI: track 57.0 -> 52.8 mm, vias 3 -> 2
- net LINE_RF: track 82.0 -> 79.6 mm, vias 3 -> 1
- net +3.3V: track 210.5 -> 208.9 mm
- net N$7: track 6.21 -> 4.66 mm
- net N$6: track 11.1 -> 9.96 mm

Commit message: Moved/Re-routed Some Parts
Moved/Re-routed Some Parts (Moved components away from the Teensy pins)
Parts:
- moved C20 2.21 mm to (9.30, 42.3), turned to 180 degrees
- moved R10 1.55 mm to (10.0, 33.7)
- moved F1 1.46 mm to (-0.60, 41.7), turned to 0 degrees
- moved C8 1.41 mm to (-8.30, 38.3)
- moved C6 1.41 mm to (-7.30, 42.3)
- moved C7 1.41 mm to (-6.30, 38.3)
- moved C19 1.06 mm to (13.2, 42.3), turned to 180 degrees
- moved R11 0.58 mm to (15.5, 33.7)
Routing:
- net N$6: track 9.96 -> 12.6 mm
- net N$7: track 4.66 -> 6.90 mm
- net GND: track 108.2 -> 106.3 mm
- net TRX1: track 24.3 -> 26.0 mm
- net LINE_RF: track 79.6 -> 81.0 mm
- net +3.3V: track 208.9 -> 209.9 mm
- net RF_INT: track 19.5 -> 20.3 mm
- net TRX2: track 41.7 -> 41.2 mm

Commit message: Replaced parts on Kirbi control board
Replaced parts on Kirbi control board/made slight changes to Gucci library
Parts:
- D1, D5: value DFLS130L-7_30V_1A -> 30; device Kirbi_ControlBoard:DFLS130L-7_30V_1A -> Kirbi_ControlBoard:DFLS130L-7
- DIST_1, DIST_2, DIST_3, DIST_4, DIST_5, DIST_6: value MOLEX_1.25MM_4PIN_SMT -> 0532610471; device Kirbi_ControlBoard:MOLEX_1.25MM_4PIN_SMT -> Kirbi_ControlBoard:0532610471
- ESC: value MOLEX_1.25MM_3PIN_SMT -> 0532610371; device Kirbi_ControlBoard:MOLEX_1.25MM_3PIN_SMT -> Kirbi_ControlBoard:0532610371
- F1: device Kirbi_ControlBoard:BEL_FUSE_C1F_3.5 -> Kirbi_ControlBoard:C1F
- LINE_LF, LINE_RF, START: value AMPHENOL_2X02_2.54MM_SHROUD -> 75869-130LF; device Gucci_ControlBoard:AMPHENOL_2X02_2.54MM_SHROUD -> Gucci_ControlBoard:75869-130LF
- MUX_RX1, MUX_RX2, MUX_TX1, MUX_TX2: value MUX_74LVC1G157GV -> 74LVC1G157GW,125; device Kirbi_ControlBoard:MUX_74LVC1G157GV -> Kirbi_ControlBoard:TSSOP6
- PDB_CONN: value AMPHENOL_2X3_2.54MM -> 71600-006LF
- POWER_CONN: value MOLEX_2.54MM_2PIN -> 1719770002; device Kirbi_ControlBoard:MOLEX_2.54MM_2PIN -> Kirbi_ControlBoard:1719770002
- U1: value TEENSY_3.6_DIL -> DEV-14057; device Teensy_3_and_LC_Series_Boards_v1.4:TEENSY_3.6_DIL -> Kirbi_ControlBoard:TEENSY_3.6_DIL
- U2: device ICM-20948:QFN40P300X300X105-25N -> Gucci_ControlBoard:24-QFN_(3X3)
- U3: value PCA9306_LSSOP -> PCA9306
- U4: value (none) -> RFM69HCW_SMT
- U5: value LM393-8-SOIC -> LM393ADR
- moved U5 0.20 mm to (12.5, 38.3)
Connections:
- net +3.3V: now also D1.2, D5.1, MUX_RX1.5, MUX_RX2.5, MUX_TX1.5, MUX_TX2.5; no longer D1.P$2, D5.P$1, MUX_RX1.P$5, MUX_RX2.P$5, MUX_TX1.P$5, MUX_TX2.P$5
- net +5V: now also D1.1, DIST_1.6, DIST_2.6, DIST_3.6, DIST_4.6, DIST_5.6, DIST_6.6, POWER_SWITCH.P, U5.8; no longer D1.P$1, DIST_1.P$6, DIST_2.P$6, DIST_3.P$6, DIST_4.P$6, DIST_5.P$6, DIST_6.P$6, POWER_SWITCH.P$2, U5.P$8
- net 1.8V: now also D5.2, U3.2; no longer D5.P$2, U3.P$2
- net GND: now also DIST_1.3, DIST_2.3, DIST_3.3, DIST_4.3, DIST_5.3, DIST_6.3, ESC.3, MUX_RX1.2, MUX_RX2.2, MUX_TX1.2, MUX_TX2.2, POWER_CONN.1, U3.1, U5.4; no longer DIST_1.P$3, DIST_2.P$3, DIST_3.P$3, DIST_4.P$3, DIST_5.P$3, DIST_6.P$3, ESC.P$3, MUX_RX1.P$2, MUX_RX2.P$2, MUX_TX1.P$2, MUX_TX2.P$2, POWER_CONN.P$2, U3.P$1, U5.P$4
- net LF_INT: now also U5.7; no longer U5.P$7
- net LINE_LF: now also U5.5; no longer U5.P$5
- net LINE_REF: now also U5.2, U5.6; no longer U5.P$2, U5.P$6
- net LINE_RF: now also U5.3; no longer U5.P$3
- net MISO: now also PDB_CONN.5; no longer PDB_CONN.P$5
- net MOSI: now also PDB_CONN.4; no longer PDB_CONN.P$4
- net MUXS1: now also MUX_RX1.6, MUX_TX1.6; no longer MUX_RX1.P$6, MUX_TX1.P$6
- net MUXS2: now also MUX_RX2.6, MUX_TX2.6; no longer MUX_RX2.P$6, MUX_TX2.P$6
- net N$4: now also U3.7, U3.8; no longer U3.P$7, U3.P$8
- net N$6: now also F1.2, POWER_SWITCH.1; no longer F1.P$2, POWER_SWITCH.P$1
- net N$7: now also F1.1, POWER_CONN.2; no longer F1.P$1, POWER_CONN.P$1
- net PDB_!CS!: now also PDB_CONN.6; no longer PDB_CONN.P$6
- net PDB_!EOC!: now also PDB_CONN.2; no longer PDB_CONN.P$2
- net PDB_START: now also PDB_CONN.1; no longer PDB_CONN.P$1
- net RF_INT: now also U5.1; no longer U5.P$1
- net RXD1: now also DIST_1.4, MUX_RX1.3; no longer DIST_1.P$4, MUX_RX1.P$3
- net RXD2: now also DIST_2.4, MUX_RX1.1; no longer DIST_2.P$4, MUX_RX1.P$1
- net RXD3: now also DIST_3.4; no longer DIST_3.P$4
- net RXD4: now also DIST_4.4; no longer DIST_4.P$4
- net RXD5: now also DIST_5.4, MUX_RX2.3; no longer DIST_5.P$4, MUX_RX2.P$3
- net RXD6: now also DIST_6.4, MUX_RX2.1; no longer DIST_6.P$4, MUX_RX2.P$1
- net S1/TRX: now also ESC.2; no longer ESC.P$2
- net S1/TTX: now also ESC.1; no longer ESC.P$1
- net SCK: now also PDB_CONN.3; no longer PDB_CONN.P$3
- net SCL1: now also U3.3; no longer U3.P$3
- net SCL2: now also U3.6; no longer U3.P$6
- net SDA1: now also U3.4; no longer U3.P$4
- net SDA2: now also U3.5; no longer U3.P$5
- net TRX1: now also MUX_RX1.4; no longer MUX_RX1.P$4
- net TRX2: now also MUX_RX2.4; no longer MUX_RX2.P$4
- net TTX1: now also MUX_TX1.4; no longer MUX_TX1.P$4
- net TTX2: now also MUX_TX2.4; no longer MUX_TX2.P$4
- net TXD1: now also DIST_1.5, MUX_TX1.3; no longer DIST_1.P$5, MUX_TX1.P$3
- net TXD2: now also DIST_2.5, MUX_TX1.1; no longer DIST_2.P$5, MUX_TX1.P$1
- net TXD3: now also DIST_3.5; no longer DIST_3.P$5
- net TXD4: now also DIST_4.5; no longer DIST_4.P$5
- net TXD5: now also DIST_5.5, MUX_TX2.3; no longer DIST_5.P$5, MUX_TX2.P$3
- net TXD6: now also DIST_6.5, MUX_TX2.1; no longer DIST_6.P$5, MUX_TX2.P$1
Routing:
- net TXD1: track 15.4 -> 17.0 mm, vias 1 -> 2
- net +3.3V: track 209.9 -> 209.0 mm
- net GND: track 106.3 -> 107.0 mm
- net SCL2: track 21.8 -> 21.1 mm
- net MUXS2: track 28.2 -> 28.8 mm
- net TXD6: track 17.2 -> 17.7 mm
- net MUXS1: track 26.6 -> 27.1 mm
