File: Kirbi/v2 pcb/Kirbi_ControlBoard.brd (EAGLE design)
At the start: 66 x 56 mm, 81 parts, among them U1 DEV-14057, U2 ICM-20948, U3 PCA9306, U4 RFM69HCW_SMT, U5 LM393ADR, U6 AP2114H-1.8TRG1, U7 AP2114H-3.3TRG1

Commit message: Fixed Diodes on Kirbi, Gucci, and PD Board
Fixed Diodes (DFLS130L-7) on Kirbi, Gucci, and PD Board from Kirbi Library
Parts:
- turned D1 to 180 degrees
- turned D5 to 90 degrees
Connections:
- net +3.3V: now also D1.1, D5.2; no longer D1.2, D5.1
- net +5V: now also D1.2; no longer D1.1
- net 1.8V: now also D5.1; no longer D5.2
Routing:
- net +5V: track 46.1 -> 46.8 mm
Changed lines of the file:
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@@
 <attribute name="VALUE" x="15.5" y="32.938" size="0.6096" layer="27" font="vector" ratio="20" align="top-center"/>
 </element>
-<element name="D5" library="Kirbi_ControlBoard" package="DFLS130L-7" value="30" x="19.2" y="18.7" smashed="yes" rot="R270">
-<attribute name="DKPN" value="DFLS130LDICT-ND" x="19.2" y="18.7" size="1.778" layer="27" rot="R270" display="off"/>
-<attribute name="NAME" x="18.5" y="20.9" size="1.016" layer="25" font="vector"/>
-<attribute name="VALUE" value="30" x="16.5" y="20.7" size="1.016" layer="27" font="vector" rot="R270"/>
-</element>
-<element name="D1" library="Kirbi_ControlBoard" package="DFLS130L-7" value="30" x="29.5" y="42" smashed="yes">
-<attribute name="DKPN" value="DFLS130LDICT-ND" x="29.5" y="42" size="1.778" layer="27" display="off"/>
-<attribute name="NAME" x="28.2" y="39.5" size="1.016" layer="25" font="vector"/>
-<attribute name="VALUE" value="30" x="27.5" y="39.3" size="1.016" layer="27" font="vector"/>
+<element name="D5" library="Kirbi_ControlBoard" package="DFLS130L-7" value="30" x="19.2" y="18.7" smashed="yes" rot="R90">
+<attribute name="DKPN" value="DFLS130LDICT-ND" x="19.2" y="18.7" size="1.778" layer="27" rot="R90" display="off"/>
+<attribute name="NAME" x="19.9" y="16.5" size="1.016" layer="25" font="vector" rot="R180"/>
+<attribute name="VALUE" value="30" x="21.9" y="16.7" size="1.016" layer="27" font="vector" rot="R90"/>
+</element>
+<element name="D1" library="Kirbi_ControlBoard" package="DFLS130L-7" value="30" x="29.5" y="42" smashed="yes" rot="R180">
+<attribute name="DKPN" value="DFLS130LDICT-ND" x="29.5" y="42" size="1.778" layer="27" rot="R180" display="off"/>
+<attribute name="NAME" x="30.3" y="40.8" size="1.016" layer="25" font="vector" rot="R180"/>
+<attribute name="VALUE" value="30" x="31.5" y="44.7" size="1.016" layer="27" font="vector" rot="R180"/>
 </element>
 <element name="R4" library="SparkFun-Resistors" library_urn="urn:adsk.eagle:library:532" package="0603" package3d_urn="urn:adsk.eagle:package:39650/1" value="1k" x="27" y="5" smashed="yes" rot="R180">
@@
 <contactref element="C25" pad="1"/>
 <contactref element="C12" pad="1"/>
-<contactref element="D1" pad="1"/>
+<contactref element="D1" pad="2"/>
 <contactref element="POWER_SWITCH" pad="P"/>
 <contactref element="5V" pad="A"/>
@@
 <via x="23" y="25" extent="1-16" drill="0.4"/>
 <wire x1="32.5" y1="42.6" x2="31.9" y2="42" width="0.2" layer="1"/>
-<wire x1="31.9" y1="42" x2="31.1" y2="42" width="0.2" layer="1"/>
 <via x="32.5" y="42.6" extent="1-16" drill="0.4"/>
 <via x="16.23561875" y="42.46438125" extent="1-16" drill="0.4"/>
@@
 <wire x1="15.2" y1="40.205" x2="15.2" y2="41.4287625" width="0.2" layer="1"/>
 <wire x1="15.2" y1="41.4287625" x2="16.23561875" y2="42.46438125" width="0.2" layer="1"/>
+<wire x1="31.9" y1="42" x2="30.45" y2="42" width="0.2" layer="1"/>
 </signal>
 <signal name="+3.3V">
@@
 <wire x1="10.9" y1="12.8" x2="9.26" y2="12.8" width="0.2" layer="16"/>
 <wire x1="9.26" y1="12.8" x2="8.73" y2="12.27" width="0.2" layer="16"/>
-<contactref element="D1" pad="2"/>
-<contactref element="D5" pad="1"/>
-<wire x1="28.55" y1="42" x2="28.55" y2="42.8" width="0.3" layer="1"/>
-<wire x1="28.55" y1="42.8" x2="27.05" y2="44.3" width="0.3" layer="1"/>
-<wire x1="27.05" y1="44.3" x2="22.35" y2="44.3" width="0.3" layer="1"/>
+<contactref element="D1" pad="1"/>
+<contactref element="D5" pad="2"/>
+<wire x1="22.35" y1="44.3" x2="27" y2="44.3" width="0.3" layer="1"/>
 <wire x1="20.65" y1="54" x2="20.65" y2="51.1" width="0.3" layer="1"/>
 <wire x1="20.65" y1="51.1" x2="20.75" y2="51" width="0.3" layer="1"/>
@@
 <wire x1="29.2" y1="17" x2="29.2" y2="13.48384375" width="0.5" layer="1"/>
 <wire x1="27.9" y1="15.7" x2="29.2" y2="17" width="0.2" layer="1"/>
-<wire x1="21.878975" y1="15.7" x2="20.478975" y2="17.1" width="0.2" layer="1"/>
-<wire x1="19.2" y1="17.1" x2="20.478975" y2="17.1" width="0.2" layer="1"/>
-<wire x1="21.878975" y1="15.7" x2="27.9" y2="15.7" width="0.2" layer="1"/>
+<wire x1="27.9" y1="15.7" x2="22" y2="15.7" width="0.2" layer="1"/>
 <wire x1="38.65" y1="18.4" x2="38.65" y2="18.7" width="0.2" layer="16"/>
 <wire x1="38.65" y1="18.7" x2="37.923" y2="19.427" width="0.2" layer="16"/>
@@
 <wire x1="4.1" y1="18.2976" x2="3.24545" y2="18.2976" width="0.2" layer="1"/>
 <wire x1="33" y1="19" x2="32.1" y2="18.1" width="0.2" layer="1"/>
+<wire x1="27" y1="44.3" x2="27.9" y2="43.4" width="0.3" layer="1"/>
+<wire x1="27.9" y1="43.4" x2="27.9" y2="42" width="0.3" layer="1"/>
+<wire x1="22" y1="15.7" x2="19.95" y2="17.75" width="0.2" layer="1"/>
+<wire x1="19.95" y1="17.75" x2="19.2" y2="17.75" width="0.2" layer="1"/>
 </signal>
 <signal name="LINE_LF">
@@
 <wire x1="25.123" y1="28" x2="24" y2="26.877" width="0.2" layer="16"/>
 <wire x1="24" y1="26.877" x2="24" y2="26.0556" width="0.2" layer="16"/>
-<contactref element="D5" pad="2"/>
+<contactref element="D5" pad="1"/>
 </signal>
 <signal name="EXP_PAD">
