File: Kirbi/v2 pcb/Kirbi_ControlBoard.sch (EAGLE design)
At the start: 57 parts, among them U1 PCA9306_LSSOP, U2 TEENSY_3.6_DIL, U5 LM393-8-SOIC, U6 AP2114H-1.8TRG1, U7 AP2114H-3.3TRG1

Commit message: Fixed Github versioning
Gucci:
V2 - 9/11/2019 (last push before competition)
V3 - current
Kirbi:
V1 - 9/11/2019 (last push before competition)
V2 - current
Parts:
- removed C13: 0.1uF, SparkFun-Capacitors:0.1UF-0603-25V-(+80/-20%)
- removed R21: 50, SparkFun-Resistors:1KOHM-0603-1/10W-1%
- added C10, C15, C25, C5, C9: 0.1uF, SparkFun-Capacitors:0.1UF-0603-25V-(+80/-20%)
- added F1: 3.5, Kirbi_ControlBoard:BEL_FUSE_C1F_3.5
- added POWER_CONN: MOLEX_2.54MM_2PIN, Kirbi_ControlBoard:MOLEX_2.54MM_2PIN
- added R10, R11, R3, R5, R6, R7: 1k, SparkFun-Resistors:1KOHM-0603-1/10W-1%
- added R2: 6.2, Kirbi_ControlBoard:6.2OHM-0603-1/10W-5%
- ESC: value MOLEX_1.25MM_4PIN_SMT -> MOLEX_1.25MM_3PIN_SMT; device Kirbi_ControlBoard:MOLEX_1.25MM_4PIN_SMT -> Kirbi_ControlBoard:MOLEX_1.25MM_3PIN_SMT
- R1: value 1.65k -> 100; device SparkFun-Resistors:1KOHM-0603-1/10W-1% -> SparkFun-Resistors:100OHM-0603-1/4W-5%
- R19: value 1.65k -> 200; device SparkFun-Resistors:1KOHM-0603-1/10W-1% -> SparkFun-Resistors:200OHM-0603-1/10W-1%
- R20: value 800 -> 100; device SparkFun-Resistors:1KOHM-0603-1/10W-1% -> SparkFun-Resistors:100OHM-0603-1/4W-5%
Connections:
- net S1/TX renamed S1/TTX
- removed net N$10: D4.C, R21.1
- new net N$6: F1.P$2, POWER.P4
- new net N$7: F1.P$1, POWER_CONN.P$1
- new net N$9: D4.C, R2.1
- new net RADIO_RESET: TRANSCEIVER.RESET, U2.29/T/PWM
- new net S1/TRX: ESC.2, U2.34/A15/RX5/CAN1-RX
- net +3.3V: now also R10.2, R11.2, R3.2, R5.2, R6.2, R7.2
- net +5V: now also C10.1, C15.1, C25.1, C5.1, C9.1; no longer C13.1
- net GND: now also C10.2, C15.2, C25.2, C5.2, C9.2, ESC.1, POWER_CONN.P$2, R2.2; no longer C13.2, R21.2
- net LF_INT: now also U2.15/A1/T; no longer U2.18/A4/T/SDA0
- net RADIO_NSS: now also U2.30/T/PWM; no longer U2.6/PWM
- net RF_INT: now also U2.16/A2/T/PWM; no longer U2.19/A5/T/SCL0
- net START: now also U2.14/A0/PWM; no longer U2.17/A3/T/PWM
- net TRX1: now also R10.1
- net TRX2: now also R11.1
- net TXD1: now also R3.1
- net TXD2: now also R5.1
- net TXD5: now also R6.1
- net TXD6: now also R7.1
Other:
- note added: "*Note: The TX and RX labels refer to the respective Teensy connection (not the sensor pins)"
- moved on the sheet: C11, C12

Commit message: Cleaned up Schematic/Silkscreen
Cleaned up Schematic/Silkscreen (moved a few things around)
Changed lines of the file:
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@@
 <part name="R11" library="SparkFun-Resistors" library_urn="urn:adsk.eagle:library:532" deviceset="1KOHM" device="-0603-1/10W-1%" package3d_urn="urn:adsk.eagle:package:39650/1" value="1k"/>
 <part name="+3V23" library="supply1" library_urn="urn:adsk.eagle:library:371" deviceset="+3V3" device=""/>
+<part name="GND27" library="supply1" library_urn="urn:adsk.eagle:library:371" deviceset="GND" device=""/>
 </parts>
 <sheets>
@@
 </instance>
 <instance part="U1" gate="G$1" x="375.92" y="96.52" smashed="yes">
-<attribute name="NAME" x="370.84" y="106.68" size="1.778" layer="95"/>
+<attribute name="NAME" x="370.84" y="107.442" size="1.778" layer="95"/>
 <attribute name="VALUE" x="370.84" y="86.36" size="1.778" layer="96"/>
 </instance>
@@
 </instance>
 <instance part="POWER" gate="G$1" x="296.672" y="105.41" smashed="yes">
-<attribute name="NAME" x="294.132" y="105.41" size="1.27" layer="97"/>
+<attribute name="NAME" x="283.972" y="113.792" size="1.27" layer="97"/>
 </instance>
 <instance part="P+3" gate="1" x="296.672" y="118.11" smashed="yes">
-<attribute name="VALUE" x="294.132" y="113.03" size="1.778" layer="96" rot="R90"/>
+<attribute name="VALUE" x="294.64" y="114.3" size="1.778" layer="96" rot="R90"/>
 </instance>
 <instance part="P+9" gate="1" x="101.6" y="205.74" smashed="yes">
@@
 <instance part="POWER_CONN" gate="G$1" x="266.7" y="101.6" smashed="yes">
 <attribute name="NAME" x="262.89" y="108.204" size="1.778" layer="95"/>
-<attribute name="VALUE" x="262.636" y="93.98" size="1.778" layer="95"/>
+<attribute name="VALUE" x="256.54" y="93.98" size="1.778" layer="95"/>
 </instance>
 <instance part="C12" gate="G$1" x="58.42" y="228.6" smashed="yes">
@@
 <instance part="+3V23" gate="G$1" x="414.02" y="237.998" smashed="yes">
 <attribute name="VALUE" x="412.496" y="233.172" size="1.778" layer="96" rot="R90"/>
+</instance>
+<instance part="GND27" gate="1" x="403.86" y="53.086" smashed="yes">
+<attribute name="VALUE" x="401.32" y="51.054" size="1.778" layer="96"/>
 </instance>
 </instances>
@@
 <wire x1="381" y1="55.88" x2="391.16" y2="55.88" width="0.1524" layer="91"/>
 <junction x="381" y="55.88"/>
-<pinref part="C11" gate="G$1" pin="2"/>
-<wire x1="391.16" y1="55.88" x2="403.86" y2="55.88" width="0.1524" layer="91"/>
-<wire x1="403.86" y1="55.88" x2="403.86" y2="58.42" width="0.1524" layer="91"/>
 <pinref part="C14" gate="G$1" pin="2"/>
 <wire x1="391.16" y1="58.42" x2="391.16" y2="55.88" width="0.1524" layer="91"/>
-<junction x="391.16" y="55.88"/>
 </segment>
 <segment>
@@
 <wire x1="316.992" y1="85.09" x2="304.292" y2="85.09" width="0.1524" layer="91"/>
 <pinref part="R1" gate="G$1" pin="1"/>
-<wire x1="304.292" y1="85.09" x2="283.972" y2="85.09" width="0.1524" layer="91"/>
+<wire x1="304.292" y1="85.09" x2="282.702" y2="85.09" width="0.1524" layer="91"/>
 <junction x="304.292" y="85.09"/>
 <pinref part="POWER_CONN" gate="G$1" pin="P$2"/>
-<wire x1="274.32" y1="99.06" x2="283.972" y2="99.06" width="0.1524" layer="91"/>
-<wire x1="283.972" y1="99.06" x2="283.972" y2="85.09" width="0.1524" layer="91"/>
+<wire x1="274.32" y1="99.06" x2="282.702" y2="99.314" width="0.1524" layer="91"/>
+<wire x1="282.702" y1="99.314" x2="282.702" y2="85.09" width="0.1524" layer="91"/>
 </segment>
 <segment>
@@
 <wire x1="279.4" y1="147.32" x2="279.908" y2="147.32" width="0.1524" layer="91"/>
 <wire x1="279.908" y1="147.32" x2="279.908" y2="139.446" width="0.1524" layer="91"/>
+</segment>
+<segment>
+<pinref part="C11" gate="G$1" pin="2"/>
+<pinref part="GND27" gate="1" pin="GND"/>
+<wire x1="403.86" y1="58.42" x2="403.86" y2="55.626" width="0.1524" layer="91"/>
 </segment>
 </net>
@@
 <wire x1="327.152" y1="97.79" x2="316.992" y2="97.79" width="0.1524" layer="91"/>
 <junction x="316.992" y="97.79"/>
-<wire x1="316.992" y1="97.79" x2="309.372" y2="97.79" width="0.1524" layer="91"/>
+<wire x1="316.992" y1="97.79" x2="314.198" y2="97.79" width="0.1524" layer="91"/>
 <junction x="316.992" y="97.79"/>
 <pinref part="P+3" gate="1" pin="+5V"/>
@@
 <junction x="296.672" y="110.49"/>
 <junction x="296.672" y="115.57"/>
-<wire x1="309.372" y1="97.79" x2="309.372" y2="115.57" width="0.1524" layer="91"/>
-<wire x1="309.372" y1="115.57" x2="296.672" y2="115.57" width="0.1524" layer="91"/>
+<wire x1="314.198" y1="97.79" x2="314.198" y2="115.57" width="0.1524" layer="91"/>
+<wire x1="314.198" y1="115.57" x2="296.672" y2="115.57" width="0.1524" layer="91"/>
 <wire x1="296.672" y1="102.87" x2="291.592" y2="102.87" width="0.1524" layer="91"/>
 <pinref part="POWER" gate="G$1" pin="P5"/>
@@
 <segment>
 <pinref part="U1" gate="G$1" pin="SCL2"/>
-<wire x1="396.24" y1="96.52" x2="401.32" y2="96.52" width="0.1524" layer="91"/>
-<label x="401.32" y="96.52" size="1.778" layer="95" xref="yes"/>
+<wire x1="396.24" y1="96.52" x2="406.4" y2="96.52" width="0.1524" layer="91"/>
+<label x="406.4" y="96.52" size="1.778" layer="95" rot="R270" xref="yes"/>
 </segment>
 </net>
@@
 <pinref part="U1" gate="G$1" pin="SDA2"/>
 <wire x1="396.24" y1="93.98" x2="401.32" y2="93.98" width="0.1524" layer="91"/>
-<label x="401.32" y="93.98" size="1.778" layer="95" xref="yes"/>
+<label x="401.32" y="93.98" size="1.778" layer="95" rot="R270" xref="yes"/>
 </segment>
 </net>
@@
 <net name="N$6" class="0">
 <segment>
-<wire x1="281.94" y1="104.14" x2="284.48" y2="104.14" width="0.1524" layer="91"/>
-<wire x1="284.48" y1="104.14" x2="284.48" y2="110.49" width="0.1524" layer="91"/>
+<wire x1="281.94" y1="104.14" x2="283.464" y2="104.14" width="0.1524" layer="91"/>
+<wire x1="283.464" y1="104.14" x2="283.464" y2="110.49" width="0.1524" layer="91"/>
 <pinref part="POWER" gate="G$1" pin="P4"/>
-<wire x1="284.48" y1="110.49" x2="286.512" y2="110.49" width="0.1524" layer="91"/>
+<wire x1="283.464" y1="110.49" x2="286.512" y2="110.49" width="0.1524" layer="91"/>
 <pinref part="F1" gate="G$1" pin="P$2"/>
 </segment>
@@
 <segment>
 <pinref part="ESC" gate="G$1" pin="3"/>
-<wire x1="279.4" y1="152.4" x2="281.94" y2="152.4" width="0.1524" layer="91"/>
-<label x="281.94" y="152.4" size="1.778" layer="95" xref="yes"/>
+<wire x1="279.4" y1="152.4" x2="284.48" y2="152.4" width="0.1524" layer="91"/>
+<label x="284.48" y="152.4" size="1.778" layer="95" rot="R90" xref="yes"/>
 </segment>
 </net>
@@
 <segment>
 <pinref part="ESC" gate="G$1" pin="2"/>
-<wire x1="279.4" y1="149.86" x2="281.94" y2="149.86" width="0.1524" layer="91"/>
-<label x="281.94" y="149.86" size="1.778" layer="95" xref="yes"/>
-</segment>
-</net>
+<wire x1="279.4" y1="149.86" x2="289.56" y2="149.86" width="0.1524" layer="91"/>
+<label x="289.56" y="149.86" size="1.778" layer="95" rot="R90" xref="yes"/>
+</segment>
+</net>

Commit message: PDB Conector/Power Switch/Resistors
Pull Up Resistor - Radio Module
Pull Down Resistors - MUXs
Power Distribution Board Connector (in Kirbi library and on schematic)
Replaced old power switch addded LED
Parts:
- removed POWER: POWER_SWITCH, Kirbi_ControlBoard:POWER_SWITCH
- added D1, D5: DFLS130L-7_30V_1A, Kirbi_ControlBoard:DFLS130L-7_30V_1A
- added D6: 5V, SparkFun-LED:LED0603
- added PDB_CONN: AMPHENOL_2X3_2.54MM, Kirbi_ControlBoard:AMPHENOL_2X3_2.54MM
- added POWER_SWITCH: GPTS202312B, Kirbi_ControlBoard:GPTS202312B
- added R12, R18, R4, R8, R9: 1k, SparkFun-Resistors:1KOHM-0603-1/10W-1%
- R1: value 100 -> 200; device SparkFun-Resistors:100OHM-0603-1/4W-5% -> SparkFun-Resistors:200OHM-0603-1/10W-1%
Connections:
- new net PDB_!CS!: PDB_CONN.1
- new net PDB_!EOC!: PDB_CONN.4
- new net PDB_MISO: PDB_CONN.2, U2.5/PWM
- new net PDB_MOSI: PDB_CONN.5, U2.21/A7/PWM
- new net PDB_SCLK: PDB_CONN.3, U2.20/A6/PWM
- new net PDB_START: PDB_CONN.6
- net +3.3V: now also D1.A, D5.C, R4.2
- net +5V: now also D1.C, D6.A, POWER_SWITCH.COMMON; no longer POWER.P3, POWER.P5
- net 1.8V: now also D5.A
- net GND: now also R12.1, R18.1, R8.1, R9.1
- net MUXS1: now also R12.2, R8.2
- net MUXS2: now also R18.2, R9.2
- net N$6: now also POWER_SWITCH.B; no longer POWER.P4
- net N$8: now also D6.C; no longer POWER.P1
- net NEO_DI: now also U2.6/PWM; no longer U2.24
- net RADIO_DIO0: now also U2.22/A8/T/PWM; no longer U2.5/PWM
- net RADIO_NSS: now also R4.1

Commit message: Routed Power Distribution Board
Routed Power Distribution Board
Connections:
- net PDB_!CS!: now also U2.17/A3/T/PWM
- net PDB_!EOC!: now also U2.18/A4/T/SDA0
- net PDB_START: now also U2.19/A5/T/SCL0
Changed lines of the file:
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@@
+</segment>
+</net>
+<net name="PDB_!CS!" class="0">
+<segment>
+<pinref part="U2" gate="G$1" pin="17/A3/T/PWM"/>
+<wire x1="165.1" y1="193.04" x2="160.02" y2="193.04" width="0.1524" layer="91"/>
+<label x="160.02" y="193.04" size="1.778" layer="95" rot="R180" xref="yes"/>
+</segment>
+</net>
+<net name="PDB_!EOC!" class="0">
+<segment>
+<pinref part="U2" gate="G$1" pin="18/A4/T/SDA0"/>
+<wire x1="165.1" y1="190.5" x2="160.02" y2="190.5" width="0.1524" layer="91"/>
+<label x="160.02" y="190.5" size="1.778" layer="95" rot="R180" xref="yes"/>
+</segment>
+</net>
+<net name="PDB_START" class="0">
+<segment>
+<pinref part="U2" gate="G$1" pin="19/A5/T/SCL0"/>
+<wire x1="165.1" y1="187.96" x2="160.02" y2="187.96" width="0.1524" layer="91"/>
+<label x="160.02" y="187.96" size="1.778" layer="95" rot="R180" xref="yes"/>
 </segment>
 </net>

Commit message: Screw Head Clearance/Silkscreen
Screw Head Clearance/Silkscreen cleaned up
Parts:
- renumbered D6 to 5V
Changed lines of the file:
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@@
 <part name="GND33" library="SparkFun-PowerSymbols" library_urn="urn:adsk.eagle:library:530" deviceset="GND" device=""/>
 <part name="POWER_SWITCH" library="Kirbi_ControlBoard" deviceset="GPTS202312B" device=""/>
-<part name="D6" library="SparkFun-LED" deviceset="LED" device="0603" value="5V"/>
+<part name="5V" library="SparkFun-LED" deviceset="LED" device="0603" value="5V"/>
 <part name="R1" library="SparkFun-Resistors" library_urn="urn:adsk.eagle:library:532" deviceset="200OHM" device="-0603-1/10W-1%" package3d_urn="urn:adsk.eagle:package:39650/1" value="200"/>
 <part name="FRAME2" library="RoboJackets-Frames" deviceset="FRAME_B_L" device=""/>
@@
 <attribute name="VALUE" x="302.006" y="109.22" size="1.778" layer="96" font="vector" rot="R180"/>
 </instance>
-<instance part="D6" gate="G$1" x="307.086" y="97.536" smashed="yes" rot="R90">
+<instance part="5V" gate="G$1" x="307.086" y="97.536" smashed="yes" rot="R90">
 <attribute name="NAME" x="311.658" y="94.107" size="1.778" layer="95" font="vector" rot="R180"/>
 <attribute name="VALUE" x="311.658" y="99.441" size="1.778" layer="96" font="vector" rot="R180" align="top-left"/>
@@
 <wire x1="304.546" y1="113.03" x2="304.546" y2="104.14" width="0.1524" layer="91"/>
 <junction x="304.292" y="113.03"/>
-<pinref part="D6" gate="G$1" pin="A"/>
+<pinref part="5V" gate="G$1" pin="A"/>
 <wire x1="304.546" y1="104.14" x2="304.546" y2="97.536" width="0.1524" layer="91"/>
 <junction x="304.546" y="104.14"/>
@@
 <net name="N$8" class="0">
 <segment>
-<pinref part="D6" gate="G$1" pin="C"/>
+<pinref part="5V" gate="G$1" pin="C"/>
 <wire x1="312.166" y1="97.536" x2="313.69" y2="97.536" width="0.1524" layer="91"/>
 <wire x1="313.69" y1="97.536" x2="313.69" y2="95.25" width="0.1524" layer="91"/>

Commit message: Renamed Parts/Routed SPI Interface
Renamed Parts (U1-U7)
Routed SPI Interface (Connectted MISO, MOSI, and SCK) (Fixed routing to avoid islands/breaks in ground plane)
Parts:
- removed IMU: ICM-20948, ICM-20948:ICM-20948
- added U3: PCA9306_LSSOP, Gucci_ControlBoard:PCA9306_LSSOP
- U1: value PCA9306_LSSOP -> TEENSY_3.6_DIL; device Gucci_ControlBoard:PCA9306_LSSOP -> Teensy_3_and_LC_Series_Boards_v1.4:TEENSY_3.6_DIL
- U2: value TEENSY_3.6_DIL -> ICM-20948; device Teensy_3_and_LC_Series_Boards_v1.4:TEENSY_3.6_DIL -> ICM-20948:ICM-20948
- renumbered TRANSCEIVER to U4
Connections:
- removed net PDB_MISO: PDB_CONN.2, U2.5/PWM
- removed net PDB_MOSI: PDB_CONN.5, U2.21/A7/PWM
- removed net PDB_SCLK: PDB_CONN.3, U2.20/A6/PWM
- removed net RADIO_SCK: U2.13/SCK0/LED, U4.SCK
- new net SCK: PDB_CONN.2, U1.13/SCK0/LED, U4.SCK
- net +5V: now also U1.VIN; no longer U2.VIN
- net 1.8V: now also U2.NCS, U2.VDD, U2.VDDIO, U3.VREF1; no longer IMU.NCS, IMU.VDD, IMU.VDDIO, U1.VREF1
- net GND: now also U1.AGND, U2.AD0/SDO, U2.FSYNC, U2.RESV_20, U3.GND; no longer IMU.AD0/SDO, IMU.FSYNC, IMU.GND, IMU.RESV_20, U2.AGND
- net LF_INT: now also U1.15/A1/T; no longer U2.15/A1/T
- net LINE_LF: now also U1.35/A16/PWM; no longer U2.35/A16/PWM
- net LINE_REF: now also U1.A22/DAC1; no longer U2.A22/DAC1
- net LINE_RF: now also U1.23/A9/T/PWM; no longer U2.23/A9/T/PWM
- net MISO: now also PDB_CONN.3, U1.12/MISO0; no longer U2.12/MISO0
- net MOSI: now also PDB_CONN.5, U1.11/MOSI0; no longer U2.11/MOSI0
- net MUXS1: now also U1.2/PWM; no longer U2.2/PWM
- net MUXS2: now also U1.25; no longer U2.25
- net N$3: now also U2.REGOUT; no longer IMU.REGOUT
- net N$4: now also U3.EN, U3.VREF2; no longer U1.EN, U1.VREF2
- net NEO_DI: now also U1.6/PWM; no longer U2.6/PWM
- net PDB_!CS!: now also U1.17/A3/T/PWM; no longer U2.17/A3/T/PWM
- net PDB_!EOC!: now also U1.18/A4/T/SDA0; no longer U2.18/A4/T/SDA0
- net PDB_START: now also U1.19/A5/T/SCL0; no longer U2.19/A5/T/SCL0
- net RADIO_DIO0: now also U1.22/A8/T/PWM; no longer U2.22/A8/T/PWM
- net RADIO_NSS: now also U1.30/T/PWM; no longer U2.30/T/PWM
- net RADIO_RESET: now also U1.29/T/PWM; no longer U2.29/T/PWM
- net RF_INT: now also U1.16/A2/T/PWM; no longer U2.16/A2/T/PWM
- net RXD3: now also U1.0/RX1/MOSI1/T; no longer U2.0/RX1/MOSI1/T
- net RXD4: now also U1.31/A12/RX4; no longer U2.31/A12/RX4
- net S1/TRX: now also U1.34/A15/RX5/CAN1-RX; no longer U2.34/A15/RX5/CAN1-RX
- net S1/TTX: now also U1.33/A14/TX5/CAN1-TX; no longer U2.33/A14/TX5/CAN1-TX
- net SCL1: now also U2.SCL/SCLK, U3.SCL1; no longer IMU.SCL/SCLK, U1.SCL1
- net SCL2: now also U1.3/CAN0-TX/SCL2/PWM, U3.SCL2; no longer U1.SCL2, U2.3/CAN0-TX/SCL2/PWM
- net SDA1: now also U2.SDA/SDI, U3.SDA1; no longer IMU.SDA/SDI, U1.SDA1
- net SDA2: now also U1.4/CAN0-RX/SDA2/PWM, U3.SDA2; no longer U1.SDA2, U2.4/CAN0-RX/SDA2/PWM
- net START: now also U1.14/A0/PWM; no longer U2.14/A0/PWM
- net TRX1: now also U1.7/RX3/PWM; no longer U2.7/RX3/PWM
- net TRX2: now also U1.9/RX2/PWM; no longer U2.9/RX2/PWM
- net TTX1: now also U1.8/TX3/PWM; no longer U2.8/TX3/PWM
- net TTX2: now also U1.10/TX2/PWM; no longer U2.10/TX2/PWM
- net TXD3: now also U1.1/TX1/MISO1/T; no longer U2.1/TX1/MISO1/T
- net TXD4: now also U1.32/A13/TX4; no longer U2.32/A13/TX4
