File: Kirbi/v2 pcb/Kirbi_ControlBoard.sch (EAGLE design)
At the start: 78 parts, among them U1 TEENSY_3.6_DIL, U2 ICM-20948, U3 PCA9306_LSSOP, U5 LM393-8-SOIC, U6 AP2114H-1.8TRG1, U7 AP2114H-3.3TRG1

Commit message: Replaced parts on Kirbi control board
Replaced parts on Kirbi control board/made slight changes to Gucci library
Parts:
- D1, D5: value DFLS130L-7_30V_1A -> 30; device Kirbi_ControlBoard:DFLS130L-7_30V_1A -> Kirbi_ControlBoard:DFLS130L-7
- DIST_1, DIST_2, DIST_3, DIST_4, DIST_5, DIST_6: value MOLEX_1.25MM_4PIN_SMT -> 0532610471; device Kirbi_ControlBoard:MOLEX_1.25MM_4PIN_SMT -> Kirbi_ControlBoard:0532610471
- ESC: value MOLEX_1.25MM_3PIN_SMT -> 0532610371; device Kirbi_ControlBoard:MOLEX_1.25MM_3PIN_SMT -> Kirbi_ControlBoard:0532610371
- F1: device Kirbi_ControlBoard:BEL_FUSE_C1F_3.5 -> Kirbi_ControlBoard:C1F3.5
- LINE_LF, LINE_RF, START: value AMPHENOL_2X02_2.54MM_SHROUD -> 75869-130LF; device Gucci_ControlBoard:AMPHENOL_2X02_2.54MM_SHROUD -> Gucci_ControlBoard:75869-130LF
- MUX_RX1, MUX_RX2, MUX_TX1, MUX_TX2: value MUX_74LVC1G157GV -> 74LVC1G157GW,125; device Kirbi_ControlBoard:MUX_74LVC1G157GV -> Kirbi_ControlBoard:74LVC1G157GW,125
- PDB_CONN: value AMPHENOL_2X3_2.54MM -> 71600-006LF; device Kirbi_ControlBoard:AMPHENOL_2X3_2.54MM -> Kirbi_ControlBoard:71600-006LF
- POWER_CONN: value MOLEX_2.54MM_2PIN -> 1719770002; device Kirbi_ControlBoard:MOLEX_2.54MM_2PIN -> Kirbi_ControlBoard:1719770002
- U1: value TEENSY_3.6_DIL -> DEV-14057; device Teensy_3_and_LC_Series_Boards_v1.4:TEENSY_3.6_DIL -> Kirbi_ControlBoard:DEV-14057
- U2: device ICM-20948:ICM-20948 -> Gucci_ControlBoard:ICM-20948
- U3: value PCA9306_LSSOP -> PCA9306; device Gucci_ControlBoard:PCA9306_LSSOP -> Gucci_ControlBoard:PCA9306
- U4: value (none) -> RFM69HCW_SMT
- U5: value LM393-8-SOIC -> LM393ADR; device Gucci_ControlBoard:LM393-8-SOIC -> Gucci_ControlBoard:LM393ADR
Connections:
- net +5V: now also U5.V+; no longer U5.VCC
- net GND: now also U5.V-; no longer U5.GND
- net LF_INT: now also U5.OUTB; no longer U5.OUT2
- net LINE_LF: now also U5.INB+; no longer U5.IN2+
- net LINE_REF: now also U5.INA-, U5.INB-; no longer U5.IN1-, U5.IN2-
- net LINE_RF: now also U5.INA+; no longer U5.IN1+
- net RF_INT: now also U5.OUTA; no longer U5.OUT1
Other:
- moved on the sheet: C19, C20, C21, C4, D1, D5, DIST_1, DIST_2, DIST_3, DIST_4, DIST_5, DIST_6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

Commit message: Fixed doubled parts in Gucci and Kirbi Library
Fixed doubled parts in Gucci and Kirbi Library (IMU, Teensy)
Parts:
- U1: value DEV-14057 -> TEENSY_3.6; device Kirbi_ControlBoard:DEV-14057 -> Gucci_ControlBoard:TEENSY_3.6
Changed lines of the file:
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@@
 </classes>
 <parts>
-<part name="U1" library="Kirbi_ControlBoard" deviceset="DEV-14057" device=""/>
+<part name="U1" library="Gucci_ControlBoard" deviceset="TEENSY_3.6" device=""/>
 <part name="GND2" library="SparkFun-PowerSymbols" library_urn="urn:adsk.eagle:library:530" deviceset="GND" device=""/>
 <part name="GND3" library="SparkFun-PowerSymbols" library_urn="urn:adsk.eagle:library:530" deviceset="GND" device=""/>
