File: PowerDistribution/powerDistribution.brd (EAGLE design)
At the start: 80 x 82 mm, 49 parts, among them J1 XT-60BATT_LABEL, J2 CONNECTOR, J3 CONNECTOR, U1 MAX11635EEE+, U2 LM2678SX-5.0/NOPB, U3 CQ2065, U4 CQ2065, U7 AP2114H-3.3TRG1

Commit message: added resistor values
Parts:
- C3, C4: value CF1 -> 1000pF
- R10, R14: value RF1 -> 100
- moved F1 0.48 mm to (27.0, 25.0)
Routing:
- net !EOC!: track 15.2 -> 11.3 mm, vias 0 -> 2
- net !CNVST!: track 18.4 -> 16.0 mm, vias 0 -> 2
- net !CS!: track 13.6 -> 15.5 mm, vias 0 -> 2
- net SCLK: track 13.2 -> 14.7 mm, vias 0 -> 2
- net MISO: track 13.4 -> 12.5 mm, vias 0 -> 2
- net AIN0: track 36.7 -> 36.3 mm, vias 2 -> 0
- net MOSI: track 13.2 -> 13.5 mm, vias 0 -> 2
- net +3V3: track 35.2 -> 35.3 mm, vias 0 -> 2
- net VREF: vias 0 -> 2

Commit message: made some design review edits
Parts:
- added D2, U$6: DFLS130L-7_30V_1A, Kirbi_ControlBoard:DFLS130L-7_30V_1A
- added R6: 1k, rcl:R0603
Connections:
- net !CS!: now also R6.1, R6.2
- net +24V: now also D2.P$1, XF1.3, XF1.4, XF2.1, XF2.2; no longer XF1.P$2, XF1.P$4, XF2.P$1, XF2.P$3
- net +3V3: now also U$6.P$2
- net +5V: now also D2.P$2, U$6.P$1
- net P1: now also XF1.1, XF1.2; no longer XF1.P$1, XF1.P$3
- net P2: now also XF2.3, XF2.4; no longer XF2.P$2, XF2.P$4
Routing:
- net +24V: track 16.8 -> 31.1 mm, vias 2 -> 4
- net +3V3: track 35.3 -> 40.0 mm
- net !CS!: track 15.5 -> 14.8 mm, vias 2 -> 3
- net !EOC!: track 11.3 -> 11.9 mm

Commit message: made more design review edits
Parts:
- +24V, +3.3V, +5V: value LED-SMD -> Green
- F1: value ERB-RE5R00V -> 5A
- J2, J3: value CONNECTOR -> (none); device CurrentSensing:XT-60 -> CurrentSensing:ESC_CONNECT
- R3: value 100Ω -> 100
- R4: value 200Ω -> 200
- R5: value 1200Ω -> 1200
- XF1, XF2: value 3550(2) -> 40A
- moved XF2 3.00 mm to (67.0, 72.0)
- moved R6 1.00 mm to (31.0, 9.00), turned to 180 degrees
- turned C1 to 180 degrees
- turned C4 to 0 degrees
- renumbered U$6 to D3
Connections:
- net !CNVST! renamed !START!
- net AIN0 renamed L_MOTOR
- net AIN1 renamed R_MOTOR
- net P1 renamed I1
- net P2 renamed I2
- removed net N1: J2.BATT, U3.7
- removed net N2: J3.BATT, U4.6
- new net L_ESC: J2.ESC, U3.7
- new net R_ESC: J3.ESC, U4.6
- net !CS!: no longer R6.2
- net +3V3: now also R6.2
- net +5V: now also C1.1, C2.1; no longer C1.2, C2.2
- net GND: now also C1.2, C2.2, U1.3, U1.4; no longer C1.1, C2.1
Routing:
- net +3V3: track 40.0 -> 44.3 mm
- net GND: track 65.4 -> 67.9 mm, vias 25 -> 27
- net !CS!: track 14.8 -> 16.3 mm
- net R_MOTOR: track 40.2 -> 40.8 mm
- added copper zone on layer 1, net L_ESC
- added copper zone on layer 1, net R_ESC
- removed copper zone on layer 1, net N1
- removed copper zone on layer 1, net N2
Other:
- board text added: "40A"
- board text added: "5A"

Commit message: added TVSDIODE
Parts:
- added D4: TVSDIODE, CurrentSensing:TVSDIODE
Connections:
- net +24V: now also D4.P$2
- net GND: now also D4.P$1
Routing:
- net GND: track 67.9 -> 70.4 mm, vias 27 -> 28
Other:
- board text added: "D4"
Changed lines of the file:
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@@
 <text x="54.9" y="75.6" size="1" layer="21" font="vector">40A</text>
 <rectangle x1="7" y1="0.4" x2="10" y2="3.4" layer="21"/>
+<text x="47" y="77" size="1" layer="21" font="vector">D4</text>
 </plain>
 <attributes>
@@
 <attribute name="VALUE" x="72.46" y="41.032" size="1" layer="27" font="vector"/>
 </element>
+<element name="D4" library="CurrentSensing" package="TVSDIODE" value="TVSDIODE" x="45" y="75" smashed="yes" rot="R90"/>
 </elements>
 <signals>
@@
 <contactref element="J2" pad="GND"/>
 <contactref element="J3" pad="GND"/>
+<contactref element="D4" pad="P$1"/>
+<wire x1="45" y1="73.0315" x2="45" y2="72" width="0.8" layer="1"/>
+<wire x1="45" y1="72" x2="46" y2="71" width="0.8" layer="1"/>
+<via x="46" y="71" extent="1-16" drill="0.8"/>
 </signal>
 <signal name="+5V">
@@
 <contactref element="XF2" pad="2"/>
 <contactref element="XF2" pad="1"/>
+<contactref element="D4" pad="P$2"/>
 </signal>
 <signal name="N$6">

Commit message: added connectors and M3 holes for mounting
Parts:
- removed JP1: (no value), pinhead:1X08/90
- added J4: MOLEX_2.54MM_2PIN, CurrentSensing:MOLEX_2.54MM_2PIN
- added J5: AMPHENOL_2X3_2.54MM, CurrentSensing:AMPHENOL_2X3_2.54MM
- moved R10 6.00 mm to (14.0, 28.0), turned to 90 degrees
- moved R7 6.00 mm to (11.0, 28.0)
- moved R8 6.00 mm to (17.0, 28.0)
- moved R9 6.00 mm to (20.0, 28.0)
- moved D4 1.00 mm to (46.0, 75.0)
- moved J1 1.00 mm to (40.0, 82.0)
Connections:
- net !CS!: now also J5.P$4; no longer JP1.7
- net !EOC!: now also J5.P$2; no longer JP1.3
- net !START!: now also J5.P$3; no longer JP1.2
- net +5V: now also J4.P$1; no longer JP1.1
- net GND: now also J4.P$2; no longer JP1.8
- net MISO: now also J5.P$1; no longer JP1.4
- net MOSI: now also J5.P$6; no longer JP1.5
- net SCLK: now also J5.P$5; no longer JP1.6
Routing:
- net !CS!: track 16.3 -> 32.9 mm, vias 3 -> 2
- net GND: track 70.4 -> 86.1 mm, vias 28 -> 27
- net L_MOTOR: track 36.1 -> 43.0 mm
- net MISO: track 12.5 -> 18.7 mm
- net SCLK: track 14.6 -> 19.8 mm, vias 2 -> 1
- net !START!: track 16.0 -> 21.0 mm, vias 2 -> 1
- net N$2: track 6.33 -> 8.74 mm
- net !EOC!: track 11.9 -> 13.2 mm
- net VREF: track 69.8 -> 68.6 mm, vias 2 -> 0
- net MOSI: track 13.5 -> 12.8 mm, vias 2 -> 1

Commit message: power distribution edits
Parts:
- moved R9 9.00 mm to (11.0, 28.0)
- moved R6 8.61 mm to (39.5, 10.4)
- moved R10 6.00 mm to (20.0, 28.0)
- moved R11 6.00 mm to (60.0, 28.0)
- moved R12 6.00 mm to (66.0, 28.0)
- moved R13 6.00 mm to (69.0, 28.0)
- moved R14 6.00 mm to (63.0, 28.0)
- moved R7 6.00 mm to (17.0, 28.0)
- moved J4 5.00 mm to (55.1, 2.10)
- moved C6 4.85 mm to (37.8, 12.5), turned to 180 degrees
- moved C5 4.24 mm to (35.5, 16.6), turned to 0 degrees
- moved U$2 3.61 mm to (64.0, 9.00)
- moved U$1 3.16 mm to (50.0, 4.00)
- moved U$4 3.16 mm to (68.5, 8.90)
- moved R8 3.00 mm to (14.0, 28.0), turned to 90 degrees
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Routing:
- net GND: track 86.1 -> 61.5 mm, vias 27 -> 28
- net !CS!: track 32.9 -> 10.1 mm, vias 2 -> 0
- net +5V: track 0.00 -> 17.0 mm, vias 0 -> 4
- net SCLK: track 19.8 -> 8.14 mm
- net R_MOTOR: track 40.8 -> 32.6 mm
- net MISO: track 18.7 -> 11.3 mm, vias 2 -> 1
- net L_MOTOR: track 43.0 -> 36.5 mm
- net !START!: track 21.0 -> 17.3 mm
- net !EOC!: track 13.2 -> 16.1 mm, vias 2 -> 0
- net N$2: track 8.74 -> 5.96 mm
- net +3V3: track 44.3 -> 43.2 mm, vias 2 -> 0
- net VREF: track 68.6 -> 69.2 mm

Commit message: updated device descriptions
Parts:
- U3, U4: device CurrentSensing:CQ2065 -> CurrentSensing:974-1092-1
Connections:
- net !CS!: now also J5.4; no longer J5.P$4
- net !EOC!: now also J5.2; no longer J5.P$2
- net !START!: now also J5.3; no longer J5.P$3
- net +5V: now also F1.2, J4.1; no longer F1.P$2, J4.P$1
- net GND: now also J4.2; no longer J4.P$2
- net MISO: now also J5.1; no longer J5.P$1
- net MOSI: now also J5.6; no longer J5.P$6
- net N$10: now also F1.1, L1.2; no longer F1.P$1, L1.P$2
- net N$6: now also L1.1; no longer L1.P$1
- net SCLK: now also J5.5; no longer J5.P$5

Commit message: Fixed Diodes on Kirbi, Gucci, and PD Board
Fixed Diodes (DFLS130L-7) on Kirbi, Gucci, and PD Board from Kirbi Library
Parts:
- D2, D3: value DFLS130L-7_30V_1A -> 30; device Kirbi_ControlBoard:DFLS130L-7_30V_1A -> Kirbi_ControlBoard:DFLS130L-7
- turned D2 to 0 degrees
- turned D3 to 90 degrees
Connections:
- net +24V: now also D2.2; no longer D2.P$1
- net +3V3: now also D3.1; no longer D3.P$2
- net +5V: now also D2.1, D3.2; no longer D2.P$2, D3.P$1
Routing:
- net +24V: track 31.1 -> 31.7 mm
