File: PowerDistribution/powerDistribution.sch (EAGLE design)
At the start: 45 parts, among them J1 XT-60BATT_LABEL, J2 CONNECTOR, J3 CONNECTOR, U1 MAX11635EEE+, U2 LM2678SX-5.0/NOPB, U3 CQ2065, U4 CQ2065, U7 AP2114H-3.3TRG1

Commit message: added resistor values
Parts:
- C3, C4: value CF1 -> 1000pF
- R10, R14: value RF1 -> 100
Other:
- note added: "0.1%"
Changed lines of the file:
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@@
 <part name="R8" library="rcl" library_urn="urn:adsk.eagle:library:334" deviceset="R-US_" device="R0603" package3d_urn="urn:adsk.eagle:package:23555/3" value="39k"/>
 <part name="R9" library="rcl" library_urn="urn:adsk.eagle:library:334" deviceset="R-US_" device="R0603" package3d_urn="urn:adsk.eagle:package:23555/3" value="20k"/>
-<part name="R10" library="rcl" library_urn="urn:adsk.eagle:library:334" deviceset="R-US_" device="R0603" package3d_urn="urn:adsk.eagle:package:23555/3" value="RF1"/>
-<part name="C3" library="rcl" library_urn="urn:adsk.eagle:library:334" deviceset="C-US" device="C0603" package3d_urn="urn:adsk.eagle:package:23616/2" value="CF1"/>
+<part name="R10" library="rcl" library_urn="urn:adsk.eagle:library:334" deviceset="R-US_" device="R0603" package3d_urn="urn:adsk.eagle:package:23555/3" value="100"/>
+<part name="C3" library="rcl" library_urn="urn:adsk.eagle:library:334" deviceset="C-US" device="C0603" package3d_urn="urn:adsk.eagle:package:23616/2" value="1000pF"/>
 <part name="U4" library="CurrentSensing" deviceset="CQ2065" device=""/>
 <part name="GND2" library="supply1" library_urn="urn:adsk.eagle:library:371" deviceset="GND" device=""/>
@@
 <part name="R12" library="rcl" library_urn="urn:adsk.eagle:library:334" deviceset="R-US_" device="R0603" package3d_urn="urn:adsk.eagle:package:23555/3" value="39k"/>
 <part name="R13" library="rcl" library_urn="urn:adsk.eagle:library:334" deviceset="R-US_" device="R0603" package3d_urn="urn:adsk.eagle:package:23555/3" value="20k"/>
-<part name="R14" library="rcl" library_urn="urn:adsk.eagle:library:334" deviceset="R-US_" device="R0603" package3d_urn="urn:adsk.eagle:package:23555/3" value="RF1"/>
-<part name="C4" library="rcl" library_urn="urn:adsk.eagle:library:334" deviceset="C-US" device="C0603" package3d_urn="urn:adsk.eagle:package:23616/2" value="CF1"/>
+<part name="R14" library="rcl" library_urn="urn:adsk.eagle:library:334" deviceset="R-US_" device="R0603" package3d_urn="urn:adsk.eagle:package:23555/3" value="100"/>
+<part name="C4" library="rcl" library_urn="urn:adsk.eagle:library:334" deviceset="C-US" device="C0603" package3d_urn="urn:adsk.eagle:package:23616/2" value="1000pF"/>
 <part name="JP1" library="pinhead" library_urn="urn:adsk.eagle:library:325" deviceset="PINHD-1X8" device="/90" package3d_urn="urn:adsk.eagle:package:22413/2"/>
 <part name="P+3" library="supply1" library_urn="urn:adsk.eagle:library:371" deviceset="+5V" device=""/>
@@
 <part name="GND15" library="supply1" library_urn="urn:adsk.eagle:library:371" deviceset="GND" device=""/>
 <part name="D1" library="CurrentSensing" deviceset="SD2114S040S8R0" device=""/>
-<part name="F1" library="CurrentSensing" deviceset="ERB-RE5R00V" device=""/>
 <part name="XF1" library="CurrentSensing" deviceset="3550(2)" device=""/>
 <part name="XF2" library="CurrentSensing" deviceset="3550(2)" device=""/>
 <part name="J2" library="CurrentSensing" deviceset="CONNECTOR" device=""/>
 <part name="J3" library="CurrentSensing" deviceset="CONNECTOR" device=""/>
+<part name="F1" library="CurrentSensing" deviceset="ERB-RE5R00V" device=""/>
 </parts>
 <sheets>
@@
 <wire x1="102.87" y1="95.25" x2="170.18" y2="95.25" width="0.1524" layer="97" style="shortdash"/>
 <wire x1="102.87" y1="95.25" x2="5.08" y2="95.25" width="0.1524" layer="97" style="shortdash"/>
+<text x="254" y="149.86" size="1.778" layer="97">0.1%</text>
+<text x="241.3" y="143.51" size="1.778" layer="97">0.1%</text>
+<text x="243.84" y="72.39" size="1.778" layer="97">0.1%</text>
+<text x="254" y="80.01" size="1.778" layer="97">0.1%</text>
 </plain>
 <instances>
@@
 <attribute name="VALUE" x="116.332" y="19.05" size="1.778" layer="96" font="vector" rot="R90" align="top-left"/>
 </instance>
-<instance part="F1" gate="G$1" x="138.43" y="43.18" smashed="yes" rot="R90">
-<attribute name="NAME" x="135.89" y="40.64" size="1.778" layer="95" rot="R90"/>
-<attribute name="VALUE" x="140.97" y="40.64" size="1.778" layer="96" rot="R90" align="top-left"/>
-</instance>
 <instance part="XF1" gate="G$1" x="207.01" y="191.77" smashed="yes">
 <attribute name="NAME" x="204.47" y="194.31" size="1.778" layer="95"/>
@@
 <attribute name="NAME" x="76.2" y="127.635" size="1.778" layer="95"/>
 <attribute name="VALUE" x="76.2" y="116.84" size="1.778" layer="96"/>
+</instance>
+<instance part="F1" gate="G$1" x="138.43" y="43.18" smashed="yes" rot="R90">
+<attribute name="NAME" x="135.89" y="40.64" size="1.778" layer="95" rot="R90"/>
+<attribute name="VALUE" x="140.97" y="40.64" size="1.778" layer="96" align="top-left"/>
 </instance>
 </instances>
@@
 </segment>
 <segment>
-<pinref part="F1" gate="G$1" pin="2"/>
 <wire x1="138.43" y1="45.72" x2="138.43" y2="48.26" width="0.1524" layer="91"/>
 <pinref part="P+6" gate="1" pin="+5V"/>
+<pinref part="F1" gate="G$1" pin="2"/>
+<junction x="138.43" y="45.72"/>
 </segment>
 </net>
@@
 <pinref part="C10" gate="G$1" pin="+"/>
 <wire x1="148.59" y1="27.94" x2="148.59" y2="24.13" width="0.1524" layer="91"/>
+<wire x1="138.43" y1="40.64" x2="138.43" y2="38.1" width="0.1524" layer="91"/>
 <pinref part="F1" gate="G$1" pin="1"/>
-<wire x1="138.43" y1="40.64" x2="138.43" y2="38.1" width="0.1524" layer="91"/>
-</segment>
-</net>
+<junction x="138.43" y="40.64"/>
+</segment>
+</net>

Commit message: made some design review edits
Parts:
- added D2, U$6: DFLS130L-7_30V_1A, Kirbi_ControlBoard:DFLS130L-7_30V_1A
- added R6: 1k, rcl:R-US_R0603
Connections:
- net !CS!: now also R6.1, R6.2
- net +24V: now also D2.C
- net +3V3: now also U$6.A
- net +5V: now also D2.A, U$6.C
Other:
- moved on the sheet: C10, C11, C12, C13, C14, C15, C7, D1, F1, L1, U2

Commit message: made more design review edits
Parts:
- +24V, +3.3V, +5V: value LED-SMD -> Green
- F1: value ERB-RE5R00V -> 5A
- J2, J3: value CONNECTOR -> CONNECTORESC_CONNECTOR; device CurrentSensing:CONNECTOR -> CurrentSensing:CONNECTORESC_CONNECTOR
- R3: value 100Ω -> 100
- R4: value 200Ω -> 200
- R5: value 1200Ω -> 1200
- XF1, XF2: value 3550(2) -> 40A
- renumbered U$6 to D3
Connections:
- net !CNVST! renamed !START!
- net AIN0 renamed L_MOTOR
- net AIN1 renamed R_MOTOR
- net N1 renamed L_ESC
- net N2 renamed R_ESC
- net P1 renamed I1
- net P2 renamed I2
- net !CS!: no longer R6.2
- net +3V3: now also R6.2
- net +5V: now also C1.1, C2.1; no longer C1.2, C2.2
- net GND: now also C1.2, C2.2, U1.AIN2, U1.AIN3; no longer C1.1, C2.1
Other:
- moved on the sheet: C1, C2, C3, C4, C6, C8, C9, J1, J2, J3, JP1, R1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

Commit message: added TVSDIODE
Parts:
- added D4: TVSDIODE, CurrentSensing:TVSDIODE
Connections:
- net +24V: now also D4.C
- net GND: now also D4.A
Changed lines of the file:
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@@
 <part name="J2" library="CurrentSensing" deviceset="CONNECTOR" device="ESC_CONNECTOR" value=""/>
 <part name="J3" library="CurrentSensing" deviceset="CONNECTOR" device="ESC_CONNECTOR" value=""/>
+<part name="D4" library="CurrentSensing" deviceset="TVSDIODE" device=""/>
 </parts>
 <sheets>
@@
 <attribute name="VALUE" x="82.55" y="116.84" size="1.778" layer="96"/>
 </instance>
+<instance part="D4" gate="G$1" x="16.51" y="35.56" smashed="yes">
+<attribute name="NAME" x="19.05" y="35.56" size="1.778" layer="95"/>
+<attribute name="VALUE" x="12.7" y="27.94" size="1.778" layer="96" rot="R90"/>
+</instance>
 </instances>
 <busses>
@@
 <wire x1="26.67" y1="21.59" x2="26.67" y2="24.13" width="0.1524" layer="91"/>
 <junction x="26.67" y="24.13"/>
+<pinref part="D4" gate="G$1" pin="A"/>
+<wire x1="16.51" y1="30.48" x2="16.51" y2="24.13" width="0.1524" layer="91"/>
+<wire x1="16.51" y1="24.13" x2="26.67" y2="24.13" width="0.1524" layer="91"/>
 </segment>
 <segment>
@@
 <wire x1="26.67" y1="45.72" x2="82.55" y2="45.72" width="0.1524" layer="91"/>
 <junction x="26.67" y="45.72"/>
-</segment>
-<segment>
+<pinref part="D4" gate="G$1" pin="C"/>
+<wire x1="26.67" y1="45.72" x2="16.51" y2="45.72" width="0.1524" layer="91"/>
+<wire x1="16.51" y1="45.72" x2="16.51" y2="38.1" width="0.1524" layer="91"/>
+</segment>
+<segment>

Commit message: added connectors and M3 holes for mounting
Parts:
- removed JP1: (no value), pinhead:PINHD-1X8/90
- added J4: MOLEX_2.54MM_2PIN, CurrentSensing:MOLEX_2.54MM_2PIN
- added J5: AMPHENOL_2X3_2.54MM, CurrentSensing:AMPHENOL_2X3_2.54MM
Connections:
- net !CS!: now also J5.5; no longer JP1.7
- net !EOC!: now also J5.4; no longer JP1.3
- net !START!: now also J5.2; no longer JP1.2
- net +5V: now also J4.P$1; no longer JP1.1
- net GND: now also J4.P$2; no longer JP1.8
- net MISO: now also J5.6; no longer JP1.4
- net MOSI: now also J5.1; no longer JP1.5
- net SCLK: now also J5.3; no longer JP1.6
Changed lines of the file:
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@@
 <part name="R10" library="rcl" library_urn="urn:adsk.eagle:library:334" deviceset="R-US_" device="R0603" package3d_urn="urn:adsk.eagle:package:23555/3" value="100"/>
 <part name="C3" library="rcl" library_urn="urn:adsk.eagle:library:334" deviceset="C-US" device="C0603" package3d_urn="urn:adsk.eagle:package:23616/2" value="1000pF"/>
-<part name="JP1" library="pinhead" library_urn="urn:adsk.eagle:library:325" deviceset="PINHD-1X8" device="/90" package3d_urn="urn:adsk.eagle:package:22413/2"/>
-<part name="P+3" library="supply1" library_urn="urn:adsk.eagle:library:371" deviceset="+5V" device=""/>
-<part name="GND7" library="SparkFun-PowerSymbols" library_urn="urn:adsk.eagle:library:530" deviceset="GND" device=""/>
 <part name="J1" library="RoboJackets-Connectors" deviceset="XT-60" device="BATT_LABEL"/>
 <part name="GND8" library="supply1" library_urn="urn:adsk.eagle:library:371" deviceset="GND" device=""/>
@@
 <part name="J3" library="CurrentSensing" deviceset="CONNECTOR" device="ESC_CONNECTOR" value=""/>
 <part name="D4" library="CurrentSensing" deviceset="TVSDIODE" device=""/>
+<part name="J5" library="CurrentSensing" deviceset="AMPHENOL_2X3_2.54MM" device=""/>
+<part name="J4" library="CurrentSensing" deviceset="MOLEX_2.54MM_2PIN" device=""/>
+<part name="P+14" library="supply1" library_urn="urn:adsk.eagle:library:371" deviceset="+5V" device=""/>
+<part name="GND2" library="supply1" library_urn="urn:adsk.eagle:library:371" deviceset="GND" device=""/>
 </parts>
 <sheets>
@@
 <wire x1="5.08" y1="2.54" x2="170.18" y2="2.54" width="0.1524" layer="97" style="shortdash"/>
 <wire x1="170.18" y1="2.54" x2="170.18" y2="45.72" width="0.1524" layer="97" style="shortdash"/>
-<wire x1="129.286" y1="165.1" x2="128.778" y2="165.1" width="0.1524" layer="97" style="shortdash"/>
 <text x="8.89" y="85.09" size="5.08" layer="97" ratio="12">Voltage Regulators</text>
 <wire x1="170.18" y1="45.72" x2="170.18" y2="95.25" width="0.1524" layer="97" style="shortdash"/>
@@
 <attribute name="VALUE" x="260.096" y="176.149" size="1.778" layer="96"/>
 </instance>
-<instance part="JP1" gate="A" x="130.81" y="173.99" smashed="yes" rot="MR0">
-<attribute name="NAME" x="137.16" y="187.325" size="1.778" layer="95" rot="MR0"/>
-<attribute name="VALUE" x="137.16" y="161.29" size="1.778" layer="96" rot="MR0"/>
-</instance>
-<instance part="P+3" gate="1" x="139.7" y="189.23" smashed="yes" rot="MR0">
-<attribute name="VALUE" x="142.24" y="184.15" size="1.778" layer="96" rot="MR90"/>
-</instance>
-<instance part="GND7" gate="1" x="139.7" y="161.29" smashed="yes" rot="MR0">
-<attribute name="VALUE" x="139.7" y="161.036" size="1.778" layer="96" rot="MR0" align="top-center"/>
-</instance>
 <instance part="J1" gate="G$1" x="26.67" y="121.92" smashed="yes">
 <attribute name="NAME" x="20.32" y="127.635" size="1.778" layer="95"/>
@@
 <attribute name="NAME" x="19.05" y="35.56" size="1.778" layer="95"/>
 <attribute name="VALUE" x="12.7" y="27.94" size="1.778" layer="96" rot="R90"/>
+</instance>
+<instance part="J5" gate="G$1" x="138.43" y="165.1" smashed="yes">
+<attribute name="VALUE" x="134.62" y="157.48" size="1.778" layer="96"/>
+<attribute name="NAME" x="134.62" y="170.942" size="1.778" layer="95"/>
+</instance>
+<instance part="J4" gate="G$1" x="138.43" y="184.15" smashed="yes">
+<attribute name="NAME" x="134.62" y="190.754" size="1.778" layer="95"/>
+<attribute name="VALUE" x="134.366" y="176.53" size="1.778" layer="95"/>
+</instance>
+<instance part="P+14" gate="1" x="149.86" y="193.04" smashed="yes">
+<attribute name="VALUE" x="147.32" y="187.96" size="1.778" layer="96" rot="R90"/>
+</instance>
+<instance part="GND2" gate="1" x="149.86" y="175.26" smashed="yes">
+<attribute name="VALUE" x="147.32" y="172.72" size="1.778" layer="96"/>
 </instance>
 </instances>
@@
 <wire x1="67.31" y1="60.96" x2="67.31" y2="53.34" width="0.1524" layer="91"/>
 <junction x="85.09" y="53.34"/>
-</segment>
-<segment>
-<pinref part="JP1" gate="A" pin="8"/>
-<pinref part="GND7" gate="1" pin="GND"/>
-<wire x1="139.7" y1="163.83" x2="139.7" y2="166.37" width="0.1524" layer="91"/>
-<wire x1="139.7" y1="166.37" x2="133.35" y2="166.37" width="0.1524" layer="91"/>
 </segment>
 <segment>
@@
 <junction x="257.81" y="128.27"/>
 </segment>
+<segment>
+<pinref part="J4" gate="G$1" pin="P$2"/>
+<wire x1="146.05" y1="181.61" x2="149.86" y2="181.61" width="0.1524" layer="91"/>
+<wire x1="149.86" y1="181.61" x2="149.86" y2="177.8" width="0.1524" layer="91"/>
+<pinref part="GND2" gate="1" pin="GND"/>
+</segment>
 </net>
 <net name="+5V" class="0">
@@
 </segment>
 <segment>
-<pinref part="JP1" gate="A" pin="1"/>
-<wire x1="133.35" y1="184.15" x2="139.7" y2="184.15" width="0.1524" layer="91"/>
-<pinref part="P+3" gate="1" pin="+5V"/>
-<wire x1="139.7" y1="186.69" x2="139.7" y2="184.15" width="0.1524" layer="91"/>
-</segment>
-<segment>
 <pinref part="P+10" gate="1" pin="+5V"/>
 <pinref part="R4" gate="G$1" pin="2"/>
@@
 <junction x="236.22" y="118.11"/>
 </segment>
+<segment>
+<pinref part="J4" gate="G$1" pin="P$1"/>
+<wire x1="146.05" y1="186.69" x2="149.86" y2="186.69" width="0.1524" layer="91"/>
+<wire x1="149.86" y1="186.69" x2="149.86" y2="190.5" width="0.1524" layer="91"/>
+<pinref part="P+14" gate="1" pin="+5V"/>
+</segment>
 </net>
 <net name="!EOC!" class="0">
@@
 </segment>
 <segment>
-<label x="139.7" y="179.07" size="1.27" layer="95" rot="MR180" xref="yes"/>
-<pinref part="JP1" gate="A" pin="3"/>
-<wire x1="139.7" y1="179.07" x2="133.35" y2="179.07" width="0.1524" layer="91"/>
+<pinref part="J5" gate="G$1" pin="4"/>
+<wire x1="130.81" y1="165.1" x2="128.27" y2="165.1" width="0.1524" layer="91"/>
+<label x="128.27" y="165.1" size="1.27" layer="95" rot="R180" xref="yes"/>
 </segment>
 </net>
@@
 </segment>
 <segment>
-<label x="139.7" y="176.53" size="1.27" layer="95" rot="MR180" xref="yes"/>
-<pinref part="JP1" gate="A" pin="4"/>
-<wire x1="139.7" y1="176.53" x2="133.35" y2="176.53" width="0.1524" layer="91"/>
+<pinref part="J5" gate="G$1" pin="6"/>
+<wire x1="130.81" y1="167.64" x2="128.27" y2="167.64" width="0.1524" layer="91"/>
+<label x="128.27" y="167.64" size="1.27" layer="95" rot="R180" xref="yes"/>
 </segment>
 </net>
@@
 </segment>
 <segment>
-<label x="139.7" y="173.99" size="1.27" layer="95" rot="MR180" xref="yes"/>
-<pinref part="JP1" gate="A" pin="5"/>
-<wire x1="139.7" y1="173.99" x2="133.35" y2="173.99" width="0.1524" layer="91"/>
+<pinref part="J5" gate="G$1" pin="1"/>
+<wire x1="146.05" y1="162.56" x2="148.59" y2="162.56" width="0.1524" layer="91"/>
+<label x="148.59" y="162.56" size="1.27" layer="95" xref="yes"/>
 </segment>
 </net>
@@
 </segment>
 <segment>
-<pinref part="JP1" gate="A" pin="6"/>
-<wire x1="139.7" y1="171.45" x2="133.35" y2="171.45" width="0.1524" layer="91"/>
-<label x="139.7" y="171.45" size="1.27" layer="95" rot="MR180" xref="yes"/>
+<pinref part="J5" gate="G$1" pin="3"/>
+<wire x1="146.05" y1="165.1" x2="148.59" y2="165.1" width="0.1524" layer="91"/>
+<label x="148.59" y="165.1" size="1.27" layer="95" xref="yes"/>
 </segment>
 </net>
@@
 </segment>
 <segment>
-<label x="139.7" y="168.91" size="1.27" layer="95" rot="MR180" xref="yes"/>
-<pinref part="JP1" gate="A" pin="7"/>
-<wire x1="139.7" y1="168.91" x2="133.35" y2="168.91" width="0.1524" layer="91"/>
+<pinref part="J5" gate="G$1" pin="5"/>
+<wire x1="146.05" y1="167.64" x2="148.59" y2="167.64" width="0.1524" layer="91"/>
+<label x="148.59" y="167.64" size="1.27" layer="95" xref="yes"/>
 </segment>
 </net>
@@
 </segment>
 <segment>
-<label x="139.7" y="181.61" size="1.27" layer="95" rot="MR180" xref="yes"/>
-<pinref part="JP1" gate="A" pin="2"/>
-<wire x1="139.7" y1="181.61" x2="133.35" y2="181.61" width="0.1524" layer="91"/>
-</segment>
-</net>
+<pinref part="J5" gate="G$1" pin="2"/>
+<wire x1="130.81" y1="162.56" x2="128.27" y2="162.56" width="0.1524" layer="91"/>
+<label x="128.27" y="162.56" size="1.27" layer="95" rot="R180" xref="yes"/>
+</segment>
+</net>

Commit message: updated device descriptions
Other:
- moved on the sheet: J4
Changed lines of the file:
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@@
 <wire x1="87.63" y1="45.72" x2="140.97" y2="45.72" width="0.1524" layer="91"/>
 <wire x1="140.97" y1="45.72" x2="140.97" y2="43.18" width="0.1524" layer="91"/>
+<junction x="140.97" y="45.72"/>
 </segment>
 <segment>
@@
 <pinref part="U1" gate="A" pin="VDD"/>
 <pinref part="+3V1" gate="G$1" pin="+3V3"/>
-<wire x1="82.55" y1="179.07" x2="106.68" y2="179.07" width="0.1524" layer="91"/>
 <wire x1="106.68" y1="179.07" x2="106.68" y2="180.34" width="0.1524" layer="91"/>
 <pinref part="C6" gate="G$1" pin="1"/>
 <junction x="106.68" y="179.07"/>
+<wire x1="82.55" y1="179.07" x2="106.68" y2="179.07" width="0.1524" layer="91"/>
 </segment>
 <segment>

Commit message: Fixed Diodes on Kirbi, Gucci, and PD Board
Fixed Diodes (DFLS130L-7) on Kirbi, Gucci, and PD Board from Kirbi Library
Parts:
- D2, D3: value DFLS130L-7_30V_1A -> 30; device Kirbi_ControlBoard:DFLS130L-7_30V_1A -> Kirbi_ControlBoard:DFLS130L-7
Changed lines of the file:
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@@
 <?xml version="1.0" encoding="utf-8"?>
 <!DOCTYPE eagle SYSTEM "eagle.dtd">
-<eagle version="9.5.2">
+<eagle version="9.5.1">
 <drawing>
 <settings>
@@
 <part name="XF1" library="CurrentSensing" deviceset="3550(2)" device="" value="40A"/>
 <part name="F1" library="CurrentSensing" deviceset="ERB-RE5R00V" device="" value="5A"/>
-<part name="D2" library="Kirbi_ControlBoard" deviceset="DFLS130L-7_30V_1A" device=""/>
-<part name="D3" library="Kirbi_ControlBoard" deviceset="DFLS130L-7_30V_1A" device=""/>
+<part name="D2" library="Kirbi_ControlBoard" deviceset="DFLS130L-7" device="" value="30"/>
+<part name="D3" library="Kirbi_ControlBoard" deviceset="DFLS130L-7" device="" value="30"/>
 <part name="R6" library="rcl" library_urn="urn:adsk.eagle:library:334" deviceset="R-US_" device="R0603" package3d_urn="urn:adsk.eagle:package:23555/3" value="1k"/>
 <part name="+3V3" library="supply1" library_urn="urn:adsk.eagle:library:371" deviceset="+3V3" device=""/>
@@
 </instance>
 <instance part="D3" gate="G$1" x="85.09" y="78.74" smashed="yes" rot="R180">
-<attribute name="NAME" x="91.44" y="77.47" size="1.27" layer="95" rot="R180"/>
+<attribute name="NAME" x="86.36" y="82.55" size="1.27" layer="95" rot="R180"/>
 <attribute name="VALUE" x="86.36" y="76.2" size="1.27" layer="96" rot="R180"/>
 </instance>
