File: Spici/v1 pcb/Spici_ControlBoard.brd (EAGLE design)
At the start: 66 x 56 mm, 81 parts, among them U1 TEENSY_3.6, U2 ICM-20948, U3 PCA9306, U4 RFM69HCW_SMT, U5 LM393ADR, U6 AP2114H-1.8TRG1, U7 AP2114H-3.3TRG1

Commit message: Added Decoder and Encoder to Spici Schematic
Added Decoder and Encoder Pin connectors to Spici schematic, added connections
Parts:
- added J1: PINHD-2X5_SMD, Spici_ControlBoard:PINHD-2X5_SMD
- added R21: 100K, Spici_ControlBoard:0603
- added U8: LS7184N-S, Spici_ControlBoard:8-SOIC
Connections:
- new net DECCLK: U1.36/A17, U8.8
- new net DECMODE: U1.27, U8.6
- new net DECUPDN: U1.26, U8.7
- new net ENCA: J1.P$6, U8.4
- new net ENCB: J1.P$8, U8.5
- new net ENCINDEX: J1.P$10, U1.28
- new net N$13: R21.2, U8.1
- net +5V: now also J1.P$2, U8.2
- net GND: now also J1.P$3, R21.1, U8.3

Commit message: Fixed Encoder Pin Layout and Added another Encoder and Decoder to Spici Schematic
Parts:
- added J2: PINHD-2X5_SMD, Spici_ControlBoard:PINHD-2X5_SMD
- added R22: 100K, Spici_ControlBoard:0603
- added R23, R27: 2k, SparkFun-Resistors:0603
- added R26, R28: 3k, SparkFun-Resistors:0603
- added U9: LS7184N-S, Spici_ControlBoard:8-SOIC
- moved J1 88.8 mm to (45.0, 52.0)
Connections:
- new net DECCLK2: U1.5, U9.8
- new net DECMODE2: U1.24, U9.6
- new net DECUPDN2: U1.39/A20, U9.7
- new net ENCA2: J2.P$8, U9.4
- new net ENCB2: J2.P$7, U9.5
- new net ENCINDEX2: R27.1, R28.2, U1.20/A6
- new net N$10: R22.2, U9.1
- new net N$12: J2.P$6, R27.2
- new net N$14: J1.P$6, R23.2
- net +5V: now also J1.P$10, J2.P$10, U9.2; no longer J1.P$2
- net ENCA: now also J1.P$8; no longer J1.P$6
- net ENCB: now also J1.P$7; no longer J1.P$8
- net ENCINDEX: now also R23.1, R26.2; no longer J1.P$10
- net GND: now also J1.P$2, J2.P$2, R22.1, R26.1, R28.1, U9.3; no longer J1.P$3
Other:
- board size 66 x 56 mm -> 66 x 64 mm

Commit message: Put Parts On Spici Board
Placed new parts on the board in eagle for spici
Parts:
- moved R28 138.8 mm to (45.0, 62.0), turned to 270 degrees
- moved R27 136.8 mm to (47.0, 62.0), turned to 90 degrees
- moved R26 135.0 mm to (49.0, 62.0), turned to 90 degrees
- moved R23 133.2 mm to (51.0, 62.0), turned to 270 degrees
- moved J2 110.3 mm to (45.0, 52.0), turned to 180 degrees
- moved U9 94.4 mm to (26.0, 60.0)
- moved R22 94.0 mm to (17.0, 59.0)
- moved R21 86.1 mm to (17.0, 62.0)
- moved U8 82.0 mm to (37.0, 60.0)
- flipped J1 to the bottom

Commit message: Shifted some parts
Shifted some parts, (moved power button down, extended ground and 5v plane)
Parts:
- moved J1 52.7 mm to (-7.20, 59.4), flipped to the top
- moved R1 4.43 mm to (-7.30, 43.8)
- moved 5V 3.39 mm to (-12.0, 45.6), turned to 270 degrees
- moved POWER_SWITCH 1.66 mm to (-6.90, 51.2)
- moved C6 0.45 mm to (-7.10, 41.9)
Routing:
- net N$8: track 1.97 -> 4.69 mm
- net N$6: track 12.6 -> 11.5 mm
- net GND: track 107.0 -> 106.2 mm
- net +5V: track 46.8 -> 46.3 mm
- added copper zone on layer 15, net 5V
- removed copper zone on layer 15, net +5V

Commit message: Connected new parts
Added routes for the parts added, removed esc connector
Parts:
- removed ESC: 0532610371, Kirbi_ControlBoard:0532610371
- moved R21 14.6 mm to (31.6, 60.8), turned to 90 degrees
- moved R22 4.25 mm to (20.8, 60.9), turned to 90 degrees
- moved R28 2.33 mm to (43.8, 60.0), turned to 90 degrees
- moved R23 2.24 mm to (50.0, 60.0), turned to 90 degrees
- moved R26 2.24 mm to (48.0, 60.0), turned to 270 degrees
- moved R27 2.24 mm to (46.0, 60.0), turned to 270 degrees
Connections:
- net GND: no longer ESC.3
- net S1/TRX: no longer ESC.2
- net S1/TTX: no longer ESC.1
Routing:
- net ENCINDEX2: track 0.00 -> 61.1 mm
- net DECCLK2: track 0.00 -> 59.4 mm, vias 0 -> 2
- net N$14: track 0.00 -> 55.1 mm
- net DECUPDN: track 0.00 -> 50.3 mm, vias 0 -> 2
- net ENCB: track 0.00 -> 48.7 mm, vias 0 -> 2
- net ENCA: track 0.00 -> 45.2 mm, vias 0 -> 2
- net ENCINDEX: track 0.00 -> 42.3 mm
- net DECMODE2: track 0.00 -> 40.2 mm
- net DECMODE: track 0.00 -> 38.1 mm, vias 0 -> 6
- net DECCLK: track 0.00 -> 37.7 mm, vias 0 -> 2
- net ENCA2: track 0.00 -> 35.3 mm, vias 0 -> 2
- net ENCB2: track 0.00 -> 21.9 mm
- net DECUPDN2: track 0.00 -> 21.3 mm, vias 0 -> 2
- net GND: track 106.2 -> 121.0 mm, vias 52 -> 59
- net N$12: track 0.00 -> 14.4 mm
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
Commit message: Fixed ratsnest
Edited polygons and made some more route adjustments
Routing:
- added copper zone on layer 15, net +5V
- removed copper zone on layer 15, net 5V
Changed lines of the file:
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@@
 <wire x1="-9.74" y1="58.36" x2="-8.6" y2="59.5" width="0.2" layer="1"/>
 <via x="-8.6" y="59.5" extent="1-16" drill="0.4"/>
-<wire x1="48" y1="57" x2="48" y2="60.85" width="0" layer="19" extent="1-1"/>
-<wire x1="44" y1="57.8" x2="48" y2="57" width="0" layer="19" extent="1-1"/>
-<wire x1="36" y1="58.838" x2="43.8" y2="59.15" width="0" layer="19" extent="1-1"/>
-<wire x1="32" y1="58.524" x2="34.3" y2="59.365" width="0" layer="19" extent="1-1"/>
-<wire x1="25" y1="59.838" x2="31.6" y2="59.95" width="0" layer="19" extent="1-1"/>
-<wire x1="21" y1="58.5" x2="23.3" y2="59.365" width="0" layer="19" extent="1-1"/>
-<wire x1="18.95" y1="54" x2="21" y2="58.5" width="0" layer="19" extent="1-1"/>
-<wire x1="26.73" y1="53.27" x2="25" y2="59.838" width="0" layer="19" extent="1-1"/>
-<wire x1="25.62" y1="45.62" x2="26.73" y2="53.27" width="0" layer="19" extent="1-1"/>
-<wire x1="26.4" y1="43.4" x2="25.62" y2="45.62" width="0" layer="19" extent="1-1"/>
-<wire x1="25.9" y1="34.75" x2="25.85" y2="42" width="0" layer="19" extent="1-1"/>
-<wire x1="28.4" y1="34.75" x2="27.2" y2="34.8" width="0" layer="19" extent="1-1"/>
-<wire x1="32.3" y1="28.6302" x2="29.7" y2="34.8" width="0" layer="19" extent="1-1"/>
-<wire x1="29.75" y1="27" x2="30.85" y2="28" width="0" layer="19" extent="1-16"/>
-<wire x1="33.45" y1="27" x2="32.3" y2="28.6302" width="0" layer="19" extent="1-1"/>
-<wire x1="27.5" y1="21.2" x2="29.3" y2="25.8" width="0" layer="19" extent="1-1"/>
-<wire x1="27.1" y1="18.8" x2="27.95" y2="19.9" width="0" layer="19" extent="1-16"/>
-<wire x1="25.5" y1="17.6" x2="25.5" y2="18.6" width="0" layer="19" extent="1-1"/>
-<wire x1="22.8" y1="19.455" x2="23.6" y2="19.455" width="0" layer="19" extent="1-1"/>
-<wire x1="25.4" y1="22.4" x2="27.5" y2="21.2" width="0" layer="19" extent="1-1"/>
-<wire x1="23.6" y1="22.545" x2="24.545" y2="22" width="0" layer="19" extent="1-1"/>
-<wire x1="22.7" y1="26.8" x2="24.8" y2="23.5" width="0" layer="19" extent="1-1"/>
-<wire x1="23.4" y1="13.4" x2="24.15" y2="17.3" width="0" layer="19" extent="1-1"/>
-<wire x1="17" y1="17.45" x2="21.1" y2="18.2" width="0" layer="19" extent="1-1"/>
-<wire x1="15.1" y1="17.1" x2="15.7" y2="15.9" width="0" layer="19" extent="1-1"/>
-<wire x1="15" y1="20.6698" x2="13.9" y2="18.025" width="0" layer="19" extent="1-1"/>
-<wire x1="13.8" y1="26.3" x2="16.45" y2="21.95" width="0" layer="19" extent="16-16"/>
-<wire x1="32.55" y1="16.6" x2="27.95" y2="19.9" width="0" layer="19" extent="1-1"/>
-<wire x1="34.9" y1="14.7" x2="33.4" y2="14.7" width="0" layer="19" extent="1-1"/>
-<wire x1="29.73" y1="12.27" x2="33.4" y2="14.7" width="0" layer="19" extent="1-1"/>
-<wire x1="39.8" y1="15.7556" x2="35" y2="17.1" width="0" layer="19" extent="1-1"/>
-<wire x1="41.640875" y1="10.8012" x2="39.8" y2="15.7556" width="0" layer="19" extent="1-1"/>
-<wire x1="37.85" y1="5.1" x2="40.1629125" y2="8.83446875" width="0" layer="19" extent="1-1"/>
-<wire x1="14.4" y1="10.35" x2="15.7" y2="15.9" width="0" layer="19" extent="1-1"/>
-<wire x1="15.3" y1="8.5" x2="13.7" y2="8.9" width="0" layer="19" extent="1-1"/>
-<wire x1="14.1" y1="5.6" x2="15.3" y2="8.5" width="0" layer="19" extent="1-1"/>
-<wire x1="10.85" y1="5.1" x2="10.9" y2="6.8" width="0" layer="19" extent="1-16"/>
-<wire x1="8.3" y1="5.05" x2="10.85" y2="5.1" width="0" layer="19" extent="1-16"/>
-<wire x1="3.725" y1="5" x2="8.3" y2="5.05" width="0" layer="19" extent="1-16"/>
-<wire x1="-1" y1="7" x2="2.3327625" y2="5.1944" width="0" layer="19" extent="1-1"/>
-<wire x1="46.601040625" y1="16.201040625" x2="40" y2="17.1" width="0" layer="19" extent="1-1"/>
-<wire x1="47" y1="19" x2="47.6" y2="17.1" width="0" layer="19" extent="1-1"/>
-<wire x1="47.007415625" y1="27.149965625" x2="47.1" y2="20.125" width="0" layer="19" extent="1-1"/>
-<wire x1="18" y1="34" x2="21.85" y2="28" width="0" layer="19" extent="16-16"/>
-<wire x1="30.625" y1="5" x2="37.85" y2="5.1" width="0" layer="19" extent="1-1"/>
-<wire x1="5.73" y1="12.27" x2="-0.49895625" y2="8.39895625" width="0" layer="19" extent="1-1"/>
-<wire x1="3.8" y1="14.9" x2="5.73" y2="12.27" width="0" layer="19" extent="1-1"/>
-<wire x1="6.3" y1="18.35" x2="3" y2="17.1" width="0" layer="19" extent="1-1"/>
-<wire x1="-2" y1="17.1" x2="3" y2="17.1" width="0" layer="19" extent="1-1"/>
-<wire x1="-6.322428125" y1="13.386225" x2="-2" y2="15.7" width="0" layer="19" extent="1-1"/>
-<wire x1="-8.6" y1="16.15" x2="-7.4" y2="14.4" width="0" layer="19" extent="1-1"/>
-<wire x1="-2" y1="22.15" x2="-2" y2="17.1" width="0" layer="19" extent="1-16"/>
-<wire x1="-5" y1="25" x2="-6.6" y2="24" width="0" layer="19" extent="1-1"/>
-<wire x1="-9.1" y1="23.875" x2="-6.6" y2="24" width="0" layer="19" extent="1-1"/>
-<wire x1="-9.94" y1="30.38" x2="-9" y2="25" width="0" layer="19" extent="1-1"/>
-<wire x1="-9.8" y1="37.5" x2="-9.94" y2="30.38" width="0" layer="19" extent="1-1"/>
-<wire x1="-6.3" y1="37.45" x2="-8.3" y2="37.45" width="0" layer="19" extent="1-1"/>
-<wire x1="-0.91" y1="36.73" x2="-5.1" y2="37.5" width="0" layer="19" extent="16-16"/>
-<wire x1="-7.95" y1="41.9" x2="-8.3" y2="37.45" width="0" layer="19" extent="1-1"/>
-<wire x1="-6.45" y1="43.8" x2="-7.95" y2="41.9" width="0" layer="19" extent="1-1"/>
-<wire x1="9.8" y1="36.395" x2="18" y2="34" width="0" layer="19" extent="1-1"/>
-<wire x1="8.45" y1="42.3" x2="9.8" y2="36.395" width="0" layer="19" extent="1-1"/>
-<wire x1="11.862" y1="43.6" x2="8.45" y2="42.3" width="0" layer="19" extent="1-1"/>
-<wire x1="-9.74" y1="57.05" x2="-7.4" y2="45.62" width="0" layer="19" extent="1-1"/>
 </signal>
 <signal name="+5V">
@@
 <wire x1="-11" y1="60.47" x2="-11" y2="60" width="0.2" layer="1"/>
 <via x="-11" y="60" extent="1-16" drill="0.4"/>
-<wire x1="36" y1="60" x2="50.08" y2="49.65" width="0" layer="19" extent="1-1"/>
-<wire x1="25" y1="61" x2="34.3" y2="60.635" width="0" layer="19" extent="1-1"/>
-<wire x1="32.5" y1="42.6" x2="36" y2="60" width="0" layer="19" extent="1-1"/>
-<wire x1="29.7" y1="36.1698" x2="30.45" y2="42" width="0" layer="19" extent="1-1"/>
-<wire x1="27.2" y1="36.1698" x2="28.4" y2="36.45" width="0" layer="19" extent="1-1"/>
-<wire x1="23.3" y1="35.975" x2="25.9" y2="36.45" width="0" layer="19" extent="1-1"/>
-<wire x1="23" y1="25" x2="24.162" y2="34" width="0" layer="19" extent="1-1"/>
-<wire x1="15.2" y1="40.205" x2="23.3" y2="35.975" width="0" layer="19" extent="1-1"/>
-<wire x1="8" y1="26.162" x2="21.35" y2="25.25" width="0" layer="19" extent="16-16"/>
-<wire x1="-6.5" y1="17.9" x2="8" y2="26.162" width="0" layer="19" extent="1-1"/>
-<wire x1="-9.1" y1="20.125" x2="-8.6" y2="17.85" width="0" layer="19" extent="1-1"/>
-<wire x1="-3.6340125" y1="10.771853125" x2="-6.5" y2="17.9" width="0" layer="19" extent="1-1"/>
-<wire x1="-4.0386375" y1="9.037575" x2="-5" y2="10" width="0" layer="19" extent="1-1"/>
-<wire x1="7.475" y1="5" x2="-1.701040625" y2="9.601040625" width="0" layer="19" extent="1-1"/>
-<wire x1="8.394" y1="3.4" x2="7.0552" y2="3.39851875" width="0" layer="19" extent="1-1"/>
-<wire x1="-6.3" y1="39.15" x2="7.123" y2="28" width="0" layer="19" extent="1-16"/>
-<wire x1="-6.6" y1="40.6" x2="-5.2" y2="40.9" width="0" layer="19" extent="1-1"/>
-<wire x1="-8.2" y1="40.6" x2="-6.6" y2="40.6" width="0" layer="19" extent="1-1"/>
-<wire x1="-9.94" y1="45.62" x2="-6.25" y2="41.9" width="0" layer="19" extent="1-1"/>
-<wire x1="-6.9" y1="51.2" x2="-9.94" y2="45.62" width="0" layer="19" extent="1-1"/>
-<wire x1="-11" y1="60" x2="-6.9" y2="51.2" width="0" layer="19" extent="1-1"/>
-<wire x1="46.99258125" y1="25.45003125" x2="29.7" y2="36.1698" width="0" layer="19" extent="1-1"/>
-<wire x1="49" y1="23.6" x2="49" y2="24.794" width="0" layer="19" extent="1-1"/>
-<wire x1="45.39895625" y1="14.99895625" x2="47.1" y2="23.875" width="0" layer="19" extent="1-1"/>
-<wire x1="45.3" y1="12" x2="46.14203125" y2="12.649040625" width="0" layer="19" extent="1-1"/>
-<wire x1="36.15" y1="5.1" x2="45.3" y2="12" width="0" layer="19" extent="1-1"/>
-<wire x1="34.362" y1="2.9" x2="35.094" y2="3.5" width="0" layer="19" extent="1-1"/>
+<polygon width="0.2" layer="15">
+<vertex x="-14" y="64"/>
+<vertex x="-14" y="14"/>
+<vertex x="0" y="0"/>
+<vertex x="38" y="0"/>
+<vertex x="52" y="14"/>
+<vertex x="52" y="64"/>
+</polygon>
 </signal>
 <signal name="+3.3V">
@@
 <via x="43.8698" y="44" extent="1-16" drill="0.4"/>
 <wire x1="46.3" y1="48.7" x2="46.5" y2="48.5" width="0.2" layer="1"/>
-<wire x1="46.5" y1="48.5" x2="46.5" y2="47.52478125" width="0.2" layer="1"/>
-<wire x1="44.9891" y1="45.1193" x2="43.8698" y2="44" width="0.2" layer="1"/>
-<wire x1="46.5" y1="47.52478125" x2="44.9891" y2="46.01388125" width="0.2" layer="1"/>
-<wire x1="44.9891" y1="46.01388125" x2="44.9891" y2="45.1193" width="0.2" layer="1"/>
+<wire x1="46.5" y1="48.5" x2="46.5" y2="48.12478125" width="0.2" layer="1"/>
+<wire x1="44.6891" y1="44.8193" x2="43.8698" y2="44" width="0.2" layer="1"/>
+<wire x1="46.5" y1="48.12478125" x2="44.6891" y2="46.31388125" width="0.2" layer="1"/>
+<wire x1="44.6891" y1="46.31388125" x2="44.6891" y2="44.8193" width="0.2" layer="1"/>
 <wire x1="43.8698" y1="44" x2="43.8698" y2="39.8698" width="0.2" layer="16"/>
 <wire x1="43.8698" y1="39.8698" x2="42" y2="38" width="0.2" layer="16"/>
@@
 <wire x1="-2.12" y1="61.88" x2="-2.12" y2="61.75" width="0.2" layer="1"/>
 </signal>
-<signal name="5V">
-<polygon width="0.2" layer="15">
-<vertex x="-14" y="64"/>
-<vertex x="-14" y="14"/>
-<vertex x="0" y="0"/>
-<vertex x="38" y="0"/>
-<vertex x="52" y="14"/>
-<vertex x="52" y="64"/>
-</polygon>
-</signal>
 </signals>

Commit message: molex
add molex connector
Parts:
- added U$2: 0532610671, Spici_ControlBoard:0532610671
Changed lines of the file:
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@@
 <attribute name="VALUE" x="44.562" y="60" size="0.6096" layer="27" font="vector" ratio="20" rot="R90" align="top-center"/>
+</element>
+<element name="U$2" library="Spici_ControlBoard" package="0532610671" value="0532610671" x="-9" y="-8" smashed="yes">
+<attribute name="DKPN" value="WM7624TR-ND" x="-9" y="-8" size="1.778" layer="27" display="off"/>
+<attribute name="NAME" x="-14.27" y="-4" size="1" layer="25" font="vector" ratio="10"/>
+<attribute name="VALUE" x="-14.27" y="-12.27" size="1" layer="27" font="vector" ratio="10" align="top-left"/>
 </element>
 </elements>
