File: Spici/v1 pcb/Spici_ControlBoard.sch (EAGLE design)
At the start: 78 parts, among them U1 TEENSY_3.6, U2 ICM-20948, U3 PCA9306, U4 RFM69HCW_SMT, U5 LM393ADR, U6 AP2114H-1.8TRG1, U7 AP2114H-3.3TRG1

Commit message: Added Decoder and Encoder to Spici Schematic
Added Decoder and Encoder Pin connectors to Spici schematic, added connections
Parts:
- added J1: PINHD-2X5_SMD, Spici_ControlBoard:PINHD-2X5_SMD
- added R21: 100K, Spici_ControlBoard:100KOHM-0603-1/10W-5%
- added U8: LS7184N-S, Spici_ControlBoard:LS7184N-S
Connections:
- new net DECCLK: U1.36/A17/PWM, U8.!CLK
- new net DECMODE: U1.27, U8.MODE
- new net DECUPDN: U1.26, U8.UP/!DN
- new net ENCA: J1.P$6, U8.A
- new net ENCB: J1.P$8, U8.B
- new net ENCINDEX: J1.P$10, U1.28
- new net N$13: R21.2, U8.RBIAS
- net +5V: now also J1.P$2, U8.VDD
- net GND: now also J1.P$3, R21.1, U8.VSS
Other:
- note added: "Quadrature Encoder/Decoder"

Commit message: Fixed Encoder Pin Layout and Added another Encoder and Decoder to Spici Schematic
Parts:
- added J2: PINHD-2X5_SMD, Spici_ControlBoard:PINHD-2X5_SMD
- added R22: 100K, Spici_ControlBoard:100KOHM-0603-1/10W-5%
- added R23, R27: 2k, SparkFun-Resistors:1KOHM-0603-1/10W-1%
- added R26, R28: 3k, SparkFun-Resistors:1KOHM-0603-1/10W-1%
- added U9: LS7184N-S, Spici_ControlBoard:LS7184N-S
Connections:
- new net DECCLK2: U1.5/PWM, U9.!CLK
- new net DECMODE2: U1.24, U9.MODE
- new net DECUPDN2: U1.39/A20, U9.UP/!DN
- new net ENCA2: J2.P$8, U9.A
- new net ENCB2: J2.P$7, U9.B
- new net ENCINDEX2: R27.1, R28.2, U1.20/A6/PWM
- new net N$10: R22.2, U9.RBIAS
- new net N$12: J2.P$6, R27.2
- new net N$14: J1.P$6, R23.2
- net +5V: now also J1.P$10, J2.P$10, U9.VDD; no longer J1.P$2
- net ENCA: now also J1.P$8; no longer J1.P$6
- net ENCB: now also J1.P$7; no longer J1.P$8
- net ENCINDEX: now also R23.1, R26.2; no longer J1.P$10
- net GND: now also J1.P$2, J2.P$2, R22.1, R26.1, R28.1, U9.VSS; no longer J1.P$3

Commit message: Connected new parts
Added routes for the parts added, removed esc connector
Parts:
- removed ESC: 0532610371, Kirbi_ControlBoard:0532610371
Connections:
- net GND: no longer ESC.1
- net S1/TRX: no longer ESC.2
- net S1/TTX: no longer ESC.3
Changed lines of the file:
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@@
 <part name="POWER_CONN" library="Kirbi_ControlBoard" deviceset="1719770002" device=""/>
 <part name="C12" library="SparkFun-Capacitors" library_urn="urn:adsk.eagle:library:510" deviceset="0.1UF" device="-0603-25V-(+80/-20%)" package3d_urn="urn:adsk.eagle:package:37414/1" value="0.1uF"/>
-<part name="ESC" library="Kirbi_ControlBoard" deviceset="0532610371" device=""/>
-<part name="GND21" library="SparkFun-PowerSymbols" library_urn="urn:adsk.eagle:library:530" deviceset="GND" device=""/>
 <part name="F1" library="Kirbi_ControlBoard" deviceset="C1F3.5" device="" value="3.5"/>
 <part name="R2" library="Kirbi_ControlBoard" deviceset="6.2OHM" device="-0603-1/10W-5%" package3d_urn="urn:adsk.eagle:package:39650/1" value="6.2"/>
@@
 <attribute name="VALUE" x="59.944" y="226.441" size="1.778" layer="96" font="vector"/>
 </instance>
-<instance part="ESC" gate="G$1" x="271.78" y="149.86" smashed="yes">
-<attribute name="VALUE" x="269.24" y="142.494" size="1.778" layer="96" font="vector"/>
-<attribute name="NAME" x="269.24" y="155.448" size="1.778" layer="95" font="vector"/>
-</instance>
-<instance part="GND21" gate="1" x="279.908" y="136.906" smashed="yes">
-<attribute name="VALUE" x="279.908" y="136.652" size="1.778" layer="96" align="top-center"/>
-</instance>
 <instance part="F1" gate="G$1" x="279.4" y="104.14" smashed="yes">
 <attribute name="NAME" x="276.86" y="106.68" size="1.778" layer="95"/>
@@
 </segment>
 <segment>
-<pinref part="ESC" gate="G$1" pin="1"/>
-<pinref part="GND21" gate="1" pin="GND"/>
-<wire x1="279.4" y1="147.32" x2="279.908" y2="147.32" width="0.1524" layer="91"/>
-<wire x1="279.908" y1="147.32" x2="279.908" y2="139.446" width="0.1524" layer="91"/>
-</segment>
-<segment>
 <pinref part="C11" gate="G$1" pin="2"/>
 <pinref part="GND27" gate="1" pin="GND"/>
@@
 <label x="160.02" y="152.4" size="1.778" layer="95" rot="R180" xref="yes"/>
 </segment>
-<segment>
-<pinref part="ESC" gate="G$1" pin="3"/>
-<wire x1="279.4" y1="152.4" x2="284.48" y2="152.4" width="0.1524" layer="91"/>
-<label x="284.48" y="152.4" size="1.778" layer="95" rot="R90" xref="yes"/>
-</segment>
 </net>
 <net name="S1/TRX" class="0">
@@
 <wire x1="165.1" y1="149.86" x2="160.02" y2="149.86" width="0.1524" layer="91"/>
 <label x="160.02" y="149.86" size="1.778" layer="95" rot="MR0" xref="yes"/>
-</segment>
-<segment>
-<pinref part="ESC" gate="G$1" pin="2"/>
-<wire x1="279.4" y1="149.86" x2="289.56" y2="149.86" width="0.1524" layer="91"/>
-<label x="289.56" y="149.86" size="1.778" layer="95" rot="R90" xref="yes"/>
 </segment>
 </net>
@@
 </sheet>
 </sheets>
-<errors>
-</errors>
 </schematic>
 </drawing>

Commit message: molex
add molex connector
Parts:
- added U$2: 0532610671, Spici_ControlBoard:0532610671
Other:
- note added: "Connectors (to PDB)"
Changed lines of the file:
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@@
 <part name="R28" library="SparkFun-Resistors" library_urn="urn:adsk.eagle:library:532" deviceset="1KOHM" device="-0603-1/10W-1%" package3d_urn="urn:adsk.eagle:package:39650/1" value="3k"/>
 <part name="GND39" library="SparkFun-PowerSymbols" library_urn="urn:adsk.eagle:library:530" deviceset="GND" device=""/>
+<part name="U$2" library="Spici_ControlBoard" deviceset="0532610671" device=""/>
 </parts>
 <sheets>
@@
 <plain>
 <text x="10.16" y="231.14" size="6.4516" layer="97">Quadrature Encoder/Decoder</text>
+<text x="58.42" y="266.7" size="6.4516" layer="97">Connectors (to PDB)</text>
 </plain>
 <instances>
@@
 <attribute name="VALUE" x="160.02" y="127.762" size="1.778" layer="96" align="top-center"/>
 </instance>
+<instance part="U$2" gate="G$1" x="91.44" y="251.46" smashed="yes">
+<attribute name="VALUE" x="88.9" y="243.84" size="1.778" layer="96" align="top-left"/>
+<attribute name="NAME" x="88.9" y="259.08" size="1.778" layer="95"/>
+</instance>
 </instances>
