File: ShawtiBoard/RatatoulliBoard/RatatoulliBoard.kicad_sch (KiCad schematic)
At the start: 50 parts, among them IC1 TEENSY_4.1, IC2 DRV8212DRLR, IC3 DRV8212DRLR, J1 BDC1, J2 BDC2, J3 LIDAR1, J4 LIDAR2, J5 LIDAR3, J6 LIDAR4, J7 LINE_RF, J8 LINE_LF, J9 Battery, U1 ADP2303ARDZ-R7, U2 ADP2303ARDZ-R7

Commit message: workin on stuff
added extra line sensors, fixed library paths for symbol and footprints as well as board layout
Parts:
- added J10: LINE_RB, phoenix:PhoenixContact_MSTBA_2,5_3-G_1x03_P5.00mm_Horizontal, symbol Connector_Generic:Conn_02x02_Odd_Even
- added J11: LINE_LB, phoenix:PhoenixContact_MSTBA_2,5_3-G_1x03_P5.00mm_Horizontal, symbol Connector_Generic:Conn_02x02_Odd_Even
- C1, C10, C13, C14, C15, C16, C17, C18, C2, C3, C4, C5, C6, C8, C9: footprint Capacitor_SMD:C_0201_0603Metric -> kicadLib:C_0805_2012Metric
- C11, C12, C7: footprint Capacitor_SMD:C_0201_0603Metric -> kicadLib:C_1210_3225Metric
- D3, D4, D5: footprint (none) -> kicadLib:C_0603_1608Metric
- F1, F2: footprint (none) -> kicadLib:C_1206_3216Metric
- IC1: footprint TEENSY41 -> Teensy4:TEENSY41
- J1, J2: footprint (none) -> phoenix:PhoenixContact_MSTBA_2,5_2-G_1x02_P5.00mm_Horizontal
- J3, J4, J5, J6: footprint (none) -> jst:JST_SH_SM04B-SRSS-TB_1x04-1MP_P1.00mm_Horizontal
- J7, J8: footprint (none) -> phoenix:PhoenixContact_MSTBA_2,5_3-G_1x03_P5.00mm_Horizontal
- J9: footprint (none) -> molex:Molex_PicoBlade_53261-0271_1x02-1MP_P1.25mm_Horizontal
- L1, L2: footprint (none) -> Inductor_SMD:L_Bourns_SRP1245A
- R1, R2, R3, R4, R5, R6, R7, R8: footprint (none) -> kicadLib:C_0805_2012Metric
- R9: footprint (none) -> kicadLib:C_0402_1005Metric
Connections:
- net +3.3V: now also J10.1 (Pin_1), J11.1 (Pin_1)
- net GND: now also J10.3 (Pin_3), J11.3 (Pin_3)
- net RB_INT: now reaches IC1.24 (A10)
- net RB_INT: now also J10.2 (Pin_2)
- net LB_INT: now reaches IC1.25 (A11)
- net LB_INT: now also J11.2 (Pin_2)
- no-connect marks 45 -> 41
Other:
- moved on the sheet: C10, C14, C15, C17, C18, C6, C7, D1, D3, D4, D5, F1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

Commit message: updates to 500g
Parts:
- removed J10: LINE_RB, phoenix:PhoenixContact_MSTBA_2,5_3-G_1x03_P5.00mm_Horizontal, symbol Connector_Generic:Conn_02x02_Odd_Even
- removed J11: LINE_LB, phoenix:PhoenixContact_MSTBA_2,5_3-G_1x03_P5.00mm_Horizontal, symbol Connector_Generic:Conn_02x02_Odd_Even
- added SW1: SW_DIP_x03, Button_Switch_SMD:SW_DIP_SPSTx03_Slide_9.78x9.8mm_W8.61mm_P2.54mm, symbol Switch:SW_DIP_x03
- added SW2: SW_SPST, Button_Switch_SMD:SW_SPST_B3S-1100, symbol Switch:SW_SPST
Connections:
- net +12V: now also SW2.1 (A); no longer J9.1 (Pin_1)
- net GND: now also SW1.1, SW1.2, SW1.3
- net at IC1.26 (A12): now also SW1.4
- net LB_INT: no longer names the net of IC1.25 (A11)
- net LB_INT: now also SW1.5
- net RB_INT: no longer names the net of IC1.24 (A10)
- net RB_INT: now also SW1.6
- new net: J9.1 (Pin_1), SW2.2 (B)
- no-connect marks 41 -> 40
Other:
- moved on the sheet: C10, C14, C15, C17, C18, C6, C7, D1, F1, J9, L1, R1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
