File: ShawtiBoard/RatatoulliBoard/RatatoulliBoard.kicad_pcb (KiCad board)
At the start: 2 copper layers, 7 parts, among them IC1 TEENSY_4.1, IC2 DRV8212DRLR, IC3 DRV8212DRLR, U1 ADP2303ARDZ-R7, U2 ADP2303ARDZ-R7

Commit message: workin on stuff
added extra line sensors, fixed library paths for symbol and footprints as well as board layout
Parts:
- added C1: 0.1uF, kicadLib:C_0805_2012Metric, F.Cu at (154.4, 104.0)
- added C10: 0.1uF, kicadLib:C_0805_2012Metric, F.Cu at (116.5, 107.0)
- added C11: 47uF, kicadLib:C_1210_3225Metric, F.Cu at (140.5, 92.0)
- added C12: 47uF, kicadLib:C_1210_3225Metric, F.Cu at (141.5, 86.0)
- added C13: 0.1uF, kicadLib:C_0805_2012Metric, F.Cu at (93.0, 127.0)
- added C14: 0.1uF, kicadLib:C_0805_2012Metric, F.Cu at (137.9, 115.5)
- added C15: 0.1uF, kicadLib:C_0805_2012Metric, F.Cu at (142.4, 57.5)
- added C16: 0.1uF, kicadLib:C_0805_2012Metric, F.Cu at (123.0, 127.6)
- added C17: 0.1uF, kicadLib:C_0805_2012Metric, F.Cu at (141.8, 73.0)
- added C18: 0.1uF, kicadLib:C_0805_2012Metric, F.Cu at (133.5, 121.5)
- added C2: 0.1uF, kicadLib:C_0805_2012Metric, F.Cu at (154.4, 101.0)
- added C3: 10uF, kicadLib:C_0805_2012Metric, F.Cu at (149.5, 72.5)
- added C4: 0.1uF, kicadLib:C_0805_2012Metric, F.Cu at (157.6, 97.7)
- added C5: 0.1uF, kicadLib:C_0805_2012Metric, F.Cu at (169.4, 69.8)
- added C6: 10uF, kicadLib:C_0805_2012Metric, F.Cu at (133.5, 115.5)
- added C7: 47uF, kicadLib:C_1210_3225Metric, F.Cu at (91.4, 119.4)
- added C8: 0.1uF, kicadLib:C_0805_2012Metric, F.Cu at (168.9, 87.5)
- added C9: 0.1uF, kicadLib:C_0805_2012Metric, F.Cu at (164.5, 87.5)
- added D3: GREEN, kicadLib:C_0603_1608Metric, F.Cu at (168.7, 90.2)
- added D4: GREEN, kicadLib:C_0603_1608Metric, F.Cu at (158.6, 100.4)
- added D5: GREEN, kicadLib:C_0603_1608Metric, F.Cu at (163.0, 96.3)
- added F1: 3A, kicadLib:C_1206_3216Metric, F.Cu at (155.0, 82.6)
- added F2: 3A, kicadLib:C_1206_3216Metric, F.Cu at (149.3, 82.6)
- added J1: BDC1, phoenix:PhoenixContact_MSTBA_2,5_2-G_1x02_P5.00mm_Horizontal, F.Cu at (47.0, 40.3)
- added J10: LINE_RB, phoenix:PhoenixContact_MSTBA_2,5_3-G_1x03_P5.00mm_Horizontal, F.Cu at (117.0, 40.8)
- added J11: LINE_LB, phoenix:PhoenixContact_MSTBA_2,5_3-G_1x03_P5.00mm_Horizontal, F.Cu at (65.5, 40.3)
- added J2: BDC2, phoenix:PhoenixContact_MSTBA_2,5_2-G_1x02_P5.00mm_Horizontal, F.Cu at (130.5, 40.8)
- added J3: LIDAR1, jst:JST_SH_SM04B-SRSS-TB_1x04-1MP_P1.00mm_Horizontal, F.Cu at (42.0, 69.0)
- added J4: LIDAR2, jst:JST_SH_SM04B-SRSS-TB_1x04-1MP_P1.00mm_Horizontal, F.Cu at (131.0, 68.5)
- added J5: LIDAR3, jst:JST_SH_SM04B-SRSS-TB_1x04-1MP_P1.00mm_Horizontal, F.Cu at (42.0, 77.5)
- added J6: LIDAR4, jst:JST_SH_SM04B-SRSS-TB_1x04-1MP_P1.00mm_Horizontal, F.Cu at (131.0, 77.0)
- added J7: LINE_RF, phoenix:PhoenixContact_MSTBA_2,5_3-G_1x03_P5.00mm_Horizontal, F.Cu at (111.5, 80.5)
- added J8: LINE_LF, phoenix:PhoenixContact_MSTBA_2,5_3-G_1x03_P5.00mm_Horizontal, F.Cu at (51.0, 80.7)
- added J9: Battery, molex:Molex_PicoBlade_53261-0271_1x02-1MP_P1.25mm_Horizontal, B.Cu at (97.5, 40.0)
- added L1: 4.7uH, Inductor_SMD:L_Bourns_SRP1245A, B.Cu at (64.5, 71.5)
- added L2: 4.7uH, Inductor_SMD:L_Bourns_SRP1245A, F.Cu at (113.5, 55.5)
- added R1: 100k, kicadLib:C_0805_2012Metric, F.Cu at (164.5, 90.5)
- added R2: 52.3k, kicadLib:C_0805_2012Metric, F.Cu at (164.9, 69.0)
- added R3: 10k, kicadLib:C_0805_2012Metric, F.Cu at (128.7, 123.1)
- added R4: 100k, kicadLib:C_0805_2012Metric, F.Cu at (133.5, 118.5)
- added R5: 31.6k, kicadLib:C_0805_2012Metric, F.Cu at (127.5, 127.6)
- added R6: 10.2k, kicadLib:C_0805_2012Metric, F.Cu at (122.5, 130.9)
- added R7: 100, kicadLib:C_0805_2012Metric, F.Cu at (118.0, 130.9)
- added R8: 200, kicadLib:C_0805_2012Metric, F.Cu at (163.2, 93.5)
- added R9: 600, kicadLib:C_0402_1005Metric, F.Cu at (145.2, 72.3)
- IC1: footprint KiCad:TEENSY41 -> Teensy4:TEENSY41
- moved IC2 148.3 mm to (54.0, 69.0)
- moved U1 123.7 mm to (64.4, 68.8)
- moved IC1 81.6 mm to (45.4, 60.6)
- moved IC3 77.9 mm to (128.5, 47.5)
- moved U2 63.9 mm to (128.5, 58.0)
- moved D1 47.6 mm to (170.0, 119.5)
- moved D2 41.8 mm to (178.0, 112.0)
Connections:
- IC1 pad 24: unconnected-(IC1-Pad24) -> RB_INT
- IC1 pad 25: unconnected-(IC1-Pad25) -> LB_INT

Commit message: updates to 500g
Parts:
- added SW1: SW_DIP_x03, Button_Switch_SMD:SW_DIP_SPSTx03_Slide_9.78x9.8mm_W8.61mm_P2.54mm, F.Cu at (80.9, 70.4)
- added SW2: SW_SPST, Button_Switch_THT:SW_DIP_SPSTx01_Slide_6.7x4.1mm_W7.62mm_P2.54mm_LowProfile, F.Cu at (83.7, 40.0)
- moved D1 71.2 mm to (163.8, 48.6)
- moved D2 58.5 mm to (164.2, 55.2)
- moved C16 41.1 mm to (96.1, 96.5)
- moved R5 41.1 mm to (100.5, 96.5)
- moved R7 41.1 mm to (91.1, 99.9)
- moved R6 41.1 mm to (95.5, 99.9)
- moved C7 31.9 mm to (65.0, 101.6)
- moved C14 31.9 mm to (111.5, 97.7)
- moved C13 21.1 mm to (88.9, 106.3)
- moved C18 13.3 mm to (133.0, 108.2)
- moved R4 13.3 mm to (133.0, 105.2)
- moved C6 13.3 mm to (133.0, 102.2)
- moved R3 13.3 mm to (128.2, 109.8)
- moved J9 0.91 mm to (97.4, 39.1)
Connections:
- IC1 pad 24: RB_INT -> Net-(IC1-Pad24)
- IC1 pad 25: LB_INT -> Net-(IC1-Pad25)
- IC1 pad 26: unconnected-(IC1-Pad26) -> Net-(IC1-Pad26)
- J9 pad 1: +12V -> Net-(J9-Pad1)

Commit message: PCB Layout
You're welcome - Rhea
Parts:
- C11, C12, C14, C15, C17, C18, C5, C7, F1, F2, L2, R2, R3, R5, R6: moved to B.Cu
- moved R1 124.9 mm to (43.2, 61.0)
- moved C9 123.0 mm to (41.6, 83.8)
- moved C8 122.6 mm to (47.3, 71.9), turned to 180 degrees
- moved D1 116.4 mm to (47.4, 46.7)
- moved C5 113.0 mm to (58.3, 49.2), turned to 180 degrees
- moved C1 110.7 mm to (58.3, 49.2)
- moved R2 105.0 mm to (60.0, 73.7), turned to 180 degrees
- moved C6 97.7 mm to (43.2, 63.8)
- moved C10 96.6 mm to (41.1, 46.6)
- moved F1 90.2 mm to (65.2, 73.7), turned to 180 degrees
- moved R7 86.7 mm to (177.8, 99.1)
- moved R3 81.9 mm to (54.7, 73.7), turned to 180 degrees
- moved C18 70.0 mm to (69.5, 78.7), turned to 180 degrees
- moved C2 64.0 mm to (116.8, 49.2), turned to 180 degrees
- moved C13 60.1 mm to (131.1, 63.5), turned to 180 degrees
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Routing:
- net +3.3V: track 0.00 -> 146.7 mm
- net TX3: track 0.00 -> 51.0 mm
- net TX1: track 0.00 -> 25.8 mm
- net RX1: track 0.00 -> 20.6 mm
- net Net-(C11-Pad1): track 0.00 -> 20.1 mm
- net +12V: track 0.00 -> 13.4 mm
- net Net-(C7-Pad1): track 0.00 -> 12.1 mm
- net Net-(C10-Pad2): track 0.00 -> 12.0 mm
- net Net-(IC1-Pad24): track 0.00 -> 10.4 mm
- net Net-(C4-Pad2): track 0.00 -> 9.07 mm
- net Net-(C10-Pad1): track 0.00 -> 8.90 mm
- net Net-(IC1-Pad25): track 0.00 -> 8.04 mm
- net Net-(J9-Pad1): track 0.00 -> 7.42 mm
- net +5V: track 0.00 -> 6.59 mm
- net Net-(C4-Pad1): track 0.00 -> 6.12 mm
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
Commit message: Spedrun board layout
minor edits to schematic for layout purposes. finally finished layout for manufacturing
Parts:
- removed J10: LINE_RB, phoenix:PhoenixContact_MSTBA_2,5_3-G_1x03_P5.00mm_Horizontal
- removed J11: LINE_LB, phoenix:PhoenixContact_MSTBA_2,5_3-G_1x03_P5.00mm_Horizontal
- R9: footprint kicadLib:C_0402_1005Metric -> Diode_SMD:D_0805_2012Metric
- SW2: footprint Button_Switch_THT:SW_DIP_SPSTx01_Slide_6.7x4.1mm_W7.62mm_P2.54mm_LowProfile -> Button_Switch_SMD:SW_SPST_B3S-1100
- moved D4 111.5 mm to (75.8, 83.1)
- moved R8 104.8 mm to (82.2, 83.8)
- moved D3 103.0 mm to (75.8, 87.3)
- moved R7 96.3 mm to (82.1, 87.8)
- moved D5 88.9 mm to (75.9, 78.9)
- moved R9 87.7 mm to (82.2, 78.7)
- moved C16 64.6 mm to (62.0, 87.5), turned to 180 degrees
- moved J8 42.9 mm to (65.3, 40.3), turned to 180 degrees
- moved J7 40.2 mm to (117.2, 40.7), turned to 180 degrees
- moved C9 20.9 mm to (61.9, 78.7), turned to 180 degrees
- moved C13 20.5 mm to (121.0, 81.3)
- moved C8 18.4 mm to (62.0, 83.0)
- moved SW2 7.89 mm to (77.1, 44.3)
- moved SW1 5.08 mm to (91.4, 83.8)
- moved C5 5.02 mm to (53.3, 48.3), turned to 0 degrees
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Connections:
- IC1 pad 18: BDC21 -> BDC22
- IC1 pad 19: BDC22 -> BDC21
- IC1 pad 22: BDC11 -> BDC12
- IC1 pad 23: BDC12 -> BDC11
Routing:
- net +12V: track 13.4 -> 221.6 mm, vias 0 -> 7
- net +5V: track 6.59 -> 184.3 mm, vias 0 -> 2
- net RX4: track 0.00 -> 64.5 mm
- net TX4: track 0.00 -> 61.6 mm
- net RX2: track 0.00 -> 54.6 mm, vias 0 -> 2
- net TX2: track 0.00 -> 52.5 mm, vias 0 -> 1
- net RF_INT: track 0.00 -> 46.2 mm, vias 0 -> 1
- net RX3: track 5.90 -> 51.1 mm, vias 0 -> 1
- net BDC21: track 0.00 -> 44.3 mm
- net BDC22: track 0.00 -> 41.5 mm
- net Net-(U2-FB): track 3.18 -> 32.2 mm, vias 0 -> 1
- net GND: track 0.00 -> 26.4 mm, vias 0 -> 2
- net Net-(U1-FB): track 3.41 -> 25.1 mm, vias 0 -> 1
- net Net-(IC2-OUT1): track 0.00 -> 17.6 mm
- net Net-(U2-SW): track 9.07 -> 26.4 mm, vias 0 -> 1
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- added copper zone on B.Cu, net GND
- added copper zone on F.Cu, net GND
Other:
- board outline added: 98.3 x 59.9 mm
- board text added: "PrototypeMiniSumo"
