File: 500g/Musubi/musubidraft3.kicad_sch (KiCad schematic)
At the start: 29 parts, among them IC2 DRV8212DRLR, IC3 DRV8212DRLR, J1 BDC1, J1 DDS3, J2 BDC2, J2 LINE_SENS1, J3 LINE_SENS2, J4 DDS1, J5 DDS2, J9 Battery, J9 DDS4, U1 DEV-16771, U2 LM2576S-5, U3 LM2576-3.3WT

Commit message: fixed all errors except voltage input error, resolved some warnings
Connections:
- net DDS3 is gone; now on net DDS_3: U1.41 (A17)
- net DDS4 is gone; now on net DDS_4: U1.40 (A16)
- net L_LINE: now also J3.4 (Pin_4)
- net R_LINE: no longer J3.4 (Pin_4)
- net IR_MOD: no longer names the net of U1.14 (A0)
- no-connect marks 4 -> 49
Other:
- note added: "AMOGUS"
