File: 3kg/Fewawi/FewawiPowerBoard/FewawiPowerBoard.kicad_pcb (KiCad board)
At the start: 2 copper layers, 22 parts, among them J1 Battery, J2 MD_Power, J3 Conn_01x02, J4 Conn_01x02, Q1 SQM40P10-40L_GE3, Q2 SQ2318AES-T1_BE3, SW1 SW_SPST, U1 L7812CV

Commit message: finished fewawi power pcb
Parts:
- removed C2, C4: 0.1uF, Capacitor_SMD:C_0805_2012Metric_Pad1.18x1.45mm_HandSolder
- moved C7 11.8 mm to (83.8, 74.8), turned to 180 degrees
- moved C5 9.55 mm to (83.8, 71.2), turned to 180 degrees
- moved C6 9.49 mm to (83.8, 67.8), turned to 180 degrees
- moved F1 2.25 mm to (98.2, 62.5)
Routing:
- net Net-(PS1-+VIN): track 5.64 -> 34.8 mm
- net 34V: track 38.1 -> 52.3 mm
- net Net-(Q1-G): track 34.0 -> 22.2 mm
- net Net-(J4-Pin_1): track 0.00 -> 11.8 mm
- net Net-(J3-Pin_1): track 0.00 -> 11.8 mm
- net Net-(J4-Pin_2): track 0.00 -> 10.8 mm
- net Net-(J3-Pin_2): track 0.00 -> 10.8 mm
- added copper zone on B.Cu, net GND
- added copper zone on F.Cu, net GND
Other:
- board outline added: 49 x 56 mm
- board text added: "Fewawi Power :3"
