File: 3kg/Fewawi/FewawiPowerBoard/FewawiPowerBoard.kicad_pcb (KiCad board)
At the start: 2 copper layers, 49 x 56 mm, 20 parts, among them J1 Battery, J2 MD_Power, J3 Conn_01x02, J4 Conn_01x02, Q1 SQM40P10-40L_GE3, Q2 SQ2318AES-T1_BE3, SW1 SW_SPST, U1 L7812CV

Commit message: added mounting holes and some text to pcbs
Parts:
- added REF**: MountingHole_3mm_Pad, MountingHole:MountingHole_3mm_Pad, F.Cu at (123.2, 85.2)
- added REF**: MountingHole_3mm_Pad, MountingHole:MountingHole_3mm_Pad, F.Cu at (85.8, 55.8)
- moved J1 4.76 mm to (115.3, 91.8)
- moved SW1 4.13 mm to (121.2, 71.4)
- moved C1 2.59 mm to (118.2, 60.8), turned to 180 degrees
Routing:
- net Net-(J1-Pin_2): track 13.4 -> 11.2 mm
- net Net-(Q1-S): track 38.6 -> 37.1 mm
- net Net-(PS1-+VIN): track 34.8 -> 33.7 mm
Other:
- board text added: "a foolish man complains about a hole in his pants a wise man uses it to scratch his balls"

Commit message: changed fuse out, fixed most errors on both pcbs
Parts:
- removed F2: Fuse, WTF:0456050.DRSD
- added F3: 3544-2, 3544_2:FUSE_3544-2, F.Cu at (108.2, 69.2)
Routing:
- net Net-(Q1-S): track 37.1 -> 46.3 mm
- net Net-(J1-Pin_2): track 11.2 -> 16.6 mm
- net GND: vias 0 -> 1

Commit message: removed fuse
Parts:
- removed F3: 3544-2, 3544_2:FUSE_3544-2
Connections:
- Q1 pad 3: Net-(Q1-S) -> Net-(J1-Pin_2)
- R2 pad 2: Net-(Q1-S) -> Net-(J1-Pin_2)
- SW1 pad 2: Net-(Q1-S) -> Net-(J1-Pin_2)
Routing:
- net Net-(Q1-S): track 46.3 -> 0.00 mm
- net Net-(J1-Pin_2): track 16.6 -> 47.3 mm
- net Net-(SW1-A): track 28.2 -> 53.6 mm
