File: 3kg/Fewawi/FewawiPowerBoard/FewawiPowerBoard.kicad_sch (KiCad schematic)
At the start: 20 parts, among them J1 Battery, J2 MD_Power, J3 Conn_01x02, J4 Conn_01x02, Q1 SQM40P10-40L_GE3, Q2 SQ2318AES-T1_BE3, SW1 SW_SPST, U1 L7812CV

Commit message: changed fuse out, fixed most errors on both pcbs
Parts:
- removed F2: Fuse, WTF:0456050.DRSD, symbol Device:Fuse
- added F3: 3544-2, 3544_2:FUSE_3544-2, symbol 3544-2:3544-2
Connections:
- net at Q1.3 (S), R2.2, SW1.2 (B): now also F3.1_1
- net at J1.2 (Pin_2): now also F3.2_2
Other:
- moved on the sheet: J1
Changed lines of the file:
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@@
+	(wire
+		(pts
+			(xy 217.17 41.91) (xy 222.25 41.91)
+		)
+		(stroke
+			(width 0)
+			(type default)
+		)
+	)
 	(wire
 		(pts
@@
 	(wire
 		(pts
-			(xy 207.01 39.37) (xy 207.01 40.64)
-		)
-		(stroke
-			(width 0)
-			(type default)
-		)
-	)
-	(wire
-		(pts
 			(xy 171.45 48.895) (xy 173.355 48.895)
 		)
@@
 	(wire
 		(pts
-			(xy 203.2 43.18) (xy 203.2 40.64)
-		)
-		(stroke
-			(width 0)
-			(type default)
-		)
-	)
-	(wire
-		(pts
 			(xy 145.415 50.8) (xy 145.415 51.435)
 		)
@@
 	(wire
 		(pts
+			(xy 222.25 39.37) (xy 217.17 39.37)
+		)
+		(stroke
+			(width 0)
+			(type default)
+		)
+	)
+	(wire
+		(pts
 			(xy 171.45 48.26) (xy 171.45 48.895)
 		)
@@
 	(wire
 		(pts
-			(xy 191.77 40.64) (xy 195.58 40.64)
+			(xy 191.77 40.64) (xy 201.93 40.64)
 		)
 		(stroke
@@
 	(wire
 		(pts
+			(xy 201.93 40.64) (xy 201.93 41.91)
+		)
+		(stroke
+			(width 0)
+			(type default)
+		)
+	)
+	(wire
+		(pts
 			(xy 191.77 68.58) (xy 191.77 57.785)
 		)
@@
 		(pts
 			(xy 161.29 40.64) (xy 156.845 40.64)
-		)
-		(stroke
-			(width 0)
-			(type default)
-		)
-	)
-	(wire
-		(pts
-			(xy 207.01 43.18) (xy 203.2 43.18)
 		)
 		(stroke
@@
 	(rectangle
 		(start 120.65 12.7)
-		(end 227.33 88.9)
+		(end 237.49 88.9)
 		(stroke
 			(width 0)
@@
 	(symbol
 		(lib_id "Connector_Generic:Conn_01x02")
-		(at 212.09 40.64 0)
+		(at 227.33 39.37 0)
 		(unit 1)
 		(exclude_from_sim no)
@@
 		(fields_autoplaced yes)
 		(property "Reference" "J1"
-			(at 214.63 40.6399 0)
+			(at 229.87 39.3699 0)
 			(effects
 				(font
@@
 		)
 		(property "Value" "Battery"
-			(at 214.63 43.1799 0)
+			(at 229.87 41.9099 0)
 			(effects
 				(font
@@
 		)
 		(property "Footprint" "Connector_AMASS:AMASS_XT60-F_1x02_P7.20mm_Vertical"
-			(at 212.09 40.64 0)
+			(at 227.33 39.37 0)
 			(effects
 				(font
@@
 		)
 		(property "Datasheet" "~"
-			(at 212.09 40.64 0)
+			(at 227.33 39.37 0)
 			(effects
 				(font
@@
 		)
 		(property "Description" ""
-			(at 212.09 40.64 0)
+			(at 227.33 39.37 0)
 			(effects
 				(font
@@
 	)
 	(symbol
+		(lib_id "3544-2:3544-2")
+		(at 209.55 41.91 0)
+		(unit 1)
+		(exclude_from_sim no)
+		(in_bom yes)
+		(on_board yes)
+		(dnp no)
+		(fields_autoplaced yes)
+		(property "Reference" "F3"
+			(at 209.55 35.56 0)
+			(effects
+				(font
+					(size 1.27 1.27)
+				)
+			)
+		)
+		(property "Value" "3544-2"
+			(at 209.55 38.1 0)
+			(effects
+				(font
+					(size 1.27 1.27)
+				)
+			)
+		)
+		(property "Footprint" "3544_2:FUSE_3544-2"
+			(at 209.55 41.91 0)
+			(effects
+				(font
+					(size 1.27 1.27)
+				)
+				(justify bottom)
+				(hide yes)
+			)
+		)
+		(property "Datasheet" ""
+			(at 209.55 41.91 0)
+			(effects
+				(font
+					(size 1.27 1.27)
+				)
+				(hide yes)
+			)
+		)
+		(property "Description" ""
+			(at 209.55 41.91 0)
+			(effects
+				(font
+					(size 1.27 1.27)
+				)
+				(hide yes)
+			)
+		)
+		(property "PARTREV" "C"
+			(at 209.55 41.91 0)
+			(effects
+				(font
+					(size 1.27 1.27)
+				)
+				(justify bottom)
+				(hide yes)
+			)
+		)
+		(property "STANDARD" "Manufacturer Recommendations"
+			(at 209.55 41.91 0)
+			(effects
+				(font
+					(size 1.27 1.27)
+				)
+				(justify bottom)
+				(hide yes)
+			)
+		)
+		(property "SNAPEDA_PN" "3544-2"
+			(at 209.55 41.91 0)
+			(effects
+				(font
+					(size 1.27 1.27)
+				)
+				(justify bottom)
+				(hide yes)
+			)
+		)
+		(property "MAXIMUM_PACKAGE_HEIGHT" "9.02mm"
+			(at 209.55 41.91 0)
+			(effects
+				(font
+					(size 1.27 1.27)
+				)
+				(justify bottom)
+				(hide yes)
+			)
+		)
+		(property "MANUFACTURER" "Keystone"
+			(at 209.55 41.91 0)
+			(effects
+				(font
+					(size 1.27 1.27)
+				)
+				(justify bottom)
+				(hide yes)
+			)
+		)
+		(pin "2_2"
+		)
+		(pin "1_1"
+		)
+		(instances
+			(project "FewawiPowerBoard"
+				(path "/d4362b00-15c8-4a73-a6ef-1b3dcaef07a6"
+					(reference "F3")
+					(unit 1)
+				)
+			)
+		)
+	)
+	(symbol
 		(lib_id "Device:R_Small_US")
 		(at 180.975 73.025 0)
@@
 	)
 	(symbol
-		(lib_id "Device:Fuse")
-		(at 199.39 40.64 90)
-		(unit 1)
-		(exclude_from_sim no)
-		(in_bom yes)
-		(on_board yes)
-		(dnp no)
-		(fields_autoplaced yes)
-		(property "Reference" "F2"
-			(at 199.39 34.29 90)
-			(effects
-				(font
-					(size 1.27 1.27)
-				)
-			)
-		)
-		(property "Value" "Fuse"
-			(at 199.39 36.83 90)
-			(effects
-				(font
-					(size 1.27 1.27)
-				)
-			)
-		)
-		(property "Footprint" "WTF:0456050.DRSD"
-			(at 199.39 42.418 90)
-			(effects
-				(font
-					(size 1.27 1.27)
-				)
-				(hide yes)
-			)
-		)
-		(property "Datasheet" "~"
-			(at 199.39 40.64 0)
-			(effects
-				(font
-					(size 1.27 1.27)
-				)
-				(hide yes)
-			)
-		)
-		(property "Description" "Fuse"
-			(at 199.39 40.64 0)
-			(effects
-				(font
-					(size 1.27 1.27)
-				)
-				(hide yes)
-			)
-		)
-		(pin "1"
-		)
-		(pin "2"
-		)
-		(instances
-			(project "FewawiPowerBoard"
-				(path "/d4362b00-15c8-4a73-a6ef-1b3dcaef07a6"
-					(reference "F2")
-					(unit 1)
-				)
-			)
-		)
-	)
-	(symbol
 		(lib_id "power:GND")
 		(at 36.83 111.76 0)
@@
 		(lib_name "GND_1")
 		(lib_id "power:GND")
-		(at 207.01 39.37 180)
+		(at 217.17 39.37 180)
 		(unit 1)
 		(exclude_from_sim no)
@@
 		(fields_autoplaced yes)
 		(property "Reference" "#PWR012"
-			(at 207.01 33.02 0)
+			(at 217.17 33.02 0)
 			(effects
 				(font
@@
 		)
 		(property "Value" "GND"
-			(at 207.01 34.29 0)
+			(at 217.17 34.29 0)
 			(effects
 				(font
@@
 		)
 		(property "Footprint" ""
-			(at 207.01 39.37 0)
+			(at 217.17 39.37 0)
 			(effects
 				(font
@@
 		)
 		(property "Datasheet" ""
-			(at 207.01 39.37 0)
+			(at 217.17 39.37 0)
 			(effects
 				(font
@@
 		)
 		(property "Description" ""
-			(at 207.01 39.37 0)
-			(effects
-				(font
+			(at 217.17 39.37 0)
+			(effects
+				(font

Commit message: removed fuse
Parts:
- removed F3: 3544-2, 3544_2:FUSE_3544-2, symbol 3544-2:3544-2
Connections:
- net at Q1.3 (S), R2.2, SW1.2 (B): now also J1.2 (Pin_2)
Changed lines of the file:
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@@
-	(wire
-		(pts
-			(xy 217.17 41.91) (xy 222.25 41.91)
-		)
-		(stroke
-			(width 0)
-			(type default)
-		)
-	)
 	(wire
 		(pts
@@
 		(pts
 			(xy 140.97 51.435) (xy 140.97 55.245)
+		)
+		(stroke
+			(width 0)
+			(type default)
+		)
+	)
+	(wire
+		(pts
+			(xy 201.93 41.91) (xy 222.25 41.91)
 		)
 		(stroke
@@
 					(unit 1)
 				)
-			)
-		)
-	)
-	(symbol
-		(lib_id "3544-2:3544-2")
-		(at 209.55 41.91 0)
-		(unit 1)
-		(exclude_from_sim no)
-		(in_bom yes)
-		(on_board yes)
-		(dnp no)
-		(fields_autoplaced yes)
-		(property "Reference" "F3"
-			(at 209.55 35.56 0)
-			(effects
-				(font
-					(size 1.27 1.27)
-				)
-			)
-		)
-		(property "Value" "3544-2"
-			(at 209.55 38.1 0)
-			(effects
-				(font
-					(size 1.27 1.27)
-				)
-			)
-		)
-		(property "Footprint" "3544_2:FUSE_3544-2"
-			(at 209.55 41.91 0)
-			(effects
-				(font
-					(size 1.27 1.27)
-				)
-				(justify bottom)
-				(hide yes)
-			)
-		)
-		(property "Datasheet" ""
-			(at 209.55 41.91 0)
-			(effects
-				(font
-					(size 1.27 1.27)
-				)
-				(hide yes)
-			)
-		)
-		(property "Description" ""
-			(at 209.55 41.91 0)
-			(effects
-				(font
-					(size 1.27 1.27)
-				)
-				(hide yes)
-			)
-		)
-		(property "PARTREV" "C"
-			(at 209.55 41.91 0)
-			(effects
-				(font
-					(size 1.27 1.27)
-				)
-				(justify bottom)
-				(hide yes)
-			)
-		)
-		(property "STANDARD" "Manufacturer Recommendations"
-			(at 209.55 41.91 0)
-			(effects
-				(font
-					(size 1.27 1.27)
-				)
-				(justify bottom)
-				(hide yes)
-			)
-		)
-		(property "SNAPEDA_PN" "3544-2"
-			(at 209.55 41.91 0)
-			(effects
-				(font
-					(size 1.27 1.27)
-				)
-				(justify bottom)
-				(hide yes)
-			)
-		)
-		(property "MAXIMUM_PACKAGE_HEIGHT" "9.02mm"
-			(at 209.55 41.91 0)
-			(effects
-				(font
-					(size 1.27 1.27)
-				)
-				(justify bottom)
-				(hide yes)
-			)
-		)
-		(property "MANUFACTURER" "Keystone"
-			(at 209.55 41.91 0)
-			(effects
-				(font
-					(size 1.27 1.27)
-				)
-				(justify bottom)
-				(hide yes)
-			)
-		)
-		(pin "2_2"
-		)
-		(pin "1_1"
-		)
-		(instances
-			(project "FewawiPowerBoard"
-				(path "/d4362b00-15c8-4a73-a6ef-1b3dcaef07a6"
-					(reference "F3")
-					(unit 1)
-				)
