File: 3kg/Fewawi/FewawiControlBoard/FewawiControlBoard.kicad_pcb (KiCad board)
At the start: 2 copper layers, 106.5 x 86 mm, 88 parts, among them J1 Encoder_Left, J10 DS_45R, J11 DS_60R, J12 DS_90R, J13 DS_FR, J14 LS_LF1, J15 LS_RF1, J16 LS_BL1, J17 LS_BR1, J18 LS_PlowLeft, J19 LS_PlowMid, J2 Encoder_Right, J20 LS_LF2, J21 LS_RF2, J22 LS_BL2, J23 LS_BR2, J24 LS_PlowRight, J25 SignalsToMD, J26 12vPower, J27 5vPower, J3 DS_FL, J4 Start Module, J5 DS_45L, J6 DS_60L, J7 DS_90L, J8 DS_Mid, J9 LCD_Screen, Q2 LTV-826S, Q3 LTV-826S, Q4 LTV-826S, Q5 LTV-826S, Q6 LTV-826S, U1 DEV-16771, U2 Button1, U4 LMV358IDGKRG4

Commit message: power connections made on control board
Parts:
- moved J1 130.0 mm to (101.2, 131.6)
- moved J2 64.0 mm to (191.5, 131.6)
- moved C1 47.2 mm to (101.5, 102.4)
- moved C10 47.2 mm to (188.5, 88.4)
- moved C11 47.2 mm to (188.4, 99.9)
- moved C12 47.2 mm to (179.5, 65.9)
- moved C13 47.2 mm to (108.5, 65.9)
- moved C14 47.2 mm to (191.0, 65.9)
- moved C15 47.2 mm to (129.5, 126.4)
- moved C16 47.2 mm to (165.0, 126.4)
- moved C17 47.2 mm to (133.5, 65.9)
- moved C18 47.2 mm to (144.5, 65.9)
- moved C19 47.2 mm to (112.0, 65.9)
- moved C2 47.2 mm to (105.0, 102.4)
- moved C20 47.2 mm to (187.5, 65.9)
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Routing:
- net +3.3V: track 0.00 -> 297.2 mm
- net +12V: track 0.00 -> 272.0 mm
- net +5V: track 0.00 -> 224.0 mm, vias 0 -> 1
- net Net-(Q6-Pad1): track 0.00 -> 26.1 mm
- net Net-(Q4-Pad1): track 0.00 -> 18.0 mm
- net Net-(Q2-Pad3): track 0.00 -> 12.8 mm
- net Net-(Q3-Pad1): track 0.00 -> 11.8 mm
- net Net-(Q3-Pad3): track 0.00 -> 11.4 mm
- net Button1: track 0.00 -> 9.57 mm
- net Net-(Q2-Pad1): track 0.00 -> 8.30 mm
- net Net-(Q5-Pad3): track 0.00 -> 8.12 mm
- net OCT_90R: track 0.00 -> 7.35 mm
- net OCT_60R: track 0.00 -> 7.15 mm
- net Net-(Q4-Pad3): track 0.00 -> 6.86 mm
- net OCT_90L: track 0.00 -> 6.77 mm
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
Commit message: fewawi pcb done (with errors
Parts:
- moved R6 6.99 mm to (102.5, 126.8), turned to 90 degrees
- moved R7 6.98 mm to (193.5, 126.4), turned to 90 degrees
- moved R2 6.52 mm to (200.0, 126.5), turned to 90 degrees
- moved R1 3.28 mm to (109.2, 126.8), turned to 90 degrees
- moved R4 3.28 mm to (105.8, 126.8), turned to 90 degrees
- moved C22 2.73 mm to (171.8, 126.5)
- moved R20 2.73 mm to (175.2, 126.5)
- moved R8 1.48 mm to (184.5, 120.5)
- moved R9 1.48 mm to (181.0, 120.5)
- moved U4 1.23 mm to (182.8, 126.0)
- moved R5 0.24 mm to (196.8, 126.5), turned to 90 degrees
Connections:
- R8 pad 2: MD_InputSignal2 -> Net-(R8-Pad2)
- R9 pad 1: MD_InputSignal1 -> Net-(R9-Pad1)
- U1 pad 0: DS_90R -> DS_45L
- U1 pad 1: DS_60R -> DS_FL
- U1 pad 11: DS_FL -> DS_60R
- U1 pad 12: DS_45L -> DS_90R
- U1 pad 14: LS_RF2 -> LS_RF1
- U1 pad 15: LS_RF1 -> LS_RF2
- U1 pad 16: LS_PlowLeft -> LS_PlowRight
- U1 pad 17: LS_PlowRight -> LS_PlowMid
- U1 pad 2: DS_FR -> DS_90L
- U1 pad 20: LS_PlowMid -> LS_PlowLeft
- U1 pad 21: LS_BR1 -> LS_LF2
- U1 pad 22: EncR_Pin2 -> LS_LF1
- U1 pad 23: LS_BR2 -> StartMod
- U1 pad 26: LS_LF1 -> LS_BR1
- U1 pad 27: LS_LF2 -> LS_BR2
- U1 pad 28: DS_60L -> DS_45R
- U1 pad 29: DS_90L -> DS_FR
- U1 pad 3: DS_45R -> DS_60L
- U1 pad 33: StartMod -> EncR_Pin2
- U1 pad 38: MD_InputSignal1 -> MD_InputSignal2
- U1 pad 39: MD_InputSignal2 -> MD_InputSignal1
- U1 pad 40: LS_BL2 -> LS_BL1
- U1 pad 41: LS_BL1 -> LS_BL2
- U1 pad 5: EncR_Pin3 -> EncL_Pin3
- U1 pad 9: EncL_Pin3 -> EncR_Pin3
- U4 pad 2: MD_InputSignal2 -> Net-(R8-Pad2)
- U4 pad 6: MD_InputSignal1 -> Net-(R9-Pad1)
Routing:
- net LS_RF1: track 0.00 -> 99.0 mm, vias 0 -> 2
- net +3.3V: track 297.2 -> 388.9 mm, vias 0 -> 3
- net LS_RF2: track 0.00 -> 91.6 mm, vias 0 -> 2
- net EncR_Pin3: track 0.00 -> 87.0 mm, vias 0 -> 5
- net StartMod: track 0.00 -> 78.0 mm, vias 0 -> 3
- net Button1: track 9.57 -> 83.7 mm, vias 0 -> 5
- net LS_PlowRight: track 0.00 -> 67.8 mm, vias 0 -> 4
- net EncR_Pin5: track 0.00 -> 66.6 mm, vias 0 -> 3
- net DS_60R: track 0.00 -> 64.3 mm, vias 0 -> 6
- net IMU_INT2: track 0.00 -> 60.8 mm, vias 0 -> 4
- net DS_45L: track 0.00 -> 58.6 mm, vias 0 -> 10
- net DS_90R: track 0.00 -> 57.8 mm, vias 0 -> 6
- net MD_InputSignal2: track 0.00 -> 57.7 mm, vias 0 -> 4
- net DS_45R: track 0.00 -> 57.5 mm, vias 0 -> 4
- net IMU_INT1: track 0.00 -> 57.3 mm, vias 0 -> 4
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
Commit message: fewawi pcb errors resolved thank god im tired and coke deprived and am dealing with pm abuse
Routing:
- net GND: track 6.95 -> 46.0 mm, vias 0 -> 6
- net +3.3V: track 388.9 -> 427.5 mm, vias 3 -> 8
- net Signal1: track 6.79 -> 12.6 mm
- net +12V: track 268.2 -> 263.4 mm
- net Button1: track 83.7 -> 84.7 mm
- added copper zone on B.Cu, net GND
- added copper zone on F.Cu, net GND

Commit message: added mounting holes and some text to pcbs
Parts:
- added REF**: MountingHole_3mm_Pad, MountingHole:MountingHole_3mm_Pad, F.Cu at (196.5, 112.0)
- added REF**: MountingHole_3mm_Pad, MountingHole:MountingHole_3mm_Pad, F.Cu at (137.0, 72.8)
- moved J26 4.95 mm to (199.2, 104.5)
Routing:
- net +12V: track 263.4 -> 256.4 mm
Other:
- board text added: "Fewawi :3 First iteration Kyle Nguyen"
- board text added: "Jinhee needs a shower, Xander is a nasty girl, Cord is the rizzler"
Changed lines of the file:
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@@
 		)
 	)
+	(footprint "MountingHole:MountingHole_3mm_Pad"
+		(layer "F.Cu")
+		(at 196.5 112)
+		(descr "Mounting Hole 3mm")
+		(tags "mounting hole 3mm")
+		(property "Reference" "REF**"
+			(at 0 -4 0)
+			(layer "F.SilkS")
+			(effects
+				(font
+					(size 1 1)
+					(thickness 0.15)
+				)
+			)
+		)
+		(property "Value" "MountingHole_3mm_Pad"
+			(at 0 4 0)
+			(layer "F.Fab")
+			(effects
+				(font
+					(size 1 1)
+					(thickness 0.15)
+				)
+			)
+		)
+		(property "Footprint" "MountingHole:MountingHole_3mm_Pad"
+			(at 0 0 0)
+			(unlocked yes)
+			(layer "F.Fab")
+			(hide yes)
+			(effects
+				(font
+					(size 1.27 1.27)
+				)
+			)
+		)
+		(property "Datasheet" ""
+			(at 0 0 0)
+			(unlocked yes)
+			(layer "F.Fab")
+			(hide yes)
+			(effects
+				(font
+					(size 1.27 1.27)
+				)
+			)
+		)
+		(property "Description" ""
+			(at 0 0 0)
+			(unlocked yes)
+			(layer "F.Fab")
+			(hide yes)
+			(effects
+				(font
+					(size 1.27 1.27)
+				)
+			)
+		)
+		(attr exclude_from_pos_files exclude_from_bom)
+		(fp_circle
+			(center 0 0)
+			(end 3 0)
+			(stroke
+				(width 0.15)
+				(type solid)
+			)
+			(fill none)
+			(layer "Cmts.User")
+		)
+		(fp_circle
+			(center 0 0)
+			(end 3.25 0)
+			(stroke
+				(width 0.05)
+				(type solid)
+			)
+			(fill none)
+			(layer "F.CrtYd")
+		)
+		(fp_text user "${REFERENCE}"
+			(at 0 0 0)
+			(layer "F.Fab")
+			(effects
+				(font
+					(size 1 1)
+					(thickness 0.15)
+				)
+			)
+		)
+		(pad "1" thru_hole circle
+			(at 0 0)
+			(size 6 6)
+			(drill 3)
+			(layers "*.Cu" "*.Mask")
+			(remove_unused_layers no)
+		)
+	)
 	(footprint "Resistor_SMD:R_0805_2012Metric_Pad1.20x1.40mm_HandSolder"
 		(layer "F.Cu")
@@
 	(footprint "Connector_AMASS:AMASS_XT30U-F_1x02_P5.0mm_Vertical"
 		(layer "F.Cu")
-		(at 199.48 109.44 180)
+		(at 199.25 104.5 180)
 		(descr "Connector XT30 Vertical Cable Female, https://www.tme.eu/en/Document/3cbfa5cfa544d79584972dd5234a409e/XT30U%20SPEC.pdf")
 		(tags "RC Connector XT30")
@@
 		)
 	)
+	(footprint "MountingHole:MountingHole_3mm_Pad"
+		(layer "F.Cu")
+		(at 137 72.75)
+		(descr "Mounting Hole 3mm")
+		(tags "mounting hole 3mm")
+		(property "Reference" "REF**"
+			(at 0 -4 0)
+			(layer "F.SilkS")
+			(effects
+				(font
+					(size 1 1)
+					(thickness 0.15)
+				)
+			)
+		)
+		(property "Value" "MountingHole_3mm_Pad"
+			(at 0 4 0)
+			(layer "F.Fab")
+			(effects
+				(font
+					(size 1 1)
+					(thickness 0.15)
+				)
+			)
+		)
+		(property "Footprint" "MountingHole:MountingHole_3mm_Pad"
+			(at 0 0 0)
+			(unlocked yes)
+			(layer "F.Fab")
+			(hide yes)
+			(effects
+				(font
+					(size 1.27 1.27)
+				)
+			)
+		)
+		(property "Datasheet" ""
+			(at 0 0 0)
+			(unlocked yes)
+			(layer "F.Fab")
+			(hide yes)
+			(effects
+				(font
+					(size 1.27 1.27)
+				)
+			)
+		)
+		(property "Description" ""
+			(at 0 0 0)
+			(unlocked yes)
+			(layer "F.Fab")
+			(hide yes)
+			(effects
+				(font
+					(size 1.27 1.27)
+				)
+			)
+		)
+		(attr exclude_from_pos_files exclude_from_bom)
+		(fp_circle
+			(center 0 0)
+			(end 3 0)
+			(stroke
+				(width 0.15)
+				(type solid)
+			)
+			(fill none)
+			(layer "Cmts.User")
+		)
+		(fp_circle
+			(center 0 0)
+			(end 3.25 0)
+			(stroke
+				(width 0.05)
+				(type solid)
+			)
+			(fill none)
+			(layer "F.CrtYd")
+		)
+		(fp_text user "${REFERENCE}"
+			(at 0 0 0)
+			(layer "F.Fab")
+			(effects
+				(font
+					(size 1 1)
+					(thickness 0.15)
+				)
+			)
+		)
+		(pad "1" thru_hole circle
+			(at 0 0)
+			(size 6 6)
+			(drill 3)
+			(layers "*.Cu" "*.Mask")
+			(remove_unused_layers no)
+		)
+	)
 	(footprint "Resistor_SMD:R_0805_2012Metric_Pad1.20x1.40mm_HandSolder"
 		(layer "F.Cu")
@@
 		(layer "Edge.Cuts")
 	)
+	(gr_text "Jinhee needs a shower, Xander is a nasty girl, Cord is the rizzler\n"
+		(at 200.25 136.5 0)
+		(layer "B.SilkS")
+		(effects
+			(font
+				(size 1 1)
+				(thickness 0.1)
+			)
+			(justify left bottom mirror)
+		)
+	)
+	(gr_text "Fewawi :3\nFirst iteration\nKyle Nguyen"
+		(at 143.25 77.25 0)
+		(layer "F.SilkS")
+		(effects
+			(font
+				(size 2 2)
+				(thickness 0.1)
+			)
+			(justify left bottom)
+		)
+	)
 	(segment
 		(start 194.48 119.94)
@@
 	)
 	(segment
+		(start 194.25 100.22)
+		(end 194.25 104.5)
+		(width 0.7)
+		(layer "F.Cu")
+		(net 4)
+	)
+	(segment
 		(start 194.53 99.94)
 		(end 196.03 98.44)
@@
 	)
 	(segment
+		(start 194.25 100.22)
+		(end 194.53 99.94)
+		(width 0.2)
+		(layer "F.Cu")
+		(net 4)
+	)
+	(segment
 		(start 154.59 57.5)
 		(end 126.87 57.5)
@@
 	)
 	(segment
-		(start 194.48 109.44)
-		(end 194.48 99.99)
-		(width 0.7)
-		(layer "F.Cu")
-		(net 4)
-	)
-	(segment
 		(start 125.48 60.89)
 		(end 124.48 59.89)
@@
 		(layer "F.Cu")
 		(net 4)
-	)
-	(segment
-		(start 194.48 99.99)
-		(end 196.03 98.44)
-		(width 0.2)
-		(layer "F.Cu")
-		(net 4)

Commit message: changed fuse out, fixed most errors on both pcbs
Routing:
- net +5V: track 243.0 -> 241.9 mm
- net GND: vias 6 -> 10
Changed lines of the file:
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@@
 			)
 		)
-		(fp_text user "-"
-			(at -4 0 180)
-			(layer "F.SilkS")
-			(effects
-				(font
-					(size 1.5 1.5)
-					(thickness 0.15)
-				)
-			)
-		)
 		(fp_text user "${REFERENCE}"
 			(at 2.5 0 180)
@@
 			(layer "F.Fab")
 		)
-		(fp_text user "-"
-			(at -4 0 180)
-			(layer "F.SilkS")
-			(effects
-				(font
-					(size 1.5 1.5)
-					(thickness 0.15)
-				)
-			)
-		)
 		(fp_text user "+"
 			(at 9 0 180)
@@
 	)
 	(segment
-		(start 191.54 117)
-		(end 191.5 117)
-		(width 0.2)
-		(layer "F.Cu")
-		(net 1)
-	)
-	(segment
 		(start 107.25 127.75)
 		(end 107.25 131.55)
@@
 	(segment
 		(start 192.27 117.73)
-		(end 191.54 117)
-		(width 0.7)
-		(layer "F.Cu")
-		(net 1)
-	)
-	(segment
-		(start 192.27 117.73)
 		(end 190.304 115.764)
 		(width 0.7)
@@
 	)
 	(via
+		(at 124.25 86)
+		(size 0.6)
+		(drill 0.3)
+		(layers "F.Cu" "B.Cu")
+		(free yes)
+		(net 2)
+	)
+	(via
 		(at 187.25 122.9)
 		(size 0.6)
@@
 	)
 	(via
+		(at 185.25 73.75)
+		(size 0.6)
+		(drill 0.3)
+		(layers "F.Cu" "B.Cu")
+		(free yes)
+		(net 2)
+	)
+	(via
 		(at 185.75 122.9)
 		(size 0.6)
@@
 	)
 	(via
+		(at 186.5 62.75)
+		(size 0.6)
+		(drill 0.3)
+		(layers "F.Cu" "B.Cu")
+		(free yes)
+		(net 2)
+	)
+	(via
 		(at 169.75 128.75)
 		(size 0.6)
@@
 		(net 2)
 	)
+	(via
+		(at 107.5 104.25)
+		(size 0.6)
+		(drill 0.3)
+		(layers "F.Cu" "B.Cu")
+		(free yes)
+		(net 2)
+	)
